File: flipdot_driver.sch (KiCad schematic (older format))
At the start: 365 parts, among them J4 Barrel_Jack, Q1 2N7002, Q2 2N7002, Q3 BUZ11, Q4 IRF9540N, Q5 BUZ11, Q6 IRF9540N, Q7 BUZ11, SW1 NP_TACTILE_SWITCH, SW2 TACTILE_SWITCH, U1 FE310-G000, U2 FT2232D, U3 IS25LP128-JBLE

Commit message: replaced relatively large power MOSFETs with much more space-efficient N P pairs in a TSOT-23-6 package
Parts:
- removed Q3, Q5, Q? (x42): BUZ11, TO_SOT_Packages_THT:TO-220-3_Horizontal, symbol BUZ11
- removed Q4, Q6, Q? (x42): IRF9540N, TO_SOT_Packages_THT:TO-220-3_Horizontal, symbol IRF9540N
- added Q? (x88): DMG6602, TSOT-23-6, symbol DMG6602

Commit message: Added DC-DC converters to attain necessary voltage rails
Parts:
- removed R14: 47k, Resistors_SMD:R_0603_HandSoldering, symbol R
- added C? (x8): 22uF, Capacitors_SMD:C_0603_HandSoldering, symbol C
- added C? (x3): 1uF, Capacitors_SMD:C_0603_HandSoldering, symbol C
- added C? (x3): 47pF, Capacitors_SMD:C_0603_HandSoldering, symbol C
- added C? (x5): 4.7uF, Capacitors_SMD:C_0603_HandSoldering, symbol C
- added C?: 4.7nF, Capacitors_SMD:C_0603_HandSoldering, symbol C
- added C?: 15nF, Capacitors_SMD:C_0603_HandSoldering, symbol C
- added C? (x2): 47uF, symbol CP1
- added C?: NP_47uF, symbol CP1
- added D?: D, symbol D
- added J?: Screw_Terminal_01x04, symbol Screw_Terminal_01x04
- added L?: 3.3uH, symbol L
- added L? (x2): 6.5uH, symbol L
- added L?: 12uH, symbol L
- added R?: 100k, Resistors_SMD:R_0603_HandSoldering, symbol R
- added R? (x3): 40.2k, Resistors_SMD:R_0603_HandSoldering, symbol R
- added R?: 32.4k, Resistors_SMD:R_0603_HandSoldering, symbol R
- added R? (x2): 47k, Resistors_SMD:R_0603_HandSoldering, symbol R
- added R?: 13k, Resistors_SMD:R_0603_HandSoldering, symbol R
- added R?: 7.68k, Resistors_SMD:R_0603_HandSoldering, symbol R
- added R?: 143k, Resistors_SMD:R_0603_HandSoldering, symbol R
- added R? (x2): 4.87k, Resistors_SMD:R_0603_HandSoldering, symbol R
- added R?: 300k, Resistors_SMD:R_0603_HandSoldering, symbol R
- added R?: 16.2k, Resistors_SMD:R_0603_HandSoldering, symbol R
- added U? (x3): AP65111A, symbol AP65111A
- added U?: TPS61175, symbol TPS61175
Connections:
- net +12V: now also J4.1, C?.1, C?.1, C?.1, C?.1, C?.1, C?.1, C?.1, C?.1, C?.1, C?.1, C?.1, J?.1 (Pin_1), J?.2 (Pin_2), L?.1, U?.1 (VIN), U?.1 (VIN), U?.1 (VIN), U?.3 (VIN)
- net +1V8: now also C?.1, C?.1, L?.2, R?.2
- net +24V: now also C?.1, C?.1, D?.1 (K), R?.1
- net +3V3: now also C?.1, C?.1, L?.2, R?.2
- net +5V: now also C?.1, C?.1, L?.2, R?.2
- net GND: now also J4.2, J4.3, C?.2, C?.2, C?.2, C?.2, C?.2, C?.2, C?.2, C?.2, C?.2, C?.2, C?.2, C?.2, C?.2, C?.2, C?.2, C?.2, C?.2, C?.2, J?.3 (Pin_3), J?.4 (Pin_4), R?.1, R?.1, R?.1, R?.1, R?.2, U?.11 (RES), U?.12 (PGND), U?.13 (PGND), U?.14 (PGND), U?.2 (GND), U?.2 (GND), U?.2 (GND), U?.6 (SYN), U?.7 (AGND)
- new net: C?.1, L?.1, U?.3 (SW) (x3)
- new net: C?.2, U?.4 (BST) (x3)
- new net: R?.2, U?.6 (FB) (x3)
- new net: C?.2, R?.1, R?.1, R?.2 (x3)
- new net: D?.2 (A), L?.2, U?.1 (SW), U?.2 (SW)
- new net: R?.2, U?.10 (FREQ)
- new net: C?.1, U?.5 (SS)
- new net: R?.2, U?.8 (COMP)
- new net: R?.1, U?.9 (FB)
- new net: C?.1, R?.1
- new net: R?.1, R?.2, R?.2
- new net EN_1V8: U?.5 (EN)
- new net EN_24V: U?.4 (EN)
- new net EN_3V3: U?.5 (EN)
- new net EN_5V: U?.5 (EN)
Other:
- note added: "LABEL POSITIVE AND\nNEGATIVE TERMINALS\nON SILKSCREEN"
- note added: "USB TO JTAG\nJTAG\nGPIO\nCONSOLE\nINPUT ESD PROTECTION\nINPUT REVERSE PROTECTION\nTESTPOINTS\nPOWER SEQUENCING\nCALCULATE MAX CLK RATE BASED ON INPUT CAPACITANCE AND RESISTANCE OF FETS."
- note removed: "USB TO JTAG\nJTAG\nconsole\n12V INPUT\nBUCK CONVERTERS\nMULTIPLEXING\nTESTPOINTS\nCALCULATE MAX CLK RATE BASED ON INPUT CAPACITANCE AND RESISTANCE OF FETS.\nMAKE SURE INRUSH CURRENT OF SWITCHING DOES NOT VIOLATE FET MAX CURRENT."
- moved on the sheet: J4

Commit message: Sprinkled in some test points on the power circuitry
Parts:
- added TP? (x8): TEST, symbol TEST
- C?: value NP_47uF -> NP_470uF
Connections:
- net +12V: now also TP1.1
- net +1V8: now also TP?.1
- net +24V: now also TP?.1
- net +3V3: now also TP?.1
- net +5V: now also TP?.1
- net at C?.2, R?.1, R?.1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: now also TP?.1 (x3)
- net at R?.1, R?.2, R?.2: now also TP?.1
Other:
- moved on the sheet: C?, TP1
Changed lines of the file:
@@
 L TEST TP1
 U 1 1 59EB83DE
-P 12250 15300
-F 0 "TP1" H 12250 15600 50  0000 C BNN
-F 1 "TEST" H 12250 15550 50  0000 C CNN
-F 2 "" H 12250 15300 50  0001 C CNN
-F 3 "" H 12250 15300 50  0001 C CNN
-	1    12250 15300
-	1    0    0    -1
+P 10000 10900
+F 0 "TP1" H 10000 11200 50  0000 C BNN
+F 1 "TEST" H 10000 11150 50  0000 C CNN
+F 2 "" H 10000 10900 50  0001 C CNN
+F 3 "" H 10000 10900 50  0001 C CNN
+	1    10000 10900
+	0    1    1    0
 $EndComp
 $Comp
@@
 L C C?
 U 1 1 5A7474C6
-P 16550 23150
-F 0 "C?" H 16575 23250 50  0000 L CNN
-F 1 "22uF" H 16575 23050 50  0000 L CNN
-F 2 "Capacitors_SMD:C_0603_HandSoldering" H 16588 23000 50  0001 C CNN
-F 3 "" H 16550 23150 50  0001 C CNN
-	1    16550 23150
+P 16800 23150
+F 0 "C?" H 16825 23250 50  0000 L CNN
+F 1 "22uF" H 16825 23050 50  0000 L CNN
+F 2 "Capacitors_SMD:C_0603_HandSoldering" H 16838 23000 50  0001 C CNN
+F 3 "" H 16800 23150 50  0001 C CNN
+	1    16800 23150
 	1    0    0    -1
 $EndComp
@@
 L +24V #PWR0197
 U 1 1 5A849187
-P 16900 22350
-F 0 "#PWR0197" H 16900 22200 50  0001 C CNN
-F 1 "+24V" H 16900 22490 50  0000 C CNN
-F 2 "" H 16900 22350 50  0001 C CNN
-F 3 "" H 16900 22350 50  0001 C CNN
-	1    16900 22350
+P 17150 22350
+F 0 "#PWR0197" H 17150 22200 50  0001 C CNN
+F 1 "+24V" H 17150 22490 50  0000 C CNN
+F 2 "" H 17150 22350 50  0001 C CNN
+F 3 "" H 17150 22350 50  0001 C CNN
+	1    17150 22350
 	1    0    0    -1
 $EndComp
@@
 L C C?
 U 1 1 5A86AFB3
-P 16900 23150
-F 0 "C?" H 16925 23250 50  0000 L CNN
-F 1 "22uF" H 16925 23050 50  0000 L CNN
-F 2 "Capacitors_SMD:C_0603_HandSoldering" H 16938 23000 50  0001 C CNN
-F 3 "" H 16900 23150 50  0001 C CNN
-	1    16900 23150
+P 17150 23150
+F 0 "C?" H 17175 23250 50  0000 L CNN
+F 1 "22uF" H 17175 23050 50  0000 L CNN
+F 2 "Capacitors_SMD:C_0603_HandSoldering" H 17188 23000 50  0001 C CNN
+F 3 "" H 17150 23150 50  0001 C CNN
+	1    17150 23150
 	1    0    0    -1
 $EndComp
@@
 	16850 25150 16850 25250
 Wire Wire Line
-	16150 25200 16850 25200
+	16150 25200 16900 25200
 Connection ~ 16850 25200
 Wire Wire Line
 	16200 26000 16200 25950
 Wire Wire Line
-	16000 25600 16450 25600
-Wire Wire Line
-	16450 25600 16450 25550
+	16450 25550 16450 25650
 Wire Wire Line
 	16200 25250 16200 25200
@@
 	16850 26800 16850 26900
 Wire Wire Line
-	16150 26850 16850 26850
+	16150 26850 16900 26850
 Connection ~ 16850 26850
 Wire Wire Line
 	16200 27650 16200 27600
 Wire Wire Line
-	16000 27250 16450 27250
-Wire Wire Line
-	16450 27250 16450 27200
+	16450 27200 16450 27300
 Wire Wire Line
 	16200 26900 16200 26850
@@
 	16900 28450 16900 28550
 Wire Wire Line
-	16200 28500 16900 28500
+	16200 28500 16950 28500
 Connection ~ 16900 28500
 Wire Wire Line
 	16250 29300 16250 29250
 Wire Wire Line
-	16050 28900 16500 28900
-Wire Wire Line
-	16500 28900 16500 28850
+	16500 28850 16500 28950
 Wire Wire Line
 	16250 28550 16250 28500
@@
 	15150 24050 15150 24150
 Wire Wire Line
-	13450 24050 16900 24050
+	13450 24050 17150 24050
 Wire Wire Line
 	14600 24050 15150 24050
@@
 	16200 22900 16200 23100
 Wire Wire Line
-	16200 23000 16050 23000
+	16050 23000 16250 23000
 Connection ~ 16200 23000
 Wire Wire Line
 	16200 22600 16200 22400
 Wire Wire Line
-	16150 22400 16900 22400
+	16150 22400 17200 22400
 Wire Wire Line
-	16550 22400 16550 23000
+	16800 22400 16800 23000
 Connection ~ 16200 22400
 Wire Wire Line
-	16550 24050 16550 23300
+	16800 24050 16800 23300
 Connection ~ 16200 24050
-Connection ~ 16550 22400
+Connection ~ 16800 22400
 Wire Wire Line
 	15750 23000 15650 23000
 Connection ~ 14600 22400
 Wire Wire Line
-	16900 22350 16900 23000
-Connection ~ 16900 22400
+	17150 22350 17150 23000
+Connection ~ 17150 22400
 Wire Wire Line
-	16900 24050 16900 23300
-Connection ~ 16550 24050
+	17150 24050 17150 23300
+Connection ~ 16800 24050
 Wire Wire Line
 	10050 10000 10050 9950
@@
 Connection ~ 10450 10350
 Wire Wire Line
-	9800 10900 9900 10900
+	9800 10900 10000 10900
 Wire Wire Line
 	9900 10900 9900 10800
@@
 $EndComp
 Wire Wire Line
-	11150 10900 11100 10900
+	11100 10900 11150 10900
 Wire Wire Line
-	11100 10900 11100 10750
+	11100 10750 11100 10900
 Wire Wire Line
 	11150 10800 11100 10800
@@
 P 9650 10150
 F 0 "C?" H 9675 10250 50  0000 L CNN
-F 1 "NP_47uF" H 9300 10050 50  0000 L CNN
+F 1 "NP_470uF" H 9250 10050 50  0000 L CNN
 F 2 "" H 9650 10150 50  0001 C CNN
 F 3 "" H 9650 10150 50  0001 C CNN
@@
 	9650 10000 9650 9950
 Connection ~ 10050 9950
+Connection ~ 9900 10900
+$Comp
+L TEST TP?
+U 1 1 5A366C4B
+P 16950 28500
+F 0 "TP?" H 16950 28800 50  0000 C BNN
+F 1 "TEST" H 16950 28750 50  0000 C CNN
+F 2 "" H 16950 28500 50  0001 C CNN
+F 3 "" H 16950 28500 50  0001 C CNN
+	1    16950 28500
+	0    1    1    0
+$EndComp
+$Comp
+L TEST TP?
+U 1 1 5A36E907
+P 16900 26850
+F 0 "TP?" H 16900 27150 50  0000 C BNN
+F 1 "TEST" H 16900 27100 50  0000 C CNN
+F 2 "" H 16900 26850 50  0001 C CNN
+F 3 "" H 16900 26850 50  0001 C CNN
+	1    16900 26850
+	0    1    1    0
+$EndComp
+$Comp
+L TEST TP?
+U 1 1 5A378CBD
+P 16900 25200
+F 0 "TP?" H 16900 25500 50  0000 C BNN
+F 1 "TEST" H 16900 25450 50  0000 C CNN
+F 2 "" H 16900 25200 50  0001 C CNN
+F 3 "" H 16900 25200 50  0001 C CNN
+	1    16900 25200
+	0    1    1    0
+$EndComp
+$Comp
+L TEST TP?
+U 1 1 5A37D933
+P 16450 27300
+F 0 "TP?" H 16450 27600 50  0000 C BNN
+F 1 "TEST" H 16450 27550 50  0000 C CNN
+F 2 "" H 16450 27300 50  0001 C CNN
+F 3 "" H 16450 27300 50  0001 C CNN
+	1    16450 27300
+	-1   0    0    1
+$EndComp
+Wire Wire Line
+	16000 27250 16450 27250
+Connection ~ 16450 27250
+Wire Wire Line
+	16000 25600 16450 25600
+Wire Wire Line
+	16050 28900 16500 28900
+$Comp
+L TEST TP?
+U 1 1 5A3A9D8A
+P 16500 28950
+F 0 "TP?" H 16500 29250 50  0000 C BNN
+F 1 "TEST" H 16500 29200 50  0000 C CNN
+F 2 "" H 16500 28950 50  0001 C CNN
+F 3 "" H 16500 28950 50  0001 C CNN
+	1    16500 28950
+	-1   0    0    1
+$EndComp
+$Comp
+L TEST TP?
+U 1 1 5A3ADF04
+P 16450 25650
+F 0 "TP?" H 16450 25950 50  0000 C BNN
+F 1 "TEST" H 16450 25900 50  0000 C CNN
+F 2 "" H 16450 25650 50  0001 C CNN
+F 3 "" H 16450 25650 50  0001 C CNN
+	1    16450 25650
+	-1   0    0    1
+$EndComp
+Connection ~ 16450 25600
+Connection ~ 16500 28900
+$Comp
+L TEST TP?
+U 1 1 5A3C186F
+P 17200 22400
+F 0 "TP?" H 17200 22700 50  0000 C BNN
+F 1 "TEST" H 17200 22650 50  0000 C CNN
+F 2 "" H 17200 22400 50  0001 C CNN
+F 3 "" H 17200 22400 50  0001 C CNN
+	1    17200 22400
+	0    1    1    0
+$EndComp
+$Comp
+L TEST TP?
+U 1 1 5A3D3A31
+P 16250 23000
+F 0 "TP?" H 16250 23300 50  0000 C BNN
+F 1 "TEST" H 16250 23250 50  0000 C CNN
+F 2 "" H 16250 23000 50  0001 C CNN
+F 3 "" H 16250 23000 50  0001 C CNN
+	1    16250 23000
+	0    1    1    0
+$EndComp
 $EndSCHEMATC

Commit message: Ignore this commit; shouldn't be any changes
Other:
- note added: "POWER INPUT"
- note added: "POWER RAIL GENERATION"
- note added: "SHIFT REGISTER"
- moved on the sheet: C?, L?, Q?, R13, R?, U2, U?

Commit message: STARTED WORK ON CLOCK CIRCUITS FOR FE310-G000 AND FTD2232D CHIPS. ALSO DECIDED TO OPTIMIZE DIGITAL BOARD/BOARD INTERFACE TO REDUCE CABLE COST BY ADDING OPTOISOLATORS ON THE BOARD, GETTING RID OF INVERTED SIGNALS (THEY CAN BE INVERTED ON THE RECEIVING BOARD), AND SETTING UP JTAG IN SUCH A WAY THAT THE CABLES FOR IT ARE OPTIONAL (USER WILL BE ABLE TO SET THE JTAG CHAIN TO PROBOGATE TO ALL OTHER CONNECTED DISPLAYS, OR JUST STAY LOCAL TO THE BOARD. ONLY THE CLOCK CIRCUITS HAVE BEEN STARTED; DIGITAL SIGNAL CHANGES SOON TO COME
Parts:
- removed J?: Conn_01x08_Male, symbol Conn_01x08_Male
- removed Q? (x2): 2N7002, TO_SOT_Packages_SMD:SOT-23_Handsoldering, symbol 2N7002
- removed R? (x4): 47k, Resistors_SMD:R_0603_HandSoldering, symbol R
- removed R? (x2): NP_47k, Resistors_SMD:R_0603_HandSoldering, symbol R
- added C? (x4): 1uF, Capacitors_SMD:C_0603_HandSoldering, symbol C
- added J?: Conn_01x09_Male, symbol Conn_01x09_Male
- added Y? (x2): Crystal, symbol Crystal
Connections:
- net !ENABLE: now also J?.5 (Pin_5)
- net COL_DATA: now also J?.3 (Pin_3)
- net COL_SHCP: now also J?.4 (Pin_4)
- net GND: now also C?.2, C?.2, C?.2, C?.2
- net ROW_DATA: now also J?.1 (Pin_1)
- net ROW_SHCP: now also J?.2 (Pin_2)
- net at U1.10 (XTAL_XO): now also C?.1, Y?.2
- net TCK: now reaches U1.13 (JTAG_TCK)
- net TCK: now also J?.6 (Pin_6)
- net TDO: now reaches U1.14 (JTAG_TDO)
- net TDO: now also J?.7 (Pin_7)
- net TMS: now reaches U1.15 (JTAG_TMS)
- net TMS: now also J?.8 (Pin_8)
- net TDI: now reaches U1.16 (JTAG_TDI)
- net TDI: now also J?.9 (Pin_9)
- net at U1.9 (XTAL_XI): now also C?.1, Y?.1
- net at U2.43 (XTIN): now also C?.1, Y?.1
- net at U2.44 (XTOUT): now also C?.1, Y?.2
- no-connect marks 6 -> 4
Other:
- moved on the sheet: C1, C2, C?, J?, R11, R15, R9, R?, SW2, U3

Commit message: cleaned up clock circuits and created a footprint for the crystals. Still considering wheter to propgate the JTAG chain through all connected boards
Parts:
- removed C? (x4): 1uF, Capacitors_SMD:C_0603_HandSoldering, symbol C
- removed Y? (x2): Crystal, symbol Crystal
- added C? (x4): 12pF, Capacitors_SMD:C_0603_HandSoldering, symbol C
- added Y?: 16MHz, symbol CRYSTAL
- added Y?: 12MHz, symbol CRYSTAL
Connections:
- net GND: now also C?.2, C?.2, C?.2, C?.2, Y?.2, Y?.2, Y?.4, Y?.4
- net TCK: no longer J?.6 (Pin_6)
- net TDI: no longer J?.9 (Pin_9)
- net TDO: no longer J?.7 (Pin_7)
- net TMS: no longer J?.8 (Pin_8)
- net at U1.10 (XTAL_XO): now also C?.1, Y?.3
- net at U1.9 (XTAL_XI): now also C?.1, Y?.1
- net at U2.43 (XTIN): now also C?.1, Y?.1
- net at U2.44 (XTOUT): now also C?.1, Y?.3

Commit message: Thank goodness for version control! Accidentally deleted the signal inverters at some point, but the initial commit still had them! Added those, beefed up circuit protection with reverse input diode, TVS diodes at plugs/ports, connected UART and JTAG between FE310 and FT2232 and minor touchups.
Parts:
- removed D?: D, symbol D
- removed J?: 10x2_1&3_loaded_2.5mm_0.1\"_female_header, symbol 10x2_1&3_loaded_2.5mm_0.1"_female_header
- removed J?: Conn_01x09_Male, symbol Conn_01x09_Male
- removed R10, R? (x4): NP_47k, Resistors_SMD:R_0603_HandSoldering, symbol R
- removed R8: NP_0, Resistors_SMD:R_0603_HandSoldering, symbol R
- removed R? (x4): 47k, Resistors_SMD:R_0603_HandSoldering, symbol R
- removed SW1: NP_TACTILE_SWITCH, CUSTOM:TACTILE_SWITCH, symbol TACTILE_SWITCH
- added C?: 33nF, Capacitors_SMD:C_0603_HandSoldering, symbol C
- added C? (x5): 0.1uF, Capacitors_SMD:C_0603_HandSoldering, symbol C
- added C? (x2): 10nF, Capacitors_SMD:C_0603_HandSoldering, symbol C
- added D?: SMAJ12A, Footprint, symbol SMAJ12A
- added D?: NP_UCLAMP2501T.TCT, Footprint, symbol UCLAMP2501T.TCT
- added D?: UCLAMP2501T.TCT, Footprint, symbol UCLAMP2501T.TCT
- added D? (x6): SMF5.0A, Footprint, symbol SMF5.0A
- added D?: RSB6.8F2T106, symbol RSB6.8F2T106
- added D? (x2): DST2080S, symbol DST2080S
- added J?: 10x2_1&3_loaded_2.5mm_0.1\"_female_header, symbol 10x2_1&3_loaded_2.5mm_0.1"_female_header
- added J?: USB-C_Connector, symbol USB-C_Connector
- added L?: FBMH4532HM681-T, symbol FBMH4532HM681-T
- added Q? (x2): 2N7002, TO_SOT_Packages_SMD:SOT-23_Handsoldering, symbol 2N7002
- added R? (x2): 47, Resistors_SMD:R_0603_HandSoldering, symbol R
- added R? (x3): NP_0, Resistors_SMD:R_0603_HandSoldering, symbol R
- added R? (x6): NP_4.7k, Resistors_SMD:R_0603_HandSoldering, symbol R
- added R? (x5): NP, Resistors_SMD:R_0603_HandSoldering, symbol R
- added R? (x2): 0, Resistors_SMD:R_0603_HandSoldering, symbol R
- added R? (x9): 4.7k, Resistors_SMD:R_0603_HandSoldering, symbol R
- added R? (x5): 47k, Resistors_SMD:R_0603_HandSoldering, symbol R
- added R?: 470, Resistors_SMD:R_0603_HandSoldering, symbol R
- added R?: 13k, Resistors_SMD:R_0603_HandSoldering, symbol R
- added SW?: NP_TACTILE_SWITCH, CUSTOM:TACTILE_SWITCH, symbol TACTILE_SWITCH
- added TP? (x16): TEST, symbol TEST
- R137: renamed from R?; value NP_47k -> NP_4.7k
- R138: renamed from R?; value 47k -> 4.7k
- Y2: renamed from Y?; value 12MHz -> 6MHz
- gave numbers to parts that had none: 317
Connections:
- net COL_RESET is gone; now on net !COL_RESET: U12.10 (MR), U13.10 (MR), U14.10 (MR), U15.10 (MR), U16.10 (MR), U17.10 (MR), U18.10 (MR)
- net EN_1V8 is gone; now on net +3V3: U4.5 (EN)
- net EN_3V3 is gone; now on net +5V: U5.5 (EN)
- net ROW_RESET is gone; now on net !ROW_RESET: U10.10 (MR), U11.10 (MR), U8.10 (MR), U9.10 (MR)
- net !COL_RESET: now also R?.1, R?.2, TP?.1
- net !COL_SHCP: now also U12.11 (SHCP), U13.11 (SHCP), U14.11 (SHCP), U15.11 (SHCP), U16.11 (SHCP), U17.11 (SHCP), U18.11 (SHCP), Q?.3 (D), R?.2, TP?.1; no longer U12.12 (STCP), U13.12 (STCP), U14.12 (STCP), U15.12 (STCP), U16.12 (STCP), U17.12 (STCP), U18.12 (STCP)
- net !ENABLE: now also R?.1, R?.2, TP?.1
- net !ROW_RESET: now also R?.1, R?.2, TP?.1
- net !ROW_SHCP: now also U10.11 (SHCP), U11.11 (SHCP), U8.11 (SHCP), U9.11 (SHCP), Q?.3 (D), R?.2, TP?.1; no longer U10.12 (STCP), U11.12 (STCP), U8.12 (STCP), U9.12 (STCP)
- net +12V: now also L?.1, R?.2, TP?.1; no longer J2.1 (Pin_1), J2.2 (Pin_2), J4.1, TP1.1
- net +1V8: now also C10.1, C11.1, C19.1, C6.1, U1.7 (PLL_AVDD), R?.1
- net +24V: now also D?.1 (K), J?.3, J?.4
- net +3V3: now also U2.14 (VCCIOA), U2.31 (VCCIOB), C?.1, C?.1, C?.1, R?.2, R?.2, R?.2; no longer C10.1, C11.1, C19.1, C6.1, U1.7 (PLL_AVDD)
- net +5V: now also U2.3 (VCC), U2.42 (VCC), C?.1, C?.1, C?.1, R?.1, R?.1, R?.1, R?.1, R?.1, R?.1, R?.1, R?.1, R?.1, R?.2
- net COL00: now also J?.37
- net COL01: now also J?.38
- net COL02: now also J?.39
- net COL03: now also J?.40
- net COL04: now also J?.41
- net COL05: now also J?.42
- net COL06: now also J?.43
- net COL07: now also J?.44
- net COL08: now also J?.45
- net COL09: now also J?.46
- net COL10: now also J?.47
- net COL11: now also J?.48
- net COL12: now also J?.49
- net COL13: now also J?.50
- net COL14: now also J?.51
- net COL15: now also J?.52
- net COL16: now also J?.53
- net COL17: now also J?.54
- net COL18: now also J?.55
- net COL19: now also J?.56
- net COL20: now also J?.57
- net COL21: now also J?.58
- net COL22: now also J?.59
- net COL23: now also J?.60
- net COL24: now also J?.61
- net COL25: now also J?.62
- net COL26: now also J?.63
- net COL27: now also J?.64
- net COL_IN: now also TP?.1
- net COL_SHCP: now also U12.12 (STCP), U13.12 (STCP), U14.12 (STCP), U15.12 (STCP), U16.12 (STCP), U17.12 (STCP), U18.12 (STCP), Q?.1 (G), R?.1, R?.2, TP?.1; no longer U12.11 (SHCP), U13.11 (SHCP), U14.11 (SHCP), U15.11 (SHCP), U16.11 (SHCP), U17.11 (SHCP), U18.11 (SHCP)
- net COL_SR_IN: now also D?.1 (K), TP?.1
- net COL_SR_OUT: now also D?.1 (K), TP?.1
- net GND: now also U2.47 (TEST), C?.2, C?.2, C?.2, C?.2, C?.2, C?.2, C?.2, C?.2, D?.2 (A), D?.2 (A), D?.2 (A), D?.2 (A), D?.2 (A), D?.2 (A), D?.2 (A), D?.2 (A), D?.2 (A), D?.3, J?.A1 (GND), J?.A12 (GND), J?.B1 (GND), J?.B12 (GND), Q?.2 (S), Q?.2 (S), R?.1, R?.1, R?.1, R?.1, R?.1, R?.2, R?.2, R?.2, R?.2, R?.2, R?.2, R?.2, R?.2
- net LED_CTL: now also J?.1, J?.2
- net ROW00N: now also J?.36
- net ROW00P: now also J?.35
- net ROW01N: now also J?.6
- net ROW01P: now also J?.5
- net ROW02N: now also J?.34
- net ROW02P: now also J?.33
- net ROW03N: now also J?.8
- net ROW03P: now also J?.7
- net ROW04N: now also J?.32
- net ROW04P: now also J?.31
- net ROW05N: now also J?.10
- net ROW05P: now also J?.9
- net ROW06N: now also J?.30
- net ROW06P: now also J?.29
- net ROW07N: now also J?.12
- net ROW07P: now also J?.11
- net ROW08N: now also J?.28
- net ROW08P: now also J?.27
- net ROW09N: now also J?.14
- net ROW09P: now also J?.13
- net ROW10N: now also J?.26
- net ROW10P: now also J?.25
- net ROW11N: now also J?.16
- net ROW11P: now also J?.15
- net ROW12N: now also J?.24
- net ROW12P: now also J?.23
- net ROW13N: now also J?.18
- net ROW13P: now also J?.17
- net ROW14N: now also J?.22
- net ROW14P: now also J?.21
- net ROW15N: now also J?.20
- net ROW15P: now also J?.19
- net ROW_IN: now also R?.1, R?.2, TP?.1
- net ROW_SHCP: now also U10.12 (STCP), U11.12 (STCP), U8.12 (STCP), U9.12 (STCP), Q?.1 (G), R?.1, R?.2, TP?.1; no longer U10.11 (SHCP), U11.11 (SHCP), U8.11 (SHCP), U9.11 (SHCP)
- net ROW_SR_IN: now also D?.1 (K), TP?.1
- net ROW_SR_OUT: now also D?.1 (K), TP?.1
- net TCK: now also U2.24 (ADBUS0)
- net TDI: now also U2.23 (ADBUS1)
- net TDO: now also U2.22 (ADBUS2)
- net TMS: now also U2.21 (ADBUS3)
- net at C21.1, U1.10 (XTAL_XO), Y1.3: now also R?.1
- net at U1.18 (AON_PMU_DWAKEUP_N): now also D?.1 (K), R?.2, SW?.3, SW?.4
- net RESET: now reaches R11.2, SW2.3, SW2.4, U1.24 (AON_ERST_N)
- net RESET: now also D?.1 (K)
- net UART_FE_RX: now reaches U1.38 (GPIO_16)
- net UART_FE_RX: now also R?.1, R?.2, R?.2, R?.2
- net UART_FE_TX: now reaches U1.39 (GPIO_17)
- net UART_FE_TX: now also R?.1, R?.2, R?.2, R?.2
- net at C20.1, U1.9 (XTAL_XI), Y1.1: now also R?.2
- net UART_FT_RX: now reaches U2.39 (BDBUS1)
- net UART_FT_RX: now also R?.1, R?.1
- net at U2.4 (~RESET): now also R?.1, R?.2
- net UART_FT_TX: now reaches U2.40 (BDBUS0)
- net UART_FT_TX: now also R?.1, R?.1
- net FT2232D_AVCC: now reaches U2.46 (AVCC)
- net FT2232D_AVCC: now also C?.1, R?.2
- net at U2.5 (~RSTOUT): now also R13.1
- net at U2.6 (3V3OUT): now also C?.1; no longer R13.1
- net at R13.2, U2.7 (USBDP): now also D?.1, R?.1
- net at U2.8 (USBDM): now also D?.2, R?.1
- net at L1.2, U7.1 (SW), U7.2 (SW): now also D?.2 (A)
- net EN_5V: no longer names the net of U6.5 (EN)
- net EN_5V: now also R?.1, R?.2
- new net: D?.2 (A), J2.1 (Pin_1), J2.2 (Pin_2), J4.1, TP1.1
- new net: R?.1, SW?.1, SW?.2
- new net: D?.1 (K), D?.1 (K), L?.2, TP?.1
- new net: D?.1 (K), TP?.1
- new net D+: J?.A6 (D+), J?.B6 (D+), R?.2
- new net D-: J?.A7 (D-), J?.B7 (D-), R?.2
- new net USB-C_VBUS: D?.1 (K), J?.A4 (VBUS), J?.A9 (VBUS), J?.B4 (VBUS), J?.B9 (VBUS), R?.1
- no-connect marks 4 -> 22
Other:
- note added: "-USB TO JTAG\n-JTAG\nGPIO\n-CONSOLE\n-INPUT ESD PROTECTION\n-INPUT REVERSE PROTECTION\n-TESTPOINTS\n-POWER SEQUENCING\nCALCULATE MAX CLK RATE BASED ON INPUT CAPACITANCE AND RESISTANCE OF FETS."
- note added: "AVOID STUBS"
- note added: "FT2232D POWER"
- note added: "SILKSCREEN:\n12V (13V MAX)"
- note added: "STRAPPING"
- note added: "UART_CYA"
- note added: "USB TO SERIAL"
- note removed: "CONSIDER LOWERING RESISTOR VALUE\nIF INPUT CAPACITANCE TO SHIFT\nREGISTER WOULD CAUSE SKEW"
- note removed: "USB TO JTAG\nJTAG\nGPIO\nCONSOLE\nINPUT ESD PROTECTION\nINPUT REVERSE PROTECTION\nTESTPOINTS\nPOWER SEQUENCING\nCALCULATE MAX CLK RATE BASED ON INPUT CAPACITANCE AND RESISTANCE OF FETS."
- moved on the sheet: C20, C21, C22, C23, C24, C25, C26, C28, C30, C33, C35, C37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
