File: flipdot_driver.sch (KiCad schematic (older format))
At the start: 436 parts, among them J2 Screw_Terminal_01x04, J4 Barrel_Jack, Q1 2N7002, Q10 2N7002, Q11 2N7002, Q12 DMG6602, Q13 DMG6602, Q14 2N7002, Q15 2N7002, Q16 DMG6602, Q17 DMG6602, Q18 2N7002, Q19 2N7002, Q2 2N7002, Q20 DMG6602, Q21 DMG6602, Q22 2N7002, Q23 2N7002, Q24 DMG6602, Q25 DMG6602, Q26 2N7002, Q27 2N7002, Q28 DMG6602, Q29 DMG6602, Q3 DMG6602, Q30 2N7002, Q31 2N7002, Q32 DMG6602, Q33 DMG6602, Q34 2N7002, Q35 2N7002, Q36 DMG6602, Q37 DMG6602, Q38 2N7002, Q39 2N7002, Q4 DMG6602, Q40 DMG6602, Q41 DMG6602, Q42 2N7002, Q43 2N7002, Q44 DMG6602, Q45 DMG6602, Q46 2N7002, Q47 2N7002, Q48 DMG6602, Q49 DMG6602, Q5 2N7002, Q50 2N7002, Q51 2N7002, Q52 DMG6602, Q53 DMG6602, Q54 2N7002, Q55 2N7002, Q56 DMG6602, Q57 DMG6602, Q58 2N7002, Q59 2N7002, Q6 2N7002, Q60 DMG6602, Q61 DMG6602, Q62 2N7002, Q63 2N7002, Q64 DMG6602, Q65 DMG6602, Q66 2N7002, Q67 2N7002, Q68 2N7002, Q69 DMG6602, Q7 BUZ11, Q70 DMG6602, Q71 DMG6602, Q72 2N7002, Q73 2N7002, Q74 2N7002, Q75 DMG6602, Q76 DMG6602, Q77 DMG6602, Q78 2N7002, Q79 2N7002, Q8 DMG6602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

Commit message: Changed bias resistors to more sane values and included my kicad library
Parts:
- removed D?: SMF5.0A, Footprint, symbol SMF5.0A
- removed R1, R100, R101, R102, R103, R104, R105, R106, R107, R108, R109, R110, R111, R112, R113, R114, R115, R116, R117, R118, R119, R120, R121, R122, R123, R124, R125, R126, R127, R128, R129, R130, R131, R132, R133, R134, R135, R136, R14, R147, R148, R149, R150, R151, R152, R153, R154, R155, R156, R157, R158, R159, R16, R160, R161, R162, R163, R164, R17, R18, R19, R2, R20, R21, R22, R23, R24, R25, R26, R27, R28, R29, R3, R30, R31, R32, R33, R34, R35, R36, R37, R38, R39, R4, R40, R41, R42, R43, R44, R47, R48, R49, R50, R51, R52, R6, R65, R66, R67, R68, R69, R70, R71, R72, R73, R74, R75, R76, R77, R78, R79, R80, R81, R82, R83, R84, R85, R86, R87, R88, R89, R90, R91, R92, R93, R94, R95, R96, R97, R98, R99: 47k, Resistors_SMD:R_0603_HandSoldering, symbol R
- removed TP?: TEST, symbol TEST
- added R? (x131): 4.7k, Resistors_SMD:R_0603_HandSoldering, symbol R
- R11, R15, R5, R7, R?: value 47k -> 4.7k
Connections:
- net !COL_RESET: now also U1.28 (GPIO_3)
- net !ENABLE: now also U1.29 (GPIO_4)
- net !ROW_RESET: now also U1.27 (GPIO_2)
- net +12V: now also R?.1, R?.1, R?.1, R?.1, R?.1, R?.1, R?.1, R?.1, R?.1, R?.1, R?.1, R?.1, R?.1, R?.1, R?.1, R?.1, R?.1, R?.1, R?.1, R?.1, R?.1, R?.1, R?.1, R?.1, R?.1, R?.1, R?.1, R?.1, R?.1, R?.1, R?.1, R?.1, R?.1, R?.1, R?.1, R?.1, R?.1, R?.1, R?.1, R?.1, R?.1, R?.1, R?.1
- net COL00_OFF: now also R?.1
- net COL00_ON: now also R?.1
- net COL01_OFF: now also R?.1
- net COL01_ON: now also R?.1
- net COL02_OFF: now also R?.1
- net COL02_ON: now also R?.1
- net COL03_OFF: now also R?.1
- net COL03_ON: now also R?.1
- net COL04_OFF: now also R?.1
- net COL04_ON: now also R?.1
- net COL05_OFF: now also R?.1
- net COL05_ON: now also R?.1
- net COL06_OFF: now also R?.1
- net COL06_ON: now also R?.1
- net COL07_OFF: now also R?.1
- net COL07_ON: now also R?.1
- net COL08_OFF: now also R?.1
- net COL08_ON: now also R?.1
- net COL09_OFF: now also R?.1
- net COL09_ON: now also R?.1
- net COL10_OFF: now also R?.1
- net COL10_ON: now also R?.1
- net COL11_OFF: now also R?.1
- net COL11_ON: now also R?.1
- net COL12_OFF: now also R?.1
- net COL12_ON: now also R?.1
- net COL13_OFF: now also R?.1
- net COL13_ON: now also R?.1
- net COL14_OFF: now also R?.1
- net COL14_ON: now also R?.1
- net COL15_OFF: now also R?.1
- net COL15_ON: now also R?.1
- net COL16_OFF: now also R?.1
- net COL16_ON: now also R?.1
- net COL17_OFF: now also R?.1
- net COL17_ON: now also R?.1
- net COL18_OFF: now also R?.1
- net COL18_ON: now also R?.1
- net COL19_OFF: now also R?.1
- net COL19_ON: now also R?.1
- net COL20_OFF: now also R?.1
- net COL20_ON: now also R?.1
- net COL21_OFF: now also R?.1
- net COL21_ON: now also R?.1
- net COL22_OFF: now also R?.1
- net COL22_ON: now also R?.1
- net COL23_OFF: now also R?.1
- net COL23_ON: now also R?.1
- net COL24_OFF: now also R?.1
- net COL24_ON: now also R?.1
- net COL25_OFF: now also R?.1
- net COL25_ON: now also R?.1
- net COL26_OFF: now also R?.1
- net COL26_ON: now also R?.1
- net COL27_OFF: now also R?.1
- net COL27_ON: now also R?.1
- net COL_IN: now also U1.33 (GPIO_9)
- net COL_SHCP: now also U1.35 (GPIO_11)
- net GND: now also R?.2, R?.2, R?.2, R?.2, R?.2, R?.2, R?.2, R?.2, R?.2, R?.2, R?.2, R?.2, R?.2, R?.2, R?.2, R?.2, R?.2, R?.2, R?.2, R?.2, R?.2, R?.2, R?.2, R?.2, R?.2, R?.2, R?.2, R?.2, R?.2, R?.2, R?.2, R?.2, R?.2, R?.2, R?.2, R?.2, R?.2, R?.2, R?.2, R?.2, R?.2, R?.2, R?.2, R?.2, R?.2, R?.2, R?.2, R?.2, R?.2, R?.2, R?.2, R?.2, R?.2, R?.2, R?.2, R?.2, R?.2, R?.2, R?.2, R?.2, R?.2, R?.2, R?.2, R?.2, R?.2, R?.2, R?.2, R?.2, R?.2, R?.2, R?.2, R?.2, R?.2, R?.2, R?.2, R?.2, R?.2, R?.2, R?.2, R?.2, R?.2, R?.2, R?.2, R?.2, R?.2, R?.2, R?.2, R?.2
- net ROW00_OFF: now also R?.1
- net ROW00_ON: now also R?.1
- net ROW01_OFF: now also R?.1
- net ROW01_ON: now also R?.1
- net ROW02_OFF: now also R?.1
- net ROW02_ON: now also R?.1
- net ROW03_OFF: now also R?.1
- net ROW03_ON: now also R?.1
- net ROW04_OFF: now also R?.1
- net ROW04_ON: now also R?.1
- net ROW05_OFF: now also R?.1
- net ROW05_ON: now also R?.1
- net ROW06_OFF: now also R?.1
- net ROW06_ON: now also R?.1
- net ROW07_OFF: now also R?.1
- net ROW07_ON: now also R?.1
- net ROW08_OFF: now also R?.1
- net ROW08_ON: now also R?.1
- net ROW09_OFF: now also R?.1
- net ROW09_ON: now also R?.1
- net ROW10_OFF: now also R?.1
- net ROW10_ON: now also R?.1
- net ROW11_OFF: now also R?.1
- net ROW11_ON: now also R?.1
- net ROW12_OFF: now also R?.1
- net ROW12_ON: now also R?.1
- net ROW13_OFF: now also R?.1
- net ROW13_ON: now also R?.1
- net ROW14_OFF: now also R?.1
- net ROW14_ON: now also R?.1
- net ROW15_OFF: now also R?.1
- net ROW15_ON: now also R?.1
- net ROW_IN: now also U1.31 (GPIO_5)
- net ROW_SHCP: now also U1.34 (GPIO_10)
- net at R12.2: now also U1.41 (GPIO_19); no longer U1.25 (GPIO_0)
- net PIEZO_1: now reaches U1.26 (GPIO_1)
- net PIEZO_2: now reaches U1.37 (GPIO_13)
- net at Q2.3 (D), Q4.3 (G): now also R?.2
- net at Q86.3 (D), Q89.3 (G): now also R?.2
- net at Q5.3 (D), Q8.3 (G): now also R?.2
- net at Q10.3 (D), Q12.3 (G): now also R?.2
- net at Q14.3 (D), Q16.3 (G): now also R?.2
- net at Q18.3 (D), Q20.3 (G): now also R?.2
- net at Q22.3 (D), Q24.3 (G): now also R?.2
- net at Q26.3 (D), Q28.3 (G): now also R?.2
- net at Q30.3 (D), Q32.3 (G): now also R?.2
- net at Q34.3 (D), Q36.3 (G): now also R?.2
- net at Q38.3 (D), Q40.3 (G): now also R?.2
- net at Q42.3 (D), Q44.3 (G): now also R?.2
- net at Q46.3 (D), Q48.3 (G): now also R?.2
- net at Q50.3 (D), Q52.3 (G): now also R?.2
- net at Q54.3 (D), Q56.3 (G): now also R?.2
- net at Q58.3 (D), Q60.3 (G): now also R?.2
- net at Q62.3 (D), Q64.3 (G): now also R?.2
- net at Q66.3 (D), Q69.3 (G): now also R?.2
- net at Q72.3 (D), Q75.3 (G): now also R?.2
- net at Q67.3 (D), Q70.3 (G): now also R?.2
- net at Q73.3 (D), Q76.3 (G): now also R?.2
- net at Q78.3 (D), Q81.3 (G): now also R?.2
- net at Q84.3 (D), Q87.3 (G): now also R?.2
- net at Q79.3 (D), Q82.3 (G): now also R?.2
- net at Q68.3 (D), Q71.3 (G): now also R?.2
- net at Q74.3 (D), Q77.3 (G): now also R?.2
- net at Q80.3 (D), Q83.3 (G): now also R?.2
- net at Q85.3 (D), Q88.3 (G): now also R?.2
- net at Q63.3 (D), Q65.3 (G): now also R?.2
- net at Q6.3 (D), Q9.3 (G): now also R?.2
- net at Q11.3 (D), Q13.3 (G): now also R?.2
- net at Q15.3 (D), Q17.3 (G): now also R?.2
- net at Q19.3 (D), Q21.3 (G): now also R?.2
- net at Q23.3 (D), Q25.3 (G): now also R?.2
- net at Q27.3 (D), Q29.3 (G): now also R?.2
- net at Q31.3 (D), Q33.3 (G): now also R?.2
- net at Q35.3 (D), Q37.3 (G): now also R?.2
- net at Q39.3 (D), Q41.3 (G): now also R?.2
- net at Q43.3 (D), Q45.3 (G): now also R?.2
- net at Q47.3 (D), Q49.3 (G): now also R?.2
- net at Q51.3 (D), Q53.3 (G): now also R?.2
- net at Q55.3 (D), Q57.3 (G): now also R?.2
- net at Q59.3 (D), Q61.3 (G): now also R?.2
- new net PIEZO_0: U1.25 (GPIO_0)
Other:
- note added: "CLOCK INVERSION"
- note added: "INTERFACE"
- note added: "PANEL EXTENSION"
- note added: "RISC-V uC"
- note added: "SHIFT REGISTERS"
- note removed: "-USB TO JTAG\n-JTAG\nGPIO\n-CONSOLE\n-INPUT ESD PROTECTION\n-INPUT REVERSE PROTECTION\n-TESTPOINTS\n-POWER SEQUENCING\nCALCULATE MAX CLK RATE BASED ON INPUT CAPACITANCE AND RESISTANCE OF FETS."
- note removed: "SHIFT REGISTER"
- moved on the sheet: C1, C10, C11, C12, C13, C14, C15, C16, C17, C18, C19, C2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
