File: flipdot_driver.sch (KiCad schematic (older format))
At the start: 434 parts, among them J2 Screw_Terminal_01x04, J4 Barrel_Jack, Q1 2N7002, Q10 2N7002, Q11 2N7002, Q12 DMG6602, Q13 DMG6602, Q14 2N7002, Q15 2N7002, Q16 DMG6602, Q17 DMG6602, Q18 2N7002, Q19 2N7002, Q2 2N7002, Q20 DMG6602, Q21 DMG6602, Q22 2N7002, Q23 2N7002, Q24 DMG6602, Q25 DMG6602, Q26 2N7002, Q27 2N7002, Q28 DMG6602, Q29 DMG6602, Q3 DMG6602, Q30 2N7002, Q31 2N7002, Q32 DMG6602, Q33 DMG6602, Q34 2N7002, Q35 2N7002, Q36 DMG6602, Q37 DMG6602, Q38 2N7002, Q39 2N7002, Q4 DMG6602, Q40 DMG6602, Q41 DMG6602, Q42 2N7002, Q43 2N7002, Q44 DMG6602, Q45 DMG6602, Q46 2N7002, Q47 2N7002, Q48 DMG6602, Q49 DMG6602, Q5 2N7002, Q50 2N7002, Q51 2N7002, Q52 DMG6602, Q53 DMG6602, Q54 2N7002, Q55 2N7002, Q56 DMG6602, Q57 DMG6602, Q58 2N7002, Q59 2N7002, Q6 2N7002, Q60 DMG6602, Q61 DMG6602, Q62 2N7002, Q63 2N7002, Q64 DMG6602, Q65 DMG6602, Q66 2N7002, Q67 2N7002, Q68 2N7002, Q69 DMG6602, Q7 BUZ11, Q70 DMG6602, Q71 DMG6602, Q72 2N7002, Q73 2N7002, Q74 2N7002, Q75 DMG6602, Q76 DMG6602, Q77 DMG6602, Q78 2N7002, Q79 2N7002, Q8 DMG6602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

Commit message: moar bugfixes
Parts:
- added J?: Conn_01x08, symbol Conn_01x08
- added L?: FBMH4532HM681-T, symbol FBMH4532HM681-T
Connections:
- net COL_SR_IN is gone; now on net COL_IN: D?.1 (K), TP?.1, U12.14 (DS), U19.3
- net ROW_SR_IN is gone; now on net ROW_IN: D?.1 (K), TP?.1, U19.1, U8.14 (DS)
- net !ENABLE: now also J?.5 (Pin_5)
- net +5V: no longer C?.1, C?.1, C?.1, R?.1, U2.3 (VCC), U2.42 (VCC)
- net COL_DATA: now also J?.3 (Pin_3)
- net COL_SHCP: now also J?.4 (Pin_4)
- net ROW_DATA: now also J?.1 (Pin_1)
- net ROW_SHCP: now also J?.2 (Pin_2)
- net UART_FE_RX: now also R?.2; no longer R?.2
- net UART_FE_TX: now also R?.2; no longer R?.2
- net COL_SR_OUT renamed COL_OUT
- net ROW_SR_OUT renamed ROW_OUT
- net USB-C_VBUS: no longer names the net of D?.1 (K), J?.A4 (VBUS), J?.A9 (VBUS), J?.B4 (VBUS), J?.B9 (VBUS)
- net USB-C_VBUS: now also L?.2; no longer R?.1
- new net FT2232D_VCC: C?.1, C?.1, C?.1, L?.1, R?.1, R?.1, U2.3 (VCC), U2.42 (VCC)
Other:
- note added: "FLIPDOT BOARD INTERFACE"
- note removed: "INTERFACE"
- moved on the sheet: D?, J?, R?

Commit message: bugfixes and added aux io
Parts:
- removed J?: Conn_01x08, symbol Conn_01x08
- added D? (x6): LED, symbol LED
- added J?: Conn_01x06, symbol Conn_01x06
- added J?: Conn_01x08_Male, symbol Conn_01x08_Male
- added R? (x6): 470, Resistors_SMD:R_0603_HandSoldering, symbol R
Connections:
- net !ENABLE: now also J?.5 (Pin_5)
- net COL_DATA: now also J?.3 (Pin_3)
- net COL_SHCP: now also J?.4 (Pin_4)
- net GND: now also D?.1 (K), D?.1 (K), D?.1 (K), D?.1 (K), D?.1 (K), D?.1 (K)
- net ROW_DATA: now also J?.1 (Pin_1)
- net ROW_SHCP: now also J?.2 (Pin_2)
- net AUX_0: now reaches U1.36 (GPIO_12)
- net AUX_0: now also J?.6 (Pin_6), R?.2
- net AUX_1: now reaches U1.40 (GPIO_18)
- net AUX_1: now also J?.5 (Pin_5), R?.2
- net AUX_2: now reaches U1.42 (GPIO_20)
- net AUX_2: now also J?.4 (Pin_4), R?.2
- net AUX_3: now reaches U1.43 (GPIO_21)
- net AUX_3: now also J?.3 (Pin_3), R?.2
- net AUX_4: now reaches U1.44 (GPIO_22)
- net AUX_4: now also J?.2 (Pin_2), R?.2
- net AUX_5: now reaches U1.45 (GPIO_23)
- net AUX_5: now also J?.1 (Pin_1), R?.2
- new net: D?.2 (A), R?.1 (x6)
Other:
- note added: "AUXILLARY IO"

Commit message: Moved my cucstom components here, and made a bunch of changes to schematic
Parts:
- removed D?: UCLAMP2501T.TCT, Footprint, symbol UCLAMP2501T.TCT
- removed D? (x6): LED, symbol LED
- removed J?: Conn_01x06, symbol Conn_01x06
- removed unit 2 of Q13
- removed unit 2 of Q17
- removed unit 2 of Q21
- removed unit 2 of Q25
- removed unit 2 of Q29
- removed unit 2 of Q33
- removed unit 2 of Q37
- removed unit 2 of Q4
- removed unit 2 of Q41
- removed unit 2 of Q45
- removed unit 2 of Q49
- removed unit 2 of Q53
- removed unit 2 of Q57
- removed unit 2 of Q65
- removed unit 2 of Q9
- removed R? (x6): 470, Resistors_SMD:R_0603_HandSoldering, symbol R
- removed U1: FE310-G000, CUSTOM:QFN-48-1EP_6x6mm_Pitch0.4mm_PadLength1.4mm, symbol FE310-G000-RESCUE-flipdot_driver
- added D? (x7): NP_UCLAMP2501T.TCT, Footprint, symbol UCLAMP2501T.TCT
- added D?: UCLAMP2501T.TCT, Footprint, symbol UCLAMP2501T.TCT
- added D? (x7): LED, symbol LED
- added D? (x32): MMBZ5243BLT1G, symbol MMBZ5243BLT1G
- added D? (x7): SMF5.0A, Footprint, symbol SMF5.0A
- added J?: NP_Conn_01x06_Male, symbol Conn_01x06_Male
- added Q? (x6): 2N7002, TO_SOT_Packages_SMD:SOT-23_Handsoldering, symbol 2N7002
- added Q? (x15): DMG6602, TSOT-23-6, symbol DMG6602
- added R? (x8): 4.7k, Resistors_SMD:R_0603_HandSoldering, symbol R
- added R? (x6): 470, Resistors_SMD:R_0603_HandSoldering, symbol R
- added R?: 2k, Resistors_SMD:R_0603_HandSoldering, symbol R
- added TP? (x17): TEST, symbol TEST
- added U?: FE310-G000, symbol FE310-G000
- R?: value NP_0 -> 4.7k
- R?: value 4.7k -> NP_0
Connections:
- net labels added: !RESET, !WAKEUP
- net labels removed: RESET
- wire segments 1601 -> 1807
Other:
- note added: "AUX IO"
- note added: "DOT DRIVERS"
- note added: "FE310"
- note added: "FE310 BYPASS"
- note added: "FT2232D BYPASS"
- note added: "INCLUDE FILLED RECTANGLES\nON SILKSCREEN NEAR EACH\nLED TO WRITE LABELS ON"
- note added: "PLACE CLOSE TO CONNECTOR"
- note added: "PUT SYMBOL FOR CENTER-POSITIVE\nCONNECTOR, VOLTAGE RANGE, AND\nBARREL JACK DIMENSIONS FOR MATE\nON SILKSCREEN"
- note added: "ROW_SHCP AND COL_SHCP\nARE PULLED DOWN IN THE\nCLOCK INVERSION SECTION"
- note added: "SILKSCREEN: POPULATE TVS DIODES\nAS APPROPRIATE FOR USE\nWITH GPIO PERIPHERALS"
- note added: "SILKSCREEN:\n0 = ROW\n1 = COL\n2 = NC\n3 = NC\nON = DUPLICATE\nOFF = EXTEND"
- note added: "SILKSCREEN:\n12V (12.9V MAX)"
- note added: "UART CYA"
- note removed: "AUXILLARY IO"
- note removed: "BYPASS CAPS FOR FE310\nPLACE AS CLOSE TO RESPECTIVE PADS AS POSSIBLE\nLEFTMOST CAPS ARE MOST CRITICAL"
- note removed: "FT2232D POWER"
- note removed: "PUT SYMBOL FOR CENTER-POSITIVE\nCONNECTOR AND VOLTAGE RANGE\nON SILKSCREEN"
- note removed: "RISC-V uC"
- note removed: "SILKSCREEN:\n12V (13V MAX)"
- note removed: "UART_CYA"
- moved on the sheet: C1, C10, C11, C12, C13, C14, C15, C16, C17, C18, C19, C2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

Commit message: Cleaned repo up some
Parts:
- U2: symbol FT2232D-RESCUE-flipdot_driver -> FT2232D
- U3: symbol IS25LP128-JBLE-RESCUE-flipdot_driver -> IS25LP128-JBLE

Commit message: updated whole project from kicad 4 to 5
Parts:
- C1, C10, C11, C12, C13, C14, C15, C16, C17, C18, C19, C2, C20, C21, C25, C26, C27, C28, C29, C3, C30, C31, C32, C33, C34, C35, C36, C37, C38, C39, C4, C40, C41, C42, C43, C44, C45, C46, C47, C48, C49, C5, C50, C51, C52, C53, C54, C55, C56, C57, C58, C59, C6, C60, C61, C62, C63, C64, C65, C66, C67, C68, C69, C7, C70, C71, C72, C73, C74, C75, C76, C77, C78, C79, C8, C80, C9, C? (x8): symbol C -> Device:C
- C22, C23, C24: symbol CP1 -> Device:CP1
- D?: symbol SMAJ12A -> custom:SMAJ12A
- D? (x9): symbol UCLAMP2501T.TCT -> custom:UCLAMP2501T.TCT
- D? (x12): symbol SMF5.0A -> custom:SMF5.0A
- D?: symbol RSB6.8F2T106 -> custom:RSB6.8F2T106
- D? (x2): symbol DST2080S -> custom:DST2080S
- D? (x7): symbol LED -> Device:LED
- D? (x32): symbol MMBZ5243BLT1G -> custom:MMBZ5243BLT1G
- J2: symbol Screw_Terminal_01x04 -> Connector:Screw_Terminal_01x04
- J4: symbol Barrel_Jack -> Connector:Barrel_Jack
- J?: value 10x2_1&3_loaded_2.5mm_0.1\"_female_header -> 10x2_1&3_loaded_2.5mm_0.1in_female_header; symbol 10x2_1&3_loaded_2.5mm_0.1"_female_header -> custom:10x2_1&3_loaded_2.5mm_0.1in_female_header
- J?: symbol Conn_01x06_Male -> Connector:Conn_01x06_Male
- J?: symbol USB-C_Connector -> custom:USB-C_Connector
- J?: symbol Conn_01x08_Male -> Connector:Conn_01x08_Male
- L1, L2, L3, L4: symbol L -> Device:L
- L? (x2): symbol FBMH4532HM681-T -> custom:FBMH4532HM681-T
- Q1, Q10, Q11, Q14, Q15, Q18, Q19, Q2, Q22, Q23, Q26, Q27, Q30, Q31, Q34, Q35, Q38, Q39, Q42, Q43, Q46, Q47, Q5, Q50, Q51, Q54, Q55, Q58, Q59, Q6, Q62, Q63, Q66, Q67, Q68, Q72, Q73, Q74, Q78, Q79, Q80, Q84, Q85, Q86, Q? (x8): symbol 2N7002 -> Transistor_FET:2N7002
- Q12, Q13, Q16, Q17, Q20, Q21, Q24, Q25, Q28, Q29, Q3, Q32, Q33, Q36, Q37, Q4, Q40, Q41, Q44, Q45, Q48, Q49, Q52, Q53, Q56, Q57, Q60, Q61, Q64, Q65, Q69, Q70, Q71, Q75, Q76, Q77, Q8, Q81, Q82, Q83, Q87, Q88, Q89, Q9, Q? (x15): symbol DMG6602 -> custom:DMG6602
- Q7: symbol BUZ11 -> Transistor_FET:BUZ11
- R11, R12, R13, R137, R138, R15, R45, R46, R5, R53, R54, R55, R56, R57, R58, R59, R60, R61, R62, R63, R64, R7, R9, R? (x180): symbol R -> Device:R
- SW2, SW?: symbol TACTILE_SWITCH -> custom:TACTILE_SWITCH
- TP1, TP2, TP3, TP4, TP5, TP6, TP7, TP8, TP9, TP? (x32): symbol TEST -> Connector:TestPoint
- U10, U11, U12, U13, U14, U15, U16, U17, U18, U8, U9: symbol 74HC595 -> custom:74HC595
- U19: symbol SPDT_DIP_SWITCH_4_CIRCUIT -> custom:SPDT_DIP_SWITCH_4_CIRCUIT
- U2: symbol FT2232D -> custom:FT2232D
- U3: symbol IS25LP128-JBLE -> custom:IS25LP128-JBLE
- U4, U5, U6: symbol AP65111A -> custom:AP65111A
- U7: symbol TPS61175 -> custom:TPS61175
- U?: symbol FE310-G000 -> custom:FE310-G000
- Y1, Y2: symbol CRYSTAL -> custom:CRYSTAL
Connections:
- wire segments 1807 -> 2479
Other:
- moved on the sheet: L1, TP1, TP2, TP3, TP4, TP5, TP6, TP7, TP8, TP9, TP?
