File: flipdot_driver.sch (KiCad schematic (older format))
At the start: 522 parts, among them J1 10x2_1&3_loaded_2.5mm_0.1in_f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, J2 Barrel_Jack, J3 Screw_Terminal_01x04, J4 Conn_01x03_Male, J5 Conn_01x08_Male, J6 Conn_01x03_Male, J7 USB-C_Connector, J8 NP_Conn_01x06_Male, Q1 DMG6602, Q10 DMG6602, Q11 DMG6602, Q12 DMG6602, Q13 DMG6602, Q14 DMG6602, Q15 DMG6602, Q16 DMG6602, Q17 DMG6602, Q18 DMG6602, Q19 DMG6602, Q2 DMG6602, Q20 DMG6602, Q21 2N7002, Q22 2N7002, Q23 2N7002, Q24 2N7002, Q25 2N7002, Q26 2N7002, Q27 2N7002, Q28 2N7002, Q29 2N7002, Q3 DMG6602, Q30 2N7002, Q31 2N7002, Q32 2N7002, Q33 2N7002, Q34 2N7002, Q35 2N7002, Q36 2N7002, Q37 2N7002, Q38 2N7002, Q39 2N7002, Q4 DMG6602, Q40 2N7002, Q41 DMG6602, Q42 DMG6602, Q43 DMG6602, Q44 DMG6602, Q45 DMG6602, Q46 DMG6602, Q47 DMG6602, Q48 DMG6602, Q49 DMG6602, Q5 DMG6602, Q50 DMG6602, Q51 DMG6602, Q52 DMG6602, Q53 DMG6602, Q54 DMG6602, Q55 DMG6602, Q56 DMG6602, Q57 DMG6602, Q58 DMG6602, Q59 DMG6602, Q6 DMG6602, Q60 DMG6602, Q61 2N7002, Q62 2N7002, Q63 2N7002, Q64 2N7002, Q65 2N7002, Q66 2N7002, Q67 2N7002, Q68 2N7002, Q69 2N7002, Q7 DMG6602, Q70 2N7002, Q71 2N7002, Q72 2N7002, Q73 2N7002, Q74 2N7002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

Commit message: continued assigning caps to actual parts
Parts:
- removed C14, C15: 47uF, symbol Device:CP1
- removed C16, C17, C34, C35, C36: 4.7uF, Capacitor_SMD:C_0603_1608Metric, symbol Device:C
- removed C30, C31, C32, C43, C44, C45, C55, C56, C65, C68, C78, C80: 0.1uF, Capacitor_SMD:C_0603_1608Metric, symbol Device:C
- removed C33, C46, C57, C59, C66, C67, C74, C79, C81: 1uF, Capacitor_SMD:C_0603_1608Metric, symbol Device:C
- removed C40, C41, C60, C62, C75, C77: 22uF, Capacitor_SMD:C_0603_1608Metric, symbol Device:C
- removed C42: 4.7nF, Capacitor_SMD:C_0603_1608Metric, symbol Device:C
- removed C50: 15nF, Capacitor_SMD:C_0603_1608Metric, symbol Device:C
- removed C61, C76: 47pF, Capacitor_SMD:C_0603_1608Metric, symbol Device:C
- removed C63, C64, C72, C73: 12pF, Capacitor_SMD:C_0603_1608Metric, symbol Device:C
- added C? (x9): CL10B105KA8NNNC, Capacitor_SMD:C_0603_1608Metric, symbol custom:CL10B105KA8NNNC
- added C? (x12): CL10B104KO8NNNC, Capacitor_SMD:C_0603_1608Metric, symbol custom:CL10B104KO8NNNC
- added C? (x2): EEE-1VA220SP, symbol custom:EEE-1VA220SP
- added C? (x4): CL21A226MOCLRNC, Capacitor_SMD:C_0805_2012Metric, symbol custom:CL21A226MOCLRNC
- added C?: 885012206087, Capacitor_SMD:C_0603_1608Metric, symbol custom:885012206087
- added C? (x2): ‎C0603C470J1GACTU‎, Capacitor_SMD:C_0603_1608Metric, symbol custom:‎C0603C470J1GACTU‎
- added C? (x4): TMK042CG120JD-W‎, Capacitor_SMD:C_01005_0402Metric, symbol custom:TMK042CG120JD-W‎
- added C? (x5): ‎CL21A475KLCLQNC‎, Capacitor_SMD:C_0805_2012Metric, symbol custom:‎CL21A475KLCLQNC‎
- added C?: ‎CL10B153KB8SFNC‎, Capacitor_SMD:C_0603_1608Metric, symbol custom:‎CL10B153KB8SFNC‎
- added C? (x2): ‎ESK476M035AC3AA‎, symbol custom:‎ESK476M035AC3AA‎
- added R?: 4.7k, Resistors_SMD:R_0603_HandSoldering, symbol Device:R
- added R?: NP, Resistors_SMD:R_0603_HandSoldering, symbol Device:R
- added TP?: TEST, symbol Connector:TestPoint
Connections:
- net labels removed: EN_24V
- wire segments 2449 -> 2457
Other:
- moved on the sheet: C13, D33, D34, D35, D40, D41, D42, D43, D44, D45, D46, D51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

Commit message: Swapped discrete TVS with arrays. Swapped LED PWM PMOS (Q89)
Parts:
- removed C54: 33nF, Capacitor_SMD:C_0603_1608Metric, symbol Device:C
- removed D10, D11, D12, D13, D14, D15, D16, D18, D19, D2, D20, D21, D22, D23, D24, D25, D26, D27, D28, D29, D3, D30, D31, D32, D4, D5, D6, D7, D8, D9: MMBZ5243BLT1G, symbol custom:MMBZ5243BLT1G
- removed D36, D37, D38, D39, D40, D41, D42, D43, D44, D45, D46: SMF5.0A, Footprint, symbol custom:SMF5.0A
- removed D59, D60, D61, D62, D63, D64: NP_UCLAMP2501T.TCT, Footprint, symbol custom:UCLAMP2501T.TCT
- removed Q10, Q11, Q12, Q13, Q14, Q15, Q16, Q17, Q18, Q19, Q2, Q20, Q3, Q4, Q41, Q42, Q43, Q44, Q46, Q47, Q48, Q49, Q5, Q50, Q51, Q52, Q53, Q54, Q55, Q56, Q57, Q58, Q59, Q6, Q60, Q7, Q8, Q81, Q82, Q83, Q84, Q9: DMG6602, Package_TO_SOT_SMD:TSOT-23-6, symbol custom:DMG6602
- removed Q21, Q22, Q23, Q24, Q25, Q26, Q27, Q28, Q29, Q30, Q31, Q32, Q33, Q34, Q35, Q36, Q37, Q38, Q39, Q40, Q61, Q62, Q63, Q64, Q65, Q66, Q67, Q68, Q69, Q70, Q71, Q72, Q73, Q74, Q75, Q76, Q77, Q78, Q79, Q80, Q85, Q86, Q87, Q88, Q90, Q91, Q92, Q93, Q94, Q95, Q96, Q97: 2N7002, TO_SOT_Packages_SMD:SOT-23_Handsoldering, symbol Transistor_FET:2N7002
- removed Q89: BUZ11, TO_SOT_Packages_THT:TO-220-3_Horizontal, symbol Transistor_FET:BUZ11
- removed R1, R10, R100, R101, R102, R103, R104, R105, R106, R107, R108, R109, R11, R110, R111, R112, R113, R114, R115, R116, R117, R118, R119, R12, R120, R121, R122, R123, R124, R125, R126, R127, R128, R129, R13, R130, R131, R132, R133, R135, R137, R138, R139, R14, R142, R146, R147, R149, R15, R150, R151, R152, R157, R16, R160, R17, R175, R18, R19, R197, R198, R199, R2, R20, R200, R201, R202, R21, R22, R23, R24, R25, R26, R27, R28, R29, R3, R30, R31, R32, R33, R34, R35, R36, R37, R38, R39, R4, R40, R41, R42, R43, R44, R45, R46, R47, R48, R49, R5, R50, R51, R52, R53, R54, R55, R56, R57, R58, R59, R6, R60, R61, R62, R63, R64, R65, R66, R67, R68, R69, R7, R70, R71, R72, R73, R74, R75, R76, R77, R78, R79, R8, R80, R81, R82, R83, R84, R85, R86, R87, R88, R89, R9, R90, R91, R92, R93, R94, R95, R96, R97, R98, R99, R?: 4.7k, Resistors_SMD:R_0603_HandSoldering, symbol Device:R
- removed R134, R136, R140, R141, R143, R144, R148: NP_4.7k, Resistors_SMD:R_0603_HandSoldering, symbol Device:R
- removed R145: 2k, Resistors_SMD:R_0603_HandSoldering, symbol Device:R
- removed R153, R192, R196: NP_0, Resistors_SMD:R_0603_HandSoldering, symbol Device:R
- removed R155: 4.87k, Resistors_SMD:R_0603_HandSoldering, symbol Device:R
- removed R161, R185, R186, R187, R188, R189, R190: 470, Resistors_SMD:R_0603_HandSoldering, symbol Device:R
- removed R162, R170, R178, R191, R193: 0, Resistors_SMD:R_0603_HandSoldering, symbol Device:R
- removed R164, R166, R177, R183, R184, R194, R195, R?: NP, Resistors_SMD:R_0603_HandSoldering, symbol Device:R
- removed R167, R172, R176, R180: 47k, Resistors_SMD:R_0603_HandSoldering, symbol Device:R
- removed TP1, TP10, TP11, TP12, TP13, TP14, TP15, TP16, TP17, TP18, TP19, TP20, TP21, TP22, TP23, TP24, TP25, TP26, TP27, TP28, TP29, TP3, TP30, TP31, TP32, TP33, TP34, TP36, TP37, TP38, TP39, TP4, TP41, TP5, TP6, TP7, TP8, TP9, TP?: TEST, symbol Connector:TestPoint
- added C?: CL10B333KB8SFNC, Capacitor_SMD:C_0603_1608Metric, symbol custom:CL10B333KB8SFNC
- added Q89, Q? (x2): DMG6602, TSOT-23-6, symbol custom:DMG6602
- added Q90, Q91, Q92, Q93, Q94, Q95, Q96, Q97: SSM3K35AMFV, symbol custom:SSM3K35AMFV
- added R1, R109, R133, R135, R137, R138, R139, R142, R145, R146, R147, R149, R150, R151, R152, R153, R158, R161, R162, R174, R176, R198, R199, R200, R201, R202, R203, R21, R22, R65, R81: CRG0603F4K7, Resistor_SMD:R_0603_1608Metric, symbol custom:CRG0603F4K7
- added R134, R136, R140, R141, R143, R144, R148, R154, R166, R168, R178, R184, R185, R193, R195, R196, R197: NP_R_0603, Resistor_SMD:R_0603_1608Metric, symbol custom:NP_R_0603
- added R156, R164, R179, R192, R194: RC0603JR-070RL, Resistor_SMD:R_0603_1608Metric, symbol custom:RC0603JR-070RL
- added R163, R186, R187, R188, R189, R190, R191: ‎RMCF0603FT470R‎, Resistor_SMD:R_0603_1608Metric, symbol flipdot_driver-rescue:‎RMCF0603FT470R‎-custom
- added R169, R177, R181: RC0603FR-0747KL, Resistor_SMD:R_0603_1608Metric, symbol custom:RC0603FR-0747KL
- added R?: RMCF0603FT470R, Resistor_SMD:R_0603_1608Metric, symbol custom:RMCF0603FT470R
- added TP1, TP10, TP11, TP12, TP13, TP14, TP15, TP16, TP17, TP18, TP19, TP20, TP21, TP22, TP23, TP24, TP25, TP26, TP27, TP28, TP29, TP3, TP30, TP31, TP32, TP33, TP34, TP35, TP36, TP37, TP38, TP4, TP40, TP42, TP5, TP6, TP7, TP8, TP9: TestPoint, symbol custom:TestPoint
- added U20, U22: NP_CM1293A-04SO, symbol custom:CM1293A-04SO
- added U7, U8, U9: CM1293A-04SO, symbol custom:CM1293A-04SO
- C14, C15: renamed from C?; symbol custom:‎ESK476M035AC3AA‎ -> flipdot_driver-rescue:‎ESK476M035AC3AA‎-custom
- C16, C17, C30, C31, C32: renamed from C?; symbol custom:‎CL21A475KLCLQNC‎ -> flipdot_driver-rescue:‎CL21A475KLCLQNC‎-custom
- C50: renamed from C?; symbol custom:‎CL10B153KB8SFNC‎ -> flipdot_driver-rescue:‎CL10B153KB8SFNC‎-custom
- C61, C76: renamed from C?; symbol custom:‎C0603C470J1GACTU‎ -> flipdot_driver-rescue:‎C0603C470J1GACTU‎-custom
- R159: value 4.87k -> 200
- R173: value 4.7k -> 59k
- gave numbers to parts that had none: 32
- renumbered C8 to C1, C26 to C10, C47 to C11, C69 to C12, C10 to C18, C12 to C2, C23 to C20, C27 to C21, C48 to C22, C70 to C23, C11 to C24, C20 to C25, C24 to C26, C28 to C27, C49 to C28, C71 to C29, C21 to C3, C2 to C37, C4 to C38, C7 to C39, C25 to C4, C1 to C47, C3 to C48, C6 to C49, C39 to C5, C29 to C51, C51 to C52, C82 to C53, C5 to C58, C58 to C6, C37 to C67, C52 to C68, C83 to C69, C9 to C7, C18 to C8, C38 to C82, C53 to C83, C22 to C9, D47 to D36, D48 to D37, D49 to D38, D50 to D39, D51 to D40, D52 to D41, D53 to D42, D54 to D43, D55 to D44, D56 to D45, D57 to D46, D58 to D47, R154 to R155, R156 to R157, R158 to R160, R163 to R165, R165 to R167, R168 to R170, R169 to R171, R171 to R172, R174 to R175, R179 to R180, R181 to R182, R182 to R183, TP35 to TP39, TP40 to TP41, U4 to U10, U8 to U11, U9 to U12, U10 to U13, U11 to U14, U12 to U15, U13 to U16, U14 to U17, U15 to U18, U16 to U19, U5 to U2, U17 to U21, U2 to U3, U6 to U4, U3 to U5, U7 to U6
Connections:
- wire segments 2457 -> 1278
- no-connect marks 22 -> 27
Other:
- note added: "0.4 V"
- moved on the sheet: C60, C75, D42, D43, D44, D45, D46, D47, J4, J5, J6, J8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

Commit message: automated commit
Parts:
- removed C63, C64: TMK042CG120JD-W‎, Capacitor_SMD:C_01005_0402Metric, symbol custom:TMK042CG120JD-W‎
- removed C70: CL10B105KA8NNNC, Capacitor_SMD:C_0603_1608Metric, symbol custom:CL10B105KA8NNNC
- removed C71: CL10B104KO8NNNC, Capacitor_SMD:C_0603_1608Metric, symbol custom:CL10B104KO8NNNC
- removed D35, D42, D43, D44, D45, D46, D47: LED, symbol Device:LED
- removed D38, D39: NP_UCLAMP2501T.TCT, Footprint, symbol custom:UCLAMP2501T.TCT
- removed D40: UCLAMP2501T.TCT, Footprint, symbol custom:UCLAMP2501T.TCT
- removed Q? (x2): DMG6602, TSOT-23-6, symbol custom:DMG6602
- removed R154, R166: NP_R_0603, Resistor_SMD:R_0603_1608Metric, symbol custom:NP_R_0603
- removed R158, R162, R176: CRG0603F4K7, Resistor_SMD:R_0603_1608Metric, symbol custom:CRG0603F4K7
- removed R164: RC0603JR-070RL, Resistor_SMD:R_0603_1608Metric, symbol custom:RC0603JR-070RL
- removed R?: RMCF0603FT470R, Resistor_SMD:R_0603_1608Metric, symbol custom:RMCF0603FT470R
- removed SW1: NP_TACTILE_SWITCH, CUSTOM:TACTILE_SWITCH, symbol custom:TACTILE_SWITCH
- removed SW2: TACTILE_SWITCH, CUSTOM:TACTILE_SWITCH, symbol custom:TACTILE_SWITCH
- removed U13: FE310-G000, symbol custom:FE310-G000
- removed U17: IS25LP128-JBLE, Housings_SOIC:SOIC-8_3.9x4.9mm_Pitch1.27mm, symbol custom:IS25LP128-JBLE
- removed Y1: 16MHz, symbol custom:CRYSTAL
- removed Y2: 6MHz, symbol custom:CRYSTAL
- added D? (x8): LED_GENERIC_0805, Diode_SMD:D_0805_2012Metric, symbol custom:LED_GENERIC_0805
- added Q? (x29): SSM3K35AMFV, symbol custom:SSM3K35AMFV
- added Q? (x24): DMG6602, Package_TO_SOT_SMD:TSOT-23-6, symbol custom:DMG6602
- added R? (x51): CRG0603F4K7, Resistor_SMD:R_0603_1608Metric, symbol custom:CRG0603F4K7
- added R?: ‎RMCF0603FT470R‎, Resistor_SMD:R_0603_1608Metric, symbol flipdot_driver-rescue:‎RMCF0603FT470R‎-custom
- added Y?: NX8045GB-6MHZ-STD-CSF-3, symbol custom:NX8045GB-6MHZ-STD-CSF-3
- TP1, TP10, TP11, TP12, TP13, TP14, TP15, TP16, TP17, TP18, TP19, TP20, TP21, TP22, TP23, TP24, TP25, TP26, TP27, TP28, TP29, TP3, TP30, TP31, TP32, TP33, TP34, TP35, TP36, TP37, TP38, TP4, TP40, TP42, TP5, TP6, TP7, TP8, TP9: symbol custom:TestPoint -> Connector:TestPoint
- U20, U22, U7, U8, U9: symbol custom:CM1293A-04SO -> custom:CM1293A-04SO_ALTERNATE_SYMBOL
Connections:
- net +12V: now also Q?.2 (S), Q?.2 (S), Q?.2 (S), Q?.2 (S), Q?.2 (S), Q?.2 (S), Q?.2 (S), Q?.2 (S), Q?.2 (S), Q?.2 (S), Q?.2 (S), Q?.2 (S), R?.1, R?.1, R?.1, R?.1, R?.1, R?.1, R?.1, R?.1, R?.1, R?.1, R?.1, R?.1
- net +3V3: now also R?.1
- net COL00: now also Q?.4 (D), Q?.4 (D), Q?.4 (D), Q?.4 (D), Q?.4 (D), Q?.4 (D), Q?.4 (D), Q?.4 (D), Q?.4 (D), Q?.4 (D), Q?.4 (D), Q?.4 (D), Q?.6 (D), Q?.6 (D), Q?.6 (D), Q?.6 (D), Q?.6 (D), Q?.6 (D), Q?.6 (D), Q?.6 (D), Q?.6 (D), Q?.6 (D), Q?.6 (D), Q?.6 (D)
- net COL00_OFF: now also R?.1, R?.1, R?.1, R?.1, R?.1, R?.1, R?.1, R?.1, R?.1, R?.1, R?.1, R?.1, R?.2, R?.2, R?.2, R?.2, R?.2, R?.2, R?.2, R?.2, R?.2, R?.2, R?.2, R?.2, R?.2; no longer Q1.1 (G)
- net COL00_ON: now also Q?.1 (G), Q?.1 (G), Q?.1 (G), Q?.1 (G), Q?.1 (G), Q?.1 (G), Q?.1 (G), Q?.1 (G), Q?.1 (G), Q?.1 (G), Q?.1 (G), Q?.1 (G), Q?.1 (G), Q?.1 (G), Q?.1 (G), Q?.1 (G), Q?.1 (G), Q?.1 (G), Q?.1 (G), Q?.1 (G), Q?.1 (G), Q?.1 (G), Q?.1 (G), Q?.1 (G), Q?.1 (G), Q?.1 (G), R?.1, R?.1, R?.1, R?.1, R?.1, R?.1, R?.1, R?.1, R?.1, R?.1, R?.1, R?.1
- net GND: now also D?.1 (K), Q?.2 (S), Q?.2 (S), Q?.2 (S), Q?.2 (S), Q?.2 (S), Q?.2 (S), Q?.2 (S), Q?.2 (S), Q?.2 (S), Q?.2 (S), Q?.2 (S), Q?.2 (S), Q?.2 (S), Q?.2 (S), Q?.2 (S), Q?.2 (S), Q?.2 (S), Q?.2 (S), Q?.2 (S), Q?.2 (S), Q?.2 (S), Q?.2 (S), Q?.2 (S), Q?.2 (S), Q?.2 (S), Q?.2 (S), Q?.2 (S), Q?.2 (S), Q?.2 (S), Q?.5 (S), Q?.5 (S), Q?.5 (S), Q?.5 (S), Q?.5 (S), Q?.5 (S), Q?.5 (S), Q?.5 (S), Q?.5 (S), Q?.5 (S), Q?.5 (S), Q?.5 (S), R?.2, R?.2, R?.2, R?.2, R?.2, R?.2, R?.2, R?.2, R?.2, R?.2, R?.2, R?.2, R?.2, R?.2, R?.2, R?.2, R?.2, R?.2, R?.2, R?.2, R?.2, R?.2, R?.2, R?.2, R?.2
- net ROW00_OFF: now also R?.2; no longer Q45.1 (G)
- net ROW00_ON: now also Q?.1 (G), Q?.1 (G)
- net at C72.1, U16.43 (XTIN): now also Y?.1
- net at C73.1, U16.44 (XTOUT): now also Y?.2
- net at Q1.3 (G), R1.2: now also Q?.3 (D)
- net at Q97.3 (D): now also D?.1 (K)
- net at R191.2: now also D?.2 (A)
- net at Q96.3 (D): now also D?.1 (K)
- net at R190.2: now also D?.2 (A)
- net at Q95.3 (D): now also D?.1 (K)
- net at R189.2: now also D?.2 (A)
- net at Q94.3 (D): now also D?.1 (K)
- net at R188.2: now also D?.2 (A)
- net at Q93.3 (D): now also D?.1 (K)
- net at R187.2: now also D?.2 (A)
- net at Q92.3 (D): now also D?.1 (K)
- net at R186.2: now also D?.2 (A)
- net at Q45.3 (G), R65.2: now also Q?.3 (D)
- net at R145.2: now also D?.2 (A)
- net TCK renamed JTAG_TCK
- net TDI renamed JTAG_TDI
- net TDO renamed JTAG_TDO
- net TMS renamed JTAG_TMS
- new net: Q1.1 (G), Q?.3 (D), R?.1
- new net: Q45.1 (G), Q?.3 (D), R?.1
- new net: D?.1 (K), Q?.3 (D)
- new net: D?.2 (A), R?.2
- new net: Q?.1 (G), Q?.3 (D), R?.1 (x12)
- new net: Q?.3 (D), Q?.3 (G), R?.2 (x12)
- new net AUX_6: Q?.1 (G), R?.1
- no-connect marks 27 -> 23
Other:
- note added: "TVS DIODES ALLOW THE ROW TRANSISTORS TO BE SHUT OFF\nBEFORE THE COLUMN TRANSISTOR. WITHOUT IT, SHUTTING OFF\nTHE ROW TRANSISTOR MAY CAUSE AN INDUCTIVE SPIKEACROSS\nTHE RESISTOR, BLOWING OUT ITS BODY DIODE."
- note removed: "FE310"
- note removed: "SILKSCREEN:\nRESET"
- note removed: "SILKSCREEN:\nWAKEUP"
- moved on the sheet: D1, D17, Q1A, Q1B, Q45A, Q45B, Q92, Q93, Q94, Q95, Q96, Q97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

Commit message: automated commit
Parts:
- removed C1, C10, C18, C21, C24, C27, C33, C34, C35, C37, C38, C4, C43, C44, C45, C47, C48, C51, C55, C56, C58, C65, C67, C7, C78, C80, C82: CL10B104KO8NNNC, Capacitor_SMD:C_0603_1608Metric, symbol custom:CL10B104KO8NNNC
- removed C11, C19, C2, C22, C25, C28, C36, C46, C5, C52, C57, C59, C66, C68, C74, C79, C8, C81, C83: CL10B105KA8NNNC, Capacitor_SMD:C_0603_1608Metric, symbol custom:CL10B105KA8NNNC
- removed C12, C20, C23, C26, C29, C3, C39, C49, C53, C6, C69, C84, C9: NP_C_0603, Capacitor_SMD:C_0603_1608Metric, symbol custom:NP_C_0603
- removed C13: NP_470uF, symbol Device:CP1
- removed C14, C15: ‎ESK476M035AC3AA‎, symbol flipdot_driver-rescue:‎ESK476M035AC3AA‎-custom
- removed C16, C17, C30, C31, C32: ‎CL21A475KLCLQNC‎, Capacitor_SMD:C_0805_2012Metric, symbol flipdot_driver-rescue:‎CL21A475KLCLQNC‎-custom
- removed C40, C41: EEE-1VA220SP, symbol custom:EEE-1VA220SP
- removed C42: 885012206087, Capacitor_SMD:C_0603_1608Metric, symbol custom:885012206087
- removed C50: ‎CL10B153KB8SFNC‎, Capacitor_SMD:C_0603_1608Metric, symbol flipdot_driver-rescue:‎CL10B153KB8SFNC‎-custom
- removed C60, C62, C75, C77: CL21A226MOCLRNC, Capacitor_SMD:C_0805_2012Metric, symbol custom:CL21A226MOCLRNC
- removed C61, C76: ‎C0603C470J1GACTU‎, Capacitor_SMD:C_0603_1608Metric, symbol flipdot_driver-rescue:‎C0603C470J1GACTU‎-custom
- removed C72, C73: TMK042CG120JD-W‎, Capacitor_SMD:C_01005_0402Metric, symbol custom:TMK042CG120JD-W‎
- removed C?: CL10B333KB8SFNC, Capacitor_SMD:C_0603_1608Metric, symbol custom:CL10B333KB8SFNC
- removed D1, D17: MMBZ5243BLT1G, symbol custom:MMBZ5243BLT1G
- removed D33, D36: DST2080S, symbol custom:DST2080S
- removed D34: SMAJ12A, Footprint, symbol custom:SMAJ12A
- removed D37: SMF5.0A, Footprint, symbol custom:SMF5.0A
- removed D41: RSB6.8F2T106, symbol custom:RSB6.8F2T106
- removed D? (x8): LED_GENERIC_0805, Diode_SMD:D_0805_2012Metric, symbol custom:LED_GENERIC_0805
- removed J1: 10x2_1&3_loaded_2.5mm_0.1in_female_header, symbol custom:10x2_1&3_loaded_2.5mm_0.1in_female_header
- removed J2: Barrel_Jack, Connectors:BARREL_JACK, symbol Connector:Barrel_Jack_Switch
- removed J3: Screw_Terminal_01x04, symbol Connector:Screw_Terminal_01x04
- removed J4, J6: Conn_01x03_Male, symbol Connector:Conn_01x03_Male
- removed J5: Conn_01x08_Male, symbol Connector:Conn_01x08_Male
- removed J7: USB-C_Connector, symbol custom:USB-C_Connector
- removed J8: NP_Conn_01x06_Male, symbol Connector:Conn_01x06_Male
- removed L1, L3: FBMH4532HM681-T, symbol custom:FBMH4532HM681-T
- removed L2: 12uH, symbol Device:L
- removed L4: 6.5uH, symbol Device:L
- removed L5: 3.3uH, symbol Device:L
- removed Q1, Q45, Q? (x24): DMG6602, Package_TO_SOT_SMD:TSOT-23-6, symbol custom:DMG6602
- removed Q89: DMG6602, TSOT-23-6, symbol custom:DMG6602
- removed Q90, Q91, Q92, Q93, Q94, Q95, Q96, Q97, Q? (x29): SSM3K35AMFV, symbol custom:SSM3K35AMFV
- removed R1, R109, R133, R135, R137, R138, R139, R142, R145, R146, R147, R149, R150, R151, R152, R153, R161, R174, R198, R199, R200, R201, R202, R203, R21, R22, R65, R81, R? (x51): CRG0603F4K7, Resistor_SMD:R_0603_1608Metric, symbol custom:CRG0603F4K7
- removed R134, R136, R140, R141, R143, R144, R148, R168, R178, R184, R185, R193, R195, R196, R197: NP_R_0603, Resistor_SMD:R_0603_1608Metric, symbol custom:NP_R_0603
- removed R155: 300k, Resistors_SMD:R_0603_HandSoldering, symbol Device:R
- removed R156, R179, R192, R194: RC0603JR-070RL, Resistor_SMD:R_0603_1608Metric, symbol custom:RC0603JR-070RL
- removed R157: 16.2k, Resistors_SMD:R_0603_HandSoldering, symbol Device:R
- removed R159: 200, Resistors_SMD:R_0603_HandSoldering, symbol Device:R
- removed R160: 143k, Resistors_SMD:R_0603_HandSoldering, symbol Device:R
- removed R163, R186, R187, R188, R189, R190, R191, R?: ‎RMCF0603FT470R‎, Resistor_SMD:R_0603_1608Metric, symbol flipdot_driver-rescue:‎RMCF0603FT470R‎-custom
- removed R165, R167: 47, Resistors_SMD:R_0603_HandSoldering, symbol Device:R
- removed R169, R177, R181: RC0603FR-0747KL, Resistor_SMD:R_0603_1608Metric, symbol custom:RC0603FR-0747KL
- removed R170, R180: 40.2k, Resistors_SMD:R_0603_HandSoldering, symbol Device:R
- removed R171: 1.5k, Resistors_SMD:R_0603_HandSoldering, symbol Device:R
- removed R172, R175: 13k, Resistors_SMD:R_0603_HandSoldering, symbol Device:R
- removed R173: 59k, Resistors_SMD:R_0603_HandSoldering, symbol Device:R
- removed R182: 100k, Resistors_SMD:R_0603_HandSoldering, symbol Device:R
- removed R183: 32.4k, Resistors_SMD:R_0603_HandSoldering, symbol Device:R
- removed TP1, TP10, TP11, TP12, TP13, TP14, TP15, TP16, TP17, TP18, TP19, TP20, TP21, TP22, TP23, TP24, TP25, TP26, TP27, TP28, TP29, TP3, TP30, TP31, TP32, TP33, TP34, TP35, TP36, TP37, TP38, TP4, TP40, TP42, TP5, TP6, TP7, TP8, TP9: TestPoint, symbol Connector:TestPoint
- removed TP2, TP39, TP41: TEST, symbol Connector:TestPoint
- removed U1, U10, U11, U14, U19, U2, U21, U3, U4, U5, U6: 74HC595, symbol custom:74HC595
- removed U12: TPS61175, symbol custom:TPS61175
- removed U15, U18: AP65111A, symbol custom:AP65111A
- removed U16: FT2232D, Housings_QFP:LQFP-48_7x7mm_Pitch0.5mm, symbol custom:FT2232D
- removed U20, U22: NP_CM1293A-04SO, symbol custom:CM1293A-04SO_ALTERNATE_SYMBOL
- removed U7, U8, U9: CM1293A-04SO, symbol custom:CM1293A-04SO_ALTERNATE_SYMBOL
- removed Y?: NX8045GB-6MHZ-STD-CSF-3, symbol custom:NX8045GB-6MHZ-STD-CSF-3
Connections:
- no-connect marks 23 -> 0
Other:
- note removed: "0.4 V"
- note removed: "AUX IO"
- note removed: "AVOID STUBS"
- note removed: "CLOCK INVERSION"
- note removed: "DOT DRIVERS"
- note removed: "FE310 BYPASS"
- note removed: "FLIPDOT BOARD INTERFACE"
- note removed: "FT2232D BYPASS"
- note removed: "INCLUDE FILLED RECTANGLES\nON SILKSCREEN NEAR EACH\nLED TO WRITE LABELS ON"
- note removed: "LABEL POSITIVE AND\nNEGATIVE TERMINALS\nON SILKSCREEN"
- note removed: "PANEL EXTENSION"
- note removed: "PLACE CLOSE TO CONNECTOR"
- note removed: "POWER INPUT"
- note removed: "POWER RAIL GENERATION"
- note removed: "PUT SYMBOL FOR CENTER-POSITIVE\nCONNECTOR, VOLTAGE RANGE, AND\nBARREL JACK DIMENSIONS FOR MATE\nON SILKSCREEN"
- note removed: "ROW_SHCP AND COL_SHCP\nARE PULLED DOWN IN THE\nCLOCK INVERSION SECTION"
- note removed: "SHIFT REGISTERS"
- note removed: "SILKSCREEN: POPULATE TVS DIODES\nAS APPROPRIATE FOR USE\nWITH GPIO PERIPHERALS"
- note removed: "SILKSCREEN:\n12V (12.9V MAX)"
- note removed: "SPACE 1x3 HEADERS SO\nAS TO PREVENT A JUMPER\nFROM CONNECTING AN\nINVALID SET OF PINS"
- note removed: "STRAPPING"
- note removed: "TVS DIODES ALLOW THE ROW TRANSISTORS TO BE SHUT OFF\nBEFORE THE COLUMN TRANSISTOR. WITHOUT IT, SHUTTING OFF\nTHE ROW TRANSISTOR MAY CAUSE AN INDUCTIVE SPIKEACROSS\nTHE RESISTOR, BLOWING OUT ITS BODY DIODE."
- note removed: "UART CYA"
- note removed: "USB TO SERIAL"

Commit message: automated commit
Changed lines of the file:
@@
 $Descr A4 11693 8268
 encoding utf-8
-Sheet 1 19
+Sheet 1 20
 Title ""
 Date ""
@@
 S 3600 3200 1300 700
 U 627E3ADC
-F0 "MISC" 50
-F1 "MISC.sch" 50
+F0 "INTERFACE" 50
+F1 "INTERFACE.sch" 50
 $EndSheet
 $Sheet
@@
 F1 "ROW_DRIVERS_3.sch" 50
 $EndSheet
+$Sheet
+S 5000 3200 1300 700
+U 5D4A63FF
+F0 "SHIFT_REGISTER_SIGNALS" 50
+F1 "SHIFT_REGISTER_SIGNALS.sch" 50
+$EndSheet
 $EndSCHEMATC
