File: AUXILIARY_IO.sch (KiCad schematic (older format))
At the start: 38 parts

Commit message: automated commit
Connections:
- wire segments 105 -> 119
Other:
- moved on the sheet: D?, J?, Q?, R?, TP?, U?

Commit message: automated commit
Parts:
- removed R? (x7): ‎RMCF0603FT470R‎, Resistor_SMD:R_0603_1608Metric, symbol flipdot_driver-rescue:‎RMCF0603FT470R‎-custom
- added R49, R50, R51, R52, R53, R54, R55: ‎RMCF0603FT470R‎, Resistor_SMD:R_0603_1608Metric, symbol custom:‎RMCF0603FT470R‎
- gave numbers to parts that had none: 31
