File: AUXILIARY_IO.sch (KiCad schematic (older format))
At the start: 38 parts, among them J4 NP_Conn_01x07_Male, Q10 SSM3K35AMFV, Q4 SSM3K35AMFV, Q5 SSM3K35AMFV, Q6 SSM3K35AMFV, Q7 SSM3K35AMFV, Q8 SSM3K35AMFV, Q9 SSM3K35AMFV, U7 NP_CM1293A-04SO, U8 NP_CM1293A-04SO

Commit message: automated commit
Parts:
- removed D14, D15, D16, D17, D18, D19: LED_GENERIC_0805, Diode_SMD:D_0805_2012Metric, symbol custom:LED_GENERIC_0805
- removed Q10, Q5, Q6, Q7, Q8, Q9: SSM3K35AMFV, symbol custom:SSM3K35AMFV
- removed R50, R51, R52, R53, R54, R55: ‎RMCF0603FT470R‎, Resistor_SMD:R_0603_1608Metric, symbol custom:‎RMCF0603FT470R‎
- removed R57, R58, R59, R60, R61, R62: CRG0603F4K7, Resistor_SMD:R_0603_1608Metric, symbol custom:CRG0603F4K7
- added D? (x6): LED_GENERIC_0805, Diode_SMD:D_0805_2012Metric, symbol custom:LED_GENERIC_0805
- added Q? (x6): SSM3K35AMFV, symbol custom:SSM3K35AMFV
- added R? (x7): NP_R_0603, 0603, symbol custom:NP_R_0603
- added R? (x6): CRG0603F4K7, Resistor_SMD:R_0603_1608Metric, symbol custom:CRG0603F4K7
- added R? (x6): ‎RMCF0603FT470R‎, Resistor_SMD:R_0603_1608Metric, symbol custom:‎RMCF0603FT470R‎
Connections:
- wire segments 119 -> 141
Other:
- moved on the sheet: D13, Q4, R49, R56, TP17, TP18, TP19, TP20, TP21, TP22, TP23, U7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

Commit message: automated commit
Parts:
- removed D? (x2): LED_GENERIC_0805, Diode_SMD:D_0805_2012Metric, symbol custom:LED_GENERIC_0805
- removed J4: NP_Conn_01x07_Male, symbol Connector:Conn_01x07_Male
- removed Q? (x2): SSM3K35AMFV, symbol custom:SSM3K35AMFV
- removed R? (x2): CRG0603F4K7, Resistor_SMD:R_0603_1608Metric, symbol custom:CRG0603F4K7
- removed R? (x2): ‎RMCF0603FT470R‎, Resistor_SMD:R_0603_1608Metric, symbol custom:‎RMCF0603FT470R‎
- removed R? (x2): NP_R_0603, 0603, symbol custom:NP_R_0603
- removed TP22, TP23: TestPoint, symbol Connector:TestPoint
- added J3: Conn_01x05_Male, symbol Connector:Conn_01x05_Male
- gave numbers to parts that had none: 21
- renumbered D13 to D11, R49 to R35, R56 to R40, TP17 to TP13, TP18 to TP14, TP19 to TP15, TP20 to TP16, TP21 to TP17, U7 to U6, U8 to U7
Connections:
- net labels removed: AUX_5, AUX_6
- wire segments 141 -> 103
- no-connect marks 1 -> 3
Other:
- moved on the sheet: D11, D12, D13, D14, D15, Q4, Q5, Q6, Q7, Q8, R35, R36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

Commit message: automated commit
Parts:
- R40, R46, R47, R48, R49: Resistance 4.7k -> (none); TOLERANCE (none) -> 5%; VALUE (none) -> 4k7
Changed lines of the file:
@@
-	1    0    0    -1
-$EndComp
-$Comp
-L custom:CRG0603F4K7 R?
-U 1 1 61EC1140
-P 2750 1950
-AR Path="/61EC1140" Ref="R?"  Part="1"
-AR Path="/61C6D021/61EC1140" Ref="R40"  Part="1"
-F 0 "R40" V 2870 1850 50  0000 L BNN
-F 1 "CRG0603F4K7" H 2000 1500 50  0001 L BNN
-F 2 "Resistor_SMD:R_0603_1608Metric" H 2000 1400 50  0001 L BNN
-F 3 "datasheets/PYu-RC_Group_51_RoHS_L_9.pdf" H 2000 1300 50  0001 L BNN
-F 4 "4.7k" V 2770 1890 39  0000 L BNN "Resistance"
-	1    2750 1950
 	1    0    0    -1
 $EndComp
@@
 $EndComp
 $Comp
-L custom:CRG0603F4K7 R?
-U 1 1 5D063603
-P 3950 2625
-AR Path="/5D063603" Ref="R?"  Part="1"
-AR Path="/61C6D021/5D063603" Ref="R46"  Part="1"
-F 0 "R46" V 4070 2525 50  0000 L BNN
-F 1 "CRG0603F4K7" H 3200 2175 50  0001 L BNN
-F 2 "Resistor_SMD:R_0603_1608Metric" H 3200 2075 50  0001 L BNN
-F 3 "datasheets/PYu-RC_Group_51_RoHS_L_9.pdf" H 3200 1975 50  0001 L BNN
-F 4 "4.7k" V 3970 2565 39  0000 L BNN "Resistance"
-	1    3950 2625
-	1    0    0    -1
-$EndComp
-$Comp
 L custom:LED_GENERIC_0805 D?
 U 1 1 5D063609
@@
 $EndComp
 $Comp
-L custom:CRG0603F4K7 R?
-U 1 1 5D07707B
-P 5150 2625
-AR Path="/5D07707B" Ref="R?"  Part="1"
-AR Path="/61C6D021/5D07707B" Ref="R47"  Part="1"
-F 0 "R47" V 5270 2525 50  0000 L BNN
-F 1 "CRG0603F4K7" H 4400 2175 50  0001 L BNN
-F 2 "Resistor_SMD:R_0603_1608Metric" H 4400 2075 50  0001 L BNN
-F 3 "datasheets/PYu-RC_Group_51_RoHS_L_9.pdf" H 4400 1975 50  0001 L BNN
-F 4 "4.7k" V 5170 2565 39  0000 L BNN "Resistance"
-	1    5150 2625
-	1    0    0    -1
-$EndComp
-$Comp
 L custom:LED_GENERIC_0805 D?
 U 1 1 5D077081
@@
 $EndComp
 $Comp
-L custom:CRG0603F4K7 R?
-U 1 1 5D0770BD
-P 6350 2625
-AR Path="/5D0770BD" Ref="R?"  Part="1"
-AR Path="/61C6D021/5D0770BD" Ref="R48"  Part="1"
-F 0 "R48" V 6470 2525 50  0000 L BNN
-F 1 "CRG0603F4K7" H 5600 2175 50  0001 L BNN
-F 2 "Resistor_SMD:R_0603_1608Metric" H 5600 2075 50  0001 L BNN
-F 3 "datasheets/PYu-RC_Group_51_RoHS_L_9.pdf" H 5600 1975 50  0001 L BNN
-F 4 "4.7k" V 6370 2565 39  0000 L BNN "Resistance"
-	1    6350 2625
-	1    0    0    -1
-$EndComp
-$Comp
 L custom:LED_GENERIC_0805 D?
 U 1 1 5D0770C3
@@
 $EndComp
 $Comp
-L custom:CRG0603F4K7 R?
-U 1 1 5D07F690
-P 7550 2625
-AR Path="/5D07F690" Ref="R?"  Part="1"
-AR Path="/61C6D021/5D07F690" Ref="R49"  Part="1"
-F 0 "R49" V 7670 2525 50  0000 L BNN
-F 1 "CRG0603F4K7" H 6800 2175 50  0001 L BNN
-F 2 "Resistor_SMD:R_0603_1608Metric" H 6800 2075 50  0001 L BNN
-F 3 "datasheets/PYu-RC_Group_51_RoHS_L_9.pdf" H 6800 1975 50  0001 L BNN
-F 4 "4.7k" V 7570 2565 39  0000 L BNN "Resistance"
-	1    7550 2625
-	1    0    0    -1
-$EndComp
-$Comp
 L custom:LED_GENERIC_0805 D?
 U 1 1 5D07F696
@@
 	-1   0    0    -1
 $EndComp
+$Comp
+L custom:CRG0603F4K7 R46
+U 1 1 5D0124E3
+P 3950 2625
+F 0 "R46" H 4020 2645 50  0000 L BNN
+F 1 "CRG0603F4K7" H 3250 2225 50  0001 L BNN
+F 2 "Resistor_SMD:R_0603_1608Metric" H 3250 2125 50  0001 L BNN
+F 3 "/home/dj/datasheets/Pyu-RC_Group_51_RoHS_L_9.pdf" H 3250 2025 50  0001 L BNN
+F 4 "4k7" V 3950 2625 50  0000 C CNN "VALUE"
+F 5 "5%" H 4070 2585 50  0000 C CNN "TOLERANCE"
+	1    3950 2625
+	1    0    0    -1
+$EndComp
+$Comp
+L custom:CRG0603F4K7 R47
+U 1 1 5D012934
+P 5150 2625
+F 0 "R47" H 5220 2645 50  0000 L BNN
+F 1 "CRG0603F4K7" H 4450 2225 50  0001 L BNN
+F 2 "Resistor_SMD:R_0603_1608Metric" H 4450 2125 50  0001 L BNN
+F 3 "/home/dj/datasheets/Pyu-RC_Group_51_RoHS_L_9.pdf" H 4450 2025 50  0001 L BNN
+F 4 "4k7" V 5150 2625 50  0000 C CNN "VALUE"
+F 5 "5%" H 5270 2585 50  0000 C CNN "TOLERANCE"
+	1    5150 2625
+	1    0    0    -1
+$EndComp
+$Comp
+L custom:CRG0603F4K7 R48
+U 1 1 5D012E81
+P 6350 2625
+F 0 "R48" H 6420 2645 50  0000 L BNN
+F 1 "CRG0603F4K7" H 5650 2225 50  0001 L BNN
+F 2 "Resistor_SMD:R_0603_1608Metric" H 5650 2125 50  0001 L BNN
+F 3 "/home/dj/datasheets/Pyu-RC_Group_51_RoHS_L_9.pdf" H 5650 2025 50  0001 L BNN
+F 4 "4k7" V 6350 2625 50  0000 C CNN "VALUE"
+F 5 "5%" H 6470 2585 50  0000 C CNN "TOLERANCE"
+	1    6350 2625
+	1    0    0    -1
+$EndComp
+$Comp
+L custom:CRG0603F4K7 R49
+U 1 1 5D0133BA
+P 7550 2625
+F 0 "R49" H 7620 2645 50  0000 L BNN
+F 1 "CRG0603F4K7" H 6850 2225 50  0001 L BNN
+F 2 "Resistor_SMD:R_0603_1608Metric" H 6850 2125 50  0001 L BNN
+F 3 "/home/dj/datasheets/Pyu-RC_Group_51_RoHS_L_9.pdf" H 6850 2025 50  0001 L BNN
+F 4 "4k7" V 7550 2625 50  0000 C CNN "VALUE"
+F 5 "5%" H 7670 2585 50  0000 C CNN "TOLERANCE"
+	1    7550 2625
+	1    0    0    -1
+$EndComp
+$Comp
+L custom:CRG0603F4K7 R40
+U 1 1 5D0137B5
+P 2750 1950
+F 0 "R40" H 2525 1975 50  0000 L BNN
+F 1 "CRG0603F4K7" H 2050 1550 50  0001 L BNN
+F 2 "Resistor_SMD:R_0603_1608Metric" H 2050 1450 50  0001 L BNN
+F 3 "/home/dj/datasheets/Pyu-RC_Group_51_RoHS_L_9.pdf" H 2050 1350 50  0001 L BNN
+F 4 "4k7" V 2750 1950 50  0000 C CNN "VALUE"
+F 5 "5%" H 2575 1925 50  0000 C CNN "TOLERANCE"
+	1    2750 1950
+	1    0    0    -1
+$EndComp
 $EndSCHEMATC

Commit message: automated commit
Parts:
- removed D11: LED_GENERIC_0805, Diode_SMD:D_0805_2012Metric, symbol custom:LED_GENERIC_0805
- removed Q4: SSM3K35AMFV, symbol custom:SSM3K35AMFV
- removed R35: ‎RMCF0603FT470R‎, Resistor_SMD:R_0603_1608Metric, symbol custom:‎RMCF0603FT470R‎
- removed R40, R46, R47, R48: CRG0603F4K7, Resistor_SMD:R_0603_1608Metric, symbol custom:CRG0603F4K7
- removed R41, R42, R43, R44, R45: NP_R_0603, 0603, symbol custom:NP_R_0603
- removed TP13, TP14, TP15, TP16, TP17: TestPoint, symbol Connector:TestPoint
- added D15: LED_GENERIC_0805, Diode_SMD:D_0805_2012Metric, symbol custom:LED_GENERIC_0805
- added J3, J4, J5, J6, J8: PTH_1.5_mm, TestPoint:TestPoint_THTPad_D3.0mm_Drill1.5mm, symbol custom:PTH_1.5_mm
- added Q8: SSM3K35AMFV, symbol custom:SSM3K35AMFV
- added R39: ‎RMCF0603FT470R‎, Resistor_SMD:R_0603_1608Metric, symbol custom:‎RMCF0603FT470R‎
- added R41, R42, R43, R44: CRG0603F4K7, Resistor_SMD:R_0603_1608Metric, symbol custom:CRG0603F4K7
- added SW3, SW4, SW5, SW6, SW7: NP_TACTILE_SWITCH, CUSTOM:TACTILE_SWITCH, symbol custom:TACTILE_SWITCH
- renumbered D15 to D11, J3 to J7, Q8 to Q4, R39 to R35, R49 to R40
Connections:
- net +3V3: now also U7.3 (CH2), U7.4 (CH3), U7.6 (CH4), R39.1, SW3.2, SW4.2, SW5.2, SW6.2, SW7.2
- net AUX_0: now also Q4.1 (G), R40.1, J3.1, SW3.1
- net AUX_1: now also J4.1, R41.1, SW4.1
- net AUX_2: now also J5.1, R42.1, SW5.1
- net AUX_3: now also J6.1, R43.1, SW6.1
- net AUX_4: now also J8.1, Q8.1 (G), R44.1, SW7.1; no longer Q4.1 (G), R40.1
- net GND: now also Q8.2 (S), R41.2, R42.2, R43.2, R44.2
- new net: D15.2 (A), R39.2
- new net: D15.1 (K), Q8.3 (D)
- no-connect marks 3 -> 0
Other:
- note added: "LABEL PINS ON SILKSCREEN"
- note added: "ROUTE 3V3 *THROUGH* FOR ALL BUTTONS"
- note removed: "AVOID STUBS"
- note removed: "PLACE CLOSE TO CONNECTOR"
- moved on the sheet: D11, Q4, R35, R40, U6, U7

Commit message: automated commit
Parts:
- J7: footprint (none) -> Connector_PinHeader_2.54mm:PinHeader_1x05_P2.54mm_Vertical
- Q4, Q5, Q6, Q7, Q8: footprint (none) -> Package_TO_SOT_SMD:SOT-723
Changed lines of the file:
@@
 F 0 "J7" H 7500 5375 50  0000 C CNN
 F 1 "Conn_01x05_Male" H 7500 4775 50  0000 C CNN
-F 2 "" H 7500 5075 50  0001 C CNN
+F 2 "Connector_PinHeader_2.54mm:PinHeader_1x05_P2.54mm_Vertical" H 7500 5075 50  0001 C CNN
 F 3 "~" H 7500 5075 50  0001 C CNN
 	1    7500 5075
@@
 F 0 "Q4" V 3175 2200 50  0000 L BNN
 F 1 "SSM3K35AMFV" V 3100 2025 50  0000 L BNN
-F 2 "" H 3050 2150 50  0001 L BIN
+F 2 "Package_TO_SOT_SMD:SOT-723" H 3050 2150 50  0001 L BIN
 F 3 "datasheets/SSM3K35AMFV.pdf" H 3050 2125 50  0001 L BNN
 	1    2850 2275
@@
 F 0 "Q5" V 4450 2200 50  0000 L BNN
 F 1 "SSM3K35AMFV" V 4375 2025 50  0000 L BNN
-F 2 "" H 4325 2150 50  0001 L BIN
+F 2 "Package_TO_SOT_SMD:SOT-723" H 4325 2150 50  0001 L BIN
 F 3 "datasheets/SSM3K35AMFV.pdf" H 4325 2125 50  0001 L BNN
 	1    4125 2275
@@
 F 0 "Q6" V 5725 2200 50  0000 L BNN
 F 1 "SSM3K35AMFV" V 5650 2025 50  0000 L BNN
-F 2 "" H 5600 2150 50  0001 L BIN
+F 2 "Package_TO_SOT_SMD:SOT-723" H 5600 2150 50  0001 L BIN
 F 3 "datasheets/SSM3K35AMFV.pdf" H 5600 2125 50  0001 L BNN
 	1    5400 2275
@@
 F 0 "Q7" V 7000 2200 50  0000 L BNN
 F 1 "SSM3K35AMFV" V 6925 2025 50  0000 L BNN
-F 2 "" H 6875 2150 50  0001 L BIN
+F 2 "Package_TO_SOT_SMD:SOT-723" H 6875 2150 50  0001 L BIN
 F 3 "datasheets/SSM3K35AMFV.pdf" H 6875 2125 50  0001 L BNN
 	1    6675 2275
@@
 F 0 "Q8" V 8275 2200 50  0000 L BNN
 F 1 "SSM3K35AMFV" V 8200 2025 50  0000 L BNN
-F 2 "" H 8150 2150 50  0001 L BIN
+F 2 "Package_TO_SOT_SMD:SOT-723" H 8150 2150 50  0001 L BIN
 F 3 "datasheets/SSM3K35AMFV.pdf" H 8150 2125 50  0001 L BNN
 	1    7950 2275

Commit message: automated commit
Parts:
- U6, U7: footprint (none) -> custom:SOT-457; TEXT (none) -> CM1293A
Changed lines of the file:
@@
 F 0 "U6" H 2725 5050 60  0000 C CNN
 F 1 "NP_CM1293A-04SO" H 2975 4550 60  0000 C CNN
-F 2 "" H 2625 4700 60  0001 C CNN
-F 3 "datasheets/CM1293A-04SO-D.PDF" H 2775 4450 60  0001 C CNN
+F 2 "custom:SOT-457" H 2625 4700 60  0001 C CNN
+F 3 "~/datasheets/CM1293A-04SO-D.PDF" H 2775 4450 60  0001 C CNN
+F 4 "CM1293A" H 2775 4800 50  0001 C CNN "TEXT"
 	1    2775 4800
 	1    0    0    -1
@@
 F 0 "U7" H 2725 6600 60  0000 C CNN
 F 1 "NP_CM1293A-04SO" H 2975 6100 60  0000 C CNN
-F 2 "" H 2625 6250 60  0001 C CNN
-F 3 "datasheets/CM1293A-04SO-D.PDF" H 2775 6000 60  0001 C CNN
+F 2 "custom:SOT-457" H 2625 6250 60  0001 C CNN
+F 3 "~/datasheets/CM1293A-04SO-D.PDF" H 2775 6000 60  0001 C CNN
+F 4 "CM1293A" H 2775 6350 50  0001 C CNN "TEXT"
 	1    2775 6350
 	1    0    0    -1

Commit message: automated commit
Parts:
- removed SW3, SW4, SW5, SW6, SW7: NP_TACTILE_SWITCH, CUSTOM:TACTILE_SWITCH, symbol custom:TACTILE_SWITCH
- added SW3, SW4, SW5, SW6, SW7: TACTILE_SWITCH_SMALL, custom:TACTILE_SWITCH_SMALL, symbol custom:TACTILE_SWITCH_SMALL
Connections:
- net +3V3: now also SW3.2, SW4.2, SW5.2, SW6.2, SW7.2
- net AUX_0: now also SW3.1
- net AUX_1: now also SW4.1
- net AUX_2: now also SW5.1
- net AUX_3: now also SW6.1
- net AUX_4: now also SW7.1
Changed lines of the file:
@@
 	1    0    0    -1
 $EndComp
-Wire Wire Line
-	2650 1925 2650 1875
-Wire Wire Line
-	2550 1875 2550 1925
-Wire Wire Line
-	2650 1425 2650 1475
-Wire Wire Line
-	2550 1475 2550 1425
-$Comp
-L custom:TACTILE_SWITCH SW?
-U 1 1 5D3F593B
-P 2600 1675
-AR Path="/64D8274A/5D3F593B" Ref="SW?"  Part="1"
-AR Path="/61C6D021/5D3F593B" Ref="SW3"  Part="1"
-F 0 "SW3" H 2500 1850 60  0000 C CNN
-F 1 "NP_TACTILE_SWITCH" H 2600 1575 39  0000 C CNN
-F 2 "CUSTOM:TACTILE_SWITCH" H 2600 1850 60  0001 C CNN
-F 3 "" H 2600 1850 60  0001 C CNN
-	1    2600 1675
-	0    -1   -1   0
-$EndComp
-Wire Wire Line
-	2550 1925 2600 1925
-Wire Wire Line
-	2550 1425 2600 1425
-Wire Wire Line
-	2600 2125 2600 1925
 Connection ~ 2600 2125
-Connection ~ 2600 1925
-Wire Wire Line
-	2600 1925 2650 1925
-Wire Wire Line
-	2600 1300 2600 1425
-Connection ~ 2600 1425
-Wire Wire Line
-	2600 1425 2650 1425
+Wire Wire Line
+	2600 1300 2600 1500
 $Comp
 L custom:CRG0603F4K7 R41
@@
 	1    0    0    -1
 $EndComp
-Wire Wire Line
-	3925 1925 3925 1875
-Wire Wire Line
-	3825 1875 3825 1925
-Wire Wire Line
-	3925 1425 3925 1475
-Wire Wire Line
-	3825 1475 3825 1425
-$Comp
-L custom:TACTILE_SWITCH SW?
-U 1 1 5D4CA4FE
-P 3875 1675
-AR Path="/64D8274A/5D4CA4FE" Ref="SW?"  Part="1"
-AR Path="/61C6D021/5D4CA4FE" Ref="SW4"  Part="1"
-F 0 "SW4" H 3775 1850 60  0000 C CNN
-F 1 "NP_TACTILE_SWITCH" H 3875 1575 39  0000 C CNN
-F 2 "CUSTOM:TACTILE_SWITCH" H 3875 1850 60  0001 C CNN
-F 3 "" H 3875 1850 60  0001 C CNN
-	1    3875 1675
-	0    -1   -1   0
-$EndComp
-Wire Wire Line
-	3825 1925 3875 1925
-Wire Wire Line
-	3825 1425 3875 1425
-Wire Wire Line
-	3875 2125 3875 1925
-Connection ~ 3875 2125
-Connection ~ 3875 1925
-Wire Wire Line
-	3875 1925 3925 1925
-Wire Wire Line
-	3875 1300 3875 1425
-Connection ~ 3875 1425
-Wire Wire Line
-	3875 1425 3925 1425
 $Comp
 L custom:SSM3K35AMFV Q?
@@
 	1    0    0    -1
 $EndComp
-Wire Wire Line
-	5200 1925 5200 1875
-Wire Wire Line
-	5100 1875 5100 1925
-Wire Wire Line
-	5200 1425 5200 1475
-Wire Wire Line
-	5100 1475 5100 1425
-$Comp
-L custom:TACTILE_SWITCH SW?
-U 1 1 5D4D26E1
-P 5150 1675
-AR Path="/64D8274A/5D4D26E1" Ref="SW?"  Part="1"
-AR Path="/61C6D021/5D4D26E1" Ref="SW5"  Part="1"
-F 0 "SW5" H 5050 1850 60  0000 C CNN
-F 1 "NP_TACTILE_SWITCH" H 5150 1575 39  0000 C CNN
-F 2 "CUSTOM:TACTILE_SWITCH" H 5150 1850 60  0001 C CNN
-F 3 "" H 5150 1850 60  0001 C CNN
-	1    5150 1675
-	0    -1   -1   0
-$EndComp
-Wire Wire Line
-	5100 1925 5150 1925
-Wire Wire Line
-	5100 1425 5150 1425
-Wire Wire Line
-	5150 2125 5150 1925
-Connection ~ 5150 2125
-Connection ~ 5150 1925
-Wire Wire Line
-	5150 1925 5200 1925
-Wire Wire Line
-	5150 1300 5150 1425
-Connection ~ 5150 1425
-Wire Wire Line
-	5150 1425 5200 1425
 $Comp
 L custom:CRG0603F4K7 R43
@@
 	1    0    0    -1
 $EndComp
-Wire Wire Line
-	6475 1925 6475 1875
-Wire Wire Line
-	6375 1875 6375 1925
-Wire Wire Line
-	6475 1425 6475 1475
-Wire Wire Line
-	6375 1475 6375 1425
-$Comp
-L custom:TACTILE_SWITCH SW?
-U 1 1 5D4DEBF4
-P 6425 1675
-AR Path="/64D8274A/5D4DEBF4" Ref="SW?"  Part="1"
-AR Path="/61C6D021/5D4DEBF4" Ref="SW6"  Part="1"
-F 0 "SW6" H 6325 1850 60  0000 C CNN
-F 1 "NP_TACTILE_SWITCH" H 6425 1575 39  0000 C CNN
-F 2 "CUSTOM:TACTILE_SWITCH" H 6425 1850 60  0001 C CNN
-F 3 "" H 6425 1850 60  0001 C CNN
-	1    6425 1675
-	0    -1   -1   0
-$EndComp
-Wire Wire Line
-	6375 1925 6425 1925
-Wire Wire Line
-	6375 1425 6425 1425
-Wire Wire Line
-	6425 2125 6425 1925
-Connection ~ 6425 2125
-Connection ~ 6425 1925
-Wire Wire Line
-	6425 1925 6475 1925
-Wire Wire Line
-	6425 1300 6425 1425
-Connection ~ 6425 1425
-Wire Wire Line
-	6425 1425 6475 1425
 $Comp
 L custom:SSM3K35AMFV Q?
@@
 	1    0    0    -1
 $EndComp
-Wire Wire Line
-	7750 1925 7750 1875
-Wire Wire Line
-	7650 1875 7650 1925
-Wire Wire Line
-	7750 1425 7750 1475
-Wire Wire Line
-	7650 1475 7650 1425
-$Comp
-L custom:TACTILE_SWITCH SW?
-U 1 1 5D4DEC46
-P 7700 1675
-AR Path="/64D8274A/5D4DEC46" Ref="SW?"  Part="1"
-AR Path="/61C6D021/5D4DEC46" Ref="SW7"  Part="1"
-F 0 "SW7" H 7600 1850 60  0000 C CNN
-F 1 "NP_TACTILE_SWITCH" H 7700 1575 39  0000 C CNN
-F 2 "CUSTOM:TACTILE_SWITCH" H 7700 1850 60  0001 C CNN
-F 3 "" H 7700 1850 60  0001 C CNN
-	1    7700 1675
-	0    -1   -1   0
-$EndComp
-Wire Wire Line
-	7650 1925 7700 1925
-Wire Wire Line
-	7650 1425 7700 1425
-Wire Wire Line
-	7700 2125 7700 1925
-Connection ~ 7700 2125
-Connection ~ 7700 1925
-Wire Wire Line
-	7700 1925 7750 1925
-Wire Wire Line
-	7700 1300 7700 1425
-Connection ~ 7700 1425
-Wire Wire Line
-	7700 1425 7750 1425
 Text Notes 7700 5100 0    60   ~ 0
 LABEL PINS ON SILKSCREEN
@@
 Wire Wire Line
 	3125 6200 3600 6200
+$Comp
+L custom:TACTILE_SWITCH_SMALL SW3
+U 1 1 5D1462DE
+P 2600 1650
+F 0 "SW3" H 2400 1800 60  0000 L BNN
+F 1 "TACTILE_SWITCH_SMALL" H 2110 1530 60  0001 L BNN
+F 2 "custom:TACTILE_SWITCH_SMALL" H 2600 1450 60  0001 C CNN
+F 3 "" H 2600 1800 60  0001 C CNN
+	1    2600 1650
+	0    -1   -1   0
+$EndComp
+Wire Wire Line
+	2600 2125 2600 1800
+Wire Wire Line
+	3875 1300 3875 1500
+$Comp
+L custom:TACTILE_SWITCH_SMALL SW4
+U 1 1 5D181AE5
+P 3875 1650
+F 0 "SW4" H 3675 1800 60  0000 L BNN
+F 1 "TACTILE_SWITCH_SMALL" H 3385 1530 60  0001 L BNN
+F 2 "custom:TACTILE_SWITCH_SMALL" H 3875 1450 60  0001 C CNN
+F 3 "" H 3875 1800 60  0001 C CNN
+	1    3875 1650
+	0    -1   -1   0
+$EndComp
+Wire Wire Line
+	3875 2125 3875 1800
+Wire Wire Line
+	5150 1300 5150 1500
+$Comp
+L custom:TACTILE_SWITCH_SMALL SW5
+U 1 1 5D18456E
+P 5150 1650
+F 0 "SW5" H 4950 1800 60  0000 L BNN
+F 1 "TACTILE_SWITCH_SMALL" H 4660 1530 60  0001 L BNN
+F 2 "custom:TACTILE_SWITCH_SMALL" H 5150 1450 60  0001 C CNN
+F 3 "" H 5150 1800 60  0001 C CNN
+	1    5150 1650
+	0    -1   -1   0
+$EndComp
+Wire Wire Line
+	5150 2125 5150 1800
+Wire Wire Line
+	6425 1300 6425 1500
+$Comp
+L custom:TACTILE_SWITCH_SMALL SW6
+U 1 1 5D18746D
+P 6425 1650
+F 0 "SW6" H 6225 1800 60  0000 L BNN
+F 1 "TACTILE_SWITCH_SMALL" H 5935 1530 60  0001 L BNN
+F 2 "custom:TACTILE_SWITCH_SMALL" H 6425 1450 60  0001 C CNN
+F 3 "" H 6425 1800 60  0001 C CNN
+	1    6425 1650
+	0    -1   -1   0
+$EndComp
+Wire Wire Line
+	6425 2125 6425 1800
+Connection ~ 6425 2125
+Connection ~ 5150 2125
+Connection ~ 3875 2125
+Wire Wire Line
+	7700 1300 7700 1500
+$Comp
+L custom:TACTILE_SWITCH_SMALL SW7
+U 1 1 5D18A7CB
+P 7700 1650
+F 0 "SW7" H 7500 1800 60  0000 L BNN
+F 1 "TACTILE_SWITCH_SMALL" H 7210 1530 60  0001 L BNN
+F 2 "custom:TACTILE_SWITCH_SMALL" H 7700 1450 60  0001 C CNN
+F 3 "" H 7700 1800 60  0001 C CNN
+	1    7700 1650
+	0    -1   -1   0
+$EndComp
+Wire Wire Line
+	7700 2125 7700 1800
+Connection ~ 7700 2125
 $EndSCHEMATC

Commit message: automated commit
Parts:
- removed D13, D14, D15: LED_GENERIC_0805, Diode_SMD:D_0805_2012Metric, symbol custom:LED_GENERIC_0805
- removed J5, J6, J8: PTH_1.5_mm, TestPoint:TestPoint_THTPad_D3.0mm_Drill1.5mm, symbol custom:PTH_1.5_mm
- removed J7: Conn_01x05_Male, Connector_PinHeader_2.54mm:PinHeader_1x05_P2.54mm_Vertical, symbol Connector:Conn_01x05_Male
- removed Q6, Q7, Q8: SSM3K35AMFV, Package_TO_SOT_SMD:SOT-723, symbol custom:SSM3K35AMFV
- removed R37, R38, R39: ‎RMCF0603FT470R‎, Resistor_SMD:R_0603_1608Metric, symbol custom:‎RMCF0603FT470R‎
- removed R42, R43, R44: CRG0603F4K7, Resistor_SMD:R_0603_1608Metric, symbol custom:CRG0603F4K7
- removed SW5, SW6, SW7: TACTILE_SWITCH_SMALL, custom:TACTILE_SWITCH_SMALL, symbol custom:TACTILE_SWITCH_SMALL
- removed U7: NP_CM1293A-04SO, custom:SOT-457, symbol custom:CM1293A-04SO_ALTERNATE_SYMBOL
- added J5: Conn_01x02_Male, Connector_PinHeader_2.54mm:PinHeader_1x02_P2.54mm_Vertical, symbol Connector:Conn_01x02_Male
Connections:
- net AUX_2 is gone; now on net +3V3: U6.4 (CH3)
- net AUX_3 is gone; now on net +3V3: U6.6 (CH4)
- net AUX_0: now also J5.1 (Pin_1)
- net AUX_1: now also J5.2 (Pin_2)
Other:
- note removed: "INCLUDE FILLED RECTANGLES\nON SILKSCREEN NEAR EACH\nLED TO WRITE LABELS ON"
- note removed: "ROUTE 3V3 *THROUGH* FOR ALL BUTTONS"
- moved on the sheet: D11, D12, J3, J4, Q4, Q5, R35, R36, R40, R41, SW3, SW4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
