File: COLUMN_DRIVERS_0.sch (KiCad schematic (older format))
At the start: 42 parts, among them Q12 DMG6602, Q13 DMG6602, Q14 DMG6602, Q15 SSM3K35AMFV, Q16 SSM3K35AMFV, Q17 SSM3K35AMFV, Q18 SSM3K35AMFV, Q19 SSM3K35AMFV, Q20 SSM3K35AMFV, Q21 DMG6602, Q22 DMG6602, Q23 DMG6602, Q24 SSM3K35AMFV, Q25 SSM3K35AMFV, Q26 SSM3K35AMFV, Q27 SSM3K35AMFV, Q28 SSM3K35AMFV, Q29 SSM3K35AMFV

Commit message: automated commit
Parts:
- renumbered Q12 to Q49, Q13 to Q50, Q14 to Q51, Q15 to Q52, Q16 to Q53, Q17 to Q54, Q18 to Q55, Q19 to Q56, Q20 to Q57, Q21 to Q58, Q22 to Q59, Q23 to Q60, Q24 to Q61, Q25 to Q62, Q26 to Q63, Q27 to Q64, Q28 to Q65, Q29 to Q66, R66 to R139, R67 to R140, R68 to R141, R69 to R142, R70 to R143, R71 to R144, R72 to R145, R73 to R146, R74 to R147, R75 to R148, R76 to R149, R77 to R150, R78 to R151, R79 to R152, R80 to R153, R81 to R154, R82 to R155, R83 to R156, R84 to R157, R85 to R158, R86 to R159, R87 to R160, R88 to R161, R89 to R162

Commit message: automated commit
Parts:
- R139, R140, R141, R142, R143, R144, R145, R146, R147, R148, R149, R150, R151, R152, R153, R154, R155, R156, R157, R158, R159, R160, R161, R162: Resistance 4.7k -> (none); TOLERANCE (none) -> 5%; VALUE (none) -> 4k7

Commit message: automated commit
Parts:
- removed R147, R148, R149, R150, R159, R160, R161, R162: CRG0603F4K7, Resistor_SMD:R_0603_1608Metric, symbol custom:CRG0603F4K7
- added R143, R144, R145, R146, R153, R154, R155, R156: CRG0603F4K7, Resistor_SMD:R_0603_1608Metric, symbol custom:CRG0603F4K7
- added TP74, TP75, TP76, TP77, TP78, TP79, TP80, TP81, TP82, TP83, TP84, TP85, TP86, TP87: TestPoint, symbol Connector:TestPoint
- renumbered R139 to R135, R140 to R136, R141 to R137, R142 to R138, R143 to R139, R144 to R140, R145 to R141, R146 to R142, R151 to R147, R152 to R148, R153 to R149, R154 to R150, R155 to R151, R156 to R152
Connections:
- net +12V: now also TP74.1, TP75.1
- net COL00: now also TP80.1
- net COL00_OFF: now also TP78.1
- net COL00_ON: now also TP79.1
- net COL01: now also TP83.1
- net COL01_OFF: now also R144.1, TP81.1
- net COL01_ON: now also R143.1, TP82.1
- net COL02_OFF: now also R146.1
- net COL02_ON: now also R145.1
- net COL03_OFF: now also R154.1; no longer R158.1
- net COL03_ON: now also R153.1; no longer R157.1
- net COL04_OFF: now also R156.1
- net COL04_ON: now also R155.1
- net COL05_OFF: now also R158.1
- net COL05_ON: now also R157.1
- net GND: now also R143.2, R144.2, R145.2, R146.2, R153.2, R154.2, R155.2, R156.2, TP86.1, TP87.1
- net at Q49.1 (G), Q55.3 (D), R138.1: now also TP84.1
- net at Q49.3 (G), Q52.3 (D), R135.2: now also TP76.1
- net at Q50.1 (G), Q56.3 (D), R139.1: now also TP85.1
- net at Q50.3 (G), Q53.3 (D), R136.2: now also TP77.1

Commit message: automated commit
Parts:
- Q52, Q53, Q54, Q55, Q56, Q57, Q61, Q62, Q63, Q64, Q65, Q66: footprint (none) -> Package_TO_SOT_SMD:SOT-723
Changed lines of the file:
@@
 F 0 "Q63" V 9675 4800 50  0000 L BNN
 F 1 "SSM3K35AMFV" V 9600 4625 50  0000 L BNN
-F 2 "" H 9550 4750 50  0001 L BIN
+F 2 "Package_TO_SOT_SMD:SOT-723" H 9550 4750 50  0001 L BIN
 F 3 "datasheets/SSM3K35AMFV.pdf" H 9550 4725 50  0001 L BNN
 	1    9350 4875
@@
 F 0 "Q66" V 9350 5425 50  0000 L BNN
 F 1 "SSM3K35AMFV" V 9275 5250 50  0000 L BNN
-F 2 "" H 9225 5375 50  0001 L BIN
+F 2 "Package_TO_SOT_SMD:SOT-723" H 9225 5375 50  0001 L BIN
 F 3 "datasheets/SSM3K35AMFV.pdf" H 9225 5350 50  0001 L BNN
 	1    9025 5500
@@
 F 0 "Q62" V 6275 4800 50  0000 L BNN
 F 1 "SSM3K35AMFV" V 6200 4625 50  0000 L BNN
-F 2 "" H 6150 4750 50  0001 L BIN
+F 2 "Package_TO_SOT_SMD:SOT-723" H 6150 4750 50  0001 L BIN
 F 3 "datasheets/SSM3K35AMFV.pdf" H 6150 4725 50  0001 L BNN
 	1    5950 4875
@@
 F 0 "Q61" V 2875 4800 50  0000 L BNN
 F 1 "SSM3K35AMFV" V 2800 4625 50  0000 L BNN
-F 2 "" H 2750 4750 50  0001 L BIN
+F 2 "Package_TO_SOT_SMD:SOT-723" H 2750 4750 50  0001 L BIN
 F 3 "datasheets/SSM3K35AMFV.pdf" H 2750 4725 50  0001 L BNN
 	1    2550 4875
@@
 F 0 "Q64" V 2550 5425 50  0000 L BNN
 F 1 "SSM3K35AMFV" V 2475 5250 50  0000 L BNN
-F 2 "" H 2425 5375 50  0001 L BIN
+F 2 "Package_TO_SOT_SMD:SOT-723" H 2425 5375 50  0001 L BIN
 F 3 "datasheets/SSM3K35AMFV.pdf" H 2425 5350 50  0001 L BNN
 	1    2225 5500
@@
 F 0 "Q54" V 9675 2200 50  0000 L BNN
 F 1 "SSM3K35AMFV" V 9600 2025 50  0000 L BNN
-F 2 "" H 9550 2150 50  0001 L BIN
+F 2 "Package_TO_SOT_SMD:SOT-723" H 9550 2150 50  0001 L BIN
 F 3 "datasheets/SSM3K35AMFV.pdf" H 9550 2125 50  0001 L BNN
 	1    9350 2275
@@
 F 0 "Q57" V 9350 2825 50  0000 L BNN
 F 1 "SSM3K35AMFV" V 9275 2650 50  0000 L BNN
-F 2 "" H 9225 2775 50  0001 L BIN
+F 2 "Package_TO_SOT_SMD:SOT-723" H 9225 2775 50  0001 L BIN
 F 3 "datasheets/SSM3K35AMFV.pdf" H 9225 2750 50  0001 L BNN
 	1    9025 2900
@@
 F 0 "Q53" V 6275 2200 50  0000 L BNN
 F 1 "SSM3K35AMFV" V 6200 2025 50  0000 L BNN
-F 2 "" H 6150 2150 50  0001 L BIN
+F 2 "Package_TO_SOT_SMD:SOT-723" H 6150 2150 50  0001 L BIN
 F 3 "datasheets/SSM3K35AMFV.pdf" H 6150 2125 50  0001 L BNN
 	1    5950 2275
@@
 F 0 "Q56" V 5950 2825 50  0000 L BNN
 F 1 "SSM3K35AMFV" V 5875 2650 50  0000 L BNN
-F 2 "" H 5825 2775 50  0001 L BIN
+F 2 "Package_TO_SOT_SMD:SOT-723" H 5825 2775 50  0001 L BIN
 F 3 "datasheets/SSM3K35AMFV.pdf" H 5825 2750 50  0001 L BNN
 	1    5625 2900
@@
 F 0 "Q52" V 2875 2200 50  0000 L BNN
 F 1 "SSM3K35AMFV" V 2800 2025 50  0000 L BNN
-F 2 "" H 2750 2150 50  0001 L BIN
+F 2 "Package_TO_SOT_SMD:SOT-723" H 2750 2150 50  0001 L BIN
 F 3 "datasheets/SSM3K35AMFV.pdf" H 2750 2125 50  0001 L BNN
 	1    2550 2275
@@
 F 0 "Q55" V 2550 2825 50  0000 L BNN
 F 1 "SSM3K35AMFV" V 2475 2650 50  0000 L BNN
-F 2 "" H 2425 2775 50  0001 L BIN
+F 2 "Package_TO_SOT_SMD:SOT-723" H 2425 2775 50  0001 L BIN
 F 3 "datasheets/SSM3K35AMFV.pdf" H 2425 2750 50  0001 L BNN
 	1    2225 2900
@@
 F 0 "Q65" V 5950 5425 50  0000 L BNN
 F 1 "SSM3K35AMFV" V 5875 5250 50  0000 L BNN
-F 2 "" H 5825 5375 50  0001 L BIN
+F 2 "Package_TO_SOT_SMD:SOT-723" H 5825 5375 50  0001 L BIN
 F 3 "datasheets/SSM3K35AMFV.pdf" H 5825 5350 50  0001 L BNN
 	1    5625 5500

Commit message: automated commit
Parts:
- TP79: renamed from TP74; footprint (none) -> custom:TestPoint_THTPad_D1.0mm_Drill0.5mm
- TP80: renamed from TP75; footprint (none) -> custom:TestPoint_THTPad_D1.0mm_Drill0.5mm
- TP81: renamed from TP76; footprint (none) -> custom:TestPoint_THTPad_D1.0mm_Drill0.5mm
- TP82: renamed from TP77; footprint (none) -> custom:TestPoint_THTPad_D1.0mm_Drill0.5mm
- TP83: renamed from TP78; footprint (none) -> custom:TestPoint_THTPad_D1.0mm_Drill0.5mm
- TP84: renamed from TP79; footprint (none) -> custom:TestPoint_THTPad_D1.0mm_Drill0.5mm
- TP85: renamed from TP80; footprint (none) -> custom:TestPoint_THTPad_D1.0mm_Drill0.5mm
- TP86: renamed from TP81; footprint (none) -> custom:TestPoint_THTPad_D1.0mm_Drill0.5mm
- TP87: renamed from TP82; footprint (none) -> custom:TestPoint_THTPad_D1.0mm_Drill0.5mm
- TP88: renamed from TP83; footprint (none) -> custom:TestPoint_THTPad_D1.0mm_Drill0.5mm
- TP89: renamed from TP84; footprint (none) -> custom:TestPoint_THTPad_D1.0mm_Drill0.5mm
- TP90: renamed from TP85; footprint (none) -> custom:TestPoint_THTPad_D1.0mm_Drill0.5mm
- TP91: renamed from TP86; footprint (none) -> custom:TestPoint_THTPad_D1.0mm_Drill0.5mm
- TP92: renamed from TP87; footprint (none) -> custom:TestPoint_THTPad_D1.0mm_Drill0.5mm
Changed lines of the file:
@@
 AR Path="/609E0ED6/5D9A7D12" Ref="TP?"  Part="1"
 AR Path="/621F0CB4/5D9A7D12" Ref="TP?"  Part="1"
-AR Path="/62A8D0C3/5D9A7D12" Ref="TP78"  Part="1"
-F 0 "TP78" V 1275 2475 50  0000 C CNN
+AR Path="/62A8D0C3/5D9A7D12" Ref="TP83"  Part="1"
+F 0 "TP83" V 1275 2475 50  0000 C CNN
 F 1 "TestPoint" H 1025 2225 50  0001 C CNN
-F 2 "" H 1475 2175 50  0001 C CNN
+F 2 "custom:TestPoint_THTPad_D1.0mm_Drill0.5mm" H 1475 2175 50  0001 C CNN
 F 3 "~" H 1475 2175 50  0001 C CNN
 	1    1275 2175
@@
 AR Path="/609E0ED6/5D9BF3B4" Ref="TP?"  Part="1"
 AR Path="/621F0CB4/5D9BF3B4" Ref="TP?"  Part="1"
-AR Path="/62A8D0C3/5D9BF3B4" Ref="TP79"  Part="1"
-F 0 "TP79" V 1425 2475 50  0000 C CNN
+AR Path="/62A8D0C3/5D9BF3B4" Ref="TP84"  Part="1"
+F 0 "TP84" V 1425 2475 50  0000 C CNN
 F 1 "TestPoint" H 1175 2225 50  0001 C CNN
-F 2 "" H 1625 2175 50  0001 C CNN
+F 2 "custom:TestPoint_THTPad_D1.0mm_Drill0.5mm" H 1625 2175 50  0001 C CNN
 F 3 "~" H 1625 2175 50  0001 C CNN
 	1    1425 2175
@@
 AR Path="/609E0ED6/5D9D75F8" Ref="TP?"  Part="1"
 AR Path="/621F0CB4/5D9D75F8" Ref="TP?"  Part="1"
-AR Path="/62A8D0C3/5D9D75F8" Ref="TP86"  Part="1"
-F 0 "TP86" V 1025 3500 50  0000 C CNN
+AR Path="/62A8D0C3/5D9D75F8" Ref="TP91"  Part="1"
+F 0 "TP91" V 1025 3500 50  0000 C CNN
 F 1 "TestPoint" H 775 3250 50  0001 C CNN
-F 2 "" H 1225 3200 50  0001 C CNN
+F 2 "custom:TestPoint_THTPad_D1.0mm_Drill0.5mm" H 1225 3200 50  0001 C CNN
 F 3 "~" H 1225 3200 50  0001 C CNN
 	1    1025 3200
@@
 AR Path="/609E0ED6/5D9E3D97" Ref="TP?"  Part="1"
 AR Path="/621F0CB4/5D9E3D97" Ref="TP?"  Part="1"
-AR Path="/62A8D0C3/5D9E3D97" Ref="TP76"  Part="1"
-F 0 "TP76" V 2550 2175 50  0000 C CNN
+AR Path="/62A8D0C3/5D9E3D97" Ref="TP81"  Part="1"
+F 0 "TP81" V 2550 2175 50  0000 C CNN
 F 1 "TestPoint" H 2300 1925 50  0001 C CNN
-F 2 "" H 2750 1875 50  0001 C CNN
+F 2 "custom:TestPoint_THTPad_D1.0mm_Drill0.5mm" H 2750 1875 50  0001 C CNN
 F 3 "~" H 2750 1875 50  0001 C CNN
 	1    2550 1875
@@
 AR Path="/609E0ED6/5D9EFED5" Ref="TP?"  Part="1"
 AR Path="/621F0CB4/5D9EFED5" Ref="TP?"  Part="1"
-AR Path="/62A8D0C3/5D9EFED5" Ref="TP74"  Part="1"
-F 0 "TP74" V 2550 1675 50  0000 C CNN
+AR Path="/62A8D0C3/5D9EFED5" Ref="TP79"  Part="1"
+F 0 "TP79" V 2550 1675 50  0000 C CNN
 F 1 "TestPoint" H 2300 1425 50  0001 C CNN
-F 2 "" H 2750 1375 50  0001 C CNN
+F 2 "custom:TestPoint_THTPad_D1.0mm_Drill0.5mm" H 2750 1375 50  0001 C CNN
 F 3 "~" H 2750 1375 50  0001 C CNN
 	1    2550 1375
@@
 AR Path="/609E0ED6/5DA08E40" Ref="TP?"  Part="1"
 AR Path="/621F0CB4/5DA08E40" Ref="TP?"  Part="1"
-AR Path="/62A8D0C3/5DA08E40" Ref="TP80"  Part="1"
-F 0 "TP80" V 3400 2475 50  0000 C CNN
+AR Path="/62A8D0C3/5DA08E40" Ref="TP85"  Part="1"
+F 0 "TP85" V 3400 2475 50  0000 C CNN
 F 1 "TestPoint" H 3150 2225 50  0001 C CNN
-F 2 "" H 3600 2175 50  0001 C CNN
+F 2 "custom:TestPoint_THTPad_D1.0mm_Drill0.5mm" H 3600 2175 50  0001 C CNN
 F 3 "~" H 3600 2175 50  0001 C CNN
 	1    3400 2175
@@
 AR Path="/609E0ED6/5DA237AD" Ref="TP?"  Part="1"
 AR Path="/621F0CB4/5DA237AD" Ref="TP?"  Part="1"
-AR Path="/62A8D0C3/5DA237AD" Ref="TP84"  Part="1"
-F 0 "TP84" H 2725 2925 50  0000 C CNN
+AR Path="/62A8D0C3/5DA237AD" Ref="TP89"  Part="1"
+F 0 "TP89" H 2725 2925 50  0000 C CNN
 F 1 "TestPoint" H 2525 2725 50  0001 C CNN
-F 2 "" H 2975 2675 50  0001 C CNN
+F 2 "custom:TestPoint_THTPad_D1.0mm_Drill0.5mm" H 2975 2675 50  0001 C CNN
 F 3 "~" H 2975 2675 50  0001 C CNN
 	1    2775 2675
@@
 AR Path="/609E0ED6/5DA46205" Ref="TP?"  Part="1"
 AR Path="/621F0CB4/5DA46205" Ref="TP?"  Part="1"
-AR Path="/62A8D0C3/5DA46205" Ref="TP81"  Part="1"
-F 0 "TP81" V 4675 2475 50  0000 C CNN
+AR Path="/62A8D0C3/5DA46205" Ref="TP86"  Part="1"
+F 0 "TP86" V 4675 2475 50  0000 C CNN
 F 1 "TestPoint" H 4425 2225 50  0001 C CNN
-F 2 "" H 4875 2175 50  0001 C CNN
+F 2 "custom:TestPoint_THTPad_D1.0mm_Drill0.5mm" H 4875 2175 50  0001 C CNN
 F 3 "~" H 4875 2175 50  0001 C CNN
 	1    4675 2175
@@
 AR Path="/609E0ED6/5DA4620E" Ref="TP?"  Part="1"
 AR Path="/621F0CB4/5DA4620E" Ref="TP?"  Part="1"
-AR Path="/62A8D0C3/5DA4620E" Ref="TP82"  Part="1"
-F 0 "TP82" V 4825 2475 50  0000 C CNN
+AR Path="/62A8D0C3/5DA4620E" Ref="TP87"  Part="1"
+F 0 "TP87" V 4825 2475 50  0000 C CNN
 F 1 "TestPoint" H 4575 2225 50  0001 C CNN
-F 2 "" H 5025 2175 50  0001 C CNN
+F 2 "custom:TestPoint_THTPad_D1.0mm_Drill0.5mm" H 5025 2175 50  0001 C CNN
 F 3 "~" H 5025 2175 50  0001 C CNN
 	1    4825 2175
@@
 AR Path="/609E0ED6/5DA46217" Ref="TP?"  Part="1"
 AR Path="/621F0CB4/5DA46217" Ref="TP?"  Part="1"
-AR Path="/62A8D0C3/5DA46217" Ref="TP87"  Part="1"
-F 0 "TP87" V 4425 3500 50  0000 C CNN
+AR Path="/62A8D0C3/5DA46217" Ref="TP92"  Part="1"
+F 0 "TP92" V 4425 3500 50  0000 C CNN
 F 1 "TestPoint" H 4175 3250 50  0001 C CNN
-F 2 "" H 4625 3200 50  0001 C CNN
+F 2 "custom:TestPoint_THTPad_D1.0mm_Drill0.5mm" H 4625 3200 50  0001 C CNN
 F 3 "~" H 4625 3200 50  0001 C CNN
 	1    4425 3200
@@
 AR Path="/609E0ED6/5DA4621F" Ref="TP?"  Part="1"
 AR Path="/621F0CB4/5DA4621F" Ref="TP?"  Part="1"
-AR Path="/62A8D0C3/5DA4621F" Ref="TP77"  Part="1"
-F 0 "TP77" V 5950 2175 50  0000 C CNN
+AR Path="/62A8D0C3/5DA4621F" Ref="TP82"  Part="1"
+F 0 "TP82" V 5950 2175 50  0000 C CNN
 F 1 "TestPoint" H 5700 1925 50  0001 C CNN
-F 2 "" H 6150 1875 50  0001 C CNN
+F 2 "custom:TestPoint_THTPad_D1.0mm_Drill0.5mm" H 6150 1875 50  0001 C CNN
 F 3 "~" H 6150 1875 50  0001 C CNN
 	1    5950 1875
@@
 AR Path="/609E0ED6/5DA46226" Ref="TP?"  Part="1"
 AR Path="/621F0CB4/5DA46226" Ref="TP?"  Part="1"
-AR Path="/62A8D0C3/5DA46226" Ref="TP75"  Part="1"
-F 0 "TP75" V 5950 1675 50  0000 C CNN
+AR Path="/62A8D0C3/5DA46226" Ref="TP80"  Part="1"
+F 0 "TP80" V 5950 1675 50  0000 C CNN
 F 1 "TestPoint" H 5700 1425 50  0001 C CNN
-F 2 "" H 6150 1375 50  0001 C CNN
+F 2 "custom:TestPoint_THTPad_D1.0mm_Drill0.5mm" H 6150 1375 50  0001 C CNN
 F 3 "~" H 6150 1375 50  0001 C CNN
 	1    5950 1375
@@
 AR Path="/609E0ED6/5DA46230" Ref="TP?"  Part="1"
 AR Path="/621F0CB4/5DA46230" Ref="TP?"  Part="1"
-AR Path="/62A8D0C3/5DA46230" Ref="TP83"  Part="1"
-F 0 "TP83" V 6800 2475 50  0000 C CNN
+AR Path="/62A8D0C3/5DA46230" Ref="TP88"  Part="1"
+F 0 "TP88" V 6800 2475 50  0000 C CNN
 F 1 "TestPoint" H 6550 2225 50  0001 C CNN
-F 2 "" H 7000 2175 50  0001 C CNN
+F 2 "custom:TestPoint_THTPad_D1.0mm_Drill0.5mm" H 7000 2175 50  0001 C CNN
 F 3 "~" H 7000 2175 50  0001 C CNN
 	1    6800 2175
@@
 AR Path="/609E0ED6/5DA4623A" Ref="TP?"  Part="1"
 AR Path="/621F0CB4/5DA4623A" Ref="TP?"  Part="1"
-AR Path="/62A8D0C3/5DA4623A" Ref="TP85"  Part="1"
-F 0 "TP85" H 6125 2925 50  0000 C CNN
+AR Path="/62A8D0C3/5DA4623A" Ref="TP90"  Part="1"
+F 0 "TP90" H 6125 2925 50  0000 C CNN
 F 1 "TestPoint" H 5925 2725 50  0001 C CNN
-F 2 "" H 6375 2675 50  0001 C CNN
+F 2 "custom:TestPoint_THTPad_D1.0mm_Drill0.5mm" H 6375 2675 50  0001 C CNN
 F 3 "~" H 6375 2675 50  0001 C CNN
 	1    6175 2675

Commit message: automated commit
Parts:
- renumbered R135 to R143, R136 to R144, R137 to R145, R138 to R146, R139 to R147, R140 to R148, R141 to R149, R142 to R150, R143 to R151, R144 to R152, R145 to R153, R146 to R154, R147 to R155, R148 to R156, R149 to R157, R150 to R158, R151 to R159, R152 to R160, R153 to R161, R154 to R162, R155 to R163, R156 to R164, R157 to R165, R158 to R166

Commit message: automated commit
Parts:
- renumbered Q49 to Q48, Q50 to Q49, Q51 to Q50, Q52 to Q51, Q53 to Q52, Q54 to Q53, Q55 to Q54, Q56 to Q55, Q57 to Q56, Q58 to Q57, Q59 to Q58, Q60 to Q59, Q61 to Q60, Q62 to Q61, Q63 to Q62, Q64 to Q63, Q65 to Q64, Q66 to Q65, R143 to R142, R144 to R143, R145 to R144, R146 to R145, R147 to R146, R148 to R147, R149 to R148, R150 to R149, R151 to R150, R152 to R151, R153 to R152, R154 to R153, R155 to R154, R156 to R155, R157 to R156, R158 to R157, R159 to R158, R160 to R159, R161 to R160, R162 to R161, R163 to R162, R164 to R163, R165 to R164, R166 to R165, TP79 to TP78, TP80 to TP79, TP81 to TP80, TP82 to TP81, TP83 to TP82, TP84 to TP83, TP85 to TP84, TP86 to TP85, TP87 to TP86, TP88 to TP87, TP89 to TP88, TP90 to TP89, TP91 to TP90, TP92 to TP91

Commit message: automated commit
Parts:
- removed TP79, TP81, TP85, TP86, TP87, TP89, TP91: TestPoint, custom:TestPoint_THTPad_D1.0mm_Drill0.5mm, symbol Connector:TestPoint
Changed lines of the file:
@@
 Wire Wire Line
 	4425 2275 4525 2275
-Wire Wire Line
-	4425 2575 4675 2575
 Text GLabel 1025 5175 0    50   Input ~ 0
 COL03_OFF
@@
 Connection ~ 5725 2575
 Wire Wire Line
-	5725 2575 6175 2575
-Wire Wire Line
 	5725 2575 5525 2575
 Wire Wire Line
@@
 	5225 2575 4825 2575
 Wire Wire Line
-	4525 2275 4825 2275
-Wire Wire Line
 	4825 3200 5725 3200
 Wire Wire Line
@@
 Wire Wire Line
 	6050 1975 6250 1975
-Wire Wire Line
-	6050 1775 6050 1875
 Connection ~ 6550 1375
 Wire Wire Line
@@
 Wire Wire Line
 	6550 2175 6550 2275
-Wire Wire Line
-	6550 2275 6700 2275
 Connection ~ 6550 2275
 Wire Wire Line
 	6550 2275 6550 2375
-$Comp
-L Connector:TestPoint TP?
-U 1 1 5DA46205
-P 4675 2175
-AR Path="/5DA46205" Ref="TP?"  Part="1"
-AR Path="/61C6D021/5DA46205" Ref="TP?"  Part="1"
-AR Path="/609E0ED6/5DA46205" Ref="TP?"  Part="1"
-AR Path="/621F0CB4/5DA46205" Ref="TP?"  Part="1"
-AR Path="/62A8D0C3/5DA46205" Ref="TP85"  Part="1"
-F 0 "TP85" V 4675 2475 50  0000 C CNN
-F 1 "TestPoint" H 4425 2225 50  0001 C CNN
-F 2 "custom:TestPoint_THTPad_D1.0mm_Drill0.5mm" H 4875 2175 50  0001 C CNN
-F 3 "~" H 4875 2175 50  0001 C CNN
-	1    4675 2175
-	-1   0    0    -1
-$EndComp
-$Comp
-L Connector:TestPoint TP?
-U 1 1 5DA4620E
-P 4825 2175
-AR Path="/5DA4620E" Ref="TP?"  Part="1"
-AR Path="/61C6D021/5DA4620E" Ref="TP?"  Part="1"
-AR Path="/609E0ED6/5DA4620E" Ref="TP?"  Part="1"
-AR Path="/621F0CB4/5DA4620E" Ref="TP?"  Part="1"
-AR Path="/62A8D0C3/5DA4620E" Ref="TP86"  Part="1"
-F 0 "TP86" V 4825 2475 50  0000 C CNN
-F 1 "TestPoint" H 4575 2225 50  0001 C CNN
-F 2 "custom:TestPoint_THTPad_D1.0mm_Drill0.5mm" H 5025 2175 50  0001 C CNN
-F 3 "~" H 5025 2175 50  0001 C CNN
-	1    4825 2175
-	-1   0    0    -1
-$EndComp
-Wire Wire Line
-	4825 2175 4825 2275
-$Comp
-L Connector:TestPoint TP?
-U 1 1 5DA46217
-P 4425 3200
-AR Path="/5DA46217" Ref="TP?"  Part="1"
-AR Path="/61C6D021/5DA46217" Ref="TP?"  Part="1"
-AR Path="/609E0ED6/5DA46217" Ref="TP?"  Part="1"
-AR Path="/621F0CB4/5DA46217" Ref="TP?"  Part="1"
-AR Path="/62A8D0C3/5DA46217" Ref="TP91"  Part="1"
-F 0 "TP91" V 4425 3500 50  0000 C CNN
-F 1 "TestPoint" H 4175 3250 50  0001 C CNN
-F 2 "custom:TestPoint_THTPad_D1.0mm_Drill0.5mm" H 4625 3200 50  0001 C CNN
-F 3 "~" H 4625 3200 50  0001 C CNN
-	1    4425 3200
-	0    -1   1    0
-$EndComp
-Wire Wire Line
-	4425 3200 4525 3200
-$Comp
-L Connector:TestPoint TP?
-U 1 1 5DA4621F
-P 5950 1875
-AR Path="/5DA4621F" Ref="TP?"  Part="1"
-AR Path="/61C6D021/5DA4621F" Ref="TP?"  Part="1"
-AR Path="/609E0ED6/5DA4621F" Ref="TP?"  Part="1"
-AR Path="/621F0CB4/5DA4621F" Ref="TP?"  Part="1"
-AR Path="/62A8D0C3/5DA4621F" Ref="TP81"  Part="1"
-F 0 "TP81" V 5950 2175 50  0000 C CNN
-F 1 "TestPoint" H 5700 1925 50  0001 C CNN
-F 2 "custom:TestPoint_THTPad_D1.0mm_Drill0.5mm" H 6150 1875 50  0001 C CNN
-F 3 "~" H 6150 1875 50  0001 C CNN
-	1    5950 1875
-	0    -1   1    0
-$EndComp
-Wire Wire Line
-	5950 1875 6050 1875
-$Comp
-L Connector:TestPoint TP?
-U 1 1 5DA46226
-P 5950 1375
-AR Path="/5DA46226" Ref="TP?"  Part="1"
-AR Path="/61C6D021/5DA46226" Ref="TP?"  Part="1"
-AR Path="/609E0ED6/5DA46226" Ref="TP?"  Part="1"
-AR Path="/621F0CB4/5DA46226" Ref="TP?"  Part="1"
-AR Path="/62A8D0C3/5DA46226" Ref="TP79"  Part="1"
-F 0 "TP79" V 5950 1675 50  0000 C CNN
-F 1 "TestPoint" H 5700 1425 50  0001 C CNN
-F 2 "custom:TestPoint_THTPad_D1.0mm_Drill0.5mm" H 6150 1375 50  0001 C CNN
-F 3 "~" H 6150 1375 50  0001 C CNN
-	1    5950 1375
-	0    -1   1    0
-$EndComp
-Wire Wire Line
-	5950 1375 6050 1375
-$Comp
-L Connector:TestPoint TP?
-U 1 1 5DA46230
-P 6800 2175
-AR Path="/5DA46230" Ref="TP?"  Part="1"
-AR Path="/61C6D021/5DA46230" Ref="TP?"  Part="1"
-AR Path="/609E0ED6/5DA46230" Ref="TP?"  Part="1"
-AR Path="/621F0CB4/5DA46230" Ref="TP?"  Part="1"
-AR Path="/62A8D0C3/5DA46230" Ref="TP87"  Part="1"
-F 0 "TP87" V 6800 2475 50  0000 C CNN
-F 1 "TestPoint" H 6550 2225 50  0001 C CNN
-F 2 "custom:TestPoint_THTPad_D1.0mm_Drill0.5mm" H 7000 2175 50  0001 C CNN
-F 3 "~" H 7000 2175 50  0001 C CNN
-	1    6800 2175
-	0    1    1    0
-$EndComp
-Wire Wire Line
-	6800 2175 6700 2175
-Wire Wire Line
-	6700 2175 6700 2275
-$Comp
-L Connector:TestPoint TP?
-U 1 1 5DA4623A
-P 6175 2675
-AR Path="/5DA4623A" Ref="TP?"  Part="1"
-AR Path="/61C6D021/5DA4623A" Ref="TP?"  Part="1"
-AR Path="/609E0ED6/5DA4623A" Ref="TP?"  Part="1"
-AR Path="/621F0CB4/5DA4623A" Ref="TP?"  Part="1"
-AR Path="/62A8D0C3/5DA4623A" Ref="TP89"  Part="1"
-F 0 "TP89" H 6125 2925 50  0000 C CNN
-F 1 "TestPoint" H 5925 2725 50  0001 C CNN
-F 2 "custom:TestPoint_THTPad_D1.0mm_Drill0.5mm" H 6375 2675 50  0001 C CNN
-F 3 "~" H 6375 2675 50  0001 C CNN
-	1    6175 2675
-	-1   0    0    1
-$EndComp
-Wire Wire Line
-	6175 2675 6175 2575
-Connection ~ 4525 3200
-Connection ~ 4825 2275
-Wire Wire Line
-	4825 2275 5075 2275
-Connection ~ 6050 1375
-Connection ~ 6050 1875
-Wire Wire Line
-	6050 1875 6050 1975
-Connection ~ 6175 2575
-Wire Wire Line
-	6175 2575 6250 2575
-Connection ~ 6700 2275
-Wire Wire Line
-	6700 2275 6825 2275
-Wire Wire Line
-	4675 2175 4675 2575
-Connection ~ 4675 2575
-Wire Wire Line
-	4675 2575 4825 2575
+Wire Wire Line
+	6050 1775 6050 1975
+Wire Wire Line
+	6550 2275 6825 2275
+Wire Wire Line
+	4425 2575 4825 2575
+Wire Wire Line
+	4525 2275 5075 2275
+Wire Wire Line
+	5725 2575 6250 2575
 $EndSCHEMATC
