File: COLUMN_DRIVERS_1.sch (KiCad schematic (older format))
At the start: 42 parts, among them Q30 DMG6602, Q31 DMG6602, Q32 DMG6602, Q33 SSM3K35AMFV, Q34 SSM3K35AMFV, Q35 SSM3K35AMFV, Q36 SSM3K35AMFV, Q37 SSM3K35AMFV, Q38 SSM3K35AMFV, Q39 DMG6602, Q40 DMG6602, Q41 DMG6602, Q42 SSM3K35AMFV, Q43 SSM3K35AMFV, Q44 SSM3K35AMFV, Q45 SSM3K35AMFV, Q46 SSM3K35AMFV, Q47 SSM3K35AMFV

Commit message: automated commit
Parts:
- renumbered Q30 to Q67, Q31 to Q68, Q32 to Q69, Q33 to Q70, Q34 to Q71, Q35 to Q72, Q36 to Q73, Q37 to Q74, Q38 to Q75, Q39 to Q76, Q40 to Q77, Q41 to Q78, Q42 to Q79, Q43 to Q80, Q44 to Q81, Q45 to Q82, Q46 to Q83, Q47 to Q84, R90 to R163, R91 to R164, R92 to R165, R93 to R166, R94 to R167, R95 to R168, R96 to R169, R97 to R170, R98 to R171, R99 to R172, R100 to R173, R101 to R174, R102 to R175, R103 to R176, R104 to R177, R105 to R178, R106 to R179, R107 to R180, R108 to R181, R109 to R182, R110 to R183, R111 to R184, R112 to R185, R113 to R186

Commit message: automated commit
Parts:
- R163, R164, R165, R166, R167, R168, R169, R170, R171, R172, R173, R174, R175, R176, R177, R178, R179, R180, R181, R182, R183, R184, R185, R186: Resistance 4.7k -> (none); TOLERANCE (none) -> 5%; VALUE (none) -> 4k7

Commit message: automated commit
Parts:
- removed R171, R172, R173, R174, R183, R184, R185, R186: CRG0603F4K7, Resistor_SMD:R_0603_1608Metric, symbol custom:CRG0603F4K7
- added R165, R166, R167, R168, R177, R178, R179, R180: CRG0603F4K7, Resistor_SMD:R_0603_1608Metric, symbol custom:CRG0603F4K7
- renumbered R163 to R159, R164 to R160, R165 to R161, R166 to R162, R167 to R163, R168 to R164, R175 to R171, R176 to R172, R177 to R173, R178 to R174, R179 to R175, R180 to R176
Connections:
- net COL06_OFF: now also R166.1; no longer R170.1
- net COL06_ON: now also R165.1; no longer R169.1
- net COL07_OFF: now also R168.1
- net COL07_ON: now also R167.1
- net COL08_OFF: now also R170.1
- net COL08_ON: now also R169.1
- net COL09_OFF: now also R178.1; no longer R182.1
- net COL09_ON: now also R177.1; no longer R181.1
- net COL10_OFF: now also R180.1
- net COL10_ON: now also R179.1
- net COL11_OFF: now also R182.1
- net COL11_ON: now also R181.1
- net GND: now also R165.2, R166.2, R167.2, R168.2, R177.2, R178.2, R179.2, R180.2

Commit message: automated commit
Parts:
- Q70, Q71, Q72, Q73, Q74, Q75, Q79, Q80, Q81, Q82, Q83, Q84: footprint (none) -> Package_TO_SOT_SMD:SOT-723
Changed lines of the file:
@@
 F 0 "Q73" V 2550 2825 50  0000 L BNN
 F 1 "SSM3K35AMFV" V 2475 2650 50  0000 L BNN
-F 2 "" H 2425 2775 50  0001 L BIN
+F 2 "Package_TO_SOT_SMD:SOT-723" H 2425 2775 50  0001 L BIN
 F 3 "datasheets/SSM3K35AMFV.pdf" H 2425 2750 50  0001 L BNN
 	1    2225 2900
@@
 F 0 "Q70" V 2875 2200 50  0000 L BNN
 F 1 "SSM3K35AMFV" V 2800 2025 50  0000 L BNN
-F 2 "" H 2750 2150 50  0001 L BIN
+F 2 "Package_TO_SOT_SMD:SOT-723" H 2750 2150 50  0001 L BIN
 F 3 "datasheets/SSM3K35AMFV.pdf" H 2750 2125 50  0001 L BNN
 	1    2550 2275
@@
 F 0 "Q74" V 5950 2825 50  0000 L BNN
 F 1 "SSM3K35AMFV" V 5875 2650 50  0000 L BNN
-F 2 "" H 5825 2775 50  0001 L BIN
+F 2 "Package_TO_SOT_SMD:SOT-723" H 5825 2775 50  0001 L BIN
 F 3 "datasheets/SSM3K35AMFV.pdf" H 5825 2750 50  0001 L BNN
 	1    5625 2900
@@
 F 0 "Q71" V 6275 2200 50  0000 L BNN
 F 1 "SSM3K35AMFV" V 6200 2025 50  0000 L BNN
-F 2 "" H 6150 2150 50  0001 L BIN
+F 2 "Package_TO_SOT_SMD:SOT-723" H 6150 2150 50  0001 L BIN
 F 3 "datasheets/SSM3K35AMFV.pdf" H 6150 2125 50  0001 L BNN
 	1    5950 2275
@@
 F 0 "Q75" V 9350 2825 50  0000 L BNN
 F 1 "SSM3K35AMFV" V 9275 2650 50  0000 L BNN
-F 2 "" H 9225 2775 50  0001 L BIN
+F 2 "Package_TO_SOT_SMD:SOT-723" H 9225 2775 50  0001 L BIN
 F 3 "datasheets/SSM3K35AMFV.pdf" H 9225 2750 50  0001 L BNN
 	1    9025 2900
@@
 F 0 "Q72" V 9675 2200 50  0000 L BNN
 F 1 "SSM3K35AMFV" V 9600 2025 50  0000 L BNN
-F 2 "" H 9550 2150 50  0001 L BIN
+F 2 "Package_TO_SOT_SMD:SOT-723" H 9550 2150 50  0001 L BIN
 F 3 "datasheets/SSM3K35AMFV.pdf" H 9550 2125 50  0001 L BNN
 	1    9350 2275
@@
 F 0 "Q82" V 2550 5425 50  0000 L BNN
 F 1 "SSM3K35AMFV" V 2475 5250 50  0000 L BNN
-F 2 "" H 2425 5375 50  0001 L BIN
+F 2 "Package_TO_SOT_SMD:SOT-723" H 2425 5375 50  0001 L BIN
 F 3 "datasheets/SSM3K35AMFV.pdf" H 2425 5350 50  0001 L BNN
 	1    2225 5500
@@
 F 0 "Q79" V 2875 4800 50  0000 L BNN
 F 1 "SSM3K35AMFV" V 2800 4625 50  0000 L BNN
-F 2 "" H 2750 4750 50  0001 L BIN
+F 2 "Package_TO_SOT_SMD:SOT-723" H 2750 4750 50  0001 L BIN
 F 3 "datasheets/SSM3K35AMFV.pdf" H 2750 4725 50  0001 L BNN
 	1    2550 4875
@@
 F 0 "Q83" V 5950 5425 50  0000 L BNN
 F 1 "SSM3K35AMFV" V 5875 5250 50  0000 L BNN
-F 2 "" H 5825 5375 50  0001 L BIN
+F 2 "Package_TO_SOT_SMD:SOT-723" H 5825 5375 50  0001 L BIN
 F 3 "datasheets/SSM3K35AMFV.pdf" H 5825 5350 50  0001 L BNN
 	1    5625 5500
@@
 F 0 "Q80" V 6275 4800 50  0000 L BNN
 F 1 "SSM3K35AMFV" V 6200 4625 50  0000 L BNN
-F 2 "" H 6150 4750 50  0001 L BIN
+F 2 "Package_TO_SOT_SMD:SOT-723" H 6150 4750 50  0001 L BIN
 F 3 "datasheets/SSM3K35AMFV.pdf" H 6150 4725 50  0001 L BNN
 	1    5950 4875
@@
 F 0 "Q84" V 9350 5425 50  0000 L BNN
 F 1 "SSM3K35AMFV" V 9275 5250 50  0000 L BNN
-F 2 "" H 9225 5375 50  0001 L BIN
+F 2 "Package_TO_SOT_SMD:SOT-723" H 9225 5375 50  0001 L BIN
 F 3 "datasheets/SSM3K35AMFV.pdf" H 9225 5350 50  0001 L BNN
 	1    9025 5500
@@
 F 0 "Q81" V 9675 4800 50  0000 L BNN
 F 1 "SSM3K35AMFV" V 9600 4625 50  0000 L BNN
-F 2 "" H 9550 4750 50  0001 L BIN
+F 2 "Package_TO_SOT_SMD:SOT-723" H 9550 4750 50  0001 L BIN
 F 3 "datasheets/SSM3K35AMFV.pdf" H 9550 4725 50  0001 L BNN
 	1    9350 4875

Commit message: automated commit
Parts:
- renumbered R159 to R167, R160 to R168, R161 to R169, R162 to R170, R163 to R171, R164 to R172, R165 to R173, R166 to R174, R167 to R175, R168 to R176, R169 to R177, R170 to R178, R171 to R179, R172 to R180, R173 to R181, R174 to R182, R175 to R183, R176 to R184, R177 to R185, R178 to R186, R179 to R187, R180 to R188, R181 to R189, R182 to R190

Commit message: automated commit
Parts:
- renumbered Q67 to Q66, Q68 to Q67, Q69 to Q68, Q70 to Q69, Q71 to Q70, Q72 to Q71, Q73 to Q72, Q74 to Q73, Q75 to Q74, Q76 to Q75, Q77 to Q76, Q78 to Q77, Q79 to Q78, Q80 to Q79, Q81 to Q80, Q82 to Q81, Q83 to Q82, Q84 to Q83, R167 to R166, R168 to R167, R169 to R168, R170 to R169, R171 to R170, R172 to R171, R173 to R172, R174 to R173, R175 to R174, R176 to R175, R177 to R176, R178 to R177, R179 to R178, R180 to R179, R181 to R180, R182 to R181, R183 to R182, R184 to R183, R185 to R184, R186 to R185, R187 to R186, R188 to R187, R189 to R188, R190 to R189
