File: COLUMN_DRIVERS_2.sch (KiCad schematic (older format))
At the start: 48 parts

Commit message: automated commit
Parts:
- removed Q? (x12): DMG6602, Package_TO_SOT_SMD:TSOT-23-6, symbol custom:DMG6602
- removed Q? (x12): SSM3K35AMFV, symbol custom:SSM3K35AMFV
- removed R? (x24): CRG0603F4K7, Resistor_SMD:R_0603_1608Metric, symbol custom:CRG0603F4K7
- added Q? (x12): DMG6602, Package_TO_SOT_SMD:TSOT-23-6, symbol custom:DMG6602
- added Q? (x12): SSM3K35AMFV, symbol custom:SSM3K35AMFV
- added R? (x24): CRG0603F4K7, Resistor_SMD:R_0603_1608Metric, symbol custom:CRG0603F4K7
Connections:
- net +12V: now also Q?.2 (S), Q?.2 (S), Q?.2 (S), Q?.2 (S), Q?.2 (S), Q?.2 (S), R?.1, R?.1, R?.1, R?.1, R?.1, R?.1
- net GND: now also Q?.2 (S), Q?.2 (S), Q?.2 (S), Q?.2 (S), Q?.2 (S), Q?.2 (S), Q?.2 (S), Q?.2 (S), Q?.2 (S), Q?.2 (S), Q?.2 (S), Q?.2 (S), Q?.5 (S), Q?.5 (S), Q?.5 (S), Q?.5 (S), Q?.5 (S), Q?.5 (S), R?.2, R?.2, R?.2, R?.2, R?.2, R?.2, R?.2, R?.2, R?.2, R?.2, R?.2, R?.2
- new net: Q?.1 (G), Q?.3 (D), R?.1 (x6)
- new net: Q?.3 (D), Q?.3 (G), R?.2 (x6)
- new net COL12: Q?.4 (D), Q?.6 (D)
- new net COL12_OFF: R?.1, R?.2
- new net COL12_ON: Q?.1 (G), Q?.1 (G), R?.1
- new net COL13: Q?.4 (D), Q?.6 (D)
- new net COL13_OFF: R?.1, R?.2
- new net COL13_ON: Q?.1 (G), Q?.1 (G), R?.1
- new net COL14: Q?.4 (D), Q?.6 (D)
- new net COL14_OFF: R?.1, R?.2
- new net COL14_ON: Q?.1 (G), Q?.1 (G), R?.1
- new net COL15: Q?.4 (D), Q?.6 (D)
- new net COL15_OFF: R?.1, R?.2
- new net COL15_ON: Q?.1 (G), Q?.1 (G), R?.1
- new net COL16: Q?.4 (D), Q?.6 (D)
- new net COL16_OFF: R?.1, R?.2
- new net COL16_ON: Q?.1 (G), Q?.1 (G), R?.1
- new net COL17: Q?.4 (D), Q?.6 (D)
- new net COL17_OFF: R?.1, R?.2
- new net COL17_ON: Q?.1 (G), Q?.1 (G), R?.1

Commit message: automated commit
Parts:
- gave numbers to parts that had none: 42
Other:
- moved on the sheet: Q48A, Q48B, Q49A, Q49B, Q50A, Q50B, Q51, Q52, Q53, Q54, Q55, Q56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
