File: COLUMN_DRIVERS_2.sch (KiCad schematic (older format))
At the start: 42 parts, among them Q48 DMG6602, Q49 DMG6602, Q50 DMG6602, Q51 SSM3K35AMFV, Q52 SSM3K35AMFV, Q53 SSM3K35AMFV, Q54 SSM3K35AMFV, Q55 SSM3K35AMFV, Q56 SSM3K35AMFV, Q57 DMG6602, Q58 DMG6602, Q59 DMG6602, Q60 SSM3K35AMFV, Q61 SSM3K35AMFV, Q62 SSM3K35AMFV, Q63 SSM3K35AMFV, Q64 SSM3K35AMFV, Q65 SSM3K35AMFV

Commit message: automated commit
Parts:
- renumbered Q63 to Q100, Q64 to Q101, Q65 to Q102, Q48 to Q85, Q49 to Q86, Q50 to Q87, Q51 to Q88, Q52 to Q89, Q53 to Q90, Q54 to Q91, Q55 to Q92, Q56 to Q93, Q57 to Q94, Q58 to Q95, Q59 to Q96, Q60 to Q97, Q61 to Q98, Q62 to Q99, R114 to R187, R115 to R188, R116 to R189, R117 to R190, R118 to R191, R119 to R192, R120 to R193, R121 to R194, R122 to R195, R123 to R196, R124 to R197, R125 to R198, R126 to R199, R127 to R200, R128 to R201, R129 to R202, R130 to R203, R131 to R204, R132 to R205, R133 to R206, R134 to R207, R135 to R208, R136 to R209, R137 to R210

Commit message: automated commit
Parts:
- R187, R188, R189, R190, R191, R192, R193, R194, R195, R196, R197, R198, R199, R200, R201, R202, R203, R204, R205, R206, R207, R208, R209, R210: Resistance 4.7k -> (none); TOLERANCE (none) -> 5%; VALUE (none) -> 4k7

Commit message: automated commit
Parts:
- removed R195, R196, R197, R198, R207, R208, R209, R210: CRG0603F4K7, Resistor_SMD:R_0603_1608Metric, symbol custom:CRG0603F4K7
- added R189, R190, R191, R192, R201, R202, R203, R204: CRG0603F4K7, Resistor_SMD:R_0603_1608Metric, symbol custom:CRG0603F4K7
- renumbered R187 to R183, R188 to R184, R189 to R185, R190 to R186, R191 to R187, R192 to R188, R199 to R195, R200 to R196, R201 to R197, R202 to R198, R203 to R199, R204 to R200
Connections:
- net COL12_OFF: now also R190.1; no longer R194.1
- net COL12_ON: now also R189.1; no longer R193.1
- net COL13_OFF: now also R192.1
- net COL13_ON: now also R191.1
- net COL14_OFF: now also R194.1
- net COL14_ON: now also R193.1
- net COL15_OFF: now also R202.1; no longer R206.1
- net COL15_ON: now also R201.1; no longer R205.1
- net COL16_OFF: now also R204.1
- net COL16_ON: now also R203.1
- net COL17_OFF: now also R206.1
- net COL17_ON: now also R205.1
- net GND: now also R189.2, R190.2, R191.2, R192.2, R201.2, R202.2, R203.2, R204.2

Commit message: automated commit
Parts:
- Q100, Q101, Q102, Q88, Q89, Q90, Q91, Q92, Q93, Q97, Q98, Q99: footprint (none) -> Package_TO_SOT_SMD:SOT-723
Changed lines of the file:
@@
 F 0 "Q91" V 2550 2825 50  0000 L BNN
 F 1 "SSM3K35AMFV" V 2475 2650 50  0000 L BNN
-F 2 "" H 2425 2775 50  0001 L BIN
+F 2 "Package_TO_SOT_SMD:SOT-723" H 2425 2775 50  0001 L BIN
 F 3 "datasheets/SSM3K35AMFV.pdf" H 2425 2750 50  0001 L BNN
 	1    2225 2900
@@
 F 0 "Q88" V 2875 2200 50  0000 L BNN
 F 1 "SSM3K35AMFV" V 2800 2025 50  0000 L BNN
-F 2 "" H 2750 2150 50  0001 L BIN
+F 2 "Package_TO_SOT_SMD:SOT-723" H 2750 2150 50  0001 L BIN
 F 3 "datasheets/SSM3K35AMFV.pdf" H 2750 2125 50  0001 L BNN
 	1    2550 2275
@@
 F 0 "Q92" V 5950 2825 50  0000 L BNN
 F 1 "SSM3K35AMFV" V 5875 2650 50  0000 L BNN
-F 2 "" H 5825 2775 50  0001 L BIN
+F 2 "Package_TO_SOT_SMD:SOT-723" H 5825 2775 50  0001 L BIN
 F 3 "datasheets/SSM3K35AMFV.pdf" H 5825 2750 50  0001 L BNN
 	1    5625 2900
@@
 F 0 "Q89" V 6275 2200 50  0000 L BNN
 F 1 "SSM3K35AMFV" V 6200 2025 50  0000 L BNN
-F 2 "" H 6150 2150 50  0001 L BIN
+F 2 "Package_TO_SOT_SMD:SOT-723" H 6150 2150 50  0001 L BIN
 F 3 "datasheets/SSM3K35AMFV.pdf" H 6150 2125 50  0001 L BNN
 	1    5950 2275
@@
 F 0 "Q93" V 9350 2825 50  0000 L BNN
 F 1 "SSM3K35AMFV" V 9275 2650 50  0000 L BNN
-F 2 "" H 9225 2775 50  0001 L BIN
+F 2 "Package_TO_SOT_SMD:SOT-723" H 9225 2775 50  0001 L BIN
 F 3 "datasheets/SSM3K35AMFV.pdf" H 9225 2750 50  0001 L BNN
 	1    9025 2900
@@
 F 0 "Q90" V 9675 2200 50  0000 L BNN
 F 1 "SSM3K35AMFV" V 9600 2025 50  0000 L BNN
-F 2 "" H 9550 2150 50  0001 L BIN
+F 2 "Package_TO_SOT_SMD:SOT-723" H 9550 2150 50  0001 L BIN
 F 3 "datasheets/SSM3K35AMFV.pdf" H 9550 2125 50  0001 L BNN
 	1    9350 2275
@@
 F 0 "Q100" V 2550 5425 50  0000 L BNN
 F 1 "SSM3K35AMFV" V 2475 5250 50  0000 L BNN
-F 2 "" H 2425 5375 50  0001 L BIN
+F 2 "Package_TO_SOT_SMD:SOT-723" H 2425 5375 50  0001 L BIN
 F 3 "datasheets/SSM3K35AMFV.pdf" H 2425 5350 50  0001 L BNN
 	1    2225 5500
@@
 F 0 "Q97" V 2875 4800 50  0000 L BNN
 F 1 "SSM3K35AMFV" V 2800 4625 50  0000 L BNN
-F 2 "" H 2750 4750 50  0001 L BIN
+F 2 "Package_TO_SOT_SMD:SOT-723" H 2750 4750 50  0001 L BIN
 F 3 "datasheets/SSM3K35AMFV.pdf" H 2750 4725 50  0001 L BNN
 	1    2550 4875
@@
 F 0 "Q101" V 5950 5425 50  0000 L BNN
 F 1 "SSM3K35AMFV" V 5875 5250 50  0000 L BNN
-F 2 "" H 5825 5375 50  0001 L BIN
+F 2 "Package_TO_SOT_SMD:SOT-723" H 5825 5375 50  0001 L BIN
 F 3 "datasheets/SSM3K35AMFV.pdf" H 5825 5350 50  0001 L BNN
 	1    5625 5500
@@
 F 0 "Q98" V 6275 4800 50  0000 L BNN
 F 1 "SSM3K35AMFV" V 6200 4625 50  0000 L BNN
-F 2 "" H 6150 4750 50  0001 L BIN
+F 2 "Package_TO_SOT_SMD:SOT-723" H 6150 4750 50  0001 L BIN
 F 3 "datasheets/SSM3K35AMFV.pdf" H 6150 4725 50  0001 L BNN
 	1    5950 4875
@@
 F 0 "Q102" V 9350 5425 50  0000 L BNN
 F 1 "SSM3K35AMFV" V 9275 5250 50  0000 L BNN
-F 2 "" H 9225 5375 50  0001 L BIN
+F 2 "Package_TO_SOT_SMD:SOT-723" H 9225 5375 50  0001 L BIN
 F 3 "datasheets/SSM3K35AMFV.pdf" H 9225 5350 50  0001 L BNN
 	1    9025 5500
@@
 F 0 "Q99" V 9675 4800 50  0000 L BNN
 F 1 "SSM3K35AMFV" V 9600 4625 50  0000 L BNN
-F 2 "" H 9550 4750 50  0001 L BIN
+F 2 "Package_TO_SOT_SMD:SOT-723" H 9550 4750 50  0001 L BIN
 F 3 "datasheets/SSM3K35AMFV.pdf" H 9550 4725 50  0001 L BNN
 	1    9350 4875

Commit message: automated commit
Parts:
- renumbered R183 to R191, R184 to R192, R185 to R193, R186 to R194, R187 to R195, R188 to R196, R189 to R197, R190 to R198, R191 to R199, R192 to R200, R193 to R201, R194 to R202, R195 to R203, R196 to R204, R197 to R205, R198 to R206, R199 to R207, R200 to R208, R201 to R209, R202 to R210, R203 to R211, R204 to R212, R205 to R213, R206 to R214

Commit message: automated commit
Parts:
- renumbered Q101 to Q100, Q102 to Q101, Q85 to Q84, Q86 to Q85, Q87 to Q86, Q88 to Q87, Q89 to Q88, Q90 to Q89, Q91 to Q90, Q92 to Q91, Q93 to Q92, Q94 to Q93, Q95 to Q94, Q96 to Q95, Q97 to Q96, Q98 to Q97, Q99 to Q98, Q100 to Q99, R191 to R190, R192 to R191, R193 to R192, R194 to R193, R195 to R194, R196 to R195, R197 to R196, R198 to R197, R199 to R198, R200 to R199, R201 to R200, R202 to R201, R203 to R202, R204 to R203, R205 to R204, R206 to R205, R207 to R206, R208 to R207, R209 to R208, R210 to R209, R211 to R210, R212 to R211, R213 to R212, R214 to R213
