File: COLUMN_DRIVERS_3.sch (KiCad schematic (older format))
At the start: 48 parts

Commit message: automated commit
Parts:
- removed Q? (x12): DMG6602, Package_TO_SOT_SMD:TSOT-23-6, symbol custom:DMG6602
- removed Q? (x12): SSM3K35AMFV, symbol custom:SSM3K35AMFV
- removed R? (x24): CRG0603F4K7, Resistor_SMD:R_0603_1608Metric, symbol custom:CRG0603F4K7
- added Q? (x12): DMG6602, Package_TO_SOT_SMD:TSOT-23-6, symbol custom:DMG6602
- added Q? (x12): SSM3K35AMFV, symbol custom:SSM3K35AMFV
- added R? (x24): CRG0603F4K7, Resistor_SMD:R_0603_1608Metric, symbol custom:CRG0603F4K7
Connections:
- net +12V: now also Q?.2 (S), Q?.2 (S), Q?.2 (S), Q?.2 (S), Q?.2 (S), Q?.2 (S), R?.1, R?.1, R?.1, R?.1, R?.1, R?.1
- net GND: now also Q?.2 (S), Q?.2 (S), Q?.2 (S), Q?.2 (S), Q?.2 (S), Q?.2 (S), Q?.2 (S), Q?.2 (S), Q?.2 (S), Q?.2 (S), Q?.2 (S), Q?.2 (S), Q?.5 (S), Q?.5 (S), Q?.5 (S), Q?.5 (S), Q?.5 (S), Q?.5 (S), R?.2, R?.2, R?.2, R?.2, R?.2, R?.2, R?.2, R?.2, R?.2, R?.2, R?.2, R?.2
- new net: Q?.1 (G), Q?.3 (D), R?.1 (x6)
- new net: Q?.3 (D), Q?.3 (G), R?.2 (x6)
- new net COL18: Q?.4 (D), Q?.6 (D)
- new net COL18_OFF: R?.1, R?.2
- new net COL18_ON: Q?.1 (G), Q?.1 (G), R?.1
- new net COL19: Q?.4 (D), Q?.6 (D)
- new net COL19_OFF: R?.1, R?.2
- new net COL19_ON: Q?.1 (G), Q?.1 (G), R?.1
- new net COL20: Q?.4 (D), Q?.6 (D)
- new net COL20_OFF: R?.1, R?.2
- new net COL20_ON: Q?.1 (G), Q?.1 (G), R?.1
- new net COL21: Q?.4 (D), Q?.6 (D)
- new net COL21_OFF: R?.1, R?.2
- new net COL21_ON: Q?.1 (G), Q?.1 (G), R?.1
- new net COL22: Q?.4 (D), Q?.6 (D)
- new net COL22_OFF: R?.1, R?.2
- new net COL22_ON: Q?.1 (G), Q?.1 (G), R?.1
- new net COL23: Q?.4 (D), Q?.6 (D)
- new net COL23_OFF: R?.1, R?.2
- new net COL23_ON: Q?.1 (G), Q?.1 (G), R?.1

Commit message: automated commit
Parts:
- gave numbers to parts that had none: 42
Other:
- moved on the sheet: Q66A, Q66B, Q67A, Q67B, Q68A, Q68B, Q69, Q70, Q71, Q72, Q73, Q74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
