File: COLUMN_DRIVERS_3.sch (KiCad schematic (older format))
At the start: 42 parts, among them Q66 DMG6602, Q67 DMG6602, Q68 DMG6602, Q69 SSM3K35AMFV, Q70 SSM3K35AMFV, Q71 SSM3K35AMFV, Q72 SSM3K35AMFV, Q73 SSM3K35AMFV, Q74 SSM3K35AMFV, Q75 DMG6602, Q76 DMG6602, Q77 DMG6602, Q78 SSM3K35AMFV, Q79 SSM3K35AMFV, Q80 SSM3K35AMFV, Q81 SSM3K35AMFV, Q82 SSM3K35AMFV, Q83 SSM3K35AMFV

Commit message: automated commit
Parts:
- renumbered Q66 to Q103, Q67 to Q104, Q68 to Q105, Q69 to Q106, Q70 to Q107, Q71 to Q108, Q72 to Q109, Q73 to Q110, Q74 to Q111, Q75 to Q112, Q76 to Q113, Q77 to Q114, Q78 to Q115, Q79 to Q116, Q80 to Q117, Q81 to Q118, Q82 to Q119, Q83 to Q120, R138 to R211, R139 to R212, R140 to R213, R141 to R214, R142 to R215, R143 to R216, R144 to R217, R145 to R218, R146 to R219, R147 to R220, R148 to R221, R149 to R222, R150 to R223, R151 to R224, R152 to R225, R153 to R226, R154 to R227, R155 to R228, R156 to R229, R157 to R230, R158 to R231, R159 to R232, R160 to R233, R161 to R234

Commit message: automated commit
Parts:
- R211, R212, R213, R214, R215, R216, R217, R218, R219, R220, R221, R222, R223, R224, R225, R226, R227, R228, R229, R230, R231, R232, R233, R234: Resistance 4.7k -> (none); TOLERANCE (none) -> 5%; VALUE (none) -> 4k7

Commit message: automated commit
Parts:
- removed R219, R220, R221, R222, R231, R232, R233, R234: CRG0603F4K7, Resistor_SMD:R_0603_1608Metric, symbol custom:CRG0603F4K7
- added R213, R214, R215, R216, R225, R226, R227, R228: CRG0603F4K7, Resistor_SMD:R_0603_1608Metric, symbol custom:CRG0603F4K7
- renumbered R211 to R207, R212 to R208, R213 to R209, R214 to R210, R215 to R211, R216 to R212, R223 to R219, R224 to R220, R225 to R221, R226 to R222, R227 to R223, R228 to R224
Connections:
- net COL18_OFF: now also R214.1; no longer R218.1
- net COL18_ON: now also R213.1; no longer R217.1
- net COL19_OFF: now also R216.1
- net COL19_ON: now also R215.1
- net COL20_OFF: now also R218.1
- net COL20_ON: now also R217.1
- net COL21_OFF: now also R226.1; no longer R230.1
- net COL21_ON: now also R225.1; no longer R229.1
- net COL22_OFF: now also R228.1
- net COL22_ON: now also R227.1
- net COL23_OFF: now also R230.1
- net COL23_ON: now also R229.1
- net GND: now also R213.2, R214.2, R215.2, R216.2, R225.2, R226.2, R227.2, R228.2

Commit message: automated commit
Parts:
- Q106, Q107, Q108, Q109, Q110, Q111, Q115, Q116, Q117, Q118, Q119, Q120: footprint (none) -> Package_TO_SOT_SMD:SOT-723
Changed lines of the file:
@@
 F 0 "Q111" V 9350 2825 50  0000 L BNN
 F 1 "SSM3K35AMFV" V 9275 2650 50  0000 L BNN
-F 2 "" H 9225 2775 50  0001 L BIN
+F 2 "Package_TO_SOT_SMD:SOT-723" H 9225 2775 50  0001 L BIN
 F 3 "datasheets/SSM3K35AMFV.pdf" H 9225 2750 50  0001 L BNN
 	1    9025 2900
@@
 F 0 "Q108" V 9675 2200 50  0000 L BNN
 F 1 "SSM3K35AMFV" V 9600 2025 50  0000 L BNN
-F 2 "" H 9550 2150 50  0001 L BIN
+F 2 "Package_TO_SOT_SMD:SOT-723" H 9550 2150 50  0001 L BIN
 F 3 "datasheets/SSM3K35AMFV.pdf" H 9550 2125 50  0001 L BNN
 	1    9350 2275
@@
 F 0 "Q120" V 9350 5425 50  0000 L BNN
 F 1 "SSM3K35AMFV" V 9275 5250 50  0000 L BNN
-F 2 "" H 9225 5375 50  0001 L BIN
+F 2 "Package_TO_SOT_SMD:SOT-723" H 9225 5375 50  0001 L BIN
 F 3 "datasheets/SSM3K35AMFV.pdf" H 9225 5350 50  0001 L BNN
 	1    9025 5500
@@
 F 0 "Q117" V 9675 4800 50  0000 L BNN
 F 1 "SSM3K35AMFV" V 9600 4625 50  0000 L BNN
-F 2 "" H 9550 4750 50  0001 L BIN
+F 2 "Package_TO_SOT_SMD:SOT-723" H 9550 4750 50  0001 L BIN
 F 3 "datasheets/SSM3K35AMFV.pdf" H 9550 4725 50  0001 L BNN
 	1    9350 4875
@@
 F 0 "Q109" V 2550 2825 50  0000 L BNN
 F 1 "SSM3K35AMFV" V 2475 2650 50  0000 L BNN
-F 2 "" H 2425 2775 50  0001 L BIN
+F 2 "Package_TO_SOT_SMD:SOT-723" H 2425 2775 50  0001 L BIN
 F 3 "datasheets/SSM3K35AMFV.pdf" H 2425 2750 50  0001 L BNN
 	1    2225 2900
@@
 F 0 "Q106" V 2875 2200 50  0000 L BNN
 F 1 "SSM3K35AMFV" V 2800 2025 50  0000 L BNN
-F 2 "" H 2750 2150 50  0001 L BIN
+F 2 "Package_TO_SOT_SMD:SOT-723" H 2750 2150 50  0001 L BIN
 F 3 "datasheets/SSM3K35AMFV.pdf" H 2750 2125 50  0001 L BNN
 	1    2550 2275
@@
 F 0 "Q110" V 5950 2825 50  0000 L BNN
 F 1 "SSM3K35AMFV" V 5875 2650 50  0000 L BNN
-F 2 "" H 5825 2775 50  0001 L BIN
+F 2 "Package_TO_SOT_SMD:SOT-723" H 5825 2775 50  0001 L BIN
 F 3 "datasheets/SSM3K35AMFV.pdf" H 5825 2750 50  0001 L BNN
 	1    5625 2900
@@
 F 0 "Q107" V 6275 2200 50  0000 L BNN
 F 1 "SSM3K35AMFV" V 6200 2025 50  0000 L BNN
-F 2 "" H 6150 2150 50  0001 L BIN
+F 2 "Package_TO_SOT_SMD:SOT-723" H 6150 2150 50  0001 L BIN
 F 3 "datasheets/SSM3K35AMFV.pdf" H 6150 2125 50  0001 L BNN
 	1    5950 2275
@@
 F 0 "Q118" V 2550 5425 50  0000 L BNN
 F 1 "SSM3K35AMFV" V 2475 5250 50  0000 L BNN
-F 2 "" H 2425 5375 50  0001 L BIN
+F 2 "Package_TO_SOT_SMD:SOT-723" H 2425 5375 50  0001 L BIN
 F 3 "datasheets/SSM3K35AMFV.pdf" H 2425 5350 50  0001 L BNN
 	1    2225 5500
@@
 F 0 "Q115" V 2875 4800 50  0000 L BNN
 F 1 "SSM3K35AMFV" V 2800 4625 50  0000 L BNN
-F 2 "" H 2750 4750 50  0001 L BIN
+F 2 "Package_TO_SOT_SMD:SOT-723" H 2750 4750 50  0001 L BIN
 F 3 "datasheets/SSM3K35AMFV.pdf" H 2750 4725 50  0001 L BNN
 	1    2550 4875
@@
 F 0 "Q119" V 5950 5425 50  0000 L BNN
 F 1 "SSM3K35AMFV" V 5875 5250 50  0000 L BNN
-F 2 "" H 5825 5375 50  0001 L BIN
+F 2 "Package_TO_SOT_SMD:SOT-723" H 5825 5375 50  0001 L BIN
 F 3 "datasheets/SSM3K35AMFV.pdf" H 5825 5350 50  0001 L BNN
 	1    5625 5500
@@
 F 0 "Q116" V 6275 4800 50  0000 L BNN
 F 1 "SSM3K35AMFV" V 6200 4625 50  0000 L BNN
-F 2 "" H 6150 4750 50  0001 L BIN
+F 2 "Package_TO_SOT_SMD:SOT-723" H 6150 4750 50  0001 L BIN
 F 3 "datasheets/SSM3K35AMFV.pdf" H 6150 4725 50  0001 L BNN
 	1    5950 4875

Commit message: automated commit
Parts:
- renumbered R207 to R215, R208 to R216, R209 to R217, R210 to R218, R211 to R219, R212 to R220, R213 to R221, R214 to R222, R215 to R223, R216 to R224, R217 to R225, R218 to R226, R219 to R227, R220 to R228, R221 to R229, R222 to R230, R223 to R231, R224 to R232, R225 to R233, R226 to R234, R227 to R235, R228 to R236, R229 to R237, R230 to R238

Commit message: automated commit
Parts:
- renumbered Q103 to Q102, Q104 to Q103, Q105 to Q104, Q106 to Q105, Q107 to Q106, Q108 to Q107, Q109 to Q108, Q110 to Q109, Q111 to Q110, Q112 to Q111, Q113 to Q112, Q114 to Q113, Q115 to Q114, Q116 to Q115, Q117 to Q116, Q118 to Q117, Q119 to Q118, Q120 to Q119, R215 to R214, R216 to R215, R217 to R216, R218 to R217, R219 to R218, R220 to R219, R221 to R220, R222 to R221, R223 to R222, R224 to R223, R225 to R224, R226 to R225, R227 to R226, R228 to R227, R229 to R228, R230 to R229, R231 to R230, R232 to R231, R233 to R232, R234 to R233, R235 to R234, R236 to R235, R237 to R236, R238 to R237
