File: COLUMN_DRIVERS_4.sch (KiCad schematic (older format))
At the start: 32 parts

Commit message: automated commit
Parts:
- removed Q? (x8): DMG6602, Package_TO_SOT_SMD:TSOT-23-6, symbol custom:DMG6602
- removed Q? (x8): SSM3K35AMFV, symbol custom:SSM3K35AMFV
- removed R? (x16): CRG0603F4K7, Resistor_SMD:R_0603_1608Metric, symbol custom:CRG0603F4K7
- added Q? (x8): DMG6602, Package_TO_SOT_SMD:TSOT-23-6, symbol custom:DMG6602
- added Q? (x8): SSM3K35AMFV, symbol custom:SSM3K35AMFV
- added R? (x16): CRG0603F4K7, Resistor_SMD:R_0603_1608Metric, symbol custom:CRG0603F4K7
Connections:
- net +12V: now also Q?.2 (S), Q?.2 (S), Q?.2 (S), Q?.2 (S), R?.1, R?.1, R?.1, R?.1
- net GND: now also Q?.2 (S), Q?.2 (S), Q?.2 (S), Q?.2 (S), Q?.2 (S), Q?.2 (S), Q?.2 (S), Q?.2 (S), Q?.5 (S), Q?.5 (S), Q?.5 (S), Q?.5 (S), R?.2, R?.2, R?.2, R?.2, R?.2, R?.2, R?.2, R?.2
- new net: Q?.1 (G), Q?.3 (D), R?.1 (x4)
- new net: Q?.3 (D), Q?.3 (G), R?.2 (x4)
- new net COL24: Q?.4 (D), Q?.6 (D)
- new net COL24_OFF: R?.1, R?.2
- new net COL24_ON: Q?.1 (G), Q?.1 (G), R?.1
- new net COL25: Q?.4 (D), Q?.6 (D)
- new net COL25_OFF: R?.1, R?.2
- new net COL25_ON: Q?.1 (G), Q?.1 (G), R?.1
- new net COL26: Q?.4 (D), Q?.6 (D)
- new net COL26_OFF: R?.1, R?.2
- new net COL26_ON: Q?.1 (G), Q?.1 (G), R?.1
- new net COL27: Q?.4 (D), Q?.6 (D)
- new net COL27_OFF: R?.1, R?.2
- new net COL27_ON: Q?.1 (G), Q?.1 (G), R?.1

Commit message: automated commit
Parts:
- gave numbers to parts that had none: 28
Other:
- moved on the sheet: Q84A, Q84B, Q85A, Q85B, Q86A, Q86B, Q87, Q88, Q89, Q90, Q91, Q92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
