File: COLUMN_DRIVERS_4.sch (KiCad schematic (older format))
At the start: 28 parts, among them Q84 DMG6602, Q85 DMG6602, Q86 DMG6602, Q87 SSM3K35AMFV, Q88 SSM3K35AMFV, Q89 SSM3K35AMFV, Q90 SSM3K35AMFV, Q91 SSM3K35AMFV, Q92 SSM3K35AMFV, Q93 DMG6602, Q94 SSM3K35AMFV, Q95 SSM3K35AMFV

Commit message: automated commit
Parts:
- renumbered Q84 to Q121, Q85 to Q122, Q86 to Q123, Q87 to Q124, Q88 to Q125, Q89 to Q126, Q90 to Q127, Q91 to Q128, Q92 to Q129, Q93 to Q130, Q94 to Q131, Q95 to Q132, R162 to R235, R163 to R236, R164 to R237, R165 to R238, R166 to R239, R167 to R240, R168 to R241, R169 to R242, R170 to R243, R171 to R244, R172 to R245, R173 to R246, R174 to R247, R175 to R248, R176 to R249, R177 to R250

Commit message: automated commit
Parts:
- R235, R236, R237, R238, R239, R240, R241, R242, R243, R244, R245, R246, R247, R248, R249, R250: Resistance 4.7k -> (none); TOLERANCE (none) -> 5%; VALUE (none) -> 4k7

Commit message: automated commit
Parts:
- removed R243, R244, R249, R250: CRG0603F4K7, Resistor_SMD:R_0603_1608Metric, symbol custom:CRG0603F4K7
- added R237, R238, R239, R240: CRG0603F4K7, Resistor_SMD:R_0603_1608Metric, symbol custom:CRG0603F4K7
- renumbered R235 to R231, R236 to R232, R237 to R233, R238 to R234, R239 to R235, R240 to R236, R247 to R243, R248 to R244
Connections:
- net COL24_OFF: now also R238.1; no longer R242.1
- net COL24_ON: now also R237.1; no longer R241.1
- net COL25_OFF: now also R240.1
- net COL25_ON: now also R239.1
- net COL26_OFF: now also R242.1; no longer R246.1
- net COL26_ON: now also R241.1; no longer R245.1
- net COL27_OFF: now also R246.1
- net COL27_ON: now also R245.1
- net GND: now also R237.2, R238.2, R239.2, R240.2

Commit message: automated commit
Parts:
- Q124, Q125, Q126, Q127, Q128, Q129, Q131, Q132: footprint (none) -> Package_TO_SOT_SMD:SOT-723
Changed lines of the file:
@@
 F 0 "Q127" V 2550 2825 50  0000 L BNN
 F 1 "SSM3K35AMFV" V 2475 2650 50  0000 L BNN
-F 2 "" H 2425 2775 50  0001 L BIN
+F 2 "Package_TO_SOT_SMD:SOT-723" H 2425 2775 50  0001 L BIN
 F 3 "datasheets/SSM3K35AMFV.pdf" H 2425 2750 50  0001 L BNN
 	1    2225 2900
@@
 F 0 "Q124" V 2875 2200 50  0000 L BNN
 F 1 "SSM3K35AMFV" V 2800 2025 50  0000 L BNN
-F 2 "" H 2750 2150 50  0001 L BIN
+F 2 "Package_TO_SOT_SMD:SOT-723" H 2750 2150 50  0001 L BIN
 F 3 "datasheets/SSM3K35AMFV.pdf" H 2750 2125 50  0001 L BNN
 	1    2550 2275
@@
 F 0 "Q128" V 5950 2825 50  0000 L BNN
 F 1 "SSM3K35AMFV" V 5875 2650 50  0000 L BNN
-F 2 "" H 5825 2775 50  0001 L BIN
+F 2 "Package_TO_SOT_SMD:SOT-723" H 5825 2775 50  0001 L BIN
 F 3 "datasheets/SSM3K35AMFV.pdf" H 5825 2750 50  0001 L BNN
 	1    5625 2900
@@
 F 0 "Q125" V 6275 2200 50  0000 L BNN
 F 1 "SSM3K35AMFV" V 6200 2025 50  0000 L BNN
-F 2 "" H 6150 2150 50  0001 L BIN
+F 2 "Package_TO_SOT_SMD:SOT-723" H 6150 2150 50  0001 L BIN
 F 3 "datasheets/SSM3K35AMFV.pdf" H 6150 2125 50  0001 L BNN
 	1    5950 2275
@@
 F 0 "Q129" V 9350 2825 50  0000 L BNN
 F 1 "SSM3K35AMFV" V 9275 2650 50  0000 L BNN
-F 2 "" H 9225 2775 50  0001 L BIN
+F 2 "Package_TO_SOT_SMD:SOT-723" H 9225 2775 50  0001 L BIN
 F 3 "datasheets/SSM3K35AMFV.pdf" H 9225 2750 50  0001 L BNN
 	1    9025 2900
@@
 F 0 "Q126" V 9675 2200 50  0000 L BNN
 F 1 "SSM3K35AMFV" V 9600 2025 50  0000 L BNN
-F 2 "" H 9550 2150 50  0001 L BIN
+F 2 "Package_TO_SOT_SMD:SOT-723" H 9550 2150 50  0001 L BIN
 F 3 "datasheets/SSM3K35AMFV.pdf" H 9550 2125 50  0001 L BNN
 	1    9350 2275
@@
 F 0 "Q132" V 2550 5425 50  0000 L BNN
 F 1 "SSM3K35AMFV" V 2475 5250 50  0000 L BNN
-F 2 "" H 2425 5375 50  0001 L BIN
+F 2 "Package_TO_SOT_SMD:SOT-723" H 2425 5375 50  0001 L BIN
 F 3 "datasheets/SSM3K35AMFV.pdf" H 2425 5350 50  0001 L BNN
 	1    2225 5500
@@
 F 0 "Q131" V 2875 4800 50  0000 L BNN
 F 1 "SSM3K35AMFV" V 2800 4625 50  0000 L BNN
-F 2 "" H 2750 4750 50  0001 L BIN
+F 2 "Package_TO_SOT_SMD:SOT-723" H 2750 4750 50  0001 L BIN
 F 3 "datasheets/SSM3K35AMFV.pdf" H 2750 4725 50  0001 L BNN
 	1    2550 4875

Commit message: automated commit
Parts:
- renumbered R231 to R239, R232 to R240, R233 to R241, R234 to R242, R235 to R243, R236 to R244, R237 to R245, R238 to R246, R239 to R247, R240 to R248, R241 to R249, R242 to R250, R243 to R251, R244 to R252, R245 to R253, R246 to R254
Changed lines of the file:
@@
 AR Path="/5D79BBAA" Ref="#PWR?"  Part="1"
 AR Path="/62A8D0C3/5D79BBAA" Ref="#PWR?"  Part="1"
-AR Path="/62C1C003/5D79BBAA" Ref="#PWR0264"  Part="1"
-F 0 "#PWR0264" H 3150 1175 50  0001 C CNN
+AR Path="/62C1C003/5D79BBAA" Ref="#PWR0266"  Part="1"
+F 0 "#PWR0266" H 3150 1175 50  0001 C CNN
 F 1 "+12V" H 3150 1465 50  0000 C CNN
 F 2 "" H 3150 1325 50  0001 C CNN
@@
 AR Path="/5D79BBD0" Ref="#PWR?"  Part="1"
 AR Path="/62A8D0C3/5D79BBD0" Ref="#PWR?"  Part="1"
-AR Path="/62C1C003/5D79BBD0" Ref="#PWR0267"  Part="1"
-F 0 "#PWR0267" H 3150 3000 50  0001 C CNN
+AR Path="/62C1C003/5D79BBD0" Ref="#PWR0269"  Part="1"
+F 0 "#PWR0269" H 3150 3000 50  0001 C CNN
 F 1 "GND" H 3150 3100 50  0000 C CNN
 F 2 "" H 3150 3250 50  0001 C CNN
@@
 AR Path="/5D79BC15" Ref="#PWR?"  Part="1"
 AR Path="/62A8D0C3/5D79BC15" Ref="#PWR?"  Part="1"
-AR Path="/62C1C003/5D79BC15" Ref="#PWR0265"  Part="1"
-F 0 "#PWR0265" H 6550 1175 50  0001 C CNN
+AR Path="/62C1C003/5D79BC15" Ref="#PWR0267"  Part="1"
+F 0 "#PWR0267" H 6550 1175 50  0001 C CNN
 F 1 "+12V" H 6550 1465 50  0000 C CNN
 F 2 "" H 6550 1325 50  0001 C CNN
@@
 AR Path="/5D79BC37" Ref="#PWR?"  Part="1"
 AR Path="/62A8D0C3/5D79BC37" Ref="#PWR?"  Part="1"
-AR Path="/62C1C003/5D79BC37" Ref="#PWR0268"  Part="1"
-F 0 "#PWR0268" H 6550 3000 50  0001 C CNN
+AR Path="/62C1C003/5D79BC37" Ref="#PWR0270"  Part="1"
+F 0 "#PWR0270" H 6550 3000 50  0001 C CNN
 F 1 "GND" H 6550 3100 50  0000 C CNN
 F 2 "" H 6550 3250 50  0001 C CNN
@@
 AR Path="/5D79BC78" Ref="#PWR?"  Part="1"
 AR Path="/62A8D0C3/5D79BC78" Ref="#PWR?"  Part="1"
-AR Path="/62C1C003/5D79BC78" Ref="#PWR0266"  Part="1"
-F 0 "#PWR0266" H 9950 1175 50  0001 C CNN
+AR Path="/62C1C003/5D79BC78" Ref="#PWR0268"  Part="1"
+F 0 "#PWR0268" H 9950 1175 50  0001 C CNN
 F 1 "+12V" H 9950 1465 50  0000 C CNN
 F 2 "" H 9950 1325 50  0001 C CNN
@@
 AR Path="/5D79BC9A" Ref="#PWR?"  Part="1"
 AR Path="/62A8D0C3/5D79BC9A" Ref="#PWR?"  Part="1"
-AR Path="/62C1C003/5D79BC9A" Ref="#PWR0269"  Part="1"
-F 0 "#PWR0269" H 9950 3000 50  0001 C CNN
+AR Path="/62C1C003/5D79BC9A" Ref="#PWR0271"  Part="1"
+F 0 "#PWR0271" H 9950 3000 50  0001 C CNN
 F 1 "GND" H 9950 3100 50  0000 C CNN
 F 2 "" H 9950 3250 50  0001 C CNN
@@
 AR Path="/5D79BCDB" Ref="#PWR?"  Part="1"
 AR Path="/62A8D0C3/5D79BCDB" Ref="#PWR?"  Part="1"
-AR Path="/62C1C003/5D79BCDB" Ref="#PWR0270"  Part="1"
-F 0 "#PWR0270" H 3150 3775 50  0001 C CNN
+AR Path="/62C1C003/5D79BCDB" Ref="#PWR0272"  Part="1"
+F 0 "#PWR0272" H 3150 3775 50  0001 C CNN
 F 1 "+12V" H 3150 4065 50  0000 C CNN
 F 2 "" H 3150 3925 50  0001 C CNN
@@
 AR Path="/5D79BCFD" Ref="#PWR?"  Part="1"
 AR Path="/62A8D0C3/5D79BCFD" Ref="#PWR?"  Part="1"
-AR Path="/62C1C003/5D79BCFD" Ref="#PWR0271"  Part="1"
-F 0 "#PWR0271" H 3150 5600 50  0001 C CNN
+AR Path="/62C1C003/5D79BCFD" Ref="#PWR0273"  Part="1"
+F 0 "#PWR0273" H 3150 5600 50  0001 C CNN
 F 1 "GND" H 3150 5700 50  0000 C CNN
 F 2 "" H 3150 5850 50  0001 C CNN
@@
 AR Path="/62A8D0C3/5D128832" Ref="R?"  Part="1"
 AR Path="/62C1BAEB/5D128832" Ref="R?"  Part="1"
-AR Path="/62C1C003/5D128832" Ref="R234"  Part="1"
-F 0 "R234" V 1950 2700 50  0000 L BNN
+AR Path="/62C1C003/5D128832" Ref="R242"  Part="1"
+F 0 "R242" V 1950 2700 50  0000 L BNN
 F 1 "CRG0603F4K7" H 1275 2175 50  0001 L BNN
 F 2 "Resistor_SMD:R_0603_1608Metric" H 1275 2075 50  0001 L BNN
@@
 AR Path="/62A8D0C3/5D12883A" Ref="R?"  Part="1"
 AR Path="/62C1BAEB/5D12883A" Ref="R?"  Part="1"
-AR Path="/62C1C003/5D12883A" Ref="R231"  Part="1"
-F 0 "R231" H 2720 1645 50  0000 L BNN
+AR Path="/62C1C003/5D12883A" Ref="R239"  Part="1"
+F 0 "R239" H 2720 1645 50  0000 L BNN
 F 1 "CRG0603F4K7" H 1950 1225 50  0001 L BNN
 F 2 "Resistor_SMD:R_0603_1608Metric" H 1950 1125 50  0001 L BNN
@@
 AR Path="/62A8D0C3/5D12D2AE" Ref="R?"  Part="1"
 AR Path="/62C1BAEB/5D12D2AE" Ref="R?"  Part="1"
-AR Path="/62C1C003/5D12D2AE" Ref="R235"  Part="1"
-F 0 "R235" V 5350 2700 50  0000 L BNN
+AR Path="/62C1C003/5D12D2AE" Ref="R243"  Part="1"
+F 0 "R243" V 5350 2700 50  0000 L BNN
 F 1 "CRG0603F4K7" H 4675 2175 50  0001 L BNN
 F 2 "Resistor_SMD:R_0603_1608Metric" H 4675 2075 50  0001 L BNN
@@
 AR Path="/62A8D0C3/5D12D2B6" Ref="R?"  Part="1"
 AR Path="/62C1BAEB/5D12D2B6" Ref="R?"  Part="1"
-AR Path="/62C1C003/5D12D2B6" Ref="R232"  Part="1"
-F 0 "R232" H 6120 1645 50  0000 L BNN
+AR Path="/62C1C003/5D12D2B6" Ref="R240"  Part="1"
+F 0 "R240" H 6120 1645 50  0000 L BNN
 F 1 "CRG0603F4K7" H 5350 1225 50  0001 L BNN
 F 2 "Resistor_SMD:R_0603_1608Metric" H 5350 1125 50  0001 L BNN
@@
 AR Path="/62A8D0C3/5D1323C4" Ref="R?"  Part="1"
 AR Path="/62C1BAEB/5D1323C4" Ref="R?"  Part="1"
-AR Path="/62C1C003/5D1323C4" Ref="R236"  Part="1"
-F 0 "R236" V 8750 2700 50  0000 L BNN
+AR Path="/62C1C003/5D1323C4" Ref="R244"  Part="1"
+F 0 "R244" V 8750 2700 50  0000 L BNN
 F 1 "CRG0603F4K7" H 8075 2175 50  0001 L BNN
 F 2 "Resistor_SMD:R_0603_1608Metric" H 8075 2075 50  0001 L BNN
@@
 AR Path="/62A8D0C3/5D1323CC" Ref="R?"  Part="1"
 AR Path="/62C1BAEB/5D1323CC" Ref="R?"  Part="1"
-AR Path="/62C1C003/5D1323CC" Ref="R233"  Part="1"
-F 0 "R233" H 9520 1645 50  0000 L BNN
+AR Path="/62C1C003/5D1323CC" Ref="R241"  Part="1"
+F 0 "R241" H 9520 1645 50  0000 L BNN
 F 1 "CRG0603F4K7" H 8750 1225 50  0001 L BNN
 F 2 "Resistor_SMD:R_0603_1608Metric" H 8750 1125 50  0001 L BNN
@@
 AR Path="/62A8D0C3/5D137A54" Ref="R?"  Part="1"
 AR Path="/62C1BAEB/5D137A54" Ref="R?"  Part="1"
-AR Path="/62C1C003/5D137A54" Ref="R244"  Part="1"
-F 0 "R244" V 1950 5300 50  0000 L BNN
+AR Path="/62C1C003/5D137A54" Ref="R252"  Part="1"
+F 0 "R252" V 1950 5300 50  0000 L BNN
 F 1 "CRG0603F4K7" H 1275 4775 50  0001 L BNN
 F 2 "Resistor_SMD:R_0603_1608Metric" H 1275 4675 50  0001 L BNN
@@
 AR Path="/62A8D0C3/5D137A5C" Ref="R?"  Part="1"
 AR Path="/62C1BAEB/5D137A5C" Ref="R?"  Part="1"
-AR Path="/62C1C003/5D137A5C" Ref="R243"  Part="1"
-F 0 "R243" H 2720 4245 50  0000 L BNN
+AR Path="/62C1C003/5D137A5C" Ref="R251"  Part="1"
+F 0 "R251" H 2720 4245 50  0000 L BNN
 F 1 "CRG0603F4K7" H 1950 3825 50  0001 L BNN
 F 2 "Resistor_SMD:R_0603_1608Metric" H 1950 3725 50  0001 L BNN
@@
 P 1125 2825
 AR Path="/62A8D0C3/5D362D02" Ref="R?"  Part="1"
-AR Path="/62C1C003/5D362D02" Ref="R237"  Part="1"
-F 0 "R237" V 1100 2500 50  0000 L BNN
+AR Path="/62C1C003/5D362D02" Ref="R245"  Part="1"
+F 0 "R245" V 1100 2500 50  0000 L BNN
 F 1 "CRG0603F4K7" H 425 2425 50  0001 L BNN
 F 2 "Resistor_SMD:R_0603_1608Metric" H 425 2325 50  0001 L BNN
@@
 P 1425 2825
 AR Path="/62A8D0C3/5D362D0A" Ref="R?"  Part="1"
-AR Path="/62C1C003/5D362D0A" Ref="R238"  Part="1"
-F 0 "R238" V 1400 2500 50  0000 L BNN
+AR Path="/62C1C003/5D362D0A" Ref="R246"  Part="1"
+F 0 "R246" V 1400 2500 50  0000 L BNN
 F 1 "CRG0603F4K7" H 725 2425 50  0001 L BNN
 F 2 "Resistor_SMD:R_0603_1608Metric" H 725 2325 50  0001 L BNN
@@
 P 4525 2825
 AR Path="/62A8D0C3/5D362D12" Ref="R?"  Part="1"
-AR Path="/62C1C003/5D362D12" Ref="R239"  Part="1"
-F 0 "R239" V 4500 2500 50  0000 L BNN
+AR Path="/62C1C003/5D362D12" Ref="R247"  Part="1"
+F 0 "R247" V 4500 2500 50  0000 L BNN
 F 1 "CRG0603F4K7" H 3825 2425 50  0001 L BNN
 F 2 "Resistor_SMD:R_0603_1608Metric" H 3825 2325 50  0001 L BNN
@@
 P 4825 2825
 AR Path="/62A8D0C3/5D362D1A" Ref="R?"  Part="1"
-AR Path="/62C1C003/5D362D1A" Ref="R240"  Part="1"
-F 0 "R240" V 4800 2500 50  0000 L BNN
+AR Path="/62C1C003/5D362D1A" Ref="R248"  Part="1"
+F 0 "R248" V 4800 2500 50  0000 L BNN
 F 1 "CRG0603F4K7" H 4125 2425 50  0001 L BNN
 F 2 "Resistor_SMD:R_0603_1608Metric" H 4125 2325 50  0001 L BNN
@@
 P 7925 2825
 AR Path="/62A8D0C3/5D362D22" Ref="R?"  Part="1"
-AR Path="/62C1C003/5D362D22" Ref="R241"  Part="1"
-F 0 "R241" V 7900 2500 50  0000 L BNN
+AR Path="/62C1C003/5D362D22" Ref="R249"  Part="1"
+F 0 "R249" V 7900 2500 50  0000 L BNN
 F 1 "CRG0603F4K7" H 7225 2425 50  0001 L BNN
 F 2 "Resistor_SMD:R_0603_1608Metric" H 7225 2325 50  0001 L BNN
@@
 P 8225 2825
 AR Path="/62A8D0C3/5D362D2A" Ref="R?"  Part="1"
-AR Path="/62C1C003/5D362D2A" Ref="R242"  Part="1"
-F 0 "R242" V 8200 2500 50  0000 L BNN
+AR Path="/62C1C003/5D362D2A" Ref="R250"  Part="1"
+F 0 "R250" V 8200 2500 50  0000 L BNN
 F 1 "CRG0603F4K7" H 7525 2425 50  0001 L BNN
 F 2 "Resistor_SMD:R_0603_1608Metric" H 7525 2325 50  0001 L BNN
@@
 P 1125 5425
 AR Path="/62A8D0C3/5D362D32" Ref="R?"  Part="1"
-AR Path="/62C1C003/5D362D32" Ref="R245"  Part="1"
-F 0 "R245" V 1100 5100 50  0000 L BNN
+AR Path="/62C1C003/5D362D32" Ref="R253"  Part="1"
+F 0 "R253" V 1100 5100 50  0000 L BNN
 F 1 "CRG0603F4K7" H 425 5025 50  0001 L BNN
 F 2 "Resistor_SMD:R_0603_1608Metric" H 425 4925 50  0001 L BNN
@@
 P 1425 5425
 AR Path="/62A8D0C3/5D362D3A" Ref="R?"  Part="1"
-AR Path="/62C1C003/5D362D3A" Ref="R246"  Part="1"
-F 0 "R246" V 1400 5100 50  0000 L BNN
+AR Path="/62C1C003/5D362D3A" Ref="R254"  Part="1"
+F 0 "R254" V 1400 5100 50  0000 L BNN
 F 1 "CRG0603F4K7" H 725 5025 50  0001 L BNN
 F 2 "Resistor_SMD:R_0603_1608Metric" H 725 4925 50  0001 L BNN

Commit message: automated commit
Parts:
- renumbered Q121 to Q120, Q122 to Q121, Q123 to Q122, Q124 to Q123, Q125 to Q124, Q126 to Q125, Q127 to Q126, Q128 to Q127, Q129 to Q128, Q130 to Q129, Q131 to Q130, Q132 to Q131, R239 to R238, R240 to R239, R241 to R240, R242 to R241, R243 to R242, R244 to R243, R245 to R244, R246 to R245, R247 to R246, R248 to R247, R249 to R248, R250 to R249, R251 to R250, R252 to R251, R253 to R252, R254 to R253
