File: FE310.sch (KiCad schematic (older format))
At the start: 26 parts

Commit message: automated commit
Parts:
- added C? (x11): CL10B104KO8NNNC, Capacitor_SMD:C_0603_1608Metric, symbol custom:CL10B104KO8NNNC
- added C? (x6): CL10B105KA8NNNC, Capacitor_SMD:C_0603_1608Metric, symbol custom:CL10B105KA8NNNC
- gave numbers to parts that had none: 26
Connections:
- net AON_VDD_FE310 is gone; now on net +1V8: U13.19 (AON_IVDD), U13.23 (AON_VDD)
- net IVDD_FE310 is gone; now on net +3V3: U13.11 (IVDD), U13.32 (IVDD), U13.47 (IVDD)
- net OTP_AIVDD_FE310 is gone; now on net +3V3: U13.12 (OTP_AIVDD)
- net PLL_AVDD_FE310 is gone; now on net +1V8: U13.7 (PLL_AVDD)
- net VDD_FE310 is gone; now on net +1V8: U13.30 (VDD), U13.46 (VDD), U13.6 (VDD)
- net +1V8: now also C?.1, C?.1, C?.1, C?.1, C?.1, C?.1, C?.1, C?.1, C?.1, C?.1, C?.1
- net +3V3: now also C?.1, C?.1, C?.1, C?.1, C?.1, C?.1
- net GND: now also C?.2, C?.2, C?.2, C?.2, C?.2, C?.2, C?.2, C?.2, C?.2, C?.2, C?.2, C?.2, C?.2, C?.2, C?.2
- net PLL_AVSS_FE310: now also C?.2, C?.2
Other:
- moved on the sheet: BZ1, BZ2, C63, C64, C70, C71, D10, D11, D12, Q43, Q44, R56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

Commit message: automated commit
Parts:
- added TP? (x2): TestPoint, symbol Connector:TestPoint
Connections:
- net !WAKEUP: now also TP?.1
Changed lines of the file:
@@
 $Descr A4 11693 8268
 encoding utf-8
-Sheet 2 19
+Sheet 2 20
 Title ""
 Date ""
@@
 Connection ~ 7875 3225
 Wire Wire Line
-	9925 3225 10150 3225
-Wire Wire Line
 	8025 4125 7125 4125
 Wire Wire Line
@@
 Text GLabel 10150 2825 2    50   Input ~ 0
 IVDD_FE310
-Text GLabel 10150 3225 2    50   Input ~ 0
-OTP_AIVDD_FE310
 Text GLabel 10150 3625 2    50   Output ~ 0
 !ROW_RESET
@@
 	1    0    0    -1
 $EndComp
+Text Label 10825 3225 2    60   ~ 0
+OTP_AIVDD_FE310
+Wire Wire Line
+	9925 3225 10825 3225
+Wire Wire Line
+	6825 2300 6825 2375
+$Comp
+L Connector:TestPoint TP?
+U 1 1 5D072151
+P 6825 2300
+AR Path="/5D072151" Ref="TP?"  Part="1"
+AR Path="/61C6D021/5D072151" Ref="TP?"  Part="1"
+AR Path="/64D8274A/5D072151" Ref="TP?"  Part="1"
+F 0 "TP?" H 6775 2525 50  0000 C CNN
+F 1 "TestPoint" H 6575 2350 50  0001 C CNN
+F 2 "" H 7025 2300 50  0001 C CNN
+F 3 "~" H 7025 2300 50  0001 C CNN
+	1    6825 2300
+	1    0    0    -1
+$EndComp
+Connection ~ 6825 2375
+Wire Wire Line
+	5950 3850 5950 3925
+$Comp
+L Connector:TestPoint TP?
+U 1 1 5D0847E2
+P 5950 3850
+AR Path="/5D0847E2" Ref="TP?"  Part="1"
+AR Path="/61C6D021/5D0847E2" Ref="TP?"  Part="1"
+AR Path="/64D8274A/5D0847E2" Ref="TP?"  Part="1"
+F 0 "TP?" H 5900 4075 50  0000 C CNN
+F 1 "TestPoint" H 5700 3900 50  0001 C CNN
+F 2 "" H 6150 3850 50  0001 C CNN
+F 3 "~" H 6150 3850 50  0001 C CNN
+	1    5950 3850
+	1    0    0    -1
+$EndComp

Commit message: automated commit
Parts:
- gave numbers to parts that had none: 19
- renumbered C63 to C12, C64 to C13, C70 to C16, C71 to C17, D10 to D1, D11 to D2, D12 to D3, Q43 to Q1, Q44 to Q2, R57 to R1, R66 to R10, R59 to R2, R60 to R3, R61 to R4, R56 to R5, R58 to R6, R62 to R7, R63 to R8, R64 to R9, U13 to U1, U17 to U2, Y2 to Y1
Connections:
- net !RESET: now also TP2.1
Other:
- moved on the sheet: BZ1, BZ2, C1, C10, C11, C12, C13, C14, C15, C16, C17, C18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
