File: FE310.sch (KiCad schematic (older format))
At the start: 45 parts, among them Q1 SSM3K35AMFV, Q2 SSM3K35AMFV, SW1 NP_TACTILE_SWITCH, SW2 TACTILE_SWITCH, U1 FE310-G000, U2 IS25LP128-JBLE, Y1 16MHz

Commit message: automated commit
Connections:
- net labels added: ROW_ON
- net labels removed: !ROW_RESET
Changed lines of the file:
@@
 IVDD_FE310
 Text GLabel 9550 3625 2    50   Output ~ 0
-!ROW_RESET
+ROW_ON
 Text GLabel 9550 3725 2    50   Output ~ 0
 !COL_RESET

Commit message: automated commit
Parts:
- removed BZ1, BZ2: Buzzer, symbol Device:Buzzer
- removed R10, R7: CRG0603F4K7, Resistor_SMD:R_0603_1608Metric, symbol custom:CRG0603F4K7
- added BZ1, BZ2: PASSIVE_BUZZER, symbol custom:PASSIVE_BUZZER
- added R31, R34: CRG0603F4K7, Resistor_SMD:R_0603_1608Metric, symbol custom:CRG0603F4K7
- renumbered C1 to C21, C2 to C22, C3 to C23, C4 to C24, C5 to C25, C6 to C26, C7 to C27, C8 to C28, C9 to C29, C10 to C30, C11 to C31, C12 to C32, C13 to C33, C14 to C34, C15 to C35, C16 to C36, C17 to C37, C18 to C38, C19 to C39, C20 to C40, C21 to C41, D3 to D10, D1 to D8, D2 to D9, Q1 to Q2, Q2 to Q3, R1 to R25, R2 to R26, R3 to R27, R4 to R28, R5 to R29, R6 to R30, R8 to R32, R9 to R33, TP1 to TP11, TP2 to TP12, U1 to U4, U2 to U5
Connections:
- net labels added: COL_MODE_SEL, ROW_MODE_SEL
- net labels removed: AUX_5, AUX_6

Commit message: automated commit
Parts:
- R30: Resistance 4.7k -> (none); TOLERANCE (none) -> 5%; VALUE (none) -> 4k7
Changed lines of the file:
@@
-	1    0    0    -1
-$EndComp
-$Comp
-L custom:CRG0603F4K7 R30
-U 1 1 65272D28
-P 5575 2675
-F 0 "R30" V 5695 2575 50  0000 L BNN
-F 1 "CRG0603F4K7" H 4825 2225 50  0001 L BNN
-F 2 "Resistor_SMD:R_0603_1608Metric" H 4825 2125 50  0001 L BNN
-F 3 "datasheets/PYu-RC_Group_51_RoHS_L_9.pdf" H 4825 2025 50  0001 L BNN
-F 4 "4.7k" V 5595 2615 39  0000 L BNN "Resistance"
-	1    5575 2675
 	1    0    0    -1
 $EndComp
@@
 	0    1    1    0
 $EndComp
+$Comp
+L custom:CRG0603F4K7 R30
+U 1 1 5D00CA6C
+P 5575 2675
+F 0 "R30" H 5645 2695 50  0000 L BNN
+F 1 "CRG0603F4K7" H 4875 2275 50  0001 L BNN
+F 2 "Resistor_SMD:R_0603_1608Metric" H 4875 2175 50  0001 L BNN
+F 3 "/home/dj/datasheets/Pyu-RC_Group_51_RoHS_L_9.pdf" H 4875 2075 50  0001 L BNN
+F 4 "4k7" V 5575 2675 50  0000 C CNN "VALUE"
+F 5 "5%" H 5695 2635 50  0000 C CNN "TOLERANCE"
+	1    5575 2675
+	1    0    0    -1
+$EndComp
 $EndSCHEMATC

Commit message: automated commit
Parts:
- D10, D8, D9: footprint Footprint -> (none)
- renumbered TP11 to TP17, TP12 to TP18
Connections:
- net !RESET: no longer names the net of D10.1 (K), R31.2, SW2.2, TP18.1, U4.24 (AON_ERST_N)
- net !WAKEUP: no longer names the net of D9.1 (K), R30.1, SW1.2, TP17.1, U4.18 (AON_PMU_DWAKEUP_N)
Other:
- note added: "!RESET"
- note added: "!WAKEUP"
Changed lines of the file:
@@
 	1    0    0    -1
 $EndComp
-Text Label 6975 3925 0    60   ~ 0
-!RESET
 $Comp
 L power:+1V8 #PWR043
@@
 F 0 "D9" H 5225 2875 50  0000 C CNN
 F 1 "NP_UCLAMP2501T.TCT" H 5275 2675 31  0000 C CNN
-F 2 "Footprint" H 5225 2575 50  0001 C CNN
+F 2 "" H 5225 2575 50  0001 C CNN
 F 3 "" H 5225 2775 50  0001 C CNN
 	1    5225 2775
@@
 F 0 "D8" H 4425 2875 50  0000 C CNN
 F 1 "NP_UCLAMP2501T.TCT" H 4400 2675 31  0000 C CNN
-F 2 "Footprint" H 4425 2575 50  0001 C CNN
+F 2 "" H 4425 2575 50  0001 C CNN
 F 3 "" H 4425 2775 50  0001 C CNN
 	1    4425 2775
@@
 F 0 "D10" H 4825 4425 50  0000 C CNN
 F 1 "UCLAMP2501T.TCT" H 4875 4225 31  0000 C CNN
-F 2 "Footprint" H 4825 4125 50  0001 C CNN
+F 2 "" H 4825 4125 50  0001 C CNN
 F 3 "" H 4825 4325 50  0001 C CNN
 	1    4825 4325
 	0    -1   -1   0
 $EndComp
-Text Label 6825 3625 0    60   ~ 0
-!WAKEUP
 Wire Wire Line
 	4575 2425 4625 2425
@@
 U 1 1 5D9D0EDA
 P 7550 1225
-F 0 "R25" V 7500 1175 50  0000 L BNN
+F 0 "R25" V 7475 1150 50  0000 L BNN
 F 1 "RC0603JR-071KL" H 7625 1150 50  0001 L BNN
 F 2 "Resistor_SMD:R_0603_1608Metric" H 7625 1225 50  0001 L BNN
@@
 U 1 1 65A6018C
 P 7100 2000
-F 0 "R27" V 7050 1950 50  0000 L BNN
+F 0 "R27" V 7025 1925 50  0000 L BNN
 F 1 "RC0603JR-071KL" H 7175 1925 50  0001 L BNN
 F 2 "Resistor_SMD:R_0603_1608Metric" H 7175 2000 50  0001 L BNN
@@
 U 1 1 5DA3C640
 P 9125 1250
-F 0 "R26" V 9075 1200 50  0000 L BNN
+F 0 "R26" V 9050 1175 50  0000 L BNN
 F 1 "RC0603JR-071KL" H 9200 1175 50  0001 L BNN
 F 2 "Resistor_SMD:R_0603_1608Metric" H 9200 1250 50  0001 L BNN
@@
 U 1 1 5DA3C662
 P 8675 2025
-F 0 "R28" V 8625 1975 50  0000 L BNN
+F 0 "R28" V 8600 1950 50  0000 L BNN
 F 1 "RC0603JR-071KL" H 8750 1950 50  0001 L BNN
 F 2 "Resistor_SMD:R_0603_1608Metric" H 8750 2025 50  0001 L BNN
@@
 AR Path="/5D072151" Ref="TP?"  Part="1"
 AR Path="/61C6D021/5D072151" Ref="TP?"  Part="1"
-AR Path="/64D8274A/5D072151" Ref="TP11"  Part="1"
-F 0 "TP11" H 6175 2525 50  0000 C CNN
+AR Path="/64D8274A/5D072151" Ref="TP17"  Part="1"
+F 0 "TP17" H 6175 2525 50  0000 C CNN
 F 1 "TestPoint" H 5975 2350 50  0001 C CNN
 F 2 "" H 6425 2300 50  0001 C CNN
@@
 AR Path="/5D0847E2" Ref="TP?"  Part="1"
 AR Path="/61C6D021/5D0847E2" Ref="TP?"  Part="1"
-AR Path="/64D8274A/5D0847E2" Ref="TP12"  Part="1"
-F 0 "TP12" H 5300 4075 50  0000 C CNN
+AR Path="/64D8274A/5D0847E2" Ref="TP18"  Part="1"
+F 0 "TP18" H 5300 4075 50  0000 C CNN
 F 1 "TestPoint" H 5100 3900 50  0001 C CNN
 F 2 "" H 5550 3850 50  0001 C CNN
@@
 	1    0    0    -1
 $EndComp
+Text Notes 6525 3625 0    60   ~ 0
+!WAKEUP
+Text Notes 6525 3925 0    60   ~ 0
+!RESET
 $EndSCHEMATC

Commit message: automated commit
Parts:
- BZ1, BZ2: footprint (none) -> custom:0.5_IN_BUZZER
- D10, D8, D9: footprint (none) -> custom:SLP1006P2T
- Q2, Q3: footprint (none) -> Package_TO_SOT_SMD:SOT-723
Changed lines of the file:
@@
 F 0 "D9" H 5225 2875 50  0000 C CNN
 F 1 "NP_UCLAMP2501T.TCT" H 5275 2675 31  0000 C CNN
-F 2 "" H 5225 2575 50  0001 C CNN
+F 2 "custom:SLP1006P2T" H 5225 2575 50  0001 C CNN
 F 3 "" H 5225 2775 50  0001 C CNN
 	1    5225 2775
@@
 F 0 "D8" H 4425 2875 50  0000 C CNN
 F 1 "NP_UCLAMP2501T.TCT" H 4400 2675 31  0000 C CNN
-F 2 "" H 4425 2575 50  0001 C CNN
+F 2 "custom:SLP1006P2T" H 4425 2575 50  0001 C CNN
 F 3 "" H 4425 2775 50  0001 C CNN
 	1    4425 2775
@@
 	1    4425 2975
 	1    0    0    -1
-$EndComp
-$Comp
-L custom:UCLAMP2501T.TCT D10
-U 1 1 65272C47
-P 4825 4325
-F 0 "D10" H 4825 4425 50  0000 C CNN
-F 1 "UCLAMP2501T.TCT" H 4875 4225 31  0000 C CNN
-F 2 "" H 4825 4125 50  0001 C CNN
-F 3 "" H 4825 4325 50  0001 C CNN
-	1    4825 4325
-	0    -1   -1   0
 $EndComp
 Wire Wire Line
@@
 F 0 "Q2" V 7775 1725 50  0000 L BNN
 F 1 "SSM3K35AMFV" V 7700 1550 50  0000 L BNN
-F 2 "" H 7650 1675 50  0001 L BIN
+F 2 "Package_TO_SOT_SMD:SOT-723" H 7650 1675 50  0001 L BIN
 F 3 "datasheets/SSM3K35AMFV.pdf" H 7650 1650 50  0001 L BNN
 	1    7450 1800
@@
 F 0 "Q3" V 9350 1750 50  0000 L BNN
 F 1 "SSM3K35AMFV" V 9275 1575 50  0000 L BNN
-F 2 "" H 9225 1700 50  0001 L BIN
+F 2 "Package_TO_SOT_SMD:SOT-723" H 9225 1700 50  0001 L BIN
 F 3 "datasheets/SSM3K35AMFV.pdf" H 9225 1675 50  0001 L BNN
 	1    9025 1825
@@
 	5350 3925 5875 3925
 $Comp
-L custom:PASSIVE_BUZZER BZ1
-U 1 1 5D66C067
-P 7925 1225
-F 0 "BZ1" H 8075 1275 50  0000 L CNN
-F 1 "PASSIVE_BUZZER" H 8075 1175 50  0001 L CNN
-F 2 "" V 7900 1325 50  0001 C CNN
-F 3 "~" V 7900 1325 50  0001 C CNN
-	1    7925 1225
-	1    0    0    -1
-$EndComp
-$Comp
-L custom:PASSIVE_BUZZER BZ2
-U 1 1 5D66C3A0
-P 9500 1250
-F 0 "BZ2" H 9650 1300 50  0000 L CNN
-F 1 "PASSIVE_BUZZER" H 9650 1200 50  0001 L CNN
-F 2 "" V 9475 1350 50  0001 C CNN
-F 3 "~" V 9475 1350 50  0001 C CNN
-	1    9500 1250
-	1    0    0    -1
-$EndComp
-$Comp
 L custom:CRG0603F4K7 R31
 U 1 1 5D66CDE1
@@
 Text Notes 6525 3925 0    60   ~ 0
 !RESET
+$Comp
+L custom:UCLAMP2501T.TCT D10
+U 1 1 65272C47
+P 4825 4325
+F 0 "D10" H 4825 4425 50  0000 C CNN
+F 1 "UCLAMP2501T.TCT" H 4875 4225 31  0000 C CNN
+F 2 "custom:SLP1006P2T" H 4825 4125 50  0001 C CNN
+F 3 "" H 4825 4325 50  0001 C CNN
+	1    4825 4325
+	0    -1   -1   0
+$EndComp
+$Comp
+L custom:PASSIVE_BUZZER BZ2
+U 1 1 5D66C3A0
+P 9500 1250
+F 0 "BZ2" H 9650 1300 50  0000 L CNN
+F 1 "PASSIVE_BUZZER" H 9650 1200 50  0001 L CNN
+F 2 "custom:0.5_IN_BUZZER" V 9475 1350 50  0001 C CNN
+F 3 "~" V 9475 1350 50  0001 C CNN
+	1    9500 1250
+	1    0    0    -1
+$EndComp
+$Comp
+L custom:PASSIVE_BUZZER BZ1
+U 1 1 5D66C067
+P 7925 1225
+F 0 "BZ1" H 8075 1275 50  0000 L CNN
+F 1 "PASSIVE_BUZZER" H 8075 1175 50  0001 L CNN
+F 2 "custom:0.5_IN_BUZZER" V 7900 1325 50  0001 C CNN
+F 3 "~" V 7900 1325 50  0001 C CNN
+	1    7925 1225
+	1    0    0    -1
+$EndComp
 $EndSCHEMATC

Commit message: automated commit
Parts:
- TP22: renamed from TP17; footprint (none) -> custom:TestPoint_THTPad_D1.0mm_Drill0.5mm
- TP23: renamed from TP18; footprint (none) -> custom:TestPoint_THTPad_D1.0mm_Drill0.5mm
- U4: footprint (none) -> Package_DFN_QFN:QFN-48-1EP_6x6mm_P0.4mm_EP4.3x4.3mm
- Y1: footprint (none) -> custom:7M-16.000MAAE-T
Changed lines of the file:
@@
 F 0 "Y1" H 5600 5025 50  0000 C CNN
 F 1 "16MHz" H 5600 4725 50  0000 C CNN
-F 2 "" H 5600 4875 50  0001 C CNN
+F 2 "custom:7M-16.000MAAE-T" H 5600 4875 50  0001 C CNN
 F 3 "~/datasheets/2015TXC_7M_17.pdf" H 5600 4875 50  0001 C CNN
 F 4 "16MHz" H 5600 4875 50  0001 C CNN "Frequency"
@@
 F 0 "U4" H 8375 5275 60  0000 C CNN
 F 1 "FE310-G000" H 8375 2175 60  0000 C CNN
-F 2 "" V 7625 4725 60  0001 C CNN
+F 2 "Package_DFN_QFN:QFN-48-1EP_6x6mm_P0.4mm_EP4.3x4.3mm" V 7625 4725 60  0001 C CNN
 F 3 "" V 7625 4725 60  0001 C CNN
 	1    8375 3975
@@
 AR Path="/5D072151" Ref="TP?"  Part="1"
 AR Path="/61C6D021/5D072151" Ref="TP?"  Part="1"
-AR Path="/64D8274A/5D072151" Ref="TP17"  Part="1"
-F 0 "TP17" H 6175 2525 50  0000 C CNN
+AR Path="/64D8274A/5D072151" Ref="TP22"  Part="1"
+F 0 "TP22" H 6175 2525 50  0000 C CNN
 F 1 "TestPoint" H 5975 2350 50  0001 C CNN
-F 2 "" H 6425 2300 50  0001 C CNN
+F 2 "custom:TestPoint_THTPad_D1.0mm_Drill0.5mm" H 6425 2300 50  0001 C CNN
 F 3 "~" H 6425 2300 50  0001 C CNN
 	1    6225 2300
@@
 AR Path="/5D0847E2" Ref="TP?"  Part="1"
 AR Path="/61C6D021/5D0847E2" Ref="TP?"  Part="1"
-AR Path="/64D8274A/5D0847E2" Ref="TP18"  Part="1"
-F 0 "TP18" H 5300 4075 50  0000 C CNN
+AR Path="/64D8274A/5D0847E2" Ref="TP23"  Part="1"
+F 0 "TP23" H 5300 4075 50  0000 C CNN
 F 1 "TestPoint" H 5100 3900 50  0001 C CNN
-F 2 "" H 5550 3850 50  0001 C CNN
+F 2 "custom:TestPoint_THTPad_D1.0mm_Drill0.5mm" H 5550 3850 50  0001 C CNN
 F 3 "~" H 5550 3850 50  0001 C CNN
 	1    5350 3850

Commit message: automated commit
Parts:
- removed SW1: NP_TACTILE_SWITCH, CUSTOM:TACTILE_SWITCH, symbol custom:TACTILE_SWITCH
- removed SW2: TACTILE_SWITCH, CUSTOM:TACTILE_SWITCH, symbol custom:TACTILE_SWITCH
- added SW1, SW2: TACTILE_SWITCH_SMALL, custom:TACTILE_SWITCH_SMALL, symbol custom:TACTILE_SWITCH_SMALL
Connections:
- net at D9.1 (K), R30.1, TP22.1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: now also SW1.2
- net at D10.1 (K), R31.2, TP23.1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: now also SW2.2
- net at R32.1: now also SW2.1
- net at D8.1 (K), R29.2: now also SW1.1
Other:
- moved on the sheet: C36, C37, D10, D9, R32, R34, U5
