File: FE310.sch (KiCad schematic (older format))
At the start: 45 parts, among them Q2 SSM3K35AMFV, Q3 SSM3K35AMFV, SW1 TACTILE_SWITCH_SMALL, SW2 TACTILE_SWITCH_SMALL, U4 FE310-G000, U5 IS25LP128-JBLE, Y1 16MHz

Commit message: automated commit
Parts:
- U5: footprint Housings_SOIC:SOIC-8_3.9x4.9mm_Pitch1.27mm -> Package_SO:SOIC-8_3.9x4.9mm_P1.27mm
Changed lines of the file:
@@
 F 0 "U5" H 5125 6625 60  0000 C CNN
 F 1 "IS25LP128-JBLE" H 5475 5925 60  0000 C CNN
-F 2 "Housings_SOIC:SOIC-8_3.9x4.9mm_Pitch1.27mm" H 5525 6325 60  0001 C CNN
+F 2 "Package_SO:SOIC-8_3.9x4.9mm_P1.27mm" H 5525 6325 60  0001 C CNN
 F 3 "" H 5525 6325 60  0001 C CNN
 	1    5475 6275

Commit message: automated commit
Parts:
- removed C38: CL10B104KO8NNNC, Capacitor_SMD:C_0603_1608Metric, symbol custom:CL10B104KO8NNNC
Changed lines of the file:
@@
 	7275 2925 7275 3025
 Wire Wire Line
-	9475 2825 9550 2825
+	9475 2825 10225 2825
 Wire Wire Line
 	9475 2925 9475 3025
@@
 	1    0    0    -1
 $EndComp
-Text GLabel 9550 2825 2    50   Input ~ 0
-IVDD_FE310
 Text GLabel 9550 3625 2    50   Output ~ 0
 ROW_ON
@@
 	1    0    0    -1
 $EndComp
-$Comp
-L custom:CL10B104KO8NNNC C34
-U 1 1 5F07D419
-P 2450 5400
-F 0 "C34" H 2565 5491 50  0000 L CNN
-F 1 "CL10B104KO8NNNC" H 1500 4950 50  0001 L BNN
-F 2 "Capacitor_SMD:C_0603_1608Metric" H 1500 4850 50  0001 L BNN
-F 3 "datasheets/CL10B104KO8NNNC.pdf" H 1500 4750 50  0001 L BNN
-F 4 "0.1uF" H 2565 5400 50  0000 L CNN "Capacitance"
-F 5 "16V" H 2565 5309 50  0000 L CNN "Rating"
-	1    2450 5400
-	1    0    0    -1
-$EndComp
-$Comp
-L custom:CL10B105KA8NNNC C35
-U 1 1 5F07D421
-P 2900 5400
-F 0 "C35" H 3015 5491 50  0000 L CNN
-F 1 "CL10B105KA8NNNC" H 1950 4950 50  0001 L BNN
-F 2 "Capacitor_SMD:C_0603_1608Metric" H 1950 4850 50  0001 L BNN
-F 3 "datasheets/CL10B105KA8NNNC.pdf" H 1950 4750 50  0001 L BNN
-F 4 "1uF" H 3015 5400 50  0000 L CNN "Capacitance"
-F 5 "25V" H 3015 5309 50  0000 L CNN "Rating"
-	1    2900 5400
-	1    0    0    -1
-$EndComp
-$Comp
-L custom:CL10B104KO8NNNC C40
-U 1 1 5F07D429
-P 2450 6650
-F 0 "C40" H 2565 6741 50  0000 L CNN
-F 1 "CL10B104KO8NNNC" H 1500 6200 50  0001 L BNN
-F 2 "Capacitor_SMD:C_0603_1608Metric" H 1500 6100 50  0001 L BNN
-F 3 "datasheets/CL10B104KO8NNNC.pdf" H 1500 6000 50  0001 L BNN
-F 4 "0.1uF" H 2565 6650 50  0000 L CNN "Capacitance"
-F 5 "16V" H 2565 6559 50  0000 L CNN "Rating"
-	1    2450 6650
-	1    0    0    -1
-$EndComp
-$Comp
-L custom:CL10B105KA8NNNC C41
-U 1 1 5F07D431
-P 2900 6650
-F 0 "C41" H 3015 6741 50  0000 L CNN
-F 1 "CL10B105KA8NNNC" H 1950 6200 50  0001 L BNN
-F 2 "Capacitor_SMD:C_0603_1608Metric" H 1950 6100 50  0001 L BNN
-F 3 "datasheets/CL10B105KA8NNNC.pdf" H 1950 6000 50  0001 L BNN
-F 4 "1uF" H 3015 6650 50  0000 L CNN "Capacitance"
-F 5 "25V" H 3015 6559 50  0000 L CNN "Rating"
-	1    2900 6650
-	1    0    0    -1
-$EndComp
-$Comp
-L custom:CL10B104KO8NNNC C38
-U 1 1 5F07D439
-P 1600 6650
-F 0 "C38" H 1715 6741 50  0000 L CNN
-F 1 "CL10B104KO8NNNC" H 650 6200 50  0001 L BNN
-F 2 "Capacitor_SMD:C_0603_1608Metric" H 650 6100 50  0001 L BNN
-F 3 "datasheets/CL10B104KO8NNNC.pdf" H 650 6000 50  0001 L BNN
-F 4 "0.1uF" H 1715 6650 50  0000 L CNN "Capacitance"
-F 5 "16V" H 1715 6559 50  0000 L CNN "Rating"
-	1    1600 6650
-	1    0    0    -1
-$EndComp
-$Comp
-L custom:CL10B105KA8NNNC C39
-U 1 1 5F07D441
-P 2050 6650
-F 0 "C39" H 2165 6741 50  0000 L CNN
-F 1 "CL10B105KA8NNNC" H 1100 6200 50  0001 L BNN
-F 2 "Capacitor_SMD:C_0603_1608Metric" H 1100 6100 50  0001 L BNN
-F 3 "datasheets/CL10B105KA8NNNC.pdf" H 1100 6000 50  0001 L BNN
-F 4 "1uF" H 2165 6650 50  0000 L CNN "Capacitance"
-F 5 "25V" H 2165 6559 50  0000 L CNN "Rating"
-	1    2050 6650
-	1    0    0    -1
-$EndComp
-Wire Wire Line
-	1600 6900 2050 6900
-Wire Wire Line
-	2900 6850 2900 6900
-Wire Wire Line
-	2900 5600 2900 5650
 Wire Wire Line
 	2900 4350 2900 4450
@@
 	2900 1350 2900 1450
 Wire Wire Line
-	2900 6400 2900 6500
-Wire Wire Line
-	2450 5150 2450 5250
-Wire Wire Line
 	2900 3100 2900 3200
 Wire Wire Line
 	2900 1850 2900 1950
-Wire Wire Line
-	1600 6500 1600 6400
-Wire Wire Line
-	1600 6800 1600 6900
 Wire Wire Line
 	2450 6400 2900 6400
 Connection ~ 2450 6400
-Wire Wire Line
-	2450 6400 2450 6500
-Wire Wire Line
-	2450 6850 2900 6850
-Wire Wire Line
-	2450 6800 2450 6850
-Wire Wire Line
-	2900 5600 2450 5600
-Connection ~ 2900 5600
-Wire Wire Line
-	2900 5550 2900 5600
-Wire Wire Line
-	2900 5150 2900 5250
 Connection ~ 2900 4350
 Wire Wire Line
@@
 	2900 1850 2900 1750
 Wire Wire Line
-	1600 6400 2050 6400
-Wire Wire Line
 	2050 6400 2450 6400
 Connection ~ 2050 6400
-Wire Wire Line
-	2050 6400 2050 6500
-Wire Wire Line
-	2050 6900 2050 6800
-Connection ~ 1600 6400
-Wire Wire Line
-	650  6400 1600 6400
-Connection ~ 2900 6850
-Wire Wire Line
-	2900 6800 2900 6850
 Connection ~ 2900 6400
 Wire Wire Line
 	2900 6300 2900 6400
-Connection ~ 1600 6900
-Wire Wire Line
-	650  6900 1600 6900
-Wire Wire Line
-	2450 5550 2450 5600
 Wire Wire Line
 	2450 5150 2900 5150
@@
 	1    0    0    -1
 $EndComp
-$Comp
-L power:GND #PWR067
-U 1 1 5F07D4B2
-P 2900 6900
-F 0 "#PWR067" H 2900 6650 50  0001 C CNN
-F 1 "GND" H 2900 6750 50  0000 C CNN
-F 2 "" H 2900 6900 50  0001 C CNN
-F 3 "" H 2900 6900 50  0001 C CNN
-	1    2900 6900
-	1    0    0    -1
-$EndComp
-Text Label 650  6900 0    60   ~ 0
-PLL_AVSS_FE310
-Text Label 650  6400 0    60   ~ 0
+Text Label 1025 6400 0    60   ~ 0
 PLL_AVDD_FE310
 $Comp
@@
 F 3 "" H 2900 5050 50  0001 C CNN
 	1    2900 5050
-	1    0    0    -1
-$EndComp
-$Comp
-L power:GND #PWR062
-U 1 1 5F07D4C0
-P 2900 5650
-F 0 "#PWR062" H 2900 5400 50  0001 C CNN
-F 1 "GND" H 2900 5500 50  0000 C CNN
-F 2 "" H 2900 5650 50  0001 C CNN
-F 3 "" H 2900 5650 50  0001 C CNN
-	1    2900 5650
 	1    0    0    -1
 $EndComp
@@
 Wire Wire Line
 	5175 2375 5575 2375
+Wire Wire Line
+	1025 6400 2050 6400
+Wire Wire Line
+	2900 5150 2900 5250
+Wire Wire Line
+	2450 5150 2450 5250
+$Comp
+L power:GND #PWR062
+U 1 1 5F07D4C0
+P 2900 5750
+F 0 "#PWR062" H 2900 5500 50  0001 C CNN
+F 1 "GND" H 2900 5600 50  0000 C CNN
+F 2 "" H 2900 5750 50  0001 C CNN
+F 3 "" H 2900 5750 50  0001 C CNN
+	1    2900 5750
+	1    0    0    -1
+$EndComp
+Wire Wire Line
+	2450 5550 2450 5650
+Wire Wire Line
+	2900 5550 2900 5650
+Connection ~ 2900 5650
+Wire Wire Line
+	2900 5650 2450 5650
+Wire Wire Line
+	2900 5650 2900 5750
+$Comp
+L custom:CL10B105KA8NNNC C35
+U 1 1 5F07D421
+P 2900 5400
+F 0 "C35" H 3015 5491 50  0000 L CNN
+F 1 "CL10B105KA8NNNC" H 1950 4950 50  0001 L BNN
+F 2 "Capacitor_SMD:C_0603_1608Metric" H 1950 4850 50  0001 L BNN
+F 3 "datasheets/CL10B105KA8NNNC.pdf" H 1950 4750 50  0001 L BNN
+F 4 "1uF" H 3015 5400 50  0000 L CNN "Capacitance"
+F 5 "25V" H 3015 5309 50  0000 L CNN "Rating"
+	1    2900 5400
+	1    0    0    -1
+$EndComp
+$Comp
+L custom:CL10B104KO8NNNC C34
+U 1 1 5F07D419
+P 2450 5400
+F 0 "C34" H 2565 5491 50  0000 L CNN
+F 1 "CL10B104KO8NNNC" H 1500 4950 50  0001 L BNN
+F 2 "Capacitor_SMD:C_0603_1608Metric" H 1500 4850 50  0001 L BNN
+F 3 "datasheets/CL10B104KO8NNNC.pdf" H 1500 4750 50  0001 L BNN
+F 4 "0.1uF" H 2565 5400 50  0000 L CNN "Capacitance"
+F 5 "16V" H 2565 5309 50  0000 L CNN "Rating"
+	1    2450 5400
+	1    0    0    -1
+$EndComp
+$Comp
+L power:GND #PWR067
+U 1 1 5F07D4B2
+P 2900 7000
+F 0 "#PWR067" H 2900 6750 50  0001 C CNN
+F 1 "GND" H 2900 6850 50  0000 C CNN
+F 2 "" H 2900 7000 50  0001 C CNN
+F 3 "" H 2900 7000 50  0001 C CNN
+	1    2900 7000
+	1    0    0    -1
+$EndComp
+Wire Wire Line
+	2900 6800 2900 6900
+Connection ~ 2900 6900
+Wire Wire Line
+	2050 6400 2050 6500
+Wire Wire Line
+	2450 6800 2450 6900
+Wire Wire Line
+	2450 6900 2900 6900
+Wire Wire Line
+	2450 6400 2450 6500
+Wire Wire Line
+	2900 6400 2900 6500
+Wire Wire Line
+	2900 6900 2900 7000
+$Comp
+L custom:CL10B105KA8NNNC C39
+U 1 1 5F07D441
+P 2050 6650
+F 0 "C39" H 2165 6741 50  0000 L CNN
+F 1 "CL10B105KA8NNNC" H 1100 6200 50  0001 L BNN
+F 2 "Capacitor_SMD:C_0603_1608Metric" H 1100 6100 50  0001 L BNN
+F 3 "datasheets/CL10B105KA8NNNC.pdf" H 1100 6000 50  0001 L BNN
+F 4 "1uF" H 2165 6650 50  0000 L CNN "Capacitance"
+F 5 "25V" H 2165 6559 50  0000 L CNN "Rating"
+	1    2050 6650
+	1    0    0    -1
+$EndComp
+$Comp
+L custom:CL10B105KA8NNNC C41
+U 1 1 5F07D431
+P 2900 6650
+F 0 "C41" H 3015 6741 50  0000 L CNN
+F 1 "CL10B105KA8NNNC" H 1950 6200 50  0001 L BNN
+F 2 "Capacitor_SMD:C_0603_1608Metric" H 1950 6100 50  0001 L BNN
+F 3 "datasheets/CL10B105KA8NNNC.pdf" H 1950 6000 50  0001 L BNN
+F 4 "1uF" H 3015 6650 50  0000 L CNN "Capacitance"
+F 5 "25V" H 3015 6559 50  0000 L CNN "Rating"
+	1    2900 6650
+	1    0    0    -1
+$EndComp
+$Comp
+L custom:CL10B104KO8NNNC C40
+U 1 1 5F07D429
+P 2450 6650
+F 0 "C40" H 2565 6741 50  0000 L CNN
+F 1 "CL10B104KO8NNNC" H 1500 6200 50  0001 L BNN
+F 2 "Capacitor_SMD:C_0603_1608Metric" H 1500 6100 50  0001 L BNN
+F 3 "datasheets/CL10B104KO8NNNC.pdf" H 1500 6000 50  0001 L BNN
+F 4 "0.1uF" H 2565 6650 50  0000 L CNN "Capacitance"
+F 5 "16V" H 2565 6559 50  0000 L CNN "Rating"
+	1    2450 6650
+	1    0    0    -1
+$EndComp
+Wire Wire Line
+	1025 6900 2050 6900
+Text Label 1025 6900 0    60   ~ 0
+PLL_AVSS_FE310
+Wire Wire Line
+	2050 6900 2050 6800
+Text Label 10225 2825 2    60   ~ 0
+IVDD_FE310
 $EndSCHEMATC

Commit message: automated commit
Connections:
- net AUX_0: now also U4.27 (GPIO_2); no longer U4.26 (GPIO_1)
- net AUX_1: now also U4.26 (GPIO_1); no longer U4.36 (GPIO_12)
- net ROW_ON: now also U4.34 (GPIO_10); no longer U4.27 (GPIO_2)
- net ROW_SHCP: now also U4.36 (GPIO_12); no longer U4.34 (GPIO_10)
- net AUX_2: no longer names the net of U4.40 (GPIO_18)
- net AUX_3: no longer names the net of U4.42 (GPIO_20)
- net AUX_4: no longer names the net of U4.43 (GPIO_21)
- no-connect marks 4 -> 7
Changed lines of the file:
@@
 	9550 5325 9325 5325
-Wire Wire Line
-	9550 5225 9325 5225
-Wire Wire Line
-	9550 5125 9325 5125
-Wire Wire Line
-	9550 4925 9325 4925
 Wire Wire Line
 	9550 5425 9325 5425
@@
 	9325 4325 9550 4325
 Wire Wire Line
-	9325 4525 10225 4525
+	9325 4525 10325 4525
 Wire Wire Line
 	9325 3425 10225 3425
@@
 	1    0    0    -1
 $EndComp
-Text GLabel 9550 3625 2    50   Output ~ 0
+Text GLabel 9550 4225 2    50   Output ~ 0
 ROW_ON
 Text GLabel 9550 3725 2    50   Output ~ 0
@@
 Text GLabel 9550 4125 2    50   Output ~ 0
 COL_IN
-Text GLabel 9550 4225 2    50   Output ~ 0
+Text GLabel 9550 4425 2    50   Output ~ 0
 ROW_SHCP
 Text GLabel 9550 4325 2    50   Output ~ 0
 COL_SHCP
-Text GLabel 9550 3525 2    50   Output ~ 0
+Text GLabel 9550 3625 2    50   Output ~ 0
 AUX_0
 Text GLabel 9550 4725 2    50   Input ~ 0
@@
 Text GLabel 9550 4825 2    50   Output ~ 0
 UART_FE_TX
-Text GLabel 9550 4425 2    50   Output ~ 0
+Text GLabel 9550 3525 2    50   Output ~ 0
 AUX_1
 Text GLabel 9550 5025 2    50   Output ~ 0
 LED_PWM
-Text GLabel 9550 4925 2    50   Output ~ 0
-AUX_2
-Text GLabel 9550 5125 2    50   Output ~ 0
-AUX_3
-Text GLabel 9550 5225 2    50   Output ~ 0
-AUX_4
 Text GLabel 9550 5325 2    50   Output ~ 0
 ROW_MODE_SEL
@@
 Text Label 10225 3425 2    50   ~ 0
 PIEZO_0
-Text Label 10225 4525 2    50   ~ 0
+Text Label 10325 4525 2    50   ~ 0
 PIEZO_1
 Text Label 6725 1800 0    50   ~ 0
@@
 Text Label 10225 2825 2    60   ~ 0
 IVDD_FE310
+NoConn ~ 9325 4925
+NoConn ~ 9325 5125
+NoConn ~ 9325 5225
 $EndSCHEMATC

Commit message: automated commit
Parts:
- removed BZ2: PASSIVE_BUZZER, custom:0.5_IN_BUZZER, symbol custom:PASSIVE_BUZZER
- removed D8: NP_UCLAMP2501T.TCT, custom:SLP1006P2T, symbol custom:UCLAMP2501T.TCT
- removed Q3: SSM3K35AMFV, Package_TO_SOT_SMD:SOT-723, symbol custom:SSM3K35AMFV
- removed R26, R28: RC0603JR-071KL, Resistor_SMD:R_0603_1608Metric, symbol custom:RC0603JR-071KL
- removed SW1: TACTILE_SWITCH_SMALL, custom:TACTILE_SWITCH_SMALL, symbol custom:TACTILE_SWITCH_SMALL
- added NP_SW1: NP_TACTILE_SWITCH_SMALL, custom:TACTILE_SWITCH_SMALL, symbol custom:NP_TACTILE_SWITCH_SMALL
- added R14: NP_R_0603, Resistor_SMD:R_0603_1608Metric, symbol custom:NP_R_0603
Connections:
- net AUX_0: now also U4.40 (GPIO_18); no longer U4.27 (GPIO_2)
- net AUX_1: now also U4.42 (GPIO_20); no longer U4.26 (GPIO_1)
- net COL_MODE_SEL: now also U4.27 (GPIO_2); no longer U4.45 (GPIO_23)
- net GND: now also R14.2
- net LED_PWM: now also U4.44 (GPIO_22); no longer U4.41 (GPIO_19)
- net ROW_MODE_SEL: now also U4.26 (GPIO_1); no longer U4.44 (GPIO_22)
- net at D9.1 (K), R30.1, TP22.1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: now also R29.2, NP_SW1.2
- net AUX_2: now reaches U4.43 (GPIO_21)
- new net: NP_SW1.1, R14.1
- no-connect marks 7 -> 6
Other:
- moved on the sheet: BZ1, Q2, R25, R27, R29
