File: FT2232.sch (KiCad schematic (older format))
At the start: 34 parts

Commit message: automated commit
Parts:
- removed R?: ‎RMCF0603FT470R‎, Resistor_SMD:R_0603_1608Metric, symbol flipdot_driver-rescue:‎RMCF0603FT470R‎-custom
- added R14: ‎RMCF0603FT470R‎, Resistor_SMD:R_0603_1608Metric, symbol custom:‎RMCF0603FT470R‎
- gave numbers to parts that had none: 33
Other:
- moved on the sheet: C27, C28, C29, C30, C31, C32, C34
