File: FT2232.sch (KiCad schematic (older format))
At the start: 34 parts, among them J3 USB-C_Connector, U3 FT2232D, Y2 NX8045GB-6MHZ-STD-CSF-3

Commit message: automated commit
Parts:
- renumbered C27 to C42, C28 to C43, C29 to C44, C30 to C45, C31 to C46, C32 to C47, C33 to C48, C34 to C49, C35 to C50, C36 to C51, D7 to D16, D8 to D17, J3 to J4, L2 to L5, R12 to R50, R13 to R51, R14 to R52, R15 to R53, R16 to R54, R17 to R55, R18 to R56, R19 to R57, R20 to R58, R21 to R59, R22 to R60, R23 to R61, R24 to R62, R25 to R63, TP6 to TP18, TP7 to TP19, TP8 to TP20, TP9 to TP21, U3 to U8

Commit message: automated commit
Parts:
- removed R53: 1.5k, Resistors_SMD:R_0603_HandSoldering, symbol Device:R
- added R53: RMCF0603FT1K50, Resistor_SMD:R_0603_1608Metric, symbol custom:RMCF0603FT1K50
- R54: Resistance 4.7k -> (none); TOLERANCE (none) -> 5%; VALUE (none) -> 4k7
- R55: Resistance 47k -> (none); TOLERANCE (none) -> 1%; VALUE (none) -> 47K0
Changed lines of the file:
@@
 $EndDescr
-$Comp
-L Device:R R53
-U 1 1 60A0D443
-P 5175 3350
-F 0 "R53" V 5255 3350 50  0000 C CNN
-F 1 "1.5k" V 5175 3350 50  0000 C CNN
-F 2 "Resistors_SMD:R_0603_HandSoldering" V 5105 3350 50  0001 C CNN
-F 3 "" H 5175 3350 50  0001 C CNN
-	1    5175 3350
-	1    0    0    1
-$EndComp
 $Comp
 L custom:FT2232D U8
@@
 Text GLabel 7475 2300 2    50   Input ~ 0
 JTAG_TDO
-$Comp
-L custom:CRG0603F4K7 R54
-U 1 1 60A0D667
-P 3525 3600
-F 0 "R54" V 3645 3500 50  0000 L BNN
-F 1 "CRG0603F4K7" H 2775 3150 50  0001 L BNN
-F 2 "Resistor_SMD:R_0603_1608Metric" H 2775 3050 50  0001 L BNN
-F 3 "datasheets/PYu-RC_Group_51_RoHS_L_9.pdf" H 2775 2950 50  0001 L BNN
-F 4 "4.7k" V 3545 3540 39  0000 L BNN "Resistance"
-	1    3525 3600
-	1    0    0    -1
-$EndComp
-$Comp
-L custom:RC0603FR-0747KL R55
-U 1 1 60A0D660
-P 3525 4100
-F 0 "R55" V 3645 4000 50  0000 L BNN
-F 1 "RC0603FR-0747KL" H 2775 3650 50  0001 L BNN
-F 2 "Resistor_SMD:R_0603_1608Metric" H 2775 3550 50  0001 L BNN
-F 3 "datasheets/‎SEI-RMCF_RMCP.pdf" H 2775 3450 50  0001 L BNN
-F 4 "47k" V 3545 4040 39  0000 L BNN "Resistance"
-	1    3525 4100
-	1    0    0    -1
-$EndComp
 Wire Wire Line
 	2875 3400 3525 3400
@@
 	1    0    0    -1
 $EndComp
+$Comp
+L custom:CRG0603F4K7 R54
+U 1 1 5D023D3B
+P 3525 3600
+F 0 "R54" H 3595 3620 50  0000 L BNN
+F 1 "CRG0603F4K7" H 2825 3200 50  0001 L BNN
+F 2 "Resistor_SMD:R_0603_1608Metric" H 2825 3100 50  0001 L BNN
+F 3 "/home/dj/datasheets/Pyu-RC_Group_51_RoHS_L_9.pdf" H 2825 3000 50  0001 L BNN
+F 4 "4k7" V 3525 3600 50  0000 C CNN "VALUE"
+F 5 "5%" H 3645 3560 50  0000 C CNN "TOLERANCE"
+	1    3525 3600
+	1    0    0    -1
+$EndComp
+$Comp
+L custom:RC0603FR-0747KL R55
+U 1 1 5D0244A5
+P 3525 4100
+F 0 "R55" H 3595 4120 50  0000 L BNN
+F 1 "RC0603FR-0747KL" H 3125 3650 50  0001 L BNN
+F 2 "Resistor_SMD:R_0603_1608Metric" H 3125 3550 50  0001 L BNN
+F 3 "" H 2825 3500 50  0001 L BNN
+F 4 "47K0" V 3525 4100 50  0000 C CNN "VALUE"
+F 5 "1%" H 3645 4060 50  0000 C CNN "TOLERANCE"
+	1    3525 4100
+	1    0    0    -1
+$EndComp
+$Comp
+L custom:RMCF0603FT1K50 R53
+U 1 1 5D02E1AF
+P 5175 3350
+F 0 "R53" H 5245 3370 50  0000 L BNN
+F 1 "RMCF0603FT1K50" H 4775 2900 50  0001 L BNN
+F 2 "Resistor_SMD:R_0603_1608Metric" H 4775 2800 50  0001 L BNN
+F 3 "" H 4475 2750 50  0001 L BNN
+F 4 "1k5" V 5175 3350 50  0000 C CNN "VALUE"
+F 5 "1%" H 5295 3310 50  0000 C CNN "TOLERANCE"
+	1    5175 3350
+	1    0    0    -1
+$EndComp

Commit message: automated commit
Parts:
- removed R55: RC0603FR-0747KL, Resistor_SMD:R_0603_1608Metric, symbol custom:RC0603FR-0747KL
- added C49: CL10B105KA8NNNC, Capacitor_SMD:C_0603_1608Metric, symbol custom:CL10B105KA8NNNC
- added R45: RC0603JR-071KL, Resistor_SMD:R_0603_1608Metric, symbol custom:RC0603JR-071KL
- added R49: RMCF0603FT10K0, 0603, symbol custom:RMCF0603FT10K0
- added TP19: TestPoint, symbol Connector:TestPoint
- C44, C47: NP NP -> NP_0603
- D16: footprint Footprint -> (none)
- R50, R51: footprint Resistors_SMD:R_0603_HandSoldering -> Resistor_SMD:R_0603_1608Metric
- renumbered C49 to C50, C50 to C51, C51 to C52, J4 to J9, R52 to R46, R53 to R47, R54 to R48, R56 to R52, R57 to R53, R58 to R54, R59 to R55, R60 to R56, R61 to R57, R62 to R58, R63 to R59, TP18 to TP20, TP19 to TP21, TP20 to TP22, TP21 to TP23
Connections:
- net labels added: USB_D+, USB_D-, USB_SHIELD
- wire segments 157 -> 169
Other:
- note added: "ROUTE THROUGH\nAVOID STUBS"
- note removed: "AVOID STUBS"
- moved on the sheet: D16, D17, R50, R51

Commit message: automated commit
Parts:
- D16: footprint (none) -> custom:SOD-123FL
- D17: footprint (none) -> Package_TO_SOT_SMD:SOT-323_SC-70
- R49: footprint 0603 -> custom:R_0603
Changed lines of the file:
@@
 F 0 "D16" H 3025 1200 50  0000 C CNN
 F 1 "SMF5.0A" H 3025 1000 50  0000 C CNN
-F 2 "" H 3025 900 50  0001 C CNN
+F 2 "custom:SOD-123FL" H 3025 900 50  0001 C CNN
 F 3 "" H 3025 1100 50  0001 C CNN
 	1    3025 1100
@@
 F 0 "R49" H 3575 4150 50  0000 L BNN
 F 1 "RMCF0603FT10K0" H 3200 3550 50  0001 L BNN
-F 2 "0603" H 3450 3475 50  0001 L BNN
+F 2 "custom:R_0603" H 3450 3475 50  0001 L BNN
 F 3 "" V 3825 3650 50  0001 L BNN
 F 4 "10k0" V 3525 4100 50  0000 C CNN "Resistance"
@@
 F 0 "D17" H 1750 5175 50  0000 C CNN
 F 1 "RSB6.8F2T106" H 1850 4775 50  0000 C CNN
-F 2 "" H 1750 5075 50  0001 C CNN
+F 2 "Package_TO_SOT_SMD:SOT-323_SC-70" H 1750 5075 50  0001 C CNN
 F 3 "" H 1750 5075 50  0001 C CNN
 	1    1750 4975

Commit message: automated commit
Parts:
- removed J9: USB-C_Connector, symbol custom:USB-C_Connector
- removed L5: FBMH4532HM681-T, symbol custom:FBMH4532HM681-T
- added J?: USB-C_2.0_Connector, custom:USB4085-GF-A, symbol custom:USB-C_2.0_Connector
- added L5: BLM31SN500SZ1L, Inductor_SMD:L_1206_3216Metric, symbol custom:BLM31SN500SZ1L
- added R? (x4): NP_R_0603, Resistor_SMD:R_0603_1608Metric, symbol custom:NP_R_0603
- added R? (x4): RC0603JR-070RL, Resistor_SMD:R_0603_1608Metric, symbol custom:RC0603JR-070RL
- TP24: renamed from TP19; footprint (none) -> custom:TestPoint_THTPad_D1.0mm_Drill0.5mm
- TP25: renamed from TP20; footprint (none) -> custom:TestPoint_THTPad_D1.0mm_Drill0.5mm
- TP26: renamed from TP21; footprint (none) -> custom:TestPoint_THTPad_D1.0mm_Drill0.5mm
- TP27: renamed from TP22; footprint (none) -> custom:TestPoint_THTPad_D1.0mm_Drill0.5mm
- TP28: renamed from TP23; footprint (none) -> custom:TestPoint_THTPad_D1.0mm_Drill0.5mm
- Y2: footprint (none) -> custom:NX8045GB
Connections:
- wire segments 169 -> 201
- no-connect marks 18 -> 10
Other:
- moved on the sheet: C48, C49, C51, C52, D16, D17, R45, R47, R48, R49, R50, R51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

Commit message: automated commit
Parts:
- gave numbers to parts that had none: 9
- renumbered C50 to C49, C49 to C50, R46 to R53, R47 to R54, R45 to R55, R48 to R56, R49 to R57, R50 to R58, R51 to R59, R52 to R60, R53 to R61, R54 to R62, R55 to R63, R56 to R64, R57 to R65, R58 to R66, R59 to R67

Commit message: automated commit
Parts:
- U8: footprint Housings_QFP:LQFP-48_7x7mm_Pitch0.5mm -> Package_QFP:LQFP-48_7x7mm_P0.5mm
Changed lines of the file:
@@
 F 0 "U8" H 6525 4125 60  0000 C CNN
 F 1 "FT2232D" H 6525 4025 60  0000 C CNN
-F 2 "Housings_QFP:LQFP-48_7x7mm_Pitch0.5mm" H 6525 4075 60  0001 C CNN
+F 2 "Package_QFP:LQFP-48_7x7mm_P0.5mm" H 6525 4075 60  0001 C CNN
 F 3 "/home/dj/datasheets/FT2232D.pdf" H 6525 4075 60  0001 C CNN
 	1    6525 4075
