File: FT2232.sch (KiCad schematic (older format))
At the start: 45 parts, among them J9 USB-C_2.0_Connector, U8 FT2232D, Y2 NX8045GB-6MHZ-STD-CSF-3

Commit message: automated commit
Parts:
- removed C52: TMK042CG120JD-W‎, Capacitor_SMD:C_01005_0402Metric, symbol custom:GRM1555C1H120JA01D
- added C38: GRM1555C1H120JA01D, Capacitor_SMD:C_0402_1005Metric, symbol custom:GRM1555C1H120JA01D
- C51: value TMK042CG120JD-W‎ -> GRM1555C1H120JA01D; footprint Capacitor_SMD:C_01005_0402Metric -> Capacitor_SMD:C_0402_1005Metric; DIELECTRIC (none) -> C0G; RATING (none) -> 50V; Rating 25V -> (none); TOLERANCE (none) -> 5%
Connections:
- net GND: now also C38.2
- net at U8.43 (XTIN), Y2.1: now also C38.1; no longer C51.1
- net at U8.44 (XTOUT), Y2.2: now also C51.1
Changed lines of the file:
@@
 $Descr USLetter 11000 8500
 encoding utf-8
-Sheet 6 20
+Sheet 5 20
 Title "FLIPDOT_DRIVER"
 Date ""
@@
 Wire Wire Line
 	4200 4875 4200 4925
-$Comp
-L custom:GRM1555C1H120JA01D C52
-U 1 1 60A0D60E
-P 4925 5075
-F 0 "C52" H 5040 5166 50  0000 L CNN
-F 1 "TMK042CG120JD-W‎" H 3975 4625 50  0001 L BNN
-F 2 "Capacitor_SMD:C_01005_0402Metric" H 3975 4525 50  0001 L BNN
-F 3 "datasheets/TMK042CG120JD-W‎.pdf" H 3975 4425 50  0001 L BNN
-F 4 "12pF" H 5040 5075 50  0000 L CNN "Capacitance"
-F 5 "25V" H 5040 4984 50  0000 L CNN "Rating"
-	1    4925 5075
-	1    0    0    -1
-$EndComp
-$Comp
-L custom:GRM1555C1H120JA01D C?
-U 1 1 60A0D606
-P 4200 5075
-AR Path="/60A0D606" Ref="C?"  Part="1"
-AR Path="/609E0ED6/60A0D606" Ref="C51"  Part="1"
-F 0 "C51" H 4315 5166 50  0000 L CNN
-F 1 "TMK042CG120JD-W‎" H 3250 4625 50  0001 L BNN
-F 2 "Capacitor_SMD:C_01005_0402Metric" H 3250 4525 50  0001 L BNN
-F 3 "datasheets/TMK042CG120JD-W‎.pdf" H 3250 4425 50  0001 L BNN
-F 4 "12pF" H 4315 5075 50  0000 L CNN "Capacitance"
-F 5 "25V" H 4315 4984 50  0000 L CNN "Rating"
-	1    4200 5075
-	-1   0    0    -1
-$EndComp
 Wire Wire Line
 	4925 5225 4925 5275
@@
 	1    0    0    -1
 $EndComp
+$Comp
+L custom:GRM1555C1H120JA01D C51
+U 1 1 5D62AE5C
+P 4925 5075
+F 0 "C51" H 5075 5125 50  0000 L BNN
+F 1 "GRM1555C1H120JA01D" H 4175 4625 50  0001 L BNN
+F 2 "Capacitor_SMD:C_0402_1005Metric" H 4175 4525 50  0001 L BNN
+F 3 "" H 4175 4425 50  0001 L BNN
+F 4 "12pF" H 5050 5050 50  0000 L BNN "Capacitance"
+F 5 "50V" H 5050 4975 50  0000 L BNN "RATING"
+F 6 "C0G" H 5125 4925 50  0001 C CNN "DIELECTRIC"
+F 7 "5%" H 5125 4850 50  0001 C CNN "TOLERANCE"
+	1    4925 5075
+	1    0    0    -1
+$EndComp
+$Comp
+L custom:GRM1555C1H120JA01D C38
+U 1 1 5D62BA28
+P 4200 5075
+F 0 "C38" H 4350 5125 50  0000 L BNN
+F 1 "GRM1555C1H120JA01D" H 3450 4625 50  0001 L BNN
+F 2 "Capacitor_SMD:C_0402_1005Metric" H 3450 4525 50  0001 L BNN
+F 3 "" H 3450 4425 50  0001 L BNN
+F 4 "12pF" H 4300 5050 50  0000 L BNN "Capacitance"
+F 5 "50V" H 4350 4975 50  0000 L BNN "RATING"
+F 6 "C0G" H 4400 4925 50  0001 C CNN "DIELECTRIC"
+F 7 "5%" H 4400 4850 50  0001 C CNN "TOLERANCE"
+	1    4200 5075
+	-1   0    0    -1
+$EndComp
 $EndSCHEMATC
