File: INTERFACE.sch (KiCad schematic (older format))
At the start: 6 parts

Commit message: automated commit
Other:
- moved on the sheet: Q?B

Commit message: automated commit
Parts:
- gave numbers to parts that had none: 5
Other:
- moved on the sheet: J8, Q11A, Q11B, R65, TP38, TP39
