File: INTERFACE.sch (KiCad schematic (older format))
At the start: 5 parts, among them J8 10x2_1&3_loaded_2.5mm_0.1in_f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, Q11 DMG6602

Commit message: automated commit
Parts:
- renumbered J8 to J6, Q11 to Q15, R65 to R89, TP38 to TP44, TP39 to TP45
Changed lines of the file:
@@
 P 3500 3150
 AR Path="/6285D04D" Ref="#PWR?"  Part="1"
-AR Path="/627E3ADC/6285D04D" Ref="#PWR0155"  Part="1"
-F 0 "#PWR0155" H 3500 2900 50  0001 C CNN
+AR Path="/627E3ADC/6285D04D" Ref="#PWR0169"  Part="1"
+F 0 "#PWR0169" H 3500 2900 50  0001 C CNN
 F 1 "GND" H 3500 3000 50  0000 C CNN
 F 2 "" H 3500 3150 50  0001 C CNN
@@
 P 5550 2025
 AR Path="/6285D053" Ref="#PWR?"  Part="1"
-AR Path="/627E3ADC/6285D053" Ref="#PWR0154"  Part="1"
-F 0 "#PWR0154" H 5550 1875 50  0001 C CNN
+AR Path="/627E3ADC/6285D053" Ref="#PWR0168"  Part="1"
+F 0 "#PWR0168" H 5550 1875 50  0001 C CNN
 F 1 "+24V" H 5550 2165 50  0000 C CNN
 F 2 "" H 5550 2025 50  0001 C CNN
@@
 P 5000 4100
 AR Path="/6285D0A2" Ref="J?"  Part="1"
-AR Path="/627E3ADC/6285D0A2" Ref="J8"  Part="1"
-F 0 "J8" H 5150 5775 60  0000 C CNN
+AR Path="/627E3ADC/6285D0A2" Ref="J6"  Part="1"
+F 0 "J6" H 5150 5775 60  0000 C CNN
 F 1 "10x2_1&3_loaded_2.5mm_0.1in_female_header" H 5050 2400 60  0000 C CNN
 F 2 "" H 5000 4750 60  0001 C CNN
@@
 P 3500 2250
 AR Path="/6285D1B8" Ref="TP?"  Part="1"
-AR Path="/627E3ADC/6285D1B8" Ref="TP38"  Part="1"
-F 0 "TP38" H 3500 2450 50  0000 C CNN
+AR Path="/627E3ADC/6285D1B8" Ref="TP44"  Part="1"
+F 0 "TP44" H 3500 2450 50  0000 C CNN
 F 1 "TestPoint" H 3250 2300 50  0001 C CNN
 F 2 "" H 3700 2250 50  0001 C CNN
@@
 P 3100 2850
 AR Path="/6285D1F0" Ref="R?"  Part="1"
-AR Path="/627E3ADC/6285D1F0" Ref="R65"  Part="1"
-F 0 "R65" V 3220 2750 50  0000 L BNN
+AR Path="/627E3ADC/6285D1F0" Ref="R89"  Part="1"
+F 0 "R89" V 3220 2750 50  0000 L BNN
 F 1 "CRG0603F4K7" H 2350 2400 50  0001 L BNN
 F 2 "Resistor_SMD:R_0603_1608Metric" H 2350 2300 50  0001 L BNN
@@
 P 3400 2600
 AR Path="/6285D241" Ref="Q?"  Part="1"
-AR Path="/627E3ADC/6285D241" Ref="Q11"  Part="1"
-F 0 "Q11" H 3600 2675 50  0000 L CNN
+AR Path="/627E3ADC/6285D241" Ref="Q15"  Part="1"
+F 0 "Q15" H 3600 2675 50  0000 L CNN
 F 1 "DMG6602" H 3600 2600 50  0000 L CNN
 F 2 "Package_TO_SOT_SMD:TSOT-23-6" H 3600 2525 50  0001 L CIN
@@
 P 2500 1500
 AR Path="/6285D247" Ref="Q?"  Part="2"
-AR Path="/627E3ADC/6285D247" Ref="Q11"  Part="2"
-F 0 "Q11" H 2700 1575 50  0000 L CNN
+AR Path="/627E3ADC/6285D247" Ref="Q15"  Part="2"
+F 0 "Q15" H 2700 1575 50  0000 L CNN
 F 1 "DMG6602" H 2700 1500 50  0000 L CNN
 F 2 "Package_TO_SOT_SMD:TSOT-23-6" H 2700 1425 50  0001 L CIN
@@
 P 2850 2550
 AR Path="/5D2073A5" Ref="TP?"  Part="1"
-AR Path="/627E3ADC/5D2073A5" Ref="TP39"  Part="1"
-F 0 "TP39" H 2850 2750 50  0000 C CNN
+AR Path="/627E3ADC/5D2073A5" Ref="TP45"  Part="1"
+F 0 "TP45" H 2850 2750 50  0000 C CNN
 F 1 "TestPoint" H 2600 2600 50  0001 C CNN
 F 2 "" H 3050 2550 50  0001 C CNN

Commit message: automated commit
Parts:
- R89: Resistance 4.7k -> (none); TOLERANCE (none) -> 5%; VALUE (none) -> 4k7
Changed lines of the file:
@@
 P 3500 3150
 AR Path="/6285D04D" Ref="#PWR?"  Part="1"
-AR Path="/627E3ADC/6285D04D" Ref="#PWR0169"  Part="1"
-F 0 "#PWR0169" H 3500 2900 50  0001 C CNN
+AR Path="/627E3ADC/6285D04D" Ref="#PWR0167"  Part="1"
+F 0 "#PWR0167" H 3500 2900 50  0001 C CNN
 F 1 "GND" H 3500 3000 50  0000 C CNN
 F 2 "" H 3500 3150 50  0001 C CNN
@@
 P 5550 2025
 AR Path="/6285D053" Ref="#PWR?"  Part="1"
-AR Path="/627E3ADC/6285D053" Ref="#PWR0168"  Part="1"
-F 0 "#PWR0168" H 5550 1875 50  0001 C CNN
+AR Path="/627E3ADC/6285D053" Ref="#PWR0166"  Part="1"
+F 0 "#PWR0166" H 5550 1875 50  0001 C CNN
 F 1 "+24V" H 5550 2165 50  0000 C CNN
 F 2 "" H 5550 2025 50  0001 C CNN
@@
 F 3 "~" H 3700 2250 50  0001 C CNN
 	1    3500 2250
-	1    0    0    -1
-$EndComp
-$Comp
-L custom:CRG0603F4K7 R?
-U 1 1 6285D1F0
-P 3100 2850
-AR Path="/6285D1F0" Ref="R?"  Part="1"
-AR Path="/627E3ADC/6285D1F0" Ref="R89"  Part="1"
-F 0 "R89" V 3220 2750 50  0000 L BNN
-F 1 "CRG0603F4K7" H 2350 2400 50  0001 L BNN
-F 2 "Resistor_SMD:R_0603_1608Metric" H 2350 2300 50  0001 L BNN
-F 3 "datasheets/PYu-RC_Group_51_RoHS_L_9.pdf" H 2350 2200 50  0001 L BNN
-F 4 "4.7k" V 3120 2790 39  0000 L BNN "Resistance"
-	1    3100 2850
 	1    0    0    -1
 $EndComp
@@
 Text GLabel 4500 5650 0    50   Input ~ 0
 COL27
+$Comp
+L custom:CRG0603F4K7 R89
+U 1 1 5D0BFF14
+P 3100 2850
+F 0 "R89" H 3170 2870 50  0000 L BNN
+F 1 "CRG0603F4K7" H 2400 2450 50  0001 L BNN
+F 2 "Resistor_SMD:R_0603_1608Metric" H 2400 2350 50  0001 L BNN
+F 3 "/home/dj/datasheets/Pyu-RC_Group_51_RoHS_L_9.pdf" H 2400 2250 50  0001 L BNN
+F 4 "4k7" V 3100 2850 50  0000 C CNN "VALUE"
+F 5 "5%" H 3220 2810 50  0000 C CNN "TOLERANCE"
+	1    3100 2850
+	1    0    0    -1
+$EndComp
 $EndSCHEMATC

Commit message: automated commit
Parts:
- renumbered J6 to J11, R89 to R85, TP44 to TP56, TP45 to TP57
Changed lines of the file:
@@
 P 5000 4100
 AR Path="/6285D0A2" Ref="J?"  Part="1"
-AR Path="/627E3ADC/6285D0A2" Ref="J6"  Part="1"
-F 0 "J6" H 5150 5775 60  0000 C CNN
+AR Path="/627E3ADC/6285D0A2" Ref="J11"  Part="1"
+F 0 "J11" H 5150 5775 60  0000 C CNN
 F 1 "10x2_1&3_loaded_2.5mm_0.1in_female_header" H 5050 2400 60  0000 C CNN
 F 2 "" H 5000 4750 60  0001 C CNN
@@
 P 3500 2250
 AR Path="/6285D1B8" Ref="TP?"  Part="1"
-AR Path="/627E3ADC/6285D1B8" Ref="TP44"  Part="1"
-F 0 "TP44" H 3500 2450 50  0000 C CNN
+AR Path="/627E3ADC/6285D1B8" Ref="TP56"  Part="1"
+F 0 "TP56" H 3500 2450 50  0000 C CNN
 F 1 "TestPoint" H 3250 2300 50  0001 C CNN
 F 2 "" H 3700 2250 50  0001 C CNN
@@
 P 2850 2550
 AR Path="/5D2073A5" Ref="TP?"  Part="1"
-AR Path="/627E3ADC/5D2073A5" Ref="TP45"  Part="1"
-F 0 "TP45" H 2850 2750 50  0000 C CNN
+AR Path="/627E3ADC/5D2073A5" Ref="TP57"  Part="1"
+F 0 "TP57" H 2850 2750 50  0000 C CNN
 F 1 "TestPoint" H 2600 2600 50  0001 C CNN
 F 2 "" H 3050 2550 50  0001 C CNN
@@
 COL27
 $Comp
-L custom:CRG0603F4K7 R89
+L custom:CRG0603F4K7 R85
 U 1 1 5D0BFF14
 P 3100 2850
-F 0 "R89" H 3170 2870 50  0000 L BNN
+F 0 "R85" H 3170 2870 50  0000 L BNN
 F 1 "CRG0603F4K7" H 2400 2450 50  0001 L BNN
 F 2 "Resistor_SMD:R_0603_1608Metric" H 2400 2350 50  0001 L BNN

Commit message: automated commit
Parts:
- removed J11: 10x2_1&3_loaded_2.5mm_0.1in_female_header, symbol custom:10x2_1&3_loaded_2.5mm_0.1in_female_header
- added J11: 3x32_1&3_loaded_2.5mm_0.1in_female_header, custom:32x3_POP_1_3, symbol custom:3x32_1&3_loaded_2.5mm_0.1in_female_header
- TP61: renamed from TP56; footprint (none) -> custom:TestPoint_THTPad_D1.0mm_Drill0.5mm
- TP62: renamed from TP57; footprint (none) -> custom:TestPoint_THTPad_D1.0mm_Drill0.5mm
Connections:
- net +24V: now also J11.3, J11.4
- net COL00: now also J11.37
- net COL01: now also J11.38
- net COL02: now also J11.39
- net COL03: now also J11.40
- net COL04: now also J11.41
- net COL05: now also J11.42
- net COL06: now also J11.43
- net COL07: now also J11.44
- net COL08: now also J11.45
- net COL09: now also J11.46
- net COL10: now also J11.47
- net COL11: now also J11.48
- net COL12: now also J11.49
- net COL13: now also J11.50
- net COL14: now also J11.51
- net COL15: now also J11.52
- net COL16: now also J11.53
- net COL17: now also J11.54
- net COL18: now also J11.55
- net COL19: now also J11.56
- net COL20: now also J11.57
- net COL21: now also J11.58
- net COL22: now also J11.59
- net COL23: now also J11.60
- net COL24: now also J11.61
- net COL25: now also J11.62
- net COL26: now also J11.63
- net COL27: now also J11.64
- net ROW00N: now also J11.36
- net ROW00P: now also J11.35
- net ROW01N: now also J11.6
- net ROW01P: now also J11.5
- net ROW02N: now also J11.34
- net ROW02P: now also J11.33
- net ROW03N: now also J11.8
- net ROW03P: now also J11.7
- net ROW04N: now also J11.32
- net ROW04P: now also J11.31
- net ROW05N: now also J11.10
- net ROW05P: now also J11.9
- net ROW06N: now also J11.30
- net ROW06P: now also J11.29
- net ROW07N: now also J11.12
- net ROW07P: now also J11.11
- net ROW08N: now also J11.28
- net ROW08P: now also J11.27
- net ROW09N: now also J11.14
- net ROW09P: now also J11.13
- net ROW10N: now also J11.26
- net ROW10P: now also J11.25
- net ROW11N: now also J11.16
- net ROW11P: now also J11.15
- net ROW12N: now also J11.24
- net ROW12P: now also J11.23
- net ROW13N: now also J11.18
- net ROW13P: now also J11.17
- net ROW14N: now also J11.22
- net ROW14P: now also J11.21
- net ROW15N: now also J11.20
- net ROW15P: now also J11.19
- net at Q15.6 (D), TP61.1: now also J11.1, J11.2

Commit message: automated commit
Parts:
- renumbered R85 to R93
Changed lines of the file:
@@
 P 3500 3150
 AR Path="/6285D04D" Ref="#PWR?"  Part="1"
-AR Path="/627E3ADC/6285D04D" Ref="#PWR0167"  Part="1"
-F 0 "#PWR0167" H 3500 2900 50  0001 C CNN
+AR Path="/627E3ADC/6285D04D" Ref="#PWR0169"  Part="1"
+F 0 "#PWR0169" H 3500 2900 50  0001 C CNN
 F 1 "GND" H 3500 3000 50  0000 C CNN
 F 2 "" H 3500 3150 50  0001 C CNN
@@
 P 5550 2025
 AR Path="/6285D053" Ref="#PWR?"  Part="1"
-AR Path="/627E3ADC/6285D053" Ref="#PWR0166"  Part="1"
-F 0 "#PWR0166" H 5550 1875 50  0001 C CNN
+AR Path="/627E3ADC/6285D053" Ref="#PWR0168"  Part="1"
+F 0 "#PWR0168" H 5550 1875 50  0001 C CNN
 F 1 "+24V" H 5550 2165 50  0000 C CNN
 F 2 "" H 5550 2025 50  0001 C CNN
@@
 $EndComp
 $Comp
-L custom:CRG0603F4K7 R85
+L custom:CRG0603F4K7 R93
 U 1 1 5D0BFF14
 P 3100 2850
-F 0 "R85" H 3170 2870 50  0000 L BNN
+F 0 "R93" H 3170 2870 50  0000 L BNN
 F 1 "CRG0603F4K7" H 2400 2450 50  0001 L BNN
 F 2 "Resistor_SMD:R_0603_1608Metric" H 2400 2350 50  0001 L BNN
