File: PANEL_EXTENSION.sch (KiCad schematic (older format))
At the start: 19 parts

Commit message: automated commit
Parts:
- removed J? (x2): Conn_01x03_Male, symbol Connector:Conn_01x03_Male
- removed TP? (x2): TestPoint, symbol Connector:TestPoint
- added J? (x2): Conn_01x03_Male, symbol Connector:Conn_01x03_Male
- added TP? (x2): TestPoint, symbol Connector:TestPoint
Connections:
- net COL_DATA: now also J?.2 (Pin_2)
- net COL_IN: now also J?.1 (Pin_1), TP?.1
- net COL_OUT: now also J?.3 (Pin_3), TP?.1
- net ROW_DATA: now also J?.2 (Pin_2)
- net ROW_IN: now also J?.1 (Pin_1)
- net ROW_OUT: now also J?.3 (Pin_3)
Other:
- moved on the sheet: J?, R?, TP?, U?

Commit message: automated commit
Parts:
- removed J?: Conn_01x03_Male, symbol Connector:Conn_01x03_Male
- removed TP? (x4): TestPoint, symbol Connector:TestPoint
- added J?: Conn_01x03_Male, symbol Connector:Conn_01x03_Male
- added TP? (x7): TestPoint, symbol Connector:TestPoint
Connections:
- net COL_DATA: now also J?.2 (Pin_2), TP?.1
- net COL_IN: now also J?.1 (Pin_1), TP?.1
- net COL_OUT: now also J?.3 (Pin_3), TP?.1
- net GND: now also TP?.1
- net ROW_DATA: now also TP?.1
- net ROW_IN: now also TP?.1
- net ROW_OUT: now also TP?.1
Other:
- note removed: "SPACE 1x3 HEADERS SO\nAS TO PREVENT A JUMPER\nFROM CONNECTING AN\nINVALID SET OF PINS"
- moved on the sheet: J?, R?, TP?, U?

Commit message: automated commit
Parts:
- gave numbers to parts that had none: 22
Other:
- moved on the sheet: J5, J6, J7, R63, R64, TP24, TP25, TP26, TP27, TP28, TP29, TP30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
