File: PANEL_EXTENSION.sch (KiCad schematic (older format))
At the start: 22 parts, among them J5 Conn_01x03_Male, J6 Conn_01x08_Male, J7 Conn_01x03_Male, U10 CM1293A-04SO, U11 CM1293A-04SO, U9 CM1293A-04SO

Commit message: automated commit
Connections:
- net labels added: ROW_ON
- net labels removed: !ROW_RESET
Changed lines of the file:
@@
 U 1 1 621E7976
 P 7375 5125
-F 0 "TP36" V 7400 5400 50  0000 L BNN
+F 0 "TP36" V 7400 5325 50  0000 L BNN
 F 1 "TestPoint" H 7125 5175 50  0001 C CNN
 F 2 "" H 7575 5125 50  0001 C CNN
@@
 U 1 1 621E797C
 P 7275 5125
-F 0 "TP35" V 7300 5400 50  0000 L BNN
+F 0 "TP35" V 7300 5325 50  0000 L BNN
 F 1 "TestPoint" H 7025 5175 50  0001 C CNN
 F 2 "" H 7475 5125 50  0001 C CNN
@@
 U 1 1 621E7982
 P 7175 5125
-F 0 "TP34" V 7200 5400 50  0000 L BNN
+F 0 "TP34" V 7200 5325 50  0000 L BNN
 F 1 "TestPoint" H 6925 5175 50  0001 C CNN
 F 2 "" H 7375 5125 50  0001 C CNN
@@
 U 1 1 621E7988
 P 7075 5125
-F 0 "TP33" V 7100 5400 50  0000 L BNN
+F 0 "TP33" V 7100 5325 50  0000 L BNN
 F 1 "TestPoint" H 6825 5175 50  0001 C CNN
 F 2 "" H 7275 5125 50  0001 C CNN
@@
 U 1 1 621E798E
 P 6975 5125
-F 0 "TP32" V 7000 5400 50  0000 L BNN
+F 0 "TP32" V 7000 5325 50  0000 L BNN
 F 1 "TestPoint" H 6725 5175 50  0001 C CNN
 F 2 "" H 7175 5125 50  0001 C CNN
@@
 U 1 1 621E7994
 P 6875 5125
-F 0 "TP31" V 6900 5400 50  0000 L BNN
+F 0 "TP31" V 6900 5325 50  0000 L BNN
 F 1 "TestPoint" H 6625 5175 50  0001 C CNN
 F 2 "" H 7075 5125 50  0001 C CNN
@@
 U 1 1 621E799A
 P 6775 5125
-F 0 "TP30" V 6800 5400 50  0000 L BNN
+F 0 "TP30" V 6800 5325 50  0000 L BNN
 F 1 "TestPoint" H 6525 5175 50  0001 C CNN
 F 2 "" H 6975 5125 50  0001 C CNN
@@
 ROW_SHCP
 Text GLabel 7575 4525 2    50   UnSpc ~ 0
-!ROW_RESET
+ROW_ON
 Text GLabel 7575 4725 2    50   UnSpc ~ 0
 COL_SHCP
@@
 ROW_SHCP
 Text GLabel 6600 2550 0    50   Input ~ 0
-!ROW_RESET
+ROW_ON
 Text GLabel 6600 2750 0    50   Input ~ 0
 COL_SHCP
@@
 U 1 1 5D298B1C
 P 7475 5125
-F 0 "TP37" V 7500 5400 50  0000 L BNN
+F 0 "TP37" V 7500 5325 50  0000 L BNN
 F 1 "TestPoint" H 7225 5175 50  0001 C CNN
 F 2 "" H 7675 5125 50  0001 C CNN

Commit message: automated commit
Parts:
- removed J5, J7: Conn_01x03_Male, symbol Connector:Conn_01x03_Male
- removed R63, R64: CRG0603F4K7, Resistor_SMD:R_0603_1608Metric, symbol custom:CRG0603F4K7
- removed TP26, TP27, TP28, TP29: TestPoint, symbol Connector:TestPoint
- added C85, C86: CL10B104KO8NNNC, Capacitor_SMD:C_0603_1608Metric, symbol custom:CL10B104KO8NNNC
- added R85, R86, R87, R88: CRG0603F4K7, Resistor_SMD:R_0603_1608Metric, symbol custom:CRG0603F4K7
- added TP34, TP35: TestPoint, symbol Connector:TestPoint
- added U20, U21: SGM3157YC6, Package_TO_SOT_SMD:SOT-363_SC-70-6, symbol custom:SGM3157YC6
- renumbered J6 to J5, TP24 to TP32, TP25 to TP33, TP30 to TP36, TP31 to TP37, TP32 to TP38, TP33 to TP39, TP34 to TP40, TP35 to TP41, TP36 to TP42, TP37 to TP43, U9 to U22, U10 to U23, U11 to U24
Connections:
- net labels added: COL_MODE_SEL, ROW_MODE_SEL
- net labels removed: CONN_GND
- wire segments 81 -> 104
- no-connect marks 0 -> 2
Other:
- note added: "CONN_GND"
- moved on the sheet: J5, TP32, TP33, TP36, TP37, TP38, TP39, TP40, TP41, TP42, TP43, U22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

Commit message: automated commit
Parts:
- removed U23: CM1293A-04SO, symbol custom:CM1293A-04SO_ALTERNATE_SYMBOL
Other:
- moved on the sheet: C85, C86, J5, R85, R86, R87, R88, TP32, TP33, TP34, TP35, TP36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

Commit message: automated commit
Parts:
- renumbered U22 to U21, U21 to U22, U24 to U23
Changed lines of the file:
@@
 	6100 4575 6000 4575
 $Comp
-L power:+3V3 #PWR0162
+L power:+3V3 #PWR0157
 U 1 1 621E790F
 P 6000 4525
-F 0 "#PWR0162" H 6000 4375 50  0001 C CNN
+F 0 "#PWR0157" H 6000 4375 50  0001 C CNN
 F 1 "+3V3" H 6000 4665 50  0000 C CNN
 F 2 "" H 6000 4525 50  0001 C CNN
@@
 	6100 5475 6000 5475
 $Comp
-L power:+3V3 #PWR0165
+L power:+3V3 #PWR0163
 U 1 1 621E7962
 P 6000 5425
-F 0 "#PWR0165" H 6000 5275 50  0001 C CNN
+F 0 "#PWR0163" H 6000 5275 50  0001 C CNN
 F 1 "+3V3" H 6000 5565 50  0000 C CNN
 F 2 "" H 6000 5425 50  0001 C CNN
@@
 	6000 5825 6000 5775
 $Comp
-L power:GND #PWR0167
+L power:GND #PWR0165
 U 1 1 621E796A
 P 6000 5825
-F 0 "#PWR0167" H 6000 5575 50  0001 C CNN
+F 0 "#PWR0165" H 6000 5575 50  0001 C CNN
 F 1 "GND" H 6000 5675 50  0000 C CNN
 F 2 "" H 6000 5825 50  0001 C CNN
@@
 $EndComp
 $Comp
-L custom:CM1293A-04SO_ALTERNATE_SYMBOL U24
+L custom:CM1293A-04SO_ALTERNATE_SYMBOL U23
 U 1 1 621E7970
 P 6450 5625
-F 0 "U24" H 6400 5875 60  0000 C CNN
+F 0 "U23" H 6400 5875 60  0000 C CNN
 F 1 "CM1293A-04SO" H 6550 5375 60  0000 C CNN
 F 2 "" H 6300 5525 60  0001 C CNN
@@
 	6000 4925 6000 4875
 $Comp
-L power:GND #PWR0163
+L power:GND #PWR0160
 U 1 1 621E79BB
 P 6000 4925
-F 0 "#PWR0163" H 6000 4675 50  0001 C CNN
+F 0 "#PWR0160" H 6000 4675 50  0001 C CNN
 F 1 "GND" H 6000 4775 50  0000 C CNN
 F 2 "" H 6000 4925 50  0001 C CNN
@@
 $EndComp
 $Comp
-L custom:CM1293A-04SO_ALTERNATE_SYMBOL U22
+L custom:CM1293A-04SO_ALTERNATE_SYMBOL U21
 U 1 1 621E79C1
 P 6450 4725
-F 0 "U22" H 6400 4975 60  0000 C CNN
+F 0 "U21" H 6400 4975 60  0000 C CNN
 F 1 "CM1293A-04SO" H 6450 4475 60  0000 C CNN
 F 2 "" H 6300 4625 60  0001 C CNN
@@
 	1875 4950 2500 4950
 $Comp
-L custom:SGM3157YC6 U21
+L custom:SGM3157YC6 U22
 U 1 1 5D536F11
 P 3325 5000
-F 0 "U21" H 3075 5250 50  0000 L BNN
+F 0 "U22" H 3075 5250 50  0000 L BNN
 F 1 "SGM3157YC6" H 3075 4800 50  0000 L BNN
 F 2 "Package_TO_SOT_SMD:SOT-363_SC-70-6" H 3075 4700 50  0001 L BNN
@@
 	2975 4850 2875 4850
 $Comp
-L power:+3V3 #PWR0156
+L power:+3V3 #PWR0158
 U 1 1 5D54B19A
 P 2875 4800
-F 0 "#PWR0156" H 2875 4650 50  0001 C CNN
+F 0 "#PWR0158" H 2875 4650 50  0001 C CNN
 F 1 "+3V3" H 2875 4940 50  0000 C CNN
 F 2 "" H 2875 4800 50  0001 C CNN
@@
 	3775 5100 3775 5050
 $Comp
-L power:GND #PWR0159
+L power:GND #PWR0161
 U 1 1 5D54CF05
 P 3775 5100
-F 0 "#PWR0159" H 3775 4850 50  0001 C CNN
+F 0 "#PWR0161" H 3775 4850 50  0001 C CNN
 F 1 "GND" H 3775 4950 50  0000 C CNN
 F 2 "" H 3775 5100 50  0001 C CNN
@@
 	2875 5475 2875 5550
 $Comp
-L power:GND #PWR0161
+L power:GND #PWR0164
 U 1 1 5D57DDBD
 P 2700 5600
-F 0 "#PWR0161" H 2700 5350 50  0001 C CNN
+F 0 "#PWR0164" H 2700 5350 50  0001 C CNN
 F 1 "GND" H 2700 5450 50  0000 C CNN
 F 2 "" H 2700 5600 50  0001 C CNN
@@
 	2900 3100 2900 3175
 $Comp
-L power:GND #PWR0155
+L power:GND #PWR0156
 U 1 1 5D5DFF1F
 P 2725 3225
-F 0 "#PWR0155" H 2725 2975 50  0001 C CNN
+F 0 "#PWR0156" H 2725 2975 50  0001 C CNN
 F 1 "GND" H 2725 3075 50  0000 C CNN
 F 2 "" H 2725 3225 50  0001 C CNN
@@
 	2700 5550 2875 5550
 $Comp
-L power:GND #PWR0158
+L power:GND #PWR0155
 U 1 1 5D5EA3CE
 P 7325 3200
-F 0 "#PWR0158" H 7325 2950 50  0001 C CNN
+F 0 "#PWR0155" H 7325 2950 50  0001 C CNN
 F 1 "GND" H 7325 3050 50  0000 C CNN
 F 2 "" H 7325 3200 50  0001 C CNN
@@
 	4700 4875 4700 4825
 $Comp
-L power:+3V3 #PWR0157
+L power:+3V3 #PWR0159
 U 1 1 5D5FC7EC
 P 4700 4825
-F 0 "#PWR0157" H 4700 4675 50  0001 C CNN
+F 0 "#PWR0159" H 4700 4675 50  0001 C CNN
 F 1 "+3V3" H 4700 4965 50  0000 C CNN
 F 2 "" H 4700 4825 50  0001 C CNN
@@
 	4700 5225 4700 5175
 $Comp
-L power:GND #PWR0160
+L power:GND #PWR0162
 U 1 1 5D5FFF0B
 P 4700 5225
-F 0 "#PWR0160" H 4700 4975 50  0001 C CNN
+F 0 "#PWR0162" H 4700 4975 50  0001 C CNN
 F 1 "GND" H 4700 5075 50  0000 C CNN
 F 2 "" H 4700 5225 50  0001 C CNN

Commit message: automated commit
Parts:
- renumbered C85 to C86, C86 to C87, J5 to J10, R85 to R81, R86 to R82, R87 to R83, R88 to R84, TP32 to TP44, TP33 to TP45, TP34 to TP46, TP35 to TP47, TP36 to TP48, TP37 to TP49, TP38 to TP50, TP39 to TP51, TP40 to TP52, TP41 to TP53, TP42 to TP54, TP43 to TP55
Changed lines of the file:
@@
 $EndComp
 $Comp
-L Connector:TestPoint TP42
+L Connector:TestPoint TP54
 U 1 1 621E7976
 P 8150 5375
-F 0 "TP42" V 8175 5575 50  0000 L BNN
+F 0 "TP54" V 8175 5575 50  0000 L BNN
 F 1 "TestPoint" H 7900 5425 50  0001 C CNN
 F 2 "" H 8350 5375 50  0001 C CNN
@@
 $EndComp
 $Comp
-L Connector:TestPoint TP41
+L Connector:TestPoint TP53
 U 1 1 621E797C
 P 8050 5375
-F 0 "TP41" V 8075 5575 50  0000 L BNN
+F 0 "TP53" V 8075 5575 50  0000 L BNN
 F 1 "TestPoint" H 7800 5425 50  0001 C CNN
 F 2 "" H 8250 5375 50  0001 C CNN
@@
 $EndComp
 $Comp
-L Connector:TestPoint TP40
+L Connector:TestPoint TP52
 U 1 1 621E7982
 P 7950 5375
-F 0 "TP40" V 7975 5575 50  0000 L BNN
+F 0 "TP52" V 7975 5575 50  0000 L BNN
 F 1 "TestPoint" H 7700 5425 50  0001 C CNN
 F 2 "" H 8150 5375 50  0001 C CNN
@@
 $EndComp
 $Comp
-L Connector:TestPoint TP39
+L Connector:TestPoint TP51
 U 1 1 621E7988
 P 7850 5375
-F 0 "TP39" V 7875 5575 50  0000 L BNN
+F 0 "TP51" V 7875 5575 50  0000 L BNN
 F 1 "TestPoint" H 7600 5425 50  0001 C CNN
 F 2 "" H 8050 5375 50  0001 C CNN
@@
 $EndComp
 $Comp
-L Connector:TestPoint TP38
+L Connector:TestPoint TP50
 U 1 1 621E798E
 P 7750 5375
-F 0 "TP38" V 7775 5575 50  0000 L BNN
+F 0 "TP50" V 7775 5575 50  0000 L BNN
 F 1 "TestPoint" H 7500 5425 50  0001 C CNN
 F 2 "" H 7950 5375 50  0001 C CNN
@@
 $EndComp
 $Comp
-L Connector:TestPoint TP37
+L Connector:TestPoint TP49
 U 1 1 621E7994
 P 7650 5375
-F 0 "TP37" V 7675 5575 50  0000 L BNN
+F 0 "TP49" V 7675 5575 50  0000 L BNN
 F 1 "TestPoint" H 7400 5425 50  0001 C CNN
 F 2 "" H 7850 5375 50  0001 C CNN
@@
 $EndComp
 $Comp
-L Connector:TestPoint TP36
+L Connector:TestPoint TP48
 U 1 1 621E799A
 P 7550 5375
-F 0 "TP36" V 7575 5575 50  0000 L BNN
+F 0 "TP48" V 7575 5575 50  0000 L BNN
 F 1 "TestPoint" H 7300 5425 50  0001 C CNN
 F 2 "" H 7750 5375 50  0001 C CNN
@@
 	7550 4575 7550 5375
 $Comp
-L Connector:Conn_01x08_Male J5
+L Connector:Conn_01x08_Male J10
 U 1 1 621E7A0B
 P 7750 2650
-F 0 "J5" H 7750 3050 50  0000 C CNN
+F 0 "J10" H 7750 3050 50  0000 C CNN
 F 1 "Conn_01x08_Male" H 7325 2625 50  0000 C CNN
 F 2 "" H 7750 2650 50  0001 C CNN
@@
 	7550 4575 9325 4575
 $Comp
-L Connector:TestPoint TP43
+L Connector:TestPoint TP55
 U 1 1 5D298B1C
 P 8250 5375
-F 0 "TP43" V 8275 5575 50  0000 L BNN
+F 0 "TP55" V 8275 5575 50  0000 L BNN
 F 1 "TestPoint" H 8000 5425 50  0001 C CNN
 F 2 "" H 8450 5375 50  0001 C CNN
@@
 	8250 5275 9325 5275
 $Comp
-L Connector:TestPoint TP33
+L Connector:TestPoint TP45
 U 1 1 5D2A7B5A
 P 3875 2375
-F 0 "TP33" V 3900 2575 50  0000 L BNN
+F 0 "TP45" V 3900 2575 50  0000 L BNN
 F 1 "TestPoint" H 3625 2425 50  0001 C CNN
 F 2 "" H 4075 2375 50  0001 C CNN
@@
 $EndComp
 $Comp
-L Connector:TestPoint TP32
+L Connector:TestPoint TP44
 U 1 1 5D2A7B60
 P 3775 2375
-F 0 "TP32" V 3800 2575 50  0000 L BNN
+F 0 "TP44" V 3800 2575 50  0000 L BNN
 F 1 "TestPoint" H 3525 2425 50  0001 C CNN
 F 2 "" H 3975 2375 50  0001 C CNN
@@
 	3875 2575 3675 2575
 $Comp
-L Connector:TestPoint TP35
+L Connector:TestPoint TP47
 U 1 1 5D55DA0B
 P 3875 4750
-F 0 "TP35" V 3900 4950 50  0000 L BNN
+F 0 "TP47" V 3900 4950 50  0000 L BNN
 F 1 "TestPoint" H 3625 4800 50  0001 C CNN
 F 2 "" H 4075 4750 50  0001 C CNN
@@
 $EndComp
 $Comp
-L Connector:TestPoint TP34
+L Connector:TestPoint TP46
 U 1 1 5D55DA11
 P 3775 4750
-F 0 "TP34" V 3800 4950 50  0000 L BNN
+F 0 "TP46" V 3800 4950 50  0000 L BNN
 F 1 "TestPoint" H 3525 4800 50  0001 C CNN
 F 2 "" H 3975 4750 50  0001 C CNN
@@
 $EndComp
 $Comp
-L custom:CRG0603F4K7 R87
+L custom:CRG0603F4K7 R83
 U 1 1 5D5808FB
 P 2500 5325
-F 0 "R87" H 2570 5345 50  0000 L BNN
+F 0 "R83" H 2570 5345 50  0000 L BNN
 F 1 "CRG0603F4K7" H 1800 4925 50  0001 L BNN
 F 2 "Resistor_SMD:R_0603_1608Metric" H 1800 4825 50  0001 L BNN
@@
 $EndComp
 $Comp
-L custom:CRG0603F4K7 R88
+L custom:CRG0603F4K7 R84
 U 1 1 5D581918
 P 2875 5325
-F 0 "R88" H 2945 5345 50  0000 L BNN
+F 0 "R84" H 2945 5345 50  0000 L BNN
 F 1 "CRG0603F4K7" H 2175 4925 50  0001 L BNN
 F 2 "Resistor_SMD:R_0603_1608Metric" H 2175 4825 50  0001 L BNN
@@
 $EndComp
 $Comp
-L custom:CRG0603F4K7 R85
+L custom:CRG0603F4K7 R81
 U 1 1 5D5DFF27
 P 2525 2950
-F 0 "R85" H 2595 2970 50  0000 L BNN
+F 0 "R81" H 2595 2970 50  0000 L BNN
 F 1 "CRG0603F4K7" H 1825 2550 50  0001 L BNN
 F 2 "Resistor_SMD:R_0603_1608Metric" H 1825 2450 50  0001 L BNN
@@
 $EndComp
 $Comp
-L custom:CRG0603F4K7 R86
+L custom:CRG0603F4K7 R82
 U 1 1 5D5DFF2F
 P 2900 2950
-F 0 "R86" H 2970 2970 50  0000 L BNN
+F 0 "R82" H 2970 2970 50  0000 L BNN
 F 1 "CRG0603F4K7" H 2200 2550 50  0001 L BNN
 F 2 "Resistor_SMD:R_0603_1608Metric" H 2200 2450 50  0001 L BNN
@@
 Wire Wire Line
 	7325 3050 7550 3050
-Text Notes 9275 5275 2    61   ~ 0
+Text Notes 9275 5275 2    60   ~ 0
 CONN_GND
-Text Notes 6400 3050 0    61   ~ 0
+Text Notes 6400 3050 0    60   ~ 0
 CONN_GND
 NoConn ~ 6350 3050
 NoConn ~ 9325 5275
 $Comp
-L custom:CL10B104KO8NNNC C86
+L custom:CL10B104KO8NNNC C87
 U 1 1 5D5FB5AF
 P 4700 5025
-F 0 "C86" H 4850 5125 50  0000 L BNN
+F 0 "C87" H 4850 5125 50  0000 L BNN
 F 1 "CL10B104KO8NNNC" H 3750 4575 50  0001 L BNN
 F 2 "Capacitor_SMD:C_0603_1608Metric" H 3750 4475 50  0001 L BNN
@@
 $EndComp
 $Comp
-L custom:CL10B104KO8NNNC C85
+L custom:CL10B104KO8NNNC C86
 U 1 1 5D605523
 P 4700 2650
-F 0 "C85" H 4850 2750 50  0000 L BNN
+F 0 "C86" H 4850 2750 50  0000 L BNN
 F 1 "CL10B104KO8NNNC" H 3750 2200 50  0001 L BNN
 F 2 "Capacitor_SMD:C_0603_1608Metric" H 3750 2100 50  0001 L BNN

Commit message: automated commit
Parts:
- J10: footprint (none) -> Connector_PinHeader_2.54mm:PinHeader_1x08_P2.54mm_Horizontal
- U21: TEXT (none) -> CM1293A
Changed lines of the file:
@@
 F 1 "CM1293A-04SO" H 6450 4475 60  0000 C CNN
 F 2 "" H 6300 4625 60  0001 C CNN
-F 3 "datasheets/CM1293A-04SO-D.PDF" H 6450 4375 60  0001 C CNN
+F 3 "~/datasheets/CM1293A-04SO-D.PDF" H 6450 4375 60  0001 C CNN
+F 4 "CM1293A" H 6450 4725 50  0001 C CNN "TEXT"
 	1    6450 4725
 	1    0    0    -1
@@
 F 0 "J10" H 7750 3050 50  0000 C CNN
 F 1 "Conn_01x08_Male" H 7325 2625 50  0000 C CNN
-F 2 "" H 7750 2650 50  0001 C CNN
+F 2 "Connector_PinHeader_2.54mm:PinHeader_1x08_P2.54mm_Horizontal" H 7750 2650 50  0001 C CNN
 F 3 "" H 7750 2650 50  0001 C CNN
 	1    7750 2650

Commit message: automated commit
Parts:
- TP49: renamed from TP44; footprint (none) -> custom:TestPoint_THTPad_D1.0mm_Drill0.5mm
- TP50: renamed from TP45; footprint (none) -> custom:TestPoint_THTPad_D1.0mm_Drill0.5mm
- TP51: renamed from TP46; footprint (none) -> custom:TestPoint_THTPad_D1.0mm_Drill0.5mm
- TP52: renamed from TP47; footprint (none) -> custom:TestPoint_THTPad_D1.0mm_Drill0.5mm
- TP53: renamed from TP48; footprint (none) -> custom:TestPoint_THTPad_D1.0mm_Drill0.5mm
- TP54: renamed from TP49; footprint (none) -> custom:TestPoint_THTPad_D1.0mm_Drill0.5mm
- TP55: renamed from TP50; footprint (none) -> custom:TestPoint_THTPad_D1.0mm_Drill0.5mm
- TP56: renamed from TP51; footprint (none) -> custom:TestPoint_THTPad_D1.0mm_Drill0.5mm
- TP57: renamed from TP52; footprint (none) -> custom:TestPoint_THTPad_D1.0mm_Drill0.5mm
- TP58: renamed from TP53; footprint (none) -> custom:TestPoint_THTPad_D1.0mm_Drill0.5mm
- TP59: renamed from TP54; footprint (none) -> custom:TestPoint_THTPad_D1.0mm_Drill0.5mm
- TP60: renamed from TP55; footprint (none) -> custom:TestPoint_THTPad_D1.0mm_Drill0.5mm
- U21: footprint (none) -> custom:SOT-457
- U23: footprint (none) -> custom:SOT-457; TEXT (none) -> CM1293A
Changed lines of the file:
@@
 F 0 "U23" H 6400 5875 60  0000 C CNN
 F 1 "CM1293A-04SO" H 6550 5375 60  0000 C CNN
-F 2 "" H 6300 5525 60  0001 C CNN
-F 3 "datasheets/CM1293A-04SO-D.PDF" H 6450 5275 60  0001 C CNN
+F 2 "custom:SOT-457" H 6300 5525 60  0001 C CNN
+F 3 "~/datasheets/CM1293A-04SO-D.PDF" H 6450 5275 60  0001 C CNN
+F 4 "CM1293A" H 6450 5625 50  0001 C CNN "TEXT"
 	1    6450 5625
 	1    0    0    -1
 $EndComp
 $Comp
-L Connector:TestPoint TP54
+L Connector:TestPoint TP59
 U 1 1 621E7976
 P 8150 5375
-F 0 "TP54" V 8175 5575 50  0000 L BNN
+F 0 "TP59" V 8175 5575 50  0000 L BNN
 F 1 "TestPoint" H 7900 5425 50  0001 C CNN
-F 2 "" H 8350 5375 50  0001 C CNN
+F 2 "custom:TestPoint_THTPad_D1.0mm_Drill0.5mm" H 8350 5375 50  0001 C CNN
 F 3 "~" H 8350 5375 50  0001 C CNN
 	1    8150 5375
@@
 $EndComp
 $Comp
-L Connector:TestPoint TP53
+L Connector:TestPoint TP58
 U 1 1 621E797C
 P 8050 5375
-F 0 "TP53" V 8075 5575 50  0000 L BNN
+F 0 "TP58" V 8075 5575 50  0000 L BNN
 F 1 "TestPoint" H 7800 5425 50  0001 C CNN
-F 2 "" H 8250 5375 50  0001 C CNN
+F 2 "custom:TestPoint_THTPad_D1.0mm_Drill0.5mm" H 8250 5375 50  0001 C CNN
 F 3 "~" H 8250 5375 50  0001 C CNN
 	1    8050 5375
@@
 $EndComp
 $Comp
-L Connector:TestPoint TP52
+L Connector:TestPoint TP57
 U 1 1 621E7982
 P 7950 5375
-F 0 "TP52" V 7975 5575 50  0000 L BNN
+F 0 "TP57" V 7975 5575 50  0000 L BNN
 F 1 "TestPoint" H 7700 5425 50  0001 C CNN
-F 2 "" H 8150 5375 50  0001 C CNN
+F 2 "custom:TestPoint_THTPad_D1.0mm_Drill0.5mm" H 8150 5375 50  0001 C CNN
 F 3 "~" H 8150 5375 50  0001 C CNN
 	1    7950 5375
@@
 $EndComp
 $Comp
-L Connector:TestPoint TP51
+L Connector:TestPoint TP56
 U 1 1 621E7988
 P 7850 5375
-F 0 "TP51" V 7875 5575 50  0000 L BNN
+F 0 "TP56" V 7875 5575 50  0000 L BNN
 F 1 "TestPoint" H 7600 5425 50  0001 C CNN
-F 2 "" H 8050 5375 50  0001 C CNN
+F 2 "custom:TestPoint_THTPad_D1.0mm_Drill0.5mm" H 8050 5375 50  0001 C CNN
 F 3 "~" H 8050 5375 50  0001 C CNN
 	1    7850 5375
@@
 $EndComp
 $Comp
-L Connector:TestPoint TP50
+L Connector:TestPoint TP55
 U 1 1 621E798E
 P 7750 5375
-F 0 "TP50" V 7775 5575 50  0000 L BNN
+F 0 "TP55" V 7775 5575 50  0000 L BNN
 F 1 "TestPoint" H 7500 5425 50  0001 C CNN
-F 2 "" H 7950 5375 50  0001 C CNN
+F 2 "custom:TestPoint_THTPad_D1.0mm_Drill0.5mm" H 7950 5375 50  0001 C CNN
 F 3 "~" H 7950 5375 50  0001 C CNN
 	1    7750 5375
@@
 $EndComp
 $Comp
-L Connector:TestPoint TP49
+L Connector:TestPoint TP54
 U 1 1 621E7994
 P 7650 5375
-F 0 "TP49" V 7675 5575 50  0000 L BNN
+F 0 "TP54" V 7675 5575 50  0000 L BNN
 F 1 "TestPoint" H 7400 5425 50  0001 C CNN
-F 2 "" H 7850 5375 50  0001 C CNN
+F 2 "custom:TestPoint_THTPad_D1.0mm_Drill0.5mm" H 7850 5375 50  0001 C CNN
 F 3 "~" H 7850 5375 50  0001 C CNN
 	1    7650 5375
@@
 $EndComp
 $Comp
-L Connector:TestPoint TP48
+L Connector:TestPoint TP53
 U 1 1 621E799A
 P 7550 5375
-F 0 "TP48" V 7575 5575 50  0000 L BNN
+F 0 "TP53" V 7575 5575 50  0000 L BNN
 F 1 "TestPoint" H 7300 5425 50  0001 C CNN
-F 2 "" H 7750 5375 50  0001 C CNN
+F 2 "custom:TestPoint_THTPad_D1.0mm_Drill0.5mm" H 7750 5375 50  0001 C CNN
 F 3 "~" H 7750 5375 50  0001 C CNN
 	1    7550 5375
@@
 F 0 "U21" H 6400 4975 60  0000 C CNN
 F 1 "CM1293A-04SO" H 6450 4475 60  0000 C CNN
-F 2 "" H 6300 4625 60  0001 C CNN
+F 2 "custom:SOT-457" H 6300 4625 60  0001 C CNN
 F 3 "~/datasheets/CM1293A-04SO-D.PDF" H 6450 4375 60  0001 C CNN
 F 4 "CM1293A" H 6450 4725 50  0001 C CNN "TEXT"
@@
 	7550 4575 9325 4575
 $Comp
-L Connector:TestPoint TP55
+L Connector:TestPoint TP60
 U 1 1 5D298B1C
 P 8250 5375
-F 0 "TP55" V 8275 5575 50  0000 L BNN
+F 0 "TP60" V 8275 5575 50  0000 L BNN
 F 1 "TestPoint" H 8000 5425 50  0001 C CNN
-F 2 "" H 8450 5375 50  0001 C CNN
+F 2 "custom:TestPoint_THTPad_D1.0mm_Drill0.5mm" H 8450 5375 50  0001 C CNN
 F 3 "~" H 8450 5375 50  0001 C CNN
 	1    8250 5375
@@
 	8250 5275 9325 5275
 $Comp
-L Connector:TestPoint TP45
+L Connector:TestPoint TP50
 U 1 1 5D2A7B5A
 P 3875 2375
-F 0 "TP45" V 3900 2575 50  0000 L BNN
+F 0 "TP50" V 3900 2575 50  0000 L BNN
 F 1 "TestPoint" H 3625 2425 50  0001 C CNN
-F 2 "" H 4075 2375 50  0001 C CNN
+F 2 "custom:TestPoint_THTPad_D1.0mm_Drill0.5mm" H 4075 2375 50  0001 C CNN
 F 3 "~" H 4075 2375 50  0001 C CNN
 	1    3875 2375
@@
 $EndComp
 $Comp
-L Connector:TestPoint TP44
+L Connector:TestPoint TP49
 U 1 1 5D2A7B60
 P 3775 2375
-F 0 "TP44" V 3800 2575 50  0000 L BNN
+F 0 "TP49" V 3800 2575 50  0000 L BNN
 F 1 "TestPoint" H 3525 2425 50  0001 C CNN
-F 2 "" H 3975 2375 50  0001 C CNN
+F 2 "custom:TestPoint_THTPad_D1.0mm_Drill0.5mm" H 3975 2375 50  0001 C CNN
 F 3 "~" H 3975 2375 50  0001 C CNN
 	1    3775 2375
@@
 	3875 2575 3675 2575
 $Comp
-L Connector:TestPoint TP47
+L Connector:TestPoint TP52
 U 1 1 5D55DA0B
 P 3875 4750
-F 0 "TP47" V 3900 4950 50  0000 L BNN
+F 0 "TP52" V 3900 4950 50  0000 L BNN
 F 1 "TestPoint" H 3625 4800 50  0001 C CNN
-F 2 "" H 4075 4750 50  0001 C CNN
+F 2 "custom:TestPoint_THTPad_D1.0mm_Drill0.5mm" H 4075 4750 50  0001 C CNN
 F 3 "~" H 4075 4750 50  0001 C CNN
 	1    3875 4750
@@
 $EndComp
 $Comp
-L Connector:TestPoint TP46
+L Connector:TestPoint TP51
 U 1 1 5D55DA11
 P 3775 4750
-F 0 "TP46" V 3800 4950 50  0000 L BNN
+F 0 "TP51" V 3800 4950 50  0000 L BNN
 F 1 "TestPoint" H 3525 4800 50  0001 C CNN
-F 2 "" H 3975 4750 50  0001 C CNN
+F 2 "custom:TestPoint_THTPad_D1.0mm_Drill0.5mm" H 3975 4750 50  0001 C CNN
 F 3 "~" H 3975 4750 50  0001 C CNN
 	1    3775 4750
