File: PANEL_EXTENSION.sch (KiCad schematic (older format))
At the start: 23 parts, among them J10 Conn_01x08_Male, U20 SGM3157YC6, U21 CM1293A-04SO, U22 SGM3157YC6, U23 CM1293A-04SO

Commit message: automated commit
Parts:
- renumbered R81 to R89, R82 to R90, R83 to R91, R84 to R92
Changed lines of the file:
@@
 	6100 4575 6000 4575
 $Comp
-L power:+3V3 #PWR0157
+L power:+3V3 #PWR0159
 U 1 1 621E790F
 P 6000 4525
-F 0 "#PWR0157" H 6000 4375 50  0001 C CNN
+F 0 "#PWR0159" H 6000 4375 50  0001 C CNN
 F 1 "+3V3" H 6000 4665 50  0000 C CNN
 F 2 "" H 6000 4525 50  0001 C CNN
@@
 	6100 5475 6000 5475
 $Comp
-L power:+3V3 #PWR0163
+L power:+3V3 #PWR0165
 U 1 1 621E7962
 P 6000 5425
-F 0 "#PWR0163" H 6000 5275 50  0001 C CNN
+F 0 "#PWR0165" H 6000 5275 50  0001 C CNN
 F 1 "+3V3" H 6000 5565 50  0000 C CNN
 F 2 "" H 6000 5425 50  0001 C CNN
@@
 	6000 5825 6000 5775
 $Comp
-L power:GND #PWR0165
+L power:GND #PWR0167
 U 1 1 621E796A
 P 6000 5825
-F 0 "#PWR0165" H 6000 5575 50  0001 C CNN
+F 0 "#PWR0167" H 6000 5575 50  0001 C CNN
 F 1 "GND" H 6000 5675 50  0000 C CNN
 F 2 "" H 6000 5825 50  0001 C CNN
@@
 	6000 4925 6000 4875
 $Comp
-L power:GND #PWR0160
+L power:GND #PWR0162
 U 1 1 621E79BB
 P 6000 4925
-F 0 "#PWR0160" H 6000 4675 50  0001 C CNN
+F 0 "#PWR0162" H 6000 4675 50  0001 C CNN
 F 1 "GND" H 6000 4775 50  0000 C CNN
 F 2 "" H 6000 4925 50  0001 C CNN
@@
 	2975 4850 2875 4850
 $Comp
-L power:+3V3 #PWR0158
+L power:+3V3 #PWR0160
 U 1 1 5D54B19A
 P 2875 4800
-F 0 "#PWR0158" H 2875 4650 50  0001 C CNN
+F 0 "#PWR0160" H 2875 4650 50  0001 C CNN
 F 1 "+3V3" H 2875 4940 50  0000 C CNN
 F 2 "" H 2875 4800 50  0001 C CNN
@@
 	3775 5100 3775 5050
 $Comp
-L power:GND #PWR0161
+L power:GND #PWR0163
 U 1 1 5D54CF05
 P 3775 5100
-F 0 "#PWR0161" H 3775 4850 50  0001 C CNN
+F 0 "#PWR0163" H 3775 4850 50  0001 C CNN
 F 1 "GND" H 3775 4950 50  0000 C CNN
 F 2 "" H 3775 5100 50  0001 C CNN
@@
 	2975 2475 2875 2475
 $Comp
-L power:+3V3 #PWR0151
+L power:+3V3 #PWR0153
 U 1 1 5D54FAD1
 P 2875 2425
-F 0 "#PWR0151" H 2875 2275 50  0001 C CNN
+F 0 "#PWR0153" H 2875 2275 50  0001 C CNN
 F 1 "+3V3" H 2875 2565 50  0000 C CNN
 F 2 "" H 2875 2425 50  0001 C CNN
@@
 	3775 2725 3775 2675
 $Comp
-L power:GND #PWR0153
+L power:GND #PWR0155
 U 1 1 5D54FAD9
 P 3775 2725
-F 0 "#PWR0153" H 3775 2475 50  0001 C CNN
+F 0 "#PWR0155" H 3775 2475 50  0001 C CNN
 F 1 "GND" H 3775 2575 50  0000 C CNN
 F 2 "" H 3775 2725 50  0001 C CNN
@@
 	2875 5475 2875 5550
 $Comp
-L power:GND #PWR0164
+L power:GND #PWR0166
 U 1 1 5D57DDBD
 P 2700 5600
-F 0 "#PWR0164" H 2700 5350 50  0001 C CNN
+F 0 "#PWR0166" H 2700 5350 50  0001 C CNN
 F 1 "GND" H 2700 5450 50  0000 C CNN
 F 2 "" H 2700 5600 50  0001 C CNN
@@
 $EndComp
 $Comp
-L custom:CRG0603F4K7 R83
+L custom:CRG0603F4K7 R91
 U 1 1 5D5808FB
 P 2500 5325
-F 0 "R83" H 2570 5345 50  0000 L BNN
+F 0 "R91" H 2570 5345 50  0000 L BNN
 F 1 "CRG0603F4K7" H 1800 4925 50  0001 L BNN
 F 2 "Resistor_SMD:R_0603_1608Metric" H 1800 4825 50  0001 L BNN
@@
 $EndComp
 $Comp
-L custom:CRG0603F4K7 R84
+L custom:CRG0603F4K7 R92
 U 1 1 5D581918
 P 2875 5325
-F 0 "R84" H 2945 5345 50  0000 L BNN
+F 0 "R92" H 2945 5345 50  0000 L BNN
 F 1 "CRG0603F4K7" H 2175 4925 50  0001 L BNN
 F 2 "Resistor_SMD:R_0603_1608Metric" H 2175 4825 50  0001 L BNN
@@
 	2900 3100 2900 3175
 $Comp
-L power:GND #PWR0156
+L power:GND #PWR0158
 U 1 1 5D5DFF1F
 P 2725 3225
-F 0 "#PWR0156" H 2725 2975 50  0001 C CNN
+F 0 "#PWR0158" H 2725 2975 50  0001 C CNN
 F 1 "GND" H 2725 3075 50  0000 C CNN
 F 2 "" H 2725 3225 50  0001 C CNN
@@
 $EndComp
 $Comp
-L custom:CRG0603F4K7 R81
+L custom:CRG0603F4K7 R89
 U 1 1 5D5DFF27
 P 2525 2950
-F 0 "R81" H 2595 2970 50  0000 L BNN
+F 0 "R89" H 2595 2970 50  0000 L BNN
 F 1 "CRG0603F4K7" H 1825 2550 50  0001 L BNN
 F 2 "Resistor_SMD:R_0603_1608Metric" H 1825 2450 50  0001 L BNN
@@
 $EndComp
 $Comp
-L custom:CRG0603F4K7 R82
+L custom:CRG0603F4K7 R90
 U 1 1 5D5DFF2F
 P 2900 2950
-F 0 "R82" H 2970 2970 50  0000 L BNN
+F 0 "R90" H 2970 2970 50  0000 L BNN
 F 1 "CRG0603F4K7" H 2200 2550 50  0001 L BNN
 F 2 "Resistor_SMD:R_0603_1608Metric" H 2200 2450 50  0001 L BNN
@@
 	2700 5550 2875 5550
 $Comp
-L power:GND #PWR0155
+L power:GND #PWR0157
 U 1 1 5D5EA3CE
 P 7325 3200
-F 0 "#PWR0155" H 7325 2950 50  0001 C CNN
+F 0 "#PWR0157" H 7325 2950 50  0001 C CNN
 F 1 "GND" H 7325 3050 50  0000 C CNN
 F 2 "" H 7325 3200 50  0001 C CNN
@@
 	4700 4875 4700 4825
 $Comp
-L power:+3V3 #PWR0159
+L power:+3V3 #PWR0161
 U 1 1 5D5FC7EC
 P 4700 4825
-F 0 "#PWR0159" H 4700 4675 50  0001 C CNN
+F 0 "#PWR0161" H 4700 4675 50  0001 C CNN
 F 1 "+3V3" H 4700 4965 50  0000 C CNN
 F 2 "" H 4700 4825 50  0001 C CNN
@@
 	4700 5225 4700 5175
 $Comp
-L power:GND #PWR0162
+L power:GND #PWR0164
 U 1 1 5D5FFF0B
 P 4700 5225
-F 0 "#PWR0162" H 4700 4975 50  0001 C CNN
+F 0 "#PWR0164" H 4700 4975 50  0001 C CNN
 F 1 "GND" H 4700 5075 50  0000 C CNN
 F 2 "" H 4700 5225 50  0001 C CNN
@@
 	4700 2500 4700 2450
 $Comp
-L power:+3V3 #PWR0152
+L power:+3V3 #PWR0154
 U 1 1 5D60552A
 P 4700 2450
-F 0 "#PWR0152" H 4700 2300 50  0001 C CNN
+F 0 "#PWR0154" H 4700 2300 50  0001 C CNN
 F 1 "+3V3" H 4700 2590 50  0000 C CNN
 F 2 "" H 4700 2450 50  0001 C CNN
@@
 	4700 2850 4700 2800
 $Comp
-L power:GND #PWR0154
+L power:GND #PWR0156
 U 1 1 5D605531
 P 4700 2850
-F 0 "#PWR0154" H 4700 2600 50  0001 C CNN
+F 0 "#PWR0156" H 4700 2600 50  0001 C CNN
 F 1 "GND" H 4700 2700 50  0000 C CNN
 F 2 "" H 4700 2850 50  0001 C CNN
