File: PANEL_EXTENSION.sch (KiCad schematic (older format))
At the start: 23 parts, among them J10 Conn_01x08_Male, U20 SGM3157YC6, U21 CM1293A-04SO, U22 SGM3157YC6, U23 CM1293A-04SO

Commit message: automated commit
Connections:
- net GND: now also TP60.1, U23.6 (CH4)
Changed lines of the file:
@@
 	-1   0    0    -1
 $EndComp
+Wire Wire Line
+	7200 5825 7200 5775
+$Comp
+L power:GND #PWR?
+U 1 1 5D1EC1AC
+P 7200 5825
+F 0 "#PWR?" H 7200 5575 50  0001 C CNN
+F 1 "GND" H 7200 5675 50  0000 C CNN
+F 2 "" H 7200 5825 50  0001 C CNN
+F 3 "" H 7200 5825 50  0001 C CNN
+	1    7200 5825
+	1    0    0    -1
+$EndComp
+Connection ~ 7200 5775
 $EndSCHEMATC

Commit message: automated commit
Connections:
- net !COL_RESET: now also J10.3 (Pin_3); no longer J10.6 (Pin_6)
- net !ENABLE: now also J10.2 (Pin_2); no longer J10.7 (Pin_7)
- net COL_DATA: now also J10.5 (Pin_5); no longer J10.4 (Pin_4)
- net COL_SHCP: now also J10.4 (Pin_4); no longer J10.5 (Pin_5)
- net GND: now also J10.1 (Pin_1); no longer J10.8 (Pin_8)
- net ROW_DATA: now also J10.8 (Pin_8); no longer J10.1 (Pin_1)
- net ROW_ON: now also J10.6 (Pin_6); no longer J10.3 (Pin_3)
- net ROW_SHCP: now also J10.7 (Pin_7); no longer J10.2 (Pin_2)
Changed lines of the file:
@@
 L Connector:Conn_01x08_Male J10
 U 1 1 621E7A0B
-P 7750 2650
-F 0 "J10" H 7750 3050 50  0000 C CNN
-F 1 "Conn_01x08_Male" H 7325 2625 50  0000 C CNN
-F 2 "Connector_PinHeader_2.54mm:PinHeader_1x08_P2.54mm_Horizontal" H 7750 2650 50  0001 C CNN
-F 3 "" H 7750 2650 50  0001 C CNN
-	1    7750 2650
-	-1   0    0    -1
+P 7750 2750
+F 0 "J10" H 7750 3150 50  0000 C CNN
+F 1 "Conn_01x08_Male" H 7325 2725 50  0000 C CNN
+F 2 "Connector_PinHeader_2.54mm:PinHeader_1x08_P2.54mm_Horizontal" H 7750 2750 50  0001 C CNN
+F 3 "" H 7750 2750 50  0001 C CNN
+	1    7750 2750
+	-1   0    0    1
 $EndComp
 Text Label 1875 4950 0    60   ~ 0
