File: POWER.sch (KiCad schematic (older format))
At the start: 48 parts

Commit message: automated commit
Parts:
- removed R?: 32.4k, Resistors_SMD:R_0603_HandSoldering, symbol Device:R
- added D10, D11, D12: LED_GENERIC_0805, Diode_SMD:D_0805_2012Metric, symbol custom:LED_GENERIC_0805
- added Q3: SSM3K35AMFV, symbol custom:SSM3K35AMFV
- added R28, R31: ‎RMCF0603FT470R‎, Resistor_SMD:R_0603_1608Metric, symbol custom:‎RMCF0603FT470R‎
- added R30: RMCF0603FT10K0, 0603, symbol custom:RMCF0603FT10K0
- added R36: CRG0603F4K7, Resistor_SMD:R_0603_1608Metric, symbol custom:CRG0603F4K7
- added R48: CR0603-FX-3242ELF, Resistor_SMD:R_0603_1608Metric, symbol custom:CR0603-FX-3242ELF
- gave numbers to parts that had none: 47
Connections:
- net +12V: now also R30.1
- net +1V8: now also Q3.1 (G), R36.1
- net +3V3: now also R28.1, R31.1
- net GND: now also D11.1 (K), D12.1 (K), Q3.2 (S), R36.2, R48.2
- net at C50.2, R45.1, R47.1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: now also R48.1
- new net: D12.2 (A), R31.2
- new net: D10.1 (K), Q3.3 (D)
- new net: D10.2 (A), R28.2
- new net: D11.2 (A), R30.2
Other:
- note added: "LABEL VOLTAGE\nDOMAINS ON\nSILKSCREEN"
