File: POWER.sch (KiCad schematic (older format))
At the start: 56 parts, among them Q3 SSM3K35AMFV, U4 TPS61175, U5 AP65111A, U6 AP65111A

Commit message: automated commit
Parts:
- renumbered C41 to C10, C42 to C11, C43 to C12, C44 to C13, C45 to C14, C46 to C15, C47 to C16, C48 to C17, C49 to C18, C50 to C19, C51 to C20, C37 to C6, C38 to C7, C39 to C8, C40 to C9, D9 to D4, D10 to D5, D11 to D6, D12 to D7, L3 to L2, L4 to L3, L5 to L4, Q3 to Q1, R34 to R10, R35 to R11, R36 to R12, R37 to R13, R38 to R14, R39 to R15, R40 to R16, R41 to R17, R42 to R18, R43 to R19, R26 to R2, R44 to R20, R45 to R21, R46 to R22, R47 to R23, R48 to R24, R27 to R3, R28 to R4, R29 to R5, R30 to R6, R31 to R7, R32 to R8, R33 to R9, TP16 to TP10, TP10 to TP4, TP11 to TP5, TP12 to TP6, TP13 to TP7, TP14 to TP8, TP15 to TP9, U4 to U1, U5 to U2, U6 to U3

Commit message: automated commit
Parts:
- removed R10: 143k, Resistors_SMD:R_0603_HandSoldering, symbol Device:R
- removed R11, R12, R2: CRG0603F4K7, Resistor_SMD:R_0603_1608Metric, symbol custom:CRG0603F4K7
- removed R13, R22: RC0603FR-0747KL, Resistor_SMD:R_0603_1608Metric, symbol custom:RC0603FR-0747KL
- removed R15, R21: 40.2k, Resistors_SMD:R_0603_HandSoldering, symbol Device:R
- removed R16, R18: 13k, Resistors_SMD:R_0603_HandSoldering, symbol Device:R
- removed R17: 59k, Resistors_SMD:R_0603_HandSoldering, symbol Device:R
- removed R23: 100k, Resistors_SMD:R_0603_HandSoldering, symbol Device:R
- removed R24: CR0603-FX-3242ELF, Resistor_SMD:R_0603_1608Metric, symbol custom:CR0603-FX-3242ELF
- removed R3: 300k, Resistors_SMD:R_0603_HandSoldering, symbol Device:R
- removed R8: 16.2k, Resistors_SMD:R_0603_HandSoldering, symbol Device:R
- removed R9: 200, Resistors_SMD:R_0603_HandSoldering, symbol Device:R
- added R? (x3): CRG0603F4K7, Resistor_SMD:R_0603_1608Metric, symbol custom:CRG0603F4K7
- added R?: RMCF0603FT16K2, custom:R_0603, symbol custom:RMCF0603FT16K2
- added R? (x2): RMCF0603JT13K0, custom:R_0603, symbol custom:RMCF0603JT13K0
- added R? (x2): RC0603FR-0747KL, Resistor_SMD:R_0603_1608Metric, symbol custom:RC0603FR-0747KL
- added R?: RMCF0603FT59K0, custom:R_0603, symbol custom:RMCF0603FT59K0
- added R? (x2): RMCF0603FT40K2, 0603, symbol custom:RMCF0603FT40K2
- added R?: CR0603-FX-3242ELF, Resistor_SMD:R_0603_1608Metric, symbol custom:CR0603-FX-3242ELF
- added R?: RMCF0603FG100K, custom:R_0603, symbol custom:RMCF0603FG100K
- added R?: CR0603-FX-3003ELF, custom:R_0603, symbol custom:CR0603-FX-3003ELF
- added R?: AC0603JR-07200RL, custom:R_0603, symbol custom:AC0603JR-07200RL
- added R?: ERJ-3EKF1433V, custom:R_0603, symbol custom:ERJ-3EKF1433V
Connections:
- net +12V: now also R?.1, R?.1
- net +1V8: now also R?.1, R?.1
- net +24V: now also R?.1
- net +3V3: now also R?.1
- net GND: now also R?.2, R?.2, R?.2, R?.2, R?.2, R?.2, R?.2, R?.2
- net at C19.2, TP10.1: now also R?.1, R?.1, R?.2
- net at R19.2, R20.2, U3.5 (EN): now also R?.1
- net at U3.6 (FB): now also R?.2
- net at R14.2, U2.5 (EN): now also R?.1, R?.2
- net at U2.6 (FB): now also R?.2
- net at C15.2, TP8.1: now also R?.1, R?.1, R?.2
- net at U1.10 (FREQ): now also R?.1
- net at TP5.1, U1.4 (EN): now also R?.1, R?.2
- net at U1.8 (COMP): now also R?.1
- net at R5.1, TP6.1: now also R?.1, R?.2
- net at C12.1: now also R?.2
Other:
- moved on the sheet: C17, C18, C19, C20, L4, R19, R20, TP10, TP9, U3

Commit message: automated commit
Parts:
- gave numbers to parts that had none: 16
Changed lines of the file:
@@
 LABEL VOLTAGE\nDOMAINS ON\nSILKSCREEN
 $Comp
-L custom:CRG0603F4K7 R?
+L custom:CRG0603F4K7 R12
 U 1 1 5D012BA6
 P 8875 3300
-F 0 "R?" H 8945 3320 50  0000 L BNN
+F 0 "R12" H 8945 3320 50  0000 L BNN
 F 1 "CRG0603F4K7" H 8175 2900 50  0001 L BNN
 F 2 "Resistor_SMD:R_0603_1608Metric" H 8175 2800 50  0001 L BNN
@@
 $EndComp
 $Comp
-L custom:CRG0603F4K7 R?
+L custom:CRG0603F4K7 R11
 U 1 1 5D0133DD
 P 2725 2975
-F 0 "R?" H 2795 2995 50  0000 L BNN
+F 0 "R11" H 2795 2995 50  0000 L BNN
 F 1 "CRG0603F4K7" H 2025 2575 50  0001 L BNN
 F 2 "Resistor_SMD:R_0603_1608Metric" H 2025 2475 50  0001 L BNN
@@
 $EndComp
 $Comp
-L custom:CRG0603F4K7 R?
+L custom:CRG0603F4K7 R2
 U 1 1 5D014677
 P 2925 2075
-F 0 "R?" H 3050 2100 50  0000 L BNN
+F 0 "R2" H 3050 2100 50  0000 L BNN
 F 1 "CRG0603F4K7" H 2225 1675 50  0001 L BNN
 F 2 "Resistor_SMD:R_0603_1608Metric" H 2225 1575 50  0001 L BNN
@@
 $EndComp
 $Comp
-L custom:RMCF0603FT16K2 R?
+L custom:RMCF0603FT16K2 R8
 U 1 1 5D02B17B
 P 4725 2875
-F 0 "R?" H 4825 2925 50  0000 C CNN
+F 0 "R8" H 4825 2925 50  0000 C CNN
 F 1 "RMCF0603FT16K2" H 4750 2375 50  0001 C CNN
 F 2 "custom:R_0603" H 4750 2300 50  0001 C CNN
@@
 $EndComp
 $Comp
-L custom:RMCF0603JT13K0 R?
+L custom:RMCF0603JT13K0 R16
 U 1 1 5D03F2FE
 P 2325 5125
-F 0 "R?" H 2425 5175 50  0000 C CNN
+F 0 "R16" H 2425 5175 50  0000 C CNN
 F 1 "RMCF0603JT13K0" H 2325 4625 50  0000 C CNN
 F 2 "custom:R_0603" H 2325 4550 50  0001 C CNN
@@
 $EndComp
 $Comp
-L custom:RC0603FR-0747KL R?
+L custom:RC0603FR-0747KL R13
 U 1 1 5D059A4F
 P 2325 4725
-F 0 "R?" H 2395 4745 50  0000 L BNN
+F 0 "R13" H 2395 4745 50  0000 L BNN
 F 1 "RC0603FR-0747KL" H 1925 4275 50  0001 L BNN
 F 2 "Resistor_SMD:R_0603_1608Metric" H 1925 4175 50  0001 L BNN
@@
 $EndComp
 $Comp
-L custom:RMCF0603FT59K0 R?
+L custom:RMCF0603FT59K0 R17
 U 1 1 5D071AFC
 P 4075 5125
-F 0 "R?" V 4125 5300 50  0000 C CNN
+F 0 "R17" V 4125 5300 50  0000 C CNN
 F 1 "RMCF0603FT59K0" H 4075 4675 50  0001 C CNN
 F 2 "custom:R_0603" H 4075 4600 50  0001 C CNN
@@
 $EndComp
 $Comp
-L custom:RMCF0603JT13K0 R?
+L custom:RMCF0603JT13K0 R18
 U 1 1 5D075C6B
 P 5325 5325
-F 0 "R?" H 5425 5375 50  0000 C CNN
+F 0 "R18" H 5425 5375 50  0000 C CNN
 F 1 "RMCF0603JT13K0" H 5325 4825 50  0000 C CNN
 F 2 "custom:R_0603" H 5325 4750 50  0001 C CNN
@@
 $EndComp
 $Comp
-L custom:RMCF0603FT40K2 R?
+L custom:RMCF0603FT40K2 R15
 U 1 1 5D080D8F
 P 5325 4925
-F 0 "R?" H 5375 4950 50  0000 L BNN
+F 0 "R15" H 5375 4950 50  0000 L BNN
 F 1 "RMCF0603FT40K2" H 5050 4425 50  0001 L BNN
 F 2 "0603" H 5050 4500 50  0001 L BNN
@@
 $EndComp
 $Comp
-L custom:RC0603FR-0747KL R?
+L custom:RC0603FR-0747KL R22
 U 1 1 5D0819DB
 P 2325 7075
-F 0 "R?" H 2395 7095 50  0000 L BNN
+F 0 "R22" H 2395 7095 50  0000 L BNN
 F 1 "RC0603FR-0747KL" H 1925 6625 50  0001 L BNN
 F 2 "Resistor_SMD:R_0603_1608Metric" H 1925 6525 50  0001 L BNN
@@
 $EndComp
 $Comp
-L custom:RMCF0603FT40K2 R?
+L custom:RMCF0603FT40K2 R21
 U 1 1 5D082BEB
 P 5325 6875
-F 0 "R?" H 5375 6900 50  0000 L BNN
+F 0 "R21" H 5375 6900 50  0000 L BNN
 F 1 "RMCF0603FT40K2" H 5050 6375 50  0001 L BNN
 F 2 "0603" H 5050 6450 50  0001 L BNN
@@
 $EndComp
 $Comp
-L custom:CR0603-FX-3242ELF R?
+L custom:CR0603-FX-3242ELF R24
 U 1 1 5D08E2D3
 P 5325 7275
-F 0 "R?" H 5395 7295 50  0000 L BNN
+F 0 "R24" H 5395 7295 50  0000 L BNN
 F 1 "CR0603-FX-3242ELF" H 4925 6825 50  0001 L BNN
 F 2 "Resistor_SMD:R_0603_1608Metric" H 4925 6725 50  0001 L BNN
@@
 $EndComp
 $Comp
-L custom:RMCF0603FG100K R?
+L custom:RMCF0603FG100K R23
 U 1 1 5D0B44A9
 P 4075 7075
-F 0 "R?" V 4125 7250 50  0000 C CNN
+F 0 "R23" V 4125 7250 50  0000 C CNN
 F 1 "RMCF0603FG100K" H 4075 6650 50  0001 C CNN
 F 2 "custom:R_0603" H 4075 6550 50  0001 C CNN
@@
 $EndComp
 $Comp
-L custom:CR0603-FX-3003ELF R?
+L custom:CR0603-FX-3003ELF R3
 U 1 1 5D0CF1A0
 P 4725 2225
-F 0 "R?" H 4825 2275 50  0000 C CNN
+F 0 "R3" H 4825 2275 50  0000 C CNN
 F 1 "CR0603-FX-3003ELF" H 4725 1750 50  0001 C CNN
 F 2 "custom:R_0603" H 4725 1675 50  0001 C CNN
@@
 $EndComp
 $Comp
-L custom:AC0603JR-07200RL R?
+L custom:AC0603JR-07200RL R9
 U 1 1 5D0E17AC
 P 1675 2975
-F 0 "R?" V 1725 3150 50  0000 C CNN
+F 0 "R9" V 1725 3150 50  0000 C CNN
 F 1 "AC0603JR-07200RL" H 1675 2525 50  0001 C CNN
 F 2 "custom:R_0603" H 1675 2450 50  0001 C CNN
@@
 $EndComp
 $Comp
-L custom:ERJ-3EKF1433V R?
+L custom:ERJ-3EKF1433V R10
 U 1 1 5D0FAA18
 P 1975 2975
-F 0 "R?" V 2025 3150 50  0000 C CNN
+F 0 "R10" V 2025 3150 50  0000 C CNN
 F 1 "ERJ-3EKF1433V" H 1975 2525 50  0001 C CNN
 F 2 "custom:R_0603" H 1975 2450 50  0001 C CNN

Commit message: automated commit
Parts:
- added TP10, TP12, TP14, TP16, TP7, TP8: TestPoint, symbol Connector:TestPoint
- R15, R21, R6: footprint 0603 -> (none)
- renumbered TP8 to TP11, TP9 to TP13, TP10 to TP15, TP7 to TP9
Connections:
- net GND: now also TP10.1, TP12.1, TP14.1, TP16.1, TP7.1, TP8.1
Other:
- note added: "LABEL VOLTAGE\nON SILKSCREEN"
- moved on the sheet: C13, C14, C15, C16, L3, R13, R14, R15, R16, R17, R18, TP11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
