File: POWER.sch (KiCad schematic (older format))
At the start: 62 parts, among them Q1 SSM3K35AMFV, U1 TPS61175, U2 AP65111A, U3 AP65111A

Commit message: automated commit
Parts:
- C10, C9: footprint (none) -> custom:EEE-1VA220SP
- D4: footprint (none) -> Package_TO_SOT_SMD:TO-277B
- Q1: footprint (none) -> Package_TO_SOT_SMD:SOT-723
- R15, R21, R6: footprint (none) -> custom:R_0603
Changed lines of the file:
@@
 	0    -1   -1   0
 $EndComp
-$Comp
-L power:+24V #PWR?
-U 1 1 60DE1CEA
-P 5775 1775
-AR Path="/60DE1CEA" Ref="#PWR?"  Part="1"
-AR Path="/60B0CF7E/60DE1CEA" Ref="#PWR011"  Part="1"
-F 0 "#PWR011" H 5775 1625 50  0001 C CNN
-F 1 "+24V" H 5775 1950 50  0000 C CNN
-F 2 "" H 5775 1775 50  0001 C CNN
-F 3 "" H 5775 1775 50  0001 C CNN
-	1    5775 1775
-	1    0    0    -1
-$EndComp
-$Comp
-L custom:DST2080S D?
-U 1 1 60DE1CF1
-P 4525 1875
-AR Path="/60DE1CF1" Ref="D?"  Part="1"
-AR Path="/60B0CF7E/60DE1CF1" Ref="D4"  Part="1"
-F 0 "D4" H 4525 1975 50  0000 C CNN
-F 1 "DST2080S" H 4525 1775 50  0000 C CNN
-F 2 "" H 4525 1875 50  0001 C CNN
-F 3 "" H 4525 1875 50  0001 C CNN
-	1    4525 1875
-	1    0    0    -1
-$EndComp
-Connection ~ 4275 1825
-Wire Wire Line
-	4325 1825 4275 1825
-Connection ~ 4275 1925
-Wire Wire Line
-	4275 1925 4325 1925
 Connection ~ 4275 2175
 Wire Wire Line
@@
 Connection ~ 4725 2475
 Wire Wire Line
-	4725 2075 4725 1875
-Wire Wire Line
-	4675 1875 4725 1875
-Wire Wire Line
-	5325 1875 5325 2475
-Connection ~ 4725 1875
-Wire Wire Line
 	5325 3525 5325 2775
 Connection ~ 4725 3525
-Connection ~ 5325 1875
 Wire Wire Line
 	4275 2475 4175 2475
 Connection ~ 3125 1825
 Wire Wire Line
-	5775 1775 5775 1875
-Connection ~ 5775 1875
-Wire Wire Line
 	5775 3525 5775 2775
 Connection ~ 5325 3525
 Wire Wire Line
-	4275 1825 4275 1925
-Wire Wire Line
-	4275 1925 4275 2175
-Wire Wire Line
 	4275 2175 4275 2325
 Wire Wire Line
@@
 	4725 2600 4775 2600
 Wire Wire Line
-	4725 1875 5075 1875
-Wire Wire Line
 	4725 3525 5325 3525
 Wire Wire Line
 	3125 1825 3125 2175
-Wire Wire Line
-	5775 1875 5775 2475
-Wire Wire Line
-	5075 1875 5075 1825
 Wire Wire Line
 	5325 3525 5775 3525
@@
 F 0 "C9" H 5440 2716 50  0000 L CNN
 F 1 "EEE-1VA220SP" H 4375 2175 50  0001 L BNN
-F 2 "" H 4375 2075 50  0001 L BNN
+F 2 "custom:EEE-1VA220SP" H 4375 2075 50  0001 L BNN
 F 3 "datasheets/EEE-1VA220SP.pdf" H 4375 1975 50  0001 L BNN
 F 4 "22uF" H 5440 2625 50  0000 L CNN "Capacitance"
@@
 F 0 "C10" H 5890 2716 50  0000 L CNN
 F 1 "EEE-1VA220SP" H 4825 2175 50  0001 L BNN
-F 2 "" H 4825 2075 50  0001 L BNN
+F 2 "custom:EEE-1VA220SP" H 4825 2075 50  0001 L BNN
 F 3 "datasheets/EEE-1VA220SP.pdf" H 4825 1975 50  0001 L BNN
 F 4 "22uF" H 5890 2625 50  0000 L CNN "Capacitance"
@@
 $Comp
 L Connector:TestPoint TP?
-U 1 1 60DE1E58
-P 5075 1825
-AR Path="/60DE1E58" Ref="TP?"  Part="1"
-AR Path="/60B0CF7E/60DE1E58" Ref="TP4"  Part="1"
-F 0 "TP4" H 5000 2050 50  0000 C CNN
-F 1 "TestPoint" H 4825 1875 50  0001 C CNN
-F 2 "" H 5275 1825 50  0001 C CNN
-F 3 "~" H 5275 1825 50  0001 C CNN
-	1    5075 1825
-	1    0    0    -1
-$EndComp
-$Comp
-L Connector:TestPoint TP?
 U 1 1 60DE1E5E
 P 4775 2600
@@
 Wire Wire Line
 	4725 2475 4725 2600
-Wire Wire Line
-	5325 1875 5775 1875
-Connection ~ 5075 1875
-Wire Wire Line
-	5075 1875 5325 1875
 Connection ~ 1525 1175
 Connection ~ 2425 1575
@@
 F 0 "Q1" V 9450 2975 50  0000 L BNN
 F 1 "SSM3K35AMFV" V 9375 2800 50  0000 L BNN
-F 2 "" H 9325 2925 50  0001 L BIN
-F 3 "datasheets/SSM3K35AMFV.pdf" H 9325 2900 50  0001 L BNN
+F 2 "Package_TO_SOT_SMD:SOT-723" H 9325 2925 50  0001 L BIN
+F 3 "/home/dj/datasheets/SSM3K35AMFV.pdf" H 9325 2900 50  0001 L BNN
 	1    9125 3050
 	1    0    0    -1
@@
 F 0 "R6" H 7850 2525 50  0000 L BNN
 F 1 "RMCF0603FT10K0" H 7450 1950 50  0001 L BNN
-F 2 "" H 7700 1875 50  0001 L BNN
+F 2 "custom:R_0603" H 7700 1875 50  0001 L BNN
 F 3 "" V 8075 2050 50  0001 L BNN
 F 4 "10k0" V 7775 2500 50  0000 C CNN "Resistance"
@@
 F 0 "R15" H 5400 4825 50  0000 L BNN
 F 1 "RMCF0603FT40K2" H 5050 4300 50  0001 L BNN
-F 2 "" H 5050 4375 50  0001 L BNN
+F 2 "custom:R_0603" H 5050 4375 50  0001 L BNN
 F 3 "/home/dj/datasheets/SEI-RMCF_RMCP.pdf" H 5050 4200 50  0001 L BNN
 F 4 "40k2" V 5325 4800 50  0000 C CNN "Resistance"
@@
 F 0 "R21" H 5375 6900 50  0000 L BNN
 F 1 "RMCF0603FT40K2" H 5050 6375 50  0001 L BNN
-F 2 "" H 5050 6450 50  0001 L BNN
+F 2 "custom:R_0603" H 5050 6450 50  0001 L BNN
 F 3 "/home/dj/datasheets/SEI-RMCF_RMCP.pdf" H 5050 6275 50  0001 L BNN
 F 4 "40k2" V 5325 6875 50  0000 C CNN "Resistance"
@@
 	-1   0    0    -1
 $EndComp
-Text Notes 4750 1450 0    60   ~ 0
-LABEL VOLTAGE\nON SILKSCREEN
 Text Notes 4950 4225 0    60   ~ 0
 LABEL VOLTAGE\nON SILKSCREEN
@@
 Connection ~ 1675 3525
 Connection ~ 2925 5000
+Text Notes 4750 1450 0    60   ~ 0
+LABEL VOLTAGE\nON SILKSCREEN
+Wire Wire Line
+	5075 1875 5325 1875
+Connection ~ 5075 1875
+Wire Wire Line
+	5325 1875 5775 1875
+$Comp
+L Connector:TestPoint TP?
+U 1 1 60DE1E58
+P 5075 1825
+AR Path="/60DE1E58" Ref="TP?"  Part="1"
+AR Path="/60B0CF7E/60DE1E58" Ref="TP4"  Part="1"
+F 0 "TP4" H 5000 2050 50  0000 C CNN
+F 1 "TestPoint" H 4825 1875 50  0001 C CNN
+F 2 "" H 5275 1825 50  0001 C CNN
+F 3 "~" H 5275 1825 50  0001 C CNN
+	1    5075 1825
+	1    0    0    -1
+$EndComp
+Wire Wire Line
+	5075 1875 5075 1825
+Wire Wire Line
+	5775 1875 5775 2475
+Wire Wire Line
+	4725 1875 5075 1875
+Connection ~ 5775 1875
+Wire Wire Line
+	5775 1775 5775 1875
+Connection ~ 5325 1875
+Wire Wire Line
+	5325 1875 5325 2475
+Wire Wire Line
+	4725 2075 4725 1875
+$Comp
+L power:+24V #PWR?
+U 1 1 60DE1CEA
+P 5775 1775
+AR Path="/60DE1CEA" Ref="#PWR?"  Part="1"
+AR Path="/60B0CF7E/60DE1CEA" Ref="#PWR011"  Part="1"
+F 0 "#PWR011" H 5775 1625 50  0001 C CNN
+F 1 "+24V" H 5775 1950 50  0000 C CNN
+F 2 "" H 5775 1775 50  0001 C CNN
+F 3 "" H 5775 1775 50  0001 C CNN
+	1    5775 1775
+	1    0    0    -1
+$EndComp
+Connection ~ 4725 1875
+Wire Wire Line
+	4675 1875 4725 1875
+Connection ~ 4275 1825
+Wire Wire Line
+	4325 1825 4275 1825
+Wire Wire Line
+	4275 1925 4275 2175
+Wire Wire Line
+	4275 1825 4275 1925
+Connection ~ 4275 1925
+Wire Wire Line
+	4275 1925 4325 1925
+$Comp
+L custom:DST2080S D?
+U 1 1 60DE1CF1
+P 4525 1875
+AR Path="/60DE1CF1" Ref="D?"  Part="1"
+AR Path="/60B0CF7E/60DE1CF1" Ref="D4"  Part="1"
+F 0 "D4" H 4525 1975 50  0000 C CNN
+F 1 "DST2080S" H 4525 1775 50  0000 C CNN
+F 2 "Package_TO_SOT_SMD:TO-277B" H 4525 1875 50  0001 C CNN
+F 3 "" H 4525 1875 50  0001 C CNN
+	1    4525 1875
+	1    0    0    -1
+$EndComp
 $EndSCHEMATC

Commit message: automated commit
Parts:
- removed L2: 12uH, symbol Device:L
- removed L3: 6.5uH, symbol Device:L
- removed L4: 3.3uH, symbol Device:L
- added L2: #B966AS-120M=P3, custom:490-14124-1-ND, symbol custom:#B966AS-120M=P3
- added L3: NRS5020T6R8MMGJ, custom:NRS5020T6R8MMGJ, symbol custom:NRS5020T6R8MMGJ
- added L4: MAKK2016T3R3M, custom:MAKK2016T3R3M, symbol custom:MAKK2016T3R3M
- added TP10, TP4, TP5, TP8, TP9: TestPoint, custom:TestPoint_THTPad_D1.0mm_Drill0.5mm, symbol Connector:TestPoint
- TP11: renamed from TP6; footprint (none) -> custom:TestPoint_THTPad_D1.0mm_Drill0.5mm
- TP12: renamed from TP7; footprint (none) -> custom:TestPoint_THTPad_D1.0mm_Drill0.5mm
- TP13: renamed from TP8; footprint (none) -> custom:TestPoint_THTPad_D1.0mm_Drill0.5mm
- TP14: renamed from TP9; footprint (none) -> custom:TestPoint_THTPad_D1.0mm_Drill0.5mm
- TP15: renamed from TP10; footprint (none) -> custom:TestPoint_THTPad_D1.0mm_Drill0.5mm
- TP16: renamed from TP11; footprint (none) -> custom:TestPoint_THTPad_D1.0mm_Drill0.5mm
- TP17: renamed from TP12; footprint (none) -> custom:TestPoint_THTPad_D1.0mm_Drill0.5mm
- TP18: renamed from TP13; footprint (none) -> custom:TestPoint_THTPad_D1.0mm_Drill0.5mm
- TP19: renamed from TP14; footprint (none) -> custom:TestPoint_THTPad_D1.0mm_Drill0.5mm
- TP20: renamed from TP15; footprint (none) -> custom:TestPoint_THTPad_D1.0mm_Drill0.5mm
- TP21: renamed from TP16; footprint (none) -> custom:TestPoint_THTPad_D1.0mm_Drill0.5mm
- TP6: renamed from TP4; footprint (none) -> custom:TestPoint_THTPad_D1.0mm_Drill0.5mm
- TP7: renamed from TP5; footprint (none) -> custom:TestPoint_THTPad_D1.0mm_Drill0.5mm
- U1: footprint (none) -> custom:HTSSOP-14
- U2, U3: footprint (none) -> Package_TO_SOT_SMD:TSOT-23-6
Connections:
- net +12V: now also L2.2, TP4.1
- net +1V8: now also L4.1
- net +3V3: now also L3.1
- net at R11.1, U1.8 (COMP): now also TP10.1
- net at R10.1, U1.10 (FREQ): now also TP8.1
- net at C17.2, U3.3 (SW): now also L4.2
- net at C13.2, U2.3 (SW): now also L3.2
- net at D4.1 (A1), D4.2 (A2), U1.1 (SW)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: now also L2.1, TP5.1
- net at C11.1, U1.5 (SS): now also TP9.1
Other:
- moved on the sheet: C11, C12, C13, C14, C17, C18, C6, C7, C8, R10, R11, R13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

Commit message: automated commit
Connections:
- net +12V: no longer R6.1
- net +24V: now also R6.1
Changed lines of the file:
@@
-$EndComp
-$Comp
-L power:+12V #PWR013
-U 1 1 5D152855
-P 7775 2250
-F 0 "#PWR013" H 7775 2100 50  0001 C CNN
-F 1 "+12V" H 7775 2390 50  0000 C CNN
-F 2 "" H 7775 2250 50  0001 C CNN
-F 3 "" H 7775 2250 50  0001 C CNN
-	1    7775 2250
-	1    0    0    -1
 $EndComp
 $Comp
@@
 	0    1    1    0
 $EndComp
+$Comp
+L power:+24V #PWR?
+U 1 1 5D1C8F9D
+P 7775 2250
+AR Path="/5D1C8F9D" Ref="#PWR?"  Part="1"
+AR Path="/60B0CF7E/5D1C8F9D" Ref="#PWR0274"  Part="1"
+F 0 "#PWR0274" H 7775 2100 50  0001 C CNN
+F 1 "+24V" H 7775 2400 50  0000 C CNN
+F 2 "" H 7775 2250 50  0001 C CNN
+F 3 "" H 7775 2250 50  0001 C CNN
+	1    7775 2250
+	1    0    0    -1
+$EndComp
 $EndSCHEMATC

Commit message: automated commit
Parts:
- removed TP12, TP15, TP19: TestPoint, custom:TestPoint_THTPad_D1.0mm_Drill0.5mm, symbol Connector:TestPoint
Changed lines of the file:
@@
 Wire Wire Line
 	5775 7250 5775 7025
-$Comp
-L Connector:TestPoint TP?
-U 1 1 5D5C44D4
-P 2675 7075
-AR Path="/5D5C44D4" Ref="TP?"  Part="1"
-AR Path="/60B0CF7E/5D5C44D4" Ref="TP19"  Part="1"
-F 0 "TP19" V 2575 7225 50  0000 C CNN
-F 1 "TestPoint" H 2425 7125 50  0001 C CNN
-F 2 "custom:TestPoint_THTPad_D1.0mm_Drill0.5mm" H 2875 7075 50  0001 C CNN
-F 3 "~" H 2875 7075 50  0001 C CNN
-	1    2675 7075
-	0    -1   1    0
-$EndComp
-Wire Wire Line
-	2675 7075 2725 7075
-Connection ~ 2725 7075
-$Comp
-L Connector:TestPoint TP?
-U 1 1 5D5CD745
-P 2675 5000
-AR Path="/5D5CD745" Ref="TP?"  Part="1"
-AR Path="/60B0CF7E/5D5CD745" Ref="TP15"  Part="1"
-F 0 "TP15" V 2575 5150 50  0000 C CNN
-F 1 "TestPoint" H 2425 5050 50  0001 C CNN
-F 2 "custom:TestPoint_THTPad_D1.0mm_Drill0.5mm" H 2875 5000 50  0001 C CNN
-F 3 "~" H 2875 5000 50  0001 C CNN
-	1    2675 5000
-	0    -1   1    0
-$EndComp
-Wire Wire Line
-	2675 5000 2725 5000
-$Comp
-L Connector:TestPoint TP?
-U 1 1 5D5D5A4A
-P 1250 3525
-AR Path="/5D5D5A4A" Ref="TP?"  Part="1"
-AR Path="/60B0CF7E/5D5D5A4A" Ref="TP12"  Part="1"
-F 0 "TP12" V 1150 3675 50  0000 C CNN
-F 1 "TestPoint" H 1000 3575 50  0001 C CNN
-F 2 "custom:TestPoint_THTPad_D1.0mm_Drill0.5mm" H 1450 3525 50  0001 C CNN
-F 3 "~" H 1450 3525 50  0001 C CNN
-	1    1250 3525
-	0    -1   1    0
-$EndComp
-Wire Wire Line
-	1250 3525 1325 3525
-Connection ~ 1325 3525
-Connection ~ 2725 5000
 Text Notes 4750 1450 0    60   ~ 0
 LABEL VOLTAGE\nON SILKSCREEN

Commit message: automated commit
Parts:
- removed R14, R20: NP_R_0603, Resistor_SMD:R_0603_1608Metric, symbol custom:NP_R_0603
Other:
- moved on the sheet: C14, C18, R13, R16, R19, R22
