File: POWER_INPUT.sch (KiCad schematic (older format))
At the start: 15 parts

Commit message: automated commit
Parts:
- gave numbers to parts that had none: 15
Other:
- moved on the sheet: J2
Changed lines of the file:
@@
 EELAYER 29 0
 EELAYER END
-$Descr A4 11693 8268
+$Descr USLetter 11000 8500
 encoding utf-8
 Sheet 3 20
-Title ""
+Title "FLIPDOT_DRIVER"
 Date ""
 Rev ""
-Comp ""
+Comp "DYLAN DAILEY"
 Comment1 ""
 Comment2 ""
@@
 $EndDescr
 $Comp
-L Connector:Barrel_Jack_Switch J?
+L Connector:Barrel_Jack_Switch J1
 U 1 1 5E580BD9
 P 4275 3975
-F 0 "J?" H 4275 4185 50  0000 C CNN
+F 0 "J1" H 4275 4185 50  0000 C CNN
 F 1 "Barrel_Jack" H 4275 3775 50  0000 C CNN
 F 2 "Connectors:BARREL_JACK" H 4325 3935 50  0001 C CNN
@@
 PUT SYMBOL FOR CENTER-POSITIVE\nCONNECTOR, VOLTAGE RANGE, AND\nBARREL JACK DIMENSIONS FOR MATE\nON SILKSCREEN
 $Comp
-L power:GND #PWR?
+L power:GND #PWR030
 U 1 1 5E580BE0
 P 6650 2875
-F 0 "#PWR?" H 6650 2625 50  0001 C CNN
+F 0 "#PWR030" H 6650 2625 50  0001 C CNN
 F 1 "GND" H 6650 2725 50  0000 C CNN
 F 2 "" H 6650 2875 50  0001 C CNN
@@
 $EndComp
 $Comp
-L power:+12V #PWR?
+L power:+12V #PWR029
 U 1 1 5E580BE6
 P 4850 2375
-F 0 "#PWR?" H 4850 2225 50  0001 C CNN
+F 0 "#PWR029" H 4850 2225 50  0001 C CNN
 F 1 "+12V" H 4850 2515 50  0000 C CNN
 F 2 "" H 4850 2375 50  0001 C CNN
@@
 $EndComp
 $Comp
-L Connector:Screw_Terminal_01x04 J?
+L Connector:Screw_Terminal_01x04 J2
 U 1 1 5E580BEC
-P 5400 4175
-F 0 "J?" H 5400 4375 50  0000 C CNN
-F 1 "Screw_Terminal_01x04" V 5500 4075 50  0001 C CNN
-F 2 "" H 5400 4175 50  0001 C CNN
-F 3 "" H 5400 4175 50  0001 C CNN
-	1    5400 4175
-	1    0    0    -1
-$EndComp
-$Comp
-L power:GND #PWR?
+P 5400 4275
+F 0 "J2" H 5400 4475 50  0000 C CNN
+F 1 "Screw_Terminal_01x04" V 5500 4175 50  0001 C CNN
+F 2 "" H 5400 4275 50  0001 C CNN
+F 3 "" H 5400 4275 50  0001 C CNN
+	1    5400 4275
+	1    0    0    -1
+$EndComp
+$Comp
+L power:GND #PWR034
 U 1 1 5E580BF2
-P 5150 4425
-F 0 "#PWR?" H 5150 4175 50  0001 C CNN
-F 1 "GND" H 5150 4275 50  0000 C CNN
-F 2 "" H 5150 4425 50  0001 C CNN
-F 3 "" H 5150 4425 50  0001 C CNN
-	1    5150 4425
-	1    0    0    -1
-$EndComp
-$Comp
-L power:GND #PWR?
+P 5150 4525
+F 0 "#PWR034" H 5150 4275 50  0001 C CNN
+F 1 "GND" H 5150 4375 50  0000 C CNN
+F 2 "" H 5150 4525 50  0001 C CNN
+F 3 "" H 5150 4525 50  0001 C CNN
+	1    5150 4525
+	1    0    0    -1
+$EndComp
+$Comp
+L power:GND #PWR032
 U 1 1 5E580BF8
 P 4675 4175
-F 0 "#PWR?" H 4675 3925 50  0001 C CNN
+F 0 "#PWR032" H 4675 3925 50  0001 C CNN
 F 1 "GND" H 4675 4025 50  0000 C CNN
 F 2 "" H 4675 4175 50  0001 C CNN
@@
 	1    0    0    -1
 $EndComp
-Text Notes 4950 4975 0    60   ~ 0
+Text Notes 4950 5075 0    60   ~ 0
 LABEL POSITIVE AND\nNEGATIVE TERMINALS\nON SILKSCREEN
 $Comp
-L Device:CP1 C?
+L Device:CP1 C22
 U 1 1 5E580BFF
 P 4850 2625
-F 0 "C?" H 4875 2725 50  0000 L CNN
+F 0 "C22" H 4875 2725 50  0000 L CNN
 F 1 "NP_470uF" H 4450 2525 50  0000 L CNN
 F 2 "" H 4850 2625 50  0001 C CNN
@@
 $EndComp
 $Comp
-L custom:SMAJ12A D?
+L custom:SMAJ12A D5
 U 1 1 5E580C05
 P 6150 4175
-F 0 "D?" H 6150 4275 50  0000 C CNN
+F 0 "D5" H 6150 4275 50  0000 C CNN
 F 1 "SMAJ12A" H 6150 4075 50  0000 C CNN
 F 2 "Footprint" H 6150 3975 50  0001 C CNN
@@
 $EndComp
 $Comp
-L power:GND #PWR?
+L power:GND #PWR033
 U 1 1 5E580C0B
 P 6150 4375
-F 0 "#PWR?" H 6150 4125 50  0001 C CNN
+F 0 "#PWR033" H 6150 4125 50  0001 C CNN
 F 1 "GND" H 6150 4225 50  0000 C CNN
 F 2 "" H 6150 4375 50  0001 C CNN
@@
 $EndComp
 $Comp
-L power:+12V #PWR?
+L power:+12V #PWR031
 U 1 1 5E580C11
 P 7450 3725
-F 0 "#PWR?" H 7450 3575 50  0001 C CNN
+F 0 "#PWR031" H 7450 3575 50  0001 C CNN
 F 1 "+12V" H 7450 3865 50  0000 C CNN
 F 2 "" H 7450 3725 50  0001 C CNN
@@
 $EndComp
 $Comp
-L custom:FBMH4532HM681-T L?
+L custom:FBMH4532HM681-T L1
 U 1 1 5E580C17
 P 6800 3875
-F 0 "L?" V 6750 3875 50  0000 C CNN
+F 0 "L1" V 6750 3875 50  0000 C CNN
 F 1 "FBMH4532HM681-T" V 6910 3875 50  0000 C CNN
 F 2 "" H 6800 3875 50  0001 C CNN
@@
 $EndComp
 $Comp
-L custom:DST2080S D?
+L custom:DST2080S D4
 U 1 1 5E580C1D
 P 5750 3875
-F 0 "D?" H 5750 3975 50  0000 C CNN
+F 0 "D4" H 5750 3975 50  0000 C CNN
 F 1 "DST2080S" H 5750 3775 50  0000 C CNN
 F 2 "" H 5750 3875 50  0001 C CNN
@@
 SILKSCREEN:\n12V (12.9V MAX)
 $Comp
-L power:GND #PWR?
+L power:GND #PWR035
 U 1 1 5E580C24
 P 7450 4725
-F 0 "#PWR?" H 7450 4475 50  0001 C CNN
+F 0 "#PWR035" H 7450 4475 50  0001 C CNN
 F 1 "GND" H 7450 4575 50  0000 C CNN
 F 2 "" H 7450 4725 50  0001 C CNN
@@
 Connection ~ 5750 2825
 Wire Wire Line
+	5150 4275 5200 4275
+Wire Wire Line
+	4900 3825 4900 3875
+Wire Wire Line
 	5150 4175 5200 4175
-Wire Wire Line
-	4900 3825 4900 3875
-Wire Wire Line
-	5150 4075 5200 4075
-Connection ~ 5150 4075
-Wire Wire Line
-	5200 4275 5150 4275
-Wire Wire Line
-	5150 4275 5150 4375
+Connection ~ 5150 4175
 Wire Wire Line
 	5200 4375 5150 4375
-Connection ~ 5150 4375
+Wire Wire Line
+	5150 4375 5150 4475
+Wire Wire Line
+	5200 4475 5150 4475
+Connection ~ 5150 4475
 Wire Wire Line
 	4675 3975 4675 4075
@@
 	6650 2825 6650 2875
 Wire Wire Line
-	5150 4075 5150 4175
-Wire Wire Line
-	5150 4375 5150 4425
+	5150 4175 5150 4275
+Wire Wire Line
+	5150 4475 5150 4525
 Wire Wire Line
 	4675 4075 4675 4175
@@
 	6150 3875 6150 4025
 Wire Wire Line
-	5150 3875 5150 4075
+	5150 3875 5150 4175
 Wire Wire Line
 	5150 3875 5500 3875
 $Comp
-L flipdot_driver-rescue:‎CL21A475KLCLQNC‎-custom C?
+L flipdot_driver-rescue:‎CL21A475KLCLQNC‎-custom C25
 U 1 1 5E580C6B
 P 6200 2625
-F 0 "C?" H 6315 2716 50  0000 L CNN
+F 0 "C25" H 6315 2716 50  0000 L CNN
 F 1 "‎CL21A475KLCLQNC‎" H 5250 2175 50  0001 L BNN
 F 2 "Capacitor_SMD:C_0805_2012Metric" H 5250 2075 50  0001 L BNN
@@
 $EndComp
 $Comp
-L flipdot_driver-rescue:‎CL21A475KLCLQNC‎-custom C?
+L flipdot_driver-rescue:‎CL21A475KLCLQNC‎-custom C26
 U 1 1 5E580C73
 P 6650 2625
-F 0 "C?" H 6765 2716 50  0000 L CNN
+F 0 "C26" H 6765 2716 50  0000 L CNN
 F 1 "‎CL21A475KLCLQNC‎" H 5700 2175 50  0001 L BNN
 F 2 "Capacitor_SMD:C_0805_2012Metric" H 5700 2075 50  0001 L BNN
@@
 $EndComp
 $Comp
-L flipdot_driver-rescue:‎ESK476M035AC3AA‎-custom C?
+L flipdot_driver-rescue:‎ESK476M035AC3AA‎-custom C23
 U 1 1 5E580C7B
 P 5300 2625
-F 0 "C?" H 5415 2716 50  0000 L CNN
+F 0 "C23" H 5415 2716 50  0000 L CNN
 F 1 "‎ESK476M035AC3AA‎" H 4350 2175 50  0001 L BNN
 F 2 "" H 4350 2075 50  0001 L BNN
@@
 $EndComp
 $Comp
-L flipdot_driver-rescue:‎ESK476M035AC3AA‎-custom C?
+L flipdot_driver-rescue:‎ESK476M035AC3AA‎-custom C24
 U 1 1 5E580C83
 P 5750 2625
-F 0 "C?" H 5865 2716 50  0000 L CNN
+F 0 "C24" H 5865 2716 50  0000 L CNN
 F 1 "‎ESK476M035AC3AA‎" H 4800 2175 50  0001 L BNN
 F 2 "" H 4800 2075 50  0001 L BNN
@@
 $EndComp
 $Comp
-L Connector:TestPoint TP?
+L Connector:TestPoint TP3
 U 1 1 5E580C89
 P 4900 3825
-F 0 "TP?" H 4900 4025 50  0000 C CNN
+F 0 "TP3" H 4900 4025 50  0000 C CNN
 F 1 "TestPoint" H 4650 3875 50  0001 C CNN
 F 2 "" H 5100 3825 50  0001 C CNN
@@
 $EndComp
 $Comp
-L Connector:TestPoint TP?
+L Connector:TestPoint TP4
 U 1 1 5E580C8F
 P 6375 3825
-F 0 "TP?" H 6375 4025 50  0000 C CNN
+F 0 "TP4" H 6375 4025 50  0000 C CNN
 F 1 "TestPoint" H 6125 3875 50  0001 C CNN
 F 2 "" H 6575 3825 50  0001 C CNN
@@
 $EndComp
 $Comp
-L custom:CRG0603F4K7 R?
+L custom:CRG0603F4K7 R11
 U 1 1 5E580C9C
 P 7450 4125
-F 0 "R?" V 7570 4025 50  0000 L BNN
+F 0 "R11" V 7570 4025 50  0000 L BNN
 F 1 "CRG0603F4K7" H 6700 3675 50  0001 L BNN
 F 2 "Resistor_SMD:R_0603_1608Metric" H 6700 3575 50  0001 L BNN
@@
 $EndComp
 $Comp
-L custom:LED_GENERIC_0805 D?
+L custom:LED_GENERIC_0805 D6
 U 1 1 5E580CA2
 P 7450 4475
-F 0 "D?" H 7510 4495 50  0000 L BNN
+F 0 "D6" H 7510 4495 50  0000 L BNN
 F 1 "LED_GENERIC_0805" H 7100 4275 50  0001 L BNN
 F 2 "Diode_SMD:D_0805_2012Metric" H 7050 4175 50  0001 L BNN
@@
 	7125 3825 7125 3875
 $Comp
-L Connector:TestPoint TP?
+L Connector:TestPoint TP5
 U 1 1 5D09BC5D
 P 7125 3825
-F 0 "TP?" H 7125 4025 50  0000 C CNN
+F 0 "TP5" H 7125 4025 50  0000 C CNN
 F 1 "TestPoint" H 6875 3875 50  0001 C CNN
 F 2 "" H 7325 3825 50  0001 C CNN
