File: POWER_INPUT.sch (KiCad schematic (older format))
At the start: 15 parts, among them J1 Barrel_Jack, J2 Screw_Terminal_01x04

Commit message: automated commit
Parts:
- removed C22: NP_470uF, symbol Device:CP1
- added C?: NP_470uF, symbol custom:NP_470uF
Other:
- note removed: "Need to make my\nown version + footprint\nof this part"
Changed lines of the file:
@@
 LABEL POSITIVE AND\nNEGATIVE TERMINALS\nON SILKSCREEN
-$Comp
-L Device:CP1 C22
-U 1 1 5E580BFF
-P 4850 2625
-F 0 "C22" H 4875 2725 50  0000 L CNN
-F 1 "NP_470uF" H 4450 2525 50  0000 L CNN
-F 2 "" H 4850 2625 50  0001 C CNN
-F 3 "" H 4850 2625 50  0001 C CNN
-	1    4850 2625
-	1    0    0    -1
-$EndComp
 $Comp
 L custom:SMAJ12A D5
@@
 	0    -1   -1   0
 $EndComp
-Text Notes 3725 2625 0    50   ~ 0
-Need to make my\nown version + footprint\nof this part
 Connection ~ 6375 3875
 Wire Wire Line
@@
 Wire Wire Line
 	4575 3875 4900 3875
+$Comp
+L custom:NP_470uF C?
+U 1 1 5CFDB81D
+P 4850 2625
+F 0 "C?" H 4875 2725 50  0000 L CNN
+F 1 "NP_470uF" H 4450 2500 50  0000 L CNN
+F 2 "" H 4850 2625 50  0001 C CNN
+F 3 "~" H 4850 2625 50  0001 C CNN
+	1    4850 2625
+	1    0    0    -1
+$EndComp
 $EndSCHEMATC

Commit message: automated commit
Parts:
- removed R11: CRG0603F4K7, Resistor_SMD:R_0603_1608Metric, symbol custom:CRG0603F4K7
- added R1: CRG0603F4K7, Resistor_SMD:R_0603_1608Metric, symbol custom:CRG0603F4K7
- gave numbers to parts that had none: 1
- renumbered C23 to C2, C24 to C3, C25 to C4, C26 to C5, D4 to D1, D5 to D2, D6 to D3, TP3 to TP1, TP4 to TP2, TP5 to TP3
Connections:
- net +12V: now also R1.1
- net at D3.2 (A): now also R1.2
Changed lines of the file:
@@
 PUT SYMBOL FOR CENTER-POSITIVE\nCONNECTOR, VOLTAGE RANGE, AND\nBARREL JACK DIMENSIONS FOR MATE\nON SILKSCREEN
 $Comp
-L power:GND #PWR030
+L power:GND #PWR02
 U 1 1 5E580BE0
 P 6650 2875
-F 0 "#PWR030" H 6650 2625 50  0001 C CNN
+F 0 "#PWR02" H 6650 2625 50  0001 C CNN
 F 1 "GND" H 6650 2725 50  0000 C CNN
 F 2 "" H 6650 2875 50  0001 C CNN
@@
 $EndComp
 $Comp
-L power:+12V #PWR029
+L power:+12V #PWR01
 U 1 1 5E580BE6
 P 4850 2375
-F 0 "#PWR029" H 4850 2225 50  0001 C CNN
+F 0 "#PWR01" H 4850 2225 50  0001 C CNN
 F 1 "+12V" H 4850 2515 50  0000 C CNN
 F 2 "" H 4850 2375 50  0001 C CNN
@@
 $EndComp
 $Comp
-L power:GND #PWR034
+L power:GND #PWR06
 U 1 1 5E580BF2
 P 5150 4525
-F 0 "#PWR034" H 5150 4275 50  0001 C CNN
+F 0 "#PWR06" H 5150 4275 50  0001 C CNN
 F 1 "GND" H 5150 4375 50  0000 C CNN
 F 2 "" H 5150 4525 50  0001 C CNN
@@
 $EndComp
 $Comp
-L power:GND #PWR032
+L power:GND #PWR04
 U 1 1 5E580BF8
 P 4675 4175
-F 0 "#PWR032" H 4675 3925 50  0001 C CNN
+F 0 "#PWR04" H 4675 3925 50  0001 C CNN
 F 1 "GND" H 4675 4025 50  0000 C CNN
 F 2 "" H 4675 4175 50  0001 C CNN
@@
 LABEL POSITIVE AND\nNEGATIVE TERMINALS\nON SILKSCREEN
 $Comp
-L custom:SMAJ12A D5
+L custom:SMAJ12A D2
 U 1 1 5E580C05
 P 6150 4175
-F 0 "D5" H 6150 4275 50  0000 C CNN
+F 0 "D2" H 6150 4275 50  0000 C CNN
 F 1 "SMAJ12A" H 6150 4075 50  0000 C CNN
 F 2 "Footprint" H 6150 3975 50  0001 C CNN
@@
 $EndComp
 $Comp
-L power:GND #PWR033
+L power:GND #PWR05
 U 1 1 5E580C0B
 P 6150 4375
-F 0 "#PWR033" H 6150 4125 50  0001 C CNN
+F 0 "#PWR05" H 6150 4125 50  0001 C CNN
 F 1 "GND" H 6150 4225 50  0000 C CNN
 F 2 "" H 6150 4375 50  0001 C CNN
@@
 $EndComp
 $Comp
-L power:+12V #PWR031
+L power:+12V #PWR03
 U 1 1 5E580C11
 P 7450 3725
-F 0 "#PWR031" H 7450 3575 50  0001 C CNN
+F 0 "#PWR03" H 7450 3575 50  0001 C CNN
 F 1 "+12V" H 7450 3865 50  0000 C CNN
 F 2 "" H 7450 3725 50  0001 C CNN
@@
 $EndComp
 $Comp
-L custom:DST2080S D4
+L custom:DST2080S D1
 U 1 1 5E580C1D
 P 5750 3875
-F 0 "D4" H 5750 3975 50  0000 C CNN
+F 0 "D1" H 5750 3975 50  0000 C CNN
 F 1 "DST2080S" H 5750 3775 50  0000 C CNN
 F 2 "" H 5750 3875 50  0001 C CNN
@@
 SILKSCREEN:\n12V (12.9V MAX)
 $Comp
-L power:GND #PWR035
+L power:GND #PWR07
 U 1 1 5E580C24
 P 7450 4725
-F 0 "#PWR035" H 7450 4475 50  0001 C CNN
+F 0 "#PWR07" H 7450 4475 50  0001 C CNN
 F 1 "GND" H 7450 4575 50  0000 C CNN
 F 2 "" H 7450 4725 50  0001 C CNN
@@
 	5150 3875 5500 3875
 $Comp
-L flipdot_driver-rescue:‎CL21A475KLCLQNC‎-custom C25
+L flipdot_driver-rescue:‎CL21A475KLCLQNC‎-custom C4
 U 1 1 5E580C6B
 P 6200 2625
-F 0 "C25" H 6315 2716 50  0000 L CNN
+F 0 "C4" H 6315 2716 50  0000 L CNN
 F 1 "‎CL21A475KLCLQNC‎" H 5250 2175 50  0001 L BNN
 F 2 "Capacitor_SMD:C_0805_2012Metric" H 5250 2075 50  0001 L BNN
@@
 $EndComp
 $Comp
-L flipdot_driver-rescue:‎CL21A475KLCLQNC‎-custom C26
+L flipdot_driver-rescue:‎CL21A475KLCLQNC‎-custom C5
 U 1 1 5E580C73
 P 6650 2625
-F 0 "C26" H 6765 2716 50  0000 L CNN
+F 0 "C5" H 6765 2716 50  0000 L CNN
 F 1 "‎CL21A475KLCLQNC‎" H 5700 2175 50  0001 L BNN
 F 2 "Capacitor_SMD:C_0805_2012Metric" H 5700 2075 50  0001 L BNN
@@
 $EndComp
 $Comp
-L flipdot_driver-rescue:‎ESK476M035AC3AA‎-custom C23
+L flipdot_driver-rescue:‎ESK476M035AC3AA‎-custom C2
 U 1 1 5E580C7B
 P 5300 2625
-F 0 "C23" H 5415 2716 50  0000 L CNN
+F 0 "C2" H 5415 2716 50  0000 L CNN
 F 1 "‎ESK476M035AC3AA‎" H 4350 2175 50  0001 L BNN
 F 2 "" H 4350 2075 50  0001 L BNN
@@
 $EndComp
 $Comp
-L flipdot_driver-rescue:‎ESK476M035AC3AA‎-custom C24
+L flipdot_driver-rescue:‎ESK476M035AC3AA‎-custom C3
 U 1 1 5E580C83
 P 5750 2625
-F 0 "C24" H 5865 2716 50  0000 L CNN
+F 0 "C3" H 5865 2716 50  0000 L CNN
 F 1 "‎ESK476M035AC3AA‎" H 4800 2175 50  0001 L BNN
 F 2 "" H 4800 2075 50  0001 L BNN
@@
 $EndComp
 $Comp
-L Connector:TestPoint TP3
+L Connector:TestPoint TP1
 U 1 1 5E580C89
 P 4900 3825
-F 0 "TP3" H 4900 4025 50  0000 C CNN
+F 0 "TP1" H 4900 4025 50  0000 C CNN
 F 1 "TestPoint" H 4650 3875 50  0001 C CNN
 F 2 "" H 5100 3825 50  0001 C CNN
@@
 $EndComp
 $Comp
-L Connector:TestPoint TP4
+L Connector:TestPoint TP2
 U 1 1 5E580C8F
 P 6375 3825
-F 0 "TP4" H 6375 4025 50  0000 C CNN
+F 0 "TP2" H 6375 4025 50  0000 C CNN
 F 1 "TestPoint" H 6125 3875 50  0001 C CNN
 F 2 "" H 6575 3825 50  0001 C CNN
@@
 $EndComp
 $Comp
-L custom:CRG0603F4K7 R11
-U 1 1 5E580C9C
-P 7450 4125
-F 0 "R11" V 7570 4025 50  0000 L BNN
-F 1 "CRG0603F4K7" H 6700 3675 50  0001 L BNN
-F 2 "Resistor_SMD:R_0603_1608Metric" H 6700 3575 50  0001 L BNN
-F 3 "datasheets/PYu-RC_Group_51_RoHS_L_9.pdf" H 6700 3475 50  0001 L BNN
-F 4 "4.7k" V 7470 4065 39  0000 L BNN "Resistance"
-	1    7450 4125
-	1    0    0    -1
-$EndComp
-$Comp
-L custom:LED_GENERIC_0805 D6
+L custom:LED_GENERIC_0805 D3
 U 1 1 5E580CA2
 P 7450 4475
-F 0 "D6" H 7510 4495 50  0000 L BNN
+F 0 "D3" H 7350 4350 50  0000 L BNN
 F 1 "LED_GENERIC_0805" H 7100 4275 50  0001 L BNN
 F 2 "Diode_SMD:D_0805_2012Metric" H 7050 4175 50  0001 L BNN
@@
 	7125 3825 7125 3875
 $Comp
-L Connector:TestPoint TP5
+L Connector:TestPoint TP3
 U 1 1 5D09BC5D
 P 7125 3825
-F 0 "TP5" H 7125 4025 50  0000 C CNN
+F 0 "TP3" H 7125 4025 50  0000 C CNN
 F 1 "TestPoint" H 6875 3875 50  0001 C CNN
 F 2 "" H 7325 3825 50  0001 C CNN
@@
 	4575 3875 4900 3875
 $Comp
-L custom:NP_470uF C?
+L custom:NP_470uF C1
 U 1 1 5CFDB81D
 P 4850 2625
-F 0 "C?" H 4875 2725 50  0000 L CNN
+F 0 "C1" H 4875 2725 50  0000 L CNN
 F 1 "NP_470uF" H 4450 2500 50  0000 L CNN
 F 2 "" H 4850 2625 50  0001 C CNN
@@
 	1    0    0    -1
 $EndComp
+$Comp
+L custom:CRG0603F4K7 R1
+U 1 1 5D63DE6F
+P 7450 4125
+F 0 "R1" H 7520 4145 50  0000 L BNN
+F 1 "CRG0603F4K7" H 6750 3725 50  0001 L BNN
+F 2 "Resistor_SMD:R_0603_1608Metric" H 6750 3625 50  0001 L BNN
+F 3 "/home/dj/datasheets/Pyu-RC_Group_51_RoHS_L_9.pdf" H 6750 3525 50  0001 L BNN
+F 4 "4k7" V 7450 4125 50  0000 C CNN "VALUE"
+F 5 "5%" H 7570 4085 50  0000 C CNN "TOLERANCE"
+	1    7450 4125
+	1    0    0    -1
+$EndComp

Commit message: automated commit
Parts:
- D2: footprint Footprint -> (none)
Other:
- note added: "LABEL VOLTAGE\nON SILKSCREEN"
- note added: "SILKSCREEN:\n12V"
Changed lines of the file:
@@
 F 0 "D2" H 6150 4275 50  0000 C CNN
 F 1 "SMAJ12A" H 6150 4075 50  0000 C CNN
-F 2 "Footprint" H 6150 3975 50  0001 C CNN
+F 2 "" H 6150 3975 50  0001 C CNN
 F 3 "" H 6150 4175 50  0001 C CNN
 	1    6150 4175
@@
 	1    0    0    -1
 $EndComp
+Text Notes 7650 4575 0    60   ~ 0
+SILKSCREEN:\n12V
+Text Notes 7250 3200 0    60   ~ 0
+LABEL VOLTAGE\nON SILKSCREEN
+Wire Notes Line
+	7275 3250 7175 3525
 $EndSCHEMATC

Commit message: automated commit
Parts:
- C1: footprint (none) -> custom:NP_470uF
- C2, C3: footprint (none) -> custom:‎ESK476M035AC3AA‎
- D1: footprint (none) -> Package_TO_SOT_SMD:TO-277B
- D2: footprint (none) -> Diode_SMD:D_SMA
- J2: footprint (none) -> custom:TERMINAL_BLOCK_5mm_1x4
Changed lines of the file:
@@
 F 0 "J2" H 5400 4475 50  0000 C CNN
 F 1 "Screw_Terminal_01x04" V 5500 4175 50  0001 C CNN
-F 2 "" H 5400 4275 50  0001 C CNN
+F 2 "custom:TERMINAL_BLOCK_5mm_1x4" H 5400 4275 50  0001 C CNN
 F 3 "" H 5400 4275 50  0001 C CNN
 	1    5400 4275
@@
 Text Notes 4950 5075 0    60   ~ 0
 LABEL POSITIVE AND\nNEGATIVE TERMINALS\nON SILKSCREEN
-$Comp
-L custom:SMAJ12A D2
-U 1 1 5E580C05
-P 6150 4175
-F 0 "D2" H 6150 4275 50  0000 C CNN
-F 1 "SMAJ12A" H 6150 4075 50  0000 C CNN
-F 2 "" H 6150 3975 50  0001 C CNN
-F 3 "" H 6150 4175 50  0001 C CNN
-	1    6150 4175
-	0    -1   -1   0
-$EndComp
 $Comp
 L power:GND #PWR05
@@
 	0    1    1    0
 $EndComp
-$Comp
-L custom:DST2080S D1
-U 1 1 5E580C1D
-P 5750 3875
-F 0 "D1" H 5750 3975 50  0000 C CNN
-F 1 "DST2080S" H 5750 3775 50  0000 C CNN
-F 2 "" H 5750 3875 50  0001 C CNN
-F 3 "" H 5750 3875 50  0001 C CNN
-	1    5750 3875
-	1    0    0    -1
-$EndComp
 Text Notes 3250 3675 0    60   ~ 0
 SILKSCREEN:\n12V (12.9V MAX)
@@
 Wire Wire Line
 	7450 4325 7450 4275
-Connection ~ 5500 3875
-Wire Wire Line
-	5500 3925 5550 3925
-Wire Wire Line
-	5500 3825 5550 3825
-Wire Wire Line
-	5500 3825 5500 3875
 Wire Wire Line
 	5300 2475 5300 2425
@@
 	4850 2475 4850 2425
 Connection ~ 5300 2425
-Wire Wire Line
-	5900 3875 6150 3875
 Wire Wire Line
 	6375 3825 6375 3875
@@
 	7450 3875 7450 3975
 Wire Wire Line
-	5500 3875 5500 3925
-Wire Wire Line
 	6200 2425 6650 2425
 Wire Wire Line
@@
 Wire Wire Line
 	5150 3875 5150 4175
-Wire Wire Line
-	5150 3875 5500 3875
 $Comp
 L flipdot_driver-rescue:‎CL21A475KLCLQNC‎-custom C4
@@
 F 0 "C2" H 5415 2716 50  0000 L CNN
 F 1 "‎ESK476M035AC3AA‎" H 4350 2175 50  0001 L BNN
-F 2 "" H 4350 2075 50  0001 L BNN
+F 2 "custom:‎ESK476M035AC3AA‎" H 4350 2075 50  0001 L BNN
 F 3 "datasheets/‎KEM_A4004_ESK.pdf" H 4350 1975 50  0001 L BNN
 F 4 "47uF" H 5415 2625 50  0000 L CNN "Capacitance"
@@
 F 0 "C3" H 5865 2716 50  0000 L CNN
 F 1 "‎ESK476M035AC3AA‎" H 4800 2175 50  0001 L BNN
-F 2 "" H 4800 2075 50  0001 L BNN
+F 2 "custom:‎ESK476M035AC3AA‎" H 4800 2075 50  0001 L BNN
 F 3 "datasheets/‎KEM_A4004_ESK.pdf" H 4800 1975 50  0001 L BNN
 F 4 "47uF" H 5865 2625 50  0000 L CNN "Capacitance"
@@
 F 0 "C1" H 4875 2725 50  0000 L CNN
 F 1 "NP_470uF" H 4450 2500 50  0000 L CNN
-F 2 "" H 4850 2625 50  0001 C CNN
+F 2 "custom:NP_470uF" H 4850 2625 50  0001 C CNN
 F 3 "~" H 4850 2625 50  0001 C CNN
 	1    4850 2625
@@
 Wire Notes Line
 	7275 3250 7175 3525
+$Comp
+L custom:SMAJ12A D2
+U 1 1 5E580C05
+P 6150 4175
+F 0 "D2" H 6150 4275 50  0000 C CNN
+F 1 "SMAJ12A" H 6150 4075 50  0000 C CNN
+F 2 "Diode_SMD:D_SMA" H 6150 3975 50  0001 C CNN
+F 3 "" H 6150 4175 50  0001 C CNN
+	1    6150 4175
+	0    -1   -1   0
+$EndComp
+Wire Wire Line
+	5900 3875 6150 3875
+Wire Wire Line
+	5150 3875 5500 3875
+Wire Wire Line
+	5500 3875 5500 3925
+Connection ~ 5500 3875
+Wire Wire Line
+	5500 3825 5500 3875
+Wire Wire Line
+	5500 3825 5550 3825
+Wire Wire Line
+	5500 3925 5550 3925
+$Comp
+L custom:DST2080S D1
+U 1 1 5E580C1D
+P 5750 3875
+F 0 "D1" H 5750 3975 50  0000 C CNN
+F 1 "DST2080S" H 5750 3775 50  0000 C CNN
+F 2 "Package_TO_SOT_SMD:TO-277B" H 5750 3875 50  0001 C CNN
+F 3 "" H 5750 3875 50  0001 C CNN
+	1    5750 3875
+	1    0    0    -1
+$EndComp
 $EndSCHEMATC

Commit message: automated commit
Parts:
- removed L1: FBMH4532HM681-T, symbol custom:FBMH4532HM681-T
- added L1: BLM31SN500SZ1L, Inductor_SMD:L_1206_3216Metric, symbol custom:BLM31SN500SZ1L
- TP1, TP2, TP3: footprint (none) -> custom:TestPoint_THTPad_D1.0mm_Drill0.5mm
Connections:
- net +12V: now also L1.1
- net at D1.3 (K), D2.1 (K), TP2.1: now also L1.2
Changed lines of the file:
@@
 	1    0    0    -1
-$EndComp
-$Comp
-L custom:FBMH4532HM681-T L1
-U 1 1 5E580C17
-P 6800 3875
-F 0 "L1" V 6750 3875 50  0000 C CNN
-F 1 "FBMH4532HM681-T" V 6910 3875 50  0000 C CNN
-F 2 "" H 6800 3875 50  0001 C CNN
-F 3 "" H 6800 3875 50  0001 C CNN
-	1    6800 3875
-	0    1    1    0
 $EndComp
 Text Notes 3250 3675 0    60   ~ 0
@@
 F 0 "TP1" H 4900 4025 50  0000 C CNN
 F 1 "TestPoint" H 4650 3875 50  0001 C CNN
-F 2 "" H 5100 3825 50  0001 C CNN
+F 2 "custom:TestPoint_THTPad_D1.0mm_Drill0.5mm" H 5100 3825 50  0001 C CNN
 F 3 "~" H 5100 3825 50  0001 C CNN
 	1    4900 3825
@@
 F 0 "TP2" H 6375 4025 50  0000 C CNN
 F 1 "TestPoint" H 6125 3875 50  0001 C CNN
-F 2 "" H 6575 3825 50  0001 C CNN
+F 2 "custom:TestPoint_THTPad_D1.0mm_Drill0.5mm" H 6575 3825 50  0001 C CNN
 F 3 "~" H 6575 3825 50  0001 C CNN
 	1    6375 3825
@@
 F 0 "TP3" H 7125 4025 50  0000 C CNN
 F 1 "TestPoint" H 6875 3875 50  0001 C CNN
-F 2 "" H 7325 3825 50  0001 C CNN
+F 2 "custom:TestPoint_THTPad_D1.0mm_Drill0.5mm" H 7325 3825 50  0001 C CNN
 F 3 "~" H 7325 3825 50  0001 C CNN
 	1    7125 3825
@@
 	1    0    0    -1
 $EndComp
+Wire Notes Line
+	7175 3250 6500 3600
+Wire Notes Line
+	7025 3250 5050 3600
+$Comp
+L custom:BLM31SN500SZ1L L1
+U 1 1 5D15E000
+P 6800 3875
+F 0 "L1" V 6750 3875 50  0000 C CNN
+F 1 "BLM31SN500SZ1L" V 6925 3875 50  0001 C CNN
+F 2 "Inductor_SMD:L_1206_3216Metric" H 6800 3425 50  0001 C CNN
+F 3 "" H 6800 3875 50  0001 C CNN
+F 4 "50ohm @ 100MHz" V 7000 3875 50  0001 C CNN "IMPEDANCE"
+	1    6800 3875
+	0    1    1    0
+$EndComp
 $EndSCHEMATC

Commit message: automated commit
Parts:
- J1: footprint Connectors:BARREL_JACK -> Connector_BarrelJack:BarrelJack_Wuerth_6941xx301002
Changed lines of the file:
@@
 F 0 "J1" H 4275 4185 50  0000 C CNN
 F 1 "Barrel_Jack" H 4275 3775 50  0000 C CNN
-F 2 "Connectors:BARREL_JACK" H 4325 3935 50  0001 C CNN
+F 2 "Connector_BarrelJack:BarrelJack_Wuerth_6941xx301002" H 4325 3935 50  0001 C CNN
 F 3 "" H 4325 3935 50  0001 C CNN
 	1    4275 3975
