File: ROW_DRIVERS_0.sch (KiCad schematic (older format))
At the start: 40 parts

Commit message: automated commit
Connections:
- net ROW00N: no longer D?.1 (K), D?.1 (K), D?.1 (K), Q?.6 (D), Q?.6 (D), Q?.6 (D)
- net ROW00P: no longer D?.2 (A), D?.2 (A), D?.2 (A), Q?.4 (D), Q?.4 (D), Q?.4 (D)
- net ROW00_OFF: no longer R?.1, R?.1, R?.1, R?.2, R?.2, R?.2
- net ROW00_ON: no longer Q?.1 (G), Q?.1 (G), Q?.1 (G), Q?.1 (G), Q?.1 (G), Q?.1 (G), R?.1, R?.1, R?.1
- new net ROW01N: D?.1 (K), Q?.6 (D)
- new net ROW01P: D?.2 (A), Q?.4 (D)
- new net ROW01_OFF: R?.1, R?.2
- new net ROW01_ON: Q?.1 (G), Q?.1 (G), R?.1
- new net ROW02N: D?.1 (K), Q?.6 (D)
- new net ROW02P: D?.2 (A), Q?.4 (D)
- new net ROW02_OFF: R?.1, R?.2
- new net ROW02_ON: Q?.1 (G), Q?.1 (G), R?.1
- new net ROW03N: D?.1 (K), Q?.6 (D)
- new net ROW03P: D?.2 (A), Q?.4 (D)
- new net ROW03_OFF: R?.1, R?.2
- new net ROW03_ON: Q?.1 (G), Q?.1 (G), R?.1
Other:
- moved on the sheet: D?, Q?, Q?A, Q?B, R?

Commit message: automated commit
Parts:
- gave numbers to parts that had none: 36
