File: ROW_DRIVERS_0.sch (KiCad schematic (older format))
At the start: 36 parts, among them Q100 SSM3K35AMFV, Q101 SSM3K35AMFV, Q102 DMG6602, Q103 DMG6602, Q104 SSM3K35AMFV, Q105 SSM3K35AMFV, Q106 SSM3K35AMFV, Q107 SSM3K35AMFV, Q96 DMG6602, Q97 DMG6602, Q98 SSM3K35AMFV, Q99 SSM3K35AMFV

Commit message: automated commit
Parts:
- removed D26, D27: MMBZ5243BLT1G, symbol custom:MMBZ5243BLT1G
- removed Q101, Q104, Q105, Q106, Q107, Q99: SSM3K35AMFV, symbol custom:SSM3K35AMFV
- removed Q102, Q103, Q97: DMG6602, Package_TO_SOT_SMD:TSOT-23-6, symbol custom:DMG6602
- removed R178, R179, R180, R181, R182, R183, R184, R185, R186, R187, R188, R189, R190, R191, R192, R193: CRG0603F4K7, Resistor_SMD:R_0603_1608Metric, symbol custom:CRG0603F4K7
- added D19, D22: MMBZ5243BLT1G, symbol custom:MMBZ5243BLT1G
- added Q17, Q21, Q22: DMG6602, Package_TO_SOT_SMD:TSOT-23-6, symbol custom:DMG6602
- added Q19, Q23, Q24: SSM3K35AMFV, symbol custom:SSM3K35AMFV
- added R100, R101, R102, R90, R91, R92, R93, R94, R95, R96, R97, R98, R99: CRG0603F4K7, Resistor_SMD:R_0603_1608Metric, symbol custom:CRG0603F4K7
- renumbered D20 to D18, D22 to D20, Q96 to Q16, Q98 to Q18, Q100 to Q20
Connections:
- net +12V: now also D23.1 (K), D19.1 (K), D22.1 (K), Q17.2 (S), Q21.2 (S), Q22.2 (S), R90.1, R91.1, R97.1, R98.1; no longer D21.1 (K), D24.1 (K), D25.1 (K)
- net GND: now also D21.2 (A), D24.2 (A), D25.2 (A), Q17.5 (S), Q19.2 (S), Q21.5 (S), Q22.5 (S), Q23.2 (S), Q24.2 (S), R100.2, R101.2, R102.2, R92.2, R93.2, R95.2, R96.2, R99.2; no longer D23.2 (A)
- net ROW00_OFF: now also R94.2, R96.1
- net ROW00_ON: now also R92.1
- net ROW01N: now also D21.1 (K), Q17.6 (D); no longer D23.1 (K)
- net ROW01P: now also D19.2 (A), Q17.4 (D); no longer D21.2 (A)
- net ROW01_OFF: now also Q17.1 (G), R95.1
- net ROW01_ON: now also Q19.1 (G), R93.1
- net ROW02N: now also D24.1 (K), Q21.6 (D)
- net ROW02P: now also D22.2 (A), Q21.4 (D); no longer D24.2 (A)
- net ROW02_OFF: now also Q21.1 (G), R101.1
- net ROW02_ON: now also Q23.1 (G), R99.1
- net ROW03N: now also D25.1 (K), Q22.6 (D)
- net ROW03P: now also D23.2 (A), Q22.4 (D); no longer D25.2 (A)
- net ROW03_OFF: now also Q22.1 (G), R102.1
- net ROW03_ON: now also Q24.1 (G), R100.1
- net at Q16.1 (G), Q20.3 (D): now also R94.1
- net at Q16.3 (G), Q18.3 (D): now also R90.2
- new net: Q17.3 (G), Q19.3 (D), R91.2
- new net: Q22.3 (G), Q24.3 (D), R98.2
- new net: Q21.3 (G), Q23.3 (D), R97.2
Other:
- note removed: "TVS DIODES ALLOW THE ROW TRANSISTORS TO BE SHUT OFF\nBEFORE THE COLUMN TRANSISTOR. WITHOUT IT, SHUTTING OFF\nTHE ROW TRANSISTOR MAY CAUSE AN INDUCTIVE SPIKEACROSS\nTHE RESISTOR, BLOWING OUT ITS BODY DIODE."
- moved on the sheet: D18, D20, Q16A, Q16B, Q18, Q20

Commit message: automated commit
Parts:
- added TP58, TP59, TP60, TP61, TP62, TP63, TP64, TP65, TP66, TP67, TP68, TP69, TP70, TP71, TP72, TP73: TestPoint, symbol Connector:TestPoint
- renumbered R90 to R86, R91 to R87, R92 to R88, R93 to R89, R94 to R90, R95 to R91, R96 to R92, R97 to R93, R98 to R94, R99 to R95, R100 to R96, R101 to R97, R102 to R98
Connections:
- net +12V: now also TP58.1
- net GND: now also TP65.1, TP66.1, TP72.1, TP73.1
- net ROW00N: now also TP68.1
- net ROW00P: now also TP63.1
- net ROW00_OFF: now also TP69.1
- net ROW00_ON: now also TP61.1
- net ROW01N: now also TP67.1
- net ROW01P: now also TP64.1
- net ROW01_OFF: now also TP71.1
- net ROW01_ON: now also TP62.1
- net at Q16.3 (G), Q18.3 (D), R86.2: now also TP59.1
- net at Q16.1 (G), Q20.3 (D), R90.1: now also TP70.1
- net at Q17.3 (G), Q19.3 (D), R87.2: now also TP60.1
Other:
- moved on the sheet: D20, Q16A, Q16B, Q17A, Q17B, Q18, Q19, Q20, R86, R87, R88, R89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

Commit message: automated commit
Parts:
- D18, D19, D20, D21, D22, D23, D24, D25: footprint (none) -> Package_TO_SOT_SMD:SOT-23
- Q18, Q19, Q20, Q23, Q24: footprint (none) -> Package_TO_SOT_SMD:SOT-723
Changed lines of the file:
@@
 F 0 "Q18" V 1950 1925 50  0000 L BNN
 F 1 "SSM3K35AMFV" V 1875 1750 50  0000 L BNN
-F 2 "" H 1825 1875 50  0001 L BIN
+F 2 "Package_TO_SOT_SMD:SOT-723" H 1825 1875 50  0001 L BIN
 F 3 "datasheets/SSM3K35AMFV.pdf" H 1825 1850 50  0001 L BNN
 	1    1625 2000
@@
 F 0 "Q20" V 2625 3625 50  0000 L BNN
 F 1 "SSM3K35AMFV" V 2550 3450 50  0000 L BNN
-F 2 "" H 2500 3575 50  0001 L BIN
+F 2 "Package_TO_SOT_SMD:SOT-723" H 2500 3575 50  0001 L BIN
 F 3 "datasheets/SSM3K35AMFV.pdf" H 2500 3550 50  0001 L BNN
 	1    2300 3700
@@
 F 0 "D20" H 3400 3275 50  0000 C CNN
 F 1 "MMBZ5243BLT1G" H 3375 3425 50  0000 C CNN
-F 2 "" V 3275 3325 50  0001 C CNN
+F 2 "Package_TO_SOT_SMD:SOT-23" V 3275 3325 50  0001 C CNN
 F 3 "" H 3275 3415 50  0001 C CNN
 F 4 "13V" H 3150 3275 39  0000 C CNN "Rating"
@@
 F 0 "Q19" V 5350 1925 50  0000 L BNN
 F 1 "SSM3K35AMFV" V 5275 1750 50  0000 L BNN
-F 2 "" H 5225 1875 50  0001 L BIN
+F 2 "Package_TO_SOT_SMD:SOT-723" H 5225 1875 50  0001 L BIN
 F 3 "datasheets/SSM3K35AMFV.pdf" H 5225 1850 50  0001 L BNN
 	1    5025 2000
@@
 F 0 "Q24" V 5250 5600 50  0000 L BNN
 F 1 "SSM3K35AMFV" V 5175 5425 50  0000 L BNN
-F 2 "" H 5125 5550 50  0001 L BIN
+F 2 "Package_TO_SOT_SMD:SOT-723" H 5125 5550 50  0001 L BIN
 F 3 "datasheets/SSM3K35AMFV.pdf" H 5125 5525 50  0001 L BNN
 	1    4925 5675
@@
 F 0 "Q23" V 1850 5600 50  0000 L BNN
 F 1 "SSM3K35AMFV" V 1775 5425 50  0000 L BNN
-F 2 "" H 1725 5550 50  0001 L BIN
+F 2 "Package_TO_SOT_SMD:SOT-723" H 1725 5550 50  0001 L BIN
 F 3 "datasheets/SSM3K35AMFV.pdf" H 1725 5525 50  0001 L BNN
 	1    1525 5675
@@
 F 0 "D18" H 2900 1575 50  0000 C CNN
 F 1 "MMBZ5243BLT1G" H 2775 1725 50  0000 C CNN
-F 2 "" V 2775 1625 50  0001 C CNN
+F 2 "Package_TO_SOT_SMD:SOT-23" V 2775 1625 50  0001 C CNN
 F 3 "" H 2775 1715 50  0001 C CNN
 F 4 "13V" H 2650 1575 39  0000 C CNN "Rating"
@@
 F 0 "D21" H 6100 3275 50  0000 C CNN
 F 1 "MMBZ5243BLT1G" H 6075 3425 50  0000 C CNN
-F 2 "" V 5975 3325 50  0001 C CNN
+F 2 "Package_TO_SOT_SMD:SOT-23" V 5975 3325 50  0001 C CNN
 F 3 "" H 5975 3415 50  0001 C CNN
 F 4 "13V" H 5850 3275 39  0000 C CNN "Rating"
@@
 F 0 "D19" H 6300 1575 50  0000 C CNN
 F 1 "MMBZ5243BLT1G" H 6175 1725 50  0000 C CNN
-F 2 "" V 6175 1625 50  0001 C CNN
+F 2 "Package_TO_SOT_SMD:SOT-23" V 6175 1625 50  0001 C CNN
 F 3 "" H 6175 1715 50  0001 C CNN
 F 4 "13V" H 6050 1575 39  0000 C CNN "Rating"
@@
 F 0 "D24" H 2600 6700 50  0000 C CNN
 F 1 "MMBZ5243BLT1G" H 2575 6850 50  0000 C CNN
-F 2 "" V 2475 6750 50  0001 C CNN
+F 2 "Package_TO_SOT_SMD:SOT-23" V 2475 6750 50  0001 C CNN
 F 3 "" H 2475 6840 50  0001 C CNN
 F 4 "13V" H 2350 6700 39  0000 C CNN "Rating"
@@
 F 0 "D22" H 2800 5250 50  0000 C CNN
 F 1 "MMBZ5243BLT1G" H 2675 5400 50  0000 C CNN
-F 2 "" V 2675 5300 50  0001 C CNN
+F 2 "Package_TO_SOT_SMD:SOT-23" V 2675 5300 50  0001 C CNN
 F 3 "" H 2675 5390 50  0001 C CNN
 F 4 "13V" H 2550 5250 39  0000 C CNN "Rating"
@@
 F 0 "D25" H 6000 6700 50  0000 C CNN
 F 1 "MMBZ5243BLT1G" H 5975 6850 50  0000 C CNN
-F 2 "" V 5875 6750 50  0001 C CNN
+F 2 "Package_TO_SOT_SMD:SOT-23" V 5875 6750 50  0001 C CNN
 F 3 "" H 5875 6840 50  0001 C CNN
 F 4 "13V" H 5750 6700 39  0000 C CNN "Rating"
@@
 F 0 "D23" H 6200 5250 50  0000 C CNN
 F 1 "MMBZ5243BLT1G" H 6075 5400 50  0000 C CNN
-F 2 "" V 6075 5300 50  0001 C CNN
+F 2 "Package_TO_SOT_SMD:SOT-23" V 6075 5300 50  0001 C CNN
 F 3 "" H 6075 5390 50  0001 C CNN
 F 4 "13V" H 5950 5250 39  0000 C CNN "Rating"

Commit message: automated commit
Parts:
- TP63: renamed from TP58; footprint (none) -> custom:TestPoint_THTPad_D1.0mm_Drill0.5mm
- TP64: renamed from TP59; footprint (none) -> custom:TestPoint_THTPad_D1.0mm_Drill0.5mm
- TP65: renamed from TP60; footprint (none) -> custom:TestPoint_THTPad_D1.0mm_Drill0.5mm
- TP66: renamed from TP61; footprint (none) -> custom:TestPoint_THTPad_D1.0mm_Drill0.5mm
- TP67: renamed from TP62; footprint (none) -> custom:TestPoint_THTPad_D1.0mm_Drill0.5mm
- TP68: renamed from TP63; footprint (none) -> custom:TestPoint_THTPad_D1.0mm_Drill0.5mm
- TP69: renamed from TP64; footprint (none) -> custom:TestPoint_THTPad_D1.0mm_Drill0.5mm
- TP70: renamed from TP65; footprint (none) -> custom:TestPoint_THTPad_D1.0mm_Drill0.5mm
- TP71: renamed from TP66; footprint (none) -> custom:TestPoint_THTPad_D1.0mm_Drill0.5mm
- TP72: renamed from TP67; footprint (none) -> custom:TestPoint_THTPad_D1.0mm_Drill0.5mm
- TP73: renamed from TP68; footprint (none) -> custom:TestPoint_THTPad_D1.0mm_Drill0.5mm
- TP74: renamed from TP69; footprint (none) -> custom:TestPoint_THTPad_D1.0mm_Drill0.5mm
- TP75: renamed from TP70; footprint (none) -> custom:TestPoint_THTPad_D1.0mm_Drill0.5mm
- TP76: renamed from TP71; footprint (none) -> custom:TestPoint_THTPad_D1.0mm_Drill0.5mm
- TP77: renamed from TP72; footprint (none) -> custom:TestPoint_THTPad_D1.0mm_Drill0.5mm
- TP78: renamed from TP73; footprint (none) -> custom:TestPoint_THTPad_D1.0mm_Drill0.5mm
Changed lines of the file:
@@
 AR Path="/609E0ED6/5D8A9673" Ref="TP?"  Part="1"
 AR Path="/621F0CB4/5D8A9673" Ref="TP?"  Part="1"
-AR Path="/62CDD30D/5D8A9673" Ref="TP58"  Part="1"
-F 0 "TP58" V 2250 1375 50  0000 C CNN
+AR Path="/62CDD30D/5D8A9673" Ref="TP63"  Part="1"
+F 0 "TP63" V 2250 1375 50  0000 C CNN
 F 1 "TestPoint" H 2100 1250 50  0001 C CNN
-F 2 "" H 2550 1200 50  0001 C CNN
+F 2 "custom:TestPoint_THTPad_D1.0mm_Drill0.5mm" H 2550 1200 50  0001 C CNN
 F 3 "~" H 2550 1200 50  0001 C CNN
 	1    2350 1200
@@
 AR Path="/609E0ED6/5D8B6234" Ref="TP?"  Part="1"
 AR Path="/621F0CB4/5D8B6234" Ref="TP?"  Part="1"
-AR Path="/62CDD30D/5D8B6234" Ref="TP59"  Part="1"
-F 0 "TP59" V 1550 1725 50  0000 C CNN
+AR Path="/62CDD30D/5D8B6234" Ref="TP64"  Part="1"
+F 0 "TP64" V 1550 1725 50  0000 C CNN
 F 1 "TestPoint" H 1400 1600 50  0001 C CNN
-F 2 "" H 1850 1550 50  0001 C CNN
+F 2 "custom:TestPoint_THTPad_D1.0mm_Drill0.5mm" H 1850 1550 50  0001 C CNN
 F 3 "~" H 1850 1550 50  0001 C CNN
 	1    1650 1550
@@
 AR Path="/609E0ED6/5D8C35A8" Ref="TP?"  Part="1"
 AR Path="/621F0CB4/5D8C35A8" Ref="TP?"  Part="1"
-AR Path="/62CDD30D/5D8C35A8" Ref="TP61"  Part="1"
-F 0 "TP61" H 1225 2150 50  0000 C CNN
+AR Path="/62CDD30D/5D8C35A8" Ref="TP66"  Part="1"
+F 0 "TP66" H 1225 2150 50  0000 C CNN
 F 1 "TestPoint" H 975 1975 50  0001 C CNN
-F 2 "" H 1425 1925 50  0001 C CNN
+F 2 "custom:TestPoint_THTPad_D1.0mm_Drill0.5mm" H 1425 1925 50  0001 C CNN
 F 3 "~" H 1425 1925 50  0001 C CNN
 	1    1225 1925
@@
 AR Path="/609E0ED6/5D8CA355" Ref="TP?"  Part="1"
 AR Path="/621F0CB4/5D8CA355" Ref="TP?"  Part="1"
-AR Path="/62CDD30D/5D8CA355" Ref="TP65"  Part="1"
-F 0 "TP65" V 1950 2500 50  0000 C CNN
+AR Path="/62CDD30D/5D8CA355" Ref="TP70"  Part="1"
+F 0 "TP70" V 1950 2500 50  0000 C CNN
 F 1 "TestPoint" H 1600 2400 50  0001 C CNN
-F 2 "" H 2050 2350 50  0001 C CNN
+F 2 "custom:TestPoint_THTPad_D1.0mm_Drill0.5mm" H 2050 2350 50  0001 C CNN
 F 3 "~" H 2050 2350 50  0001 C CNN
 	1    1850 2350
@@
 AR Path="/609E0ED6/5D8DEDF0" Ref="TP?"  Part="1"
 AR Path="/621F0CB4/5D8DEDF0" Ref="TP?"  Part="1"
-AR Path="/62CDD30D/5D8DEDF0" Ref="TP63"  Part="1"
-F 0 "TP63" H 2150 2200 50  0000 C CNN
+AR Path="/62CDD30D/5D8DEDF0" Ref="TP68"  Part="1"
+F 0 "TP68" H 2150 2200 50  0000 C CNN
 F 1 "TestPoint" H 2025 2100 50  0001 C CNN
-F 2 "" H 2475 2050 50  0001 C CNN
+F 2 "custom:TestPoint_THTPad_D1.0mm_Drill0.5mm" H 2475 2050 50  0001 C CNN
 F 3 "~" H 2475 2050 50  0001 C CNN
 	1    2275 2050
@@
 AR Path="/609E0ED6/5D8F3B29" Ref="TP?"  Part="1"
 AR Path="/621F0CB4/5D8F3B29" Ref="TP?"  Part="1"
-AR Path="/62CDD30D/5D8F3B29" Ref="TP68"  Part="1"
-F 0 "TP68" V 2625 3200 50  0000 C CNN
+AR Path="/62CDD30D/5D8F3B29" Ref="TP73"  Part="1"
+F 0 "TP73" V 2625 3200 50  0000 C CNN
 F 1 "TestPoint" H 2475 3075 50  0001 C CNN
-F 2 "" H 2925 3025 50  0001 C CNN
+F 2 "custom:TestPoint_THTPad_D1.0mm_Drill0.5mm" H 2925 3025 50  0001 C CNN
 F 3 "~" H 2925 3025 50  0001 C CNN
 	1    2725 3025
@@
 AR Path="/609E0ED6/5D8FAF4C" Ref="TP?"  Part="1"
 AR Path="/621F0CB4/5D8FAF4C" Ref="TP?"  Part="1"
-AR Path="/62CDD30D/5D8FAF4C" Ref="TP72"  Part="1"
-F 0 "TP72" H 3275 3975 50  0000 C CNN
+AR Path="/62CDD30D/5D8FAF4C" Ref="TP77"  Part="1"
+F 0 "TP77" H 3275 3975 50  0000 C CNN
 F 1 "TestPoint" H 3025 3800 50  0001 C CNN
-F 2 "" H 3475 3750 50  0001 C CNN
+F 2 "custom:TestPoint_THTPad_D1.0mm_Drill0.5mm" H 3475 3750 50  0001 C CNN
 F 3 "~" H 3475 3750 50  0001 C CNN
 	1    3275 3750
@@
 AR Path="/609E0ED6/5D9267BD" Ref="TP?"  Part="1"
 AR Path="/621F0CB4/5D9267BD" Ref="TP?"  Part="1"
-AR Path="/62CDD30D/5D9267BD" Ref="TP69"  Part="1"
-F 0 "TP69" H 1425 3475 50  0000 C CNN
+AR Path="/62CDD30D/5D9267BD" Ref="TP74"  Part="1"
+F 0 "TP74" H 1425 3475 50  0000 C CNN
 F 1 "TestPoint" H 1175 3300 50  0001 C CNN
-F 2 "" H 1625 3250 50  0001 C CNN
+F 2 "custom:TestPoint_THTPad_D1.0mm_Drill0.5mm" H 1625 3250 50  0001 C CNN
 F 3 "~" H 1625 3250 50  0001 C CNN
 	1    1425 3250
@@
 AR Path="/609E0ED6/5D92DD7D" Ref="TP?"  Part="1"
 AR Path="/621F0CB4/5D92DD7D" Ref="TP?"  Part="1"
-AR Path="/62CDD30D/5D92DD7D" Ref="TP70"  Part="1"
-F 0 "TP70" H 2225 3475 50  0000 C CNN
+AR Path="/62CDD30D/5D92DD7D" Ref="TP75"  Part="1"
+F 0 "TP75" H 2225 3475 50  0000 C CNN
 F 1 "TestPoint" H 1975 3300 50  0001 C CNN
-F 2 "" H 2425 3250 50  0001 C CNN
+F 2 "custom:TestPoint_THTPad_D1.0mm_Drill0.5mm" H 2425 3250 50  0001 C CNN
 F 3 "~" H 2425 3250 50  0001 C CNN
 	1    2225 3250
@@
 AR Path="/609E0ED6/5D9363B5" Ref="TP?"  Part="1"
 AR Path="/621F0CB4/5D9363B5" Ref="TP?"  Part="1"
-AR Path="/62CDD30D/5D9363B5" Ref="TP60"  Part="1"
-F 0 "TP60" V 4950 1725 50  0000 C CNN
+AR Path="/62CDD30D/5D9363B5" Ref="TP65"  Part="1"
+F 0 "TP65" V 4950 1725 50  0000 C CNN
 F 1 "TestPoint" H 4800 1600 50  0001 C CNN
-F 2 "" H 5250 1550 50  0001 C CNN
+F 2 "custom:TestPoint_THTPad_D1.0mm_Drill0.5mm" H 5250 1550 50  0001 C CNN
 F 3 "~" H 5250 1550 50  0001 C CNN
 	1    5050 1550
@@
 AR Path="/609E0ED6/5D9363BC" Ref="TP?"  Part="1"
 AR Path="/621F0CB4/5D9363BC" Ref="TP?"  Part="1"
-AR Path="/62CDD30D/5D9363BC" Ref="TP62"  Part="1"
-F 0 "TP62" H 4625 2150 50  0000 C CNN
+AR Path="/62CDD30D/5D9363BC" Ref="TP67"  Part="1"
+F 0 "TP67" H 4625 2150 50  0000 C CNN
 F 1 "TestPoint" H 4375 1975 50  0001 C CNN
-F 2 "" H 4825 1925 50  0001 C CNN
+F 2 "custom:TestPoint_THTPad_D1.0mm_Drill0.5mm" H 4825 1925 50  0001 C CNN
 F 3 "~" H 4825 1925 50  0001 C CNN
 	1    4625 1925
@@
 AR Path="/609E0ED6/5D94EF08" Ref="TP?"  Part="1"
 AR Path="/621F0CB4/5D94EF08" Ref="TP?"  Part="1"
-AR Path="/62CDD30D/5D94EF08" Ref="TP66"  Part="1"
-F 0 "TP66" V 5350 2500 50  0000 C CNN
+AR Path="/62CDD30D/5D94EF08" Ref="TP71"  Part="1"
+F 0 "TP71" V 5350 2500 50  0000 C CNN
 F 1 "TestPoint" H 5000 2400 50  0001 C CNN
-F 2 "" H 5450 2350 50  0001 C CNN
+F 2 "custom:TestPoint_THTPad_D1.0mm_Drill0.5mm" H 5450 2350 50  0001 C CNN
 F 3 "~" H 5450 2350 50  0001 C CNN
 	1    5250 2350
@@
 AR Path="/609E0ED6/5D94EF0F" Ref="TP?"  Part="1"
 AR Path="/621F0CB4/5D94EF0F" Ref="TP?"  Part="1"
-AR Path="/62CDD30D/5D94EF0F" Ref="TP64"  Part="1"
-F 0 "TP64" H 5550 2200 50  0000 C CNN
+AR Path="/62CDD30D/5D94EF0F" Ref="TP69"  Part="1"
+F 0 "TP69" H 5550 2200 50  0000 C CNN
 F 1 "TestPoint" H 5425 2100 50  0001 C CNN
-F 2 "" H 5875 2050 50  0001 C CNN
+F 2 "custom:TestPoint_THTPad_D1.0mm_Drill0.5mm" H 5875 2050 50  0001 C CNN
 F 3 "~" H 5875 2050 50  0001 C CNN
 	1    5675 2050
@@
 AR Path="/609E0ED6/5D95F68E" Ref="TP?"  Part="1"
 AR Path="/621F0CB4/5D95F68E" Ref="TP?"  Part="1"
-AR Path="/62CDD30D/5D95F68E" Ref="TP71"  Part="1"
-F 0 "TP71" H 4925 3475 50  0000 C CNN
+AR Path="/62CDD30D/5D95F68E" Ref="TP76"  Part="1"
+F 0 "TP76" H 4925 3475 50  0000 C CNN
 F 1 "TestPoint" H 4675 3300 50  0001 C CNN
-F 2 "" H 5125 3250 50  0001 C CNN
+F 2 "custom:TestPoint_THTPad_D1.0mm_Drill0.5mm" H 5125 3250 50  0001 C CNN
 F 3 "~" H 5125 3250 50  0001 C CNN
 	1    4925 3250
@@
 AR Path="/609E0ED6/5D96862D" Ref="TP?"  Part="1"
 AR Path="/621F0CB4/5D96862D" Ref="TP?"  Part="1"
-AR Path="/62CDD30D/5D96862D" Ref="TP73"  Part="1"
-F 0 "TP73" H 5975 3975 50  0000 C CNN
+AR Path="/62CDD30D/5D96862D" Ref="TP78"  Part="1"
+F 0 "TP78" H 5975 3975 50  0000 C CNN
 F 1 "TestPoint" H 5725 3800 50  0001 C CNN
-F 2 "" H 6175 3750 50  0001 C CNN
+F 2 "custom:TestPoint_THTPad_D1.0mm_Drill0.5mm" H 6175 3750 50  0001 C CNN
 F 3 "~" H 6175 3750 50  0001 C CNN
 	1    5975 3750
@@
 AR Path="/609E0ED6/5D971623" Ref="TP?"  Part="1"
 AR Path="/621F0CB4/5D971623" Ref="TP?"  Part="1"
-AR Path="/62CDD30D/5D971623" Ref="TP67"  Part="1"
-F 0 "TP67" H 5750 3175 50  0000 C CNN
+AR Path="/62CDD30D/5D971623" Ref="TP72"  Part="1"
+F 0 "TP72" H 5750 3175 50  0000 C CNN
 F 1 "TestPoint" H 5500 3000 50  0001 C CNN
-F 2 "" H 5950 2950 50  0001 C CNN
+F 2 "custom:TestPoint_THTPad_D1.0mm_Drill0.5mm" H 5950 2950 50  0001 C CNN
 F 3 "~" H 5950 2950 50  0001 C CNN
 	1    5750 2950
