File: ROW_DRIVERS_0.sch (KiCad schematic (older format))
At the start: 46 parts, among them Q16 DMG6602, Q17 DMG6602, Q18 SSM3K35AMFV, Q19 SSM3K35AMFV, Q20 SSM3K35AMFV, Q21 DMG6602, Q22 DMG6602, Q23 SSM3K35AMFV, Q24 SSM3K35AMFV

Commit message: automated commit
Parts:
- renumbered R92 to R100, R93 to R101, R94 to R102, R95 to R103, R96 to R104, R97 to R105, R98 to R106, R86 to R94, R87 to R95, R88 to R96, R89 to R97, R90 to R98, R91 to R99
Changed lines of the file:
@@
 $EndDescr
 $Comp
-L power:GND #PWR0173
+L power:GND #PWR0175
 U 1 1 62CEC058
 P 2800 4025
-F 0 "#PWR0173" H 2800 3775 50  0001 C CNN
+F 0 "#PWR0175" H 2800 3775 50  0001 C CNN
 F 1 "GND" H 2800 3875 50  0000 C CNN
 F 2 "" H 2800 4025 50  0001 C CNN
@@
 $EndComp
 $Comp
-L power:+12V #PWR0168
+L power:+12V #PWR0170
 U 1 1 62CEC05E
 P 2275 950
-F 0 "#PWR0168" H 2275 800 50  0001 C CNN
+F 0 "#PWR0170" H 2275 800 50  0001 C CNN
 F 1 "+12V" H 2275 1090 50  0000 C CNN
 F 2 "" H 2275 950 50  0001 C CNN
@@
 $EndComp
 $Comp
-L power:GND #PWR0170
+L power:GND #PWR0172
 U 1 1 62CEC068
 P 1725 2500
-F 0 "#PWR0170" H 1725 2250 50  0001 C CNN
+F 0 "#PWR0172" H 1725 2250 50  0001 C CNN
 F 1 "GND" H 1725 2350 50  0000 C CNN
 F 2 "" H 1725 2500 50  0001 C CNN
@@
 	2000 3700 2100 3700
 $Comp
-L power:GND #PWR0172
+L power:GND #PWR0174
 U 1 1 5D2F8FAD
 P 5500 3850
-F 0 "#PWR0172" H 5500 3600 50  0001 C CNN
+F 0 "#PWR0174" H 5500 3600 50  0001 C CNN
 F 1 "GND" H 5500 3700 50  0000 C CNN
 F 2 "" H 5500 3850 50  0001 C CNN
@@
 	5100 3800 5500 3800
 $Comp
-L custom:CRG0603F4K7 R88
+L custom:CRG0603F4K7 R96
 U 1 1 5D34D3B4
 P 1375 2250
-F 0 "R88" H 1445 2270 50  0000 L BNN
+F 0 "R96" H 1445 2270 50  0000 L BNN
 F 1 "CRG0603F4K7" H 675 1850 50  0001 L BNN
 F 2 "Resistor_SMD:R_0603_1608Metric" H 675 1750 50  0001 L BNN
@@
 $EndComp
 $Comp
-L custom:CRG0603F4K7 R86
+L custom:CRG0603F4K7 R94
 U 1 1 5D34D8B8
 P 1725 1300
-F 0 "R86" H 1795 1320 50  0000 L BNN
+F 0 "R94" H 1795 1320 50  0000 L BNN
 F 1 "CRG0603F4K7" H 1025 900 50  0001 L BNN
 F 2 "Resistor_SMD:R_0603_1608Metric" H 1025 800 50  0001 L BNN
@@
 $EndComp
 $Comp
-L custom:CRG0603F4K7 R92
+L custom:CRG0603F4K7 R100
 U 1 1 5D34DD9B
 P 1225 3675
-F 0 "R92" H 1295 3695 50  0000 L BNN
+F 0 "R100" H 1295 3695 50  0000 L BNN
 F 1 "CRG0603F4K7" H 525 3275 50  0001 L BNN
 F 2 "Resistor_SMD:R_0603_1608Metric" H 525 3175 50  0001 L BNN
@@
 $EndComp
 $Comp
-L custom:CRG0603F4K7 R90
+L custom:CRG0603F4K7 R98
 U 1 1 5D34E19D
 P 1900 3325
-F 0 "R90" V 1875 3050 50  0000 L BNN
+F 0 "R98" V 1875 3050 50  0000 L BNN
 F 1 "CRG0603F4K7" H 1200 2925 50  0001 L BNN
 F 2 "Resistor_SMD:R_0603_1608Metric" H 1200 2825 50  0001 L BNN
@@
 	1225 3975 2400 3975
 $Comp
-L power:+12V #PWR0169
+L power:+12V #PWR0171
 U 1 1 5D3649D3
 P 5675 950
-F 0 "#PWR0169" H 5675 800 50  0001 C CNN
+F 0 "#PWR0171" H 5675 800 50  0001 C CNN
 F 1 "+12V" H 5675 1090 50  0000 C CNN
 F 2 "" H 5675 950 50  0001 C CNN
@@
 $EndComp
 $Comp
-L power:GND #PWR0171
+L power:GND #PWR0173
 U 1 1 5D3649D9
 P 5125 2500
-F 0 "#PWR0171" H 5125 2250 50  0001 C CNN
+F 0 "#PWR0173" H 5125 2250 50  0001 C CNN
 F 1 "GND" H 5125 2350 50  0000 C CNN
 F 2 "" H 5125 2500 50  0001 C CNN
@@
 ROW01_ON
 $Comp
-L custom:CRG0603F4K7 R89
+L custom:CRG0603F4K7 R97
 U 1 1 5D364A11
 P 4775 2250
-F 0 "R89" H 4845 2270 50  0000 L BNN
+F 0 "R97" H 4845 2270 50  0000 L BNN
 F 1 "CRG0603F4K7" H 4075 1850 50  0001 L BNN
 F 2 "Resistor_SMD:R_0603_1608Metric" H 4075 1750 50  0001 L BNN
@@
 $EndComp
 $Comp
-L custom:CRG0603F4K7 R87
+L custom:CRG0603F4K7 R95
 U 1 1 5D364A19
 P 5125 1300
-F 0 "R87" H 5195 1320 50  0000 L BNN
+F 0 "R95" H 5195 1320 50  0000 L BNN
 F 1 "CRG0603F4K7" H 4425 900 50  0001 L BNN
 F 2 "Resistor_SMD:R_0603_1608Metric" H 4425 800 50  0001 L BNN
@@
 $EndComp
 $Comp
-L custom:CRG0603F4K7 R91
+L custom:CRG0603F4K7 R99
 U 1 1 5D365F82
 P 5100 3550
-F 0 "R91" H 5170 3570 50  0000 L BNN
+F 0 "R99" H 5170 3570 50  0000 L BNN
 F 1 "CRG0603F4K7" H 4400 3150 50  0001 L BNN
 F 2 "Resistor_SMD:R_0603_1608Metric" H 4400 3050 50  0001 L BNN
@@
 ROW01P
 $Comp
-L power:GND #PWR0179
+L power:GND #PWR0181
 U 1 1 5D3CB903
 P 5400 7275
-F 0 "#PWR0179" H 5400 7025 50  0001 C CNN
+F 0 "#PWR0181" H 5400 7025 50  0001 C CNN
 F 1 "GND" H 5400 7125 50  0000 C CNN
 F 2 "" H 5400 7275 50  0001 C CNN
@@
 	5000 7225 5400 7225
 $Comp
-L power:+12V #PWR0175
+L power:+12V #PWR0177
 U 1 1 5D3CB92A
 P 5575 4625
-F 0 "#PWR0175" H 5575 4475 50  0001 C CNN
+F 0 "#PWR0177" H 5575 4475 50  0001 C CNN
 F 1 "+12V" H 5575 4765 50  0000 C CNN
 F 2 "" H 5575 4625 50  0001 C CNN
@@
 $EndComp
 $Comp
-L power:GND #PWR0177
+L power:GND #PWR0179
 U 1 1 5D3CB930
 P 5025 6175
-F 0 "#PWR0177" H 5025 5925 50  0001 C CNN
+F 0 "#PWR0179" H 5025 5925 50  0001 C CNN
 F 1 "GND" H 5025 6025 50  0000 C CNN
 F 2 "" H 5025 6175 50  0001 C CNN
@@
 Connection ~ 6075 5675
 $Comp
-L custom:CRG0603F4K7 R96
+L custom:CRG0603F4K7 R104
 U 1 1 5D3CB967
 P 4675 5925
-F 0 "R96" H 4745 5945 50  0000 L BNN
+F 0 "R104" H 4745 5945 50  0000 L BNN
 F 1 "CRG0603F4K7" H 3975 5525 50  0001 L BNN
 F 2 "Resistor_SMD:R_0603_1608Metric" H 3975 5425 50  0001 L BNN
@@
 $EndComp
 $Comp
-L custom:CRG0603F4K7 R94
+L custom:CRG0603F4K7 R102
 U 1 1 5D3CB96F
 P 5025 4975
-F 0 "R94" H 5095 4995 50  0000 L BNN
+F 0 "R102" H 5095 4995 50  0000 L BNN
 F 1 "CRG0603F4K7" H 4325 4575 50  0001 L BNN
 F 2 "Resistor_SMD:R_0603_1608Metric" H 4325 4475 50  0001 L BNN
@@
 $EndComp
 $Comp
-L custom:CRG0603F4K7 R98
+L custom:CRG0603F4K7 R106
 U 1 1 5D3CB977
 P 5000 6975
-F 0 "R98" H 5070 6995 50  0000 L BNN
+F 0 "R106" H 5070 6995 50  0000 L BNN
 F 1 "CRG0603F4K7" H 4300 6575 50  0001 L BNN
 F 2 "Resistor_SMD:R_0603_1608Metric" H 4300 6475 50  0001 L BNN
@@
 ROW03P
 $Comp
-L power:GND #PWR0178
+L power:GND #PWR0180
 U 1 1 5D3F720D
 P 2000 7275
-F 0 "#PWR0178" H 2000 7025 50  0001 C CNN
+F 0 "#PWR0180" H 2000 7025 50  0001 C CNN
 F 1 "GND" H 2000 7125 50  0000 C CNN
 F 2 "" H 2000 7275 50  0001 C CNN
@@
 	1600 7225 2000 7225
 $Comp
-L power:+12V #PWR0174
+L power:+12V #PWR0176
 U 1 1 5D3F7234
 P 2175 4625
-F 0 "#PWR0174" H 2175 4475 50  0001 C CNN
+F 0 "#PWR0176" H 2175 4475 50  0001 C CNN
 F 1 "+12V" H 2175 4765 50  0000 C CNN
 F 2 "" H 2175 4625 50  0001 C CNN
@@
 $EndComp
 $Comp
-L power:GND #PWR0176
+L power:GND #PWR0178
 U 1 1 5D3F723A
 P 1625 6175
-F 0 "#PWR0176" H 1625 5925 50  0001 C CNN
+F 0 "#PWR0178" H 1625 5925 50  0001 C CNN
 F 1 "GND" H 1625 6025 50  0000 C CNN
 F 2 "" H 1625 6175 50  0001 C CNN
@@
 ROW02_ON
 $Comp
-L custom:CRG0603F4K7 R95
+L custom:CRG0603F4K7 R103
 U 1 1 5D3F7271
 P 1275 5925
-F 0 "R95" H 1345 5945 50  0000 L BNN
+F 0 "R103" H 1345 5945 50  0000 L BNN
 F 1 "CRG0603F4K7" H 575 5525 50  0001 L BNN
 F 2 "Resistor_SMD:R_0603_1608Metric" H 575 5425 50  0001 L BNN
@@
 $EndComp
 $Comp
-L custom:CRG0603F4K7 R93
+L custom:CRG0603F4K7 R101
 U 1 1 5D3F7279
 P 1625 4975
-F 0 "R93" H 1695 4995 50  0000 L BNN
+F 0 "R101" H 1695 4995 50  0000 L BNN
 F 1 "CRG0603F4K7" H 925 4575 50  0001 L BNN
 F 2 "Resistor_SMD:R_0603_1608Metric" H 925 4475 50  0001 L BNN
@@
 $EndComp
 $Comp
-L custom:CRG0603F4K7 R97
+L custom:CRG0603F4K7 R105
 U 1 1 5D3F7281
 P 1600 6975
-F 0 "R97" H 1670 6995 50  0000 L BNN
+F 0 "R105" H 1670 6995 50  0000 L BNN
 F 1 "CRG0603F4K7" H 900 6575 50  0001 L BNN
 F 2 "Resistor_SMD:R_0603_1608Metric" H 900 6475 50  0001 L BNN

Commit message: automated commit
Parts:
- removed Q20: SSM3K35AMFV, Package_TO_SOT_SMD:SOT-723, symbol custom:SSM3K35AMFV
- removed R100: CRG0603F4K7, Resistor_SMD:R_0603_1608Metric, symbol custom:CRG0603F4K7
- removed TP73, TP75, TP77: TestPoint, custom:TestPoint_THTPad_D1.0mm_Drill0.5mm, symbol Connector:TestPoint
- added TP72, TP76: TestPoint, custom:TestPoint_THTPad_D1.0mm_Drill0.5mm, symbol Connector:TestPoint
- renumbered Q21 to Q20, Q22 to Q21, Q23 to Q22, Q24 to Q23, R101 to R100, R102 to R101, R103 to R102, R104 to R103, R105 to R104, R106 to R105, TP72 to TP73, TP76 to TP75, TP78 to TP77
Connections:
- net GND: now also R98.2, TP76.1
- net ROW00N: now also TP72.1
- net ROW00_OFF: now also Q16.1 (G), R98.1; no longer R98.2

Commit message: automated commit
Parts:
- removed TP65, TP67, TP69, TP71, TP73, TP75, TP76, TP77: TestPoint, custom:TestPoint_THTPad_D1.0mm_Drill0.5mm, symbol Connector:TestPoint
Changed lines of the file:
@@
 	5100 3800 5100 3700
-Wire Wire Line
-	4775 3325 4925 3325
 Wire Wire Line
 	5100 3400 5100 3325
@@
 Wire Wire Line
 	5975 3225 5975 3025
-Wire Wire Line
-	5975 3025 5750 3025
 Connection ~ 5975 3025
 Wire Wire Line
@@
 Connection ~ 5675 1050
 Wire Wire Line
-	5125 1450 5125 1550
-Wire Wire Line
 	5125 1650 5375 1650
 Connection ~ 5125 1650
 Wire Wire Line
-	5125 2200 5125 2350
-Wire Wire Line
 	4775 2450 5125 2450
 Wire Wire Line
@@
 	4775 2100 4775 2000
 Connection ~ 5125 2450
-Wire Wire Line
-	4500 2000 4625 2000
 Connection ~ 4775 2000
 Wire Wire Line
@@
 	1075 2000 1225 2000
 $Comp
-L Connector:TestPoint TP?
-U 1 1 5D9363B5
-P 5050 1550
-AR Path="/5D9363B5" Ref="TP?"  Part="1"
-AR Path="/61C6D021/5D9363B5" Ref="TP?"  Part="1"
-AR Path="/609E0ED6/5D9363B5" Ref="TP?"  Part="1"
-AR Path="/621F0CB4/5D9363B5" Ref="TP?"  Part="1"
-AR Path="/62CDD30D/5D9363B5" Ref="TP65"  Part="1"
-F 0 "TP65" V 4950 1725 50  0000 C CNN
-F 1 "TestPoint" H 4800 1600 50  0001 C CNN
-F 2 "custom:TestPoint_THTPad_D1.0mm_Drill0.5mm" H 5250 1550 50  0001 C CNN
-F 3 "~" H 5250 1550 50  0001 C CNN
-	1    5050 1550
-	0    -1   1    0
-$EndComp
-Wire Wire Line
-	5050 1550 5125 1550
-$Comp
-L Connector:TestPoint TP?
-U 1 1 5D9363BC
-P 4625 1925
-AR Path="/5D9363BC" Ref="TP?"  Part="1"
-AR Path="/61C6D021/5D9363BC" Ref="TP?"  Part="1"
-AR Path="/609E0ED6/5D9363BC" Ref="TP?"  Part="1"
-AR Path="/621F0CB4/5D9363BC" Ref="TP?"  Part="1"
-AR Path="/62CDD30D/5D9363BC" Ref="TP67"  Part="1"
-F 0 "TP67" H 4625 2150 50  0000 C CNN
-F 1 "TestPoint" H 4375 1975 50  0001 C CNN
-F 2 "custom:TestPoint_THTPad_D1.0mm_Drill0.5mm" H 4825 1925 50  0001 C CNN
-F 3 "~" H 4825 1925 50  0001 C CNN
-	1    4625 1925
-	-1   0    0    -1
-$EndComp
-Wire Wire Line
-	4625 1925 4625 2000
-Connection ~ 5125 1550
-Wire Wire Line
-	5125 1550 5125 1650
-Connection ~ 4625 2000
-Wire Wire Line
-	4625 2000 4775 2000
-$Comp
-L Connector:TestPoint TP?
-U 1 1 5D94EF08
-P 5250 2350
-AR Path="/5D94EF08" Ref="TP?"  Part="1"
-AR Path="/61C6D021/5D94EF08" Ref="TP?"  Part="1"
-AR Path="/609E0ED6/5D94EF08" Ref="TP?"  Part="1"
-AR Path="/621F0CB4/5D94EF08" Ref="TP?"  Part="1"
-AR Path="/62CDD30D/5D94EF08" Ref="TP71"  Part="1"
-F 0 "TP71" V 5350 2500 50  0000 C CNN
-F 1 "TestPoint" H 5000 2400 50  0001 C CNN
-F 2 "custom:TestPoint_THTPad_D1.0mm_Drill0.5mm" H 5450 2350 50  0001 C CNN
-F 3 "~" H 5450 2350 50  0001 C CNN
-	1    5250 2350
-	0    1    1    0
-$EndComp
-Wire Wire Line
-	5250 2350 5125 2350
-$Comp
-L Connector:TestPoint TP?
-U 1 1 5D94EF0F
-P 5675 2050
-AR Path="/5D94EF0F" Ref="TP?"  Part="1"
-AR Path="/61C6D021/5D94EF0F" Ref="TP?"  Part="1"
-AR Path="/609E0ED6/5D94EF0F" Ref="TP?"  Part="1"
-AR Path="/621F0CB4/5D94EF0F" Ref="TP?"  Part="1"
-AR Path="/62CDD30D/5D94EF0F" Ref="TP69"  Part="1"
-F 0 "TP69" H 5550 2200 50  0000 C CNN
-F 1 "TestPoint" H 5425 2100 50  0001 C CNN
-F 2 "custom:TestPoint_THTPad_D1.0mm_Drill0.5mm" H 5875 2050 50  0001 C CNN
-F 3 "~" H 5875 2050 50  0001 C CNN
-	1    5675 2050
-	-1   0    0    1
-$EndComp
-Wire Wire Line
-	5675 2050 5675 2000
-Connection ~ 5675 2000
-Connection ~ 5125 2350
-Wire Wire Line
-	5125 2350 5125 2450
-$Comp
-L Connector:TestPoint TP?
-U 1 1 5D95F68E
-P 4925 3250
-AR Path="/5D95F68E" Ref="TP?"  Part="1"
-AR Path="/61C6D021/5D95F68E" Ref="TP?"  Part="1"
-AR Path="/609E0ED6/5D95F68E" Ref="TP?"  Part="1"
-AR Path="/621F0CB4/5D95F68E" Ref="TP?"  Part="1"
-AR Path="/62CDD30D/5D95F68E" Ref="TP75"  Part="1"
-F 0 "TP75" H 4925 3475 50  0000 C CNN
-F 1 "TestPoint" H 4675 3300 50  0001 C CNN
-F 2 "custom:TestPoint_THTPad_D1.0mm_Drill0.5mm" H 5125 3250 50  0001 C CNN
-F 3 "~" H 5125 3250 50  0001 C CNN
-	1    4925 3250
-	-1   0    0    -1
-$EndComp
-Wire Wire Line
-	4925 3250 4925 3325
-Connection ~ 4925 3325
-Wire Wire Line
-	4925 3325 5100 3325
-$Comp
-L Connector:TestPoint TP?
-U 1 1 5D96862D
-P 5975 3750
-AR Path="/5D96862D" Ref="TP?"  Part="1"
-AR Path="/61C6D021/5D96862D" Ref="TP?"  Part="1"
-AR Path="/609E0ED6/5D96862D" Ref="TP?"  Part="1"
-AR Path="/621F0CB4/5D96862D" Ref="TP?"  Part="1"
-AR Path="/62CDD30D/5D96862D" Ref="TP77"  Part="1"
-F 0 "TP77" H 5975 3975 50  0000 C CNN
-F 1 "TestPoint" H 5725 3800 50  0001 C CNN
-F 2 "custom:TestPoint_THTPad_D1.0mm_Drill0.5mm" H 6175 3750 50  0001 C CNN
-F 3 "~" H 6175 3750 50  0001 C CNN
-	1    5975 3750
-	1    0    0    1
-$EndComp
-Wire Wire Line
-	5975 3750 5975 3675
-Connection ~ 5975 3675
-$Comp
-L Connector:TestPoint TP?
-U 1 1 5D971623
-P 5750 2950
-AR Path="/5D971623" Ref="TP?"  Part="1"
-AR Path="/61C6D021/5D971623" Ref="TP?"  Part="1"
-AR Path="/609E0ED6/5D971623" Ref="TP?"  Part="1"
-AR Path="/621F0CB4/5D971623" Ref="TP?"  Part="1"
-AR Path="/62CDD30D/5D971623" Ref="TP73"  Part="1"
-F 0 "TP73" H 5750 3175 50  0000 C CNN
-F 1 "TestPoint" H 5500 3000 50  0001 C CNN
-F 2 "custom:TestPoint_THTPad_D1.0mm_Drill0.5mm" H 5950 2950 50  0001 C CNN
-F 3 "~" H 5950 2950 50  0001 C CNN
-	1    5750 2950
-	-1   0    0    -1
-$EndComp
-Wire Wire Line
-	5750 2950 5750 3025
-Connection ~ 5750 3025
-Wire Wire Line
-	5750 3025 5500 3025
-$Comp
 L power:GND #PWR0174
 U 1 1 5D17FE95
@@
 $Comp
 L Connector:TestPoint TP?
-U 1 1 5D17FECD
-P 2575 3750
-AR Path="/5D17FECD" Ref="TP?"  Part="1"
-AR Path="/61C6D021/5D17FECD" Ref="TP?"  Part="1"
-AR Path="/609E0ED6/5D17FECD" Ref="TP?"  Part="1"
-AR Path="/621F0CB4/5D17FECD" Ref="TP?"  Part="1"
-AR Path="/62CDD30D/5D17FECD" Ref="TP76"  Part="1"
-F 0 "TP76" H 2575 3975 50  0000 C CNN
-F 1 "TestPoint" H 2325 3800 50  0001 C CNN
-F 2 "custom:TestPoint_THTPad_D1.0mm_Drill0.5mm" H 2775 3750 50  0001 C CNN
-F 3 "~" H 2775 3750 50  0001 C CNN
-	1    2575 3750
-	1    0    0    1
-$EndComp
-Wire Wire Line
-	2575 3750 2575 3675
-Connection ~ 2575 3675
-$Comp
-L Connector:TestPoint TP?
 U 1 1 5D17FED5
 P 2350 2950
@@
 Wire Wire Line
 	2350 3025 2100 3025
+Wire Wire Line
+	4775 3325 5100 3325
+Wire Wire Line
+	5500 3025 5975 3025
+Wire Wire Line
+	4500 2000 4775 2000
+Wire Wire Line
+	5125 1450 5125 1650
+Wire Wire Line
+	5125 2200 5125 2450
 $EndSCHEMATC
