File: ROW_DRIVERS_1.sch (KiCad schematic (older format))
At the start: 36 parts, among them Q108 DMG6602, Q109 DMG6602, Q110 SSM3K35AMFV, Q111 SSM3K35AMFV, Q112 SSM3K35AMFV, Q113 SSM3K35AMFV, Q114 DMG6602, Q115 DMG6602, Q116 SSM3K35AMFV, Q117 SSM3K35AMFV, Q118 SSM3K35AMFV, Q119 SSM3K35AMFV

Commit message: automated commit
Parts:
- removed D34, D35: MMBZ5243BLT1G, symbol custom:MMBZ5243BLT1G
- removed Q108, Q109, Q114, Q115: DMG6602, Package_TO_SOT_SMD:TSOT-23-6, symbol custom:DMG6602
- removed Q110, Q111, Q112, Q113, Q116, Q117, Q118, Q119: SSM3K35AMFV, symbol custom:SSM3K35AMFV
- removed R194, R195, R196, R197, R198, R199, R200, R201, R202, R203, R204, R205, R206, R207, R208, R209: CRG0603F4K7, Resistor_SMD:R_0603_1608Metric, symbol custom:CRG0603F4K7
- added D26, D27: MMBZ5243BLT1G, symbol custom:MMBZ5243BLT1G
- added Q25, Q26, Q29, Q30: DMG6602, Package_TO_SOT_SMD:TSOT-23-6, symbol custom:DMG6602
- added Q27, Q28, Q31, Q32: SSM3K35AMFV, symbol custom:SSM3K35AMFV
- added R103, R104, R105, R106, R107, R108, R109, R110, R111, R112, R113, R114: CRG0603F4K7, Resistor_SMD:R_0603_1608Metric, symbol custom:CRG0603F4K7
Connections:
- net +12V: now also D30.1 (K), D31.1 (K), D26.1 (K), D27.1 (K), Q25.2 (S), Q26.2 (S), Q29.2 (S), Q30.2 (S), R103.1, R104.1, R109.1, R110.1; no longer D28.1 (K), D29.1 (K), D32.1 (K), D33.1 (K)
- net GND: now also D28.2 (A), D29.2 (A), D32.2 (A), D33.2 (A), Q25.5 (S), Q26.5 (S), Q27.2 (S), Q28.2 (S), Q29.5 (S), Q30.5 (S), Q31.2 (S), Q32.2 (S), R105.2, R106.2, R107.2, R108.2, R111.2, R112.2, R113.2, R114.2; no longer D30.2 (A), D31.2 (A)
- net ROW04N: now also D28.1 (K), Q25.6 (D); no longer D30.1 (K)
- net ROW04P: now also D26.2 (A), Q25.4 (D); no longer D28.2 (A)
- net ROW04_OFF: now also Q25.1 (G), R107.1
- net ROW04_ON: now also Q27.1 (G), R105.1
- net ROW05N: now also D29.1 (K), Q26.6 (D); no longer D31.1 (K)
- net ROW05P: now also D27.2 (A), Q26.4 (D); no longer D29.2 (A)
- net ROW05_OFF: now also Q26.1 (G), R108.1
- net ROW05_ON: now also Q28.1 (G), R106.1
- net ROW06N: now also D32.1 (K), Q29.6 (D)
- net ROW06P: now also D30.2 (A), Q29.4 (D); no longer D32.2 (A)
- net ROW06_OFF: now also Q29.1 (G), R113.1
- net ROW06_ON: now also Q31.1 (G), R111.1
- net ROW07N: now also D33.1 (K), Q30.6 (D)
- net ROW07P: now also D31.2 (A), Q30.4 (D); no longer D33.2 (A)
- net ROW07_OFF: now also Q30.1 (G), R114.1
- net ROW07_ON: now also Q32.1 (G), R112.1
- new net: Q26.3 (G), Q28.3 (D), R104.2
- new net: Q30.3 (G), Q32.3 (D), R110.2
- new net: Q29.3 (G), Q31.3 (D), R109.2
- new net: Q25.3 (G), Q27.3 (D), R103.2

Commit message: automated commit
Parts:
- renumbered R104 to R100, R105 to R101, R106 to R102, R107 to R103, R108 to R104, R109 to R105, R110 to R106, R111 to R107, R112 to R108, R113 to R109, R114 to R110, R103 to R99

Commit message: automated commit
Parts:
- D26, D27, D28, D29, D30, D31, D32, D33: footprint (none) -> Package_TO_SOT_SMD:SOT-23
- Q27, Q28, Q31, Q32: footprint (none) -> Package_TO_SOT_SMD:SOT-723
Changed lines of the file:
@@
 F 0 "Q28" V 5250 1925 50  0000 L BNN
 F 1 "SSM3K35AMFV" V 5175 1750 50  0000 L BNN
-F 2 "" H 5125 1875 50  0001 L BIN
+F 2 "Package_TO_SOT_SMD:SOT-723" H 5125 1875 50  0001 L BIN
 F 3 "datasheets/SSM3K35AMFV.pdf" H 5125 1850 50  0001 L BNN
 	1    4925 2000
@@
 F 0 "Q32" V 5250 5300 50  0000 L BNN
 F 1 "SSM3K35AMFV" V 5175 5125 50  0000 L BNN
-F 2 "" H 5125 5250 50  0001 L BIN
+F 2 "Package_TO_SOT_SMD:SOT-723" H 5125 5250 50  0001 L BIN
 F 3 "datasheets/SSM3K35AMFV.pdf" H 5125 5225 50  0001 L BNN
 	1    4925 5375
@@
 F 0 "Q31" V 1850 5300 50  0000 L BNN
 F 1 "SSM3K35AMFV" V 1775 5125 50  0000 L BNN
-F 2 "" H 1725 5250 50  0001 L BIN
+F 2 "Package_TO_SOT_SMD:SOT-723" H 1725 5250 50  0001 L BIN
 F 3 "datasheets/SSM3K35AMFV.pdf" H 1725 5225 50  0001 L BNN
 	1    1525 5375
@@
 F 0 "Q27" V 1850 1925 50  0000 L BNN
 F 1 "SSM3K35AMFV" V 1775 1750 50  0000 L BNN
-F 2 "" H 1725 1875 50  0001 L BIN
+F 2 "Package_TO_SOT_SMD:SOT-723" H 1725 1875 50  0001 L BIN
 F 3 "datasheets/SSM3K35AMFV.pdf" H 1725 1850 50  0001 L BNN
 	1    1525 2000
@@
 F 0 "D26" H 2800 1575 50  0000 C CNN
 F 1 "MMBZ5243BLT1G" H 2675 1725 50  0000 C CNN
-F 2 "" V 2675 1625 50  0001 C CNN
+F 2 "Package_TO_SOT_SMD:SOT-23" V 2675 1625 50  0001 C CNN
 F 3 "" H 2675 1715 50  0001 C CNN
 F 4 "13V" H 2550 1575 39  0000 C CNN "Rating"
@@
 F 0 "D29" H 6000 3025 50  0000 C CNN
 F 1 "MMBZ5243BLT1G" H 5975 3175 50  0000 C CNN
-F 2 "" V 5875 3075 50  0001 C CNN
+F 2 "Package_TO_SOT_SMD:SOT-23" V 5875 3075 50  0001 C CNN
 F 3 "" H 5875 3165 50  0001 C CNN
 F 4 "13V" H 5750 3025 39  0000 C CNN "Rating"
@@
 F 0 "D27" H 6200 1575 50  0000 C CNN
 F 1 "MMBZ5243BLT1G" H 6075 1725 50  0000 C CNN
-F 2 "" V 6075 1625 50  0001 C CNN
+F 2 "Package_TO_SOT_SMD:SOT-23" V 6075 1625 50  0001 C CNN
 F 3 "" H 6075 1715 50  0001 C CNN
 F 4 "13V" H 5950 1575 39  0000 C CNN "Rating"
@@
 F 0 "D28" H 2600 3025 50  0000 C CNN
 F 1 "MMBZ5243BLT1G" H 2575 3175 50  0000 C CNN
-F 2 "" V 2475 3075 50  0001 C CNN
+F 2 "Package_TO_SOT_SMD:SOT-23" V 2475 3075 50  0001 C CNN
 F 3 "" H 2475 3165 50  0001 C CNN
 F 4 "13V" H 2350 3025 39  0000 C CNN "Rating"
@@
 F 0 "D32" H 2600 6400 50  0000 C CNN
 F 1 "MMBZ5243BLT1G" H 2575 6550 50  0000 C CNN
-F 2 "" V 2475 6450 50  0001 C CNN
+F 2 "Package_TO_SOT_SMD:SOT-23" V 2475 6450 50  0001 C CNN
 F 3 "" H 2475 6540 50  0001 C CNN
 F 4 "13V" H 2350 6400 39  0000 C CNN "Rating"
@@
 F 0 "D30" H 2800 4950 50  0000 C CNN
 F 1 "MMBZ5243BLT1G" H 2675 5100 50  0000 C CNN
-F 2 "" V 2675 5000 50  0001 C CNN
+F 2 "Package_TO_SOT_SMD:SOT-23" V 2675 5000 50  0001 C CNN
 F 3 "" H 2675 5090 50  0001 C CNN
 F 4 "13V" H 2550 4950 39  0000 C CNN "Rating"
@@
 F 0 "D33" H 6000 6400 50  0000 C CNN
 F 1 "MMBZ5243BLT1G" H 5975 6550 50  0000 C CNN
-F 2 "" V 5875 6450 50  0001 C CNN
+F 2 "Package_TO_SOT_SMD:SOT-23" V 5875 6450 50  0001 C CNN
 F 3 "" H 5875 6540 50  0001 C CNN
 F 4 "13V" H 5750 6400 39  0000 C CNN "Rating"
@@
 F 0 "D31" H 6200 4950 50  0000 C CNN
 F 1 "MMBZ5243BLT1G" H 6075 5100 50  0000 C CNN
-F 2 "" V 6075 5000 50  0001 C CNN
+F 2 "Package_TO_SOT_SMD:SOT-23" V 6075 5000 50  0001 C CNN
 F 3 "" H 6075 5090 50  0001 C CNN
 F 4 "13V" H 5950 4950 39  0000 C CNN "Rating"

Commit message: automated commit
Parts:
- renumbered R99 to R107, R100 to R108, R101 to R109, R102 to R110, R103 to R111, R104 to R112, R105 to R113, R106 to R114, R107 to R115, R108 to R116, R109 to R117, R110 to R118
Changed lines of the file:
@@
 P 5400 3600
 AR Path="/62CDD30D/5D477EE1" Ref="#PWR?"  Part="1"
-AR Path="/62D7188C/5D477EE1" Ref="#PWR0185"  Part="1"
-F 0 "#PWR0185" H 5400 3350 50  0001 C CNN
+AR Path="/62D7188C/5D477EE1" Ref="#PWR0187"  Part="1"
+F 0 "#PWR0187" H 5400 3350 50  0001 C CNN
 F 1 "GND" H 5400 3450 50  0000 C CNN
 F 2 "" H 5400 3600 50  0001 C CNN
@@
 P 5575 950
 AR Path="/62CDD30D/5D477F2D" Ref="#PWR?"  Part="1"
-AR Path="/62D7188C/5D477F2D" Ref="#PWR0181"  Part="1"
-F 0 "#PWR0181" H 5575 800 50  0001 C CNN
+AR Path="/62D7188C/5D477F2D" Ref="#PWR0183"  Part="1"
+F 0 "#PWR0183" H 5575 800 50  0001 C CNN
 F 1 "+12V" H 5575 1090 50  0000 C CNN
 F 2 "" H 5575 950 50  0001 C CNN
@@
 P 5025 2500
 AR Path="/62CDD30D/5D477F33" Ref="#PWR?"  Part="1"
-AR Path="/62D7188C/5D477F33" Ref="#PWR0183"  Part="1"
-F 0 "#PWR0183" H 5025 2250 50  0001 C CNN
+AR Path="/62D7188C/5D477F33" Ref="#PWR0185"  Part="1"
+F 0 "#PWR0185" H 5025 2250 50  0001 C CNN
 F 1 "GND" H 5025 2350 50  0000 C CNN
 F 2 "" H 5025 2500 50  0001 C CNN
@@
 P 4675 2250
 AR Path="/62CDD30D/5D477F6A" Ref="R?"  Part="1"
-AR Path="/62D7188C/5D477F6A" Ref="R102"  Part="1"
-F 0 "R102" H 4745 2270 50  0000 L BNN
+AR Path="/62D7188C/5D477F6A" Ref="R110"  Part="1"
+F 0 "R110" H 4745 2270 50  0000 L BNN
 F 1 "CRG0603F4K7" H 3975 1850 50  0001 L BNN
 F 2 "Resistor_SMD:R_0603_1608Metric" H 3975 1750 50  0001 L BNN
@@
 P 5025 1300
 AR Path="/62CDD30D/5D477F72" Ref="R?"  Part="1"
-AR Path="/62D7188C/5D477F72" Ref="R100"  Part="1"
-F 0 "R100" H 5095 1320 50  0000 L BNN
+AR Path="/62D7188C/5D477F72" Ref="R108"  Part="1"
+F 0 "R108" H 5095 1320 50  0000 L BNN
 F 1 "CRG0603F4K7" H 4325 900 50  0001 L BNN
 F 2 "Resistor_SMD:R_0603_1608Metric" H 4325 800 50  0001 L BNN
@@
 P 5000 3300
 AR Path="/62CDD30D/5D477F7A" Ref="R?"  Part="1"
-AR Path="/62D7188C/5D477F7A" Ref="R104"  Part="1"
-F 0 "R104" H 5070 3320 50  0000 L BNN
+AR Path="/62D7188C/5D477F7A" Ref="R112"  Part="1"
+F 0 "R112" H 5070 3320 50  0000 L BNN
 F 1 "CRG0603F4K7" H 4300 2900 50  0001 L BNN
 F 2 "Resistor_SMD:R_0603_1608Metric" H 4300 2800 50  0001 L BNN
@@
 P 5400 6975
 AR Path="/62CDD30D/5D477F81" Ref="#PWR?"  Part="1"
-AR Path="/62D7188C/5D477F81" Ref="#PWR0191"  Part="1"
-F 0 "#PWR0191" H 5400 6725 50  0001 C CNN
+AR Path="/62D7188C/5D477F81" Ref="#PWR0193"  Part="1"
+F 0 "#PWR0193" H 5400 6725 50  0001 C CNN
 F 1 "GND" H 5400 6825 50  0000 C CNN
 F 2 "" H 5400 6975 50  0001 C CNN
@@
 P 5575 4325
 AR Path="/62CDD30D/5D477FA8" Ref="#PWR?"  Part="1"
-AR Path="/62D7188C/5D477FA8" Ref="#PWR0187"  Part="1"
-F 0 "#PWR0187" H 5575 4175 50  0001 C CNN
+AR Path="/62D7188C/5D477FA8" Ref="#PWR0189"  Part="1"
+F 0 "#PWR0189" H 5575 4175 50  0001 C CNN
 F 1 "+12V" H 5575 4465 50  0000 C CNN
 F 2 "" H 5575 4325 50  0001 C CNN
@@
 P 5025 5875
 AR Path="/62CDD30D/5D477FAE" Ref="#PWR?"  Part="1"
-AR Path="/62D7188C/5D477FAE" Ref="#PWR0189"  Part="1"
-F 0 "#PWR0189" H 5025 5625 50  0001 C CNN
+AR Path="/62D7188C/5D477FAE" Ref="#PWR0191"  Part="1"
+F 0 "#PWR0191" H 5025 5625 50  0001 C CNN
 F 1 "GND" H 5025 5725 50  0000 C CNN
 F 2 "" H 5025 5875 50  0001 C CNN
@@
 P 4675 5625
 AR Path="/62CDD30D/5D477FE4" Ref="R?"  Part="1"
-AR Path="/62D7188C/5D477FE4" Ref="R108"  Part="1"
-F 0 "R108" H 4745 5645 50  0000 L BNN
+AR Path="/62D7188C/5D477FE4" Ref="R116"  Part="1"
+F 0 "R116" H 4745 5645 50  0000 L BNN
 F 1 "CRG0603F4K7" H 3975 5225 50  0001 L BNN
 F 2 "Resistor_SMD:R_0603_1608Metric" H 3975 5125 50  0001 L BNN
@@
 P 5025 4675
 AR Path="/62CDD30D/5D477FEC" Ref="R?"  Part="1"
-AR Path="/62D7188C/5D477FEC" Ref="R106"  Part="1"
-F 0 "R106" H 5095 4695 50  0000 L BNN
+AR Path="/62D7188C/5D477FEC" Ref="R114"  Part="1"
+F 0 "R114" H 5095 4695 50  0000 L BNN
 F 1 "CRG0603F4K7" H 4325 4275 50  0001 L BNN
 F 2 "Resistor_SMD:R_0603_1608Metric" H 4325 4175 50  0001 L BNN
@@
 P 5000 6675
 AR Path="/62CDD30D/5D477FF4" Ref="R?"  Part="1"
-AR Path="/62D7188C/5D477FF4" Ref="R110"  Part="1"
-F 0 "R110" H 5070 6695 50  0000 L BNN
+AR Path="/62D7188C/5D477FF4" Ref="R118"  Part="1"
+F 0 "R118" H 5070 6695 50  0000 L BNN
 F 1 "CRG0603F4K7" H 4300 6275 50  0001 L BNN
 F 2 "Resistor_SMD:R_0603_1608Metric" H 4300 6175 50  0001 L BNN
@@
 P 2000 6975
 AR Path="/62CDD30D/5D477FFB" Ref="#PWR?"  Part="1"
-AR Path="/62D7188C/5D477FFB" Ref="#PWR0190"  Part="1"
-F 0 "#PWR0190" H 2000 6725 50  0001 C CNN
+AR Path="/62D7188C/5D477FFB" Ref="#PWR0192"  Part="1"
+F 0 "#PWR0192" H 2000 6725 50  0001 C CNN
 F 1 "GND" H 2000 6825 50  0000 C CNN
 F 2 "" H 2000 6975 50  0001 C CNN
@@
 P 2175 4325
 AR Path="/62CDD30D/5D478022" Ref="#PWR?"  Part="1"
-AR Path="/62D7188C/5D478022" Ref="#PWR0186"  Part="1"
-F 0 "#PWR0186" H 2175 4175 50  0001 C CNN
+AR Path="/62D7188C/5D478022" Ref="#PWR0188"  Part="1"
+F 0 "#PWR0188" H 2175 4175 50  0001 C CNN
 F 1 "+12V" H 2175 4465 50  0000 C CNN
 F 2 "" H 2175 4325 50  0001 C CNN
@@
 P 1625 5875
 AR Path="/62CDD30D/5D478028" Ref="#PWR?"  Part="1"
-AR Path="/62D7188C/5D478028" Ref="#PWR0188"  Part="1"
-F 0 "#PWR0188" H 1625 5625 50  0001 C CNN
+AR Path="/62D7188C/5D478028" Ref="#PWR0190"  Part="1"
+F 0 "#PWR0190" H 1625 5625 50  0001 C CNN
 F 1 "GND" H 1625 5725 50  0000 C CNN
 F 2 "" H 1625 5875 50  0001 C CNN
@@
 P 1275 5625
 AR Path="/62CDD30D/5D47805F" Ref="R?"  Part="1"
-AR Path="/62D7188C/5D47805F" Ref="R107"  Part="1"
-F 0 "R107" H 1345 5645 50  0000 L BNN
+AR Path="/62D7188C/5D47805F" Ref="R115"  Part="1"
+F 0 "R115" H 1345 5645 50  0000 L BNN
 F 1 "CRG0603F4K7" H 575 5225 50  0001 L BNN
 F 2 "Resistor_SMD:R_0603_1608Metric" H 575 5125 50  0001 L BNN
@@
 P 1625 4675
 AR Path="/62CDD30D/5D478067" Ref="R?"  Part="1"
-AR Path="/62D7188C/5D478067" Ref="R105"  Part="1"
-F 0 "R105" H 1695 4695 50  0000 L BNN
+AR Path="/62D7188C/5D478067" Ref="R113"  Part="1"
+F 0 "R113" H 1695 4695 50  0000 L BNN
 F 1 "CRG0603F4K7" H 925 4275 50  0001 L BNN
 F 2 "Resistor_SMD:R_0603_1608Metric" H 925 4175 50  0001 L BNN
@@
 P 1600 6675
 AR Path="/62CDD30D/5D47806F" Ref="R?"  Part="1"
-AR Path="/62D7188C/5D47806F" Ref="R109"  Part="1"
-F 0 "R109" H 1670 6695 50  0000 L BNN
+AR Path="/62D7188C/5D47806F" Ref="R117"  Part="1"
+F 0 "R117" H 1670 6695 50  0000 L BNN
 F 1 "CRG0603F4K7" H 900 6275 50  0001 L BNN
 F 2 "Resistor_SMD:R_0603_1608Metric" H 900 6175 50  0001 L BNN
@@
 P 2000 3600
 AR Path="/62CDD30D/5D493974" Ref="#PWR?"  Part="1"
-AR Path="/62D7188C/5D493974" Ref="#PWR0184"  Part="1"
-F 0 "#PWR0184" H 2000 3350 50  0001 C CNN
+AR Path="/62D7188C/5D493974" Ref="#PWR0186"  Part="1"
+F 0 "#PWR0186" H 2000 3350 50  0001 C CNN
 F 1 "GND" H 2000 3450 50  0000 C CNN
 F 2 "" H 2000 3600 50  0001 C CNN
@@
 P 2175 950
 AR Path="/62CDD30D/5D49399B" Ref="#PWR?"  Part="1"
-AR Path="/62D7188C/5D49399B" Ref="#PWR0180"  Part="1"
-F 0 "#PWR0180" H 2175 800 50  0001 C CNN
+AR Path="/62D7188C/5D49399B" Ref="#PWR0182"  Part="1"
+F 0 "#PWR0182" H 2175 800 50  0001 C CNN
 F 1 "+12V" H 2175 1090 50  0000 C CNN
 F 2 "" H 2175 950 50  0001 C CNN
@@
 P 1625 2500
 AR Path="/62CDD30D/5D4939A1" Ref="#PWR?"  Part="1"
-AR Path="/62D7188C/5D4939A1" Ref="#PWR0182"  Part="1"
-F 0 "#PWR0182" H 1625 2250 50  0001 C CNN
+AR Path="/62D7188C/5D4939A1" Ref="#PWR0184"  Part="1"
+F 0 "#PWR0184" H 1625 2250 50  0001 C CNN
 F 1 "GND" H 1625 2350 50  0000 C CNN
 F 2 "" H 1625 2500 50  0001 C CNN
@@
 P 1275 2250
 AR Path="/62CDD30D/5D4939D8" Ref="R?"  Part="1"
-AR Path="/62D7188C/5D4939D8" Ref="R101"  Part="1"
-F 0 "R101" H 1345 2270 50  0000 L BNN
+AR Path="/62D7188C/5D4939D8" Ref="R109"  Part="1"
+F 0 "R109" H 1345 2270 50  0000 L BNN
 F 1 "CRG0603F4K7" H 575 1850 50  0001 L BNN
 F 2 "Resistor_SMD:R_0603_1608Metric" H 575 1750 50  0001 L BNN
@@
 P 1625 1300
 AR Path="/62CDD30D/5D4939E0" Ref="R?"  Part="1"
-AR Path="/62D7188C/5D4939E0" Ref="R99"  Part="1"
-F 0 "R99" H 1695 1320 50  0000 L BNN
+AR Path="/62D7188C/5D4939E0" Ref="R107"  Part="1"
+F 0 "R107" H 1695 1320 50  0000 L BNN
 F 1 "CRG0603F4K7" H 925 900 50  0001 L BNN
 F 2 "Resistor_SMD:R_0603_1608Metric" H 925 800 50  0001 L BNN
@@
 P 1600 3300
 AR Path="/62CDD30D/5D4939E8" Ref="R?"  Part="1"
-AR Path="/62D7188C/5D4939E8" Ref="R103"  Part="1"
-F 0 "R103" H 1670 3320 50  0000 L BNN
+AR Path="/62D7188C/5D4939E8" Ref="R111"  Part="1"
+F 0 "R111" H 1670 3320 50  0000 L BNN
 F 1 "CRG0603F4K7" H 900 2900 50  0001 L BNN
 F 2 "Resistor_SMD:R_0603_1608Metric" H 900 2800 50  0001 L BNN

Commit message: automated commit
Parts:
- renumbered Q25 to Q24, Q26 to Q25, Q27 to Q26, Q28 to Q27, Q29 to Q28, Q30 to Q29, Q31 to Q30, Q32 to Q31, R107 to R106, R108 to R107, R109 to R108, R110 to R109, R111 to R110, R112 to R111, R113 to R112, R114 to R113, R115 to R114, R116 to R115, R117 to R116, R118 to R117
Changed lines of the file:
@@
 P 5300 3075
 AR Path="/62CDD30D/5D477EE7" Ref="Q?"  Part="1"
-AR Path="/62D7188C/5D477EE7" Ref="Q26"  Part="1"
-F 0 "Q26" V 5550 2975 50  0000 L CNN
+AR Path="/62D7188C/5D477EE7" Ref="Q25"  Part="1"
+F 0 "Q25" V 5550 2975 50  0000 L CNN
 F 1 "DMG6602" V 5650 2900 50  0000 L CNN
 F 2 "Package_TO_SOT_SMD:TSOT-23-6" H 5500 3000 50  0001 L CIN
@@
 P 5475 1650
 AR Path="/62CDD30D/5D477F39" Ref="Q?"  Part="2"
-AR Path="/62D7188C/5D477F39" Ref="Q26"  Part="2"
-F 0 "Q26" V 5725 1550 50  0000 L CNN
+AR Path="/62D7188C/5D477F39" Ref="Q25"  Part="2"
+F 0 "Q25" V 5725 1550 50  0000 L CNN
 F 1 "DMG6602" V 5825 1500 50  0000 L CNN
 F 2 "Package_TO_SOT_SMD:TSOT-23-6" H 5675 1575 50  0001 L CIN
@@
 P 4925 2000
 AR Path="/62CDD30D/5D477F59" Ref="Q?"  Part="1"
-AR Path="/62D7188C/5D477F59" Ref="Q28"  Part="1"
-F 0 "Q28" V 5250 1925 50  0000 L BNN
+AR Path="/62D7188C/5D477F59" Ref="Q27"  Part="1"
+F 0 "Q27" V 5250 1925 50  0000 L BNN
 F 1 "SSM3K35AMFV" V 5175 1750 50  0000 L BNN
 F 2 "Package_TO_SOT_SMD:SOT-723" H 5125 1875 50  0001 L BIN
@@
 P 4675 2250
 AR Path="/62CDD30D/5D477F6A" Ref="R?"  Part="1"
-AR Path="/62D7188C/5D477F6A" Ref="R110"  Part="1"
-F 0 "R110" H 4745 2270 50  0000 L BNN
+AR Path="/62D7188C/5D477F6A" Ref="R109"  Part="1"
+F 0 "R109" H 4745 2270 50  0000 L BNN
 F 1 "CRG0603F4K7" H 3975 1850 50  0001 L BNN
 F 2 "Resistor_SMD:R_0603_1608Metric" H 3975 1750 50  0001 L BNN
@@
 P 5025 1300
 AR Path="/62CDD30D/5D477F72" Ref="R?"  Part="1"
-AR Path="/62D7188C/5D477F72" Ref="R108"  Part="1"
-F 0 "R108" H 5095 1320 50  0000 L BNN
+AR Path="/62D7188C/5D477F72" Ref="R107"  Part="1"
+F 0 "R107" H 5095 1320 50  0000 L BNN
 F 1 "CRG0603F4K7" H 4325 900 50  0001 L BNN
 F 2 "Resistor_SMD:R_0603_1608Metric" H 4325 800 50  0001 L BNN
@@
 P 5000 3300
 AR Path="/62CDD30D/5D477F7A" Ref="R?"  Part="1"
-AR Path="/62D7188C/5D477F7A" Ref="R112"  Part="1"
-F 0 "R112" H 5070 3320 50  0000 L BNN
+AR Path="/62D7188C/5D477F7A" Ref="R111"  Part="1"
+F 0 "R111" H 5070 3320 50  0000 L BNN
 F 1 "CRG0603F4K7" H 4300 2900 50  0001 L BNN
 F 2 "Resistor_SMD:R_0603_1608Metric" H 4300 2800 50  0001 L BNN
@@
 P 5300 6450
 AR Path="/62CDD30D/5D477F87" Ref="Q?"  Part="1"
-AR Path="/62D7188C/5D477F87" Ref="Q30"  Part="1"
-F 0 "Q30" V 5550 6350 50  0000 L CNN
+AR Path="/62D7188C/5D477F87" Ref="Q29"  Part="1"
+F 0 "Q29" V 5550 6350 50  0000 L CNN
 F 1 "DMG6602" V 5650 6275 50  0000 L CNN
 F 2 "Package_TO_SOT_SMD:TSOT-23-6" H 5500 6375 50  0001 L CIN
@@
 P 5475 5025
 AR Path="/62CDD30D/5D477FB4" Ref="Q?"  Part="2"
-AR Path="/62D7188C/5D477FB4" Ref="Q30"  Part="2"
-F 0 "Q30" V 5725 4925 50  0000 L CNN
+AR Path="/62D7188C/5D477FB4" Ref="Q29"  Part="2"
+F 0 "Q29" V 5725 4925 50  0000 L CNN
 F 1 "DMG6602" V 5825 4875 50  0000 L CNN
 F 2 "Package_TO_SOT_SMD:TSOT-23-6" H 5675 4950 50  0001 L CIN
@@
 P 4925 5375
 AR Path="/62CDD30D/5D477FD4" Ref="Q?"  Part="1"
-AR Path="/62D7188C/5D477FD4" Ref="Q32"  Part="1"
-F 0 "Q32" V 5250 5300 50  0000 L BNN
+AR Path="/62D7188C/5D477FD4" Ref="Q31"  Part="1"
+F 0 "Q31" V 5250 5300 50  0000 L BNN
 F 1 "SSM3K35AMFV" V 5175 5125 50  0000 L BNN
 F 2 "Package_TO_SOT_SMD:SOT-723" H 5125 5250 50  0001 L BIN
@@
 P 4675 5625
 AR Path="/62CDD30D/5D477FE4" Ref="R?"  Part="1"
-AR Path="/62D7188C/5D477FE4" Ref="R116"  Part="1"
-F 0 "R116" H 4745 5645 50  0000 L BNN
+AR Path="/62D7188C/5D477FE4" Ref="R115"  Part="1"
+F 0 "R115" H 4745 5645 50  0000 L BNN
 F 1 "CRG0603F4K7" H 3975 5225 50  0001 L BNN
 F 2 "Resistor_SMD:R_0603_1608Metric" H 3975 5125 50  0001 L BNN
@@
 P 5025 4675
 AR Path="/62CDD30D/5D477FEC" Ref="R?"  Part="1"
-AR Path="/62D7188C/5D477FEC" Ref="R114"  Part="1"
-F 0 "R114" H 5095 4695 50  0000 L BNN
+AR Path="/62D7188C/5D477FEC" Ref="R113"  Part="1"
+F 0 "R113" H 5095 4695 50  0000 L BNN
 F 1 "CRG0603F4K7" H 4325 4275 50  0001 L BNN
 F 2 "Resistor_SMD:R_0603_1608Metric" H 4325 4175 50  0001 L BNN
@@
 P 5000 6675
 AR Path="/62CDD30D/5D477FF4" Ref="R?"  Part="1"
-AR Path="/62D7188C/5D477FF4" Ref="R118"  Part="1"
-F 0 "R118" H 5070 6695 50  0000 L BNN
+AR Path="/62D7188C/5D477FF4" Ref="R117"  Part="1"
+F 0 "R117" H 5070 6695 50  0000 L BNN
 F 1 "CRG0603F4K7" H 4300 6275 50  0001 L BNN
 F 2 "Resistor_SMD:R_0603_1608Metric" H 4300 6175 50  0001 L BNN
@@
 P 1900 6450
 AR Path="/62CDD30D/5D478001" Ref="Q?"  Part="1"
-AR Path="/62D7188C/5D478001" Ref="Q29"  Part="1"
-F 0 "Q29" V 2150 6350 50  0000 L CNN
+AR Path="/62D7188C/5D478001" Ref="Q28"  Part="1"
+F 0 "Q28" V 2150 6350 50  0000 L CNN
 F 1 "DMG6602" V 2250 6275 50  0000 L CNN
 F 2 "Package_TO_SOT_SMD:TSOT-23-6" H 2100 6375 50  0001 L CIN
@@
 P 2075 5025
 AR Path="/62CDD30D/5D47802E" Ref="Q?"  Part="2"
-AR Path="/62D7188C/5D47802E" Ref="Q29"  Part="2"
-F 0 "Q29" V 2325 4925 50  0000 L CNN
+AR Path="/62D7188C/5D47802E" Ref="Q28"  Part="2"
+F 0 "Q28" V 2325 4925 50  0000 L CNN
 F 1 "DMG6602" V 2425 4875 50  0000 L CNN
 F 2 "Package_TO_SOT_SMD:TSOT-23-6" H 2275 4950 50  0001 L CIN
@@
 P 1525 5375
 AR Path="/62CDD30D/5D47804E" Ref="Q?"  Part="1"
-AR Path="/62D7188C/5D47804E" Ref="Q31"  Part="1"
-F 0 "Q31" V 1850 5300 50  0000 L BNN
+AR Path="/62D7188C/5D47804E" Ref="Q30"  Part="1"
+F 0 "Q30" V 1850 5300 50  0000 L BNN
 F 1 "SSM3K35AMFV" V 1775 5125 50  0000 L BNN
 F 2 "Package_TO_SOT_SMD:SOT-723" H 1725 5250 50  0001 L BIN
@@
 P 1275 5625
 AR Path="/62CDD30D/5D47805F" Ref="R?"  Part="1"
-AR Path="/62D7188C/5D47805F" Ref="R115"  Part="1"
-F 0 "R115" H 1345 5645 50  0000 L BNN
+AR Path="/62D7188C/5D47805F" Ref="R114"  Part="1"
+F 0 "R114" H 1345 5645 50  0000 L BNN
 F 1 "CRG0603F4K7" H 575 5225 50  0001 L BNN
 F 2 "Resistor_SMD:R_0603_1608Metric" H 575 5125 50  0001 L BNN
@@
 P 1625 4675
 AR Path="/62CDD30D/5D478067" Ref="R?"  Part="1"
-AR Path="/62D7188C/5D478067" Ref="R113"  Part="1"
-F 0 "R113" H 1695 4695 50  0000 L BNN
+AR Path="/62D7188C/5D478067" Ref="R112"  Part="1"
+F 0 "R112" H 1695 4695 50  0000 L BNN
 F 1 "CRG0603F4K7" H 925 4275 50  0001 L BNN
 F 2 "Resistor_SMD:R_0603_1608Metric" H 925 4175 50  0001 L BNN
@@
 P 1600 6675
 AR Path="/62CDD30D/5D47806F" Ref="R?"  Part="1"
-AR Path="/62D7188C/5D47806F" Ref="R117"  Part="1"
-F 0 "R117" H 1670 6695 50  0000 L BNN
+AR Path="/62D7188C/5D47806F" Ref="R116"  Part="1"
+F 0 "R116" H 1670 6695 50  0000 L BNN
 F 1 "CRG0603F4K7" H 900 6275 50  0001 L BNN
 F 2 "Resistor_SMD:R_0603_1608Metric" H 900 6175 50  0001 L BNN
@@
 P 1900 3075
 AR Path="/62CDD30D/5D49397A" Ref="Q?"  Part="1"
-AR Path="/62D7188C/5D49397A" Ref="Q25"  Part="1"
-F 0 "Q25" V 2150 2975 50  0000 L CNN
+AR Path="/62D7188C/5D49397A" Ref="Q24"  Part="1"
+F 0 "Q24" V 2150 2975 50  0000 L CNN
 F 1 "DMG6602" V 2250 2900 50  0000 L CNN
 F 2 "Package_TO_SOT_SMD:TSOT-23-6" H 2100 3000 50  0001 L CIN
@@
 P 2075 1650
 AR Path="/62CDD30D/5D4939A7" Ref="Q?"  Part="2"
-AR Path="/62D7188C/5D4939A7" Ref="Q25"  Part="2"
-F 0 "Q25" V 2325 1550 50  0000 L CNN
+AR Path="/62D7188C/5D4939A7" Ref="Q24"  Part="2"
+F 0 "Q24" V 2325 1550 50  0000 L CNN
 F 1 "DMG6602" V 2425 1500 50  0000 L CNN
 F 2 "Package_TO_SOT_SMD:TSOT-23-6" H 2275 1575 50  0001 L CIN
@@
 P 1525 2000
 AR Path="/62CDD30D/5D4939C7" Ref="Q?"  Part="1"
-AR Path="/62D7188C/5D4939C7" Ref="Q27"  Part="1"
-F 0 "Q27" V 1850 1925 50  0000 L BNN
+AR Path="/62D7188C/5D4939C7" Ref="Q26"  Part="1"
+F 0 "Q26" V 1850 1925 50  0000 L BNN
 F 1 "SSM3K35AMFV" V 1775 1750 50  0000 L BNN
 F 2 "Package_TO_SOT_SMD:SOT-723" H 1725 1875 50  0001 L BIN
@@
 P 1275 2250
 AR Path="/62CDD30D/5D4939D8" Ref="R?"  Part="1"
-AR Path="/62D7188C/5D4939D8" Ref="R109"  Part="1"
-F 0 "R109" H 1345 2270 50  0000 L BNN
+AR Path="/62D7188C/5D4939D8" Ref="R108"  Part="1"
+F 0 "R108" H 1345 2270 50  0000 L BNN
 F 1 "CRG0603F4K7" H 575 1850 50  0001 L BNN
 F 2 "Resistor_SMD:R_0603_1608Metric" H 575 1750 50  0001 L BNN
@@
 P 1625 1300
 AR Path="/62CDD30D/5D4939E0" Ref="R?"  Part="1"
-AR Path="/62D7188C/5D4939E0" Ref="R107"  Part="1"
-F 0 "R107" H 1695 1320 50  0000 L BNN
+AR Path="/62D7188C/5D4939E0" Ref="R106"  Part="1"
+F 0 "R106" H 1695 1320 50  0000 L BNN
 F 1 "CRG0603F4K7" H 925 900 50  0001 L BNN
 F 2 "Resistor_SMD:R_0603_1608Metric" H 925 800 50  0001 L BNN
@@
 P 1600 3300
 AR Path="/62CDD30D/5D4939E8" Ref="R?"  Part="1"
-AR Path="/62D7188C/5D4939E8" Ref="R111"  Part="1"
-F 0 "R111" H 1670 3320 50  0000 L BNN
+AR Path="/62D7188C/5D4939E8" Ref="R110"  Part="1"
+F 0 "R110" H 1670 3320 50  0000 L BNN
 F 1 "CRG0603F4K7" H 900 2900 50  0001 L BNN
 F 2 "Resistor_SMD:R_0603_1608Metric" H 900 2800 50  0001 L BNN
