File: ROW_DRIVERS_2.sch (KiCad schematic (older format))
At the start: 36 parts, among them Q120 DMG6602, Q121 DMG6602, Q122 SSM3K35AMFV, Q123 SSM3K35AMFV, Q124 SSM3K35AMFV, Q125 SSM3K35AMFV, Q126 DMG6602, Q127 DMG6602, Q128 SSM3K35AMFV, Q129 SSM3K35AMFV, Q130 SSM3K35AMFV, Q131 SSM3K35AMFV

Commit message: automated commit
Parts:
- removed D42, D43: MMBZ5243BLT1G, symbol custom:MMBZ5243BLT1G
- removed Q120, Q121, Q126, Q127: DMG6602, Package_TO_SOT_SMD:TSOT-23-6, symbol custom:DMG6602
- removed Q122, Q123, Q124, Q125, Q128, Q129, Q130, Q131: SSM3K35AMFV, symbol custom:SSM3K35AMFV
- removed R210, R211, R212, R213, R214, R215, R216, R217, R218, R219, R220, R221, R222, R223, R224, R225: CRG0603F4K7, Resistor_SMD:R_0603_1608Metric, symbol custom:CRG0603F4K7
- added D34, D35: MMBZ5243BLT1G, symbol custom:MMBZ5243BLT1G
- added Q33, Q34, Q37, Q38: DMG6602, Package_TO_SOT_SMD:TSOT-23-6, symbol custom:DMG6602
- added Q35, Q36, Q39, Q40: SSM3K35AMFV, symbol custom:SSM3K35AMFV
- added R115, R116, R117, R118, R119, R120, R121, R122, R123, R124, R125, R126: CRG0603F4K7, Resistor_SMD:R_0603_1608Metric, symbol custom:CRG0603F4K7
Connections:
- net +12V: now also D38.1 (K), D39.1 (K), D34.1 (K), D35.1 (K), Q33.2 (S), Q34.2 (S), Q37.2 (S), Q38.2 (S), R115.1, R116.1, R121.1, R122.1; no longer D36.1 (K), D37.1 (K), D40.1 (K), D41.1 (K)
- net GND: now also D36.2 (A), D37.2 (A), D40.2 (A), D41.2 (A), Q33.5 (S), Q34.5 (S), Q35.2 (S), Q36.2 (S), Q37.5 (S), Q38.5 (S), Q39.2 (S), Q40.2 (S), R117.2, R118.2, R119.2, R120.2, R123.2, R124.2, R125.2, R126.2; no longer D38.2 (A), D39.2 (A)
- net ROW08N: now also D36.1 (K), Q33.6 (D); no longer D38.1 (K)
- net ROW08P: now also D34.2 (A), Q33.4 (D); no longer D36.2 (A)
- net ROW08_OFF: now also Q33.1 (G), R119.1
- net ROW08_ON: now also Q35.1 (G), R117.1
- net ROW09N: now also D37.1 (K), Q34.6 (D); no longer D39.1 (K)
- net ROW09P: now also D35.2 (A), Q34.4 (D); no longer D37.2 (A)
- net ROW09_OFF: now also Q34.1 (G), R120.1
- net ROW09_ON: now also Q36.1 (G), R118.1
- net ROW10N: now also D40.1 (K), Q37.6 (D)
- net ROW10P: now also D38.2 (A), Q37.4 (D); no longer D40.2 (A)
- net ROW10_OFF: now also Q37.1 (G), R125.1
- net ROW10_ON: now also Q39.1 (G), R123.1
- net ROW11N: now also D41.1 (K), Q38.6 (D)
- net ROW11P: now also D39.2 (A), Q38.4 (D); no longer D41.2 (A)
- net ROW11_OFF: now also Q38.1 (G), R126.1
- net ROW11_ON: now also Q40.1 (G), R124.1
- new net: Q34.3 (G), Q36.3 (D), R116.2
- new net: Q38.3 (G), Q40.3 (D), R122.2
- new net: Q37.3 (G), Q39.3 (D), R121.2
- new net: Q33.3 (G), Q35.3 (D), R115.2

Commit message: automated commit
Parts:
- renumbered R115 to R111, R116 to R112, R117 to R113, R118 to R114, R119 to R115, R120 to R116, R121 to R117, R122 to R118, R123 to R119, R124 to R120, R125 to R121, R126 to R122

Commit message: automated commit
Parts:
- D34, D35, D36, D37, D38, D39, D40, D41: footprint (none) -> Package_TO_SOT_SMD:SOT-23
- Q35, Q36, Q39, Q40: footprint (none) -> Package_TO_SOT_SMD:SOT-723
Changed lines of the file:
@@
 F 0 "Q36" V 5250 1925 50  0000 L BNN
 F 1 "SSM3K35AMFV" V 5175 1750 50  0000 L BNN
-F 2 "" H 5125 1875 50  0001 L BIN
+F 2 "Package_TO_SOT_SMD:SOT-723" H 5125 1875 50  0001 L BIN
 F 3 "datasheets/SSM3K35AMFV.pdf" H 5125 1850 50  0001 L BNN
 	1    4925 2000
@@
 F 0 "Q40" V 5250 5300 50  0000 L BNN
 F 1 "SSM3K35AMFV" V 5175 5125 50  0000 L BNN
-F 2 "" H 5125 5250 50  0001 L BIN
+F 2 "Package_TO_SOT_SMD:SOT-723" H 5125 5250 50  0001 L BIN
 F 3 "datasheets/SSM3K35AMFV.pdf" H 5125 5225 50  0001 L BNN
 	1    4925 5375
@@
 F 0 "Q39" V 1850 5300 50  0000 L BNN
 F 1 "SSM3K35AMFV" V 1775 5125 50  0000 L BNN
-F 2 "" H 1725 5250 50  0001 L BIN
+F 2 "Package_TO_SOT_SMD:SOT-723" H 1725 5250 50  0001 L BIN
 F 3 "datasheets/SSM3K35AMFV.pdf" H 1725 5225 50  0001 L BNN
 	1    1525 5375
@@
 F 0 "Q35" V 1850 1925 50  0000 L BNN
 F 1 "SSM3K35AMFV" V 1775 1750 50  0000 L BNN
-F 2 "" H 1725 1875 50  0001 L BIN
+F 2 "Package_TO_SOT_SMD:SOT-723" H 1725 1875 50  0001 L BIN
 F 3 "datasheets/SSM3K35AMFV.pdf" H 1725 1850 50  0001 L BNN
 	1    1525 2000
@@
 F 0 "D36" H 2600 3025 50  0000 C CNN
 F 1 "MMBZ5243BLT1G" H 2575 3175 50  0000 C CNN
-F 2 "" V 2475 3075 50  0001 C CNN
+F 2 "Package_TO_SOT_SMD:SOT-23" V 2475 3075 50  0001 C CNN
 F 3 "" H 2475 3165 50  0001 C CNN
 F 4 "13V" H 2350 3025 39  0000 C CNN "Rating"
@@
 F 0 "D34" H 2800 1575 50  0000 C CNN
 F 1 "MMBZ5243BLT1G" H 2675 1725 50  0000 C CNN
-F 2 "" V 2675 1625 50  0001 C CNN
+F 2 "Package_TO_SOT_SMD:SOT-23" V 2675 1625 50  0001 C CNN
 F 3 "" H 2675 1715 50  0001 C CNN
 F 4 "13V" H 2550 1575 39  0000 C CNN "Rating"
@@
 F 0 "D37" H 6000 3025 50  0000 C CNN
 F 1 "MMBZ5243BLT1G" H 5975 3175 50  0000 C CNN
-F 2 "" V 5875 3075 50  0001 C CNN
+F 2 "Package_TO_SOT_SMD:SOT-23" V 5875 3075 50  0001 C CNN
 F 3 "" H 5875 3165 50  0001 C CNN
 F 4 "13V" H 5750 3025 39  0000 C CNN "Rating"
@@
 F 0 "D35" H 6200 1575 50  0000 C CNN
 F 1 "MMBZ5243BLT1G" H 6075 1725 50  0000 C CNN
-F 2 "" V 6075 1625 50  0001 C CNN
+F 2 "Package_TO_SOT_SMD:SOT-23" V 6075 1625 50  0001 C CNN
 F 3 "" H 6075 1715 50  0001 C CNN
 F 4 "13V" H 5950 1575 39  0000 C CNN "Rating"
@@
 F 0 "D40" H 2600 6400 50  0000 C CNN
 F 1 "MMBZ5243BLT1G" H 2575 6550 50  0000 C CNN
-F 2 "" V 2475 6450 50  0001 C CNN
+F 2 "Package_TO_SOT_SMD:SOT-23" V 2475 6450 50  0001 C CNN
 F 3 "" H 2475 6540 50  0001 C CNN
 F 4 "13V" H 2350 6400 39  0000 C CNN "Rating"
@@
 F 0 "D38" H 2800 4950 50  0000 C CNN
 F 1 "MMBZ5243BLT1G" H 2675 5100 50  0000 C CNN
-F 2 "" V 2675 5000 50  0001 C CNN
+F 2 "Package_TO_SOT_SMD:SOT-23" V 2675 5000 50  0001 C CNN
 F 3 "" H 2675 5090 50  0001 C CNN
 F 4 "13V" H 2550 4950 39  0000 C CNN "Rating"
@@
 F 0 "D41" H 6000 6400 50  0000 C CNN
 F 1 "MMBZ5243BLT1G" H 5975 6550 50  0000 C CNN
-F 2 "" V 5875 6450 50  0001 C CNN
+F 2 "Package_TO_SOT_SMD:SOT-23" V 5875 6450 50  0001 C CNN
 F 3 "" H 5875 6540 50  0001 C CNN
 F 4 "13V" H 5750 6400 39  0000 C CNN "Rating"
@@
 F 0 "D39" H 6200 4950 50  0000 C CNN
 F 1 "MMBZ5243BLT1G" H 6075 5100 50  0000 C CNN
-F 2 "" V 6075 5000 50  0001 C CNN
+F 2 "Package_TO_SOT_SMD:SOT-23" V 6075 5000 50  0001 C CNN
 F 3 "" H 6075 5090 50  0001 C CNN
 F 4 "13V" H 5950 4950 39  0000 C CNN "Rating"

Commit message: automated commit
Parts:
- renumbered R111 to R119, R112 to R120, R113 to R121, R114 to R122, R115 to R123, R116 to R124, R117 to R125, R118 to R126, R119 to R127, R120 to R128, R121 to R129, R122 to R130
Changed lines of the file:
@@
 P 5400 3600
 AR Path="/62CDD30D/5D4D3501" Ref="#PWR?"  Part="1"
-AR Path="/62D71929/5D4D3501" Ref="#PWR0197"  Part="1"
-F 0 "#PWR0197" H 5400 3350 50  0001 C CNN
+AR Path="/62D71929/5D4D3501" Ref="#PWR0199"  Part="1"
+F 0 "#PWR0199" H 5400 3350 50  0001 C CNN
 F 1 "GND" H 5400 3450 50  0000 C CNN
 F 2 "" H 5400 3600 50  0001 C CNN
@@
 P 5575 950
 AR Path="/62CDD30D/5D4D3528" Ref="#PWR?"  Part="1"
-AR Path="/62D71929/5D4D3528" Ref="#PWR0193"  Part="1"
-F 0 "#PWR0193" H 5575 800 50  0001 C CNN
+AR Path="/62D71929/5D4D3528" Ref="#PWR0195"  Part="1"
+F 0 "#PWR0195" H 5575 800 50  0001 C CNN
 F 1 "+12V" H 5575 1090 50  0000 C CNN
 F 2 "" H 5575 950 50  0001 C CNN
@@
 P 5025 2500
 AR Path="/62CDD30D/5D4D352E" Ref="#PWR?"  Part="1"
-AR Path="/62D71929/5D4D352E" Ref="#PWR0195"  Part="1"
-F 0 "#PWR0195" H 5025 2250 50  0001 C CNN
+AR Path="/62D71929/5D4D352E" Ref="#PWR0197"  Part="1"
+F 0 "#PWR0197" H 5025 2250 50  0001 C CNN
 F 1 "GND" H 5025 2350 50  0000 C CNN
 F 2 "" H 5025 2500 50  0001 C CNN
@@
 P 4675 2250
 AR Path="/62CDD30D/5D4D3564" Ref="R?"  Part="1"
-AR Path="/62D71929/5D4D3564" Ref="R114"  Part="1"
-F 0 "R114" H 4745 2270 50  0000 L BNN
+AR Path="/62D71929/5D4D3564" Ref="R122"  Part="1"
+F 0 "R122" H 4745 2270 50  0000 L BNN
 F 1 "CRG0603F4K7" H 3975 1850 50  0001 L BNN
 F 2 "Resistor_SMD:R_0603_1608Metric" H 3975 1750 50  0001 L BNN
@@
 P 5025 1300
 AR Path="/62CDD30D/5D4D356C" Ref="R?"  Part="1"
-AR Path="/62D71929/5D4D356C" Ref="R112"  Part="1"
-F 0 "R112" H 5095 1320 50  0000 L BNN
+AR Path="/62D71929/5D4D356C" Ref="R120"  Part="1"
+F 0 "R120" H 5095 1320 50  0000 L BNN
 F 1 "CRG0603F4K7" H 4325 900 50  0001 L BNN
 F 2 "Resistor_SMD:R_0603_1608Metric" H 4325 800 50  0001 L BNN
@@
 P 5000 3300
 AR Path="/62CDD30D/5D4D3574" Ref="R?"  Part="1"
-AR Path="/62D71929/5D4D3574" Ref="R116"  Part="1"
-F 0 "R116" H 5070 3320 50  0000 L BNN
+AR Path="/62D71929/5D4D3574" Ref="R124"  Part="1"
+F 0 "R124" H 5070 3320 50  0000 L BNN
 F 1 "CRG0603F4K7" H 4300 2900 50  0001 L BNN
 F 2 "Resistor_SMD:R_0603_1608Metric" H 4300 2800 50  0001 L BNN
@@
 P 5400 6975
 AR Path="/62CDD30D/5D4D357B" Ref="#PWR?"  Part="1"
-AR Path="/62D71929/5D4D357B" Ref="#PWR0203"  Part="1"
-F 0 "#PWR0203" H 5400 6725 50  0001 C CNN
+AR Path="/62D71929/5D4D357B" Ref="#PWR0205"  Part="1"
+F 0 "#PWR0205" H 5400 6725 50  0001 C CNN
 F 1 "GND" H 5400 6825 50  0000 C CNN
 F 2 "" H 5400 6975 50  0001 C CNN
@@
 P 5575 4325
 AR Path="/62CDD30D/5D4D35A2" Ref="#PWR?"  Part="1"
-AR Path="/62D71929/5D4D35A2" Ref="#PWR0199"  Part="1"
-F 0 "#PWR0199" H 5575 4175 50  0001 C CNN
+AR Path="/62D71929/5D4D35A2" Ref="#PWR0201"  Part="1"
+F 0 "#PWR0201" H 5575 4175 50  0001 C CNN
 F 1 "+12V" H 5575 4465 50  0000 C CNN
 F 2 "" H 5575 4325 50  0001 C CNN
@@
 P 5025 5875
 AR Path="/62CDD30D/5D4D35A8" Ref="#PWR?"  Part="1"
-AR Path="/62D71929/5D4D35A8" Ref="#PWR0201"  Part="1"
-F 0 "#PWR0201" H 5025 5625 50  0001 C CNN
+AR Path="/62D71929/5D4D35A8" Ref="#PWR0203"  Part="1"
+F 0 "#PWR0203" H 5025 5625 50  0001 C CNN
 F 1 "GND" H 5025 5725 50  0000 C CNN
 F 2 "" H 5025 5875 50  0001 C CNN
@@
 P 4675 5625
 AR Path="/62CDD30D/5D4D35DE" Ref="R?"  Part="1"
-AR Path="/62D71929/5D4D35DE" Ref="R120"  Part="1"
-F 0 "R120" H 4745 5645 50  0000 L BNN
+AR Path="/62D71929/5D4D35DE" Ref="R128"  Part="1"
+F 0 "R128" H 4745 5645 50  0000 L BNN
 F 1 "CRG0603F4K7" H 3975 5225 50  0001 L BNN
 F 2 "Resistor_SMD:R_0603_1608Metric" H 3975 5125 50  0001 L BNN
@@
 P 5025 4675
 AR Path="/62CDD30D/5D4D35E6" Ref="R?"  Part="1"
-AR Path="/62D71929/5D4D35E6" Ref="R118"  Part="1"
-F 0 "R118" H 5095 4695 50  0000 L BNN
+AR Path="/62D71929/5D4D35E6" Ref="R126"  Part="1"
+F 0 "R126" H 5095 4695 50  0000 L BNN
 F 1 "CRG0603F4K7" H 4325 4275 50  0001 L BNN
 F 2 "Resistor_SMD:R_0603_1608Metric" H 4325 4175 50  0001 L BNN
@@
 P 5000 6675
 AR Path="/62CDD30D/5D4D35EE" Ref="R?"  Part="1"
-AR Path="/62D71929/5D4D35EE" Ref="R122"  Part="1"
-F 0 "R122" H 5070 6695 50  0000 L BNN
+AR Path="/62D71929/5D4D35EE" Ref="R130"  Part="1"
+F 0 "R130" H 5070 6695 50  0000 L BNN
 F 1 "CRG0603F4K7" H 4300 6275 50  0001 L BNN
 F 2 "Resistor_SMD:R_0603_1608Metric" H 4300 6175 50  0001 L BNN
@@
 P 2000 6975
 AR Path="/62CDD30D/5D4D35F5" Ref="#PWR?"  Part="1"
-AR Path="/62D71929/5D4D35F5" Ref="#PWR0202"  Part="1"
-F 0 "#PWR0202" H 2000 6725 50  0001 C CNN
+AR Path="/62D71929/5D4D35F5" Ref="#PWR0204"  Part="1"
+F 0 "#PWR0204" H 2000 6725 50  0001 C CNN
 F 1 "GND" H 2000 6825 50  0000 C CNN
 F 2 "" H 2000 6975 50  0001 C CNN
@@
 P 2175 4325
 AR Path="/62CDD30D/5D4D361C" Ref="#PWR?"  Part="1"
-AR Path="/62D71929/5D4D361C" Ref="#PWR0198"  Part="1"
-F 0 "#PWR0198" H 2175 4175 50  0001 C CNN
+AR Path="/62D71929/5D4D361C" Ref="#PWR0200"  Part="1"
+F 0 "#PWR0200" H 2175 4175 50  0001 C CNN
 F 1 "+12V" H 2175 4465 50  0000 C CNN
 F 2 "" H 2175 4325 50  0001 C CNN
@@
 P 1625 5875
 AR Path="/62CDD30D/5D4D3622" Ref="#PWR?"  Part="1"
-AR Path="/62D71929/5D4D3622" Ref="#PWR0200"  Part="1"
-F 0 "#PWR0200" H 1625 5625 50  0001 C CNN
+AR Path="/62D71929/5D4D3622" Ref="#PWR0202"  Part="1"
+F 0 "#PWR0202" H 1625 5625 50  0001 C CNN
 F 1 "GND" H 1625 5725 50  0000 C CNN
 F 2 "" H 1625 5875 50  0001 C CNN
@@
 P 1275 5625
 AR Path="/62CDD30D/5D4D3659" Ref="R?"  Part="1"
-AR Path="/62D71929/5D4D3659" Ref="R119"  Part="1"
-F 0 "R119" H 1345 5645 50  0000 L BNN
+AR Path="/62D71929/5D4D3659" Ref="R127"  Part="1"
+F 0 "R127" H 1345 5645 50  0000 L BNN
 F 1 "CRG0603F4K7" H 575 5225 50  0001 L BNN
 F 2 "Resistor_SMD:R_0603_1608Metric" H 575 5125 50  0001 L BNN
@@
 P 1625 4675
 AR Path="/62CDD30D/5D4D3661" Ref="R?"  Part="1"
-AR Path="/62D71929/5D4D3661" Ref="R117"  Part="1"
-F 0 "R117" H 1695 4695 50  0000 L BNN
+AR Path="/62D71929/5D4D3661" Ref="R125"  Part="1"
+F 0 "R125" H 1695 4695 50  0000 L BNN
 F 1 "CRG0603F4K7" H 925 4275 50  0001 L BNN
 F 2 "Resistor_SMD:R_0603_1608Metric" H 925 4175 50  0001 L BNN
@@
 P 1600 6675
 AR Path="/62CDD30D/5D4D3669" Ref="R?"  Part="1"
-AR Path="/62D71929/5D4D3669" Ref="R121"  Part="1"
-F 0 "R121" H 1670 6695 50  0000 L BNN
+AR Path="/62D71929/5D4D3669" Ref="R129"  Part="1"
+F 0 "R129" H 1670 6695 50  0000 L BNN
 F 1 "CRG0603F4K7" H 900 6275 50  0001 L BNN
 F 2 "Resistor_SMD:R_0603_1608Metric" H 900 6175 50  0001 L BNN
@@
 P 2000 3600
 AR Path="/62CDD30D/5D4D3671" Ref="#PWR?"  Part="1"
-AR Path="/62D71929/5D4D3671" Ref="#PWR0196"  Part="1"
-F 0 "#PWR0196" H 2000 3350 50  0001 C CNN
+AR Path="/62D71929/5D4D3671" Ref="#PWR0198"  Part="1"
+F 0 "#PWR0198" H 2000 3350 50  0001 C CNN
 F 1 "GND" H 2000 3450 50  0000 C CNN
 F 2 "" H 2000 3600 50  0001 C CNN
@@
 P 2175 950
 AR Path="/62CDD30D/5D4D3698" Ref="#PWR?"  Part="1"
-AR Path="/62D71929/5D4D3698" Ref="#PWR0192"  Part="1"
-F 0 "#PWR0192" H 2175 800 50  0001 C CNN
+AR Path="/62D71929/5D4D3698" Ref="#PWR0194"  Part="1"
+F 0 "#PWR0194" H 2175 800 50  0001 C CNN
 F 1 "+12V" H 2175 1090 50  0000 C CNN
 F 2 "" H 2175 950 50  0001 C CNN
@@
 P 1625 2500
 AR Path="/62CDD30D/5D4D369E" Ref="#PWR?"  Part="1"
-AR Path="/62D71929/5D4D369E" Ref="#PWR0194"  Part="1"
-F 0 "#PWR0194" H 1625 2250 50  0001 C CNN
+AR Path="/62D71929/5D4D369E" Ref="#PWR0196"  Part="1"
+F 0 "#PWR0196" H 1625 2250 50  0001 C CNN
 F 1 "GND" H 1625 2350 50  0000 C CNN
 F 2 "" H 1625 2500 50  0001 C CNN
@@
 P 1275 2250
 AR Path="/62CDD30D/5D4D36D5" Ref="R?"  Part="1"
-AR Path="/62D71929/5D4D36D5" Ref="R113"  Part="1"
-F 0 "R113" H 1345 2270 50  0000 L BNN
+AR Path="/62D71929/5D4D36D5" Ref="R121"  Part="1"
+F 0 "R121" H 1345 2270 50  0000 L BNN
 F 1 "CRG0603F4K7" H 575 1850 50  0001 L BNN
 F 2 "Resistor_SMD:R_0603_1608Metric" H 575 1750 50  0001 L BNN
@@
 P 1625 1300
 AR Path="/62CDD30D/5D4D36DD" Ref="R?"  Part="1"
-AR Path="/62D71929/5D4D36DD" Ref="R111"  Part="1"
-F 0 "R111" H 1695 1320 50  0000 L BNN
+AR Path="/62D71929/5D4D36DD" Ref="R119"  Part="1"
+F 0 "R119" H 1695 1320 50  0000 L BNN
 F 1 "CRG0603F4K7" H 925 900 50  0001 L BNN
 F 2 "Resistor_SMD:R_0603_1608Metric" H 925 800 50  0001 L BNN
@@
 P 1600 3300
 AR Path="/62CDD30D/5D4D36E5" Ref="R?"  Part="1"
-AR Path="/62D71929/5D4D36E5" Ref="R115"  Part="1"
-F 0 "R115" H 1670 3320 50  0000 L BNN
+AR Path="/62D71929/5D4D36E5" Ref="R123"  Part="1"
+F 0 "R123" H 1670 3320 50  0000 L BNN
 F 1 "CRG0603F4K7" H 900 2900 50  0001 L BNN
 F 2 "Resistor_SMD:R_0603_1608Metric" H 900 2800 50  0001 L BNN

Commit message: automated commit
Parts:
- renumbered Q33 to Q32, Q34 to Q33, Q35 to Q34, Q36 to Q35, Q37 to Q36, Q38 to Q37, Q39 to Q38, Q40 to Q39, R119 to R118, R120 to R119, R121 to R120, R122 to R121, R123 to R122, R124 to R123, R125 to R124, R126 to R125, R127 to R126, R128 to R127, R129 to R128, R130 to R129
Changed lines of the file:
@@
 P 5300 3075
 AR Path="/62CDD30D/5D4D3507" Ref="Q?"  Part="1"
-AR Path="/62D71929/5D4D3507" Ref="Q34"  Part="1"
-F 0 "Q34" V 5550 2975 50  0000 L CNN
+AR Path="/62D71929/5D4D3507" Ref="Q33"  Part="1"
+F 0 "Q33" V 5550 2975 50  0000 L CNN
 F 1 "DMG6602" V 5650 2900 50  0000 L CNN
 F 2 "Package_TO_SOT_SMD:TSOT-23-6" H 5500 3000 50  0001 L CIN
@@
 P 5475 1650
 AR Path="/62CDD30D/5D4D3534" Ref="Q?"  Part="2"
-AR Path="/62D71929/5D4D3534" Ref="Q34"  Part="2"
-F 0 "Q34" V 5725 1550 50  0000 L CNN
+AR Path="/62D71929/5D4D3534" Ref="Q33"  Part="2"
+F 0 "Q33" V 5725 1550 50  0000 L CNN
 F 1 "DMG6602" V 5825 1500 50  0000 L CNN
 F 2 "Package_TO_SOT_SMD:TSOT-23-6" H 5675 1575 50  0001 L CIN
@@
 P 4925 2000
 AR Path="/62CDD30D/5D4D3554" Ref="Q?"  Part="1"
-AR Path="/62D71929/5D4D3554" Ref="Q36"  Part="1"
-F 0 "Q36" V 5250 1925 50  0000 L BNN
+AR Path="/62D71929/5D4D3554" Ref="Q35"  Part="1"
+F 0 "Q35" V 5250 1925 50  0000 L BNN
 F 1 "SSM3K35AMFV" V 5175 1750 50  0000 L BNN
 F 2 "Package_TO_SOT_SMD:SOT-723" H 5125 1875 50  0001 L BIN
@@
 P 4675 2250
 AR Path="/62CDD30D/5D4D3564" Ref="R?"  Part="1"
-AR Path="/62D71929/5D4D3564" Ref="R122"  Part="1"
-F 0 "R122" H 4745 2270 50  0000 L BNN
+AR Path="/62D71929/5D4D3564" Ref="R121"  Part="1"
+F 0 "R121" H 4745 2270 50  0000 L BNN
 F 1 "CRG0603F4K7" H 3975 1850 50  0001 L BNN
 F 2 "Resistor_SMD:R_0603_1608Metric" H 3975 1750 50  0001 L BNN
@@
 P 5025 1300
 AR Path="/62CDD30D/5D4D356C" Ref="R?"  Part="1"
-AR Path="/62D71929/5D4D356C" Ref="R120"  Part="1"
-F 0 "R120" H 5095 1320 50  0000 L BNN
+AR Path="/62D71929/5D4D356C" Ref="R119"  Part="1"
+F 0 "R119" H 5095 1320 50  0000 L BNN
 F 1 "CRG0603F4K7" H 4325 900 50  0001 L BNN
 F 2 "Resistor_SMD:R_0603_1608Metric" H 4325 800 50  0001 L BNN
@@
 P 5000 3300
 AR Path="/62CDD30D/5D4D3574" Ref="R?"  Part="1"
-AR Path="/62D71929/5D4D3574" Ref="R124"  Part="1"
-F 0 "R124" H 5070 3320 50  0000 L BNN
+AR Path="/62D71929/5D4D3574" Ref="R123"  Part="1"
+F 0 "R123" H 5070 3320 50  0000 L BNN
 F 1 "CRG0603F4K7" H 4300 2900 50  0001 L BNN
 F 2 "Resistor_SMD:R_0603_1608Metric" H 4300 2800 50  0001 L BNN
@@
 P 5300 6450
 AR Path="/62CDD30D/5D4D3581" Ref="Q?"  Part="1"
-AR Path="/62D71929/5D4D3581" Ref="Q38"  Part="1"
-F 0 "Q38" V 5550 6350 50  0000 L CNN
+AR Path="/62D71929/5D4D3581" Ref="Q37"  Part="1"
+F 0 "Q37" V 5550 6350 50  0000 L CNN
 F 1 "DMG6602" V 5650 6275 50  0000 L CNN
 F 2 "Package_TO_SOT_SMD:TSOT-23-6" H 5500 6375 50  0001 L CIN
@@
 P 5475 5025
 AR Path="/62CDD30D/5D4D35AE" Ref="Q?"  Part="2"
-AR Path="/62D71929/5D4D35AE" Ref="Q38"  Part="2"
-F 0 "Q38" V 5725 4925 50  0000 L CNN
+AR Path="/62D71929/5D4D35AE" Ref="Q37"  Part="2"
+F 0 "Q37" V 5725 4925 50  0000 L CNN
 F 1 "DMG6602" V 5825 4875 50  0000 L CNN
 F 2 "Package_TO_SOT_SMD:TSOT-23-6" H 5675 4950 50  0001 L CIN
@@
 P 4925 5375
 AR Path="/62CDD30D/5D4D35CE" Ref="Q?"  Part="1"
-AR Path="/62D71929/5D4D35CE" Ref="Q40"  Part="1"
-F 0 "Q40" V 5250 5300 50  0000 L BNN
+AR Path="/62D71929/5D4D35CE" Ref="Q39"  Part="1"
+F 0 "Q39" V 5250 5300 50  0000 L BNN
 F 1 "SSM3K35AMFV" V 5175 5125 50  0000 L BNN
 F 2 "Package_TO_SOT_SMD:SOT-723" H 5125 5250 50  0001 L BIN
@@
 P 4675 5625
 AR Path="/62CDD30D/5D4D35DE" Ref="R?"  Part="1"
-AR Path="/62D71929/5D4D35DE" Ref="R128"  Part="1"
-F 0 "R128" H 4745 5645 50  0000 L BNN
+AR Path="/62D71929/5D4D35DE" Ref="R127"  Part="1"
+F 0 "R127" H 4745 5645 50  0000 L BNN
 F 1 "CRG0603F4K7" H 3975 5225 50  0001 L BNN
 F 2 "Resistor_SMD:R_0603_1608Metric" H 3975 5125 50  0001 L BNN
@@
 P 5025 4675
 AR Path="/62CDD30D/5D4D35E6" Ref="R?"  Part="1"
-AR Path="/62D71929/5D4D35E6" Ref="R126"  Part="1"
-F 0 "R126" H 5095 4695 50  0000 L BNN
+AR Path="/62D71929/5D4D35E6" Ref="R125"  Part="1"
+F 0 "R125" H 5095 4695 50  0000 L BNN
 F 1 "CRG0603F4K7" H 4325 4275 50  0001 L BNN
 F 2 "Resistor_SMD:R_0603_1608Metric" H 4325 4175 50  0001 L BNN
@@
 P 5000 6675
 AR Path="/62CDD30D/5D4D35EE" Ref="R?"  Part="1"
-AR Path="/62D71929/5D4D35EE" Ref="R130"  Part="1"
-F 0 "R130" H 5070 6695 50  0000 L BNN
+AR Path="/62D71929/5D4D35EE" Ref="R129"  Part="1"
+F 0 "R129" H 5070 6695 50  0000 L BNN
 F 1 "CRG0603F4K7" H 4300 6275 50  0001 L BNN
 F 2 "Resistor_SMD:R_0603_1608Metric" H 4300 6175 50  0001 L BNN
@@
 P 1900 6450
 AR Path="/62CDD30D/5D4D35FB" Ref="Q?"  Part="1"
-AR Path="/62D71929/5D4D35FB" Ref="Q37"  Part="1"
-F 0 "Q37" V 2150 6350 50  0000 L CNN
+AR Path="/62D71929/5D4D35FB" Ref="Q36"  Part="1"
+F 0 "Q36" V 2150 6350 50  0000 L CNN
 F 1 "DMG6602" V 2250 6275 50  0000 L CNN
 F 2 "Package_TO_SOT_SMD:TSOT-23-6" H 2100 6375 50  0001 L CIN
@@
 P 2075 5025
 AR Path="/62CDD30D/5D4D3628" Ref="Q?"  Part="2"
-AR Path="/62D71929/5D4D3628" Ref="Q37"  Part="2"
-F 0 "Q37" V 2325 4925 50  0000 L CNN
+AR Path="/62D71929/5D4D3628" Ref="Q36"  Part="2"
+F 0 "Q36" V 2325 4925 50  0000 L CNN
 F 1 "DMG6602" V 2425 4875 50  0000 L CNN
 F 2 "Package_TO_SOT_SMD:TSOT-23-6" H 2275 4950 50  0001 L CIN
@@
 P 1525 5375
 AR Path="/62CDD30D/5D4D3648" Ref="Q?"  Part="1"
-AR Path="/62D71929/5D4D3648" Ref="Q39"  Part="1"
-F 0 "Q39" V 1850 5300 50  0000 L BNN
+AR Path="/62D71929/5D4D3648" Ref="Q38"  Part="1"
+F 0 "Q38" V 1850 5300 50  0000 L BNN
 F 1 "SSM3K35AMFV" V 1775 5125 50  0000 L BNN
 F 2 "Package_TO_SOT_SMD:SOT-723" H 1725 5250 50  0001 L BIN
@@
 P 1275 5625
 AR Path="/62CDD30D/5D4D3659" Ref="R?"  Part="1"
-AR Path="/62D71929/5D4D3659" Ref="R127"  Part="1"
-F 0 "R127" H 1345 5645 50  0000 L BNN
+AR Path="/62D71929/5D4D3659" Ref="R126"  Part="1"
+F 0 "R126" H 1345 5645 50  0000 L BNN
 F 1 "CRG0603F4K7" H 575 5225 50  0001 L BNN
 F 2 "Resistor_SMD:R_0603_1608Metric" H 575 5125 50  0001 L BNN
@@
 P 1625 4675
 AR Path="/62CDD30D/5D4D3661" Ref="R?"  Part="1"
-AR Path="/62D71929/5D4D3661" Ref="R125"  Part="1"
-F 0 "R125" H 1695 4695 50  0000 L BNN
+AR Path="/62D71929/5D4D3661" Ref="R124"  Part="1"
+F 0 "R124" H 1695 4695 50  0000 L BNN
 F 1 "CRG0603F4K7" H 925 4275 50  0001 L BNN
 F 2 "Resistor_SMD:R_0603_1608Metric" H 925 4175 50  0001 L BNN
@@
 P 1600 6675
 AR Path="/62CDD30D/5D4D3669" Ref="R?"  Part="1"
-AR Path="/62D71929/5D4D3669" Ref="R129"  Part="1"
-F 0 "R129" H 1670 6695 50  0000 L BNN
+AR Path="/62D71929/5D4D3669" Ref="R128"  Part="1"
+F 0 "R128" H 1670 6695 50  0000 L BNN
 F 1 "CRG0603F4K7" H 900 6275 50  0001 L BNN
 F 2 "Resistor_SMD:R_0603_1608Metric" H 900 6175 50  0001 L BNN
@@
 P 1900 3075
 AR Path="/62CDD30D/5D4D3677" Ref="Q?"  Part="1"
-AR Path="/62D71929/5D4D3677" Ref="Q33"  Part="1"
-F 0 "Q33" V 2150 2975 50  0000 L CNN
+AR Path="/62D71929/5D4D3677" Ref="Q32"  Part="1"
+F 0 "Q32" V 2150 2975 50  0000 L CNN
 F 1 "DMG6602" V 2250 2900 50  0000 L CNN
 F 2 "Package_TO_SOT_SMD:TSOT-23-6" H 2100 3000 50  0001 L CIN
@@
 P 2075 1650
 AR Path="/62CDD30D/5D4D36A4" Ref="Q?"  Part="2"
-AR Path="/62D71929/5D4D36A4" Ref="Q33"  Part="2"
-F 0 "Q33" V 2325 1550 50  0000 L CNN
+AR Path="/62D71929/5D4D36A4" Ref="Q32"  Part="2"
+F 0 "Q32" V 2325 1550 50  0000 L CNN
 F 1 "DMG6602" V 2425 1500 50  0000 L CNN
 F 2 "Package_TO_SOT_SMD:TSOT-23-6" H 2275 1575 50  0001 L CIN
@@
 P 1525 2000
 AR Path="/62CDD30D/5D4D36C4" Ref="Q?"  Part="1"
-AR Path="/62D71929/5D4D36C4" Ref="Q35"  Part="1"
-F 0 "Q35" V 1850 1925 50  0000 L BNN
+AR Path="/62D71929/5D4D36C4" Ref="Q34"  Part="1"
+F 0 "Q34" V 1850 1925 50  0000 L BNN
 F 1 "SSM3K35AMFV" V 1775 1750 50  0000 L BNN
 F 2 "Package_TO_SOT_SMD:SOT-723" H 1725 1875 50  0001 L BIN
@@
 P 1275 2250
 AR Path="/62CDD30D/5D4D36D5" Ref="R?"  Part="1"
-AR Path="/62D71929/5D4D36D5" Ref="R121"  Part="1"
-F 0 "R121" H 1345 2270 50  0000 L BNN
+AR Path="/62D71929/5D4D36D5" Ref="R120"  Part="1"
+F 0 "R120" H 1345 2270 50  0000 L BNN
 F 1 "CRG0603F4K7" H 575 1850 50  0001 L BNN
 F 2 "Resistor_SMD:R_0603_1608Metric" H 575 1750 50  0001 L BNN
@@
 P 1625 1300
 AR Path="/62CDD30D/5D4D36DD" Ref="R?"  Part="1"
-AR Path="/62D71929/5D4D36DD" Ref="R119"  Part="1"
-F 0 "R119" H 1695 1320 50  0000 L BNN
+AR Path="/62D71929/5D4D36DD" Ref="R118"  Part="1"
+F 0 "R118" H 1695 1320 50  0000 L BNN
 F 1 "CRG0603F4K7" H 925 900 50  0001 L BNN
 F 2 "Resistor_SMD:R_0603_1608Metric" H 925 800 50  0001 L BNN
@@
 P 1600 3300
 AR Path="/62CDD30D/5D4D36E5" Ref="R?"  Part="1"
-AR Path="/62D71929/5D4D36E5" Ref="R123"  Part="1"
-F 0 "R123" H 1670 3320 50  0000 L BNN
+AR Path="/62D71929/5D4D36E5" Ref="R122"  Part="1"
+F 0 "R122" H 1670 3320 50  0000 L BNN
 F 1 "CRG0603F4K7" H 900 2900 50  0001 L BNN
 F 2 "Resistor_SMD:R_0603_1608Metric" H 900 2800 50  0001 L BNN
