File: ROW_DRIVERS_3.sch (KiCad schematic (older format))
At the start: 40 parts

Commit message: automated commit
Parts:
- removed D? (x8): MMBZ5243BLT1G, symbol custom:MMBZ5243BLT1G
- removed Q? (x8): DMG6602, Package_TO_SOT_SMD:TSOT-23-6, symbol custom:DMG6602
- removed Q? (x8): SSM3K35AMFV, symbol custom:SSM3K35AMFV
- removed R? (x16): CRG0603F4K7, Resistor_SMD:R_0603_1608Metric, symbol custom:CRG0603F4K7
- added D? (x8): MMBZ5243BLT1G, symbol custom:MMBZ5243BLT1G
- added Q? (x8): DMG6602, Package_TO_SOT_SMD:TSOT-23-6, symbol custom:DMG6602
- added Q? (x8): SSM3K35AMFV, symbol custom:SSM3K35AMFV
- added R? (x16): CRG0603F4K7, Resistor_SMD:R_0603_1608Metric, symbol custom:CRG0603F4K7
Connections:
- net +12V: now also D?.1 (K), D?.1 (K), D?.1 (K), D?.1 (K), Q?.2 (S), Q?.2 (S), Q?.2 (S), Q?.2 (S), R?.1, R?.1, R?.1, R?.1
- net GND: now also D?.2 (A), D?.2 (A), D?.2 (A), D?.2 (A), Q?.2 (S), Q?.2 (S), Q?.2 (S), Q?.2 (S), Q?.2 (S), Q?.2 (S), Q?.2 (S), Q?.2 (S), Q?.5 (S), Q?.5 (S), Q?.5 (S), Q?.5 (S), R?.2, R?.2, R?.2, R?.2, R?.2, R?.2, R?.2, R?.2
- new net: Q?.1 (G), Q?.3 (D), R?.1 (x4)
- new net: Q?.3 (D), Q?.3 (G), R?.2 (x4)
- new net ROW12N: D?.1 (K), Q?.6 (D)
- new net ROW12P: D?.2 (A), Q?.4 (D)
- new net ROW12_OFF: R?.1, R?.2
- new net ROW12_ON: Q?.1 (G), Q?.1 (G), R?.1
- new net ROW13N: D?.1 (K), Q?.6 (D)
- new net ROW13P: D?.2 (A), Q?.4 (D)
- new net ROW13_OFF: R?.1, R?.2
- new net ROW13_ON: Q?.1 (G), Q?.1 (G), R?.1
- new net ROW14N: D?.1 (K), Q?.6 (D)
- new net ROW14P: D?.2 (A), Q?.4 (D)
- new net ROW14_OFF: R?.1, R?.2
- new net ROW14_ON: Q?.1 (G), Q?.1 (G), R?.1
- new net ROW15N: D?.1 (K), Q?.6 (D)
- new net ROW15P: D?.2 (A), Q?.4 (D)
- new net ROW15_OFF: R?.1, R?.2
- new net ROW15_ON: Q?.1 (G), Q?.1 (G), R?.1

Commit message: automated commit
Parts:
- gave numbers to parts that had none: 36
