File: ROW_DRIVERS_3.sch (KiCad schematic (older format))
At the start: 36 parts, among them Q132 DMG6602, Q133 DMG6602, Q134 SSM3K35AMFV, Q135 SSM3K35AMFV, Q136 SSM3K35AMFV, Q137 SSM3K35AMFV, Q138 DMG6602, Q139 DMG6602, Q140 SSM3K35AMFV, Q141 SSM3K35AMFV, Q142 SSM3K35AMFV, Q143 SSM3K35AMFV

Commit message: automated commit
Parts:
- removed D50, D51: MMBZ5243BLT1G, symbol custom:MMBZ5243BLT1G
- removed Q132, Q133, Q138, Q139: DMG6602, Package_TO_SOT_SMD:TSOT-23-6, symbol custom:DMG6602
- removed Q134, Q135, Q136, Q137, Q140, Q141, Q142, Q143: SSM3K35AMFV, symbol custom:SSM3K35AMFV
- removed R226, R227, R228, R229, R230, R231, R232, R233, R234, R235, R236, R237, R238, R239, R240, R241: CRG0603F4K7, Resistor_SMD:R_0603_1608Metric, symbol custom:CRG0603F4K7
- added D42, D43: MMBZ5243BLT1G, symbol custom:MMBZ5243BLT1G
- added Q41, Q42, Q45, Q46: DMG6602, Package_TO_SOT_SMD:TSOT-23-6, symbol custom:DMG6602
- added Q43, Q44, Q47, Q48: SSM3K35AMFV, symbol custom:SSM3K35AMFV
- added R127, R128, R129, R130, R131, R132, R133, R134, R135, R136, R137, R138: CRG0603F4K7, Resistor_SMD:R_0603_1608Metric, symbol custom:CRG0603F4K7
Connections:
- net +12V: now also D46.1 (K), D47.1 (K), D42.1 (K), D43.1 (K), Q41.2 (S), Q42.2 (S), Q45.2 (S), Q46.2 (S), R127.1, R128.1, R133.1, R134.1; no longer D44.1 (K), D45.1 (K), D48.1 (K), D49.1 (K)
- net GND: now also D44.2 (A), D45.2 (A), D48.2 (A), D49.2 (A), Q41.5 (S), Q42.5 (S), Q43.2 (S), Q44.2 (S), Q45.5 (S), Q46.5 (S), Q47.2 (S), Q48.2 (S), R129.2, R130.2, R131.2, R132.2, R135.2, R136.2, R137.2, R138.2; no longer D46.2 (A), D47.2 (A)
- net ROW12N: now also D44.1 (K), Q41.6 (D); no longer D46.1 (K)
- net ROW12P: now also D42.2 (A), Q41.4 (D); no longer D44.2 (A)
- net ROW12_OFF: now also Q41.1 (G), R131.1
- net ROW12_ON: now also Q43.1 (G), R129.1
- net ROW13N: now also D45.1 (K), Q42.6 (D); no longer D47.1 (K)
- net ROW13P: now also D43.2 (A), Q42.4 (D); no longer D45.2 (A)
- net ROW13_OFF: now also Q42.1 (G), R132.1
- net ROW13_ON: now also Q44.1 (G), R130.1
- net ROW14N: now also D48.1 (K), Q45.6 (D)
- net ROW14P: now also D46.2 (A), Q45.4 (D); no longer D48.2 (A)
- net ROW14_OFF: now also Q45.1 (G), R137.1
- net ROW14_ON: now also Q47.1 (G), R135.1
- net ROW15N: now also D49.1 (K), Q46.6 (D)
- net ROW15P: now also D47.2 (A), Q46.4 (D); no longer D49.2 (A)
- net ROW15_OFF: now also Q46.1 (G), R138.1
- net ROW15_ON: now also Q48.1 (G), R136.1
- new net: Q42.3 (G), Q44.3 (D), R128.2
- new net: Q46.3 (G), Q48.3 (D), R134.2
- new net: Q45.3 (G), Q47.3 (D), R133.2
- new net: Q41.3 (G), Q43.3 (D), R127.2

Commit message: automated commit
Parts:
- renumbered R127 to R123, R128 to R124, R129 to R125, R130 to R126, R131 to R127, R132 to R128, R133 to R129, R134 to R130, R135 to R131, R136 to R132, R137 to R133, R138 to R134

Commit message: automated commit
Parts:
- D42, D43, D44, D45, D46, D47, D48, D49: footprint (none) -> Package_TO_SOT_SMD:SOT-23
- Q43, Q44, Q47, Q48: footprint (none) -> Package_TO_SOT_SMD:SOT-723
Changed lines of the file:
@@
 F 0 "Q44" V 5250 1925 50  0000 L BNN
 F 1 "SSM3K35AMFV" V 5175 1750 50  0000 L BNN
-F 2 "" H 5125 1875 50  0001 L BIN
+F 2 "Package_TO_SOT_SMD:SOT-723" H 5125 1875 50  0001 L BIN
 F 3 "datasheets/SSM3K35AMFV.pdf" H 5125 1850 50  0001 L BNN
 	1    4925 2000
@@
 F 0 "Q48" V 5250 5300 50  0000 L BNN
 F 1 "SSM3K35AMFV" V 5175 5125 50  0000 L BNN
-F 2 "" H 5125 5250 50  0001 L BIN
+F 2 "Package_TO_SOT_SMD:SOT-723" H 5125 5250 50  0001 L BIN
 F 3 "datasheets/SSM3K35AMFV.pdf" H 5125 5225 50  0001 L BNN
 	1    4925 5375
@@
 F 0 "Q47" V 1850 5300 50  0000 L BNN
 F 1 "SSM3K35AMFV" V 1775 5125 50  0000 L BNN
-F 2 "" H 1725 5250 50  0001 L BIN
+F 2 "Package_TO_SOT_SMD:SOT-723" H 1725 5250 50  0001 L BIN
 F 3 "datasheets/SSM3K35AMFV.pdf" H 1725 5225 50  0001 L BNN
 	1    1525 5375
@@
 F 0 "Q43" V 1850 1925 50  0000 L BNN
 F 1 "SSM3K35AMFV" V 1775 1750 50  0000 L BNN
-F 2 "" H 1725 1875 50  0001 L BIN
+F 2 "Package_TO_SOT_SMD:SOT-723" H 1725 1875 50  0001 L BIN
 F 3 "datasheets/SSM3K35AMFV.pdf" H 1725 1850 50  0001 L BNN
 	1    1525 2000
@@
 F 0 "D44" H 2600 3025 50  0000 C CNN
 F 1 "MMBZ5243BLT1G" H 2575 3175 50  0000 C CNN
-F 2 "" V 2475 3075 50  0001 C CNN
+F 2 "Package_TO_SOT_SMD:SOT-23" V 2475 3075 50  0001 C CNN
 F 3 "" H 2475 3165 50  0001 C CNN
 F 4 "13V" H 2350 3025 39  0000 C CNN "Rating"
@@
 F 0 "D42" H 2800 1575 50  0000 C CNN
 F 1 "MMBZ5243BLT1G" H 2675 1725 50  0000 C CNN
-F 2 "" V 2675 1625 50  0001 C CNN
+F 2 "Package_TO_SOT_SMD:SOT-23" V 2675 1625 50  0001 C CNN
 F 3 "" H 2675 1715 50  0001 C CNN
 F 4 "13V" H 2550 1575 39  0000 C CNN "Rating"
@@
 F 0 "D45" H 6000 3025 50  0000 C CNN
 F 1 "MMBZ5243BLT1G" H 5975 3175 50  0000 C CNN
-F 2 "" V 5875 3075 50  0001 C CNN
+F 2 "Package_TO_SOT_SMD:SOT-23" V 5875 3075 50  0001 C CNN
 F 3 "" H 5875 3165 50  0001 C CNN
 F 4 "13V" H 5750 3025 39  0000 C CNN "Rating"
@@
 F 0 "D43" H 6200 1575 50  0000 C CNN
 F 1 "MMBZ5243BLT1G" H 6075 1725 50  0000 C CNN
-F 2 "" V 6075 1625 50  0001 C CNN
+F 2 "Package_TO_SOT_SMD:SOT-23" V 6075 1625 50  0001 C CNN
 F 3 "" H 6075 1715 50  0001 C CNN
 F 4 "13V" H 5950 1575 39  0000 C CNN "Rating"
@@
 F 0 "D48" H 2600 6400 50  0000 C CNN
 F 1 "MMBZ5243BLT1G" H 2575 6550 50  0000 C CNN
-F 2 "" V 2475 6450 50  0001 C CNN
+F 2 "Package_TO_SOT_SMD:SOT-23" V 2475 6450 50  0001 C CNN
 F 3 "" H 2475 6540 50  0001 C CNN
 F 4 "13V" H 2350 6400 39  0000 C CNN "Rating"
@@
 F 0 "D46" H 2800 4950 50  0000 C CNN
 F 1 "MMBZ5243BLT1G" H 2675 5100 50  0000 C CNN
-F 2 "" V 2675 5000 50  0001 C CNN
+F 2 "Package_TO_SOT_SMD:SOT-23" V 2675 5000 50  0001 C CNN
 F 3 "" H 2675 5090 50  0001 C CNN
 F 4 "13V" H 2550 4950 39  0000 C CNN "Rating"
@@
 F 0 "D49" H 6000 6400 50  0000 C CNN
 F 1 "MMBZ5243BLT1G" H 5975 6550 50  0000 C CNN
-F 2 "" V 5875 6450 50  0001 C CNN
+F 2 "Package_TO_SOT_SMD:SOT-23" V 5875 6450 50  0001 C CNN
 F 3 "" H 5875 6540 50  0001 C CNN
 F 4 "13V" H 5750 6400 39  0000 C CNN "Rating"
@@
 F 0 "D47" H 6200 4950 50  0000 C CNN
 F 1 "MMBZ5243BLT1G" H 6075 5100 50  0000 C CNN
-F 2 "" V 6075 5000 50  0001 C CNN
+F 2 "Package_TO_SOT_SMD:SOT-23" V 6075 5000 50  0001 C CNN
 F 3 "" H 6075 5090 50  0001 C CNN
 F 4 "13V" H 5950 4950 39  0000 C CNN "Rating"

Commit message: automated commit
Parts:
- renumbered R123 to R131, R124 to R132, R125 to R133, R126 to R134, R127 to R135, R128 to R136, R129 to R137, R130 to R138, R131 to R139, R132 to R140, R133 to R141, R134 to R142
Changed lines of the file:
@@
 P 5400 3600
 AR Path="/62CDD30D/5D4FC77B" Ref="#PWR?"  Part="1"
-AR Path="/62D719E9/5D4FC77B" Ref="#PWR0209"  Part="1"
-F 0 "#PWR0209" H 5400 3350 50  0001 C CNN
+AR Path="/62D719E9/5D4FC77B" Ref="#PWR0211"  Part="1"
+F 0 "#PWR0211" H 5400 3350 50  0001 C CNN
 F 1 "GND" H 5400 3450 50  0000 C CNN
 F 2 "" H 5400 3600 50  0001 C CNN
@@
 P 5575 950
 AR Path="/62CDD30D/5D4FC7A2" Ref="#PWR?"  Part="1"
-AR Path="/62D719E9/5D4FC7A2" Ref="#PWR0205"  Part="1"
-F 0 "#PWR0205" H 5575 800 50  0001 C CNN
+AR Path="/62D719E9/5D4FC7A2" Ref="#PWR0207"  Part="1"
+F 0 "#PWR0207" H 5575 800 50  0001 C CNN
 F 1 "+12V" H 5575 1090 50  0000 C CNN
 F 2 "" H 5575 950 50  0001 C CNN
@@
 P 5025 2500
 AR Path="/62CDD30D/5D4FC7A8" Ref="#PWR?"  Part="1"
-AR Path="/62D719E9/5D4FC7A8" Ref="#PWR0207"  Part="1"
-F 0 "#PWR0207" H 5025 2250 50  0001 C CNN
+AR Path="/62D719E9/5D4FC7A8" Ref="#PWR0209"  Part="1"
+F 0 "#PWR0209" H 5025 2250 50  0001 C CNN
 F 1 "GND" H 5025 2350 50  0000 C CNN
 F 2 "" H 5025 2500 50  0001 C CNN
@@
 P 4675 2250
 AR Path="/62CDD30D/5D4FC7DE" Ref="R?"  Part="1"
-AR Path="/62D719E9/5D4FC7DE" Ref="R126"  Part="1"
-F 0 "R126" H 4745 2270 50  0000 L BNN
+AR Path="/62D719E9/5D4FC7DE" Ref="R134"  Part="1"
+F 0 "R134" H 4745 2270 50  0000 L BNN
 F 1 "CRG0603F4K7" H 3975 1850 50  0001 L BNN
 F 2 "Resistor_SMD:R_0603_1608Metric" H 3975 1750 50  0001 L BNN
@@
 P 5025 1300
 AR Path="/62CDD30D/5D4FC7E6" Ref="R?"  Part="1"
-AR Path="/62D719E9/5D4FC7E6" Ref="R124"  Part="1"
-F 0 "R124" H 5095 1320 50  0000 L BNN
+AR Path="/62D719E9/5D4FC7E6" Ref="R132"  Part="1"
+F 0 "R132" H 5095 1320 50  0000 L BNN
 F 1 "CRG0603F4K7" H 4325 900 50  0001 L BNN
 F 2 "Resistor_SMD:R_0603_1608Metric" H 4325 800 50  0001 L BNN
@@
 P 5000 3300
 AR Path="/62CDD30D/5D4FC7EE" Ref="R?"  Part="1"
-AR Path="/62D719E9/5D4FC7EE" Ref="R128"  Part="1"
-F 0 "R128" H 5070 3320 50  0000 L BNN
+AR Path="/62D719E9/5D4FC7EE" Ref="R136"  Part="1"
+F 0 "R136" H 5070 3320 50  0000 L BNN
 F 1 "CRG0603F4K7" H 4300 2900 50  0001 L BNN
 F 2 "Resistor_SMD:R_0603_1608Metric" H 4300 2800 50  0001 L BNN
@@
 P 5400 6975
 AR Path="/62CDD30D/5D4FC7F5" Ref="#PWR?"  Part="1"
-AR Path="/62D719E9/5D4FC7F5" Ref="#PWR0215"  Part="1"
-F 0 "#PWR0215" H 5400 6725 50  0001 C CNN
+AR Path="/62D719E9/5D4FC7F5" Ref="#PWR0217"  Part="1"
+F 0 "#PWR0217" H 5400 6725 50  0001 C CNN
 F 1 "GND" H 5400 6825 50  0000 C CNN
 F 2 "" H 5400 6975 50  0001 C CNN
@@
 P 5575 4325
 AR Path="/62CDD30D/5D4FC81C" Ref="#PWR?"  Part="1"
-AR Path="/62D719E9/5D4FC81C" Ref="#PWR0211"  Part="1"
-F 0 "#PWR0211" H 5575 4175 50  0001 C CNN
+AR Path="/62D719E9/5D4FC81C" Ref="#PWR0213"  Part="1"
+F 0 "#PWR0213" H 5575 4175 50  0001 C CNN
 F 1 "+12V" H 5575 4465 50  0000 C CNN
 F 2 "" H 5575 4325 50  0001 C CNN
@@
 P 5025 5875
 AR Path="/62CDD30D/5D4FC822" Ref="#PWR?"  Part="1"
-AR Path="/62D719E9/5D4FC822" Ref="#PWR0213"  Part="1"
-F 0 "#PWR0213" H 5025 5625 50  0001 C CNN
+AR Path="/62D719E9/5D4FC822" Ref="#PWR0215"  Part="1"
+F 0 "#PWR0215" H 5025 5625 50  0001 C CNN
 F 1 "GND" H 5025 5725 50  0000 C CNN
 F 2 "" H 5025 5875 50  0001 C CNN
@@
 P 4675 5625
 AR Path="/62CDD30D/5D4FC858" Ref="R?"  Part="1"
-AR Path="/62D719E9/5D4FC858" Ref="R132"  Part="1"
-F 0 "R132" H 4745 5645 50  0000 L BNN
+AR Path="/62D719E9/5D4FC858" Ref="R140"  Part="1"
+F 0 "R140" H 4745 5645 50  0000 L BNN
 F 1 "CRG0603F4K7" H 3975 5225 50  0001 L BNN
 F 2 "Resistor_SMD:R_0603_1608Metric" H 3975 5125 50  0001 L BNN
@@
 P 5025 4675
 AR Path="/62CDD30D/5D4FC860" Ref="R?"  Part="1"
-AR Path="/62D719E9/5D4FC860" Ref="R130"  Part="1"
-F 0 "R130" H 5095 4695 50  0000 L BNN
+AR Path="/62D719E9/5D4FC860" Ref="R138"  Part="1"
+F 0 "R138" H 5095 4695 50  0000 L BNN
 F 1 "CRG0603F4K7" H 4325 4275 50  0001 L BNN
 F 2 "Resistor_SMD:R_0603_1608Metric" H 4325 4175 50  0001 L BNN
@@
 P 5000 6675
 AR Path="/62CDD30D/5D4FC868" Ref="R?"  Part="1"
-AR Path="/62D719E9/5D4FC868" Ref="R134"  Part="1"
-F 0 "R134" H 5070 6695 50  0000 L BNN
+AR Path="/62D719E9/5D4FC868" Ref="R142"  Part="1"
+F 0 "R142" H 5070 6695 50  0000 L BNN
 F 1 "CRG0603F4K7" H 4300 6275 50  0001 L BNN
 F 2 "Resistor_SMD:R_0603_1608Metric" H 4300 6175 50  0001 L BNN
@@
 P 2000 6975
 AR Path="/62CDD30D/5D4FC86F" Ref="#PWR?"  Part="1"
-AR Path="/62D719E9/5D4FC86F" Ref="#PWR0214"  Part="1"
-F 0 "#PWR0214" H 2000 6725 50  0001 C CNN
+AR Path="/62D719E9/5D4FC86F" Ref="#PWR0216"  Part="1"
+F 0 "#PWR0216" H 2000 6725 50  0001 C CNN
 F 1 "GND" H 2000 6825 50  0000 C CNN
 F 2 "" H 2000 6975 50  0001 C CNN
@@
 P 2175 4325
 AR Path="/62CDD30D/5D4FC896" Ref="#PWR?"  Part="1"
-AR Path="/62D719E9/5D4FC896" Ref="#PWR0210"  Part="1"
-F 0 "#PWR0210" H 2175 4175 50  0001 C CNN
+AR Path="/62D719E9/5D4FC896" Ref="#PWR0212"  Part="1"
+F 0 "#PWR0212" H 2175 4175 50  0001 C CNN
 F 1 "+12V" H 2175 4465 50  0000 C CNN
 F 2 "" H 2175 4325 50  0001 C CNN
@@
 P 1625 5875
 AR Path="/62CDD30D/5D4FC89C" Ref="#PWR?"  Part="1"
-AR Path="/62D719E9/5D4FC89C" Ref="#PWR0212"  Part="1"
-F 0 "#PWR0212" H 1625 5625 50  0001 C CNN
+AR Path="/62D719E9/5D4FC89C" Ref="#PWR0214"  Part="1"
+F 0 "#PWR0214" H 1625 5625 50  0001 C CNN
 F 1 "GND" H 1625 5725 50  0000 C CNN
 F 2 "" H 1625 5875 50  0001 C CNN
@@
 P 1275 5625
 AR Path="/62CDD30D/5D4FC8D3" Ref="R?"  Part="1"
-AR Path="/62D719E9/5D4FC8D3" Ref="R131"  Part="1"
-F 0 "R131" H 1345 5645 50  0000 L BNN
+AR Path="/62D719E9/5D4FC8D3" Ref="R139"  Part="1"
+F 0 "R139" H 1345 5645 50  0000 L BNN
 F 1 "CRG0603F4K7" H 575 5225 50  0001 L BNN
 F 2 "Resistor_SMD:R_0603_1608Metric" H 575 5125 50  0001 L BNN
@@
 P 1625 4675
 AR Path="/62CDD30D/5D4FC8DB" Ref="R?"  Part="1"
-AR Path="/62D719E9/5D4FC8DB" Ref="R129"  Part="1"
-F 0 "R129" H 1695 4695 50  0000 L BNN
+AR Path="/62D719E9/5D4FC8DB" Ref="R137"  Part="1"
+F 0 "R137" H 1695 4695 50  0000 L BNN
 F 1 "CRG0603F4K7" H 925 4275 50  0001 L BNN
 F 2 "Resistor_SMD:R_0603_1608Metric" H 925 4175 50  0001 L BNN
@@
 P 1600 6675
 AR Path="/62CDD30D/5D4FC8E3" Ref="R?"  Part="1"
-AR Path="/62D719E9/5D4FC8E3" Ref="R133"  Part="1"
-F 0 "R133" H 1670 6695 50  0000 L BNN
+AR Path="/62D719E9/5D4FC8E3" Ref="R141"  Part="1"
+F 0 "R141" H 1670 6695 50  0000 L BNN
 F 1 "CRG0603F4K7" H 900 6275 50  0001 L BNN
 F 2 "Resistor_SMD:R_0603_1608Metric" H 900 6175 50  0001 L BNN
@@
 P 2000 3600
 AR Path="/62CDD30D/5D4FC8EB" Ref="#PWR?"  Part="1"
-AR Path="/62D719E9/5D4FC8EB" Ref="#PWR0208"  Part="1"
-F 0 "#PWR0208" H 2000 3350 50  0001 C CNN
+AR Path="/62D719E9/5D4FC8EB" Ref="#PWR0210"  Part="1"
+F 0 "#PWR0210" H 2000 3350 50  0001 C CNN
 F 1 "GND" H 2000 3450 50  0000 C CNN
 F 2 "" H 2000 3600 50  0001 C CNN
@@
 P 2175 950
 AR Path="/62CDD30D/5D4FC912" Ref="#PWR?"  Part="1"
-AR Path="/62D719E9/5D4FC912" Ref="#PWR0204"  Part="1"
-F 0 "#PWR0204" H 2175 800 50  0001 C CNN
+AR Path="/62D719E9/5D4FC912" Ref="#PWR0206"  Part="1"
+F 0 "#PWR0206" H 2175 800 50  0001 C CNN
 F 1 "+12V" H 2175 1090 50  0000 C CNN
 F 2 "" H 2175 950 50  0001 C CNN
@@
 P 1625 2500
 AR Path="/62CDD30D/5D4FC918" Ref="#PWR?"  Part="1"
-AR Path="/62D719E9/5D4FC918" Ref="#PWR0206"  Part="1"
-F 0 "#PWR0206" H 1625 2250 50  0001 C CNN
+AR Path="/62D719E9/5D4FC918" Ref="#PWR0208"  Part="1"
+F 0 "#PWR0208" H 1625 2250 50  0001 C CNN
 F 1 "GND" H 1625 2350 50  0000 C CNN
 F 2 "" H 1625 2500 50  0001 C CNN
@@
 P 1275 2250
 AR Path="/62CDD30D/5D4FC94F" Ref="R?"  Part="1"
-AR Path="/62D719E9/5D4FC94F" Ref="R125"  Part="1"
-F 0 "R125" H 1345 2270 50  0000 L BNN
+AR Path="/62D719E9/5D4FC94F" Ref="R133"  Part="1"
+F 0 "R133" H 1345 2270 50  0000 L BNN
 F 1 "CRG0603F4K7" H 575 1850 50  0001 L BNN
 F 2 "Resistor_SMD:R_0603_1608Metric" H 575 1750 50  0001 L BNN
@@
 P 1625 1300
 AR Path="/62CDD30D/5D4FC957" Ref="R?"  Part="1"
-AR Path="/62D719E9/5D4FC957" Ref="R123"  Part="1"
-F 0 "R123" H 1695 1320 50  0000 L BNN
+AR Path="/62D719E9/5D4FC957" Ref="R131"  Part="1"
+F 0 "R131" H 1695 1320 50  0000 L BNN
 F 1 "CRG0603F4K7" H 925 900 50  0001 L BNN
 F 2 "Resistor_SMD:R_0603_1608Metric" H 925 800 50  0001 L BNN
@@
 P 1600 3300
 AR Path="/62CDD30D/5D4FC95F" Ref="R?"  Part="1"
-AR Path="/62D719E9/5D4FC95F" Ref="R127"  Part="1"
-F 0 "R127" H 1670 3320 50  0000 L BNN
+AR Path="/62D719E9/5D4FC95F" Ref="R135"  Part="1"
+F 0 "R135" H 1670 3320 50  0000 L BNN
 F 1 "CRG0603F4K7" H 900 2900 50  0001 L BNN
 F 2 "Resistor_SMD:R_0603_1608Metric" H 900 2800 50  0001 L BNN
