File: ROW_DRIVERS_3.sch (KiCad schematic (older format))
At the start: 28 parts, among them Q41 DMG6602, Q42 DMG6602, Q43 SSM3K35AMFV, Q44 SSM3K35AMFV, Q45 DMG6602, Q46 DMG6602, Q47 SSM3K35AMFV, Q48 SSM3K35AMFV

Commit message: automated commit
Parts:
- Q44: renamed from Q45; footprint Package_TO_SOT_SMD:TSOT-23-6 -> TSOT-23-6
- renumbered Q41 to Q40, Q42 to Q41, Q43 to Q42, Q44 to Q43, Q46 to Q45, Q47 to Q46, Q48 to Q47, R131 to R130, R132 to R131, R133 to R132, R134 to R133, R135 to R134, R136 to R135, R137 to R136, R138 to R137, R139 to R138, R140 to R139, R141 to R140, R142 to R141
Changed lines of the file:
@@
 P 5300 3075
 AR Path="/62CDD30D/5D4FC781" Ref="Q?"  Part="1"
-AR Path="/62D719E9/5D4FC781" Ref="Q42"  Part="1"
-F 0 "Q42" V 5550 2975 50  0000 L CNN
+AR Path="/62D719E9/5D4FC781" Ref="Q41"  Part="1"
+F 0 "Q41" V 5550 2975 50  0000 L CNN
 F 1 "DMG6602" V 5650 2900 50  0000 L CNN
 F 2 "Package_TO_SOT_SMD:TSOT-23-6" H 5500 3000 50  0001 L CIN
@@
 P 5475 1650
 AR Path="/62CDD30D/5D4FC7AE" Ref="Q?"  Part="2"
-AR Path="/62D719E9/5D4FC7AE" Ref="Q42"  Part="2"
-F 0 "Q42" V 5725 1550 50  0000 L CNN
+AR Path="/62D719E9/5D4FC7AE" Ref="Q41"  Part="2"
+F 0 "Q41" V 5725 1550 50  0000 L CNN
 F 1 "DMG6602" V 5825 1500 50  0000 L CNN
 F 2 "Package_TO_SOT_SMD:TSOT-23-6" H 5675 1575 50  0001 L CIN
@@
 P 4925 2000
 AR Path="/62CDD30D/5D4FC7CE" Ref="Q?"  Part="1"
-AR Path="/62D719E9/5D4FC7CE" Ref="Q44"  Part="1"
-F 0 "Q44" V 5250 1925 50  0000 L BNN
+AR Path="/62D719E9/5D4FC7CE" Ref="Q43"  Part="1"
+F 0 "Q43" V 5250 1925 50  0000 L BNN
 F 1 "SSM3K35AMFV" V 5175 1750 50  0000 L BNN
 F 2 "Package_TO_SOT_SMD:SOT-723" H 5125 1875 50  0001 L BIN
@@
 P 4675 2250
 AR Path="/62CDD30D/5D4FC7DE" Ref="R?"  Part="1"
-AR Path="/62D719E9/5D4FC7DE" Ref="R134"  Part="1"
-F 0 "R134" H 4745 2270 50  0000 L BNN
+AR Path="/62D719E9/5D4FC7DE" Ref="R133"  Part="1"
+F 0 "R133" H 4745 2270 50  0000 L BNN
 F 1 "CRG0603F4K7" H 3975 1850 50  0001 L BNN
 F 2 "Resistor_SMD:R_0603_1608Metric" H 3975 1750 50  0001 L BNN
@@
 P 5025 1300
 AR Path="/62CDD30D/5D4FC7E6" Ref="R?"  Part="1"
-AR Path="/62D719E9/5D4FC7E6" Ref="R132"  Part="1"
-F 0 "R132" H 5095 1320 50  0000 L BNN
+AR Path="/62D719E9/5D4FC7E6" Ref="R131"  Part="1"
+F 0 "R131" H 5095 1320 50  0000 L BNN
 F 1 "CRG0603F4K7" H 4325 900 50  0001 L BNN
 F 2 "Resistor_SMD:R_0603_1608Metric" H 4325 800 50  0001 L BNN
@@
 P 5000 3300
 AR Path="/62CDD30D/5D4FC7EE" Ref="R?"  Part="1"
-AR Path="/62D719E9/5D4FC7EE" Ref="R136"  Part="1"
-F 0 "R136" H 5070 3320 50  0000 L BNN
+AR Path="/62D719E9/5D4FC7EE" Ref="R135"  Part="1"
+F 0 "R135" H 5070 3320 50  0000 L BNN
 F 1 "CRG0603F4K7" H 4300 2900 50  0001 L BNN
 F 2 "Resistor_SMD:R_0603_1608Metric" H 4300 2800 50  0001 L BNN
@@
 P 5300 6450
 AR Path="/62CDD30D/5D4FC7FB" Ref="Q?"  Part="1"
-AR Path="/62D719E9/5D4FC7FB" Ref="Q46"  Part="1"
-F 0 "Q46" V 5550 6350 50  0000 L CNN
+AR Path="/62D719E9/5D4FC7FB" Ref="Q45"  Part="1"
+F 0 "Q45" V 5550 6350 50  0000 L CNN
 F 1 "DMG6602" V 5650 6275 50  0000 L CNN
 F 2 "Package_TO_SOT_SMD:TSOT-23-6" H 5500 6375 50  0001 L CIN
@@
 P 5475 5025
 AR Path="/62CDD30D/5D4FC828" Ref="Q?"  Part="2"
-AR Path="/62D719E9/5D4FC828" Ref="Q46"  Part="2"
-F 0 "Q46" V 5725 4925 50  0000 L CNN
+AR Path="/62D719E9/5D4FC828" Ref="Q45"  Part="2"
+F 0 "Q45" V 5725 4925 50  0000 L CNN
 F 1 "DMG6602" V 5825 4875 50  0000 L CNN
 F 2 "Package_TO_SOT_SMD:TSOT-23-6" H 5675 4950 50  0001 L CIN
@@
 P 4925 5375
 AR Path="/62CDD30D/5D4FC848" Ref="Q?"  Part="1"
-AR Path="/62D719E9/5D4FC848" Ref="Q48"  Part="1"
-F 0 "Q48" V 5250 5300 50  0000 L BNN
+AR Path="/62D719E9/5D4FC848" Ref="Q47"  Part="1"
+F 0 "Q47" V 5250 5300 50  0000 L BNN
 F 1 "SSM3K35AMFV" V 5175 5125 50  0000 L BNN
 F 2 "Package_TO_SOT_SMD:SOT-723" H 5125 5250 50  0001 L BIN
@@
 P 4675 5625
 AR Path="/62CDD30D/5D4FC858" Ref="R?"  Part="1"
-AR Path="/62D719E9/5D4FC858" Ref="R140"  Part="1"
-F 0 "R140" H 4745 5645 50  0000 L BNN
+AR Path="/62D719E9/5D4FC858" Ref="R139"  Part="1"
+F 0 "R139" H 4745 5645 50  0000 L BNN
 F 1 "CRG0603F4K7" H 3975 5225 50  0001 L BNN
 F 2 "Resistor_SMD:R_0603_1608Metric" H 3975 5125 50  0001 L BNN
@@
 P 5025 4675
 AR Path="/62CDD30D/5D4FC860" Ref="R?"  Part="1"
-AR Path="/62D719E9/5D4FC860" Ref="R138"  Part="1"
-F 0 "R138" H 5095 4695 50  0000 L BNN
+AR Path="/62D719E9/5D4FC860" Ref="R137"  Part="1"
+F 0 "R137" H 5095 4695 50  0000 L BNN
 F 1 "CRG0603F4K7" H 4325 4275 50  0001 L BNN
 F 2 "Resistor_SMD:R_0603_1608Metric" H 4325 4175 50  0001 L BNN
@@
 P 5000 6675
 AR Path="/62CDD30D/5D4FC868" Ref="R?"  Part="1"
-AR Path="/62D719E9/5D4FC868" Ref="R142"  Part="1"
-F 0 "R142" H 5070 6695 50  0000 L BNN
+AR Path="/62D719E9/5D4FC868" Ref="R141"  Part="1"
+F 0 "R141" H 5070 6695 50  0000 L BNN
 F 1 "CRG0603F4K7" H 4300 6275 50  0001 L BNN
 F 2 "Resistor_SMD:R_0603_1608Metric" H 4300 6175 50  0001 L BNN
@@
 P 1900 6450
 AR Path="/62CDD30D/5D4FC875" Ref="Q?"  Part="1"
-AR Path="/62D719E9/5D4FC875" Ref="Q45"  Part="1"
-F 0 "Q45" V 2150 6350 50  0000 L CNN
+AR Path="/62D719E9/5D4FC875" Ref="Q44"  Part="1"
+F 0 "Q44" V 2150 6350 50  0000 L CNN
 F 1 "DMG6602" V 2250 6275 50  0000 L CNN
-F 2 "Package_TO_SOT_SMD:TSOT-23-6" H 2100 6375 50  0001 L CIN
-F 3 "" H 1900 6450 50  0001 L CNN
+F 2 "TSOT-23-6" H 2100 6375 50  0001 L CIN
+F 3 "/home/dj/datasheets/DMG6602SVT.pdf" H 1900 6450 50  0001 L CNN
 	1    1900 6450
 	1    0    0    -1
@@
 P 2075 5025
 AR Path="/62CDD30D/5D4FC8A2" Ref="Q?"  Part="2"
-AR Path="/62D719E9/5D4FC8A2" Ref="Q45"  Part="2"
-F 0 "Q45" V 2325 4925 50  0000 L CNN
+AR Path="/62D719E9/5D4FC8A2" Ref="Q44"  Part="2"
+F 0 "Q44" V 2325 4925 50  0000 L CNN
 F 1 "DMG6602" V 2425 4875 50  0000 L CNN
-F 2 "Package_TO_SOT_SMD:TSOT-23-6" H 2275 4950 50  0001 L CIN
-F 3 "" H 2075 5025 50  0001 L CNN
+F 2 "TSOT-23-6" H 2275 4950 50  0001 L CIN
+F 3 "/home/dj/datasheets/DMG6602SVT.pdf" H 2075 5025 50  0001 L CNN
 	2    2075 5025
 	1    0    0    -1
@@
 P 1525 5375
 AR Path="/62CDD30D/5D4FC8C2" Ref="Q?"  Part="1"
-AR Path="/62D719E9/5D4FC8C2" Ref="Q47"  Part="1"
-F 0 "Q47" V 1850 5300 50  0000 L BNN
+AR Path="/62D719E9/5D4FC8C2" Ref="Q46"  Part="1"
+F 0 "Q46" V 1850 5300 50  0000 L BNN
 F 1 "SSM3K35AMFV" V 1775 5125 50  0000 L BNN
 F 2 "Package_TO_SOT_SMD:SOT-723" H 1725 5250 50  0001 L BIN
@@
 P 1275 5625
 AR Path="/62CDD30D/5D4FC8D3" Ref="R?"  Part="1"
-AR Path="/62D719E9/5D4FC8D3" Ref="R139"  Part="1"
-F 0 "R139" H 1345 5645 50  0000 L BNN
+AR Path="/62D719E9/5D4FC8D3" Ref="R138"  Part="1"
+F 0 "R138" H 1345 5645 50  0000 L BNN
 F 1 "CRG0603F4K7" H 575 5225 50  0001 L BNN
 F 2 "Resistor_SMD:R_0603_1608Metric" H 575 5125 50  0001 L BNN
@@
 P 1625 4675
 AR Path="/62CDD30D/5D4FC8DB" Ref="R?"  Part="1"
-AR Path="/62D719E9/5D4FC8DB" Ref="R137"  Part="1"
-F 0 "R137" H 1695 4695 50  0000 L BNN
+AR Path="/62D719E9/5D4FC8DB" Ref="R136"  Part="1"
+F 0 "R136" H 1695 4695 50  0000 L BNN
 F 1 "CRG0603F4K7" H 925 4275 50  0001 L BNN
 F 2 "Resistor_SMD:R_0603_1608Metric" H 925 4175 50  0001 L BNN
@@
 P 1600 6675
 AR Path="/62CDD30D/5D4FC8E3" Ref="R?"  Part="1"
-AR Path="/62D719E9/5D4FC8E3" Ref="R141"  Part="1"
-F 0 "R141" H 1670 6695 50  0000 L BNN
+AR Path="/62D719E9/5D4FC8E3" Ref="R140"  Part="1"
+F 0 "R140" H 1670 6695 50  0000 L BNN
 F 1 "CRG0603F4K7" H 900 6275 50  0001 L BNN
 F 2 "Resistor_SMD:R_0603_1608Metric" H 900 6175 50  0001 L BNN
@@
 P 1900 3075
 AR Path="/62CDD30D/5D4FC8F1" Ref="Q?"  Part="1"
-AR Path="/62D719E9/5D4FC8F1" Ref="Q41"  Part="1"
-F 0 "Q41" V 2150 2975 50  0000 L CNN
+AR Path="/62D719E9/5D4FC8F1" Ref="Q40"  Part="1"
+F 0 "Q40" V 2150 2975 50  0000 L CNN
 F 1 "DMG6602" V 2250 2900 50  0000 L CNN
 F 2 "Package_TO_SOT_SMD:TSOT-23-6" H 2100 3000 50  0001 L CIN
@@
 P 2075 1650
 AR Path="/62CDD30D/5D4FC91E" Ref="Q?"  Part="2"
-AR Path="/62D719E9/5D4FC91E" Ref="Q41"  Part="2"
-F 0 "Q41" V 2325 1550 50  0000 L CNN
+AR Path="/62D719E9/5D4FC91E" Ref="Q40"  Part="2"
+F 0 "Q40" V 2325 1550 50  0000 L CNN
 F 1 "DMG6602" V 2425 1500 50  0000 L CNN
 F 2 "Package_TO_SOT_SMD:TSOT-23-6" H 2275 1575 50  0001 L CIN
@@
 P 1525 2000
 AR Path="/62CDD30D/5D4FC93E" Ref="Q?"  Part="1"
-AR Path="/62D719E9/5D4FC93E" Ref="Q43"  Part="1"
-F 0 "Q43" V 1850 1925 50  0000 L BNN
+AR Path="/62D719E9/5D4FC93E" Ref="Q42"  Part="1"
+F 0 "Q42" V 1850 1925 50  0000 L BNN
 F 1 "SSM3K35AMFV" V 1775 1750 50  0000 L BNN
 F 2 "Package_TO_SOT_SMD:SOT-723" H 1725 1875 50  0001 L BIN
@@
 P 1275 2250
 AR Path="/62CDD30D/5D4FC94F" Ref="R?"  Part="1"
-AR Path="/62D719E9/5D4FC94F" Ref="R133"  Part="1"
-F 0 "R133" H 1345 2270 50  0000 L BNN
+AR Path="/62D719E9/5D4FC94F" Ref="R132"  Part="1"
+F 0 "R132" H 1345 2270 50  0000 L BNN
 F 1 "CRG0603F4K7" H 575 1850 50  0001 L BNN
 F 2 "Resistor_SMD:R_0603_1608Metric" H 575 1750 50  0001 L BNN
@@
 P 1625 1300
 AR Path="/62CDD30D/5D4FC957" Ref="R?"  Part="1"
-AR Path="/62D719E9/5D4FC957" Ref="R131"  Part="1"
-F 0 "R131" H 1695 1320 50  0000 L BNN
+AR Path="/62D719E9/5D4FC957" Ref="R130"  Part="1"
+F 0 "R130" H 1695 1320 50  0000 L BNN
 F 1 "CRG0603F4K7" H 925 900 50  0001 L BNN
 F 2 "Resistor_SMD:R_0603_1608Metric" H 925 800 50  0001 L BNN
@@
 P 1600 3300
 AR Path="/62CDD30D/5D4FC95F" Ref="R?"  Part="1"
-AR Path="/62D719E9/5D4FC95F" Ref="R135"  Part="1"
-F 0 "R135" H 1670 3320 50  0000 L BNN
+AR Path="/62D719E9/5D4FC95F" Ref="R134"  Part="1"
+F 0 "R134" H 1670 3320 50  0000 L BNN
 F 1 "CRG0603F4K7" H 900 2900 50  0001 L BNN
 F 2 "Resistor_SMD:R_0603_1608Metric" H 900 2800 50  0001 L BNN

Commit message: automated commit
Parts:
- Q44: footprint TSOT-23-6 -> Package_TO_SOT_SMD:TSOT-23-6
Changed lines of the file:
@@
 F 0 "Q44" V 2150 6350 50  0000 L CNN
 F 1 "DMG6602" V 2250 6275 50  0000 L CNN
-F 2 "TSOT-23-6" H 2100 6375 50  0001 L CIN
+F 2 "Package_TO_SOT_SMD:TSOT-23-6" H 2100 6375 50  0001 L CIN
 F 3 "/home/dj/datasheets/DMG6602SVT.pdf" H 1900 6450 50  0001 L CNN
 	1    1900 6450
@@
 F 0 "Q44" V 2325 4925 50  0000 L CNN
 F 1 "DMG6602" V 2425 4875 50  0000 L CNN
-F 2 "TSOT-23-6" H 2275 4950 50  0001 L CIN
+F 2 "Package_TO_SOT_SMD:TSOT-23-6" H 2275 4950 50  0001 L CIN
 F 3 "/home/dj/datasheets/DMG6602SVT.pdf" H 2075 5025 50  0001 L CNN
 	2    2075 5025
