File: SHIFT_REGISTER_SIGNALS.sch (KiCad schematic (older format))
At the start: 27 parts, among them Q144 SSM3K35AMFV, Q145 SSM3K35AMFV

Commit message: automated commit
Parts:
- removed Q145: SSM3K35AMFV, symbol custom:SSM3K35AMFV
- removed R246, R249: NP_R_0603, Resistor_SMD:R_0603_1608Metric, symbol custom:NP_R_0603
- removed R250, R255, R257: CRG0603F4K7, Resistor_SMD:R_0603_1608Metric, symbol custom:CRG0603F4K7
- removed TP40, TP46, TP48: TestPoint, symbol Connector:TestPoint
- added Q? (x2): SSM3K35AMFV, symbol custom:SSM3K35AMFV
- added R? (x2): NP_R_0603, Resistor_SMD:R_0603_1608Metric, symbol custom:NP_R_0603
- added R? (x4): CRG0603F4K7, Resistor_SMD:R_0603_1608Metric, symbol custom:CRG0603F4K7
- added TP? (x4): TestPoint, symbol Connector:TestPoint
Connections:
- net !ROW_SHCP: now also Q?.3 (D), R?.2, TP?.1
- net +3V3: now also R?.1, R?.1, R?.1, R?.1
- net GND: now also Q?.2 (S), Q?.2 (S), R?.2, R?.2
- net ROW_SHCP: now also Q?.1 (G), R?.1, R?.2, TP?.1
- new net ROW_OFF: Q?.3 (D), R?.2, TP?.1
- new net ROW_ON: Q?.1 (G), R?.1, R?.2, TP?.1
Other:
- moved on the sheet: Q144, R242, R243, R244, R245, R247, R248, R251, R252, R253, R254, R256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

Commit message: automated commit
Parts:
- gave numbers to parts that had none: 12
- renumbered Q144 to Q11, R242 to R64, R243 to R65, R244 to R66, R245 to R67, R251 to R70, R252 to R71, R253 to R72, R254 to R73, R247 to R77, R248 to R78, R256 to R80, TP41 to TP22, TP42 to TP23, TP43 to TP24, TP44 to TP25, TP45 to TP30, TP47 to TP31

Commit message: automated commit
Parts:
- R66, R69, R70, R71, R73, R74, R76, R78, R79, R80: Resistance 4.7k -> (none); TOLERANCE (none) -> 5%; VALUE (none) -> 4k7

Commit message: automated commit
Parts:
- renumbered R64 to R60, R65 to R61, R66 to R62, R67 to R63, R68 to R64, R69 to R65, R70 to R66, R71 to R67, R72 to R68, R73 to R69, R74 to R70, R75 to R71, R76 to R72, R77 to R73, R78 to R74, R79 to R75, R80 to R76, TP22 to TP24, TP23 to TP25, TP24 to TP26, TP25 to TP27, TP26 to TP28, TP27 to TP29, TP28 to TP30, TP29 to TP31, TP30 to TP32, TP31 to TP33
Connections:
- net ROW_OFF renamed !ROW_ON
Changed lines of the file:
@@
 AR Path="/627E3ADC/5D4AE4D2" Ref="R?"  Part="1"
 AR Path="/620EB9A4/5D4AE4D2" Ref="R?"  Part="1"
-AR Path="/5D4A63FF/5D4AE4D2" Ref="R77"  Part="1"
-F 0 "R77" V 6820 4475 50  0000 L BNN
+AR Path="/5D4A63FF/5D4AE4D2" Ref="R73"  Part="1"
+F 0 "R73" V 6820 4475 50  0000 L BNN
 F 1 "NP_R_0603" H 5950 4125 50  0001 L BNN
 F 2 "Resistor_SMD:R_0603_1608Metric" H 5950 4025 50  0001 L BNN
@@
 AR Path="/627E3ADC/5D4AE55B" Ref="TP?"  Part="1"
 AR Path="/620EB9A4/5D4AE55B" Ref="TP?"  Part="1"
-AR Path="/5D4A63FF/5D4AE55B" Ref="TP30"  Part="1"
-F 0 "TP30" V 6325 4925 50  0000 C CNN
+AR Path="/5D4A63FF/5D4AE55B" Ref="TP32"  Part="1"
+F 0 "TP32" V 6325 4925 50  0000 C CNN
 F 1 "TestPoint" H 6150 4850 50  0001 C CNN
 F 2 "" H 6600 4800 50  0001 C CNN
@@
 P 3225 2425
 AR Path="/620EB9A4/5D4AE578" Ref="TP?"  Part="1"
-AR Path="/5D4A63FF/5D4AE578" Ref="TP22"  Part="1"
-F 0 "TP22" V 3250 2650 50  0000 L BNN
+AR Path="/5D4A63FF/5D4AE578" Ref="TP24"  Part="1"
+F 0 "TP24" V 3250 2650 50  0000 L BNN
 F 1 "TestPoint" H 2975 2475 50  0001 C CNN
 F 2 "" H 3425 2425 50  0001 C CNN
@@
 P 3325 2425
 AR Path="/620EB9A4/5D4AE57E" Ref="TP?"  Part="1"
-AR Path="/5D4A63FF/5D4AE57E" Ref="TP23"  Part="1"
-F 0 "TP23" V 3350 2650 50  0000 L BNN
+AR Path="/5D4A63FF/5D4AE57E" Ref="TP25"  Part="1"
+F 0 "TP25" V 3350 2650 50  0000 L BNN
 F 1 "TestPoint" H 3075 2475 50  0001 C CNN
 F 2 "" H 3525 2425 50  0001 C CNN
@@
 P 3425 2425
 AR Path="/620EB9A4/5D4AE584" Ref="TP?"  Part="1"
-AR Path="/5D4A63FF/5D4AE584" Ref="TP24"  Part="1"
-F 0 "TP24" V 3450 2650 50  0000 L BNN
+AR Path="/5D4A63FF/5D4AE584" Ref="TP26"  Part="1"
+F 0 "TP26" V 3450 2650 50  0000 L BNN
 F 1 "TestPoint" H 3175 2475 50  0001 C CNN
 F 2 "" H 3625 2425 50  0001 C CNN
@@
 P 3525 2425
 AR Path="/620EB9A4/5D4AE58A" Ref="TP?"  Part="1"
-AR Path="/5D4A63FF/5D4AE58A" Ref="TP25"  Part="1"
-F 0 "TP25" V 3550 2650 50  0000 L BNN
+AR Path="/5D4A63FF/5D4AE58A" Ref="TP27"  Part="1"
+F 0 "TP27" V 3550 2650 50  0000 L BNN
 F 1 "TestPoint" H 3275 2475 50  0001 C CNN
 F 2 "" H 3725 2425 50  0001 C CNN
@@
 AR Path="/627E3ADC/5D4AE567" Ref="TP?"  Part="1"
 AR Path="/620EB9A4/5D4AE567" Ref="TP?"  Part="1"
-AR Path="/5D4A63FF/5D4AE567" Ref="TP31"  Part="1"
-F 0 "TP31" V 7325 4925 50  0000 C CNN
+AR Path="/5D4A63FF/5D4AE567" Ref="TP33"  Part="1"
+F 0 "TP33" V 7325 4925 50  0000 C CNN
 F 1 "TestPoint" H 7150 4850 50  0001 C CNN
 F 2 "" H 7600 4800 50  0001 C CNN
@@
 AR Path="/627E3ADC/5D0ECA8D" Ref="R?"  Part="1"
 AR Path="/620EB9A4/5D0ECA8D" Ref="R?"  Part="1"
-AR Path="/5D4A63FF/5D0ECA8D" Ref="R68"  Part="1"
-F 0 "R68" V 6820 2225 50  0000 L BNN
+AR Path="/5D4A63FF/5D0ECA8D" Ref="R64"  Part="1"
+F 0 "R64" V 6820 2225 50  0000 L BNN
 F 1 "NP_R_0603" H 5950 1875 50  0001 L BNN
 F 2 "Resistor_SMD:R_0603_1608Metric" H 5950 1775 50  0001 L BNN
@@
 AR Path="/627E3ADC/5D0ECAA7" Ref="TP?"  Part="1"
 AR Path="/620EB9A4/5D0ECAA7" Ref="TP?"  Part="1"
-AR Path="/5D4A63FF/5D0ECAA7" Ref="TP26"  Part="1"
-F 0 "TP26" V 6325 2675 50  0000 C CNN
+AR Path="/5D4A63FF/5D0ECAA7" Ref="TP28"  Part="1"
+F 0 "TP28" V 6325 2675 50  0000 C CNN
 F 1 "TestPoint" H 6150 2600 50  0001 C CNN
 F 2 "" H 6600 2550 50  0001 C CNN
@@
 AR Path="/627E3ADC/5D0ECABB" Ref="TP?"  Part="1"
 AR Path="/620EB9A4/5D0ECABB" Ref="TP?"  Part="1"
-AR Path="/5D4A63FF/5D0ECABB" Ref="TP27"  Part="1"
-F 0 "TP27" V 7325 2675 50  0000 C CNN
+AR Path="/5D4A63FF/5D0ECABB" Ref="TP29"  Part="1"
+F 0 "TP29" V 7325 2675 50  0000 C CNN
 F 1 "TestPoint" H 7150 2600 50  0001 C CNN
 F 2 "" H 7600 2550 50  0001 C CNN
@@
 AR Path="/627E3ADC/5D11F45B" Ref="R?"  Part="1"
 AR Path="/620EB9A4/5D11F45B" Ref="R?"  Part="1"
-AR Path="/5D4A63FF/5D11F45B" Ref="R75"  Part="1"
-F 0 "R75" V 3395 4475 50  0000 L BNN
+AR Path="/5D4A63FF/5D11F45B" Ref="R71"  Part="1"
+F 0 "R71" V 3395 4475 50  0000 L BNN
 F 1 "NP_R_0603" H 2525 4125 50  0001 L BNN
 F 2 "Resistor_SMD:R_0603_1608Metric" H 2525 4025 50  0001 L BNN
@@
 AR Path="/627E3ADC/5D11F475" Ref="TP?"  Part="1"
 AR Path="/620EB9A4/5D11F475" Ref="TP?"  Part="1"
-AR Path="/5D4A63FF/5D11F475" Ref="TP28"  Part="1"
-F 0 "TP28" V 2900 4925 50  0000 C CNN
+AR Path="/5D4A63FF/5D11F475" Ref="TP30"  Part="1"
+F 0 "TP30" V 2900 4925 50  0000 C CNN
 F 1 "TestPoint" H 2725 4850 50  0001 C CNN
 F 2 "" H 3175 4800 50  0001 C CNN
@@
 ROW_ON
 Text GLabel 4150 4875 2    50   Output ~ 0
-ROW_OFF
+!ROW_ON
 Connection ~ 3975 4875
 Wire Wire Line
@@
 AR Path="/627E3ADC/5D11F489" Ref="TP?"  Part="1"
 AR Path="/620EB9A4/5D11F489" Ref="TP?"  Part="1"
-AR Path="/5D4A63FF/5D11F489" Ref="TP29"  Part="1"
-F 0 "TP29" V 3900 4925 50  0000 C CNN
+AR Path="/5D4A63FF/5D11F489" Ref="TP31"  Part="1"
+F 0 "TP31" V 3900 4925 50  0000 C CNN
 F 1 "TestPoint" H 3725 4850 50  0001 C CNN
 F 2 "" H 4175 4800 50  0001 C CNN
@@
 AR Path="/627E3ADC/5D4AE4FC" Ref="R?"  Part="1"
 AR Path="/620EB9A4/5D4AE4FC" Ref="R?"  Part="1"
-AR Path="/5D4A63FF/5D4AE4FC" Ref="R72"  Part="1"
-F 0 "R72" V 4500 2875 50  0000 L BNN
+AR Path="/5D4A63FF/5D4AE4FC" Ref="R68"  Part="1"
+F 0 "R68" V 4500 2875 50  0000 L BNN
 F 1 "NP_R_0603" H 3625 2525 50  0001 L BNN
 F 2 "Resistor_SMD:R_0603_1608Metric" H 3625 2425 50  0001 L BNN
@@
 $EndComp
 $Comp
-L custom:CRG0603F4K7 R73
+L custom:CRG0603F4K7 R69
 U 1 1 5D03699A
 P 4575 2975
-F 0 "R73" V 4700 2875 50  0000 L BNN
+F 0 "R69" V 4700 2875 50  0000 L BNN
 F 1 "CRG0603F4K7" H 3875 2575 50  0001 L BNN
 F 2 "Resistor_SMD:R_0603_1608Metric" H 3875 2475 50  0001 L BNN
@@
 $EndComp
 $Comp
-L custom:CRG0603F4K7 R71
+L custom:CRG0603F4K7 R67
 U 1 1 5D0366BC
 P 4175 2975
-F 0 "R71" V 4300 2875 50  0000 L BNN
+F 0 "R67" V 4300 2875 50  0000 L BNN
 F 1 "CRG0603F4K7" H 3475 2575 50  0001 L BNN
 F 2 "Resistor_SMD:R_0603_1608Metric" H 3475 2475 50  0001 L BNN
@@
 $EndComp
 $Comp
-L custom:CRG0603F4K7 R70
+L custom:CRG0603F4K7 R66
 U 1 1 5D03573E
 P 3975 2975
-F 0 "R70" V 4100 2875 50  0000 L BNN
+F 0 "R66" V 4100 2875 50  0000 L BNN
 F 1 "CRG0603F4K7" H 3275 2575 50  0001 L BNN
 F 2 "Resistor_SMD:R_0603_1608Metric" H 3275 2475 50  0001 L BNN
@@
 AR Path="/627E3ADC/5D4AE4EE" Ref="R?"  Part="1"
 AR Path="/620EB9A4/5D4AE4EE" Ref="R?"  Part="1"
-AR Path="/5D4A63FF/5D4AE4EE" Ref="R67"  Part="1"
-F 0 "R67" V 4695 2175 50  0000 L BNN
+AR Path="/5D4A63FF/5D4AE4EE" Ref="R63"  Part="1"
+F 0 "R63" V 4695 2175 50  0000 L BNN
 F 1 "NP_R_0603" H 3825 1825 50  0001 L BNN
 F 2 "Resistor_SMD:R_0603_1608Metric" H 3825 1725 50  0001 L BNN
@@
 AR Path="/627E3ADC/5D4AE4E7" Ref="R?"  Part="1"
 AR Path="/620EB9A4/5D4AE4E7" Ref="R?"  Part="1"
-AR Path="/5D4A63FF/5D4AE4E7" Ref="R65"  Part="1"
-F 0 "R65" V 4295 2175 50  0000 L BNN
+AR Path="/5D4A63FF/5D4AE4E7" Ref="R61"  Part="1"
+F 0 "R61" V 4295 2175 50  0000 L BNN
 F 1 "NP_R_0603" H 3425 1825 50  0001 L BNN
 F 2 "Resistor_SMD:R_0603_1608Metric" H 3425 1725 50  0001 L BNN
@@
 AR Path="/627E3ADC/5D4AE4E0" Ref="R?"  Part="1"
 AR Path="/620EB9A4/5D4AE4E0" Ref="R?"  Part="1"
-AR Path="/5D4A63FF/5D4AE4E0" Ref="R64"  Part="1"
-F 0 "R64" V 4095 2175 50  0000 L BNN
+AR Path="/5D4A63FF/5D4AE4E0" Ref="R60"  Part="1"
+F 0 "R60" V 4095 2175 50  0000 L BNN
 F 1 "NP_R_0603" H 3225 1825 50  0001 L BNN
 F 2 "Resistor_SMD:R_0603_1608Metric" H 3225 1725 50  0001 L BNN
@@
 	4175 2125 4175 2075
 $Comp
-L custom:CRG0603F4K7 R66
+L custom:CRG0603F4K7 R62
 U 1 1 5D037099
 P 4375 2275
-F 0 "R66" V 4500 2175 50  0000 L BNN
+F 0 "R62" V 4500 2175 50  0000 L BNN
 F 1 "CRG0603F4K7" H 3675 1875 50  0001 L BNN
 F 2 "Resistor_SMD:R_0603_1608Metric" H 3675 1775 50  0001 L BNN
@@
 $EndComp
 $Comp
-L custom:CRG0603F4K7 R69
+L custom:CRG0603F4K7 R65
 U 1 1 5D04A2E0
 P 7100 2325
-F 0 "R69" V 7225 2225 50  0000 L BNN
+F 0 "R65" V 7225 2225 50  0000 L BNN
 F 1 "CRG0603F4K7" H 6400 1925 50  0001 L BNN
 F 2 "Resistor_SMD:R_0603_1608Metric" H 6400 1825 50  0001 L BNN
@@
 $EndComp
 $Comp
-L custom:CRG0603F4K7 R74
+L custom:CRG0603F4K7 R70
 U 1 1 5D04ABB5
 P 6700 3250
-F 0 "R74" V 6825 3150 50  0000 L BNN
+F 0 "R70" V 6825 3150 50  0000 L BNN
 F 1 "CRG0603F4K7" H 6000 2850 50  0001 L BNN
 F 2 "Resistor_SMD:R_0603_1608Metric" H 6000 2750 50  0001 L BNN
@@
 $EndComp
 $Comp
-L custom:CRG0603F4K7 R76
+L custom:CRG0603F4K7 R72
 U 1 1 5D04B149
 P 3675 4575
-F 0 "R76" V 3800 4475 50  0000 L BNN
+F 0 "R72" V 3800 4475 50  0000 L BNN
 F 1 "CRG0603F4K7" H 2975 4175 50  0001 L BNN
 F 2 "Resistor_SMD:R_0603_1608Metric" H 2975 4075 50  0001 L BNN
@@
 $EndComp
 $Comp
-L custom:CRG0603F4K7 R79
+L custom:CRG0603F4K7 R75
 U 1 1 5D04B871
 P 3275 5500
-F 0 "R79" V 3400 5400 50  0000 L BNN
+F 0 "R75" V 3400 5400 50  0000 L BNN
 F 1 "CRG0603F4K7" H 2575 5100 50  0001 L BNN
 F 2 "Resistor_SMD:R_0603_1608Metric" H 2575 5000 50  0001 L BNN
@@
 $EndComp
 $Comp
-L custom:CRG0603F4K7 R80
+L custom:CRG0603F4K7 R76
 U 1 1 5D04BCA3
 P 6700 5500
-F 0 "R80" V 6825 5400 50  0000 L BNN
+F 0 "R76" V 6825 5400 50  0000 L BNN
 F 1 "CRG0603F4K7" H 6000 5100 50  0001 L BNN
 F 2 "Resistor_SMD:R_0603_1608Metric" H 6000 5000 50  0001 L BNN
@@
 $EndComp
 $Comp
-L custom:CRG0603F4K7 R78
+L custom:CRG0603F4K7 R74
 U 1 1 5D04C10F
 P 7100 4575
-F 0 "R78" V 7225 4475 50  0000 L BNN
+F 0 "R74" V 7225 4475 50  0000 L BNN
 F 1 "CRG0603F4K7" H 6400 4175 50  0001 L BNN
 F 2 "Resistor_SMD:R_0603_1608Metric" H 6400 4075 50  0001 L BNN

Commit message: automated commit
Parts:
- Q10, Q11, Q9: footprint (none) -> Package_TO_SOT_SMD:SOT-723
Changed lines of the file:
@@
 F 0 "Q11" V 7325 5150 50  0000 L BNN
 F 1 "SSM3K35AMFV" V 7250 4975 50  0000 L BNN
-F 2 "" H 7200 5100 50  0001 L BIN
+F 2 "Package_TO_SOT_SMD:SOT-723" H 7200 5100 50  0001 L BIN
 F 3 "datasheets/SSM3K35AMFV.pdf" H 7200 5075 50  0001 L BNN
 	1    7000 5225
@@
 F 0 "Q9" V 7325 2900 50  0000 L BNN
 F 1 "SSM3K35AMFV" V 7250 2725 50  0000 L BNN
-F 2 "" H 7200 2850 50  0001 L BIN
+F 2 "Package_TO_SOT_SMD:SOT-723" H 7200 2850 50  0001 L BIN
 F 3 "datasheets/SSM3K35AMFV.pdf" H 7200 2825 50  0001 L BNN
 	1    7000 2975
@@
 F 0 "Q10" V 3900 5150 50  0000 L BNN
 F 1 "SSM3K35AMFV" V 3825 4975 50  0000 L BNN
-F 2 "" H 3775 5100 50  0001 L BIN
+F 2 "Package_TO_SOT_SMD:SOT-723" H 3775 5100 50  0001 L BIN
 F 3 "datasheets/SSM3K35AMFV.pdf" H 3775 5075 50  0001 L BNN
 	1    3575 5225

Commit message: automated commit
Parts:
- TP29: renamed from TP24; footprint (none) -> custom:TestPoint_THTPad_D1.0mm_Drill0.5mm
- TP30: renamed from TP25; footprint (none) -> custom:TestPoint_THTPad_D1.0mm_Drill0.5mm
- TP31: renamed from TP26; footprint (none) -> custom:TestPoint_THTPad_D1.0mm_Drill0.5mm
- TP32: renamed from TP27; footprint (none) -> custom:TestPoint_THTPad_D1.0mm_Drill0.5mm
- TP33: renamed from TP28; footprint (none) -> custom:TestPoint_THTPad_D1.0mm_Drill0.5mm
- TP34: renamed from TP29; footprint (none) -> custom:TestPoint_THTPad_D1.0mm_Drill0.5mm
- TP35: renamed from TP30; footprint (none) -> custom:TestPoint_THTPad_D1.0mm_Drill0.5mm
- TP36: renamed from TP31; footprint (none) -> custom:TestPoint_THTPad_D1.0mm_Drill0.5mm
- TP37: renamed from TP32; footprint (none) -> custom:TestPoint_THTPad_D1.0mm_Drill0.5mm
- TP38: renamed from TP33; footprint (none) -> custom:TestPoint_THTPad_D1.0mm_Drill0.5mm
Changed lines of the file:
@@
 AR Path="/627E3ADC/5D4AE55B" Ref="TP?"  Part="1"
 AR Path="/620EB9A4/5D4AE55B" Ref="TP?"  Part="1"
-AR Path="/5D4A63FF/5D4AE55B" Ref="TP32"  Part="1"
-F 0 "TP32" V 6325 4925 50  0000 C CNN
+AR Path="/5D4A63FF/5D4AE55B" Ref="TP37"  Part="1"
+F 0 "TP37" V 6325 4925 50  0000 C CNN
 F 1 "TestPoint" H 6150 4850 50  0001 C CNN
-F 2 "" H 6600 4800 50  0001 C CNN
+F 2 "custom:TestPoint_THTPad_D1.0mm_Drill0.5mm" H 6600 4800 50  0001 C CNN
 F 3 "~" H 6600 4800 50  0001 C CNN
 	1    6400 4800
@@
 P 3225 2425
 AR Path="/620EB9A4/5D4AE578" Ref="TP?"  Part="1"
-AR Path="/5D4A63FF/5D4AE578" Ref="TP24"  Part="1"
-F 0 "TP24" V 3250 2650 50  0000 L BNN
+AR Path="/5D4A63FF/5D4AE578" Ref="TP29"  Part="1"
+F 0 "TP29" V 3250 2650 50  0000 L BNN
 F 1 "TestPoint" H 2975 2475 50  0001 C CNN
-F 2 "" H 3425 2425 50  0001 C CNN
+F 2 "custom:TestPoint_THTPad_D1.0mm_Drill0.5mm" H 3425 2425 50  0001 C CNN
 F 3 "~" H 3425 2425 50  0001 C CNN
 	1    3225 2425
@@
 P 3325 2425
 AR Path="/620EB9A4/5D4AE57E" Ref="TP?"  Part="1"
-AR Path="/5D4A63FF/5D4AE57E" Ref="TP25"  Part="1"
-F 0 "TP25" V 3350 2650 50  0000 L BNN
+AR Path="/5D4A63FF/5D4AE57E" Ref="TP30"  Part="1"
+F 0 "TP30" V 3350 2650 50  0000 L BNN
 F 1 "TestPoint" H 3075 2475 50  0001 C CNN
-F 2 "" H 3525 2425 50  0001 C CNN
+F 2 "custom:TestPoint_THTPad_D1.0mm_Drill0.5mm" H 3525 2425 50  0001 C CNN
 F 3 "~" H 3525 2425 50  0001 C CNN
 	1    3325 2425
@@
 P 3425 2425
 AR Path="/620EB9A4/5D4AE584" Ref="TP?"  Part="1"
-AR Path="/5D4A63FF/5D4AE584" Ref="TP26"  Part="1"
-F 0 "TP26" V 3450 2650 50  0000 L BNN
+AR Path="/5D4A63FF/5D4AE584" Ref="TP31"  Part="1"
+F 0 "TP31" V 3450 2650 50  0000 L BNN
 F 1 "TestPoint" H 3175 2475 50  0001 C CNN
-F 2 "" H 3625 2425 50  0001 C CNN
+F 2 "custom:TestPoint_THTPad_D1.0mm_Drill0.5mm" H 3625 2425 50  0001 C CNN
 F 3 "~" H 3625 2425 50  0001 C CNN
 	1    3425 2425
@@
 P 3525 2425
 AR Path="/620EB9A4/5D4AE58A" Ref="TP?"  Part="1"
-AR Path="/5D4A63FF/5D4AE58A" Ref="TP27"  Part="1"
-F 0 "TP27" V 3550 2650 50  0000 L BNN
+AR Path="/5D4A63FF/5D4AE58A" Ref="TP32"  Part="1"
+F 0 "TP32" V 3550 2650 50  0000 L BNN
 F 1 "TestPoint" H 3275 2475 50  0001 C CNN
-F 2 "" H 3725 2425 50  0001 C CNN
+F 2 "custom:TestPoint_THTPad_D1.0mm_Drill0.5mm" H 3725 2425 50  0001 C CNN
 F 3 "~" H 3725 2425 50  0001 C CNN
 	1    3525 2425
@@
 AR Path="/627E3ADC/5D4AE567" Ref="TP?"  Part="1"
 AR Path="/620EB9A4/5D4AE567" Ref="TP?"  Part="1"
-AR Path="/5D4A63FF/5D4AE567" Ref="TP33"  Part="1"
-F 0 "TP33" V 7325 4925 50  0000 C CNN
+AR Path="/5D4A63FF/5D4AE567" Ref="TP38"  Part="1"
+F 0 "TP38" V 7325 4925 50  0000 C CNN
 F 1 "TestPoint" H 7150 4850 50  0001 C CNN
-F 2 "" H 7600 4800 50  0001 C CNN
+F 2 "custom:TestPoint_THTPad_D1.0mm_Drill0.5mm" H 7600 4800 50  0001 C CNN
 F 3 "~" H 7600 4800 50  0001 C CNN
 	1    7400 4800
@@
 AR Path="/627E3ADC/5D0ECAA7" Ref="TP?"  Part="1"
 AR Path="/620EB9A4/5D0ECAA7" Ref="TP?"  Part="1"
-AR Path="/5D4A63FF/5D0ECAA7" Ref="TP28"  Part="1"
-F 0 "TP28" V 6325 2675 50  0000 C CNN
+AR Path="/5D4A63FF/5D0ECAA7" Ref="TP33"  Part="1"
+F 0 "TP33" V 6325 2675 50  0000 C CNN
 F 1 "TestPoint" H 6150 2600 50  0001 C CNN
-F 2 "" H 6600 2550 50  0001 C CNN
+F 2 "custom:TestPoint_THTPad_D1.0mm_Drill0.5mm" H 6600 2550 50  0001 C CNN
 F 3 "~" H 6600 2550 50  0001 C CNN
 	1    6400 2550
@@
 AR Path="/627E3ADC/5D0ECABB" Ref="TP?"  Part="1"
 AR Path="/620EB9A4/5D0ECABB" Ref="TP?"  Part="1"
-AR Path="/5D4A63FF/5D0ECABB" Ref="TP29"  Part="1"
-F 0 "TP29" V 7325 2675 50  0000 C CNN
+AR Path="/5D4A63FF/5D0ECABB" Ref="TP34"  Part="1"
+F 0 "TP34" V 7325 2675 50  0000 C CNN
 F 1 "TestPoint" H 7150 2600 50  0001 C CNN
-F 2 "" H 7600 2550 50  0001 C CNN
+F 2 "custom:TestPoint_THTPad_D1.0mm_Drill0.5mm" H 7600 2550 50  0001 C CNN
 F 3 "~" H 7600 2550 50  0001 C CNN
 	1    7400 2550
@@
 AR Path="/627E3ADC/5D11F475" Ref="TP?"  Part="1"
 AR Path="/620EB9A4/5D11F475" Ref="TP?"  Part="1"
-AR Path="/5D4A63FF/5D11F475" Ref="TP30"  Part="1"
-F 0 "TP30" V 2900 4925 50  0000 C CNN
+AR Path="/5D4A63FF/5D11F475" Ref="TP35"  Part="1"
+F 0 "TP35" V 2900 4925 50  0000 C CNN
 F 1 "TestPoint" H 2725 4850 50  0001 C CNN
-F 2 "" H 3175 4800 50  0001 C CNN
+F 2 "custom:TestPoint_THTPad_D1.0mm_Drill0.5mm" H 3175 4800 50  0001 C CNN
 F 3 "~" H 3175 4800 50  0001 C CNN
 	1    2975 4800
@@
 AR Path="/627E3ADC/5D11F489" Ref="TP?"  Part="1"
 AR Path="/620EB9A4/5D11F489" Ref="TP?"  Part="1"
-AR Path="/5D4A63FF/5D11F489" Ref="TP31"  Part="1"
-F 0 "TP31" V 3900 4925 50  0000 C CNN
+AR Path="/5D4A63FF/5D11F489" Ref="TP36"  Part="1"
+F 0 "TP36" V 3900 4925 50  0000 C CNN
 F 1 "TestPoint" H 3725 4850 50  0001 C CNN
-F 2 "" H 4175 4800 50  0001 C CNN
+F 2 "custom:TestPoint_THTPad_D1.0mm_Drill0.5mm" H 4175 4800 50  0001 C CNN
 F 3 "~" H 4175 4800 50  0001 C CNN
 	1    3975 4800
