File: SHIFT_REGISTER_SIGNALS.sch (KiCad schematic (older format))
At the start: 30 parts, among them Q10 SSM3K35AMFV, Q11 SSM3K35AMFV, Q9 SSM3K35AMFV

Commit message: automated commit
Parts:
- renumbered R60 to R68, R61 to R69, R62 to R70, R63 to R71, R64 to R72, R65 to R73, R66 to R74, R67 to R75, R68 to R76, R69 to R77, R70 to R78, R71 to R79, R72 to R80, R73 to R81, R74 to R82, R75 to R83, R76 to R84
Changed lines of the file:
@@
 AR Path="/627E3ADC/5D4AE45E" Ref="#PWR?"  Part="1"
 AR Path="/620EB9A4/5D4AE45E" Ref="#PWR?"  Part="1"
-AR Path="/5D4A63FF/5D4AE45E" Ref="#PWR0104"  Part="1"
-F 0 "#PWR0104" H 6900 5550 50  0001 C CNN
+AR Path="/5D4A63FF/5D4AE45E" Ref="#PWR0106"  Part="1"
+F 0 "#PWR0106" H 6900 5550 50  0001 C CNN
 F 1 "GND" H 6900 5650 50  0000 C CNN
 F 2 "" H 6900 5800 50  0001 C CNN
@@
 AR Path="/627E3ADC/5D4AE4C5" Ref="#PWR?"  Part="1"
 AR Path="/620EB9A4/5D4AE4C5" Ref="#PWR?"  Part="1"
-AR Path="/5D4A63FF/5D4AE4C5" Ref="#PWR0102"  Part="1"
-F 0 "#PWR0102" H 6900 4125 50  0001 C CNN
+AR Path="/5D4A63FF/5D4AE4C5" Ref="#PWR0104"  Part="1"
+F 0 "#PWR0104" H 6900 4125 50  0001 C CNN
 F 1 "+3V3" H 6900 4415 50  0000 C CNN
 F 2 "" H 6900 4275 50  0001 C CNN
@@
 AR Path="/627E3ADC/5D4AE4D2" Ref="R?"  Part="1"
 AR Path="/620EB9A4/5D4AE4D2" Ref="R?"  Part="1"
-AR Path="/5D4A63FF/5D4AE4D2" Ref="R73"  Part="1"
-F 0 "R73" V 6820 4475 50  0000 L BNN
+AR Path="/5D4A63FF/5D4AE4D2" Ref="R81"  Part="1"
+F 0 "R81" V 6820 4475 50  0000 L BNN
 F 1 "NP_R_0603" H 5950 4125 50  0001 L BNN
 F 2 "Resistor_SMD:R_0603_1608Metric" H 5950 4025 50  0001 L BNN
@@
 AR Path="/627E3ADC/5D0ECA6F" Ref="#PWR?"  Part="1"
 AR Path="/620EB9A4/5D0ECA6F" Ref="#PWR?"  Part="1"
-AR Path="/5D4A63FF/5D0ECA6F" Ref="#PWR0100"  Part="1"
-F 0 "#PWR0100" H 6900 3300 50  0001 C CNN
+AR Path="/5D4A63FF/5D0ECA6F" Ref="#PWR0102"  Part="1"
+F 0 "#PWR0102" H 6900 3300 50  0001 C CNN
 F 1 "GND" H 6900 3400 50  0000 C CNN
 F 2 "" H 6900 3550 50  0001 C CNN
@@
 AR Path="/627E3ADC/5D0ECA86" Ref="#PWR?"  Part="1"
 AR Path="/620EB9A4/5D0ECA86" Ref="#PWR?"  Part="1"
-AR Path="/5D4A63FF/5D0ECA86" Ref="#PWR098"  Part="1"
-F 0 "#PWR098" H 6900 1875 50  0001 C CNN
+AR Path="/5D4A63FF/5D0ECA86" Ref="#PWR0100"  Part="1"
+F 0 "#PWR0100" H 6900 1875 50  0001 C CNN
 F 1 "+3V3" H 6900 2165 50  0000 C CNN
 F 2 "" H 6900 2025 50  0001 C CNN
@@
 AR Path="/627E3ADC/5D0ECA8D" Ref="R?"  Part="1"
 AR Path="/620EB9A4/5D0ECA8D" Ref="R?"  Part="1"
-AR Path="/5D4A63FF/5D0ECA8D" Ref="R64"  Part="1"
-F 0 "R64" V 6820 2225 50  0000 L BNN
+AR Path="/5D4A63FF/5D0ECA8D" Ref="R72"  Part="1"
+F 0 "R72" V 6820 2225 50  0000 L BNN
 F 1 "NP_R_0603" H 5950 1875 50  0001 L BNN
 F 2 "Resistor_SMD:R_0603_1608Metric" H 5950 1775 50  0001 L BNN
@@
 AR Path="/627E3ADC/5D11F43D" Ref="#PWR?"  Part="1"
 AR Path="/620EB9A4/5D11F43D" Ref="#PWR?"  Part="1"
-AR Path="/5D4A63FF/5D11F43D" Ref="#PWR0103"  Part="1"
-F 0 "#PWR0103" H 3475 5550 50  0001 C CNN
+AR Path="/5D4A63FF/5D11F43D" Ref="#PWR0105"  Part="1"
+F 0 "#PWR0105" H 3475 5550 50  0001 C CNN
 F 1 "GND" H 3475 5650 50  0000 C CNN
 F 2 "" H 3475 5800 50  0001 C CNN
@@
 AR Path="/627E3ADC/5D11F454" Ref="#PWR?"  Part="1"
 AR Path="/620EB9A4/5D11F454" Ref="#PWR?"  Part="1"
-AR Path="/5D4A63FF/5D11F454" Ref="#PWR0101"  Part="1"
-F 0 "#PWR0101" H 3475 4125 50  0001 C CNN
+AR Path="/5D4A63FF/5D11F454" Ref="#PWR0103"  Part="1"
+F 0 "#PWR0103" H 3475 4125 50  0001 C CNN
 F 1 "+3V3" H 3475 4415 50  0000 C CNN
 F 2 "" H 3475 4275 50  0001 C CNN
@@
 AR Path="/627E3ADC/5D11F45B" Ref="R?"  Part="1"
 AR Path="/620EB9A4/5D11F45B" Ref="R?"  Part="1"
-AR Path="/5D4A63FF/5D11F45B" Ref="R71"  Part="1"
-F 0 "R71" V 3395 4475 50  0000 L BNN
+AR Path="/5D4A63FF/5D11F45B" Ref="R79"  Part="1"
+F 0 "R79" V 3395 4475 50  0000 L BNN
 F 1 "NP_R_0603" H 2525 4125 50  0001 L BNN
 F 2 "Resistor_SMD:R_0603_1608Metric" H 2525 4025 50  0001 L BNN
@@
 AR Path="/627E3ADC/5D4AE4FC" Ref="R?"  Part="1"
 AR Path="/620EB9A4/5D4AE4FC" Ref="R?"  Part="1"
-AR Path="/5D4A63FF/5D4AE4FC" Ref="R68"  Part="1"
-F 0 "R68" V 4500 2875 50  0000 L BNN
+AR Path="/5D4A63FF/5D4AE4FC" Ref="R76"  Part="1"
+F 0 "R76" V 4500 2875 50  0000 L BNN
 F 1 "NP_R_0603" H 3625 2525 50  0001 L BNN
 F 2 "Resistor_SMD:R_0603_1608Metric" H 3625 2425 50  0001 L BNN
@@
 AR Path="/627E3ADC/5D4AE458" Ref="#PWR?"  Part="1"
 AR Path="/620EB9A4/5D4AE458" Ref="#PWR?"  Part="1"
-AR Path="/5D4A63FF/5D4AE458" Ref="#PWR099"  Part="1"
-F 0 "#PWR099" H 4575 2975 50  0001 C CNN
+AR Path="/5D4A63FF/5D4AE458" Ref="#PWR0101"  Part="1"
+F 0 "#PWR0101" H 4575 2975 50  0001 C CNN
 F 1 "GND" H 4575 3075 50  0000 C CNN
 F 2 "" H 4575 3225 50  0001 C CNN
@@
 $EndComp
 $Comp
-L custom:CRG0603F4K7 R69
+L custom:CRG0603F4K7 R77
 U 1 1 5D03699A
 P 4575 2975
-F 0 "R69" V 4700 2875 50  0000 L BNN
+F 0 "R77" V 4700 2875 50  0000 L BNN
 F 1 "CRG0603F4K7" H 3875 2575 50  0001 L BNN
 F 2 "Resistor_SMD:R_0603_1608Metric" H 3875 2475 50  0001 L BNN
@@
 $EndComp
 $Comp
-L custom:CRG0603F4K7 R67
+L custom:CRG0603F4K7 R75
 U 1 1 5D0366BC
 P 4175 2975
-F 0 "R67" V 4300 2875 50  0000 L BNN
+F 0 "R75" V 4300 2875 50  0000 L BNN
 F 1 "CRG0603F4K7" H 3475 2575 50  0001 L BNN
 F 2 "Resistor_SMD:R_0603_1608Metric" H 3475 2475 50  0001 L BNN
@@
 $EndComp
 $Comp
-L custom:CRG0603F4K7 R66
+L custom:CRG0603F4K7 R74
 U 1 1 5D03573E
 P 3975 2975
-F 0 "R66" V 4100 2875 50  0000 L BNN
+F 0 "R74" V 4100 2875 50  0000 L BNN
 F 1 "CRG0603F4K7" H 3275 2575 50  0001 L BNN
 F 2 "Resistor_SMD:R_0603_1608Metric" H 3275 2475 50  0001 L BNN
@@
 AR Path="/627E3ADC/5D4AE4EE" Ref="R?"  Part="1"
 AR Path="/620EB9A4/5D4AE4EE" Ref="R?"  Part="1"
-AR Path="/5D4A63FF/5D4AE4EE" Ref="R63"  Part="1"
-F 0 "R63" V 4695 2175 50  0000 L BNN
+AR Path="/5D4A63FF/5D4AE4EE" Ref="R71"  Part="1"
+F 0 "R71" V 4695 2175 50  0000 L BNN
 F 1 "NP_R_0603" H 3825 1825 50  0001 L BNN
 F 2 "Resistor_SMD:R_0603_1608Metric" H 3825 1725 50  0001 L BNN
@@
 AR Path="/627E3ADC/5D4AE4E7" Ref="R?"  Part="1"
 AR Path="/620EB9A4/5D4AE4E7" Ref="R?"  Part="1"
-AR Path="/5D4A63FF/5D4AE4E7" Ref="R61"  Part="1"
-F 0 "R61" V 4295 2175 50  0000 L BNN
+AR Path="/5D4A63FF/5D4AE4E7" Ref="R69"  Part="1"
+F 0 "R69" V 4295 2175 50  0000 L BNN
 F 1 "NP_R_0603" H 3425 1825 50  0001 L BNN
 F 2 "Resistor_SMD:R_0603_1608Metric" H 3425 1725 50  0001 L BNN
@@
 AR Path="/627E3ADC/5D4AE4E0" Ref="R?"  Part="1"
 AR Path="/620EB9A4/5D4AE4E0" Ref="R?"  Part="1"
-AR Path="/5D4A63FF/5D4AE4E0" Ref="R60"  Part="1"
-F 0 "R60" V 4095 2175 50  0000 L BNN
+AR Path="/5D4A63FF/5D4AE4E0" Ref="R68"  Part="1"
+F 0 "R68" V 4095 2175 50  0000 L BNN
 F 1 "NP_R_0603" H 3225 1825 50  0001 L BNN
 F 2 "Resistor_SMD:R_0603_1608Metric" H 3225 1725 50  0001 L BNN
@@
 AR Path="/627E3ADC/5D4AE4CB" Ref="#PWR?"  Part="1"
 AR Path="/620EB9A4/5D4AE4CB" Ref="#PWR?"  Part="1"
-AR Path="/5D4A63FF/5D4AE4CB" Ref="#PWR097"  Part="1"
-F 0 "#PWR097" H 3975 1875 50  0001 C CNN
+AR Path="/5D4A63FF/5D4AE4CB" Ref="#PWR099"  Part="1"
+F 0 "#PWR099" H 3975 1875 50  0001 C CNN
 F 1 "+3V3" H 3975 2165 50  0000 C CNN
 F 2 "" H 3975 2025 50  0001 C CNN
@@
 	4175 2125 4175 2075
 $Comp
-L custom:CRG0603F4K7 R62
+L custom:CRG0603F4K7 R70
 U 1 1 5D037099
 P 4375 2275
-F 0 "R62" V 4500 2175 50  0000 L BNN
+F 0 "R70" V 4500 2175 50  0000 L BNN
 F 1 "CRG0603F4K7" H 3675 1875 50  0001 L BNN
 F 2 "Resistor_SMD:R_0603_1608Metric" H 3675 1775 50  0001 L BNN
@@
 $EndComp
 $Comp
-L custom:CRG0603F4K7 R65
+L custom:CRG0603F4K7 R73
 U 1 1 5D04A2E0
 P 7100 2325
-F 0 "R65" V 7225 2225 50  0000 L BNN
+F 0 "R73" V 7225 2225 50  0000 L BNN
 F 1 "CRG0603F4K7" H 6400 1925 50  0001 L BNN
 F 2 "Resistor_SMD:R_0603_1608Metric" H 6400 1825 50  0001 L BNN
@@
 $EndComp
 $Comp
-L custom:CRG0603F4K7 R70
+L custom:CRG0603F4K7 R78
 U 1 1 5D04ABB5
 P 6700 3250
-F 0 "R70" V 6825 3150 50  0000 L BNN
+F 0 "R78" V 6825 3150 50  0000 L BNN
 F 1 "CRG0603F4K7" H 6000 2850 50  0001 L BNN
 F 2 "Resistor_SMD:R_0603_1608Metric" H 6000 2750 50  0001 L BNN
@@
 $EndComp
 $Comp
-L custom:CRG0603F4K7 R72
+L custom:CRG0603F4K7 R80
 U 1 1 5D04B149
 P 3675 4575
-F 0 "R72" V 3800 4475 50  0000 L BNN
+F 0 "R80" V 3800 4475 50  0000 L BNN
 F 1 "CRG0603F4K7" H 2975 4175 50  0001 L BNN
 F 2 "Resistor_SMD:R_0603_1608Metric" H 2975 4075 50  0001 L BNN
@@
 $EndComp
 $Comp
-L custom:CRG0603F4K7 R75
+L custom:CRG0603F4K7 R83
 U 1 1 5D04B871
 P 3275 5500
-F 0 "R75" V 3400 5400 50  0000 L BNN
+F 0 "R83" V 3400 5400 50  0000 L BNN
 F 1 "CRG0603F4K7" H 2575 5100 50  0001 L BNN
 F 2 "Resistor_SMD:R_0603_1608Metric" H 2575 5000 50  0001 L BNN
@@
 $EndComp
 $Comp
-L custom:CRG0603F4K7 R76
+L custom:CRG0603F4K7 R84
 U 1 1 5D04BCA3
 P 6700 5500
-F 0 "R76" V 6825 5400 50  0000 L BNN
+F 0 "R84" V 6825 5400 50  0000 L BNN
 F 1 "CRG0603F4K7" H 6000 5100 50  0001 L BNN
 F 2 "Resistor_SMD:R_0603_1608Metric" H 6000 5000 50  0001 L BNN
@@
 $EndComp
 $Comp
-L custom:CRG0603F4K7 R74
+L custom:CRG0603F4K7 R82
 U 1 1 5D04C10F
 P 7100 4575
-F 0 "R74" V 7225 4475 50  0000 L BNN
+F 0 "R82" V 7225 4475 50  0000 L BNN
 F 1 "CRG0603F4K7" H 6400 4175 50  0001 L BNN
 F 2 "Resistor_SMD:R_0603_1608Metric" H 6400 4075 50  0001 L BNN
