File: ROW_SHIFT_REGISTER.sch (KiCad schematic (older format))
At the start: 27 parts, among them Q12 AO3407A, Q13 SSM3K35AMFV, Q14 SSM3K35AMFV, U10 74HC595, U11 74HC595, U12 74HC595, U9 74HC595

Commit message: automated commit
Parts:
- TP39: renamed from TP34; footprint (none) -> custom:TestPoint_THTPad_D1.0mm_Drill0.5mm
- TP40: renamed from TP35; footprint (none) -> custom:TestPoint_THTPad_D1.0mm_Drill0.5mm
- TP41: renamed from TP36; footprint (none) -> custom:TestPoint_THTPad_D1.0mm_Drill0.5mm
- TP42: renamed from TP37; footprint (none) -> custom:TestPoint_THTPad_D1.0mm_Drill0.5mm
Changed lines of the file:
@@
 AR Path="/61C6D021/5D6F7153" Ref="TP?"  Part="1"
 AR Path="/609E0ED6/5D6F7153" Ref="TP?"  Part="1"
-AR Path="/621F0CB4/5D6F7153" Ref="TP34"  Part="1"
-F 0 "TP34" V 1425 3675 50  0000 C CNN
+AR Path="/621F0CB4/5D6F7153" Ref="TP39"  Part="1"
+F 0 "TP39" V 1425 3675 50  0000 C CNN
 F 1 "TestPoint" H 1275 3550 50  0001 C CNN
-F 2 "" H 1725 3500 50  0001 C CNN
+F 2 "custom:TestPoint_THTPad_D1.0mm_Drill0.5mm" H 1725 3500 50  0001 C CNN
 F 3 "~" H 1725 3500 50  0001 C CNN
 	1    1525 3500
@@
 AR Path="/61C6D021/5D702E1C" Ref="TP?"  Part="1"
 AR Path="/609E0ED6/5D702E1C" Ref="TP?"  Part="1"
-AR Path="/621F0CB4/5D702E1C" Ref="TP35"  Part="1"
-F 0 "TP35" V 4575 3675 50  0000 C CNN
+AR Path="/621F0CB4/5D702E1C" Ref="TP40"  Part="1"
+F 0 "TP40" V 4575 3675 50  0000 C CNN
 F 1 "TestPoint" H 4425 3550 50  0001 C CNN
-F 2 "" H 4875 3500 50  0001 C CNN
+F 2 "custom:TestPoint_THTPad_D1.0mm_Drill0.5mm" H 4875 3500 50  0001 C CNN
 F 3 "~" H 4875 3500 50  0001 C CNN
 	1    4675 3500
@@
 AR Path="/61C6D021/5D723118" Ref="TP?"  Part="1"
 AR Path="/609E0ED6/5D723118" Ref="TP?"  Part="1"
-AR Path="/621F0CB4/5D723118" Ref="TP36"  Part="1"
-F 0 "TP36" H 1425 6075 50  0000 C CNN
+AR Path="/621F0CB4/5D723118" Ref="TP41"  Part="1"
+F 0 "TP41" H 1425 6075 50  0000 C CNN
 F 1 "TestPoint" H 1150 5900 50  0001 C CNN
-F 2 "" H 1600 5850 50  0001 C CNN
+F 2 "custom:TestPoint_THTPad_D1.0mm_Drill0.5mm" H 1600 5850 50  0001 C CNN
 F 3 "~" H 1600 5850 50  0001 C CNN
 	1    1400 5850
@@
 AR Path="/61C6D021/5D72F4B0" Ref="TP?"  Part="1"
 AR Path="/609E0ED6/5D72F4B0" Ref="TP?"  Part="1"
-AR Path="/621F0CB4/5D72F4B0" Ref="TP37"  Part="1"
-F 0 "TP37" H 4575 6075 50  0000 C CNN
+AR Path="/621F0CB4/5D72F4B0" Ref="TP42"  Part="1"
+F 0 "TP42" H 4575 6075 50  0000 C CNN
 F 1 "TestPoint" H 4300 5900 50  0001 C CNN
-F 2 "" H 4750 5850 50  0001 C CNN
+F 2 "custom:TestPoint_THTPad_D1.0mm_Drill0.5mm" H 4750 5850 50  0001 C CNN
 F 3 "~" H 4750 5850 50  0001 C CNN
 	1    4550 5850

Commit message: automated commit
Parts:
- renumbered R77 to R85, R78 to R86, R79 to R87, R80 to R88
Changed lines of the file:
@@
 P 1875 3100
 AR Path="/622B9CF4" Ref="#PWR?"  Part="1"
-AR Path="/621F0CB4/622B9CF4" Ref="#PWR0112"  Part="1"
-F 0 "#PWR0112" H 1875 2850 50  0001 C CNN
+AR Path="/621F0CB4/622B9CF4" Ref="#PWR0114"  Part="1"
+F 0 "#PWR0114" H 1875 2850 50  0001 C CNN
 F 1 "GND" H 1875 2950 50  0000 C CNN
 F 2 "" H 1875 3100 50  0001 C CNN
@@
 P 1875 6025
 AR Path="/622B9CFD" Ref="#PWR?"  Part="1"
-AR Path="/621F0CB4/622B9CFD" Ref="#PWR0121"  Part="1"
-F 0 "#PWR0121" H 1875 5775 50  0001 C CNN
+AR Path="/621F0CB4/622B9CFD" Ref="#PWR0123"  Part="1"
+F 0 "#PWR0123" H 1875 5775 50  0001 C CNN
 F 1 "GND" H 1875 5875 50  0000 C CNN
 F 2 "" H 1875 6025 50  0001 C CNN
@@
 P 5025 3100
 AR Path="/622B9D05" Ref="#PWR?"  Part="1"
-AR Path="/621F0CB4/622B9D05" Ref="#PWR0113"  Part="1"
-F 0 "#PWR0113" H 5025 2850 50  0001 C CNN
+AR Path="/621F0CB4/622B9D05" Ref="#PWR0115"  Part="1"
+F 0 "#PWR0115" H 5025 2850 50  0001 C CNN
 F 1 "GND" H 5025 2950 50  0000 C CNN
 F 2 "" H 5025 3100 50  0001 C CNN
@@
 P 1875 5025
 AR Path="/622B9E98" Ref="#PWR?"  Part="1"
-AR Path="/621F0CB4/622B9E98" Ref="#PWR0119"  Part="1"
-F 0 "#PWR0119" H 1875 4875 50  0001 C CNN
+AR Path="/621F0CB4/622B9E98" Ref="#PWR0121"  Part="1"
+F 0 "#PWR0121" H 1875 4875 50  0001 C CNN
 F 1 "+3V3" H 1875 5165 50  0000 C CNN
 F 2 "" H 1875 5025 50  0001 C CNN
@@
 P 5025 2100
 AR Path="/622B9E9E" Ref="#PWR?"  Part="1"
-AR Path="/621F0CB4/622B9E9E" Ref="#PWR0110"  Part="1"
-F 0 "#PWR0110" H 5025 1950 50  0001 C CNN
+AR Path="/621F0CB4/622B9E9E" Ref="#PWR0112"  Part="1"
+F 0 "#PWR0112" H 5025 1950 50  0001 C CNN
 F 1 "+3V3" H 5025 2240 50  0000 C CNN
 F 2 "" H 5025 2100 50  0001 C CNN
@@
 P 5025 5025
 AR Path="/622B9EB0" Ref="#PWR?"  Part="1"
-AR Path="/621F0CB4/622B9EB0" Ref="#PWR0120"  Part="1"
-F 0 "#PWR0120" H 5025 4875 50  0001 C CNN
+AR Path="/621F0CB4/622B9EB0" Ref="#PWR0122"  Part="1"
+F 0 "#PWR0122" H 5025 4875 50  0001 C CNN
 F 1 "+3V3" H 5025 5165 50  0000 C CNN
 F 2 "" H 5025 5025 50  0001 C CNN
@@
 P 1875 2100
 AR Path="/622B9EC8" Ref="#PWR?"  Part="1"
-AR Path="/621F0CB4/622B9EC8" Ref="#PWR0109"  Part="1"
-F 0 "#PWR0109" H 1875 1950 50  0001 C CNN
+AR Path="/621F0CB4/622B9EC8" Ref="#PWR0111"  Part="1"
+F 0 "#PWR0111" H 1875 1950 50  0001 C CNN
 F 1 "+3V3" H 1875 2240 50  0000 C CNN
 F 2 "" H 1875 2100 50  0001 C CNN
@@
 P 1925 1250
 AR Path="/622B9ED4" Ref="#PWR?"  Part="1"
-AR Path="/621F0CB4/622B9ED4" Ref="#PWR0105"  Part="1"
-F 0 "#PWR0105" H 1925 1100 50  0001 C CNN
+AR Path="/621F0CB4/622B9ED4" Ref="#PWR0107"  Part="1"
+F 0 "#PWR0107" H 1925 1100 50  0001 C CNN
 F 1 "+3V3" H 1925 1390 50  0000 C CNN
 F 2 "" H 1925 1250 50  0001 C CNN
@@
 P 2825 1800
 AR Path="/622B9F05" Ref="#PWR?"  Part="1"
-AR Path="/621F0CB4/622B9F05" Ref="#PWR0107"  Part="1"
-F 0 "#PWR0107" H 2825 1550 50  0001 C CNN
+AR Path="/621F0CB4/622B9F05" Ref="#PWR0109"  Part="1"
+F 0 "#PWR0109" H 2825 1550 50  0001 C CNN
 F 1 "GND" H 2825 1650 50  0000 C CNN
 F 2 "" H 2825 1800 50  0001 C CNN
@@
 P 1925 4175
 AR Path="/622B9F0B" Ref="#PWR?"  Part="1"
-AR Path="/621F0CB4/622B9F0B" Ref="#PWR0114"  Part="1"
-F 0 "#PWR0114" H 1925 4025 50  0001 C CNN
+AR Path="/621F0CB4/622B9F0B" Ref="#PWR0116"  Part="1"
+F 0 "#PWR0116" H 1925 4025 50  0001 C CNN
 F 1 "+3V3" H 1925 4315 50  0000 C CNN
 F 2 "" H 1925 4175 50  0001 C CNN
@@
 P 2825 4725
 AR Path="/622B9F3C" Ref="#PWR?"  Part="1"
-AR Path="/621F0CB4/622B9F3C" Ref="#PWR0117"  Part="1"
-F 0 "#PWR0117" H 2825 4475 50  0001 C CNN
+AR Path="/621F0CB4/622B9F3C" Ref="#PWR0119"  Part="1"
+F 0 "#PWR0119" H 2825 4475 50  0001 C CNN
 F 1 "GND" H 2825 4575 50  0000 C CNN
 F 2 "" H 2825 4725 50  0001 C CNN
@@
 P 5075 1250
 AR Path="/622B9F42" Ref="#PWR?"  Part="1"
-AR Path="/621F0CB4/622B9F42" Ref="#PWR0106"  Part="1"
-F 0 "#PWR0106" H 5075 1100 50  0001 C CNN
+AR Path="/621F0CB4/622B9F42" Ref="#PWR0108"  Part="1"
+F 0 "#PWR0108" H 5075 1100 50  0001 C CNN
 F 1 "+3V3" H 5075 1390 50  0000 C CNN
 F 2 "" H 5075 1250 50  0001 C CNN
@@
 P 5975 1800
 AR Path="/622B9F73" Ref="#PWR?"  Part="1"
-AR Path="/621F0CB4/622B9F73" Ref="#PWR0108"  Part="1"
-F 0 "#PWR0108" H 5975 1550 50  0001 C CNN
+AR Path="/621F0CB4/622B9F73" Ref="#PWR0110"  Part="1"
+F 0 "#PWR0110" H 5975 1550 50  0001 C CNN
 F 1 "GND" H 5975 1650 50  0000 C CNN
 F 2 "" H 5975 1800 50  0001 C CNN
@@
 P 5075 4175
 AR Path="/622B9F79" Ref="#PWR?"  Part="1"
-AR Path="/621F0CB4/622B9F79" Ref="#PWR0115"  Part="1"
-F 0 "#PWR0115" H 5075 4025 50  0001 C CNN
+AR Path="/621F0CB4/622B9F79" Ref="#PWR0117"  Part="1"
+F 0 "#PWR0117" H 5075 4025 50  0001 C CNN
 F 1 "+3V3" H 5075 4315 50  0000 C CNN
 F 2 "" H 5075 4175 50  0001 C CNN
@@
 P 5975 4725
 AR Path="/622B9FAA" Ref="#PWR?"  Part="1"
-AR Path="/621F0CB4/622B9FAA" Ref="#PWR0118"  Part="1"
-F 0 "#PWR0118" H 5975 4475 50  0001 C CNN
+AR Path="/621F0CB4/622B9FAA" Ref="#PWR0120"  Part="1"
+F 0 "#PWR0120" H 5975 4475 50  0001 C CNN
 F 1 "GND" H 5975 4575 50  0000 C CNN
 F 2 "" H 5975 4725 50  0001 C CNN
@@
 P 5025 6025
 AR Path="/622B9D0C" Ref="#PWR?"  Part="1"
-AR Path="/621F0CB4/622B9D0C" Ref="#PWR0122"  Part="1"
-F 0 "#PWR0122" H 5025 5775 50  0001 C CNN
+AR Path="/621F0CB4/622B9D0C" Ref="#PWR0124"  Part="1"
+F 0 "#PWR0124" H 5025 5775 50  0001 C CNN
 F 1 "GND" H 5025 5875 50  0000 C CNN
 F 2 "" H 5025 6025 50  0001 C CNN
@@
 	7275 3775 7850 3775
 $Comp
-L custom:CRG0603F4K7 R79
+L custom:CRG0603F4K7 R87
 U 1 1 5D1EAA64
 P 7850 4325
-F 0 "R79" H 7920 4345 50  0000 L BNN
+F 0 "R87" H 7920 4345 50  0000 L BNN
 F 1 "CRG0603F4K7" H 7150 3925 50  0001 L BNN
 F 2 "Resistor_SMD:R_0603_1608Metric" H 7150 3825 50  0001 L BNN
@@
 $EndComp
 $Comp
-L custom:CRG0603F4K7 R80
+L custom:CRG0603F4K7 R88
 U 1 1 5D1EB3B5
 P 8250 4325
-F 0 "R80" H 8320 4345 50  0000 L BNN
+F 0 "R88" H 8320 4345 50  0000 L BNN
 F 1 "CRG0603F4K7" H 7550 3925 50  0001 L BNN
 F 2 "Resistor_SMD:R_0603_1608Metric" H 7550 3825 50  0001 L BNN
@@
 P 9450 4600
 AR Path="/5D2066B7" Ref="#PWR?"  Part="1"
-AR Path="/621F0CB4/5D2066B7" Ref="#PWR0116"  Part="1"
-F 0 "#PWR0116" H 9450 4350 50  0001 C CNN
+AR Path="/621F0CB4/5D2066B7" Ref="#PWR0118"  Part="1"
+F 0 "#PWR0118" H 9450 4350 50  0001 C CNN
 F 1 "GND" H 9450 4450 50  0000 C CNN
 F 2 "" H 9450 4600 50  0001 C CNN
@@
 	8600 4550 9050 4550
 $Comp
-L custom:CRG0603F4K7 R77
+L custom:CRG0603F4K7 R85
 U 1 1 5D2191D0
 P 8600 3175
-F 0 "R77" H 8670 3195 50  0000 L BNN
+F 0 "R85" H 8670 3195 50  0000 L BNN
 F 1 "CRG0603F4K7" H 7900 2775 50  0001 L BNN
 F 2 "Resistor_SMD:R_0603_1608Metric" H 7900 2675 50  0001 L BNN
@@
 	9050 3425 8600 3425
 $Comp
-L custom:CRG0603F4K7 R78
+L custom:CRG0603F4K7 R86
 U 1 1 5D22CE7A
 P 9450 4150
-F 0 "R78" H 9520 4170 50  0000 L BNN
+F 0 "R86" H 9520 4170 50  0000 L BNN
 F 1 "CRG0603F4K7" H 8750 3750 50  0001 L BNN
 F 2 "Resistor_SMD:R_0603_1608Metric" H 8750 3650 50  0001 L BNN
@@
 P 9450 2900
 AR Path="/5D242AE4" Ref="#PWR?"  Part="1"
-AR Path="/621F0CB4/5D242AE4" Ref="#PWR0111"  Part="1"
-F 0 "#PWR0111" H 9450 2750 50  0001 C CNN
+AR Path="/621F0CB4/5D242AE4" Ref="#PWR0113"  Part="1"
+F 0 "#PWR0113" H 9450 2750 50  0001 C CNN
 F 1 "+3V3" H 9450 3040 50  0000 C CNN
 F 2 "" H 9450 2900 50  0001 C CNN

Commit message: automated commit
Connections:
- net ROW00_OFF: now also U12.7 (Q7); no longer U10.15 (Q0)
- net ROW01_OFF: now also U10.15 (Q0); no longer U10.1 (Q1)
- net ROW01_ON: now also U11.7 (Q7); no longer U9.1 (Q1)
- net ROW02_OFF: now also U12.6 (Q6); no longer U10.2 (Q2)
- net ROW02_ON: now also U9.1 (Q1); no longer U9.2 (Q2)
- net ROW03_OFF: now also U10.1 (Q1); no longer U10.3 (Q3)
- net ROW03_ON: now also U11.6 (Q6); no longer U9.3 (Q3)
- net ROW04_OFF: now also U12.5 (Q5); no longer U10.4 (Q4)
- net ROW04_ON: now also U9.2 (Q2); no longer U9.4 (Q4)
- net ROW05_OFF: now also U10.2 (Q2); no longer U10.5 (Q5)
- net ROW05_ON: now also U11.5 (Q5); no longer U9.5 (Q5)
- net ROW06_OFF: now also U12.4 (Q4); no longer U10.6 (Q6)
- net ROW06_ON: now also U9.3 (Q3); no longer U9.6 (Q6)
- net ROW07_OFF: now also U10.3 (Q3); no longer U10.7 (Q7)
- net ROW07_ON: now also U11.4 (Q4); no longer U9.7 (Q7)
- net ROW08_OFF: now also U12.3 (Q3); no longer U12.15 (Q0)
- net ROW08_ON: now also U9.4 (Q4); no longer U11.15 (Q0)
- net ROW09_OFF: now also U10.4 (Q4); no longer U12.1 (Q1)
- net ROW09_ON: now also U11.3 (Q3); no longer U11.1 (Q1)
- net ROW10_ON: now also U9.5 (Q5); no longer U11.2 (Q2)
- net ROW11_OFF: now also U10.5 (Q5); no longer U12.3 (Q3)
- net ROW11_ON: now also U11.2 (Q2); no longer U11.3 (Q3)
- net ROW12_OFF: now also U12.1 (Q1); no longer U12.4 (Q4)
- net ROW12_ON: now also U9.6 (Q6); no longer U11.4 (Q4)
- net ROW13_OFF: now also U10.6 (Q6); no longer U12.5 (Q5)
- net ROW13_ON: now also U11.1 (Q1); no longer U11.5 (Q5)
- net ROW14_OFF: now also U12.15 (Q0); no longer U12.6 (Q6)
- net ROW14_ON: now also U9.7 (Q7); no longer U11.6 (Q6)
- net ROW15_OFF: now also U10.7 (Q7); no longer U12.7 (Q7)
- net ROW15_ON: now also U11.15 (Q0); no longer U11.7 (Q7)
Changed lines of the file:
@@
 	2925 5875 2825 5875
 Wire Wire Line
-	5975 2250 6075 2250
-Wire Wire Line
-	5975 2350 6075 2350
-Wire Wire Line
-	5975 2450 6075 2450
+	5975 5875 6075 5875
+Wire Wire Line
+	5975 5775 6075 5775
+Wire Wire Line
+	5975 5675 6075 5675
+Wire Wire Line
+	6075 5575 5975 5575
+Wire Wire Line
+	5975 5475 6075 5475
+Wire Wire Line
+	6075 5375 5975 5375
+Wire Wire Line
+	6075 5275 5975 5275
+Wire Wire Line
+	6075 5175 5975 5175
+Wire Wire Line
+	6075 2950 5975 2950
+Wire Wire Line
+	6075 2850 5975 2850
+Wire Wire Line
+	6075 2750 5975 2750
+Wire Wire Line
+	6075 2650 5975 2650
 Wire Wire Line
 	6075 2550 5975 2550
 Wire Wire Line
-	5975 2650 6075 2650
-Wire Wire Line
-	6075 2750 5975 2750
-Wire Wire Line
-	6075 2850 5975 2850
-Wire Wire Line
-	6075 2950 5975 2950
-Wire Wire Line
-	6075 5175 5975 5175
-Wire Wire Line
-	6075 5275 5975 5275
-Wire Wire Line
-	6075 5375 5975 5375
-Wire Wire Line
-	6075 5475 5975 5475
-Wire Wire Line
-	6075 5575 5975 5575
-Wire Wire Line
-	6075 5675 5975 5675
-Wire Wire Line
-	6075 5775 5975 5775
-Wire Wire Line
-	6075 5875 5975 5875
+	6075 2450 5975 2450
+Wire Wire Line
+	6075 2350 5975 2350
+Wire Wire Line
+	6075 2250 5975 2250
 $Comp
 L power:+3V3 #PWR?
@@
 Text GLabel 2925 2250 2    50   Output ~ 0
 ROW00_ON
-Text GLabel 2925 2350 2    50   Output ~ 0
-ROW01_ON
 Text GLabel 2925 2450 2    50   Output ~ 0
-ROW02_ON
+ROW04_ON
 Text GLabel 2925 2550 2    50   Output ~ 0
-ROW03_ON
+ROW06_ON
 Text GLabel 2925 2650 2    50   Output ~ 0
-ROW04_ON
+ROW08_ON
 Text GLabel 2925 2750 2    50   Output ~ 0
-ROW05_ON
+ROW10_ON
 Text GLabel 2925 2850 2    50   Output ~ 0
-ROW06_ON
+ROW12_ON
 Text GLabel 2925 2950 2    50   Output ~ 0
-ROW07_ON
-Text GLabel 2925 5175 2    50   Output ~ 0
-ROW08_ON
-Text GLabel 2925 5275 2    50   Output ~ 0
-ROW09_ON
-Text GLabel 2925 5375 2    50   Output ~ 0
-ROW10_ON
-Text GLabel 2925 5475 2    50   Output ~ 0
-ROW11_ON
-Text GLabel 2925 5575 2    50   Output ~ 0
-ROW12_ON
-Text GLabel 2925 5675 2    50   Output ~ 0
-ROW13_ON
-Text GLabel 2925 5775 2    50   Output ~ 0
 ROW14_ON
-Text GLabel 2925 5875 2    50   Output ~ 0
-ROW15_ON
-Text GLabel 6075 5175 2    50   Output ~ 0
+Text GLabel 6075 5475 2    50   Output ~ 0
 ROW08_OFF
-Text GLabel 6075 5275 2    50   Output ~ 0
+Text GLabel 6075 2650 2    50   Output ~ 0
 ROW09_OFF
 Text GLabel 6075 5375 2    50   Output ~ 0
 ROW10_OFF
-Text GLabel 6075 5475 2    50   Output ~ 0
+Text GLabel 6075 2750 2    50   Output ~ 0
 ROW11_OFF
+Text GLabel 6075 5275 2    50   Output ~ 0
+ROW12_OFF
+Text GLabel 6075 2850 2    50   Output ~ 0
+ROW13_OFF
+Text GLabel 6075 5175 2    50   Output ~ 0
+ROW14_OFF
+Text GLabel 6075 2950 2    50   Output ~ 0
+ROW15_OFF
+Text GLabel 6075 5875 2    50   Output ~ 0
+ROW00_OFF
+Text GLabel 6075 2250 2    50   Output ~ 0
+ROW01_OFF
+Text GLabel 6075 5775 2    50   Output ~ 0
+ROW02_OFF
+Text GLabel 6075 2350 2    50   Output ~ 0
+ROW03_OFF
+Text GLabel 6075 5675 2    50   Output ~ 0
+ROW04_OFF
+Text GLabel 6075 2450 2    50   Output ~ 0
+ROW05_OFF
 Text GLabel 6075 5575 2    50   Output ~ 0
-ROW12_OFF
-Text GLabel 6075 5675 2    50   Output ~ 0
-ROW13_OFF
-Text GLabel 6075 5775 2    50   Output ~ 0
-ROW14_OFF
-Text GLabel 6075 5875 2    50   Output ~ 0
-ROW15_OFF
-Text GLabel 6075 2250 2    50   Output ~ 0
-ROW00_OFF
-Text GLabel 6075 2350 2    50   Output ~ 0
-ROW01_OFF
-Text GLabel 6075 2450 2    50   Output ~ 0
-ROW02_OFF
+ROW06_OFF
 Text GLabel 6075 2550 2    50   Output ~ 0
-ROW03_OFF
-Text GLabel 6075 2650 2    50   Output ~ 0
-ROW04_OFF
-Text GLabel 6075 2750 2    50   Output ~ 0
-ROW05_OFF
-Text GLabel 6075 2850 2    50   Output ~ 0
-ROW06_OFF
-Text GLabel 6075 2950 2    50   Output ~ 0
 ROW07_OFF
 Wire Wire Line
@@
 Wire Wire Line
 	1825 2350 1925 2350
+Text GLabel 2925 5875 2    50   Output ~ 0
+ROW01_ON
+Text GLabel 2925 5775 2    50   Output ~ 0
+ROW03_ON
+Text GLabel 2925 5675 2    50   Output ~ 0
+ROW05_ON
+Text GLabel 2925 5575 2    50   Output ~ 0
+ROW07_ON
+Text GLabel 2925 5475 2    50   Output ~ 0
+ROW09_ON
+Text GLabel 2925 5375 2    50   Output ~ 0
+ROW11_ON
+Text GLabel 2925 5275 2    50   Output ~ 0
+ROW13_ON
+Text GLabel 2925 5175 2    50   Output ~ 0
+ROW15_ON
+Text GLabel 2925 2350 2    50   Output ~ 0
+ROW02_ON
 $EndSCHEMATC
