File: COLUMN_SHIFT_REGISTER.sch (KiCad schematic (older format))
At the start: 28 parts

Commit message: automated commit
Other:
- moved on the sheet: C?, U?

Commit message: automated commit
Parts:
- gave numbers to parts that had none: 28
Other:
- moved on the sheet: C64, C65, C66, C67, C68, C69, C70, C71, C72, C73, C74, C75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

Commit message: automated commit
Parts:
- renumbered U16 to U13, U17 to U14, U18 to U15, U19 to U16, U20 to U17, U21 to U18, U22 to U19

Commit message: automated commit
Parts:
- C66, C69, C72, C75, C78, C81, C84: value NP_C_0603 -> NP_0603
Changed lines of the file:
@@
-	1    0    0    -1
-$EndComp
-$Comp
-L custom:NP_C_0603 C?
-U 1 1 626060EE
-P 2450 1100
-AR Path="/626060EE" Ref="C?"  Part="1"
-AR Path="/621F0CB4/626060EE" Ref="C?"  Part="1"
-AR Path="/625CA44F/626060EE" Ref="C66"  Part="1"
-F 0 "C66" H 2565 1146 50  0000 L CNN
-F 1 "NP_C_0603" H 1500 650 50  0001 L BNN
-F 2 "Capacitor_SMD:C_0603_1608Metric" H 1500 550 50  0001 L BNN
-F 3 "" H 1500 450 50  0001 L BNN
-F 4 "NP" H 2565 1055 50  0000 L CNN "NP"
-	1    2450 1100
 	1    0    0    -1
 $EndComp
@@
 	1    0    0    -1
 $EndComp
-$Comp
-L custom:NP_C_0603 C?
-U 1 1 62606125
-P 2450 3500
-AR Path="/62606125" Ref="C?"  Part="1"
-AR Path="/621F0CB4/62606125" Ref="C?"  Part="1"
-AR Path="/625CA44F/62606125" Ref="C75"  Part="1"
-F 0 "C75" H 2565 3546 50  0000 L CNN
-F 1 "NP_C_0603" H 1500 3050 50  0001 L BNN
-F 2 "Capacitor_SMD:C_0603_1608Metric" H 1500 2950 50  0001 L BNN
-F 3 "" H 1500 2850 50  0001 L BNN
-F 4 "NP" H 2565 3455 50  0000 L CNN "NP"
-	1    2450 3500
-	1    0    0    -1
-$EndComp
 Wire Wire Line
 	2000 3650 2000 3700
@@
 	1    0    0    -1
 $EndComp
-$Comp
-L custom:NP_C_0603 C?
-U 1 1 6260615C
-P 2450 5900
-AR Path="/6260615C" Ref="C?"  Part="1"
-AR Path="/621F0CB4/6260615C" Ref="C?"  Part="1"
-AR Path="/625CA44F/6260615C" Ref="C81"  Part="1"
-F 0 "C81" H 2565 5946 50  0000 L CNN
-F 1 "NP_C_0603" H 1500 5450 50  0001 L BNN
-F 2 "Capacitor_SMD:C_0603_1608Metric" H 1500 5350 50  0001 L BNN
-F 3 "" H 1500 5250 50  0001 L BNN
-F 4 "NP" H 2565 5855 50  0000 L CNN "NP"
-	1    2450 5900
-	1    0    0    -1
-$EndComp
 Wire Wire Line
 	2000 6050 2000 6100
@@
 Wire Wire Line
 	7675 1250 7675 1300
-$Comp
-L custom:NP_C_0603 C?
-U 1 1 62606197
-P 8125 1100
-AR Path="/62606197" Ref="C?"  Part="1"
-AR Path="/621F0CB4/62606197" Ref="C?"  Part="1"
-AR Path="/625CA44F/62606197" Ref="C72"  Part="1"
-F 0 "C72" H 8240 1146 50  0000 L CNN
-F 1 "NP_C_0603" H 7175 650 50  0001 L BNN
-F 2 "Capacitor_SMD:C_0603_1608Metric" H 7175 550 50  0001 L BNN
-F 3 "" H 7175 450 50  0001 L BNN
-F 4 "NP" H 8240 1055 50  0000 L CNN "NP"
-	1    8125 1100
-	1    0    0    -1
-$EndComp
 $Comp
 L custom:CL10B104KO8NNNC C?
@@
 	4825 6050 4825 6100
 $Comp
-L custom:NP_C_0603 C?
-U 1 1 626061CE
-P 5275 5900
-AR Path="/626061CE" Ref="C?"  Part="1"
-AR Path="/621F0CB4/626061CE" Ref="C?"  Part="1"
-AR Path="/625CA44F/626061CE" Ref="C84"  Part="1"
-F 0 "C84" H 5390 5946 50  0000 L CNN
-F 1 "NP_C_0603" H 4325 5450 50  0001 L BNN
-F 2 "Capacitor_SMD:C_0603_1608Metric" H 4325 5350 50  0001 L BNN
-F 3 "" H 4325 5250 50  0001 L BNN
-F 4 "NP" H 5390 5855 50  0000 L CNN "NP"
-	1    5275 5900
-	1    0    0    -1
-$EndComp
-$Comp
 L custom:CL10B104KO8NNNC C?
 U 1 1 626061D6
@@
 	4825 3650 4825 3700
 $Comp
-L custom:NP_C_0603 C?
-U 1 1 62606205
-P 5275 3500
-AR Path="/62606205" Ref="C?"  Part="1"
-AR Path="/621F0CB4/62606205" Ref="C?"  Part="1"
-AR Path="/625CA44F/62606205" Ref="C78"  Part="1"
-F 0 "C78" H 5390 3546 50  0000 L CNN
-F 1 "NP_C_0603" H 4325 3050 50  0001 L BNN
-F 2 "Capacitor_SMD:C_0603_1608Metric" H 4325 2950 50  0001 L BNN
-F 3 "" H 4325 2850 50  0001 L BNN
-F 4 "NP" H 5390 3455 50  0000 L CNN "NP"
-	1    5275 3500
-	1    0    0    -1
-$EndComp
-$Comp
 L custom:CL10B104KO8NNNC C?
 U 1 1 6260620D
@@
 Wire Wire Line
 	4825 1250 4825 1300
-$Comp
-L custom:NP_C_0603 C?
-U 1 1 6260623C
-P 5275 1100
-AR Path="/6260623C" Ref="C?"  Part="1"
-AR Path="/621F0CB4/6260623C" Ref="C?"  Part="1"
-AR Path="/625CA44F/6260623C" Ref="C69"  Part="1"
-F 0 "C69" H 5390 1146 50  0000 L CNN
-F 1 "NP_C_0603" H 4325 650 50  0001 L BNN
-F 2 "Capacitor_SMD:C_0603_1608Metric" H 4325 550 50  0001 L BNN
-F 3 "" H 4325 450 50  0001 L BNN
-F 4 "NP" H 5390 1055 50  0000 L CNN "NP"
-	1    5275 1100
-	1    0    0    -1
-$EndComp
 $Comp
 L custom:CL10B104KO8NNNC C?
@@
 Text GLabel 1475 1900 0    50   Input ~ 0
 COL_IN
+$Comp
+L custom:NP_C_0603 C?
+U 1 1 5D061C7A
+P 2450 1100
+AR Path="/5D061C7A" Ref="C?"  Part="1"
+AR Path="/621F0CB4/5D061C7A" Ref="C?"  Part="1"
+AR Path="/625CA44F/5D061C7A" Ref="C66"  Part="1"
+F 0 "C66" H 2565 1146 50  0000 L CNN
+F 1 "NP_0603" H 2500 975 50  0000 L BNN
+F 2 "Capacitor_SMD:C_0603_1608Metric" H 1500 550 50  0001 L BNN
+F 3 "" H 1500 450 50  0001 L BNN
+F 4 "NP" H 2565 1055 50  0001 L CNN "NP"
+	1    2450 1100
+	1    0    0    -1
+$EndComp
+$Comp
+L custom:NP_C_0603 C?
+U 1 1 5D06EE2A
+P 5275 1100
+AR Path="/5D06EE2A" Ref="C?"  Part="1"
+AR Path="/621F0CB4/5D06EE2A" Ref="C?"  Part="1"
+AR Path="/625CA44F/5D06EE2A" Ref="C69"  Part="1"
+F 0 "C69" H 5390 1146 50  0000 L CNN
+F 1 "NP_0603" H 5325 975 50  0000 L BNN
+F 2 "Capacitor_SMD:C_0603_1608Metric" H 4325 550 50  0001 L BNN
+F 3 "" H 4325 450 50  0001 L BNN
+F 4 "NP" H 5390 1055 50  0001 L CNN "NP"
+	1    5275 1100
+	1    0    0    -1
+$EndComp
+$Comp
+L custom:NP_C_0603 C?
+U 1 1 5D07BF71
+P 8125 1100
+AR Path="/5D07BF71" Ref="C?"  Part="1"
+AR Path="/621F0CB4/5D07BF71" Ref="C?"  Part="1"
+AR Path="/625CA44F/5D07BF71" Ref="C72"  Part="1"
+F 0 "C72" H 8240 1146 50  0000 L CNN
+F 1 "NP_0603" H 8175 975 50  0000 L BNN
+F 2 "Capacitor_SMD:C_0603_1608Metric" H 7175 550 50  0001 L BNN
+F 3 "" H 7175 450 50  0001 L BNN
+F 4 "NP" H 8240 1055 50  0001 L CNN "NP"
+	1    8125 1100
+	1    0    0    -1
+$EndComp
+$Comp
+L custom:NP_C_0603 C?
+U 1 1 5D088D64
+P 5275 3500
+AR Path="/5D088D64" Ref="C?"  Part="1"
+AR Path="/621F0CB4/5D088D64" Ref="C?"  Part="1"
+AR Path="/625CA44F/5D088D64" Ref="C78"  Part="1"
+F 0 "C78" H 5390 3546 50  0000 L CNN
+F 1 "NP_0603" H 5325 3375 50  0000 L BNN
+F 2 "Capacitor_SMD:C_0603_1608Metric" H 4325 2950 50  0001 L BNN
+F 3 "" H 4325 2850 50  0001 L BNN
+F 4 "NP" H 5390 3455 50  0001 L CNN "NP"
+	1    5275 3500
+	1    0    0    -1
+$EndComp
+$Comp
+L custom:NP_C_0603 C?
+U 1 1 5D095C9B
+P 2450 3500
+AR Path="/5D095C9B" Ref="C?"  Part="1"
+AR Path="/621F0CB4/5D095C9B" Ref="C?"  Part="1"
+AR Path="/625CA44F/5D095C9B" Ref="C75"  Part="1"
+F 0 "C75" H 2565 3546 50  0000 L CNN
+F 1 "NP_0603" H 2500 3375 50  0000 L BNN
+F 2 "Capacitor_SMD:C_0603_1608Metric" H 1500 2950 50  0001 L BNN
+F 3 "" H 1500 2850 50  0001 L BNN
+F 4 "NP" H 2565 3455 50  0001 L CNN "NP"
+	1    2450 3500
+	1    0    0    -1
+$EndComp
+$Comp
+L custom:NP_C_0603 C?
+U 1 1 5D0A2AF4
+P 2450 5900
+AR Path="/5D0A2AF4" Ref="C?"  Part="1"
+AR Path="/621F0CB4/5D0A2AF4" Ref="C?"  Part="1"
+AR Path="/625CA44F/5D0A2AF4" Ref="C81"  Part="1"
+F 0 "C81" H 2565 5946 50  0000 L CNN
+F 1 "NP_0603" H 2500 5775 50  0000 L BNN
+F 2 "Capacitor_SMD:C_0603_1608Metric" H 1500 5350 50  0001 L BNN
+F 3 "" H 1500 5250 50  0001 L BNN
+F 4 "NP" H 2565 5855 50  0001 L CNN "NP"
+	1    2450 5900
+	1    0    0    -1
+$EndComp
+$Comp
+L custom:NP_C_0603 C?
+U 1 1 5D0AFB4B
+P 5275 5900
+AR Path="/5D0AFB4B" Ref="C?"  Part="1"
+AR Path="/621F0CB4/5D0AFB4B" Ref="C?"  Part="1"
+AR Path="/625CA44F/5D0AFB4B" Ref="C84"  Part="1"
+F 0 "C84" H 5390 5946 50  0000 L CNN
+F 1 "NP_0603" H 5325 5775 50  0000 L BNN
+F 2 "Capacitor_SMD:C_0603_1608Metric" H 4325 5350 50  0001 L BNN
+F 3 "" H 4325 5250 50  0001 L BNN
+F 4 "NP" H 5390 5855 50  0001 L CNN "NP"
+	1    5275 5900
+	1    0    0    -1
+$EndComp
 $EndSCHEMATC

Commit message: automated commit
Parts:
- added TP38, TP39, TP40, TP41, TP42, TP43: TestPoint, symbol Connector:TestPoint
- renumbered C64 to C65, C65 to C66, C66 to C67, C67 to C68, C68 to C69, C69 to C70, C70 to C71, C71 to C72, C72 to C73, C73 to C74, C74 to C75, C75 to C76, C76 to C77, C77 to C78, C78 to C79, C79 to C80, C80 to C81, C81 to C82, C82 to C83, C83 to C84, C84 to C85
Connections:
- net COL_SR_CHAIN_0: now also TP38.1
- net COL_SR_CHAIN_1: now also TP39.1
- net at U13.9 (Q7S), U16.14 (DS): now also TP40.1
- net at U16.9 (Q7S), U18.14 (DS): now also TP42.1
- net at U17.9 (Q7S), U19.14 (DS): now also TP43.1
- net at U14.9 (Q7S), U17.14 (DS): now also TP41.1

Commit message: automated commit
Parts:
- U13, U14, U15, U16, U17, U18, U19: footprint (none) -> Package_SO:SOIC-16_3.9x9.9mm_P1.27mm
Changed lines of the file:
@@
 F 0 "U13" H 1950 2600 60  0000 C CNN
 F 1 "74HC595" H 2000 1650 60  0000 C CNN
-F 2 "" H 1700 2200 60  0001 C CNN
+F 2 "Package_SO:SOIC-16_3.9x9.9mm_P1.27mm" H 1700 2200 60  0001 C CNN
 F 3 "~/datasheets/74HC_HCT595.pdf" H 1700 2200 60  0001 C CNN
 	1    2000 2150
@@
 F 0 "U16" H 1950 5000 60  0000 C CNN
 F 1 "74HC595" H 2000 4050 60  0000 C CNN
-F 2 "" H 1700 4600 60  0001 C CNN
+F 2 "Package_SO:SOIC-16_3.9x9.9mm_P1.27mm" H 1700 4600 60  0001 C CNN
 F 3 "" H 1700 4600 60  0001 C CNN
 	1    2000 4550
@@
 F 0 "U18" H 1950 7400 60  0000 C CNN
 F 1 "74HC595" H 2000 6450 60  0000 C CNN
-F 2 "" H 1700 7000 60  0001 C CNN
+F 2 "Package_SO:SOIC-16_3.9x9.9mm_P1.27mm" H 1700 7000 60  0001 C CNN
 F 3 "" H 1700 7000 60  0001 C CNN
 	1    2000 6950
@@
 F 0 "U15" H 7625 2600 60  0000 C CNN
 F 1 "74HC595" H 7675 1650 60  0000 C CNN
-F 2 "" H 7375 2200 60  0001 C CNN
+F 2 "Package_SO:SOIC-16_3.9x9.9mm_P1.27mm" H 7375 2200 60  0001 C CNN
 F 3 "" H 7375 2200 60  0001 C CNN
 	1    7675 2150
@@
 F 0 "U19" H 4775 7400 60  0000 C CNN
 F 1 "74HC595" H 4825 6450 60  0000 C CNN
-F 2 "" H 4525 7000 60  0001 C CNN
+F 2 "Package_SO:SOIC-16_3.9x9.9mm_P1.27mm" H 4525 7000 60  0001 C CNN
 F 3 "" H 4525 7000 60  0001 C CNN
 	1    4825 6950
@@
 F 0 "U17" H 4775 5000 60  0000 C CNN
 F 1 "74HC595" H 4825 4050 60  0000 C CNN
-F 2 "" H 4525 4600 60  0001 C CNN
+F 2 "Package_SO:SOIC-16_3.9x9.9mm_P1.27mm" H 4525 4600 60  0001 C CNN
 F 3 "" H 4525 4600 60  0001 C CNN
 	1    4825 4550
@@
 F 0 "U14" H 4775 2600 60  0000 C CNN
 F 1 "74HC595" H 4825 1650 60  0000 C CNN
-F 2 "" H 4525 2200 60  0001 C CNN
+F 2 "Package_SO:SOIC-16_3.9x9.9mm_P1.27mm" H 4525 2200 60  0001 C CNN
 F 3 "" H 4525 2200 60  0001 C CNN
 	1    4825 2150

Commit message: automated commit
Parts:
- TP43: renamed from TP38; footprint (none) -> custom:TestPoint_THTPad_D1.0mm_Drill0.5mm
- TP44: renamed from TP39; footprint (none) -> custom:TestPoint_THTPad_D1.0mm_Drill0.5mm
- TP45: renamed from TP40; footprint (none) -> custom:TestPoint_THTPad_D1.0mm_Drill0.5mm
- TP46: renamed from TP41; footprint (none) -> custom:TestPoint_THTPad_D1.0mm_Drill0.5mm
- TP47: renamed from TP42; footprint (none) -> custom:TestPoint_THTPad_D1.0mm_Drill0.5mm
- TP48: renamed from TP43; footprint (none) -> custom:TestPoint_THTPad_D1.0mm_Drill0.5mm
Changed lines of the file:
@@
 AR Path="/61C6D021/5D749936" Ref="TP?"  Part="1"
 AR Path="/609E0ED6/5D749936" Ref="TP?"  Part="1"
-AR Path="/625CA44F/5D749936" Ref="TP40"  Part="1"
-F 0 "TP40" V 1175 3175 50  0000 C CNN
+AR Path="/625CA44F/5D749936" Ref="TP45"  Part="1"
+F 0 "TP45" V 1175 3175 50  0000 C CNN
 F 1 "TestPoint" H 850 3025 50  0001 C CNN
-F 2 "" H 1300 2975 50  0001 C CNN
+F 2 "custom:TestPoint_THTPad_D1.0mm_Drill0.5mm" H 1300 2975 50  0001 C CNN
 F 3 "~" H 1300 2975 50  0001 C CNN
 	1    1100 2975
@@
 AR Path="/61C6D021/5D77DC3E" Ref="TP?"  Part="1"
 AR Path="/609E0ED6/5D77DC3E" Ref="TP?"  Part="1"
-AR Path="/625CA44F/5D77DC3E" Ref="TP42"  Part="1"
-F 0 "TP42" V 1175 5575 50  0000 C CNN
+AR Path="/625CA44F/5D77DC3E" Ref="TP47"  Part="1"
+F 0 "TP47" V 1175 5575 50  0000 C CNN
 F 1 "TestPoint" H 850 5425 50  0001 C CNN
-F 2 "" H 1300 5375 50  0001 C CNN
+F 2 "custom:TestPoint_THTPad_D1.0mm_Drill0.5mm" H 1300 5375 50  0001 C CNN
 F 3 "~" H 1300 5375 50  0001 C CNN
 	1    1100 5375
@@
 AR Path="/61C6D021/5D78B104" Ref="TP?"  Part="1"
 AR Path="/609E0ED6/5D78B104" Ref="TP?"  Part="1"
-AR Path="/625CA44F/5D78B104" Ref="TP43"  Part="1"
-F 0 "TP43" V 4000 5575 50  0000 C CNN
+AR Path="/625CA44F/5D78B104" Ref="TP48"  Part="1"
+F 0 "TP48" V 4000 5575 50  0000 C CNN
 F 1 "TestPoint" H 3675 5425 50  0001 C CNN
-F 2 "" H 4125 5375 50  0001 C CNN
+F 2 "custom:TestPoint_THTPad_D1.0mm_Drill0.5mm" H 4125 5375 50  0001 C CNN
 F 3 "~" H 4125 5375 50  0001 C CNN
 	1    3925 5375
@@
 AR Path="/61C6D021/5D798E78" Ref="TP?"  Part="1"
 AR Path="/609E0ED6/5D798E78" Ref="TP?"  Part="1"
-AR Path="/625CA44F/5D798E78" Ref="TP41"  Part="1"
-F 0 "TP41" V 4000 3175 50  0000 C CNN
+AR Path="/625CA44F/5D798E78" Ref="TP46"  Part="1"
+F 0 "TP46" V 4000 3175 50  0000 C CNN
 F 1 "TestPoint" H 3675 3025 50  0001 C CNN
-F 2 "" H 4125 2975 50  0001 C CNN
+F 2 "custom:TestPoint_THTPad_D1.0mm_Drill0.5mm" H 4125 2975 50  0001 C CNN
 F 3 "~" H 4125 2975 50  0001 C CNN
 	1    3925 2975
@@
 AR Path="/61C6D021/5D7A81F4" Ref="TP?"  Part="1"
 AR Path="/609E0ED6/5D7A81F4" Ref="TP?"  Part="1"
-AR Path="/625CA44F/5D7A81F4" Ref="TP38"  Part="1"
-F 0 "TP38" V 3575 2100 50  0000 C CNN
+AR Path="/625CA44F/5D7A81F4" Ref="TP43"  Part="1"
+F 0 "TP43" V 3575 2100 50  0000 C CNN
 F 1 "TestPoint" H 3250 1950 50  0001 C CNN
-F 2 "" H 3700 1900 50  0001 C CNN
+F 2 "custom:TestPoint_THTPad_D1.0mm_Drill0.5mm" H 3700 1900 50  0001 C CNN
 F 3 "~" H 3700 1900 50  0001 C CNN
 	1    3500 1900
@@
 AR Path="/61C6D021/5D7C4799" Ref="TP?"  Part="1"
 AR Path="/609E0ED6/5D7C4799" Ref="TP?"  Part="1"
-AR Path="/625CA44F/5D7C4799" Ref="TP39"  Part="1"
-F 0 "TP39" V 6425 2100 50  0000 C CNN
+AR Path="/625CA44F/5D7C4799" Ref="TP44"  Part="1"
+F 0 "TP44" V 6425 2100 50  0000 C CNN
 F 1 "TestPoint" H 6100 1950 50  0001 C CNN
-F 2 "" H 6550 1900 50  0001 C CNN
+F 2 "custom:TestPoint_THTPad_D1.0mm_Drill0.5mm" H 6550 1900 50  0001 C CNN
 F 3 "~" H 6550 1900 50  0001 C CNN
 	1    6350 1900
