File: flipdot_driver.kicad_pcb (KiCad board)
At the start: 4 copper layers, 662 parts, among them J1 Barrel_Jack, J10 Conn_01x08_Male, J11 3x32_1&3_loaded_2.5mm_0.1in_f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, J2 Screw_Terminal_01x04, J3 PTH_1.5_mm, J4 PTH_1.5_mm, J5 PTH_1.5_mm, J6 PTH_1.5_mm, J7 Conn_01x05_Male, J8 PTH_1.5_mm, J9 USB-C_2.0_Connector, Q1 SSM3K35AMFV, Q10 SSM3K35AMFV, Q100 SSM3K35AMFV, Q101 SSM3K35AMFV, Q102 SSM3K35AMFV, Q103 DMG6602, Q104 DMG6602, Q105 DMG6602, Q106 SSM3K35AMFV, Q107 SSM3K35AMFV, Q108 SSM3K35AMFV, Q109 SSM3K35AMFV, Q11 SSM3K35AMFV, Q110 SSM3K35AMFV, Q111 SSM3K35AMFV, Q112 DMG6602, Q113 DMG6602, Q114 DMG6602, Q115 SSM3K35AMFV, Q116 SSM3K35AMFV, Q117 SSM3K35AMFV, Q118 SSM3K35AMFV, Q119 SSM3K35AMFV, Q12 AO3407A, Q120 SSM3K35AMFV, Q121 DMG6602, Q122 DMG6602, Q123 DMG6602, Q124 SSM3K35AMFV, Q125 SSM3K35AMFV, Q126 SSM3K35AMFV, Q127 SSM3K35AMFV, Q128 SSM3K35AMFV, Q129 SSM3K35AMFV, Q13 SSM3K35AMFV, Q130 DMG6602, Q131 SSM3K35AMFV, Q132 SSM3K35AMFV, Q14 SSM3K35AMFV, Q15 DMG6602, Q16 DMG6602, Q17 DMG6602, Q18 SSM3K35AMFV, Q19 SSM3K35AMFV, Q2 SSM3K35AMFV, Q20 SSM3K35AMFV, Q21 DMG6602, Q22 DMG6602, Q23 SSM3K35AMFV, Q24 SSM3K35AMFV, Q25 DMG6602, Q26 DMG6602, Q27 SSM3K35AMFV, Q28 SSM3K35AMFV, Q29 DMG6602, Q3 SSM3K35AMFV, Q30 DMG6602, Q31 SSM3K35AMFV, Q32 SSM3K35AMFV, Q33 DMG6602, Q34 DMG6602, Q35 SSM3K35AMFV, Q36 SSM3K35AMFV, Q37 DMG6602, Q38 DMG6602, Q39 SSM3K35AMFV, Q4 SSM3K35AMFV, Q40 SSM3K35AMFV, Q41 DMG6602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

Commit message: automated commit
Parts:
- removed Q58: DMG6602, Package_TO_SOT_SMD:TSOT-23-6
- removed Q61, Q64: SSM3K35AMFV, Package_TO_SOT_SMD:SOT-723
- removed R155, R158, R161, R162: CRG0603F4K7, Resistor_SMD:R_0603_1608Metric
- added Q0: SSM3K35AMFV, Package_TO_SOT_SMD:SOT-723, F.Cu at (94.2, -7.10)
- added Q0: DMG6602, Package_TO_SOT_SMD:TSOT-23-6, F.Cu at (82.8, -7.35)
- added Q0: DMG6602, Package_TO_SOT_SMD:TSOT-23-6, B.Cu at (105.6, -10.1)
- added Q0: DMG6602, Package_TO_SOT_SMD:TSOT-23-6, F.Cu at (108.5, -7.35)
- added Q0: SSM3K35AMFV, Package_TO_SOT_SMD:SOT-723, F.Cu at (94.0, -9.00)
- added Q0: DMG6602, Package_TO_SOT_SMD:TSOT-23-6, B.Cu at (88.5, -10.1)
- added Q0: SSM3K35AMFV, Package_TO_SOT_SMD:SOT-723, B.Cu at (85.7, -9.80)
- added Q0: SSM3K35AMFV, Package_TO_SOT_SMD:SOT-723, B.Cu at (94.3, -11.7)
- added Q0: SSM3K35AMFV, Package_TO_SOT_SMD:SOT-723, B.Cu at (68.6, -9.80)
- added Q0: SSM3K35AMFV, Package_TO_SOT_SMD:SOT-723, B.Cu at (77.2, -9.80)
- added Q0: SSM3K35AMFV, Package_TO_SOT_SMD:SOT-723, F.Cu at (77.0, -9.00)
- added Q0: SSM3K35AMFV, Package_TO_SOT_SMD:SOT-723, B.Cu at (60.1, -11.7)
- added Q0: SSM3K35AMFV, Package_TO_SOT_SMD:SOT-723, B.Cu at (111.3, -9.80)
- added Q0: SSM3K35AMFV, Package_TO_SOT_SMD:SOT-723, B.Cu at (68.7, -11.7)
- added Q0: SSM3K35AMFV, Package_TO_SOT_SMD:SOT-723, B.Cu at (94.2, -9.80)
- added Q0: SSM3K35AMFV, Package_TO_SOT_SMD:SOT-723, F.Cu at (119.7, -9.00)
- added Q0: SSM3K35AMFV, Package_TO_SOT_SMD:SOT-723, F.Cu at (85.5, -9.00)
- added Q0: DMG6602, Package_TO_SOT_SMD:TSOT-23-6, F.Cu at (99.9, -7.35)
- added Q0: SSM3K35AMFV, Package_TO_SOT_SMD:SOT-723, B.Cu at (111.5, -11.7)
- added Q0: SSM3K35AMFV, Package_TO_SOT_SMD:SOT-723, F.Cu at (68.5, -7.10)
- added Q0: DMG6602, Package_TO_SOT_SMD:TSOT-23-6, F.Cu at (74.2, -7.35)
- added Q0: DMG6602, Package_TO_SOT_SMD:TSOT-23-6, B.Cu at (80.0, -10.1)
- added Q0: DMG6602, Package_TO_SOT_SMD:TSOT-23-6, B.Cu at (71.4, -10.1)
- added Q0: SSM3K35AMFV, Package_TO_SOT_SMD:SOT-723, F.Cu at (68.4, -9.00)
- added Q0: SSM3K35AMFV, Package_TO_SOT_SMD:SOT-723, F.Cu at (111.2, -7.10)
- added Q0: SSM3K35AMFV, Package_TO_SOT_SMD:SOT-723, F.Cu at (85.6, -7.10)
- added Q0: SSM3K35AMFV, Package_TO_SOT_SMD:SOT-723, B.Cu at (60.0, -9.80)
- added Q0: SSM3K35AMFV, Package_TO_SOT_SMD:SOT-723, F.Cu at (119.8, -7.10)
- added Q0: SSM3K35AMFV, Package_TO_SOT_SMD:SOT-723, F.Cu at (77.0, -7.10)
- added Q0: DMG6602, Package_TO_SOT_SMD:TSOT-23-6, F.Cu at (91.3, -7.35)
- added Q0: DMG6602, Package_TO_SOT_SMD:TSOT-23-6, B.Cu at (114.2, -10.1)
- added Q0: DMG6602, Package_TO_SOT_SMD:TSOT-23-6, B.Cu at (62.9, -10.1)
- added Q0: DMG6602, Package_TO_SOT_SMD:TSOT-23-6, F.Cu at (65.7, -7.35)
- added Q0: SSM3K35AMFV, Package_TO_SOT_SMD:SOT-723, B.Cu at (85.8, -11.7)
- added Q0: SSM3K35AMFV, Package_TO_SOT_SMD:SOT-723, F.Cu at (111.2, -9.00)
- added Q0: SSM3K35AMFV, Package_TO_SOT_SMD:SOT-723, F.Cu at (102.7, -7.10)
- added Q0: DMG6602, Package_TO_SOT_SMD:TSOT-23-6, F.Cu at (117.0, -7.35)
- added Q0: SSM3K35AMFV, Package_TO_SOT_SMD:SOT-723, B.Cu at (94.2, 32.1)
- added Q0: SSM3K35AMFV, Package_TO_SOT_SMD:SOT-723, B.Cu at (102.6, 34.0)
- added Q0: DMG6602, Package_TO_SOT_SMD:TSOT-23-6, B.Cu at (82.8, 32.4)
- added Q0: DMG6602, Package_TO_SOT_SMD:TSOT-23-6, B.Cu at (108.5, 32.4)
- added Q0: SSM3K35AMFV, Package_TO_SOT_SMD:SOT-723, B.Cu at (94.0, 34.0)
- added Q0: SSM3K35AMFV, Package_TO_SOT_SMD:SOT-723, B.Cu at (77.0, 34.0)
- added Q0: SSM3K35AMFV, Package_TO_SOT_SMD:SOT-723, B.Cu at (119.7, 34.0)
- added Q0: SSM3K35AMFV, Package_TO_SOT_SMD:SOT-723, F.Cu at (102.6, -9.00)
- added Q0: SSM3K35AMFV, Package_TO_SOT_SMD:SOT-723, B.Cu at (85.5, 34.0)
- added Q0: DMG6602, Package_TO_SOT_SMD:TSOT-23-6, B.Cu at (99.9, 32.4)
- added Q0: SSM3K35AMFV, Package_TO_SOT_SMD:SOT-723, B.Cu at (68.5, 32.1)
- added Q0: DMG6602, Package_TO_SOT_SMD:TSOT-23-6, B.Cu at (74.2, 32.4)
- added Q0: SSM3K35AMFV, Package_TO_SOT_SMD:SOT-723, B.Cu at (68.4, 34.0)
- added Q0: SSM3K35AMFV, Package_TO_SOT_SMD:SOT-723, B.Cu at (111.2, 32.1)
- added Q0: SSM3K35AMFV, Package_TO_SOT_SMD:SOT-723, B.Cu at (85.6, 32.1)
- added Q0: SSM3K35AMFV, Package_TO_SOT_SMD:SOT-723, B.Cu at (119.8, 32.1)
- added Q0: SSM3K35AMFV, Package_TO_SOT_SMD:SOT-723, B.Cu at (77.0, 32.1)
- added Q0: DMG6602, Package_TO_SOT_SMD:TSOT-23-6, B.Cu at (91.3, 32.4)
- added Q0: SSM3K35AMFV, Package_TO_SOT_SMD:SOT-723, B.Cu at (102.9, -11.7)
- added Q0: DMG6602, Package_TO_SOT_SMD:TSOT-23-6, B.Cu at (65.7, 32.4)
- added Q0: SSM3K35AMFV, Package_TO_SOT_SMD:SOT-723, B.Cu at (111.2, 34.0)
- added Q0: SSM3K35AMFV, Package_TO_SOT_SMD:SOT-723, B.Cu at (102.7, 32.1)
- added Q0: DMG6602, Package_TO_SOT_SMD:TSOT-23-6, B.Cu at (117.0, 32.4)
- added Q0: SSM3K35AMFV, Package_TO_SOT_SMD:SOT-723, F.Cu at (111.5, 31.4)
- added Q0: DMG6602, Package_TO_SOT_SMD:TSOT-23-6, F.Cu at (105.6, 29.7)
- added Q0: SSM3K35AMFV, Package_TO_SOT_SMD:SOT-723, F.Cu at (94.3, 31.4)
- added Q0: DMG6602, Package_TO_SOT_SMD:TSOT-23-6, F.Cu at (114.2, 29.7)
- added Q0: SSM3K35AMFV, Package_TO_SOT_SMD:SOT-723, F.Cu at (102.8, 29.4)
- added Q0: SSM3K35AMFV, Package_TO_SOT_SMD:SOT-723, F.Cu at (94.2, 29.4)
- added Q0: SSM3K35AMFV, Package_TO_SOT_SMD:SOT-723, B.Cu at (77.2, -11.7)
- added Q0: SSM3K35AMFV, Package_TO_SOT_SMD:SOT-723, F.Cu at (102.9, 31.4)
- added Q0: SSM3K35AMFV, Package_TO_SOT_SMD:SOT-723, F.Cu at (111.3, 29.4)
- added Q0: DMG6602, Package_TO_SOT_SMD:TSOT-23-6, F.Cu at (97.0, 29.7)
- added Q0: DMG6602, Package_TO_SOT_SMD:TSOT-23-6, F.Cu at (88.5, 29.7)
- added Q0: SSM3K35AMFV, Package_TO_SOT_SMD:SOT-723, F.Cu at (77.2, 31.4)
- added Q0: SSM3K35AMFV, Package_TO_SOT_SMD:SOT-723, F.Cu at (85.7, 29.4)
- added Q0: SSM3K35AMFV, Package_TO_SOT_SMD:SOT-723, F.Cu at (77.2, 29.4)
- added Q0: SSM3K35AMFV, Package_TO_SOT_SMD:SOT-723, F.Cu at (85.8, 31.4)
- added Q0: DMG6602, Package_TO_SOT_SMD:TSOT-23-6, F.Cu at (80.0, 29.7)
- added Q0: SSM3K35AMFV, Package_TO_SOT_SMD:SOT-723, F.Cu at (68.7, 31.4)
- added Q0: DMG6602, Package_TO_SOT_SMD:TSOT-23-6, B.Cu at (97.0, -10.1)
- added Q0: SSM3K35AMFV, Package_TO_SOT_SMD:SOT-723, F.Cu at (68.6, 29.4)
- added Q0: DMG6602, Package_TO_SOT_SMD:TSOT-23-6, F.Cu at (71.4, 29.7)
- added Q0: DMG6602, Package_TO_SOT_SMD:TSOT-23-6, F.Cu at (62.9, 29.7)
- added Q0: SSM3K35AMFV, Package_TO_SOT_SMD:SOT-723, F.Cu at (60.1, 31.4)
- added Q0: SSM3K35AMFV, Package_TO_SOT_SMD:SOT-723, F.Cu at (60.0, 29.4)
- added Q0: SSM3K35AMFV, Package_TO_SOT_SMD:SOT-723, B.Cu at (102.8, -9.80)
- added R0: CRG0603F4K7, Resistor_SMD:R_0603_1608Metric, F.Cu at (100.9, -11.1)
- added R0: CRG0603F4K7, Resistor_SMD:R_0603_1608Metric, B.Cu at (101.1, -11.6)
- added R0: CRG0603F4K7, Resistor_SMD:R_0603_1608Metric, F.Cu at (82.5, 32.0)
- added R0: CRG0603F4K7, Resistor_SMD:R_0603_1608Metric, F.Cu at (75.5, 31.2)
- added R0: CRG0603F4K7, Resistor_SMD:R_0603_1608Metric, F.Cu at (84.0, 31.2)
- added R0: CRG0603F4K7, Resistor_SMD:R_0603_1608Metric, F.Cu at (77.3, 33.9)
- added R0: CRG0603F4K7, Resistor_SMD:R_0603_1608Metric, F.Cu at (87.5, 33.5)
- added R0: CRG0603F4K7, Resistor_SMD:R_0603_1608Metric, F.Cu at (70.4, 33.5)
- added R0: CRG0603F4K7, Resistor_SMD:R_0603_1608Metric, F.Cu at (73.9, 32.0)
- added R0: CRG0603F4K7, Resistor_SMD:R_0603_1608Metric, F.Cu at (66.9, 31.2)
- added R0: CRG0603F4K7, Resistor_SMD:R_0603_1608Metric, F.Cu at (68.8, 33.9)
- added R0: CRG0603F4K7, Resistor_SMD:R_0603_1608Metric, F.Cu at (58.4, 31.2)
- added R0: CRG0603F4K7, Resistor_SMD:R_0603_1608Metric, B.Cu at (85.9, -14.2)
- added R0: CRG0603F4K7, Resistor_SMD:R_0603_1608Metric, F.Cu at (60.2, 33.9)
- added R0: CRG0603F4K7, Resistor_SMD:R_0603_1608Metric, F.Cu at (65.3, 32.0)
- added R0: CRG0603F4K7, Resistor_SMD:R_0603_1608Metric, F.Cu at (61.9, 33.5)
- added R0: CRG0603F4K7, Resistor_SMD:R_0603_1608Metric, B.Cu at (77.3, -14.2)
- added R0: CRG0603F4K7, Resistor_SMD:R_0603_1608Metric, B.Cu at (94.5, -14.2)
- added R0: CRG0603F4K7, Resistor_SMD:R_0603_1608Metric, F.Cu at (102.5, -11.5)
- added R0: CRG0603F4K7, Resistor_SMD:R_0603_1608Metric, B.Cu at (113.2, -13.8)
- added R0: CRG0603F4K7, Resistor_SMD:R_0603_1608Metric, B.Cu at (109.7, -11.6)
- added R0: CRG0603F4K7, Resistor_SMD:R_0603_1608Metric, F.Cu at (85.4, -11.5)
- added R0: CRG0603F4K7, Resistor_SMD:R_0603_1608Metric, F.Cu at (76.8, -11.5)
- added R0: CRG0603F4K7, Resistor_SMD:R_0603_1608Metric, B.Cu at (66.9, -11.6)
- added R0: CRG0603F4K7, Resistor_SMD:R_0603_1608Metric, F.Cu at (78.8, -8.90)
- added R0: CRG0603F4K7, Resistor_SMD:R_0603_1608Metric, B.Cu at (99.5, -12.3)
- added R0: CRG0603F4K7, Resistor_SMD:R_0603_1608Metric, B.Cu at (84.0, -11.6)
- added R0: CRG0603F4K7, Resistor_SMD:R_0603_1608Metric, B.Cu at (79.0, -13.8)
- added R0: CRG0603F4K7, Resistor_SMD:R_0603_1608Metric, B.Cu at (73.9, -12.3)
- added R0: CRG0603F4K7, Resistor_SMD:R_0603_1608Metric, F.Cu at (80.3, -9.65)
- added R0: CRG0603F4K7, Resistor_SMD:R_0603_1608Metric, F.Cu at (95.8, -8.90)
- added R0: CRG0603F4K7, Resistor_SMD:R_0603_1608Metric, B.Cu at (87.5, -13.8)
- added R0: CRG0603F4K7, Resistor_SMD:R_0603_1608Metric, F.Cu at (75.2, -11.1)
- added R0: CRG0603F4K7, Resistor_SMD:R_0603_1608Metric, B.Cu at (96.0, -13.8)
- added R0: CRG0603F4K7, Resistor_SMD:R_0603_1608Metric, B.Cu at (92.5, -11.6)
- added R0: CRG0603F4K7, Resistor_SMD:R_0603_1608Metric, B.Cu at (111.5, -14.2)
- added R0: CRG0603F4K7, Resistor_SMD:R_0603_1608Metric, B.Cu at (91.0, -12.3)
- added R0: CRG0603F4K7, Resistor_SMD:R_0603_1608Metric, F.Cu at (118.0, -11.1)
- added R0: CRG0603F4K7, Resistor_SMD:R_0603_1608Metric, F.Cu at (111.0, -11.5)
- added R0: CRG0603F4K7, Resistor_SMD:R_0603_1608Metric, F.Cu at (68.3, -11.5)
- added R0: CRG0603F4K7, Resistor_SMD:R_0603_1608Metric, F.Cu at (66.7, -11.1)
- added R0: CRG0603F4K7, Resistor_SMD:R_0603_1608Metric, F.Cu at (70.2, -8.90)
- added R0: CRG0603F4K7, Resistor_SMD:R_0603_1608Metric, F.Cu at (106.0, -9.65)
- added R0: CRG0603F4K7, Resistor_SMD:R_0603_1608Metric, F.Cu at (92.3, -11.1)
- added R0: CRG0603F4K7, Resistor_SMD:R_0603_1608Metric, B.Cu at (116.7, -12.3)
- added R0: CRG0603F4K7, Resistor_SMD:R_0603_1608Metric, B.Cu at (70.4, -13.8)
- added R0: CRG0603F4K7, Resistor_SMD:R_0603_1608Metric, F.Cu at (94.0, -11.5)
- added R0: CRG0603F4K7, Resistor_SMD:R_0603_1608Metric, F.Cu at (114.5, -9.65)
- added R0: CRG0603F4K7, Resistor_SMD:R_0603_1608Metric, F.Cu at (121.5, -8.90)
- added R0: CRG0603F4K7, Resistor_SMD:R_0603_1608Metric, B.Cu at (82.5, -12.3)
- added R0: CRG0603F4K7, Resistor_SMD:R_0603_1608Metric, B.Cu at (58.4, -11.6)
- added R0: CRG0603F4K7, Resistor_SMD:R_0603_1608Metric, B.Cu at (108.1, -12.3)
- added R0: CRG0603F4K7, Resistor_SMD:R_0603_1608Metric, F.Cu at (71.8, -9.65)
- added R0: CRG0603F4K7, Resistor_SMD:R_0603_1608Metric, F.Cu at (113.0, -8.90)
- added R0: CRG0603F4K7, Resistor_SMD:R_0603_1608Metric, F.Cu at (87.3, -8.90)
- added R0: CRG0603F4K7, Resistor_SMD:R_0603_1608Metric, F.Cu at (97.4, -9.65)
- added R0: CRG0603F4K7, Resistor_SMD:R_0603_1608Metric, B.Cu at (75.5, -11.6)
- added R0: CRG0603F4K7, Resistor_SMD:R_0603_1608Metric, B.Cu at (103.0, -14.2)
- added R0: CRG0603F4K7, Resistor_SMD:R_0603_1608Metric, F.Cu at (83.8, -11.1)
- added R0: CRG0603F4K7, Resistor_SMD:R_0603_1608Metric, F.Cu at (63.2, -9.65)
- added R0: CRG0603F4K7, Resistor_SMD:R_0603_1608Metric, F.Cu at (88.8, -9.65)
- added R0: CRG0603F4K7, Resistor_SMD:R_0603_1608Metric, F.Cu at (104.4, -8.90)
- added R0: CRG0603F4K7, Resistor_SMD:R_0603_1608Metric, F.Cu at (119.6, -11.5)
- added R0: CRG0603F4K7, Resistor_SMD:R_0603_1608Metric, F.Cu at (109.5, -11.1)
- added R0: CRG0603F4K7, Resistor_SMD:R_0603_1608Metric, B.Cu at (65.3, -12.3)
- added R0: CRG0603F4K7, Resistor_SMD:R_0603_1608Metric, B.Cu at (100.9, 36.1)
- added R0: CRG0603F4K7, Resistor_SMD:R_0603_1608Metric, B.Cu at (78.8, 34.0)
- added R0: CRG0603F4K7, Resistor_SMD:R_0603_1608Metric, B.Cu at (94.0, 36.5)
- added R0: CRG0603F4K7, Resistor_SMD:R_0603_1608Metric, B.Cu at (60.2, -14.2)
- added R0: CRG0603F4K7, Resistor_SMD:R_0603_1608Metric, B.Cu at (102.5, 36.5)
- added R0: CRG0603F4K7, Resistor_SMD:R_0603_1608Metric, B.Cu at (85.4, 36.5)
- added R0: CRG0603F4K7, Resistor_SMD:R_0603_1608Metric, B.Cu at (76.8, 36.5)
- added R0: CRG0603F4K7, Resistor_SMD:R_0603_1608Metric, B.Cu at (80.3, 34.7)
- added R0: CRG0603F4K7, Resistor_SMD:R_0603_1608Metric, B.Cu at (95.8, 34.0)
- added R0: CRG0603F4K7, Resistor_SMD:R_0603_1608Metric, B.Cu at (75.2, 36.1)
- added R0: CRG0603F4K7, Resistor_SMD:R_0603_1608Metric, B.Cu at (118.0, 36.1)
- added R0: CRG0603F4K7, Resistor_SMD:R_0603_1608Metric, B.Cu at (111.0, 36.5)
- added R0: CRG0603F4K7, Resistor_SMD:R_0603_1608Metric, B.Cu at (68.3, 36.5)
- added R0: CRG0603F4K7, Resistor_SMD:R_0603_1608Metric, B.Cu at (66.7, 36.1)
- added R0: CRG0603F4K7, Resistor_SMD:R_0603_1608Metric, B.Cu at (104.6, -13.8)
- added R0: CRG0603F4K7, Resistor_SMD:R_0603_1608Metric, B.Cu at (70.2, 34.0)
- added R0: CRG0603F4K7, Resistor_SMD:R_0603_1608Metric, B.Cu at (106.0, 34.7)
- added R0: CRG0603F4K7, Resistor_SMD:R_0603_1608Metric, B.Cu at (92.3, 36.1)
- added R0: CRG0603F4K7, Resistor_SMD:R_0603_1608Metric, B.Cu at (114.5, 34.7)
- added R0: CRG0603F4K7, Resistor_SMD:R_0603_1608Metric, B.Cu at (121.5, 34.0)
- added R0: CRG0603F4K7, Resistor_SMD:R_0603_1608Metric, B.Cu at (71.8, 34.7)
- added R0: CRG0603F4K7, Resistor_SMD:R_0603_1608Metric, B.Cu at (113.0, 34.0)
- added R0: CRG0603F4K7, Resistor_SMD:R_0603_1608Metric, B.Cu at (87.3, 34.0)
- added R0: CRG0603F4K7, Resistor_SMD:R_0603_1608Metric, B.Cu at (97.4, 34.7)
- added R0: CRG0603F4K7, Resistor_SMD:R_0603_1608Metric, B.Cu at (83.8, 36.1)
- added R0: CRG0603F4K7, Resistor_SMD:R_0603_1608Metric, B.Cu at (61.9, -13.8)
- added R0: CRG0603F4K7, Resistor_SMD:R_0603_1608Metric, B.Cu at (63.2, 34.7)
- added R0: CRG0603F4K7, Resistor_SMD:R_0603_1608Metric, B.Cu at (88.8, 34.7)
- added R0: CRG0603F4K7, Resistor_SMD:R_0603_1608Metric, B.Cu at (104.4, 34.0)
- added R0: CRG0603F4K7, Resistor_SMD:R_0603_1608Metric, B.Cu at (119.6, 36.5)
- added R0: CRG0603F4K7, Resistor_SMD:R_0603_1608Metric, B.Cu at (109.5, 36.1)
- added R0: CRG0603F4K7, Resistor_SMD:R_0603_1608Metric, F.Cu at (113.2, 33.5)
- added R0: CRG0603F4K7, Resistor_SMD:R_0603_1608Metric, F.Cu at (111.5, 33.9)
- added R0: CRG0603F4K7, Resistor_SMD:R_0603_1608Metric, F.Cu at (96.0, 33.5)
- added R0: CRG0603F4K7, Resistor_SMD:R_0603_1608Metric, F.Cu at (103.0, 33.9)
- added R0: CRG0603F4K7, Resistor_SMD:R_0603_1608Metric, F.Cu at (108.1, 32.0)
- added R0: CRG0603F4K7, Resistor_SMD:R_0603_1608Metric, B.Cu at (68.8, -14.2)
- added R0: CRG0603F4K7, Resistor_SMD:R_0603_1608Metric, F.Cu at (99.5, 32.0)
- added R0: CRG0603F4K7, Resistor_SMD:R_0603_1608Metric, F.Cu at (92.5, 31.2)
- added R0: CRG0603F4K7, Resistor_SMD:R_0603_1608Metric, F.Cu at (101.1, 31.2)
- added R0: CRG0603F4K7, Resistor_SMD:R_0603_1608Metric, F.Cu at (116.7, 32.0)
- added R0: CRG0603F4K7, Resistor_SMD:R_0603_1608Metric, F.Cu at (109.7, 31.2)
- added R0: CRG0603F4K7, Resistor_SMD:R_0603_1608Metric, F.Cu at (94.5, 33.9)
- added R0: CRG0603F4K7, Resistor_SMD:R_0603_1608Metric, F.Cu at (104.6, 33.5)
- added R0: CRG0603F4K7, Resistor_SMD:R_0603_1608Metric, F.Cu at (79.0, 33.5)
- added R0: CRG0603F4K7, Resistor_SMD:R_0603_1608Metric, F.Cu at (85.9, 33.9)
- added R0: CRG0603F4K7, Resistor_SMD:R_0603_1608Metric, F.Cu at (91.0, 32.0)
- moved J11 27.6 mm to (73.8, 3.75)
Routing:
- net (no net): track 0.00 -> 868.2 mm, vias 0 -> 156
- net Net-(Q58-Pad3): track 13.9 -> 6.96 mm
- net GND: track 12.3 -> 6.15 mm, vias 8 -> 4
- net +12V: track 7.98 -> 3.99 mm, vias 4 -> 2
- net COL03: track 7.42 -> 3.71 mm
- net Net-(Q58-Pad1): track 6.19 -> 3.09 mm
- net COL03_ON: track 4.77 -> 2.38 mm
- net COL03_OFF: track 3.53 -> 1.77 mm
- added copper zone on B.Cu, net (none)
- added copper zone on F.Cu, net (none)

Commit message: automated commit
Parts:
- renumbered Q0 to Q100, Q0 to Q102, Q0 to Q112, Q0 to Q115, Q0 to Q118, Q0 to Q122, Q0 to Q125, Q0 to Q128, Q0 to Q50, Q0 to Q53, Q0 to Q56, Q0 to Q58, Q0 to Q60, Q0 to Q61, Q0 to Q63, Q0 to Q64, Q0 to Q66, Q0 to Q68, Q0 to Q71, Q0 to Q74, Q0 to Q76, Q0 to Q78, Q0 to Q79, Q0 to Q81, Q0 to Q82, Q0 to Q84, Q0 to Q86, Q0 to Q89, Q0 to Q92, Q0 to Q94, Q0 to Q96, Q0 to Q97, Q0 to Q99, R0 to R144, R0 to R147, R0 to R151, R0 to R152, R0 to R155, R0 to R157, R0 to R158, R0 to R160, R0 to R161, R0 to R162, R0 to R165, R0 to R166, R0 to R168, R0 to R171, R0 to R175, R0 to R176, R0 to R179, R0 to R181, R0 to R182, R0 to R184, R0 to R185, R0 to R186, R0 to R189, R0 to R190, R0 to R192, R0 to R195, R0 to R199, R0 to R200, R0 to R203, R0 to R205, R0 to R206, R0 to R208, R0 to R209, R0 to R210, R0 to R213, R0 to R214, R0 to R227, R0 to R230, R0 to R233, R0 to R234, R0 to R240, R0 to R243, R0 to R247, R0 to R248

Commit message: automated commit
Parts:
- renumbered Q0 to Q104, Q0 to Q107, Q0 to Q114, Q0 to Q117, Q0 to Q120, Q0 to Q130, Q0 to Q131, Q0 to Q132, Q0 to Q229, R0 to R216, R0 to R219, R0 to R223, R0 to R224, R0 to R232, R0 to R237, R0 to R238, R0 to R251, R0 to R252, R0 to R253, R0 to R254
Changed lines of the file:
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@@
     (pad_to_mask_clearance 0)
     (aux_axis_origin 0 0)
-    (visible_elements FFFFFF7F)
+    (visible_elements FFFFF77F)
     (pcbplotparams
       (layerselection 0x010fc_ffffffff)
@@
     (tags resistor)
     (attr smd)
-    (fp_text reference R0 (at 3.7 0 270) (layer B.SilkS)
+    (fp_text reference R219 (at 3.7 0 270) (layer B.SilkS)
       (effects (font (size 1 1) (thickness 0.15)) (justify mirror))
     )
@@
     (tags "sot 723")
     (attr smd)
-    (fp_text reference Q0 (at -1.4 -3 270) (layer B.SilkS)
+    (fp_text reference Q229 (at -1.4 -3 270) (layer B.SilkS)
       (effects (font (size 1 1) (thickness 0.15)) (justify mirror))
     )
@@
     (tags resistor)
     (attr smd)
-    (fp_text reference R0 (at -3.8 -0.1 270) (layer B.SilkS)
+    (fp_text reference R224 (at -3.8 -0.1 270) (layer B.SilkS)
       (effects (font (size 1 1) (thickness 0.15)) (justify mirror))
     )
@@
     (tags "TSOT-23-6 MK06A TSOT-6")
     (attr smd)
-    (fp_text reference Q0 (at 0.75 -2.5 270) (layer B.SilkS)
+    (fp_text reference Q114 (at 0.75 -2.5 270) (layer B.SilkS)
       (effects (font (size 1 1) (thickness 0.15)) (justify mirror))
     )
@@
     (tags resistor)
     (attr smd)
-    (fp_text reference R0 (at 3.7 0 270) (layer B.SilkS)
+    (fp_text reference R252 (at 3.7 0 270) (layer B.SilkS)
       (effects (font (size 1 1) (thickness 0.15)) (justify mirror))
     )
@@
     (tags resistor)
     (attr smd)
-    (fp_text reference R0 (at -3.8 -0.1 270) (layer B.SilkS)
+    (fp_text reference R238 (at -3.8 -0.1 270) (layer B.SilkS)
       (effects (font (size 1 1) (thickness 0.15)) (justify mirror))
     )
@@
     (tags "sot 723")
     (attr smd)
-    (fp_text reference Q0 (at -1.4 -3 270) (layer B.SilkS)
+    (fp_text reference Q132 (at -1.4 -3 270) (layer B.SilkS)
       (effects (font (size 1 1) (thickness 0.15)) (justify mirror))
     )
@@
     (tags "TSOT-23-6 MK06A TSOT-6")
     (attr smd)
-    (fp_text reference Q0 (at 0.75 -2.5 270) (layer B.SilkS)
+    (fp_text reference Q104 (at 0.75 -2.5 270) (layer B.SilkS)
       (effects (font (size 1 1) (thickness 0.15)) (justify mirror))
     )
@@
     (tags resistor)
     (attr smd)
-    (fp_text reference R0 (at -3.6 0 270) (layer B.SilkS)
+    (fp_text reference R251 (at -3.6 0 270) (layer B.SilkS)
       (effects (font (size 1 1) (thickness 0.15)) (justify mirror))
     )
@@
     (tags resistor)
     (attr smd)
-    (fp_text reference R0 (at -3.55 0 270) (layer B.SilkS)
+    (fp_text reference R253 (at -3.55 0 270) (layer B.SilkS)
       (effects (font (size 1 1) (thickness 0.15)) (justify mirror))
     )
@@
     (tags "sot 723")
     (attr smd)
-    (fp_text reference Q0 (at 2.7 0.05 270) (layer B.SilkS)
+    (fp_text reference Q117 (at 2.7 0.05 270) (layer B.SilkS)
       (effects (font (size 1 1) (thickness 0.15)) (justify mirror))
     )
@@
     (tags resistor)
     (attr smd)
-    (fp_text reference R0 (at -3.55 0 270) (layer B.SilkS)
+    (fp_text reference R237 (at -3.55 0 270) (layer B.SilkS)
       (effects (font (size 1 1) (thickness 0.15)) (justify mirror))
     )
@@
     (tags resistor)
     (attr smd)
-    (fp_text reference R0 (at -3.6 0 270) (layer B.SilkS)
+    (fp_text reference R216 (at -3.6 0 270) (layer B.SilkS)
       (effects (font (size 1 1) (thickness 0.15)) (justify mirror))
     )
@@
     (tags "sot 723")
     (attr smd)
-    (fp_text reference Q0 (at 2.7 0.05 270) (layer B.SilkS)
+    (fp_text reference Q131 (at 2.7 0.05 270) (layer B.SilkS)
       (effects (font (size 1 1) (thickness 0.15)) (justify mirror))
     )
@@
     (tags resistor)
     (attr smd)
-    (fp_text reference R0 (at -3.55 0 270) (layer B.SilkS)
+    (fp_text reference R223 (at -3.55 0 270) (layer B.SilkS)
       (effects (font (size 1 1) (thickness 0.15)) (justify mirror))
     )
@@
     (tags "sot 723")
     (attr smd)
-    (fp_text reference Q0 (at -1.4 -3 270) (layer B.SilkS)
+    (fp_text reference Q120 (at -1.4 -3 270) (layer B.SilkS)
       (effects (font (size 1 1) (thickness 0.15)) (justify mirror))
     )
@@
     (tags "sot 723")
     (attr smd)
-    (fp_text reference Q0 (at 2.7 0.05 270) (layer B.SilkS)
+    (fp_text reference Q107 (at 2.7 0.05 270) (layer B.SilkS)
       (effects (font (size 1 1) (thickness 0.15)) (justify mirror))
     )
@@
     (tags resistor)
     (attr smd)
-    (fp_text reference R0 (at -3.8 -0.1 270) (layer B.SilkS)
+    (fp_text reference R254 (at -3.8 -0.1 270) (layer B.SilkS)
       (effects (font (size 1 1) (thickness 0.15)) (justify mirror))
     )
@@
     (tags resistor)
     (attr smd)
-    (fp_text reference R0 (at 3.7 0 270) (layer B.SilkS)
+    (fp_text reference R232 (at 3.7 0 270) (layer B.SilkS)
       (effects (font (size 1 1) (thickness 0.15)) (justify mirror))
     )
@@
     (tags "TSOT-23-6 MK06A TSOT-6")
     (attr smd)
-    (fp_text reference Q0 (at 0.75 -2.5 270) (layer B.SilkS)
+    (fp_text reference Q130 (at 0.75 -2.5 270) (layer B.SilkS)
       (effects (font (size 1 1) (thickness 0.15)) (justify mirror))
     )

Commit message: automated commit
Parts:
- removed Q229: SSM3K35AMFV, Package_TO_SOT_SMD:SOT-723
- removed R0 (x4): CRG0603F4K7, Resistor_SMD:R_0603_1608Metric
- removed the R207 at (355.1, 233.1)
- removed the R242 at (330.9, 327.5)
- removed the R245 at (326.9, 329.4)
- added Q58: DMG6602, Package_TO_SOT_SMD:TSOT-23-6, B.Cu at (255.5, -78.3)
- added Q61: SSM3K35AMFV, Package_TO_SOT_SMD:SOT-723, B.Cu at (258.3, -78.6)
- added Q64: SSM3K35AMFV, Package_TO_SOT_SMD:SOT-723, B.Cu at (258.2, -76.7)
- added R155: CRG0603F4K7, Resistor_SMD:R_0603_1608Metric, B.Cu at (253.0, -76.0)
- added R158: CRG0603F4K7, Resistor_SMD:R_0603_1608Metric, B.Cu at (256.5, -74.6)
- added R161: CRG0603F4K7, Resistor_SMD:R_0603_1608Metric, B.Cu at (260.0, -76.8)
- added R162: CRG0603F4K7, Resistor_SMD:R_0603_1608Metric, B.Cu at (258.1, -74.2)
- added R207: CRG0603F4K7, Resistor_SMD:R_0603_1608Metric, B.Cu at (285.2, -112.5)
- added R207: CRG0603F4K7, Resistor_SMD:R_0603_1608Metric, B.Cu at (103.8, -14.7)
- added R242: CRG0603F4K7, Resistor_SMD:R_0603_1608Metric, B.Cu at (302.3, -112.5)
- added R242: CRG0603F4K7, Resistor_SMD:R_0603_1608Metric, B.Cu at (120.8, -14.7)
- added R245: CRG0603F4K7, Resistor_SMD:R_0603_1608Metric, B.Cu at (298.8, -110.3)
- added R245: CRG0603F4K7, Resistor_SMD:R_0603_1608Metric, B.Cu at (117.3, -12.4)
- Q100, Q101, Q104, Q105, Q107, Q108, Q111, Q114, Q117, Q120, Q121, Q124, Q127, Q130, Q131, Q132, Q49, Q52, Q55, Q59, Q62, Q65, Q68, Q69, Q71, Q72, Q74, Q75, Q78, Q81, Q84, Q85, Q88, Q91, Q94, Q95, Q97, Q98, R143, R146, R149, R150, R156, R159, R163, R164, R168, R169, R171, R172, R175, R176, R177, R178, R181, R184, R189, R190, R191, R194, R197, R198, R203, R204, R206, R209, R210, R211, R212, R216, R217, R219, R220, R223, R224, R225, R226, R232, R237, R238, R239, R246, R251, R252, R253, R254: moved to B.Cu
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- renumbered Q0 to Q101, Q0 to Q103, Q0 to Q105, Q0 to Q106, Q0 to Q108, Q0 to Q109, Q0 to Q111, Q0 to Q113, Q0 to Q116, Q0 to Q119, Q0 to Q121, Q0 to Q123, Q0 to Q124, Q0 to Q126, Q0 to Q127, Q0 to Q129, Q0 to Q49, Q0 to Q51, Q0 to Q52, Q0 to Q54, Q0 to Q55, Q0 to Q57, Q0 to Q59, Q0 to Q62, Q0 to Q65, Q0 to Q67, Q0 to Q69, Q0 to Q70, Q0 to Q72, Q0 to Q73, Q0 to Q75, Q0 to Q77, Q0 to Q80, Q0 to Q83, Q0 to Q85, Q0 to Q87, Q0 to Q88, Q0 to Q90, Q0 to Q91, Q0 to Q93, Q0 to Q95, Q0 to Q98, R0 to R143, R0 to R145, R0 to R146, R0 to R148, R0 to R149, R0 to R150, R0 to R153, R0 to R154, R0 to R156, R0 to R159, R0 to R163, R0 to R164, R0 to R167, R0 to R169, R0 to R170, R0 to R172, R0 to R173, R0 to R174, R0 to R177, R0 to R178, R0 to R180, R0 to R183, R0 to R187, R0 to R188, R0 to R191, R0 to R193, R0 to R194, R0 to R196, R0 to R197, R0 to R198, R0 to R201, R0 to R202, R0 to R204, R0 to R211, R0 to R212, R0 to R215, R0 to R217, R0 to R218, R0 to R220, R0 to R221, R0 to R222, R0 to R225, R0 to R226, R0 to R228, R0 to R231, R0 to R235, R0 to R236, R0 to R239, R0 to R241, R0 to R244, R0 to R246, R0 to R249, R0 to R250
Connections:
- Q100 pad 1: COL15_ON -> (no net)
- Q100 pad 2: GND -> (no net)
- Q100 pad 3: Net-(Q100-Pad3) -> (no net)
- Q100 pad 1: (no net) -> COL15_ON
- Q100 pad 2: (no net) -> GND
- Q100 pad 3: (no net) -> Net-(Q100-Pad3)
- Q101 pad 1: COL16_ON -> (no net)
- Q101 pad 2: GND -> (no net)
- Q101 pad 3: Net-(Q101-Pad3) -> (no net)
- Q101 pad 1: (no net) -> COL16_ON
- Q101 pad 2: (no net) -> GND
- Q101 pad 3: (no net) -> Net-(Q101-Pad3)
- Q102 pad 1: COL17_ON -> (no net)
- Q102 pad 2: GND -> (no net)
- Q102 pad 3: Net-(Q102-Pad3) -> (no net)
- Q102 pad 1: (no net) -> COL17_ON
- Q102 pad 2: (no net) -> GND
- Q102 pad 3: (no net) -> Net-(Q102-Pad3)
- Q103 pad 1: Net-(Q103-Pad1) -> (no net)
- Q103 pad 2: +12V -> (no net)
- Q103 pad 3: Net-(Q103-Pad3) -> (no net)
- Q103 pad 4: COL18 -> (no net)
- Q103 pad 5: GND -> (no net)
- Q103 pad 6: COL18 -> (no net)
- Q103 pad 1: (no net) -> Net-(Q103-Pad1)
- Q103 pad 2: (no net) -> +12V
- Q103 pad 3: (no net) -> Net-(Q103-Pad3)
- Q103 pad 4: (no net) -> COL18
- Q103 pad 5: (no net) -> GND
- Q103 pad 6: (no net) -> COL18
- Q104 pad 1: Net-(Q104-Pad1) -> (no net)
- Q104 pad 2: +12V -> (no net)
- Q104 pad 3: Net-(Q104-Pad3) -> (no net)
- Q104 pad 4: COL19 -> (no net)
- Q104 pad 5: GND -> (no net)
- Q104 pad 6: COL19 -> (no net)
- Q104 pad 1: (no net) -> Net-(Q104-Pad1)
- Q104 pad 2: (no net) -> +12V
- Q104 pad 3: (no net) -> Net-(Q104-Pad3)
- Q104 pad 4: (no net) -> COL19
- Q104 pad 5: (no net) -> GND
- Q104 pad 6: (no net) -> COL19
- Q105 pad 1: Net-(Q105-Pad1) -> (no net)
- Q105 pad 2: +12V -> (no net)
- Q105 pad 3: Net-(Q105-Pad3) -> (no net)
- Q105 pad 4: COL20 -> (no net)
- Q105 pad 5: GND -> (no net)
- Q105 pad 6: COL20 -> (no net)
- Q105 pad 1: (no net) -> Net-(Q105-Pad1)
- Q105 pad 2: (no net) -> +12V
- Q105 pad 3: (no net) -> Net-(Q105-Pad3)
- Q105 pad 4: (no net) -> COL20
- Q105 pad 5: (no net) -> GND
- Q105 pad 6: (no net) -> COL20
- Q106 pad 1: COL18_ON -> (no net)
- Q106 pad 2: GND -> (no net)
- Q106 pad 3: Net-(Q103-Pad3) -> (no net)
- Q106 pad 1: (no net) -> COL18_ON
- Q106 pad 2: (no net) -> GND
- Q106 pad 3: (no net) -> Net-(Q103-Pad3)
- Q107 pad 1: COL19_ON -> (no net)
- Q107 pad 2: GND -> (no net)
- Q107 pad 3: Net-(Q104-Pad3) -> (no net)
- Q107 pad 1: (no net) -> COL19_ON
- Q107 pad 2: (no net) -> GND
- Q107 pad 3: (no net) -> Net-(Q104-Pad3)
- Q108 pad 1: COL20_ON -> (no net)
- Q108 pad 2: GND -> (no net)
- Q108 pad 3: Net-(Q105-Pad3) -> (no net)
- Q108 pad 1: (no net) -> COL20_ON
- Q108 pad 2: (no net) -> GND
- Q108 pad 3: (no net) -> Net-(Q105-Pad3)
- Q109 pad 1: COL18_ON -> (no net)
- Q109 pad 2: GND -> (no net)
- Q109 pad 3: Net-(Q103-Pad1) -> (no net)
- Q109 pad 1: (no net) -> COL18_ON
- Q109 pad 2: (no net) -> GND
- Q109 pad 3: (no net) -> Net-(Q103-Pad1)
- Q111 pad 1: COL20_ON -> (no net)
- Q111 pad 2: GND -> (no net)
- Q111 pad 3: Net-(Q105-Pad1) -> (no net)
- Q111 pad 1: (no net) -> COL20_ON
- Q111 pad 2: (no net) -> GND
- Q111 pad 3: (no net) -> Net-(Q105-Pad1)
- Q112 pad 1: Net-(Q112-Pad1) -> (no net)
- Q112 pad 2: +12V -> (no net)
- Q112 pad 3: Net-(Q112-Pad3) -> (no net)
- Q112 pad 4: COL21 -> (no net)
- Q112 pad 5: GND -> (no net)
- Q112 pad 6: COL21 -> (no net)
- Q112 pad 1: (no net) -> Net-(Q112-Pad1)
- Q112 pad 2: (no net) -> +12V
- Q112 pad 3: (no net) -> Net-(Q112-Pad3)
- Q112 pad 4: (no net) -> COL21
- Q112 pad 5: (no net) -> GND
- Q112 pad 6: (no net) -> COL21
- Q113 pad 1: Net-(Q113-Pad1) -> (no net)
- Q113 pad 2: +12V -> (no net)
- Q113 pad 3: Net-(Q113-Pad3) -> (no net)
- Q113 pad 4: COL22 -> (no net)
- Q113 pad 5: GND -> (no net)
- Q113 pad 6: COL22 -> (no net)
- Q113 pad 1: (no net) -> Net-(Q113-Pad1)
- Q113 pad 2: (no net) -> +12V
- Q113 pad 3: (no net) -> Net-(Q113-Pad3)
- Q113 pad 4: (no net) -> COL22
- Q113 pad 5: (no net) -> GND
- Q113 pad 6: (no net) -> COL22
- Q114 pad 1: Net-(Q114-Pad1) -> (no net)
- Q114 pad 2: +12V -> (no net)
- Q114 pad 3: Net-(Q114-Pad3) -> (no net)
- Q114 pad 4: COL23 -> (no net)
- Q114 pad 5: GND -> (no net)
- Q114 pad 6: COL23 -> (no net)
- Q114 pad 1: (no net) -> Net-(Q114-Pad1)
- Q114 pad 2: (no net) -> +12V
- Q114 pad 3: (no net) -> Net-(Q114-Pad3)
- Q114 pad 4: (no net) -> COL23
- Q114 pad 5: (no net) -> GND
- Q114 pad 6: (no net) -> COL23
- Q115 pad 1: COL21_ON -> (no net)
- Q115 pad 2: GND -> (no net)
- Q115 pad 3: Net-(Q112-Pad3) -> (no net)
- Q115 pad 1: (no net) -> COL21_ON
- Q115 pad 2: (no net) -> GND
- Q115 pad 3: (no net) -> Net-(Q112-Pad3)
- Q116 pad 1: COL22_ON -> (no net)
- Q116 pad 2: GND -> (no net)
- Q116 pad 3: Net-(Q113-Pad3) -> (no net)
- Q116 pad 1: (no net) -> COL22_ON
- Q116 pad 2: (no net) -> GND
- Q116 pad 3: (no net) -> Net-(Q113-Pad3)
- Q117 pad 1: COL23_ON -> (no net)
- Q117 pad 2: GND -> (no net)
- Q117 pad 3: Net-(Q114-Pad3) -> (no net)
- Q117 pad 1: (no net) -> COL23_ON
- Q117 pad 2: (no net) -> GND
- Q117 pad 3: (no net) -> Net-(Q114-Pad3)
- Q118 pad 1: COL21_ON -> (no net)
- Q118 pad 2: GND -> (no net)
- Q118 pad 3: Net-(Q112-Pad1) -> (no net)
- Q118 pad 1: (no net) -> COL21_ON
- Q118 pad 2: (no net) -> GND
- Q118 pad 3: (no net) -> Net-(Q112-Pad1)
- Q119 pad 1: COL22_ON -> (no net)
- Q119 pad 2: GND -> (no net)
- Q119 pad 3: Net-(Q113-Pad1) -> (no net)
- Q119 pad 1: (no net) -> COL22_ON
- Q119 pad 2: (no net) -> GND
- Q119 pad 3: (no net) -> Net-(Q113-Pad1)
- Q120 pad 1: COL23_ON -> (no net)
- Q120 pad 2: GND -> (no net)
- Q120 pad 3: Net-(Q114-Pad1) -> (no net)
- Q120 pad 1: (no net) -> COL23_ON
- Q120 pad 2: (no net) -> GND
- Q120 pad 3: (no net) -> Net-(Q114-Pad1)
- Q121 pad 1: Net-(Q121-Pad1) -> (no net)
- Q121 pad 2: +12V -> (no net)
- Q121 pad 3: Net-(Q121-Pad3) -> (no net)
- Q121 pad 4: COL24 -> (no net)
- Q121 pad 5: GND -> (no net)
- Q121 pad 6: COL24 -> (no net)
- Q121 pad 1: (no net) -> Net-(Q121-Pad1)
- Q121 pad 2: (no net) -> +12V
- Q121 pad 3: (no net) -> Net-(Q121-Pad3)
- Q121 pad 4: (no net) -> COL24
- Q121 pad 5: (no net) -> GND
- Q121 pad 6: (no net) -> COL24
- Q122 pad 1: Net-(Q122-Pad1) -> (no net)
- Q122 pad 2: +12V -> (no net)
- Q122 pad 3: Net-(Q122-Pad3) -> (no net)
- Q122 pad 4: COL25 -> (no net)
- Q122 pad 5: GND -> (no net)
- Q122 pad 6: COL25 -> (no net)
- Q122 pad 1: (no net) -> Net-(Q122-Pad1)
- Q122 pad 2: (no net) -> +12V
- Q122 pad 3: (no net) -> Net-(Q122-Pad3)
- Q122 pad 4: (no net) -> COL25
- Q122 pad 5: (no net) -> GND
- Q122 pad 6: (no net) -> COL25
- Q123 pad 1: Net-(Q123-Pad1) -> (no net)
- Q123 pad 2: +12V -> (no net)
- Q123 pad 3: Net-(Q123-Pad3) -> (no net)
- Q123 pad 4: COL26 -> (no net)
- Q123 pad 5: GND -> (no net)
- Q123 pad 6: COL26 -> (no net)
- Q123 pad 1: (no net) -> Net-(Q123-Pad1)
- Q123 pad 2: (no net) -> +12V
- Q123 pad 3: (no net) -> Net-(Q123-Pad3)
- Q123 pad 4: (no net) -> COL26
- Q123 pad 5: (no net) -> GND
- Q123 pad 6: (no net) -> COL26
- Q124 pad 1: COL24_ON -> (no net)
- Q124 pad 2: GND -> (no net)
- Q124 pad 3: Net-(Q121-Pad3) -> (no net)
- Q124 pad 1: (no net) -> COL24_ON
- Q124 pad 2: (no net) -> GND
- Q124 pad 3: (no net) -> Net-(Q121-Pad3)
- Q125 pad 1: COL25_ON -> (no net)
- Q125 pad 2: GND -> (no net)
- Q125 pad 3: Net-(Q122-Pad3) -> (no net)
- Q125 pad 1: (no net) -> COL25_ON
- Q125 pad 2: (no net) -> GND
- Q125 pad 3: (no net) -> Net-(Q122-Pad3)
- Q126 pad 1: COL26_ON -> (no net)
- Q126 pad 2: GND -> (no net)
- Q126 pad 3: Net-(Q123-Pad3) -> (no net)
- Q126 pad 1: (no net) -> COL26_ON
- Q126 pad 2: (no net) -> GND
- Q126 pad 3: (no net) -> Net-(Q123-Pad3)
- Q127 pad 1: COL24_ON -> (no net)
- Q127 pad 2: GND -> (no net)
- Q127 pad 3: Net-(Q121-Pad1) -> (no net)
- Q127 pad 1: (no net) -> COL24_ON
- Q127 pad 2: (no net) -> GND
- Q127 pad 3: (no net) -> Net-(Q121-Pad1)
- Q128 pad 1: COL25_ON -> (no net)
- Q128 pad 2: GND -> (no net)
- Q128 pad 3: Net-(Q122-Pad1) -> (no net)
- Q128 pad 1: (no net) -> COL25_ON
- Q128 pad 2: (no net) -> GND
- Q128 pad 3: (no net) -> Net-(Q122-Pad1)
- Q129 pad 1: COL26_ON -> (no net)
- Q129 pad 2: GND -> (no net)
- Q129 pad 3: Net-(Q123-Pad1) -> (no net)
- Q129 pad 1: (no net) -> COL26_ON
- Q129 pad 2: (no net) -> GND
- Q129 pad 3: (no net) -> Net-(Q123-Pad1)
- Q130 pad 1: Net-(Q130-Pad1) -> (no net)
- Q130 pad 2: +12V -> (no net)
- Q130 pad 3: Net-(Q130-Pad3) -> (no net)
- Q130 pad 4: COL27 -> (no net)
- Q130 pad 5: GND -> (no net)
- Q130 pad 6: COL27 -> (no net)
- Q130 pad 1: (no net) -> Net-(Q130-Pad1)
- Q130 pad 2: (no net) -> +12V
- Q130 pad 3: (no net) -> Net-(Q130-Pad3)
- Q130 pad 4: (no net) -> COL27
- Q130 pad 5: (no net) -> GND
- Q130 pad 6: (no net) -> COL27
- Q131 pad 1: COL27_ON -> (no net)
- Q131 pad 2: GND -> (no net)
- Q131 pad 3: Net-(Q130-Pad3) -> (no net)
- Q131 pad 1: (no net) -> COL27_ON
- Q131 pad 2: (no net) -> GND
- Q131 pad 3: (no net) -> Net-(Q130-Pad3)
- Q132 pad 1: COL27_ON -> (no net)
- Q132 pad 2: GND -> (no net)
- Q132 pad 3: Net-(Q130-Pad1) -> (no net)
- Q132 pad 1: (no net) -> COL27_ON
- Q132 pad 2: (no net) -> GND
- Q132 pad 3: (no net) -> Net-(Q130-Pad1)
- Q49 pad 1: Net-(Q49-Pad1) -> (no net)
- Q49 pad 2: +12V -> (no net)
- Q49 pad 3: Net-(Q49-Pad3) -> (no net)
- Q49 pad 4: COL00 -> (no net)
- Q49 pad 5: GND -> (no net)
- Q49 pad 6: COL00 -> (no net)
- Q49 pad 1: (no net) -> Net-(Q49-Pad1)
- Q49 pad 2: (no net) -> +12V
- Q49 pad 3: (no net) -> Net-(Q49-Pad3)
- Q49 pad 4: (no net) -> COL00
- Q49 pad 5: (no net) -> GND
- Q49 pad 6: (no net) -> COL00
- Q50 pad 1: Net-(Q50-Pad1) -> (no net)
- Q50 pad 2: +12V -> (no net)
- Q50 pad 3: Net-(Q50-Pad3) -> (no net)
- Q50 pad 4: COL01 -> (no net)
- Q50 pad 5: GND -> (no net)
- Q50 pad 6: COL01 -> (no net)
- Q50 pad 1: (no net) -> Net-(Q50-Pad1)
- Q50 pad 2: (no net) -> +12V
- Q50 pad 3: (no net) -> Net-(Q50-Pad3)
- Q50 pad 4: (no net) -> COL01
- Q50 pad 5: (no net) -> GND
- Q50 pad 6: (no net) -> COL01
- Q51 pad 1: Net-(Q51-Pad1) -> (no net)
- Q51 pad 2: +12V -> (no net)
- Q51 pad 3: Net-(Q51-Pad3) -> (no net)
- Q51 pad 4: COL02 -> (no net)
- Q51 pad 5: GND -> (no net)
- Q51 pad 6: COL02 -> (no net)
- Q51 pad 1: (no net) -> Net-(Q51-Pad1)
- Q51 pad 2: (no net) -> +12V
- Q51 pad 3: (no net) -> Net-(Q51-Pad3)
- Q51 pad 4: (no net) -> COL02
- Q51 pad 5: (no net) -> GND
- Q51 pad 6: (no net) -> COL02
- Q52 pad 1: COL00_ON -> (no net)
- Q52 pad 2: GND -> (no net)
- Q52 pad 3: Net-(Q49-Pad3) -> (no net)
- Q52 pad 1: (no net) -> COL00_ON
- Q52 pad 2: (no net) -> GND
- Q52 pad 3: (no net) -> Net-(Q49-Pad3)
- Q53 pad 1: COL01_ON -> (no net)
- Q53 pad 2: GND -> (no net)
- Q53 pad 3: Net-(Q50-Pad3) -> (no net)
- Q53 pad 1: (no net) -> COL01_ON
- Q53 pad 2: (no net) -> GND
- Q53 pad 3: (no net) -> Net-(Q50-Pad3)
- Q54 pad 1: COL02_ON -> (no net)
- Q54 pad 2: GND -> (no net)
- Q54 pad 3: Net-(Q51-Pad3) -> (no net)
- Q54 pad 1: (no net) -> COL02_ON
- Q54 pad 2: (no net) -> GND
- Q54 pad 3: (no net) -> Net-(Q51-Pad3)
- Q55 pad 1: COL00_ON -> (no net)
- Q55 pad 2: GND -> (no net)
- Q55 pad 3: Net-(Q49-Pad1) -> (no net)
- Q55 pad 1: (no net) -> COL00_ON
- Q55 pad 2: (no net) -> GND
- Q55 pad 3: (no net) -> Net-(Q49-Pad1)
- Q56 pad 1: COL01_ON -> (no net)
- Q56 pad 2: GND -> (no net)
- Q56 pad 3: Net-(Q50-Pad1) -> (no net)
- Q56 pad 1: (no net) -> COL01_ON
- Q56 pad 2: (no net) -> GND
- Q56 pad 3: (no net) -> Net-(Q50-Pad1)
- Q57 pad 1: COL02_ON -> (no net)
- Q57 pad 2: GND -> (no net)
- Q57 pad 3: Net-(Q51-Pad1) -> (no net)
- Q57 pad 1: (no net) -> COL02_ON
- Q57 pad 2: (no net) -> GND
- Q57 pad 3: (no net) -> Net-(Q51-Pad1)
- Q58 pad 1: (no net) -> Net-(Q58-Pad1)
- Q58 pad 2: (no net) -> +12V
- Q58 pad 3: (no net) -> Net-(Q58-Pad3)
- Q58 pad 4: (no net) -> COL03
- Q58 pad 5: (no net) -> GND
- Q58 pad 6: (no net) -> COL03
- Q59 pad 1: Net-(Q59-Pad1) -> (no net)
- Q59 pad 2: +12V -> (no net)
- Q59 pad 3: Net-(Q59-Pad3) -> (no net)
- Q59 pad 4: COL04 -> (no net)
- Q59 pad 5: GND -> (no net)
- Q59 pad 6: COL04 -> (no net)
- Q59 pad 1: (no net) -> Net-(Q59-Pad1)
- Q59 pad 2: (no net) -> +12V
- Q59 pad 3: (no net) -> Net-(Q59-Pad3)
- Q59 pad 4: (no net) -> COL04
- Q59 pad 5: (no net) -> GND
- Q59 pad 6: (no net) -> COL04
- Q60 pad 1: Net-(Q60-Pad1) -> (no net)
- Q60 pad 2: +12V -> (no net)
- Q60 pad 3: Net-(Q60-Pad3) -> (no net)
- Q60 pad 4: COL05 -> (no net)
- Q60 pad 5: GND -> (no net)
- Q60 pad 6: COL05 -> (no net)
- Q60 pad 1: (no net) -> Net-(Q60-Pad1)
- Q60 pad 2: (no net) -> +12V
- Q60 pad 3: (no net) -> Net-(Q60-Pad3)
- Q60 pad 4: (no net) -> COL05
- Q60 pad 5: (no net) -> GND
- Q60 pad 6: (no net) -> COL05
- Q61 pad 1: (no net) -> COL03_ON
- Q61 pad 2: (no net) -> GND
- Q61 pad 3: (no net) -> Net-(Q58-Pad3)
- Q62 pad 1: COL04_ON -> (no net)
- Q62 pad 2: GND -> (no net)
- Q62 pad 3: Net-(Q59-Pad3) -> (no net)
- Q62 pad 1: (no net) -> COL04_ON
- Q62 pad 2: (no net) -> GND
- Q62 pad 3: (no net) -> Net-(Q59-Pad3)
- Q63 pad 1: COL05_ON -> (no net)
- Q63 pad 2: GND -> (no net)
- Q63 pad 3: Net-(Q60-Pad3) -> (no net)
- Q63 pad 1: (no net) -> COL05_ON
- Q63 pad 2: (no net) -> GND
- Q63 pad 3: (no net) -> Net-(Q60-Pad3)
- Q64 pad 1: (no net) -> COL03_ON
- Q64 pad 2: (no net) -> GND
- Q64 pad 3: (no net) -> Net-(Q58-Pad1)
- Q65 pad 1: COL04_ON -> (no net)
- Q65 pad 2: GND -> (no net)
- Q65 pad 3: Net-(Q59-Pad1) -> (no net)
- Q65 pad 1: (no net) -> COL04_ON
- Q65 pad 2: (no net) -> GND
- Q65 pad 3: (no net) -> Net-(Q59-Pad1)
- Q66 pad 1: COL05_ON -> (no net)
- Q66 pad 2: GND -> (no net)
- Q66 pad 3: Net-(Q60-Pad1) -> (no net)
- Q66 pad 1: (no net) -> COL05_ON
- Q66 pad 2: (no net) -> GND
- Q66 pad 3: (no net) -> Net-(Q60-Pad1)
- Q67 pad 1: Net-(Q67-Pad1) -> (no net)
- Q67 pad 2: +12V -> (no net)
- Q67 pad 3: Net-(Q67-Pad3) -> (no net)
- Q67 pad 4: COL06 -> (no net)
- Q67 pad 5: GND -> (no net)
- Q67 pad 6: COL06 -> (no net)
- Q67 pad 1: (no net) -> Net-(Q67-Pad1)
- Q67 pad 2: (no net) -> +12V
- Q67 pad 3: (no net) -> Net-(Q67-Pad3)
- Q67 pad 4: (no net) -> COL06
- Q67 pad 5: (no net) -> GND
- Q67 pad 6: (no net) -> COL06
- Q68 pad 1: Net-(Q68-Pad1) -> (no net)
- Q68 pad 2: +12V -> (no net)
- Q68 pad 3: Net-(Q68-Pad3) -> (no net)
- Q68 pad 4: COL07 -> (no net)
- Q68 pad 5: GND -> (no net)
- Q68 pad 6: COL07 -> (no net)
- Q68 pad 1: (no net) -> Net-(Q68-Pad1)
- Q68 pad 2: (no net) -> +12V
- Q68 pad 3: (no net) -> Net-(Q68-Pad3)
- Q68 pad 4: (no net) -> COL07
- Q68 pad 5: (no net) -> GND
- Q68 pad 6: (no net) -> COL07
- Q69 pad 1: Net-(Q69-Pad1) -> (no net)
- Q69 pad 2: +12V -> (no net)
- Q69 pad 3: Net-(Q69-Pad3) -> (no net)
- Q69 pad 4: COL08 -> (no net)
- Q69 pad 5: GND -> (no net)
- Q69 pad 6: COL08 -> (no net)
- Q69 pad 1: (no net) -> Net-(Q69-Pad1)
- Q69 pad 2: (no net) -> +12V
- Q69 pad 3: (no net) -> Net-(Q69-Pad3)
- Q69 pad 4: (no net) -> COL08
- Q69 pad 5: (no net) -> GND
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Routing:
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- added copper zone on B.Cu, net +12V
- added copper zone on B.Cu, net GND
