File: flipdot_driver.kicad_pcb (KiCad board)
At the start: 4 copper layers, 856 parts, among them J1 Barrel_Jack, J10 Conn_01x08_Male, J11 3x32_1&3_loaded_2.5mm_0.1in_f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, J2 Screw_Terminal_01x04, J3 PTH_1.5_mm, J4 PTH_1.5_mm, J5 PTH_1.5_mm, J6 PTH_1.5_mm, J7 Conn_01x05_Male, J8 PTH_1.5_mm, J9 USB-C_2.0_Connector, Q1 SSM3K35AMFV, Q10 SSM3K35AMFV, Q100 SSM3K35AMFV, Q101 SSM3K35AMFV, Q102 SSM3K35AMFV, Q103 DMG6602, Q104 DMG6602, Q105 DMG6602, Q106 SSM3K35AMFV, Q107 SSM3K35AMFV, Q108 SSM3K35AMFV, Q109 SSM3K35AMFV, Q11 SSM3K35AMFV, Q110 SSM3K35AMFV, Q111 SSM3K35AMFV, Q112 DMG6602, Q113 DMG6602, Q114 DMG6602, Q115 SSM3K35AMFV, Q116 SSM3K35AMFV, Q117 SSM3K35AMFV, Q118 SSM3K35AMFV, Q119 SSM3K35AMFV, Q12 AO3407A, Q120 SSM3K35AMFV, Q121 DMG6602, Q122 DMG6602, Q123 DMG6602, Q124 SSM3K35AMFV, Q125 SSM3K35AMFV, Q126 SSM3K35AMFV, Q127 SSM3K35AMFV, Q128 SSM3K35AMFV, Q129 SSM3K35AMFV, Q13 SSM3K35AMFV, Q130 DMG6602, Q131 SSM3K35AMFV, Q132 SSM3K35AMFV, Q14 SSM3K35AMFV, Q15 DMG6602, Q16 DMG6602, Q17 DMG6602, Q18 SSM3K35AMFV, Q19 SSM3K35AMFV, Q2 SSM3K35AMFV, Q20 SSM3K35AMFV, Q21 DMG6602, Q22 DMG6602, Q23 SSM3K35AMFV, Q24 SSM3K35AMFV, Q25 DMG6602, Q26 DMG6602, Q27 SSM3K35AMFV, Q28 SSM3K35AMFV, Q29 DMG6602, Q3 SSM3K35AMFV, Q30 DMG6602, Q31 SSM3K35AMFV, Q32 SSM3K35AMFV, Q33 DMG6602, Q34 DMG6602, Q35 SSM3K35AMFV, Q36 SSM3K35AMFV, Q37 DMG6602, Q38 DMG6602, Q39 SSM3K35AMFV, Q4 SSM3K35AMFV, Q40 SSM3K35AMFV, Q41 DMG6602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

Commit message: automated commit
Parts:
- removed the Q100 at (102.5, 21.2)
- removed the Q101 at (102.0, -12.6)
- removed the Q102 at (102.8, 18.5)
- removed the Q103 at (107.6, -8.20)
- removed the Q104 at (108.3, 19.6)
- removed the Q105 at (113.3, -10.9)
- removed the Q106 at (110.4, -7.95)
- removed the Q107 at (111.1, 19.3)
- removed the Q108 at (110.5, -10.7)
- removed the Q109 at (110.3, -9.85)
- removed the Q111 at (110.6, -12.6)
- removed the Q112 at (114.0, 16.9)
- removed the Q113 at (116.2, -8.20)
- removed the Q114 at (116.8, 19.6)
- removed the Q115 at (111.2, 16.6)
- removed the Q116 at (119.0, -7.95)
- removed the Q117 at (119.7, 19.3)
- removed the Q118 at (111.3, 18.5)
- removed the Q119 at (118.8, -9.85)
- removed the Q120 at (119.5, 21.2)
- removed the Q121 at (121.8, -10.9)
- removed the Q122 at (122.5, 16.9)
- removed the Q123 at (124.7, -8.20)
- removed the Q124 at (119.0, -10.7)
- removed the Q125 at (119.8, 16.6)
- removed the Q126 at (127.5, -7.95)
- removed the Q127 at (119.2, -12.6)
- removed the Q128 at (119.8, 18.5)
- removed the Q129 at (127.4, -9.85)
- removed the Q130 at (125.4, 19.6)
- removed the Q131 at (128.2, 19.3)
- removed the Q132 at (128.1, 21.2)
- removed the Q49 at (70.5, -10.9)
- removed the Q50 at (172.1, -77.8)
- removed the Q50 at (71.2, 16.9)
- removed the Q51 at (73.4, -8.20)
- removed the Q52 at (67.8, -10.7)
- removed the Q53 at (169.3, -78.1)
- removed the Q53 at (68.5, 16.6)
- removed the Q54 at (76.2, -7.95)
- removed the Q55 at (67.8, -12.6)
- removed the Q56 at (169.4, -76.2)
- removed the Q56 at (68.5, 18.5)
- removed the Q57 at (76.1, -9.85)
- removed the Q58 at (74.1, 19.6)
- removed the Q59 at (79.1, -10.9)
- removed the Q60 at (79.8, 16.9)
- removed the Q61 at (76.9, 19.3)
- removed the Q62 at (76.3, -10.7)
- removed the Q63 at (77.0, 16.6)
- removed the Q64 at (76.8, 21.2)
- removed the Q65 at (76.4, -12.6)
- removed the Q66 at (77.1, 18.5)
- removed the Q67 at (82.0, -8.20)
- removed the Q68 at (82.7, 19.6)
- removed the Q69 at (87.7, -10.9)
- removed the Q70 at (84.8, -7.95)
- removed the Q71 at (85.5, 19.3)
- removed the Q72 at (84.8, -10.7)
- removed the Q73 at (84.7, -9.85)
- removed the Q74 at (85.3, 21.2)
- removed the Q75 at (85.0, -12.6)
- removed the Q76 at (88.3, 16.9)
- removed the Q77 at (90.5, -8.20)
- removed the Q78 at (91.2, 19.6)
- removed the Q79 at (85.5, 16.6)
- removed the Q80 at (93.2, -9.85)
- removed the Q81 at (94.0, 19.3)
- removed the Q82 at (85.7, 18.5)
- removed the Q83 at (93.3, -7.95)
- removed the Q84 at (93.9, 21.2)
- removed the Q85 at (96.2, -10.9)
- removed the Q86 at (96.9, 16.9)
- removed the Q87 at (99.0, -8.20)
- removed the Q88 at (93.4, -10.7)
- removed the Q89 at (94.1, 16.6)
- removed the Q90 at (101.8, -7.95)
- removed the Q91 at (93.5, -12.6)
- removed the Q92 at (94.2, 18.5)
- removed the Q93 at (101.8, -9.85)
- removed the Q94 at (99.8, 19.6)
- removed the Q95 at (104.8, -10.9)
- removed the Q96 at (105.5, 16.9)
- removed the Q97 at (102.5, 19.3)
- removed the Q98 at (102.0, -10.7)
- removed the Q99 at (102.7, 16.6)
- removed the R143 at (73.0, -13.2)
- removed the R144 at (174.6, -75.5)
- removed the R144 at (73.8, 19.1)
- removed the R145 at (70.9, -10.5)
- removed the R146 at (69.5, -14.7)
- removed the R147 at (171.1, -74.1)
- removed the R147 at (70.2, 20.6)
- removed the R148 at (74.4, -11.9)
- removed the R149 at (66.0, -12.4)
- removed the R150 at (68.0, -15.1)
- removed the R151 at (167.6, -76.3)
- removed the R151 at (66.8, 18.4)
- removed the R152 at (169.5, -73.7)
- removed the R152 at (68.7, 21.0)
- removed the R153 at (77.9, -9.75)
- removed the R154 at (76.0, -12.3)
- removed the R155 at (71.6, 21.9)
- removed the R156 at (81.6, -13.2)
- removed the R157 at (82.3, 19.1)
- removed the R158 at (75.1, 23.3)
- removed the R159 at (78.1, -14.7)
- removed the R160 at (78.8, 20.6)
- removed the R161 at (78.6, 21.1)
- removed the R162 at (76.7, 23.7)
- removed the R163 at (74.6, -12.4)
- removed the R164 at (76.5, -15.1)
- removed the R165 at (75.3, 18.4)
- removed the R166 at (77.2, 21.0)
- removed the R167 at (79.5, -10.5)
- removed the R168 at (80.2, 21.9)
- removed the R169 at (90.2, -13.2)
- removed the R170 at (83.0, -11.9)
- removed the R171 at (83.7, 23.3)
- removed the R172 at (86.7, -14.7)
- removed the R173 at (86.5, -9.75)
- removed the R174 at (84.5, -12.3)
- removed the R175 at (87.2, 21.1)
- removed the R176 at (85.2, 23.7)
- removed the R177 at (83.2, -12.4)
- removed the R178 at (85.0, -15.1)
- removed the R179 at (90.8, 19.1)
- removed the R180 at (88.0, -10.5)
- removed the R181 at (88.7, 21.9)
- removed the R182 at (87.3, 20.6)
- removed the R183 at (91.5, -11.9)
- removed the R184 at (92.2, 23.3)
- removed the R185 at (83.8, 18.4)
- removed the R186 at (85.8, 21.0)
- removed the R187 at (95.0, -9.75)
- removed the R188 at (93.1, -12.3)
- removed the R189 at (95.7, 21.1)
- removed the R190 at (93.8, 23.7)
- removed the R191 at (98.7, -13.2)
- removed the R192 at (99.4, 19.1)
- removed the R193 at (96.5, -10.5)
- removed the R194 at (95.2, -14.7)
- removed the R195 at (95.9, 20.6)
- removed the R196 at (100.0, -11.9)
- removed the R197 at (91.7, -12.4)
- removed the R198 at (93.6, -15.1)
- removed the R199 at (92.4, 18.4)
- removed the R200 at (94.3, 21.0)
- removed the R201 at (103.5, -9.75)
- removed the R202 at (101.7, -12.3)
- removed the R203 at (97.2, 21.9)
- removed the R204 at (107.2, -13.2)
- removed the R205 at (108.0, 19.1)
- removed the R206 at (100.8, 23.3)
- removed the R207 at (103.8, -14.7)
- removed the R208 at (104.5, 20.6)
- removed the R209 at (104.2, 21.1)
- removed the R210 at (102.3, 23.7)
- removed the R211 at (100.2, -12.4)
- removed the R212 at (102.2, -15.1)
- removed the R213 at (101.0, 18.4)
- removed the R214 at (102.8, 21.0)
- removed the R215 at (105.1, -10.5)
- removed the R216 at (287.2, -76.0)
- removed the R216 at (105.8, 21.9)
- removed the R217 at (115.8, -13.2)
- removed the R218 at (108.6, -11.9)
- removed the R219 at (109.3, 23.3)
- removed the R220 at (112.3, -14.7)
- removed the R221 at (112.1, -9.75)
- removed the R222 at (110.2, -12.3)
- removed the R223 at (112.8, 21.1)
- removed the R224 at (110.9, 23.7)
- removed the R225 at (108.8, -12.4)
- removed the R226 at (110.7, -15.1)
- removed the R227 at (116.5, 19.1)
- removed the R228 at (113.7, -10.5)
- removed the R230 at (113.0, 20.6)
- removed the R231 at (117.2, -11.9)
- removed the R232 at (117.8, 23.3)
- removed the R233 at (109.5, 18.4)
- removed the R234 at (111.4, 21.0)
- removed the R235 at (120.7, -9.75)
- removed the R236 at (118.8, -12.3)
- removed the R237 at (121.3, 21.1)
- removed the R238 at (119.5, 23.7)
- removed the R239 at (124.3, -13.2)
- removed the R240 at (125.0, 19.1)
- removed the R241 at (122.2, -10.5)
- removed the R242 at (120.8, -14.7)
- removed the R243 at (121.5, 20.6)
- removed the R244 at (125.7, -11.9)
- removed the R245 at (117.3, -12.4)
- removed the R246 at (119.2, -15.1)
- removed the R247 at (118.0, 18.4)
- removed the R248 at (120.0, 21.0)
- removed the R249 at (129.2, -9.75)
- removed the R250 at (127.3, -12.3)
- removed the R251 at (122.9, 21.9)
- removed the R252 at (126.4, 23.3)
- removed the R253 at (129.9, 21.1)
- removed the R254 at (128.0, 23.7)
- added Q50: DMG6602, Package_TO_SOT_SMD:TSOT-23-6, F.Cu at (466.1, -118.5)
- added Q53: SSM3K35AMFV, Package_TO_SOT_SMD:SOT-723, F.Cu at (465.9, -115.7)
- added Q56: SSM3K35AMFV, Package_TO_SOT_SMD:SOT-723, F.Cu at (467.8, -115.8)
- added R144: CRG0603F4K7, Resistor_SMD:R_0603_1608Metric, F.Cu at (468.4, -121.0)
- added R147: CRG0603F4K7, Resistor_SMD:R_0603_1608Metric, F.Cu at (469.9, -117.5)
- added R151: CRG0603F4K7, Resistor_SMD:R_0603_1608Metric, F.Cu at (467.7, -114.0)
- added R152: CRG0603F4K7, Resistor_SMD:R_0603_1608Metric, F.Cu at (470.3, -115.9)
- added R216: CRG0603F4K7, Resistor_SMD:R_0603_1608Metric, B.Cu at (443.5, -153.1)
- J11, Q102, Q112, Q115, Q118, Q122, Q125, Q128, Q51, Q54, Q57, Q67, Q70, Q73, Q77, Q80, Q83, Q96, Q99, R145, R148, R153, R154, R167, R170, R173, R174, R180, R183, R187, R188, R205, R208, R213, R214, R227, R229, R230, R233, R234, R240, R243, R247, R248, U13, U14, U15, U16, U17, U18, U19: moved to B.Cu
- Q101, Q105, Q108, Q111, Q121, Q124, Q127, Q58, Q61, Q64, Q68, Q71, Q74, Q78, Q81, Q84, Q95, Q98, R155, R158, R161, R162, R168, R171, R175, R176, R181, R184, R189, R190, R204, R207, R211, R212, R217, R220, R225, R226, R239, R242, R245, R246: moved to F.Cu
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Connections:
- Q100 pad 1: (no net) -> COL15_ON
- Q100 pad 2: (no net) -> GND
- Q100 pad 3: (no net) -> Net-(Q100-Pad3)
- Q101 pad 1: (no net) -> COL16_ON
- Q101 pad 2: (no net) -> GND
- Q101 pad 3: (no net) -> Net-(Q101-Pad3)
- Q102 pad 1: (no net) -> COL17_ON
- Q102 pad 2: (no net) -> GND
- Q102 pad 3: (no net) -> Net-(Q102-Pad3)
- Q103 pad 1: (no net) -> Net-(Q103-Pad1)
- Q103 pad 2: (no net) -> +12V
- Q103 pad 3: (no net) -> Net-(Q103-Pad3)
- Q103 pad 4: (no net) -> COL18
- Q103 pad 5: (no net) -> GND
- Q103 pad 6: (no net) -> COL18
- Q104 pad 1: (no net) -> Net-(Q104-Pad1)
- Q104 pad 2: (no net) -> +12V
- Q104 pad 3: (no net) -> Net-(Q104-Pad3)
- Q104 pad 4: (no net) -> COL19
- Q104 pad 5: (no net) -> GND
- Q104 pad 6: (no net) -> COL19
- Q105 pad 1: (no net) -> Net-(Q105-Pad1)
- Q105 pad 2: (no net) -> +12V
- Q105 pad 3: (no net) -> Net-(Q105-Pad3)
- Q105 pad 4: (no net) -> COL20
- Q105 pad 5: (no net) -> GND
- Q105 pad 6: (no net) -> COL20
- Q106 pad 1: (no net) -> COL18_ON
- Q106 pad 2: (no net) -> GND
- Q106 pad 3: (no net) -> Net-(Q103-Pad3)
- Q107 pad 1: (no net) -> COL19_ON
- Q107 pad 2: (no net) -> GND
- Q107 pad 3: (no net) -> Net-(Q104-Pad3)
- Q108 pad 1: (no net) -> COL20_ON
- Q108 pad 2: (no net) -> GND
- Q108 pad 3: (no net) -> Net-(Q105-Pad3)
- Q109 pad 1: (no net) -> COL18_ON
- Q109 pad 2: (no net) -> GND
- Q109 pad 3: (no net) -> Net-(Q103-Pad1)
- Q111 pad 1: (no net) -> COL20_ON
- Q111 pad 2: (no net) -> GND
- Q111 pad 3: (no net) -> Net-(Q105-Pad1)
- Q112 pad 1: (no net) -> Net-(Q112-Pad1)
- Q112 pad 2: (no net) -> +12V
- Q112 pad 3: (no net) -> Net-(Q112-Pad3)
- Q112 pad 4: (no net) -> COL21
- Q112 pad 5: (no net) -> GND
- Q112 pad 6: (no net) -> COL21
- Q113 pad 1: (no net) -> Net-(Q113-Pad1)
- Q113 pad 2: (no net) -> +12V
- Q113 pad 3: (no net) -> Net-(Q113-Pad3)
- Q113 pad 4: (no net) -> COL22
- Q113 pad 5: (no net) -> GND
- Q113 pad 6: (no net) -> COL22
- Q114 pad 1: (no net) -> Net-(Q114-Pad1)
- Q114 pad 2: (no net) -> +12V
- Q114 pad 3: (no net) -> Net-(Q114-Pad3)
- Q114 pad 4: (no net) -> COL23
- Q114 pad 5: (no net) -> GND
- Q114 pad 6: (no net) -> COL23
- Q115 pad 1: (no net) -> COL21_ON
- Q115 pad 2: (no net) -> GND
- Q115 pad 3: (no net) -> Net-(Q112-Pad3)
- Q116 pad 1: (no net) -> COL22_ON
- Q116 pad 2: (no net) -> GND
- Q116 pad 3: (no net) -> Net-(Q113-Pad3)
- Q117 pad 1: (no net) -> COL23_ON
- Q117 pad 2: (no net) -> GND
- Q117 pad 3: (no net) -> Net-(Q114-Pad3)
- Q118 pad 1: (no net) -> COL21_ON
- Q118 pad 2: (no net) -> GND
- Q118 pad 3: (no net) -> Net-(Q112-Pad1)
- Q119 pad 1: (no net) -> COL22_ON
- Q119 pad 2: (no net) -> GND
- Q119 pad 3: (no net) -> Net-(Q113-Pad1)
- Q120 pad 1: (no net) -> COL23_ON
- Q120 pad 2: (no net) -> GND
- Q120 pad 3: (no net) -> Net-(Q114-Pad1)
- Q121 pad 1: (no net) -> Net-(Q121-Pad1)
- Q121 pad 2: (no net) -> +12V
- Q121 pad 3: (no net) -> Net-(Q121-Pad3)
- Q121 pad 4: (no net) -> COL24
- Q121 pad 5: (no net) -> GND
- Q121 pad 6: (no net) -> COL24
- Q122 pad 1: (no net) -> Net-(Q122-Pad1)
- Q122 pad 2: (no net) -> +12V
- Q122 pad 3: (no net) -> Net-(Q122-Pad3)
- Q122 pad 4: (no net) -> COL25
- Q122 pad 5: (no net) -> GND
- Q122 pad 6: (no net) -> COL25
- Q123 pad 1: (no net) -> Net-(Q123-Pad1)
- Q123 pad 2: (no net) -> +12V
- Q123 pad 3: (no net) -> Net-(Q123-Pad3)
- Q123 pad 4: (no net) -> COL26
- Q123 pad 5: (no net) -> GND
- Q123 pad 6: (no net) -> COL26
- Q124 pad 1: (no net) -> COL24_ON
- Q124 pad 2: (no net) -> GND
- Q124 pad 3: (no net) -> Net-(Q121-Pad3)
- Q125 pad 1: (no net) -> COL25_ON
- Q125 pad 2: (no net) -> GND
- Q125 pad 3: (no net) -> Net-(Q122-Pad3)
- Q126 pad 1: (no net) -> COL26_ON
- Q126 pad 2: (no net) -> GND
- Q126 pad 3: (no net) -> Net-(Q123-Pad3)
- Q127 pad 1: (no net) -> COL24_ON
- Q127 pad 2: (no net) -> GND
- Q127 pad 3: (no net) -> Net-(Q121-Pad1)
- Q128 pad 1: (no net) -> COL25_ON
- Q128 pad 2: (no net) -> GND
- Q128 pad 3: (no net) -> Net-(Q122-Pad1)
- Q129 pad 1: (no net) -> COL26_ON
- Q129 pad 2: (no net) -> GND
- Q129 pad 3: (no net) -> Net-(Q123-Pad1)
- Q130 pad 1: (no net) -> Net-(Q130-Pad1)
- Q130 pad 2: (no net) -> +12V
- Q130 pad 3: (no net) -> Net-(Q130-Pad3)
- Q130 pad 4: (no net) -> COL27
- Q130 pad 5: (no net) -> GND
- Q130 pad 6: (no net) -> COL27
- Q131 pad 1: (no net) -> COL27_ON
- Q131 pad 2: (no net) -> GND
- Q131 pad 3: (no net) -> Net-(Q130-Pad3)
- Q132 pad 1: (no net) -> COL27_ON
- Q132 pad 2: (no net) -> GND
- Q132 pad 3: (no net) -> Net-(Q130-Pad1)
- Q49 pad 1: (no net) -> Net-(Q49-Pad1)
- Q49 pad 2: (no net) -> +12V
- Q49 pad 3: (no net) -> Net-(Q49-Pad3)
- Q49 pad 4: (no net) -> COL00
- Q49 pad 5: (no net) -> GND
- Q49 pad 6: (no net) -> COL00
- Q51 pad 1: (no net) -> Net-(Q51-Pad1)
- Q51 pad 2: (no net) -> +12V
- Q51 pad 3: (no net) -> Net-(Q51-Pad3)
- Q51 pad 4: (no net) -> COL02
- Q51 pad 5: (no net) -> GND
- Q51 pad 6: (no net) -> COL02
- Q52 pad 1: (no net) -> COL00_ON
- Q52 pad 2: (no net) -> GND
- Q52 pad 3: (no net) -> Net-(Q49-Pad3)
- Q54 pad 1: (no net) -> COL02_ON
- Q54 pad 2: (no net) -> GND
- Q54 pad 3: (no net) -> Net-(Q51-Pad3)
- Q55 pad 1: (no net) -> COL00_ON
- Q55 pad 2: (no net) -> GND
- Q55 pad 3: (no net) -> Net-(Q49-Pad1)
- Q57 pad 1: (no net) -> COL02_ON
- Q57 pad 2: (no net) -> GND
- Q57 pad 3: (no net) -> Net-(Q51-Pad1)
- Q58 pad 1: (no net) -> Net-(Q58-Pad1)
- Q58 pad 2: (no net) -> +12V
- Q58 pad 3: (no net) -> Net-(Q58-Pad3)
- Q58 pad 4: (no net) -> COL03
- Q58 pad 5: (no net) -> GND
- Q58 pad 6: (no net) -> COL03
- Q59 pad 1: (no net) -> Net-(Q59-Pad1)
- Q59 pad 2: (no net) -> +12V
- Q59 pad 3: (no net) -> Net-(Q59-Pad3)
- Q59 pad 4: (no net) -> COL04
- Q59 pad 5: (no net) -> GND
- Q59 pad 6: (no net) -> COL04
- Q60 pad 1: (no net) -> Net-(Q60-Pad1)
- Q60 pad 2: (no net) -> +12V
- Q60 pad 3: (no net) -> Net-(Q60-Pad3)
- Q60 pad 4: (no net) -> COL05
- Q60 pad 5: (no net) -> GND
- Q60 pad 6: (no net) -> COL05
- Q61 pad 1: (no net) -> COL03_ON
- Q61 pad 2: (no net) -> GND
- Q61 pad 3: (no net) -> Net-(Q58-Pad3)
- Q62 pad 1: (no net) -> COL04_ON
- Q62 pad 2: (no net) -> GND
- Q62 pad 3: (no net) -> Net-(Q59-Pad3)
- Q63 pad 1: (no net) -> COL05_ON
- Q63 pad 2: (no net) -> GND
- Q63 pad 3: (no net) -> Net-(Q60-Pad3)
- Q64 pad 1: (no net) -> COL03_ON
- Q64 pad 2: (no net) -> GND
- Q64 pad 3: (no net) -> Net-(Q58-Pad1)
- Q65 pad 1: (no net) -> COL04_ON
- Q65 pad 2: (no net) -> GND
- Q65 pad 3: (no net) -> Net-(Q59-Pad1)
- Q66 pad 1: (no net) -> COL05_ON
- Q66 pad 2: (no net) -> GND
- Q66 pad 3: (no net) -> Net-(Q60-Pad1)
- Q67 pad 1: (no net) -> Net-(Q67-Pad1)
- Q67 pad 2: (no net) -> +12V
- Q67 pad 3: (no net) -> Net-(Q67-Pad3)
- Q67 pad 4: (no net) -> COL06
- Q67 pad 5: (no net) -> GND
- Q67 pad 6: (no net) -> COL06
- Q68 pad 1: (no net) -> Net-(Q68-Pad1)
- Q68 pad 2: (no net) -> +12V
- Q68 pad 3: (no net) -> Net-(Q68-Pad3)
- Q68 pad 4: (no net) -> COL07
- Q68 pad 5: (no net) -> GND
- Q68 pad 6: (no net) -> COL07
- Q69 pad 1: (no net) -> Net-(Q69-Pad1)
- Q69 pad 2: (no net) -> +12V
- Q69 pad 3: (no net) -> Net-(Q69-Pad3)
- Q69 pad 4: (no net) -> COL08
- Q69 pad 5: (no net) -> GND
- Q69 pad 6: (no net) -> COL08
- Q70 pad 1: (no net) -> COL06_ON
- Q70 pad 2: (no net) -> GND
- Q70 pad 3: (no net) -> Net-(Q67-Pad3)
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Routing:
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- removed copper zone on F.Cu, net (none)

Commit message: automated commit
Parts:
- removed the Q17 at (492.7, -99.7)
- removed the Q20 at (151.9, 274.2)
- removed the Q22 at (85.7, 285.4)
- removed the Q24 at (115.5, 293.7)
- removed the Q26 at (124.0, 294.3)
- removed the Q28 at (145.1, 295.0)
- removed the Q30 at (124.0, 289.8)
- removed the Q32 at (141.0, 296.7)
- removed the Q34 at (172.6, 255.4)
- removed the Q36 at (184.3, 266.7)
- removed the Q38 at (167.2, 255.4)
- removed the Q40 at (188.3, 265.0)
- removed the Q42 at (167.2, 279.6)
- removed the Q44 at (192.7, 279.4)
- removed the Q46 at (167.2, 284.1)
- added D18: MMBZ5243BLT1G, Package_TO_SOT_SMD:SOT-23, F.Cu at (476.8, -117.4)
- added D19: MMBZ5243BLT1G, Package_TO_SOT_SMD:SOT-23, F.Cu at (517.0, -7.18)
- added D20: MMBZ5243BLT1G, Package_TO_SOT_SMD:SOT-23, F.Cu at (480.3, -117.4)
- added D21: MMBZ5243BLT1G, Package_TO_SOT_SMD:SOT-23, F.Cu at (522.4, -11.6)
- added D22: MMBZ5243BLT1G, Package_TO_SOT_SMD:SOT-23, B.Cu at (482.9, -107.6)
- added D23: MMBZ5243BLT1G, Package_TO_SOT_SMD:SOT-23, F.Cu at (533.1, -117.4)
- added D24: MMBZ5243BLT1G, Package_TO_SOT_SMD:SOT-23, B.Cu at (479.4, -107.6)
- added D25: MMBZ5243BLT1G, Package_TO_SOT_SMD:SOT-23, F.Cu at (536.7, -117.4)
- added D26: MMBZ5243BLT1G, Package_TO_SOT_SMD:SOT-23, F.Cu at (484.8, -117.4)
- added D27: MMBZ5243BLT1G, Package_TO_SOT_SMD:SOT-23, B.Cu at (531.2, -107.6)
- added D28: MMBZ5243BLT1G, Package_TO_SOT_SMD:SOT-23, F.Cu at (488.4, -117.4)
- added D29: MMBZ5243BLT1G, Package_TO_SOT_SMD:SOT-23, B.Cu at (527.7, -107.6)
- added D30: MMBZ5243BLT1G, Package_TO_SOT_SMD:SOT-23, B.Cu at (491.0, -107.6)
- added D31: MMBZ5243BLT1G, Package_TO_SOT_SMD:SOT-23, F.Cu at (525.1, -117.4)
- added D32: MMBZ5243BLT1G, Package_TO_SOT_SMD:SOT-23, B.Cu at (487.4, -107.6)
- added D33: MMBZ5243BLT1G, Package_TO_SOT_SMD:SOT-23, F.Cu at (528.6, -117.4)
- added D34: MMBZ5243BLT1G, Package_TO_SOT_SMD:SOT-23, F.Cu at (492.9, -117.4)
- added D35: MMBZ5243BLT1G, Package_TO_SOT_SMD:SOT-23, B.Cu at (523.2, -107.6)
- added D36: MMBZ5243BLT1G, Package_TO_SOT_SMD:SOT-23, F.Cu at (496.4, -117.4)
- added D37: MMBZ5243BLT1G, Package_TO_SOT_SMD:SOT-23, B.Cu at (519.6, -107.6)
- added D38: MMBZ5243BLT1G, Package_TO_SOT_SMD:SOT-23, B.Cu at (499.0, -107.6)
- added D39: MMBZ5243BLT1G, Package_TO_SOT_SMD:SOT-23, F.Cu at (517.0, -117.4)
- added D40: MMBZ5243BLT1G, Package_TO_SOT_SMD:SOT-23, B.Cu at (495.5, -107.6)
- added D41: MMBZ5243BLT1G, Package_TO_SOT_SMD:SOT-23, F.Cu at (520.6, -117.4)
- added D42: MMBZ5243BLT1G, Package_TO_SOT_SMD:SOT-23, F.Cu at (500.9, -117.4)
- added D43: MMBZ5243BLT1G, Package_TO_SOT_SMD:SOT-23, B.Cu at (515.1, -107.6)
- added D44: MMBZ5243BLT1G, Package_TO_SOT_SMD:SOT-23, F.Cu at (504.5, -117.4)
- added D45: MMBZ5243BLT1G, Package_TO_SOT_SMD:SOT-23, B.Cu at (511.6, -107.6)
- added D46: MMBZ5243BLT1G, Package_TO_SOT_SMD:SOT-23, B.Cu at (507.1, -107.6)
- added D47: MMBZ5243BLT1G, Package_TO_SOT_SMD:SOT-23, F.Cu at (509.0, -117.4)
- added D48: MMBZ5243BLT1G, Package_TO_SOT_SMD:SOT-23, B.Cu at (503.5, -107.6)
- added D49: MMBZ5243BLT1G, Package_TO_SOT_SMD:SOT-23, F.Cu at (512.5, -117.4)
- added Q16: DMG6602, Package_TO_SOT_SMD:TSOT-23-6, F.Cu at (478.5, -121.3)
- added Q17: DMG6602, Package_TO_SOT_SMD:TSOT-23-6, B.Cu at (537.5, -111.5)
- added Q17: DMG6602, Package_TO_SOT_SMD:TSOT-23-6, F.Cu at (517.5, -11.7)
- added Q18: SSM3K35AMFV, Package_TO_SOT_SMD:SOT-723, F.Cu at (475.9, -122.5)
- added Q19: SSM3K35AMFV, Package_TO_SOT_SMD:SOT-723, F.Cu at (528.7, -9.97)
- added Q20: DMG6602, Package_TO_SOT_SMD:TSOT-23-6, B.Cu at (481.2, -111.6)
- added Q20: DMG6602, Package_TO_SOT_SMD:TSOT-23-6, F.Cu at (152.3, 272.4)
- added Q21: DMG6602, Package_TO_SOT_SMD:TSOT-23-6, F.Cu at (534.9, -121.3)
- added Q22: SSM3K35AMFV, Package_TO_SOT_SMD:SOT-723, B.Cu at (483.8, -112.8)
- added Q22: SSM3K35AMFV, Package_TO_SOT_SMD:SOT-723, F.Cu at (85.7, 285.4)
- added Q23: SSM3K35AMFV, Package_TO_SOT_SMD:SOT-723, F.Cu at (532.2, -122.6)
- added Q24: DMG6602, Package_TO_SOT_SMD:TSOT-23-6, F.Cu at (486.6, -121.3)
- added Q24: DMG6602, Package_TO_SOT_SMD:TSOT-23-6, F.Cu at (115.5, 293.7)
- added Q25: DMG6602, Package_TO_SOT_SMD:TSOT-23-6, B.Cu at (529.5, -111.5)
- added Q26: SSM3K35AMFV, Package_TO_SOT_SMD:SOT-723, F.Cu at (483.9, -122.5)
- added Q26: SSM3K35AMFV, Package_TO_SOT_SMD:SOT-723, F.Cu at (124.0, 294.3)
- added Q27: SSM3K35AMFV, Package_TO_SOT_SMD:SOT-723, B.Cu at (532.1, -112.8)
- added Q28: DMG6602, Package_TO_SOT_SMD:TSOT-23-6, B.Cu at (489.2, -111.5)
- added Q28: DMG6602, Package_TO_SOT_SMD:TSOT-23-6, F.Cu at (145.1, 295.0)
- added Q29: DMG6602, Package_TO_SOT_SMD:TSOT-23-6, F.Cu at (526.8, -121.3)
- added Q30: SSM3K35AMFV, Package_TO_SOT_SMD:SOT-723, B.Cu at (491.9, -112.8)
- added Q30: SSM3K35AMFV, Package_TO_SOT_SMD:SOT-723, F.Cu at (124.0, 289.8)
- added Q31: SSM3K35AMFV, Package_TO_SOT_SMD:SOT-723, F.Cu at (524.2, -122.6)
- added Q32: DMG6602, Package_TO_SOT_SMD:TSOT-23-6, F.Cu at (494.6, -121.3)
- added Q32: DMG6602, Package_TO_SOT_SMD:TSOT-23-6, F.Cu at (141.0, 296.7)
- added Q33: DMG6602, Package_TO_SOT_SMD:TSOT-23-6, B.Cu at (521.4, -111.5)
- added Q34: SSM3K35AMFV, Package_TO_SOT_SMD:SOT-723, F.Cu at (492.0, -122.5)
- added Q34: SSM3K35AMFV, Package_TO_SOT_SMD:SOT-723, F.Cu at (172.6, 255.4)
- added Q35: SSM3K35AMFV, Package_TO_SOT_SMD:SOT-723, B.Cu at (524.1, -112.8)
- added Q36: DMG6602, Package_TO_SOT_SMD:TSOT-23-6, B.Cu at (497.3, -111.5)
- added Q36: DMG6602, Package_TO_SOT_SMD:TSOT-23-6, F.Cu at (184.3, 266.7)
- added Q37: DMG6602, Package_TO_SOT_SMD:TSOT-23-6, F.Cu at (518.8, -121.3)
- added Q38: SSM3K35AMFV, Package_TO_SOT_SMD:SOT-723, B.Cu at (499.9, -112.8)
- added Q38: SSM3K35AMFV, Package_TO_SOT_SMD:SOT-723, F.Cu at (167.2, 255.4)
- added Q39: SSM3K35AMFV, Package_TO_SOT_SMD:SOT-723, F.Cu at (516.1, -122.6)
- added Q40: DMG6602, Package_TO_SOT_SMD:TSOT-23-6, F.Cu at (502.7, -121.3)
- added Q40: DMG6602, Package_TO_SOT_SMD:TSOT-23-6, F.Cu at (188.3, 265.0)
- added Q41: DMG6602, Package_TO_SOT_SMD:TSOT-23-6, B.Cu at (513.3, -111.5)
- added Q42: SSM3K35AMFV, Package_TO_SOT_SMD:SOT-723, F.Cu at (500.0, -122.5)
- added Q42: SSM3K35AMFV, Package_TO_SOT_SMD:SOT-723, F.Cu at (167.2, 279.6)
- added Q43: SSM3K35AMFV, Package_TO_SOT_SMD:SOT-723, B.Cu at (516.0, -112.8)
- added Q44: DMG6602, TSOT-23-6, B.Cu at (505.3, -111.5)
- added Q44: DMG6602, TSOT-23-6, F.Cu at (192.7, 279.4)
- added Q45: DMG6602, Package_TO_SOT_SMD:TSOT-23-6, F.Cu at (510.7, -121.3)
- added Q46: SSM3K35AMFV, Package_TO_SOT_SMD:SOT-723, B.Cu at (508.0, -112.8)
- added Q46: SSM3K35AMFV, Package_TO_SOT_SMD:SOT-723, F.Cu at (167.2, 284.1)
- added Q47: SSM3K35AMFV, Package_TO_SOT_SMD:SOT-723, F.Cu at (508.1, -122.6)
- added R100: CRG0603F4K7, Resistor_SMD:R_0603_1608Metric, B.Cu at (482.3, -114.5)
- added R101: CRG0603F4K7, Resistor_SMD:R_0603_1608Metric, F.Cu at (533.7, -124.3)
- added R102: CRG0603F4K7, Resistor_SMD:R_0603_1608Metric, B.Cu at (484.4, -111.1)
- added R103: CRG0603F4K7, Resistor_SMD:R_0603_1608Metric, F.Cu at (531.6, -120.9)
- added R104: CRG0603F4K7, Resistor_SMD:R_0603_1608Metric, B.Cu at (478.7, -112.2)
- added R105: CRG0603F4K7, Resistor_SMD:R_0603_1608Metric, F.Cu at (537.4, -122.0)
- added R106: CRG0603F4K7, Resistor_SMD:R_0603_1608Metric, F.Cu at (485.5, -124.3)
- added R107: CRG0603F4K7, Resistor_SMD:R_0603_1608Metric, B.Cu at (530.6, -114.5)
- added R108: CRG0603F4K7, Resistor_SMD:R_0603_1608Metric, F.Cu at (483.4, -120.8)
- added R109: CRG0603F4K7, Resistor_SMD:R_0603_1608Metric, B.Cu at (532.7, -111.1)
- added R110: CRG0603F4K7, Resistor_SMD:R_0603_1608Metric, F.Cu at (489.1, -122.0)
- added R111: CRG0603F4K7, Resistor_SMD:R_0603_1608Metric, B.Cu at (526.9, -112.2)
- added R112: CRG0603F4K7, Resistor_SMD:R_0603_1608Metric, B.Cu at (490.3, -114.5)
- added R113: CRG0603F4K7, Resistor_SMD:R_0603_1608Metric, F.Cu at (525.7, -124.3)
- added R114: CRG0603F4K7, Resistor_SMD:R_0603_1608Metric, B.Cu at (492.4, -111.1)
- added R115: CRG0603F4K7, Resistor_SMD:R_0603_1608Metric, F.Cu at (523.6, -120.9)
- added R116: CRG0603F4K7, Resistor_SMD:R_0603_1608Metric, B.Cu at (486.7, -112.2)
- added R117: CRG0603F4K7, Resistor_SMD:R_0603_1608Metric, F.Cu at (529.4, -122.0)
- added R118: CRG0603F4K7, Resistor_SMD:R_0603_1608Metric, F.Cu at (493.5, -124.3)
- added R119: CRG0603F4K7, Resistor_SMD:R_0603_1608Metric, B.Cu at (522.5, -114.5)
- added R120: CRG0603F4K7, Resistor_SMD:R_0603_1608Metric, F.Cu at (491.4, -120.8)
- added R121: CRG0603F4K7, Resistor_SMD:R_0603_1608Metric, B.Cu at (524.6, -111.1)
- added R122: CRG0603F4K7, Resistor_SMD:R_0603_1608Metric, F.Cu at (497.2, -122.0)
- added R123: CRG0603F4K7, Resistor_SMD:R_0603_1608Metric, B.Cu at (518.9, -112.2)
- added R124: CRG0603F4K7, Resistor_SMD:R_0603_1608Metric, B.Cu at (498.4, -114.5)
- added R125: CRG0603F4K7, Resistor_SMD:R_0603_1608Metric, F.Cu at (517.7, -124.3)
- added R126: CRG0603F4K7, Resistor_SMD:R_0603_1608Metric, B.Cu at (500.5, -111.1)
- added R127: CRG0603F4K7, Resistor_SMD:R_0603_1608Metric, F.Cu at (515.5, -120.9)
- added R128: CRG0603F4K7, Resistor_SMD:R_0603_1608Metric, B.Cu at (494.7, -112.2)
- added R129: CRG0603F4K7, Resistor_SMD:R_0603_1608Metric, F.Cu at (521.3, -122.0)
- added R130: CRG0603F4K7, Resistor_SMD:R_0603_1608Metric, F.Cu at (501.6, -124.3)
- added R131: CRG0603F4K7, Resistor_SMD:R_0603_1608Metric, B.Cu at (514.5, -114.5)
- added R132: CRG0603F4K7, Resistor_SMD:R_0603_1608Metric, F.Cu at (499.5, -120.8)
- added R133: CRG0603F4K7, Resistor_SMD:R_0603_1608Metric, B.Cu at (516.6, -111.1)
- added R134: CRG0603F4K7, Resistor_SMD:R_0603_1608Metric, F.Cu at (505.2, -122.0)
- added R135: CRG0603F4K7, Resistor_SMD:R_0603_1608Metric, B.Cu at (510.8, -112.2)
- added R136: CRG0603F4K7, Resistor_SMD:R_0603_1608Metric, B.Cu at (506.4, -114.5)
- added R137: CRG0603F4K7, Resistor_SMD:R_0603_1608Metric, F.Cu at (509.6, -124.3)
- added R138: CRG0603F4K7, Resistor_SMD:R_0603_1608Metric, B.Cu at (508.5, -111.1)
- added R139: CRG0603F4K7, Resistor_SMD:R_0603_1608Metric, F.Cu at (507.5, -120.8)
- added R140: CRG0603F4K7, Resistor_SMD:R_0603_1608Metric, B.Cu at (502.8, -112.2)
- added R141: CRG0603F4K7, Resistor_SMD:R_0603_1608Metric, F.Cu at (513.3, -122.0)
- added R94: CRG0603F4K7, Resistor_SMD:R_0603_1608Metric, F.Cu at (477.4, -124.3)
- added R95: CRG0603F4K7, Resistor_SMD:R_0603_1608Metric, F.Cu at (521.3, -8.10)
- added R96: CRG0603F4K7, Resistor_SMD:R_0603_1608Metric, F.Cu at (475.3, -120.8)
- added R97: CRG0603F4K7, Resistor_SMD:R_0603_1608Metric, F.Cu at (526.7, -12.6)
- added R98: CRG0603F4K7, Resistor_SMD:R_0603_1608Metric, F.Cu at (481.1, -122.0)
- added R99: CRG0603F4K7, Resistor_SMD:R_0603_1608Metric, F.Cu at (525.3, -8.10)
- D19, D21, Q19, R95, R97, R99, U10, U12: moved to B.Cu
- Q102, Q111, Q120, Q129, Q48, Q57, Q66, Q75, Q84, Q93: value SSM3K35AMFV -> DMG6602; footprint Package_TO_SOT_SMD:SOT-723 -> Package_TO_SOT_SMD:TSOT-23-6
- Q105, Q114, Q123, Q130, Q51, Q60, Q69, Q78, Q87, Q96: value DMG6602 -> SSM3K35AMFV; footprint Package_TO_SOT_SMD:TSOT-23-6 -> Package_TO_SOT_SMD:SOT-723
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Connections:
- Q100 pad 1: COL15_ON -> COL16_ON
- Q101 pad 1: COL16_ON -> COL17_ON
- Q102 pad 1: COL17_ON -> Net-(Q102-Pad1)
- Q102 pad 2: GND -> +12V
- Q103 pad 4: COL18 -> COL19
- Q103 pad 6: COL18 -> COL19
- Q104 pad 4: COL19 -> COL20
- Q104 pad 6: COL19 -> COL20
- Q105 pad 1: Net-(Q105-Pad1) -> COL18_ON
- Q105 pad 2: +12V -> GND
- Q105 pad 3: Net-(Q105-Pad3) -> Net-(Q102-Pad3)
- Q106 pad 1: COL18_ON -> COL19_ON
- Q107 pad 1: COL19_ON -> COL20_ON
- Q108 pad 1: COL20_ON -> COL18_ON
- Q108 pad 3: Net-(Q105-Pad3) -> Net-(Q102-Pad1)
- Q109 pad 1: COL18_ON -> COL19_ON
- Q110 pad 1: COL19_ON -> COL20_ON
- Q111 pad 1: COL20_ON -> Net-(Q111-Pad1)
- Q111 pad 2: GND -> +12V
- Q111 pad 3: Net-(Q105-Pad1) -> Net-(Q111-Pad3)
- Q112 pad 4: COL21 -> COL22
- Q112 pad 6: COL21 -> COL22
- Q113 pad 4: COL22 -> COL23
- Q113 pad 6: COL22 -> COL23
- Q114 pad 1: Net-(Q114-Pad1) -> COL21_ON
- Q114 pad 2: +12V -> GND
- Q114 pad 3: Net-(Q114-Pad3) -> Net-(Q111-Pad3)
- Q115 pad 1: COL21_ON -> COL22_ON
- Q116 pad 1: COL22_ON -> COL23_ON
- Q117 pad 1: COL23_ON -> COL21_ON
- Q117 pad 3: Net-(Q114-Pad3) -> Net-(Q111-Pad1)
- Q118 pad 1: COL21_ON -> COL22_ON
- Q119 pad 1: COL22_ON -> COL23_ON
- Q120 pad 1: COL23_ON -> Net-(Q120-Pad1)
- Q120 pad 2: GND -> +12V
- Q120 pad 3: Net-(Q114-Pad1) -> Net-(Q120-Pad3)
- Q121 pad 4: COL24 -> COL25
- Q121 pad 6: COL24 -> COL25
- Q122 pad 4: COL25 -> COL26
- Q122 pad 6: COL25 -> COL26
- Q123 pad 1: Net-(Q123-Pad1) -> COL24_ON
- Q123 pad 2: +12V -> GND
- Q123 pad 3: Net-(Q123-Pad3) -> Net-(Q120-Pad3)
- Q124 pad 1: COL24_ON -> COL25_ON
- Q125 pad 1: COL25_ON -> COL26_ON
- Q126 pad 1: COL26_ON -> COL24_ON
- Q126 pad 3: Net-(Q123-Pad3) -> Net-(Q120-Pad1)
- Q127 pad 1: COL24_ON -> COL25_ON
- Q128 pad 1: COL25_ON -> COL26_ON
- Q129 pad 1: COL26_ON -> Net-(Q129-Pad1)
- Q129 pad 2: GND -> +12V
- Q129 pad 3: Net-(Q123-Pad1) -> Net-(Q129-Pad3)
- Q130 pad 1: Net-(Q130-Pad1) -> COL27_ON
- Q130 pad 2: +12V -> GND
- Q130 pad 3: Net-(Q130-Pad3) -> Net-(Q129-Pad3)
- Q131 pad 3: Net-(Q130-Pad3) -> Net-(Q129-Pad1)
- Q16 pad 1: Net-(Q16-Pad1) -> ROW00_OFF
- Q21 pad 1: ROW02_OFF -> ROW03_OFF
- Q21 pad 4: ROW02P -> ROW03P
- Q21 pad 6: ROW02N -> ROW03N
- Q23 pad 1: ROW02_ON -> ROW03_ON
- Q25 pad 1: ROW04_OFF -> ROW05_OFF
- Q25 pad 4: ROW04P -> ROW05P
- Q25 pad 6: ROW04N -> ROW05N
- Q27 pad 1: ROW04_ON -> ROW05_ON
- Q29 pad 1: ROW06_OFF -> ROW07_OFF
- Q29 pad 4: ROW06P -> ROW07P
- Q29 pad 6: ROW06N -> ROW07N
- Q31 pad 1: ROW06_ON -> ROW07_ON
- Q33 pad 1: ROW08_OFF -> ROW09_OFF
- Q33 pad 4: ROW08P -> ROW09P
- Q33 pad 6: ROW08N -> ROW09N
- Q35 pad 1: ROW08_ON -> ROW09_ON
- Q37 pad 1: ROW10_OFF -> ROW11_OFF
- Q37 pad 4: ROW10P -> ROW11P
- Q37 pad 6: ROW10N -> ROW11N
- Q39 pad 1: ROW10_ON -> ROW11_ON
- Q41 pad 1: ROW12_OFF -> ROW13_OFF
- Q41 pad 4: ROW12P -> ROW13P
- Q41 pad 6: ROW12N -> ROW13N
- Q43 pad 1: ROW12_ON -> ROW13_ON
- Q45 pad 1: ROW14_OFF -> ROW15_OFF
- Q45 pad 4: ROW14P -> ROW15P
- Q45 pad 6: ROW14N -> ROW15N
- Q47 pad 1: ROW14_ON -> ROW15_ON
- Q48 pad 1: ROW15_ON -> Net-(Q48-Pad1)
- Q48 pad 2: GND -> +12V
- Q48 pad 3: Net-(Q46-Pad3) -> Net-(Q48-Pad3)
- Q49 pad 4: COL00 -> COL01
- Q49 pad 6: COL00 -> COL01
- Q50 pad 4: COL01 -> COL02
- Q50 pad 6: COL01 -> COL02
- Q51 pad 1: Net-(Q51-Pad1) -> COL00_ON
- Q51 pad 2: +12V -> GND
- Q51 pad 3: Net-(Q51-Pad3) -> Net-(Q48-Pad3)
- Q52 pad 1: COL00_ON -> COL01_ON
- Q53 pad 1: COL01_ON -> COL02_ON
- Q54 pad 1: COL02_ON -> COL00_ON
- Q54 pad 3: Net-(Q51-Pad3) -> Net-(Q48-Pad1)
- Q55 pad 1: COL00_ON -> COL01_ON
- Q56 pad 1: COL01_ON -> COL02_ON
- Q57 pad 1: COL02_ON -> Net-(Q57-Pad1)
- Q57 pad 2: GND -> +12V
- Q57 pad 3: Net-(Q51-Pad1) -> Net-(Q57-Pad3)
- Q58 pad 4: COL03 -> COL04
- Q58 pad 6: COL03 -> COL04
- Q59 pad 4: COL04 -> COL05
- Q59 pad 6: COL04 -> COL05
- Q60 pad 1: Net-(Q60-Pad1) -> COL03_ON
- Q60 pad 2: +12V -> GND
- Q60 pad 3: Net-(Q60-Pad3) -> Net-(Q57-Pad3)
- Q61 pad 1: COL03_ON -> COL04_ON
- Q62 pad 1: COL04_ON -> COL05_ON
- Q63 pad 1: COL05_ON -> COL03_ON
- Q63 pad 3: Net-(Q60-Pad3) -> Net-(Q57-Pad1)
- Q64 pad 1: COL03_ON -> COL04_ON
- Q65 pad 1: COL04_ON -> COL05_ON
- Q66 pad 1: COL05_ON -> Net-(Q66-Pad1)
- Q66 pad 2: GND -> +12V
- Q66 pad 3: Net-(Q60-Pad1) -> Net-(Q66-Pad3)
- Q67 pad 4: COL06 -> COL07
- Q67 pad 6: COL06 -> COL07
- Q68 pad 4: COL07 -> COL08
- Q68 pad 6: COL07 -> COL08
- Q69 pad 1: Net-(Q69-Pad1) -> COL06_ON
- Q69 pad 2: +12V -> GND
- Q69 pad 3: Net-(Q69-Pad3) -> Net-(Q66-Pad3)
- Q70 pad 1: COL06_ON -> COL07_ON
- Q71 pad 1: COL07_ON -> COL08_ON
- Q72 pad 1: COL08_ON -> COL06_ON
- Q72 pad 3: Net-(Q69-Pad3) -> Net-(Q66-Pad1)
- Q73 pad 1: COL06_ON -> COL07_ON
- Q74 pad 1: COL07_ON -> COL08_ON
- Q75 pad 1: COL08_ON -> Net-(Q75-Pad1)
- Q75 pad 2: GND -> +12V
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Routing:
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
Commit message: automated commit
Parts:
- removed the D18 at (151.7, 262.5)
- removed the D20 at (154.7, 278.5)
- removed the D22 at (100.5, 285.4)
- removed the D23 at (89.7, 299.0)
- removed the D24 at (99.6, 290.0)
- removed the D25 at (90.7, 289.9)
- removed the D26 at (143.2, 285.4)
- removed the D27 at (133.4, 294.5)
- removed the D28 at (137.8, 290.0)
- removed the D29 at (138.8, 285.4)
- removed the D30 at (133.4, 290.0)
- removed the D31 at (128.9, 294.4)
- removed the D32 at (134.3, 285.4)
- removed the D33 at (128.9, 289.9)
- removed the D34 at (172.1, 259.9)
- removed the D35 at (177.5, 255.5)
- removed the D36 at (172.1, 264.5)
- removed the D37 at (176.6, 260.0)
- removed the D38 at (181.0, 260.0)
- removed the D39 at (176.6, 264.6)
- removed the D40 at (186.4, 255.5)
- removed the D41 at (182.0, 255.5)
- removed the D42 at (182.0, 275.2)
- removed the D43 at (181.0, 279.8)
- removed the D44 at (176.6, 284.3)
- removed the D45 at (186.4, 275.2)
- removed the D46 at (177.5, 275.2)
- removed the D47 at (172.1, 279.7)
- removed the D48 at (172.1, 284.2)
- removed the D49 at (176.6, 279.8)
- removed the Q16 at (147.2, 258.0)
- removed the Q18 at (146.0, 260.7)
- removed the Q20 at (152.3, 272.4)
- removed the Q21 at (85.7, 294.3)
- removed the Q22 at (85.7, 285.4)
- removed the Q23 at (112.6, 296.8)
- removed the Q24 at (115.5, 293.7)
- removed the Q25 at (129.4, 285.4)
- removed the Q26 at (124.0, 294.3)
- removed the Q27 at (145.5, 292.1)
- removed the Q28 at (145.1, 295.0)
- removed the Q29 at (124.0, 285.4)
- removed the Q30 at (124.0, 289.8)
- removed the Q31 at (149.5, 289.6)
- removed the Q32 at (141.0, 296.7)
- removed the Q33 at (167.2, 264.3)
- removed the Q34 at (172.6, 255.4)
- removed the Q35 at (188.7, 262.2)
- removed the Q36 at (184.3, 266.7)
- removed the Q37 at (167.2, 259.9)
- removed the Q38 at (167.2, 255.4)
- removed the Q39 at (192.7, 259.6)
- removed the Q40 at (188.3, 265.0)
- removed the Q41 at (167.2, 275.2)
- removed the Q42 at (167.2, 279.6)
- removed the Q43 at (188.3, 284.7)
- removed the Q44 at (192.7, 279.4)
- removed the Q45 at (172.6, 275.2)
- removed the Q46 at (167.2, 284.1)
- removed the Q47 at (184.3, 286.4)
- removed the R100 at (144.6, 278.8)
- removed the R101 at (108.7, 284.4)
- removed the R102 at (94.9, 293.5)
- removed the R103 at (112.8, 284.4)
- removed the R104 at (102.9, 293.5)
- removed the R105 at (98.9, 296.0)
- removed the R106 at (94.0, 301.1)
- removed the R107 at (127.3, 298.0)
- removed the R108 at (137.6, 293.5)
- removed the R109 at (142.1, 289.0)
- removed the R110 at (131.3, 298.1)
- removed the R111 at (123.3, 297.8)
- removed the R112 at (147.5, 284.4)
- removed the R113 at (137.6, 296.0)
- removed the R114 at (142.1, 291.5)
- removed the R115 at (146.1, 289.4)
- removed the R116 at (147.5, 286.9)
- removed the R117 at (135.4, 298.5)
- removed the R118 at (141.6, 294.0)
- removed the R119 at (180.8, 263.6)
- removed the R120 at (170.5, 268.0)
- removed the R121 at (190.7, 257.0)
- removed the R122 at (178.6, 268.6)
- removed the R123 at (185.3, 259.0)
- removed the R124 at (166.5, 267.8)
- removed the R125 at (190.7, 254.5)
- removed the R126 at (184.8, 264.0)
- removed the R127 at (189.3, 259.5)
- removed the R128 at (494.7, -112.2)
- removed the R128 at (180.8, 266.1)
- removed the R129 at (185.3, 261.5)
- removed the R130 at (174.6, 268.1)
- removed the R131 at (189.3, 279.2)
- removed the R132 at (170.5, 287.7)
- removed the R133 at (178.6, 288.3)
- removed the R134 at (190.7, 276.7)
- removed the R135 at (185.3, 281.2)
- removed the R136 at (180.8, 285.8)
- removed the R137 at (190.7, 274.2)
- removed the R138 at (174.6, 287.8)
- removed the R139 at (185.3, 278.7)
- removed the R140 at (180.8, 283.3)
- removed the R141 at (166.5, 287.5)
- removed the R94 at (144.3, 259.0)
- removed the R96 at (143.5, 264.3)
- removed the R98 at (148.3, 244.1)
- removed TP92: TestPoint, custom:TestPoint_THTPad_D1.0mm_Drill0.5mm
- added R128: CRG0603F4K7, Resistor_SMD:R_0603_1608Metric, B.Cu at (493.1, -109.1)
- moved C62 546.8 mm to (495.2, -134.7), turned to 90 degrees
- moved C59 545.6 mm to (507.9, -135.5)
- moved C61 545.5 mm to (507.9, -138.5)
- moved C63 543.4 mm to (493.6, -134.7), turned to 90 degrees
- moved C64 542.7 mm to (492.1, -134.7), turned to 90 degrees
- moved C60 542.1 mm to (507.8, -137.0)
- moved R61 130.7 mm to (259.3, 282.1)
- moved R14 129.9 mm to (229.1, 242.8)
- moved C13 129.7 mm to (230.1, 247.8)
- moved TP78 126.2 mm to (232.8, 301.8)
- moved C11 126.0 mm to (230.1, 245.3)
- moved R15 122.8 mm to (226.1, 245.3)
- moved C16 121.0 mm to (220.9, 243.0)
- moved D11 120.7 mm to (258.9, 258.8)
- moved SW6 119.1 mm to (256.7, 249.5)
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Routing:
- net ROW03N: track 3.67 -> 50.5 mm, vias 0 -> 2
- net ROW07N: track 3.67 -> 48.5 mm, vias 0 -> 2
- net ROW11N: track 3.67 -> 45.1 mm, vias 1 -> 3
- net ROW01_ON: track 1.53 -> 42.1 mm, vias 0 -> 1
- net ROW02_OFF: track 1.64 -> 40.0 mm
- net ROW15N: track 3.67 -> 41.6 mm, vias 0 -> 2
- net ROW03P: track 3.67 -> 41.2 mm, vias 0 -> 1
- net ROW02_ON: track 1.53 -> 38.9 mm, vias 0 -> 1
- net ROW01_OFF: track 1.64 -> 38.4 mm
- net ROW01N: track 3.67 -> 39.6 mm, vias 0 -> 2
- net ROW00_ON: track 1.53 -> 37.3 mm
- net ROW12N: track 3.67 -> 38.4 mm, vias 0 -> 2
- net ROW05_ON: track 1.53 -> 35.6 mm, vias 0 -> 1
- net ROW07P: track 3.67 -> 37.7 mm, vias 0 -> 1
- net ROW08N: track 3.67 -> 37.2 mm, vias 0 -> 2
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- added copper zone on F.Cu, net IVDD_FE310

Commit message: automated commit
Parts:
- removed the D19 at (517.0, -7.18)
- removed the D21 at (522.4, -11.6)
- removed Q132: SSM3K35AMFV, Package_TO_SOT_SMD:SOT-723
- removed the Q17 at (517.5, -11.7)
- removed the Q19 at (528.7, -9.97)
- removed R254: CRG0603F4K7, Resistor_SMD:R_0603_1608Metric
- removed the R95 at (521.3, -8.10)
- removed the R97 at (526.7, -12.6)
- removed the R99 at (525.3, -8.10)
- added U5: IS25LP128-JBLE, Package_SO:SOIC-8_3.9x4.9mm_P1.27mm, F.Cu at (443.1, 294.9)
- added U8: FT2232D, Package_QFP:LQFP-48_7x7mm_P0.5mm, F.Cu at (537.7, 275.4)
- Q100, Q102, Q104, Q107, Q112, Q115, Q118, Q120, Q122, Q125, Q128, Q49, Q52, Q55, Q57, Q59, Q62, Q65, Q67, Q70, Q73, Q75, Q77, Q80, Q83, Q85, Q88, Q91, Q94, Q97, R143, R146, R150, R154, R156, R159, R164, R167, R170, R174, R178, R180, R183, R188, R191, R194, R198, R203, R206, R210, R214, R216, R219, R224, R227, R230, R234, R238, R240, R243, R248: moved to F.Cu
- Q101, Q103, Q106, Q109, Q111, Q113, Q116, Q119, Q121, Q124, Q127, Q129, Q48, Q50, Q53, Q56, Q58, Q61, Q64, Q66, Q68, Q71, Q74, Q76, Q79, Q82, Q84, Q87, Q90, Q93, Q95, Q98, R142, R144, R147, R152, R155, R158, R162, R166, R168, R171, R176, R179, R182, R186, R190, R193, R196, R202, R204, R207, R212, R215, R218, R222, R226, R228, R231, R236, R239, R242, R246, R250: moved to B.Cu
- moved C66 554.1 mm to (502.4, 307.1)
- moved C67 552.8 mm to (498.3, 309.6)
- moved C65 547.9 mm to (494.3, 309.6)
- moved C75 547.0 mm to (502.4, 304.6)
- moved C82 538.5 mm to (498.3, 304.6)
- moved C80 538.1 mm to (502.4, 299.5)
- moved C68 536.8 mm to (506.4, 302.0)
- moved C74 536.8 mm to (494.3, 299.5)
- moved C76 536.1 mm to (490.3, 302.0)
- moved C81 535.5 mm to (494.3, 307.1)
- moved C70 528.8 mm to (498.3, 307.1)
- moved C85 525.5 mm to (506.4, 299.5)
- moved C53 525.0 mm to (525.8, 302.0)
- moved C83 522.4 mm to (502.4, 302.0)
- moved C78 521.6 mm to (498.3, 302.0)
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Routing:
- net (no net): track 10.2 -> 0.00 mm, vias 0 -> 1
- net Net-(Q60-Pad3): track 7.13 -> 0.00 mm
- net Net-(Q114-Pad3): track 7.13 -> 0.00 mm
- net Net-(Q93-Pad3): track 0.00 -> 7.13 mm
- net Net-(Q84-Pad3): track 0.00 -> 7.13 mm
- net Net-(Q77-Pad3): track 0.00 -> 7.13 mm
- net Net-(Q69-Pad3): track 7.13 -> 0.00 mm
- net Net-(Q57-Pad3): track 0.00 -> 7.13 mm
- net Net-(Q120-Pad3): track 0.00 -> 7.13 mm
- net Net-(Q111-Pad3): track 0.00 -> 7.13 mm
- net Net-(Q48-Pad3): track 0.00 -> 7.13 mm
- net Net-(Q96-Pad3): track 7.13 -> 0.00 mm
- net Net-(Q78-Pad3): track 7.13 -> 0.00 mm
- net Net-(Q66-Pad3): track 0.00 -> 7.13 mm
- net Net-(Q87-Pad3): track 7.13 -> 0.00 mm
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- added copper zone on F.Cu, net (none)
