File: flipdot_driver.kicad_pcb (KiCad board)
At the start: 4 copper layers, 661 parts, among them J1 Barrel_Jack, J10 Conn_01x08_Male, J11 3x32_1&3_loaded_2.5mm_0.1in_f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, J2 Screw_Terminal_01x04, J3 PTH_1.5_mm, J4 PTH_1.5_mm, J5 PTH_1.5_mm, J6 PTH_1.5_mm, J7 Conn_01x05_Male, J8 PTH_1.5_mm, J9 USB-C_2.0_Connector, Q1 SSM3K35AMFV, Q10 SSM3K35AMFV, Q100 SSM3K35AMFV, Q101 SSM3K35AMFV, Q102 DMG6602, Q103 DMG6602, Q104 DMG6602, Q105 SSM3K35AMFV, Q106 SSM3K35AMFV, Q107 SSM3K35AMFV, Q108 SSM3K35AMFV, Q109 SSM3K35AMFV, Q11 SSM3K35AMFV, Q110 SSM3K35AMFV, Q111 DMG6602, Q112 DMG6602, Q113 DMG6602, Q114 SSM3K35AMFV, Q115 SSM3K35AMFV, Q116 SSM3K35AMFV, Q117 SSM3K35AMFV, Q118 SSM3K35AMFV, Q119 SSM3K35AMFV, Q12 AO3407A, Q120 DMG6602, Q121 DMG6602, Q122 DMG6602, Q123 SSM3K35AMFV, Q124 SSM3K35AMFV, Q125 SSM3K35AMFV, Q126 SSM3K35AMFV, Q127 SSM3K35AMFV, Q128 SSM3K35AMFV, Q129 DMG6602, Q13 SSM3K35AMFV, Q130 SSM3K35AMFV, Q131 SSM3K35AMFV, Q14 SSM3K35AMFV, Q15 DMG6602, Q16 DMG6602, Q17 DMG6602, Q18 SSM3K35AMFV, Q19 SSM3K35AMFV, Q2 SSM3K35AMFV, Q20 DMG6602, Q21 DMG6602, Q22 SSM3K35AMFV, Q23 SSM3K35AMFV, Q24 DMG6602, Q25 DMG6602, Q26 SSM3K35AMFV, Q27 SSM3K35AMFV, Q28 DMG6602, Q29 DMG6602, Q3 SSM3K35AMFV, Q30 SSM3K35AMFV, Q31 SSM3K35AMFV, Q32 DMG6602, Q33 DMG6602, Q34 SSM3K35AMFV, Q35 SSM3K35AMFV, Q36 DMG6602, Q37 DMG6602, Q38 SSM3K35AMFV, Q39 SSM3K35AMFV, Q4 SSM3K35AMFV, Q40 DMG6602, Q41 DMG6602, Q42 SSM3K35AMFV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

Commit message: automated commit
Parts:
- removed C38: CL10B104KO8NNNC, Capacitor_SMD:C_0603_1608Metric
- C21, C22, C23, C24, C25, C26, C27, C28, C29, C30, C31, C34, C35, C39, C40, C41, C65, C66, C67, C68, C69, C70, C71, C72, C73, C77, C78, C79, C80, C81, C82, C83, C84, C85: moved to B.Cu
- moved C37 501.9 mm to (24.2, 65.8), turned to 90 degrees
- moved C85 499.0 mm to (88.1, 27.5), turned to 270 degrees
- moved C78 498.3 mm to (89.6, 17.0), turned to 270 degrees
- moved C79 497.4 mm to (88.1, 17.0), turned to 270 degrees
- moved C36 495.7 mm to (22.6, 65.8), turned to 90 degrees
- moved C77 495.3 mm to (91.2, 16.9), turned to 270 degrees
- moved C83 494.5 mm to (91.1, 27.5), turned to 270 degrees
- moved C33 492.9 mm to (22.2, 75.9), turned to 135 degrees
- moved C21 491.5 mm to (34.0, 71.0), turned to 90 degrees
- moved C23 490.4 mm to (37.4, 69.8), turned to 270 degrees
- moved C68 489.7 mm to (124.9, -5.00), turned to 180 degrees
- moved C70 488.7 mm to (124.8, -8.05), turned to 180 degrees
- moved C32 488.6 mm to (22.5, 71.9), turned to 225 degrees
- moved C27 487.6 mm to (35.5, 69.3), turned to 270 degrees
- moved C24 487.3 mm to (39.9, 71.1), turned to 270 degrees
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Connections:
- net IVDD_FE310 renamed +3V3
Routing:
- net COL13: track 14.8 -> 99.0 mm
- net COL14: track 7.05 -> 88.4 mm
- net COL15: track 14.8 -> 93.9 mm
- net COL12: track 7.05 -> 85.0 mm
- net COL11: track 14.8 -> 90.1 mm
- net COL16: track 7.05 -> 78.9 mm
- net COL10: track 7.05 -> 76.1 mm
- net COL17: track 14.8 -> 83.4 mm
- net COL09: track 14.8 -> 81.2 mm
- net COL18: track 7.05 -> 68.5 mm
- net COL08: track 7.05 -> 67.2 mm
- net COL19: track 14.8 -> 73.0 mm
- net COL07: track 14.8 -> 72.2 mm
- net COL06: track 7.05 -> 58.3 mm
- net COL20: track 7.05 -> 58.0 mm
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- added copper zone on B.Cu, net +1V8
- added copper zone on F.Cu, net +1V8
- added copper zone on B.Cu, net +3V3
- removed copper zone on B.Cu, net (none)
- removed copper zone on F.Cu, net (none)

Commit message: automated commit
Parts:
- C15, C42, C43, C44, C45, C46, C47, C48, C49, C50, R10, R13, R14, R15, R16, R17, R18, R2, R3, R45, R46, R47, R48, R49, R5, R50, R51, R52, R55, R63, R67, R8, R9: moved to B.Cu
- moved J1 234.8 mm to (-101.6, 120.0), turned to 270 degrees
- moved J2 220.6 mm to (-104.6, 142.8), turned to 90 degrees
- moved L1 220.4 mm to (-77.0, 120.7), turned to 180 degrees
- moved D1 213.0 mm to (-91.2, 120.5), turned to 90 degrees
- moved D2 211.1 mm to (-81.9, 123.0), turned to 270 degrees
- moved R3 175.3 mm to (-42.7, 223.3), turned to 270 degrees
- moved R9 165.3 mm to (-37.7, 226.5), turned to 90 degrees
- moved C9 163.1 mm to (-50.5, 225.0)
- moved R5 161.8 mm to (-41.3, 225.6)
- moved L2 157.8 mm to (-42.7, 232.3), turned to 270 degrees
- moved C10 156.7 mm to (-57.8, 224.9)
- moved R8 152.4 mm to (-41.2, 223.3), turned to 90 degrees
- moved C11 151.8 mm to (-36.8, 229.6)
- moved C15 149.2 mm to (-48.6, 77.9), turned to 90 degrees
- moved R17 148.7 mm to (-47.0, 77.9), turned to 90 degrees
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Connections:
- R47 pad 2: Net-(J9-PadS0) -> Net-(J9-PadS)
- R48 pad 2: Net-(J9-PadS2) -> Net-(J9-PadS)
- R50 pad 1: Net-(J9-PadS0) -> Net-(J9-PadS)
- R51 pad 1: Net-(J9-PadS2) -> Net-(J9-PadS)
- U1 pad 15: (no net) -> GND
Routing:
- net Net-(J9-PadS): track 0.00 -> 23.4 mm
- net Net-(J9-PadB1): track 0.00 -> 21.5 mm
- net GND: track 294.7 -> 315.9 mm, vias 215 -> 244
- net Net-(D16-Pad1): track 0.00 -> 20.7 mm
- net Net-(C51-Pad1): track 0.00 -> 13.9 mm
- net Net-(C52-Pad1): track 0.00 -> 13.9 mm
- net UART_FE_RX: track 0.00 -> 13.5 mm, vias 0 -> 1
- net Net-(J9-PadA1): track 0.00 -> 13.4 mm
- net UART_FE_TX: track 0.00 -> 9.76 mm, vias 0 -> 1
- net ROW_IN: track 9.06 -> 0.00 mm
- net /FT2232/USB_D-: track 0.00 -> 8.43 mm
- net /FT2232/USB_D+: track 0.00 -> 8.43 mm
- net Net-(R2-Pad2): track 0.00 -> 8.25 mm, vias 0 -> 1
- net +3V3: track 5.76 -> 13.5 mm, vias 33 -> 39
- net /FT2232/USB_SHIELD: track 0.00 -> 7.65 mm
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- added copper zone on F.Cu, net +24V
- added copper zone on F.Cu, net Net-(C13-Pad2)
- added copper zone on F.Cu, net Net-(D4-Pad1)

Commit message: automated commit
Parts:
- C14, C18, C19, Q2, Q3, Q4, Q5, Q6, Q7, Q8, R19, R20, R21, R22, R23, R24, R25, R26, R27, R28, R35, R36, R37, R38, R39, R40, R41, R42, R43, R44, R74, R75, R76, R77: moved to B.Cu
- moved L2 312.3 mm to (224.4, 70.5), turned to 0 degrees
- moved C10 307.6 mm to (214.9, 82.7), turned to 90 degrees
- moved C11 306.4 mm to (219.5, 61.7), turned to 90 degrees
- moved R2 306.1 mm to (218.8, 64.0), turned to 180 degrees
- moved C9 304.6 mm to (214.9, 75.4), turned to 90 degrees
- moved R9 302.4 mm to (216.5, 62.6), turned to 180 degrees
- moved R5 302.2 mm to (215.5, 66.2), turned to 90 degrees
- moved U1 300.5 mm to (214.9, 63.3), turned to 90 degrees
- moved C12 300.3 mm to (215.5, 59.8), turned to 0 degrees
- moved D4 299.6 mm to (212.8, 69.5), turned to 270 degrees
- moved R3 299.6 mm to (213.2, 67.6), turned to 0 degrees
- moved R8 299.1 mm to (213.2, 66.1), turned to 180 degrees
- moved R10 298.1 mm to (213.3, 62.6), turned to 0 degrees
- moved R11 296.1 mm to (212.5, 59.8), turned to 0 degrees
- moved R35 274.4 mm to (-6.20, 316.7), turned to 90 degrees
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Routing:
- net GND: track 315.9 -> 360.0 mm, vias 244 -> 269
- net +3V3: track 13.5 -> 34.4 mm, vias 39 -> 52
- net +12V: track 211.1 -> 229.4 mm, vias 98 -> 108
- net !COL_RESET: track 0.00 -> 8.23 mm
- net !ENABLE: track 0.00 -> 8.23 mm
- net ROW_IN: track 0.00 -> 8.22 mm
- net COL_IN: track 0.00 -> 8.21 mm
- net Net-(R23-Pad2): track 0.00 -> 7.53 mm, vias 0 -> 1
- net Net-(D11-Pad2): track 0.00 -> 7.10 mm, vias 0 -> 1
- net Net-(D14-Pad2): track 0.00 -> 7.10 mm, vias 0 -> 1
- net Net-(D12-Pad2): track 0.00 -> 7.10 mm, vias 0 -> 1
- net Net-(D15-Pad2): track 0.00 -> 7.10 mm, vias 0 -> 1
- net Net-(D13-Pad2): track 0.00 -> 7.10 mm, vias 0 -> 1
- net Net-(D15-Pad1): track 0.00 -> 6.23 mm, vias 0 -> 1
- net Net-(D13-Pad1): track 0.00 -> 6.23 mm, vias 0 -> 1
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- added copper zone on In2.Cu, net +24V
- added copper zone on F.Cu, net Net-(C17-Pad2)
- added copper zone on F.Cu, net Net-(J11-Pad1)
Other:
- board text added: "12V"

Commit message: automated commit
Parts:
- moved C22 149.8 mm to (184.5, 24.1)
- moved C26 149.8 mm to (184.4, 22.5)
- moved C28 149.8 mm to (175.4, 18.6)
- moved C29 149.8 mm to (181.3, 26.6)
- moved C32 149.8 mm to (166.6, 22.6)
- moved C36 149.8 mm to (164.1, 16.5)
- moved U5 149.8 mm to (170.1, 15.3)
- moved Y1 149.8 mm to (168.3, 24.5)
- moved C21 149.8 mm to (175.5, 21.7)
- moved C23 149.8 mm to (178.8, 20.5)
- moved C24 149.8 mm to (181.3, 21.7)
- moved C25 149.8 mm to (177.4, 26.0)
- moved C27 149.8 mm to (177.0, 20.0)
- moved C30 149.8 mm to (179.7, 26.6)
- moved C31 149.8 mm to (180.5, 29.0)
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
Commit message: automated commit
Parts:
- C53, C54, C55, C56, C57, C58, C86, C87, R89, R90, R91, R92, U20, U21, U22, U23, U6, U7: moved to B.Cu
- moved J2 407.0 mm to (267.0, -23.1), turned to 270 degrees
- moved C2 390.0 mm to (254.5, -29.5), turned to 180 degrees
- moved J1 384.9 mm to (264.0, -0.22), turned to 90 degrees
- moved C3 376.8 mm to (247.0, -29.6), turned to 180 degrees
- moved C1 374.4 mm to (252.7, -15.3), turned to 180 degrees
- moved TP1 370.8 mm to (257.9, 3.60), turned to 180 degrees
- moved D1 365.4 mm to (253.6, -0.70), turned to 270 degrees
- moved C4 362.0 mm to (242.1, -23.0), turned to 180 degrees
- moved C5 354.9 mm to (241.7, -15.8), turned to 180 degrees
- moved D2 349.8 mm to (244.3, -3.23), turned to 90 degrees
- moved TP2 342.5 mm to (242.2, 1.60), turned to 180 degrees
- moved L1 339.0 mm to (239.4, -0.94), turned to 0 degrees
- moved TP3 330.1 mm to (235.6, 1.60), turned to 180 degrees
- moved TP24 299.1 mm to (-48.9, 276.7)
- moved TP28 297.9 mm to (-45.9, 277.3)
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Connections:
- R6 pad 1: +12V -> +24V
- TP60 pad 1: Net-(TP60-Pad1) -> GND
- U23 pad 6: Net-(TP60-Pad1) -> GND
Routing:
- net AUX_0: track 5.66 -> 81.0 mm, vias 1 -> 2
- net AUX_1: track 5.66 -> 65.8 mm, vias 1 -> 2
- net AUX_2: track 5.66 -> 51.6 mm, vias 1 -> 2
- net AUX_3: track 5.66 -> 38.3 mm, vias 1 -> 2
- net GND: track 360.0 -> 388.3 mm, vias 269 -> 294
- net +3V3: track 34.4 -> 53.2 mm, vias 52 -> 65
- net AUX_4: track 5.66 -> 22.6 mm, vias 1 -> 2
- net /PANEL_EXTENSION/ROW_DATA: track 0.00 -> 12.8 mm
- net /PANEL_EXTENSION/COL_DATA: track 0.00 -> 12.1 mm
- net Net-(TP40-Pad1): track 0.00 -> 7.76 mm, vias 0 -> 2
- net COL_SHCP: track 3.25 -> 10.8 mm
- net !ENABLE: track 8.23 -> 14.8 mm
- net !COL_RESET: track 8.23 -> 14.7 mm
- net ROW_ON: track 3.25 -> 9.59 mm
- net ROW_SHCP: track 3.25 -> 9.58 mm
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Other:
- board text added: "AUX_0"
- board text added: "AUX_1"
- board text added: "AUX_2"
- board text added: "AUX_3"
- board text added: "AUX_4"

Commit message: automated commit
Parts:
- removed the C74 at (-29.7, 272.6)
- removed the C75 at (-29.7, 275.1)
- removed the C76 at (-25.7, 272.6)
- removed TP12, TP15, TP19: TestPoint, custom:TestPoint_THTPad_D1.0mm_Drill0.5mm
- added C65: CL10B104KO8NNNC, Capacitor_SMD:C_0603_1608Metric, B.Cu at (99.4, 111.0)
- added C66: CL10B105KA8NNNC, Capacitor_SMD:C_0603_1608Metric, B.Cu at (100.9, 111.0)
- added C67: NP_0603, Capacitor_SMD:C_0603_1608Metric, B.Cu at (102.4, 111.0)
- C4, C5, R53, R60, R61, R62, R64, R65, R66: moved to B.Cu
- R63, R67: moved to F.Cu
- moved TP34 408.6 mm to (360.2, 130.7), turned to 270 degrees
- moved TP38 407.4 mm to (359.6, 144.3), turned to 270 degrees
- moved TP33 406.2 mm to (354.7, 128.4), turned to 90 degrees
- moved TP37 404.8 mm to (354.2, 142.1), turned to 90 degrees
- moved TP41 396.5 mm to (344.7, 108.8)
- moved TP42 396.5 mm to (341.6, 111.8)
- moved TP36 392.3 mm to (345.7, 143.9), turned to 270 degrees
- moved TP35 389.9 mm to (340.2, 141.6), turned to 90 degrees
- moved TP49 378.6 mm to (73.1, -67.9)
- moved TP50 378.6 mm to (79.2, -70.9)
- moved TP51 378.6 mm to (76.2, -64.8)
- moved TP52 378.6 mm to (85.3, -70.9)
- moved TP53 378.6 mm to (73.1, -70.9)
- moved TP54 378.6 mm to (82.3, -67.9)
- moved TP55 378.6 mm to (79.2, -64.8)
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- renumbered C65 to C74, C66 to C75, C67 to C76
Routing:
- net GND: track 388.3 -> 414.9 mm, vias 294 -> 312
- net /FT2232/D-: track 5.02 -> 13.2 mm
- net Net-(R2-Pad2): track 8.25 -> 16.0 mm
- net Net-(TP39-Pad1): track 8.38 -> 15.9 mm
- net Net-(TP45-Pad1): track 7.90 -> 15.4 mm
- net Net-(TP40-Pad1): track 7.76 -> 15.1 mm
- net Net-(TP48-Pad1): track 7.41 -> 14.8 mm
- net /COLUMN_SHIFT_REGISTER/COL_SR_CHAIN_1: track 7.62 -> 14.9 mm
- net Net-(TP47-Pad1): track 7.82 -> 15.1 mm
- net +12V: track 229.4 -> 236.5 mm, vias 108 -> 118
- net /FT2232/D+: track 5.85 -> 12.9 mm
- net Net-(D10-Pad1): track 0.00 -> 5.25 mm
- net /FT2232/UART_FT_TX: track 6.06 -> 11.1 mm, vias 1 -> 0
- net Net-(R3-Pad2): track 3.63 -> 8.63 mm
- net Net-(D9-Pad1): track 0.00 -> 5.00 mm
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- added copper zone on In1.Cu, net +24V
- added copper zone on F.Cu, net Net-(D1-Pad1)
- added copper zone on F.Cu, net Net-(D1-Pad3)
- removed copper zone on In2.Cu, net +24V
Other:
- board text added: "1V8"
- board text added: "24V"

Commit message: automated commit
Parts:
- removed TP65, TP67, TP69, TP71, TP73, TP75, TP76, TP77, TP79, TP81, TP85, TP86, TP87, TP89, TP91: TestPoint, custom:TestPoint_THTPad_D1.0mm_Drill0.5mm
- C86, C87, R89, R90, R91, R92, U20, U21, U22, U23: moved to F.Cu
- Q12, Q13, Q14, R85, R86, R87, R88, TP49, TP50, TP51, TP52, TP53, TP54, TP55, TP56, TP57, TP58, TP59, TP60: moved to B.Cu
- moved R87 244.7 mm to (106.2, 117.3)
- moved R88 242.9 mm to (109.5, 117.3), turned to 90 degrees
- moved Q12 240.1 mm to (106.0, 109.2), turned to 90 degrees
- moved R86 237.8 mm to (108.5, 109.0), turned to 270 degrees
- moved R85 237.6 mm to (106.0, 111.8), turned to 0 degrees
- moved TP41 237.1 mm to (107.7, 118.0)
- moved Q13 237.0 mm to (105.0, 113.5), turned to 90 degrees
- moved Q14 235.2 mm to (106.8, 113.5), turned to 90 degrees
- moved TP42 232.1 mm to (109.5, 114.9)
- moved TP84 231.0 mm to (92.5, 151.3)
- moved TP78 220.3 mm to (84.8, 145.5)
- moved R56 219.4 mm to (163.6, 67.2)
- moved R57 219.2 mm to (163.6, 68.8), turned to 180 degrees
- moved TP82 219.0 mm to (87.2, 142.1)
- moved R54 218.4 mm to (166.9, 65.7), turned to 180 degrees
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Connections:
- J10 pad 1: /PANEL_EXTENSION/ROW_DATA -> GND
- J10 pad 2: ROW_SHCP -> !ENABLE
- J10 pad 3: ROW_ON -> !COL_RESET
- J10 pad 4: /PANEL_EXTENSION/COL_DATA -> COL_SHCP
- J10 pad 5: COL_SHCP -> /PANEL_EXTENSION/COL_DATA
- J10 pad 6: !COL_RESET -> ROW_ON
- J10 pad 7: !ENABLE -> ROW_SHCP
- J10 pad 8: GND -> /PANEL_EXTENSION/ROW_DATA
Routing:
- net /ROW_SHIFT_REGISTER/SR_OUT_0: track 0.00 -> 36.2 mm, vias 0 -> 1
- net +1V8: track 17.0 -> 33.3 mm, vias 11 -> 16
- net /ROW_SHIFT_REGISTER/SR_OUT_1: track 0.00 -> 15.5 mm
- net GND: track 414.9 -> 425.8 mm, vias 312 -> 315
- net Net-(D9-Pad1): track 5.00 -> 14.1 mm
- net Net-(R56-Pad2): track 0.00 -> 8.13 mm
- net ROW_ON: track 9.59 -> 16.5 mm
- net ROW_SHCP: track 9.58 -> 16.5 mm
- net /PANEL_EXTENSION/ROW_DATA: track 12.8 -> 19.7 mm
- net COL_SHCP: track 10.8 -> 17.7 mm
- net !ENABLE: track 14.8 -> 21.7 mm
- net /PANEL_EXTENSION/COL_DATA: track 12.1 -> 18.9 mm
- net !COL_RESET: track 14.7 -> 21.5 mm
- net Net-(R54-Pad2): track 0.00 -> 5.19 mm
- net +12V: track 236.5 -> 240.5 mm, vias 118 -> 117
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- added copper zone on In1.Cu, net +1V8
