File: flipdot_driver.kicad_pcb (KiCad board)
At the start: 4 copper layers, 642 parts, among them J1 Barrel_Jack, J10 Conn_01x08_Male, J11 3x32_1&3_loaded_2.5mm_0.1in_f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, J2 Screw_Terminal_01x04, J3 PTH_1.5_mm, J4 PTH_1.5_mm, J5 PTH_1.5_mm, J6 PTH_1.5_mm, J7 Conn_01x05_Male, J8 PTH_1.5_mm, J9 USB-C_2.0_Connector, Q1 SSM3K35AMFV, Q10 SSM3K35AMFV, Q100 SSM3K35AMFV, Q101 SSM3K35AMFV, Q102 DMG6602, Q103 DMG6602, Q104 DMG6602, Q105 SSM3K35AMFV, Q106 SSM3K35AMFV, Q107 SSM3K35AMFV, Q108 SSM3K35AMFV, Q109 SSM3K35AMFV, Q11 SSM3K35AMFV, Q110 SSM3K35AMFV, Q111 DMG6602, Q112 DMG6602, Q113 DMG6602, Q114 SSM3K35AMFV, Q115 SSM3K35AMFV, Q116 SSM3K35AMFV, Q117 SSM3K35AMFV, Q118 SSM3K35AMFV, Q119 SSM3K35AMFV, Q12 AO3407A, Q120 DMG6602, Q121 DMG6602, Q122 DMG6602, Q123 SSM3K35AMFV, Q124 SSM3K35AMFV, Q125 SSM3K35AMFV, Q126 SSM3K35AMFV, Q127 SSM3K35AMFV, Q128 SSM3K35AMFV, Q129 DMG6602, Q13 SSM3K35AMFV, Q130 SSM3K35AMFV, Q131 SSM3K35AMFV, Q14 SSM3K35AMFV, Q15 DMG6602, Q16 DMG6602, Q17 DMG6602, Q18 SSM3K35AMFV, Q19 SSM3K35AMFV, Q2 SSM3K35AMFV, Q20 DMG6602, Q21 DMG6602, Q22 SSM3K35AMFV, Q23 SSM3K35AMFV, Q24 DMG6602, Q25 DMG6602, Q26 SSM3K35AMFV, Q27 SSM3K35AMFV, Q28 DMG6602, Q29 DMG6602, Q3 SSM3K35AMFV, Q30 SSM3K35AMFV, Q31 SSM3K35AMFV, Q32 DMG6602, Q33 DMG6602, Q34 SSM3K35AMFV, Q35 SSM3K35AMFV, Q36 DMG6602, Q37 DMG6602, Q38 SSM3K35AMFV, Q39 SSM3K35AMFV, Q4 SSM3K35AMFV, Q40 DMG6602, Q41 DMG6602, Q42 SSM3K35AMFV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

Commit message: automated commit
Parts:
- Q44: footprint TSOT-23-6 -> Package_TO_SOT_SMD:TSOT-23-6
- R30, TP23: moved to B.Cu
- moved R34 144.2 mm to (192.5, -15.3), turned to 0 degrees
- moved C36 142.5 mm to (188.5, -16.8), turned to 0 degrees
- moved C37 139.8 mm to (188.5, -15.3), turned to 0 degrees
- moved TP21 135.0 mm to (180.1, -28.3), turned to 0 degrees
- moved C33 134.3 mm to (183.7, -18.0), turned to 315 degrees
- moved R20 133.9 mm to (180.7, -25.2), turned to 180 degrees
- moved U5 133.7 mm to (189.7, -10.8), turned to 90 degrees
- moved R19 133.1 mm to (180.7, -23.7), turned to 180 degrees
- moved R22 132.3 mm to (180.7, -22.1), turned to 0 degrees
- moved C32 132.2 mm to (183.4, -14.1), turned to 45 degrees
- moved U3 131.8 mm to (179.1, -25.2), turned to 0 degrees
- moved C18 131.2 mm to (178.2, -26.1), turned to 270 degrees
- moved Y1 130.8 mm to (181.7, -16.0), turned to 45 degrees
- moved C17 130.5 mm to (179.1, -22.7), turned to 180 degrees
- moved R4 128.8 mm to (174.8, -29.1), turned to 0 degrees
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Routing:
- net GND: track 425.8 -> 449.0 mm, vias 315 -> 326
- net +1V8: track 33.3 -> 14.2 mm, vias 16 -> 14
- net Net-(D9-Pad1): track 14.1 -> 3.34 mm
- net Net-(U4-Pad48): track 7.18 -> 16.7 mm
- net Net-(U4-Pad1): track 14.7 -> 22.5 mm
- net Net-(U4-Pad2): track 11.3 -> 18.5 mm
- net Net-(U4-Pad3): track 14.8 -> 21.3 mm
- net Net-(D10-Pad1): track 7.20 -> 13.4 mm
- net Net-(R34-Pad1): track 16.8 -> 22.6 mm
- net Net-(U4-Pad5): track 13.2 -> 18.4 mm
- net Net-(D8-Pad1): track 2.95 -> 6.88 mm
- net +3V3: track 56.8 -> 55.7 mm, vias 70 -> 69
- net COL14: track 88.4 -> 89.3 mm
- added copper zone on In1.Cu, net +12V
- added copper zone on In1.Cu, net +3V3
- added copper zone on In2.Cu, net GND

Commit message: automated commit
Parts:
- moved C18 41.8 mm to (137.2, -17.9)
- moved C20 41.8 mm to (132.9, -16.9)
- moved C23 41.8 mm to (130.3, -3.71)
- moved C25 41.8 mm to (131.7, -9.21)
- moved C30 41.8 mm to (129.4, -9.89)
- moved C37 41.8 mm to (147.6, -7.03)
- moved C40 41.8 mm to (131.3, -5.98)
- moved D10 41.8 mm to (118.6, -10.9)
- moved D5 41.8 mm to (133.4, -19.1)
- moved L4 41.8 mm to (134.3, -14.5)
- moved Q1 41.8 mm to (130.7, -19.2)
- moved R12 41.8 mm to (130.7, -20.9)
- moved R19 41.8 mm to (139.7, -15.4)
- moved R22 41.8 mm to (139.7, -13.9)
- moved R29 41.8 mm to (128.2, -18.3)
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Routing:
- net Net-(D10-Pad1): track 13.4 -> 3.23 mm, vias 0 -> 2
- net GND: vias 326 -> 322
- net Net-(U4-Pad1): vias 0 -> 1
- net Net-(R32-Pad1): vias 0 -> 2
- net +3V3: vias 69 -> 68

Commit message: automated commit
Parts:
- Q10, R79, R80, R83, TP35, TP36: moved to B.Cu
- moved R80 111.3 mm to (112.8, 107.7), turned to 0 degrees
- moved R79 109.6 mm to (112.8, 106.1), turned to 0 degrees
- moved TP36 109.2 mm to (115.3, 108.3), turned to 0 degrees
- moved C19 109.1 mm to (124.2, 92.7)
- moved C20 109.1 mm to (124.8, 91.9)
- moved C22 109.1 mm to (116.5, 101.5)
- moved C34 109.1 mm to (123.5, 98.1)
- moved C35 109.1 mm to (123.5, 96.5)
- moved C41 109.1 mm to (123.1, 101.3)
- moved D8 109.1 mm to (115.8, 87.7)
- moved D9 109.1 mm to (114.7, 97.9)
- moved R12 109.1 mm to (122.5, 87.9)
- moved R20 109.1 mm to (131.6, 91.9)
- moved R22 109.1 mm to (131.6, 94.9)
- moved R23 109.1 mm to (125.8, 92.7)
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Routing:
- net !COL_RESET: track 21.5 -> 153.4 mm, vias 0 -> 7
- net COL_SHCP: track 17.7 -> 148.9 mm, vias 0 -> 7
- net !COL_SHCP: track 1.98 -> 129.8 mm, vias 0 -> 7
- net !ENABLE: track 21.7 -> 120.3 mm, vias 0 -> 7
- net ROW_ON: track 16.5 -> 60.9 mm, vias 0 -> 2
- net !ROW_ON: track 1.98 -> 30.2 mm
- net Net-(J9-PadS): track 23.4 -> 8.00 mm
- net (no net): track 0.00 -> 15.4 mm
- net Net-(TP40-Pad1): track 15.1 -> 19.4 mm
- net GND: track 449.0 -> 446.7 mm, vias 322 -> 325
- net COL16_ON: track 21.7 -> 20.7 mm
- net COL13_OFF: track 22.4 -> 21.5 mm
- net Net-(TP39-Pad1): track 15.9 -> 16.7 mm
- net +3V3: vias 68 -> 69
- net Net-(D10-Pad1): vias 2 -> 0
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Other:
- board text added: "3V3"

Commit message: automated commit
Parts:
- moved C2 4.09 mm to (90.5, 145.9)
- moved TP68 3.44 mm to (95.1, 143.4)
- turned TP78 to 90 degrees
Routing:
- net ROW00P: track 29.2 -> 27.0 mm

Commit message: automated commit
Parts:
- removed C51, C52: TMK042CG120JD-W‎, Capacitor_SMD:C_01005_0402Metric
- removed TP74: TestPoint, custom:TestPoint_THTPad_D1.0mm_Drill0.5mm
- Q11, Q9, R72, R73, R78, R81, R82, R84, TP33, TP34, TP37, TP38: moved to B.Cu
- moved R71 131.3 mm to (92.7, 112.4), turned to 0 degrees
- moved R77 131.3 mm to (95.3, 119.8), turned to 270 degrees
- moved R70 130.3 mm to (92.7, 114.0), turned to 0 degrees
- moved R76 130.3 mm to (96.8, 119.8), turned to 270 degrees
- moved R81 129.3 mm to (106.8, 105.0), turned to 90 degrees
- moved R82 129.3 mm to (108.3, 105.0), turned to 90 degrees
- moved R69 129.2 mm to (92.7, 115.5), turned to 0 degrees
- moved R75 129.2 mm to (98.4, 119.8), turned to 270 degrees
- moved Q11 128.9 mm to (107.0, 102.6)
- moved R84 128.9 mm to (105.2, 102.6), turned to 90 degrees
- moved TP38 128.9 mm to (108.9, 102.5), turned to 90 degrees
- moved TP37 128.9 mm to (103.8, 104.7), turned to 270 degrees
- moved R68 128.2 mm to (92.7, 117.0), turned to 0 degrees
- moved R74 128.2 mm to (100.0, 119.7), turned to 270 degrees
- moved TP29 127.0 mm to (95.3, 112.4), turned to 180 degrees
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Routing:
- net COL_IN: track 10.4 -> 124.4 mm, vias 0 -> 2
- net !ENABLE: track 120.3 -> 206.7 mm, vias 7 -> 11
- net LED_PWM: track 3.66 -> 85.8 mm
- net COL_OUT: track 2.09 -> 76.8 mm
- net ROW_IN: track 10.1 -> 73.4 mm, vias 0 -> 5
- net ROW_SHCP: track 16.5 -> 56.0 mm, vias 0 -> 3
- net !ROW_SHCP: track 1.98 -> 41.2 mm, vias 0 -> 2
- net !COL_RESET: track 153.4 -> 188.1 mm, vias 7 -> 9
- net COL_SHCP: track 148.9 -> 173.1 mm, vias 7 -> 8
- net /FE310/PIEZO_0: track 1.32 -> 24.5 mm, vias 0 -> 1
- net !COL_SHCP: track 129.8 -> 144.1 mm, vias 7 -> 8
- net Net-(D9-Pad1): track 3.34 -> 14.5 mm
- net ROW_ON: track 60.9 -> 69.7 mm
- net Net-(C51-Pad1): track 13.9 -> 11.1 mm
- net Net-(C52-Pad1): track 13.9 -> 11.2 mm
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